File: nutrient V0.1f.kicad_pcb (KiCad board)
At the start: 2 copper layers, 99.1 x 71.1 mm, 84 parts, among them J1 Conn_01x04_Female, J2 Conn_01x04_Female, J3 Conn_01x04_Female, J4 Conn_01x04_Female, J5 Conn_01x04_Female, J6 Conn_01x04_Female, J7 Conn_01x03_Male, J8 Conn_01x03_Male, P1 SolderJumper_2_Open, P2 SolderJumper_2_Bridged, P3 SolderJumper_2_Bridged, Q1 Q_NMOS_DGS, Q10 Q_NMOS_DGS, Q2 Q_NMOS_DGS, Q3 Q_NMOS_DGS, Q4 Q_NMOS_DGS, Q5 Q_NMOS_DGS, Q6 Q_NMOS_DGS, Q7 Q_NMOS_DGS, Q8 2N3904, U1 23LC512, U2 DS1307+, Y1 Crystal_Small

Commit message: New schematics for specto
Parts:
- R10: footprint Resistor_THT:R_Axial_DIN0204_L3.6mm_D1.6mm_P5.08mm_Horizontal -> Resistor_THT:R_Axial_DIN0204_L3.6mm_D1.6mm_P3.30mm_Horizontal
- moved R10 0.52 mm to (140.6, 82.5)
Routing:
- net Net-(Q4-Pad2): track 4.32 -> 3.05 mm
- net GND: track 719.1 -> 718.0 mm
- net /5V2: track 123.5 -> 122.8 mm
- net /D16: track 1.92 -> 1.27 mm
- net /GND3: track 24.1 -> 23.6 mm
