File: SpectDrone/SpectDrone.kicad_pcb (KiCad board)
At the start: 2 copper layers, 11 parts, among them J1 Camera, J2 GPS, J3 APC220, J4 BME280, J5-1 BNO055-1, J5-2 BNO055-2, U1 C12666MA, U2 C12666MA

Commit message: SpectDrone Development
Parts:
- added H1: MountingHole, MountingHole:MountingHole_2.2mm_M2_ISO14580_Pad_TopBottom, F.Cu at (215.8, 134.9)
- added H2: MountingHole, MountingHole:MountingHole_2.2mm_M2_ISO14580_Pad_TopBottom, F.Cu at (215.8, 68.9)
- added H3: MountingHole, MountingHole:MountingHole_2.2mm_M2_ISO14580_Pad_TopBottom, F.Cu at (121.8, 68.9)
- added H4: MountingHole, MountingHole:MountingHole_2.2mm_M2_ISO14580_Pad_TopBottom, F.Cu at (121.8, 134.9)
- added JAPC1: Conn_01x04_Male, Connector_PinHeader_2.54mm:PinHeader_1x04_P2.54mm_Vertical, B.Cu at (191.5, 111.0)
- JA1: value Conn_01x04_Female -> Conn_01x04_Male; footprint Connector_JST:JST_XH_B4B-XH-A_1x04_P2.50mm_Vertical -> Connector_PinHeader_2.54mm:PinHeader_1x04_P2.54mm_Vertical; moved to B.Cu
- JAUX1: value GPS -> AUX; moved to B.Cu
- JGPS1: moved to B.Cu
- moved J3 97.0 mm to (184.2, 111.0), turned to -90 degrees
- moved J1 89.8 mm to (165.1, 134.6), turned to 180 degrees
- moved U1 63.1 mm to (223.5, 97.8)
- moved J4 47.0 mm to (147.3, 85.1), turned to -90 degrees
- moved U2 41.3 mm to (223.5, 105.4), turned to 0 degrees
- turned JA1 to 180 degrees
- turned JAUX1 to 0 degrees
- turned JGPS1 to 180 degrees
Connections:
- J4 pad 4: /BMESCK -> /SCL
- J4 pad 6: /BMESDI -> /SDA
- JAUX1 pad 10: /OPT_EXT -> /CLK2
- JAUX1 pad 11: /D12 -> /CLK1
- JAUX1 pad 4: /SS_AUX -> /CAMRX
- JAUX1 pad 8: /XCL -> /CAMTX
- U1 pad 4: /OPT_EXT -> /CLK1
- U1 pad 5: unconnected-(U1-Pad5) -> /GND3
- U2 pad 4: /D12 -> /CLK2
- U2 pad 5: unconnected-(U2-Pad5) -> /GND3
Routing:
- net /GND3: track 45.4 -> 270.4 mm
- net /5V3: track 42.2 -> 205.6 mm
- net /CLK1: track 0.00 -> 92.3 mm
- net /ST: track 36.7 -> 120.7 mm
- net /CLK2: track 0.00 -> 76.9 mm
- net /SCL: track 0.00 -> 46.0 mm
- net /D12: track 45.4 -> 0.00 mm
- net /SDA: track 0.00 -> 43.1 mm
- net /A1: track 58.7 -> 32.5 mm
- net /OPT_EXT: track 22.7 -> 0.00 mm
- net /CAMTX: track 0.00 -> 16.9 mm
- net /CAMRX: track 0.00 -> 13.8 mm
- net /GAIN: track 46.8 -> 58.2 mm
- net /A2: track 37.8 -> 35.7 mm
Other:
- board outline added: 115.7 x 71.1 mm

Commit message: SpectDrone development
Parts:
- added H10: MountingHole, MountingHole:MountingHole_2.2mm_M2_ISO14580_Pad_TopBottom, F.Cu at (181.4, 71.8)
- added H11: MountingHole, MountingHole:MountingHole_2.2mm_M2_ISO14580_Pad_TopBottom, F.Cu at (181.4, 99.8)
- added H12: MountingHole, MountingHole:MountingHole_2.2mm_M2_ISO14580_Pad_TopBottom, F.Cu at (153.4, 71.8)
- added H5: MountingHole, MountingHole:MountingHole_2.2mm_M2_ISO14580_Pad_TopBottom, F.Cu at (188.4, 116.1)
- added H6: MountingHole, MountingHole:MountingHole_2.2mm_M2_ISO14580_Pad_TopBottom, F.Cu at (216.4, 88.1)
- added H7: MountingHole, MountingHole:MountingHole_2.2mm_M2_ISO14580_Pad_TopBottom, F.Cu at (216.4, 116.1)
- added H8: MountingHole, MountingHole:MountingHole_2.2mm_M2_ISO14580_Pad_TopBottom, F.Cu at (188.4, 88.1)
- added H9: MountingHole, MountingHole:MountingHole_2.2mm_M2_ISO14580_Pad_TopBottom, F.Cu at (153.4, 99.8)
- added JIR1: Conn_01x04_Male, Connector_PinHeader_2.54mm:PinHeader_1x04_P2.54mm_Horizontal, B.Cu at (135.3, 72.4)
- J1: footprint Connector_PinHeader_2.54mm:PinHeader_1x04_P2.54mm_Vertical -> Connector_JST:JST_XH_B4B-XH-A_1x04_P2.50mm_Vertical; moved to B.Cu
- J2: footprint Connector_PinHeader_2.54mm:PinHeader_1x04_P2.54mm_Vertical -> Connector_JST:JST_XH_B6B-XH-A_1x06_P2.50mm_Vertical; moved to B.Cu
- J3, J4: footprint Connector_PinHeader_2.54mm:PinHeader_1x07_P2.54mm_Vertical -> Connector_PinSocket_2.54mm:PinSocket_1x07_P2.54mm_Vertical; moved to B.Cu
- J5-1: footprint Connector_PinHeader_2.54mm:PinHeader_1x06_P2.54mm_Vertical -> Connector_PinSocket_2.54mm:PinSocket_1x06_P2.54mm_Vertical; moved to B.Cu
- J5-2: footprint Connector_PinHeader_2.54mm:PinHeader_1x04_P2.54mm_Vertical -> Connector_PinSocket_2.54mm:PinSocket_1x04_P2.54mm_Vertical; moved to B.Cu
- JA1, JAPC1, JAUX1: moved to F.Cu
- JGPS1: footprint Connector_PinSocket_2.54mm:PinSocket_1x05_P2.54mm_Vertical -> Connector_PinHeader_2.54mm:PinHeader_1x05_P2.54mm_Vertical; moved to F.Cu
- moved JAPC1 14.8 mm to (194.3, 125.5), turned to 0 degrees
- moved J5-1 10.5 mm to (142.2, 99.1)
- moved J2 9.76 mm to (134.6, 122.1), turned to -90 degrees
- moved J5-2 5.68 mm to (124.3, 101.6)
- moved JA1 4.82 mm to (186.7, 96.3), turned to 0 degrees
- moved J1 3.65 mm to (162.6, 132.0), turned to 90 degrees
- moved J4 1.91 mm to (145.4, 85.1), turned to 90 degrees
- moved J3 1.29 mm to (182.9, 111.0), turned to 90 degrees
- moved U2 0.76 mm to (223.5, 106.2)
- turned JAUX1 to 180 degrees
- turned JGPS1 to 0 degrees
Connections:
- J2 pad 1: /GND -> /PPS
- J2 pad 2: /GPSTX -> /5V2
- J2 pad 3: /GPSRX -> /5V2
- J2 pad 4: /5V2 -> /GPSRX
- J3 pad 3: /APCEN -> /APCTX
- J3 pad 5: /APCTX -> /APCEN
- J4 pad 4: /SCL -> /BMESCK
- J4 pad 6: /SDA -> /BMESDI
- J5-1 pad 1: /5V3 -> /BNORST
- J5-1 pad 2: /BNO3VO -> /BMESCK
- J5-1 pad 3: /GND3 -> /BMESDI
- J5-1 pad 4: /SDA -> /GND3
- J5-1 pad 5: /SCL -> /BNO3VO
- J5-1 pad 6: /BNORST -> /5V3
- J5-2 pad 1: /PS0 -> /ADR
- J5-2 pad 2: /PS1 -> /INT
- J5-2 pad 3: /INT -> /PS1
- J5-2 pad 4: /ADR -> /PS0
- JAPC1 pad 1: /APCRX -> /APCTX
- JAPC1 pad 2: /APCTX -> /APCRX
- JAUX1 pad 6: /SCL -> /BMESCK
- JAUX1 pad 7: /SDA -> /BMESDI
Routing:
- net /BMESDI: track 0.00 -> 53.3 mm
- net /BMESCK: track 0.00 -> 51.6 mm
- net /SCL: track 46.0 -> 0.00 mm
- net /SDA: track 43.1 -> 0.00 mm
- net /GND3: track 270.4 -> 310.4 mm
- net /5V3: track 205.6 -> 241.1 mm
- net /APCRX: track 0.00 -> 26.1 mm
- net /APCTX: track 0.00 -> 22.5 mm
- net /PPS: track 0.00 -> 19.7 mm
- net /CLK1: track 92.3 -> 81.1 mm
- net /GPSTX: track 12.5 -> 6.15 mm
- net /GPSRX: track 12.5 -> 6.17 mm
- net /GAIN: track 58.2 -> 63.4 mm
- net /A2: track 35.7 -> 40.9 mm
- net /A1: track 32.5 -> 37.3 mm
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Other:
- outline, holes or cut-outs redrawn
- board text added: "5V"
- board text added: "APC220"
- board text added: "APC_RX"
- board text added: "APC_TX"
- board text added: "BME_SCK"
- board text added: "BME_SDA"
- board text added: "BNO_SCK"
- board text added: "BNO_SDA"
- board text added: "CAM_RX"
- board text added: "CAM_TX"
- board text added: "CLK1"
- board text added: "CLK2"
- board text added: "Camera"
- board text added: "GAIN"
- board text added: "GND"
- board text added: "GPS"
- board text added: "GPS_RX"
- board text added: "GPS_TX"
- board text added: "IR_SCL"
- board text added: "IR_SDA"
- board text added: "MISO"
- board text added: "MOSI"
- board text added: "RX"
- board text added: "SCL"
- board text added: "SDA"
- board text added: "SPECT_VIDEO_1"
- board text added: "SPECT_VIDEO_2"
- board text added: "ST"
- board text added: "TX"
- board text added: "WHITE"

Commit message: SpectDrone development
Routing:
- net /GND3: track 310.4 -> 0.00 mm
- net /5V3: track 241.1 -> 0.00 mm
- net /CLK1: track 81.1 -> 85.6 mm
- net /CAMTX: track 13.3 -> 16.3 mm
- net /GAIN: track 63.4 -> 64.5 mm
- net /BMESCK: track 51.6 -> 52.4 mm
- net /BMESDI: track 53.3 -> 52.6 mm
- net /CLK2: track 78.8 -> 78.3 mm
- added copper zone on B.Cu, net /5V3
- added copper zone on F.Cu, net /GND3
Other:
- board text added: "CAMERA"
- board text added: "GPS_5V"
- board text added: "GPS_GND"
- board text added: "Infrared"
- board text added: "Orientation"
- board text added: "Radio"
- board text added: "SCK"
- board text added: "TempHumPres"
- board text removed: "APC220"
- board text removed: "BME_SCK"
- board text removed: "BME_SDA"
- board text removed: "BNO_SCK"
- board text removed: "BNO_SDA"

Commit message: SpectDrone Development
Parts:
- added C1: 0.1uF, Capacitor_SMD:C_0603_1608Metric_Pad1.08x0.95mm_HandSolder, B.Cu at (222.6, 101.9)
- added C2: 10uF, Capacitor_Tantalum_SMD:CP_EIA-3216-10_Kemet-I_Pad1.58x1.35mm_HandSolder, B.Cu at (227.1, 101.9)
- added C3: C_Small, Capacitor_THT:C_Disc_D5.0mm_W2.5mm_P2.50mm, B.Cu at (188.6, 83.1)
- added C4: C_Small, Capacitor_THT:C_Disc_D5.0mm_W2.5mm_P2.50mm, B.Cu at (188.6, 74.3)
- added JDC1: Conn_01x02_Female, Connector_PinSocket_2.54mm:PinSocket_1x02_P2.54mm_Vertical, F.Cu at (138.0, 78.5)
- added U3: LM7805_TO220, Package_TO_SOT_THT:TO-220-3_Vertical, B.Cu at (195.6, 81.3)
- moved JIR1 1.91 mm to (133.3, 72.4)
Connections:
- J1 pad 2: /GND3 -> /GND2
- J3 pad 7: /GND3 -> /GND2
- J4 pad 3: /GND3 -> /GND2
- J5-1 pad 4: /GND3 -> /GND2
- JIR1 pad 2: /GND3 -> /GND2
- U1 pad 3: /GND3 -> /GND2
- U1 pad 5: /GND3 -> /GND2
- U2 pad 3: /GND3 -> /GND2
- U2 pad 5: /GND3 -> /GND2
Routing:
- net /VIN: track 0.00 -> 7.76 mm
- net /GND2: track 0.00 -> 3.37 mm, vias 0 -> 2
- net /BMESCK: track 52.4 -> 53.5 mm
- net /BMESDI: track 52.6 -> 51.6 mm
- added copper zone on F.Cu, net /GND2
- removed copper zone on F.Cu, net /GND3

Commit message: SpectDrone Development
Parts:
- removed JDC1: Conn_01x02_Female, Connector_PinSocket_2.54mm:PinSocket_1x02_P2.54mm_Vertical
- added D1: D, Diode_THT:D_T-1_P5.08mm_Horizontal, B.Cu at (192.0, 83.8)
- added JBAT1: Conn_01x02_Female, Connector_Molex:Molex_Micro-Fit_3.0_43045-0200_2x01_P3.00mm_Horizontal, B.Cu at (144.0, 76.2)
- added Q1: FDN340P, Package_TO_SOT_SMD:SOT-23, B.Cu at (197.8, 71.1)
- added R1: 100K, Resistor_THT:R_Axial_DIN0204_L3.6mm_D1.6mm_P5.08mm_Horizontal, B.Cu at (192.0, 74.9)
- added U4: MCP112-300E/TO, Package_TO_SOT_THT:TO-92_Inline, B.Cu at (196.6, 73.9)
- C3: value C_Small -> 0.1uF
- C4: value C_Small -> 10uF
- moved U3 5.08 mm to (200.7, 81.3)
- moved C4 2.41 mm to (188.6, 76.7), turned to 90 degrees
- moved J5-2 1.80 mm to (125.5, 100.3)
- moved J5-1 1.80 mm to (143.5, 97.8)
- moved J1 1.27 mm to (161.3, 132.0)
- moved C1 0.91 mm to (221.7, 101.9)
- moved C2 0.91 mm to (226.2, 101.9)
- moved C3 0.64 mm to (188.6, 83.8)
Connections:
- C3 pad 1: /VIN -> /GND2
- C3 pad 2: /GND2 -> /VBAT
- C4 pad 1: /5V3 -> /VOUT
- JAUX1 pad 2: /GND3 -> /GND2
- U3 pad 1: /VIN -> /VBAT
- U3 pad 3: /5V3 -> /VOUT
Routing:
- net /VBAT: track 0.00 -> 58.7 mm
- net /VOUT: track 0.00 -> 19.7 mm
- net /GND2: track 3.37 -> 14.7 mm
- net /VIN: track 7.76 -> 0.00 mm
- net Net-(U4-Pad1): track 0.00 -> 3.84 mm
- net /CAMTX: track 16.3 -> 15.0 mm
- net /CAMRX: track 10.1 -> 8.87 mm
- net /BMESCK: track 53.5 -> 52.4 mm
Other:
- board text added: "C12666MA"
- board text added: "GROUND"
- board text added: "SKY"

Commit message: SpectDrone Development
Parts:
- added C5: 0.1uF, Capacitor_THT:C_Disc_D5.0mm_W2.5mm_P2.50mm, B.Cu at (130.2, 84.3)
- added C6: 10uF, Capacitor_THT:C_Disc_D5.0mm_W2.5mm_P2.50mm, B.Cu at (130.2, 77.2)
- added D2: D, Diode_THT:D_T-1_P5.08mm_Horizontal, B.Cu at (133.6, 84.3)
- added JAPC-2: APC220, Connector_PinSocket_2.54mm:PinSocket_1x07_P2.54mm_Vertical, B.Cu at (150.5, 111.0)
- added JBAT2: Conn_01x02_Female, Connector_Molex:Molex_Micro-Fit_3.0_43045-0200_2x01_P3.00mm_Horizontal, B.Cu at (150.4, 76.2)
- added JD1: Display, Connector_PinSocket_2.54mm:PinSocket_1x08_P2.54mm_Vertical, B.Cu at (111.7, 72.1)
- added JD2: Display, Connector_PinSocket_2.54mm:PinSocket_1x11_P2.54mm_Vertical, B.Cu at (123.2, 75.6)
- added Q2: FDN340P, Package_TO_SOT_SMD:SOT-23, B.Cu at (139.4, 71.6)
- added R2: 100K, Resistor_THT:R_Axial_DIN0204_L3.6mm_D1.6mm_P5.08mm_Horizontal, B.Cu at (133.6, 75.4)
- added R3: 330, Resistor_THT:R_Axial_DIN0204_L3.6mm_D1.6mm_P5.08mm_Horizontal, B.Cu at (94.0, 113.0)
- added R4: 10K, Resistor_THT:R_Axial_DIN0204_L3.6mm_D1.6mm_P5.08mm_Horizontal, B.Cu at (78.7, 108.7)
- added SW1: SW_Push, Button_Switch_THT:SW_PUSH_6mm_H5mm, B.Cu at (69.6, 113.5)
- added U5: MCP112-300E/TO, Package_TO_SOT_THT:TO-92_Inline, B.Cu at (138.2, 74.4)
- added U6: LM7805_TO220, Package_TO_SOT_THT:TO-220-3_Vertical, B.Cu at (142.2, 81.8)
- added U7: Teensy3.2, Teensy:Teensy30_31_32_LC, B.Cu at (108.0, 125.7)
- moved C1 40.6 mm to (262.3, 101.9)
- moved C2 40.6 mm to (266.9, 101.9)
- moved C3 40.6 mm to (229.2, 83.8)
- moved C4 40.6 mm to (229.2, 76.7)
- moved H1 40.6 mm to (256.4, 134.9)
- moved H2 40.6 mm to (256.4, 68.9)
- moved H5 40.6 mm to (229.1, 116.1)
- moved H6 40.6 mm to (257.1, 88.1)
- moved H7 40.6 mm to (257.1, 116.1)
- moved H8 40.6 mm to (229.1, 88.1)
- moved J1 40.6 mm to (201.9, 132.0)
- moved J4 40.6 mm to (186.1, 85.1)
- moved J5-1 40.6 mm to (184.2, 97.8)
- moved JAPC-1 40.6 mm to (223.5, 111.0)
- moved JAPC1 40.6 mm to (235.0, 125.5)
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- renumbered J3 to JAPC-1
Connections:
- D1 pad 1: /GND2 -> /5V3
- D1 pad 2: /5V3 -> /VIN1
- Q1 pad 2: /GND2 -> /5V3
- R1 pad 1: /5V3 -> /VIN1
- U4 pad 2: /5V3 -> /VIN1
Routing:
- net /SCLK: track 0.00 -> 114.2 mm
- net /MOSI_T: track 0.00 -> 104.2 mm
- net /D/C: track 0.00 -> 86.0 mm
- net /RST: track 0.00 -> 82.3 mm
- net /3V: track 0.00 -> 62.1 mm
- net /SCE: track 0.00 -> 48.1 mm
- net /APC2TX: track 0.00 -> 41.8 mm
- net /APC2RX: track 0.00 -> 41.5 mm
- net /SW2: track 0.00 -> 41.0 mm
- net /LED: track 0.00 -> 39.0 mm
- net Net-(JD1-Pad8): track 0.00 -> 35.8 mm
- net /MISO_T: track 0.00 -> 34.5 mm
- net /VBAT2: track 0.00 -> 27.6 mm
- net /SW1: track 0.00 -> 26.9 mm
- net /VOUT2: track 0.00 -> 19.7 mm
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- added copper zone on B.Cu, net /5V4
- added copper zone on F.Cu, net /GND4
Other:
- board size 115.7 x 71.1 mm -> 208.6 x 71.1 mm
- board text added: "3V"
- board text added: "3Vo"
- board text added: "D/C"
- board text added: "LED"
- board text added: "RST"
- board text added: "SCE"
- board text added: "SCLK"

Commit message: SpectDrone Development
Parts:
- added BT1: Battery_Cell, Battery:BatteryHolder_Keystone_500, B.Cu at (133.3, 96.5)
- added H13: MountingHole, MountingHole:MountingHole_2.2mm_M2_ISO14580_Pad_TopBottom, F.Cu at (156.9, 68.9)
- added H14: MountingHole, MountingHole:MountingHole_2.2mm_M2_ISO14580_Pad_TopBottom, F.Cu at (69.5, 68.9)
- added H15: MountingHole, MountingHole:MountingHole_2.2mm_M2_ISO14580_Pad_TopBottom, F.Cu at (69.5, 135.2)
- added H16: MountingHole, MountingHole:MountingHole_2.2mm_M2_ISO14580_Pad_TopBottom, F.Cu at (156.9, 134.9)
- added H17: MountingHole, MountingHole:MountingHole_2.5mm, F.Cu at (123.2, 73.0)
- added H18: MountingHole, MountingHole:MountingHole_2.5mm, F.Cu at (123.2, 104.8)
- added H19: MountingHole, MountingHole:MountingHole_2.5mm, F.Cu at (71.2, 104.8)
- added H20: MountingHole, MountingHole:MountingHole_2.5mm, F.Cu at (71.2, 73.0)
- added SW2: SW_Push, Button_Switch_THT:SW_PUSH_6mm_H4.3mm, B.Cu at (86.4, 118.1)
- added SW3: SW_Push, Button_Switch_THT:SW_PUSH_6mm_H4.3mm, B.Cu at (76.2, 118.1)
- added SW4: SW_Push, Button_Switch_THT:SW_PUSH_6mm_H4.3mm, B.Cu at (66.0, 118.1)
- added SW5: SW_Push, Button_Switch_THT:SW_PUSH_6mm_H4.3mm, B.Cu at (76.2, 126.3)
- added SW6: SW_Push, Button_Switch_THT:SW_PUSH_6mm_H4.3mm, B.Cu at (86.4, 126.3)
- SW1: footprint Button_Switch_THT:SW_PUSH_6mm_H5mm -> Button_Switch_THT:SW_PUSH_6mm_H4.3mm
- moved R4 26.7 mm to (88.9, 133.3), turned to 180 degrees
- moved SW1 7.53 mm to (76.2, 109.8), turned to 180 degrees
- moved R3 1.80 mm to (95.2, 114.3)
- moved JD1 0.88 mm to (112.2, 72.9)
- moved R2 0.76 mm to (133.6, 76.2)
- moved R1 0.63 mm to (232.7, 75.6)
- moved JD2 0.61 mm to (123.2, 76.2)
Connections:
- JD1 pad 3: /SCE -> /DCS
- JD2 pad 7: /TCS -> /DCS
- R4 pad 1: Net-(R4-Pad1) -> /5V4
- R4 pad 2: /SW1 -> Net-(SW1-Pad1)
- SW1 pad 1: /SW2 -> Net-(SW1-Pad1)
- SW1 pad 2: Net-(R4-Pad1) -> /SW1
- U7 pad 10: unconnected-(U7-Pad10) -> /SDCS
- U7 pad 15: unconnected-(U7-Pad15) -> /VBAT_RTC
- U7 pad 22: unconnected-(U7-Pad22) -> /SW1
- U7 pad 23: unconnected-(U7-Pad23) -> /SW2
- U7 pad 24: unconnected-(U7-Pad24) -> /SW3
- U7 pad 25: unconnected-(U7-Pad25) -> /SW4
- U7 pad 26: unconnected-(U7-Pad26) -> /SW5
- U7 pad 29: /SW2 -> unconnected-(U7-Pad29)
- U7 pad 31: /SW1 -> unconnected-(U7-Pad31)
- U7 pad 37: unconnected-(U7-Pad37) -> /SW6
- U7 pad 9: /SCE -> /DCS
Routing:
- net Net-(SW1-Pad1): track 0.00 -> 101.3 mm
- net /DCS: track 0.00 -> 56.7 mm
- net /SW4: track 0.00 -> 56.7 mm
- net /SW3: track 0.00 -> 49.0 mm
- net /SCE: track 48.1 -> 0.00 mm
- net /SW5: track 0.00 -> 42.9 mm
- net /SW1: track 26.9 -> 57.6 mm
- net /VBAT_RTC: track 0.00 -> 29.1 mm
- net /SW6: track 0.00 -> 26.2 mm
- net /SDCS: track 0.00 -> 22.7 mm
- net /GND4: track 8.13 -> 0.00 mm
- net /VIN1: track 0.00 -> 7.90 mm
- net /VIN2: track 0.00 -> 7.83 mm
- net /VOUT: track 19.7 -> 21.5 mm
- net /VOUT2: track 19.7 -> 21.4 mm
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Other:
- board size 208.6 x 71.1 mm -> 220.1 x 71.1 mm
- board text added: "BKL"
- board text added: "DCS"
- board text added: "SDCS"

Commit message: SpectDrone Development
Parts:
- added D3: Ge, Diode_THT:D_T-1_P5.08mm_Horizontal, B.Cu at (170.9, 142.5)
- added SW0: SW_Push, Button_Switch_THT:SW_PUSH_6mm_H4.3mm, B.Cu at (52.2, 109.2)
- added SW7: SW_Push, Button_Switch_THT:SW_PUSH_6mm_H4.3mm, B.Cu at (72.5, 134.0)
- added SW8: SW_Push, Button_Switch_THT:SW_PUSH_6mm_H4.3mm, B.Cu at (62.4, 134.0)
- added SW9: SW_Push, Button_Switch_THT:SW_PUSH_6mm_H4.3mm, B.Cu at (52.2, 134.0)
- moved RSW1 46.7 mm to (51.4, 105.4)
- moved SW6 34.1 mm to (52.2, 125.7)
- moved H14 26.0 mm to (44.7, 76.8)
- moved H15 25.9 mm to (44.7, 142.9)
- moved SW3 24.0 mm to (52.2, 117.5)
- moved SW2 24.0 mm to (62.4, 117.5)
- moved JBAT2 20.4 mm to (131.6, 84.1)
- moved C1 19.9 mm to (244.0, 109.8)
- moved C2 19.9 mm to (248.6, 109.8)
- moved H1 19.9 mm to (238.1, 142.9)
- moved H13 19.9 mm to (138.7, 76.8)
- moved H16 19.9 mm to (138.7, 142.9)
- moved H2 19.9 mm to (238.1, 76.8)
- moved H3 19.9 mm to (144.2, 76.8)
- moved H4 19.9 mm to (144.2, 142.9)
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- renumbered R4 to RSW1
Connections:
- BT1 pad 2: /GND4 -> /GND2
- C1 pad 2: /GND2 -> /GND1
- C2 pad 2: /GND2 -> /GND1
- C3 pad 1: /GND2 -> /GND1
- C4 pad 2: /GND2 -> /GND1
- C5 pad 1: /GND4 -> /GND2
- C6 pad 2: /GND4 -> /GND2
- J1 pad 2: /GND2 -> /GND1
- J4 pad 3: /GND2 -> /GND1
- J5-1 pad 4: /GND2 -> /GND1
- JAPC-1 pad 7: /GND2 -> /GND1
- JAPC-2 pad 7: /GND4 -> /GND2
- JAUX1 pad 1: /5V3 -> Net-(JAUX1-Pad1)
- JAUX1 pad 2: /GND2 -> /GND1
- JBAT1 pad 2: /GND2 -> /GND1
- JBAT2 pad 2: /GND4 -> /GND2
- JD1 pad 2: /GND4 -> /GND2
- JD2 pad 3: /GND4 -> /GND2
- JIR1 pad 2: /GND2 -> /GND1
- R1 pad 2: /GND2 -> /GND1
- R2 pad 2: /GND4 -> /GND2
- RSW1 pad 1: /5V4 -> /GND2
- RSW1 pad 2: Net-(SW1-Pad1) -> Net-(RSW1-Pad2)
- SW1 pad 1: Net-(SW1-Pad1) -> /SW1
- SW1 pad 2: /SW1 -> Net-(RSW1-Pad2)
- SW2 pad 1: Net-(SW1-Pad1) -> /SW2
- SW2 pad 2: /SW2 -> Net-(RSW1-Pad2)
- SW3 pad 1: Net-(SW1-Pad1) -> /SW3
- SW3 pad 2: /SW3 -> Net-(RSW1-Pad2)
- SW4 pad 1: Net-(SW1-Pad1) -> /SW4
- SW4 pad 2: /SW4 -> Net-(RSW1-Pad2)
- SW5 pad 1: Net-(SW1-Pad1) -> /SW5
- SW5 pad 2: /SW5 -> Net-(RSW1-Pad2)
- SW6 pad 1: Net-(SW1-Pad1) -> /SW6
- SW6 pad 2: /SW6 -> Net-(RSW1-Pad2)
- U1 pad 3: /GND2 -> /GND1
- U1 pad 5: /GND2 -> /GND1
- U2 pad 3: /GND2 -> /GND1
- U2 pad 5: /GND2 -> /GND1
- U3 pad 2: /GND2 -> /GND1
- U4 pad 3: /GND2 -> /GND1
- U5 pad 3: /GND4 -> /GND2
- U6 pad 2: /GND4 -> /GND2
- U7 pad 1: /GND4 -> /GND2
- U7 pad 17: /GND4 -> /GND2
- U7 pad 22: /SW1 -> /SW0
- U7 pad 23: /SW2 -> /SW1
- U7 pad 24: /SW3 -> /SW2
- U7 pad 25: /SW4 -> /SW3
- U7 pad 26: /SW5 -> /SW4
- U7 pad 27: unconnected-(U7-Pad27) -> /SW6
- U7 pad 28: unconnected-(U7-Pad28) -> /SW7
- U7 pad 29: unconnected-(U7-Pad29) -> /SW8
- U7 pad 30: unconnected-(U7-Pad30) -> /SW9
- U7 pad 37: /SW6 -> /SW5
Routing:
- net Net-(RSW1-Pad2): track 0.00 -> 125.3 mm
- net Net-(SW1-Pad1): track 101.3 -> 0.00 mm
- net /SW0: track 0.00 -> 81.0 mm
- net /SW9: track 0.00 -> 36.7 mm
- net /SW8: track 0.00 -> 35.6 mm
- net /SW6: track 26.2 -> 55.0 mm
- net /SW7: track 0.00 -> 28.7 mm
- net /SW4: track 56.7 -> 37.0 mm
- net /SW2: track 41.4 -> 59.3 mm
- net /SW3: track 49.0 -> 66.8 mm
- net /SW1: track 57.6 -> 51.7 mm
- net /VBAT_RTC: track 29.1 -> 25.3 mm
- net Net-(JAUX1-Pad1): track 0.00 -> 3.81 mm
- net /GND1: track 0.00 -> 3.37 mm, vias 0 -> 2
- net /GND2: track 3.37 -> 0.00 mm, vias 2 -> 0
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- added copper zone on F.Cu, net /GND1
- removed copper zone on F.Cu, net /GND4
Other:
- board size 220.1 x 71.1 mm -> 215 x 71.1 mm
