File: SpectDrone/SpectDrone.kicad_pcb (KiCad board)
At the start: 2 copper layers, 215 x 71.1 mm, 69 parts, among them J1 Camera, J2 GPS, J4 BME280, J5-1 BNO055-1, J5-2 BNO055-2, Q1 FDN340P, Q2 FDN340P, SW0 SW_Push, SW1 SW_Push, SW2 SW_Push, SW3 SW_Push, SW4 SW_Push, SW5 SW_Push, SW6 SW_Push, SW7 SW_Push, SW8 SW_Push, SW9 SW_Push, U1 C12666MA, U2 C12666MA, U3 LM7805_TO220, U4 MCP112-300E/TO, U5 MCP112-300E/TO, U6 LM7805_TO220, U7 Teensy3.2

Commit message: SpectDrone Development
Parts:
- added SW10: SW_Push, Button_Switch_THT:SW_PUSH_6mm_H4.3mm, B.Cu at (52.2, 101.5)
- added TP1: TestPoint, TestPoint:TestPoint_Keystone_5000-5004_Miniature, B.Cu at (221.7, 79.5)
- moved RSW1 7.24 mm to (51.3, 98.2)
- moved C3 3.18 mm to (207.8, 91.7)
- moved C4 3.18 mm to (207.8, 84.6)
- moved D1 3.18 mm to (211.2, 91.7)
- moved R1 3.18 mm to (211.2, 83.5)
- moved U3 3.18 mm to (219.8, 89.2)
- moved U4 3.18 mm to (215.8, 81.8)
- moved Q1 3.17 mm to (217.0, 79.0)
- moved SW9 0.81 mm to (52.7, 134.6)
- moved H17 0.64 mm to (110.0, 81.7)
- moved H20 0.64 mm to (58.0, 81.7)
- moved JD2 0.64 mm to (110.0, 84.9)
- moved SW0 0.64 mm to (52.2, 109.9)
- moved SW1 0.64 mm to (72.5, 118.1)
- moved SW2 0.64 mm to (62.4, 118.1)
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Connections:
- U7 pad 22: /SW0 -> /SW10
- U7 pad 23: /SW1 -> /SW0
- U7 pad 24: /SW2 -> /SW1
- U7 pad 25: /SW3 -> /SW2
- U7 pad 26: /SW4 -> /SW3
- U7 pad 27: /SW6 -> /SW5
- U7 pad 36: unconnected-(U7-Pad36) -> /SW6
- U7 pad 37: /SW5 -> /SW4
Routing:
- net /SW10: track 0.00 -> 88.3 mm
- net Net-(SW10-Pad2): track 125.3 -> 140.9 mm
- net /SW6: track 55.0 -> 48.4 mm
- net /SW4: track 37.0 -> 30.6 mm
- net /SW9: track 36.7 -> 42.4 mm
- net /VOUT: track 21.5 -> 25.6 mm
- net /SW5: track 41.0 -> 44.7 mm
- net /SW2: track 59.3 -> 55.7 mm
- net /SW1: track 51.7 -> 48.2 mm
- net /SW3: track 66.8 -> 63.4 mm
- net /SW0: track 81.0 -> 77.8 mm
- net /VBAT: track 58.5 -> 55.9 mm
- net /3V: track 62.5 -> 63.1 mm
- net /RST: track 80.7 -> 80.1 mm
- net /D/C: track 85.5 -> 86.2 mm
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
Commit message: SpectDrone Development
Parts:
- added JAPC-2: APC220, Connector_PinSocket_2.54mm:PinSocket_1x07_P2.54mm_Vertical, B.Cu at (134.1, 109.7)
- JAPC-3: renamed from JAPC-2; moved to F.Cu
- moved BT1 23.2 mm to (117.0, 130.3)
- moved JAPC-3 9.31 mm to (134.1, 109.7), turned to -90 degrees
- moved JAPC-1 9.31 mm to (203.7, 109.7)
- moved H10 2.91 mm to (203.8, 76.8)
- moved H11 2.91 mm to (203.8, 104.8)
- moved H12 2.91 mm to (175.8, 76.8)
- moved H9 2.91 mm to (175.8, 104.8)
Routing:
- net /VBAT_RTC: track 25.3 -> 6.38 mm
- net /APC2RX: track 40.2 -> 51.8 mm
- net /APC2TX: track 40.4 -> 52.0 mm
- net /ST: track 125.4 -> 136.9 mm
- net /CLK2: track 78.3 -> 87.9 mm
- net /APCRX: track 26.1 -> 34.8 mm
- net /APCTX: track 22.5 -> 31.2 mm

Commit message: SpectDrone Development
Parts:
- added JVIN1: Conn_01x01_Male, Connector_PinHeader_2.54mm:PinHeader_1x01_P2.54mm_Vertical, F.Cu at (227.7, 82.4)
- added TP2: TestPoint, TestPoint:TestPoint_Keystone_5000-5004_Miniature, B.Cu at (227.7, 79.5)
- added TP3: TestPoint, TestPoint:TestPoint_Keystone_5000-5004_Miniature, B.Cu at (232.3, 79.5)
- moved C3 1.40 mm to (209.2, 91.7)
- moved C4 1.40 mm to (209.2, 84.6)
- moved D1 1.40 mm to (212.6, 91.7)
- moved R1 1.40 mm to (212.6, 83.5)
- moved TP1 1.40 mm to (223.1, 79.5)
- moved U3 1.40 mm to (221.2, 89.2)
- moved Q1 1.40 mm to (218.4, 79.0)
- moved U4 1.40 mm to (217.2, 81.8)
- moved H17 0.64 mm to (110.0, 81.1)
- moved H20 0.64 mm to (58.0, 81.1)
- moved JD2 0.64 mm to (110.0, 84.2)
- moved H18 0.63 mm to (110.0, 112.8)
- moved H19 0.63 mm to (58.0, 112.8)
Routing:
- net /VIN1: track 7.90 -> 33.4 mm
- net /VBAT: track 55.9 -> 57.3 mm
- net /DCS: track 56.7 -> 58.0 mm
- net /RST: track 80.1 -> 80.7 mm
- net /SDCS: track 22.1 -> 22.7 mm
- net /D/C: track 86.2 -> 85.6 mm
- net /MOSI_T: track 103.1 -> 103.6 mm
- net /MISO_T: track 33.7 -> 34.2 mm
Other:
- board text added: "Display"
- board text added: "VIN"

Commit message: SpectDrone Development
Parts:
- moved Q1 9.71 mm to (208.7, 78.9), turned to 180 degrees
- moved J1 4.88 mm to (178.8, 140.6)
- moved JAUX1 4.86 mm to (169.9, 143.2)
- moved J2 4.83 mm to (152.1, 130.1)
- moved JGPS1 4.82 mm to (157.2, 129.9)
- moved U3 4.64 mm to (216.8, 90.5)
- moved D3 4.39 mm to (166.6, 141.7)
- moved U4 3.04 mm to (216.5, 78.9), turned to 0 degrees
- moved C4 1.35 mm to (209.2, 86.0)
- moved JAPC-1 0.13 mm to (203.7, 109.9)
- moved JAPC-2 0.13 mm to (134.1, 109.9)
- moved JAPC-3 0.13 mm to (134.1, 109.9)
Connections:
- C3 pad 2: /VBAT -> /7-12V
- C4 pad 1: /VOUT -> /5V3
- D1 pad 1: /5V3 -> /7-12V
- Q1 pad 2: /5V3 -> /7-12V
- Q1 pad 3: /VOUT -> /VBAT
- TP1 pad 1: /VOUT -> /5V3
- U3 pad 1: /VBAT -> /7-12V
- U3 pad 3: /VOUT -> /5V3
Routing:
- net /5V3: track 0.00 -> 30.9 mm
- net /VOUT: track 25.6 -> 0.00 mm
- net /7-12V: track 0.00 -> 20.4 mm
- net /VBAT: track 57.3 -> 43.5 mm
- net /VIN1: track 33.4 -> 26.6 mm
- net /CLK2: track 87.9 -> 94.1 mm
- net /ST: track 136.9 -> 142.8 mm
- net Net-(Q1-Pad1): track 3.84 -> 8.23 mm
- net /CLK1: track 85.1 -> 87.7 mm
- net /BMESDI: track 51.6 -> 49.5 mm
- net /BMESCK: track 52.4 -> 51.1 mm
- net /DCS: track 58.0 -> 56.8 mm
- net /VBAT2: track 26.6 -> 26.1 mm
Other:
- outline, holes or cut-outs redrawn

Commit message: SpectDrone Development
Parts:
- added J3: Barrel_Jack, Connector_BarrelJack:BarrelJack_Horizontal, B.Cu at (52.1, 88.3)
- U4, U5: footprint Package_TO_SOT_THT:TO-92_Inline -> Package_TO_SOT_SMD:SOT-89-3
- moved C6 21.1 mm to (136.5, 95.8), turned to 180 degrees
- moved Q2 18.6 mm to (135.0, 100.0), turned to 180 degrees
- moved D2 17.8 mm to (135.9, 104.1), turned to 180 degrees
- moved R2 17.0 mm to (131.5, 100.9)
- moved D1 14.5 mm to (210.2, 77.5), turned to 0 degrees
- moved U5 13.9 mm to (127.0, 100.4), turned to 90 degrees
- moved C5 12.6 mm to (128.9, 95.8), turned to 180 degrees
- moved R3 10.9 mm to (90.9, 128.7), turned to 180 degrees
- moved C3 9.99 mm to (217.2, 85.7), turned to 0 degrees
- moved U6 3.94 mm to (128.9, 90.2), turned to 0 degrees
- moved JD1 3.87 mm to (102.9, 80.9)
- moved H19 3.87 mm to (61.9, 112.8)
- moved H20 3.87 mm to (61.9, 81.1)
- moved H17 3.87 mm to (113.9, 81.1)
- moved H18 3.87 mm to (113.9, 112.8)
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Connections:
- net /7-12V renamed /7-12V1
- C5 pad 2: /VBAT2 -> /7-12V2
- C6 pad 1: /VOUT2 -> /5V4
- D2 pad 1: /5V4 -> /7-12V2
- JD1 pad 8: Net-(JD1-Pad8) -> /BKL
- Q2 pad 2: /5V4 -> /7-12V2
- Q2 pad 3: /VOUT2 -> /VBAT2
- R3 pad 2: Net-(JD1-Pad8) -> /BKL
- U6 pad 1: /VBAT2 -> /7-12V2
- U6 pad 3: /VOUT2 -> /5V4
- U7 pad 21: /LED -> unconnected-(U7-Pad21)
- U7 pad 5: /D/C -> unconnected-(U7-Pad5)
- U7 pad 6: unconnected-(U7-Pad6) -> /LED
- U7 pad 7: unconnected-(U7-Pad7) -> /D/C
Routing:
- net /VIN2: track 7.83 -> 123.0 mm
- net /BKL: track 0.00 -> 82.0 mm, vias 0 -> 4
- net Net-(JD1-Pad8): track 36.7 -> 0.00 mm
- net /LED: track 37.2 -> 2.55 mm
- net /7-12V2: track 0.00 -> 31.3 mm
- net /GND2: track 0.00 -> 22.8 mm
- net /GND1: track 3.37 -> 26.2 mm
- net /VOUT2: track 21.4 -> 0.00 mm
- net /VBAT: track 43.5 -> 56.8 mm
- net /7-12V1: track 20.4 -> 31.2 mm
- net /VBAT2: track 26.1 -> 36.4 mm
- net /5V4: track 0.00 -> 6.63 mm
- net Net-(Q2-Pad1): track 3.84 -> 9.96 mm
- net /5V3: track 30.9 -> 26.9 mm
- net /VIN1: track 26.6 -> 22.9 mm
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Other:
- board text removed: "BKL"

Commit message: SpectDrone Development
Parts:
- removed JAPC-3: APC220, Connector_PinSocket_2.54mm:PinSocket_1x07_P2.54mm_Vertical
- JIR1: value Conn_01x04_Male -> Infrared
Connections:
- net /VBAT renamed /VBAT1
Routing:
- net /BMESCK: track 52.0 -> 51.4 mm
- net /BKL: vias 4 -> 2

Commit message: SpectDrone Development
Parts:
- moved J5-2 18.3 mm to (162.7, 97.4), turned to 90 degrees
- moved J5-1 9.75 mm to (165.2, 115.4), turned to 90 degrees
- moved R3 7.90 mm to (88.9, 121.1)
- moved JBAT1 0.63 mm to (165.7, 84.1)
- moved J4 0.63 mm to (167.1, 93.0)
- moved TP1 0.39 mm to (223.5, 79.5)
- moved TP3 0.35 mm to (231.9, 79.5)
- moved C4 0.22 mm to (209.4, 85.8)
- moved C3 0.21 mm to (217.4, 85.8)
- moved C5 0.21 mm to (128.7, 95.8)
- moved C6 0.21 mm to (136.7, 95.8)
- moved D1 0.06 mm to (210.2, 77.5)
- moved R1 0.06 mm to (214.6, 80.7)
- moved U3 0.06 mm to (217.2, 91.4)
- moved U4 0.06 mm to (219.1, 81.2)
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Routing:
- net /BKL: track 82.0 -> 76.6 mm
- net /LED: track 2.52 -> 5.94 mm
- net /BMESCK: track 51.4 -> 50.4 mm
Other:
- board text added: "PPS"

Commit message: SpectDrone Development
Parts:
- removed J1: Camera, Connector_JST:JST_XH_B4B-XH-A_1x04_P2.50mm_Vertical
- added H5: MountingHole, MountingHole:MountingHole_2.2mm_M2_ISO14580_Pad_TopBottom, F.Cu at (242.3, 124.6)
- added H6: MountingHole, MountingHole:MountingHole_2.2mm_M2_ISO14580_Pad_TopBottom, F.Cu at (270.3, 96.6)
- added H7: MountingHole, MountingHole:MountingHole_2.2mm_M2_ISO14580_Pad_TopBottom, F.Cu at (270.3, 124.6)
- added H8: MountingHole, MountingHole:MountingHole_2.2mm_M2_ISO14580_Pad_TopBottom, F.Cu at (242.3, 96.6)
- added JCAM1: Conn_01x04_Male, Connector_PinHeader_2.54mm:PinHeader_1x04_P2.54mm_Vertical, F.Cu at (198.2, 134.2)
- added JCAM2: Camera, Connector_JST:JST_XH_B4B-XH-A_1x04_P2.50mm_Vertical, B.Cu at (205.7, 132.1)
- added JCAM3: Camera, Connector_JST:JST_XH_B4B-XH-A_1x04_P2.50mm_Vertical, B.Cu at (205.7, 140.9)
- added JD1: Conn_01x04_Male, Connector_PinHeader_2.54mm:PinHeader_1x04_P2.54mm_Vertical, F.Cu at (198.1, 105.0)
- H21: renamed from H8; moved to B.Cu
- H22: renamed from H6; moved to B.Cu
- H23: renamed from H7; moved to B.Cu
- H24: renamed from H5; moved to B.Cu
- moved H21 59.6 mm to (270.4, 96.6), turned to 180 degrees
- moved H24 59.6 mm to (270.4, 124.6), turned to 180 degrees
- moved JAPC1 26.1 mm to (190.6, 134.2)
- moved Q2 18.5 mm to (116.6, 100.8)
- moved SW1 18.5 mm to (52.1, 118.9)
- moved SW4 18.5 mm to (52.1, 127.1)
- moved BT1 18.5 mm to (98.5, 131.1)
- moved C1 18.5 mm to (225.6, 110.6)
- moved C2 18.5 mm to (230.1, 110.6)
- moved C3 18.5 mm to (198.9, 86.5)
- moved C4 18.5 mm to (190.9, 86.5)
- moved C5 18.5 mm to (110.3, 96.6)
- moved C6 18.5 mm to (118.3, 96.6)
- moved D1 18.5 mm to (191.7, 78.3)
- moved D3 18.5 mm to (148.2, 142.5)
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- renumbered JD1 to JDIS1, JD2 to JDIS2
Connections:
- JA1 pad 1: /A1 -> unconnected-(JA1-Pad1)
- JA1 pad 2: /A2 -> /A1
- JA1 pad 3: /GAIN -> /A2
- JAUX1 pad 10: /CLK2 -> /OPT_EXT
- JAUX1 pad 11: /CLK1 -> /D12
- JAUX1 pad 4: /CAMRX -> /SS_AUX
- JAUX1 pad 8: /CAMTX -> /XCL
- JAUX1 pad 9: /ST -> /XDA
Routing:
- net /ST: track 142.8 -> 82.1 mm
- net /CLK2: track 94.1 -> 35.5 mm
- net /CLK1: track 87.7 -> 34.0 mm
- net /CAM1TX: track 0.00 -> 17.5 mm
- net /CAM1RX: track 0.00 -> 15.6 mm
- net /CAM2TX: track 0.00 -> 15.3 mm
- net /CAM2RX: track 0.00 -> 14.1 mm
- net /CAMTX: track 12.1 -> 0.00 mm
- net /CAMRX: track 8.87 -> 0.00 mm
- net /GAIN: track 64.5 -> 57.1 mm
- net /APCTX: track 31.1 -> 27.9 mm
- net /APCRX: track 34.7 -> 31.5 mm
- net /5V3: track 27.0 -> 25.3 mm
- net /A1: track 37.3 -> 38.3 mm
- net /GND1: track 26.2 -> 25.4 mm
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Other:
- board size 215 x 71.1 mm -> 250.4 x 71.1 mm
- board text added: "GROUND CAMERA"
- board text added: "Ground Camera"
- board text added: "SKY CAMERA"
- board text added: "SPECT_ VIDEO_1"
- board text added: "SPECT_ VIDEO_2"
- board text added: "Sky Camera"
- board text removed: "CAMERA"
- board text removed: "Camera"
- board text removed: "SPECT_VIDEO_1"
- board text removed: "SPECT_VIDEO_2"
