File: SpectDrone/SpectDrone.kicad_pcb (KiCad board)
At the start: 2 copper layers, 250.4 x 71.1 mm, 82 parts, among them J2 GPS, J3 Barrel_Jack, J4 BME280, J5-1 BNO055-1, J5-2 BNO055-2, Q1 FDN340P, Q2 FDN340P, SW0 SW_Push, SW1 SW_Push, SW10 SW_Push, SW2 SW_Push, SW3 SW_Push, SW4 SW_Push, SW5 SW_Push, SW6 SW_Push, SW7 SW_Push, SW8 SW_Push, SW9 SW_Push, U1 C12666MA, U2 C12666MA, U3 LM7805_TO220, U4 MCP112-300E/TO, U5 MCP112-300E/TO, U6 LM7805_TO220, U7 Teensy3.2

Commit message: SpectDrone Development
Parts:
- added R6: R, Resistor_SMD:R_0603_1608Metric_Pad0.98x0.95mm_HandSolder, B.Cu at (210.8, 101.8)
- added RV1: R_Potentiometer, Potentiometer_THT:Potentiometer_Bourns_3296W_Vertical, B.Cu at (205.7, 67.5)
- added TP4: TestPoint, TestPoint:TestPoint_Keystone_5000-5004_Miniature, B.Cu at (213.3, 84.7)
- added U8: ADR510, Package_TO_SOT_SMD:SOT-23, B.Cu at (206.6, 62.3)
- added U9: AD8620, Package_DIP:DIP-8_W7.62mm, B.Cu at (203.2, 98.0)
- H21, H22, H23, H24: footprint MountingHole:MountingHole_2.2mm_M2_ISO14580_Pad_TopBottom -> MountingHole:MountingHole_2.5mm
Connections:
- JA1 pad 1: unconnected-(JA1-Pad1) -> /PD1
- JA1 pad 4: unconnected-(JA1-Pad4) -> /PD2
Routing:
- net /1.0V: track 0.00 -> 20.0 mm
- net /PD1: track 0.00 -> 2.54 mm
- net /PD2: track 0.00 -> 2.54 mm
Other:
- board text added: "1.000V"

Commit message: SpectDrone Development
Parts:
- added D4: S1336-18BK, Package_TO_SOT_THT:TO-18-4_Lens, B.Cu at (225.8, 138.1)
- added D5: S1336-18BK, Package_TO_SOT_THT:TO-18-4_Lens, F.Cu at (225.8, 83.2)
- added R10: R, Resistor_SMD:R_0603_1608Metric_Pad0.98x0.95mm_HandSolder, B.Cu at (215.5, 90.6)
- added R4: R, Resistor_SMD:R_0603_1608Metric_Pad0.98x0.95mm_HandSolder, B.Cu at (209.0, 96.5)
- added R5: R, Resistor_SMD:R_0603_1608Metric_Pad0.98x0.95mm_HandSolder, B.Cu at (215.5, 89.0)
- added R9: R, Resistor_SMD:R_0603_1608Metric_Pad0.98x0.95mm_HandSolder, B.Cu at (215.5, 96.7)
- U9: value AD8620 -> MIC863; footprint Package_DIP:DIP-8_W7.62mm -> Package_TO_SOT_SMD:SOT-23-8
- moved U8 34.1 mm to (211.9, 96.0), turned to -90 degrees
- moved RV1 24.5 mm to (211.1, 91.5), turned to 0 degrees
- moved R6 14.5 mm to (210.1, 87.3), turned to 0 degrees
- moved U9 13.0 mm to (215.5, 93.7), turned to 90 degrees
- moved JAPC-1 1.64 mm to (183.6, 110.6)
- moved H10 1.20 mm to (184.1, 77.6)
- moved H11 1.20 mm to (184.1, 105.6)
- moved H12 1.20 mm to (156.1, 77.6)
- moved H9 1.20 mm to (156.1, 105.6)
- moved TP4 0.18 mm to (213.5, 84.8)
Connections:
- JA1 pad 1: /PD1 -> /S2
- JA1 pad 4: /PD2 -> /S1
- U9 pad 1: /PD1 -> /S1
- U9 pad 2: /PD1 -> Net-(D4-Pad1)
- U9 pad 6: /PD2 -> Net-(D5-Pad1)
- U9 pad 7: /PD2 -> /S2
Routing:
- net /1.0V: track 20.0 -> 128.0 mm
- net Net-(D4-Pad1): track 0.00 -> 98.4 mm
- net /S1: track 0.00 -> 42.2 mm
- net /S2: track 0.00 -> 39.7 mm
- net /GND1: track 25.4 -> 49.8 mm
- net Net-(D5-Pad1): track 0.00 -> 18.7 mm
- net Net-(RV1-Pad2): track 0.00 -> 4.61 mm
- net /PD1: track 2.54 -> 0.00 mm
- net /PD2: track 2.54 -> 0.00 mm
- net /APCTX: track 27.9 -> 29.3 mm
- net /CLK2: track 35.5 -> 36.5 mm
- net /APCRX: track 31.5 -> 32.2 mm

Commit message: SpectDrone development
Parts:
- renumbered D5 to PD1, D4 to PD2
Connections:
- JA1 pad 1: /S2 -> /S1
- JA1 pad 4: /S1 -> /S2
- R10 pad 2: /S2 -> /S1
- R9 pad 1: /S1 -> /S2
- U9 pad 1: /S1 -> /S2
- U9 pad 7: /S2 -> /S1
Routing:
- net /S1: track 42.2 -> 39.7 mm
- net /S2: track 39.7 -> 42.1 mm
- net /APC2TX: track 52.0 -> 51.3 mm
- net /ST: track 82.1 -> 82.6 mm
Other:
- outline, holes or cut-outs redrawn
- board text added: "LONG- WAVE_1"
- board text added: "LONG- WAVE_2"

Commit message: SpectDrone Development
Parts:
- removed JCAM1: Conn_01x04_Male, Connector_PinHeader_2.54mm:PinHeader_1x04_P2.54mm_Vertical
- added J1: Conn_01x01_Male, Connector_PinHeader_2.54mm:PinHeader_1x01_P2.54mm_Vertical, F.Cu at (152.9, 98.2)
- added JI2C1: Conn_01x04_Male, Connector_PinHeader_2.54mm:PinHeader_1x04_P2.54mm_Vertical, B.Cu at (155.7, 138.9)
- added JI2C3-1: Conn_01x04_Male, Connector_PinHeader_2.54mm:PinHeader_1x04_P2.54mm_Vertical, B.Cu at (163.8, 138.9)
- added U10: PCA9306DC, Package_SO:VSSOP-8_2.3x2mm_P0.5mm, B.Cu at (159.7, 137.9)
- JAUX1: footprint Connector_PinHeader_2.54mm:PinHeader_1x11_P2.54mm_Vertical -> Connector_PinHeader_2.54mm:PinHeader_1x12_P2.54mm_Vertical
- moved JAPC1 14.5 mm to (190.6, 119.7)
- moved JCAM2 6.23 mm to (209.5, 127.2)
- moved JCAM3 6.12 mm to (209.5, 136.1)
- moved PD2 4.10 mm to (229.8, 138.6)
- moved PD1 4.08 mm to (229.8, 82.8)
Connections:
- net /3V renamed /3V2
- JAUX1 pad 10: /OPT_EXT -> /CAM2TX
- JAUX1 pad 11: /D12 -> /CAM2RX
- JAUX1 pad 8: /XCL -> /CAM1TX
- JAUX1 pad 9: /XDA -> /CAM1RX
- JCAM2 pad 3: /CAM1RX -> /CAM2TX
- JCAM2 pad 4: /CAM1TX -> /CAM2RX
- JCAM3 pad 3: /CAM2RX -> /CAM1TX
- JCAM3 pad 4: /CAM2TX -> /CAM1RX
Routing:
- net /3V1: track 0.00 -> 64.7 mm, vias 0 -> 1
- net /CAM2RX: track 14.1 -> 73.9 mm
- net /CAM1RX: track 15.6 -> 71.4 mm
- net /CAM2TX: track 15.3 -> 70.0 mm
- net /CAM1TX: track 17.5 -> 67.9 mm
- net /BMESCK: track 50.4 -> 75.1 mm
- net /BMESDI: track 49.8 -> 64.2 mm
- net /APCTX: track 29.3 -> 15.8 mm
- net /APCRX: track 32.2 -> 19.4 mm
- net /GND1: track 49.8 -> 58.1 mm
- net /1.0V: track 127.7 -> 134.1 mm
- net /5V3: track 25.3 -> 31.4 mm
- net /SDA3: track 0.00 -> 6.00 mm
- net /SCL3: track 0.00 -> 4.79 mm
- net Net-(PD1-Pad1): track 18.7 -> 23.0 mm
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Other:
- outline, holes or cut-outs redrawn
- board text added: "3.3V"
- board text added: "CAM1"
- board text added: "CAM1_RX"
- board text added: "CAM1_TX"
- board text added: "CAM2"
- board text added: "CAM2_RX"
- board text added: "CAM2_TX"
- board text added: "PWM"
- board text added: "SS"
- board text removed: "CAM_RX"
- board text removed: "CAM_TX"

Commit message: SpectDrone development
Parts:
- moved JI2C1 1.02 mm to (155.7, 139.9)
- moved JI2C3-1 1.02 mm to (163.8, 139.9)
- moved U10 1.02 mm to (159.7, 138.9)
Routing:
- net /GND1: track 58.1 -> 41.8 mm, vias 2 -> 4
- net /3V1: track 64.7 -> 67.1 mm
- net /5V3: track 31.4 -> 29.3 mm
- net /BMESCK: track 75.1 -> 77.1 mm
- net /BMESDI: track 64.2 -> 65.2 mm

Commit message: SpectDrone Development
Parts:
- added TP5: TestPoint, TestPoint:TestPoint_Keystone_5000-5004_Miniature, B.Cu at (205.1, 84.8)
Routing:
- net /3V1: track 67.1 -> 138.8 mm
Changed lines of the file:
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@@
     (property "Sheetname" "")
     (attr smd)
-    (fp_text reference "U4" (at 0.702 -3.305 90) (layer "B.SilkS")
+    (fp_text reference "U4" (at 0.5896 -3.18 90) (layer "B.SilkS")
       (effects (font (size 1 1) (thickness 0.15)) (justify mirror))
     )
@@
     (property "Sheetname" "")
     (attr through_hole)
-    (fp_text reference "C3" (at 4.98 -0.03 90) (layer "B.SilkS")
+    (fp_text reference "C3" (at 4.748 0.4226 90) (layer "B.SilkS")
       (effects (font (size 1 1) (thickness 0.15)) (justify mirror))
     )
@@
     )
   )
+  (footprint "TestPoint:TestPoint_Keystone_5000-5004_Miniature" (layer "B.Cu")
+    (at 205.0809 84.7977 180)
+    (descr "Keystone Miniature THM Test Point 5000-5004, http://www.keyelco.com/product-pdf.cfm?p=1309")
+    (tags "Through Hole Mount Test Points")
+    (property "Sheetfile" "SpectDrone.kicad_sch")
+    (property "Sheetname" "")
+    (attr through_hole)
+    (fp_text reference "TP5" (at 0 2.5) (layer "B.SilkS") hide
+      (effects (font (size 1 1) (thickness 0.15)) (justify mirror))
+    )
+    (fp_text value "TestPoint" (at 0 -2.5) (layer "B.Fab")
+      (effects (font (size 1 1) (thickness 0.15)) (justify mirror))
+    )
+    (fp_text user "${REFERENCE}" (at 0 2.5) (layer "B.Fab")
+      (effects (font (size 1 1) (thickness 0.15)) (justify mirror))
+    )
+    (fp_circle (center 0 0) (end 1.4 0) (layer "B.SilkS") (width 0.15) (fill none))
+    (fp_circle (center 0 0) (end 1.65 0) (layer "B.CrtYd") (width 0.05) (fill none))
+    (fp_line (start -0.75 -0.25) (end -0.75 0.25) (layer "B.Fab") (width 0.15))
+    (fp_line (start 0.75 -0.25) (end -0.75 -0.25) (layer "B.Fab") (width 0.15))
+    (fp_line (start -0.75 0.25) (end 0.75 0.25) (layer "B.Fab") (width 0.15))
+    (fp_line (start 0.75 0.25) (end 0.75 -0.25) (layer "B.Fab") (width 0.15))
+    (fp_circle (center 0 0) (end 1.25 0) (layer "B.Fab") (width 0.15) (fill none))
+    (pad "1" thru_hole circle (at 0 0 180) (size 2 2) (drill 1) (layers *.Cu *.Mask)
+      (net 105 "/3V1") (pinfunction "1") (pintype "passive"))
+    (model "${KICAD6_3DMODEL_DIR}/TestPoint.3dshapes/TestPoint_Keystone_5000-5004_Miniature.wrl"
+      (offset (xyz 0 0 0))
+      (scale (xyz 1 1 1))
+      (rotate (xyz 0 0 0))
+    )
+  )
   (footprint "Connector_PinHeader_2.54mm:PinHeader_1x04_P2.54mm_Vertical" (layer "B.Cu")
     (at 155.6779 139.9157)
@@
     (effects (font (size 1 1) (thickness 0.15)) (justify mirror))
   )
+  (gr_text "3.3V" (at 205.8429 82.7657) (layer "B.SilkS")
+    (effects (font (size 0.5 0.5) (thickness 0.125)) (justify mirror))
+  )
   (gr_text "Sky Camera" (at 213.3359 139.9157) (layer "B.SilkS")
     (effects (font (size 1 1) (thickness 0.15)) (justify mirror))
@@
   (segment (start 165.0539 141.4397) (end 165.5839 140.9097) (width 0.25) (layer "B.Cu") (net 105))
   (segment (start 165.5839 135.3437) (end 165.0499 134.8097) (width 0.25) (layer "B.Cu") (net 105))
+  (segment (start 181.6621 87.2869) (end 189.2059 94.8307) (width 1) (layer "B.Cu") (net 105))
+  (segment (start 202.5409 92.2907) (end 202.5409 89.1157) (width 1) (layer "B.Cu") (net 105))
   (segment (start 160.4919 140.4497) (end 160.5299 140.4497) (width 0.25) (layer "B.Cu") (net 105))
   (segment (start 160.5039 143.3447) (end 160.4919 143.3327) (width 0.25) (layer "B.Cu") (net 105))
   (segment (start 165.0499 134.8097) (end 163.8099 134.8097) (width 0.25) (layer "B.Cu") (net 105))
+  (segment (start 205.0809 86.5757) (end 205.0809 84.7977) (width 1) (layer "B.Cu") (net 105))
   (segment (start 160.4919 143.3327) (end 160.4919 140.4497) (width 0.25) (layer "B.Cu") (net 105))
+  (segment (start 155.5763 87.2869) (end 181.6621 87.2869) (width 1) (layer "B.Cu") (net 105))
+  (segment (start 152.8859 89.9773) (end 155.5763 87.2869) (width 1) (layer "B.Cu") (net 105))
   (segment (start 160.5299 140.4497) (end 161.5199 141.4397) (width 0.25) (layer "B.Cu") (net 105))
+  (segment (start 202.5409 89.1157) (end 205.0809 86.5757) (width 1) (layer "B.Cu") (net 105))
   (segment (start 161.5199 141.4397) (end 165.0539 141.4397) (width 0.25) (layer "B.Cu") (net 105))
   (segment (start 165.5839 140.9097) (end 165.5839 135.3437) (width 0.25) (layer "B.Cu") (net 105))
+  (segment (start 152.8859 98.2241) (end 152.8859 89.9773) (width 1) (layer "B.Cu") (net 105))
+  (segment (start 200.0009 94.8307) (end 202.5409 92.2907) (width 1) (layer "B.Cu") (net 105))
+  (segment (start 189.2059 94.8307) (end 200.0009 94.8307) (width 1) (layer "B.Cu") (net 105))
   (zone (net 0) (net_name "") (layers F&B.Cu) (hatch edge 0.508)
     (connect_pads (clearance 0))

Commit message: SpectDrone Development
Connections:
- JAPC1 pad 1: /APCTX -> /APCRX
- JAPC1 pad 2: /APCRX -> /APCTX
- JAUX1 pad 10: /CAM2TX -> /CAM2RX
- JAUX1 pad 11: /CAM2RX -> /CAM2TX
- JAUX1 pad 8: /CAM1TX -> /CAM1RX
- JAUX1 pad 9: /CAM1RX -> /CAM1TX
Routing:
- net /CAM2RX: track 73.9 -> 70.9 mm
- net /CAM1TX: track 67.9 -> 69.3 mm
- net /APCTX: track 15.8 -> 16.9 mm
- net /CAM2TX: track 70.0 -> 69.1 mm
- net /APCRX: track 19.4 -> 20.2 mm
Other:
- board text removed: "APC_RX"
- board text removed: "APC_TX"
