File: SpectDrone/SpectDrone.kicad_sch (KiCad schematic)
At the start: 71 parts, among them J1 Camera, J2 GPS, J4 BME280, J5-1 BNO055-1, J5-2 BNO055-2, Q1 FDN340P, Q2 FDN340P, SW0 SW_Push, SW1 SW_Push, SW10 SW_Push, SW2 SW_Push, SW3 SW_Push, SW4 SW_Push, SW5 SW_Push, SW6 SW_Push, SW7 SW_Push, SW8 SW_Push, SW9 SW_Push, U1 C12666MA, U2 C12666MA, U3 LM7805_TO220, U4 MCP112-300E/TO, U5 MCP112-300E/TO, U6 LM7805_TO220, U7 Teensy3.2

Commit message: SpectDrone Development
Parts:
- added JAPC-3: APC220, Connector_PinSocket_2.54mm:PinSocket_1x07_P2.54mm_Vertical, symbol Connector:Conn_01x07_Female
Connections:
- net 5V4: now also JAPC-3.6 (Pin_6)
- net APC2AUX: now also JAPC-3.2 (Pin_2)
- net APC2EN: now also JAPC-3.5 (Pin_5)
- net APC2RX: now also JAPC-3.4 (Pin_4)
- net APC2SET: now also JAPC-3.1 (Pin_1)
- net APC2TX: now also JAPC-3.3 (Pin_3)
- net GND2: now also JAPC-3.7 (Pin_7)
- no-connect marks 51 -> 54
Changed lines of the file:
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@@
   (no_connect (at 267.97 73.66))
   (no_connect (at 232.41 100.33))
+  (no_connect (at 173.99 95.25))
   (no_connect (at 267.97 88.9))
   (no_connect (at 267.97 86.36))
@@
   (no_connect (at 101.6 179.07))
   (no_connect (at 19.05 115.57))
+  (no_connect (at 173.99 97.79))
   (no_connect (at 19.05 80.01))
   (no_connect (at 214.63 34.29))
@@
   (no_connect (at 50.8 158.75))
   (no_connect (at 50.8 161.29))
+  (no_connect (at 173.99 105.41))
   (no_connect (at 19.05 29.21))
   (no_connect (at 19.05 34.29))
@@
     (stroke (width 0) (type default) (color 0 0 0 0))
   )
+  (wire (pts (xy 173.99 107.95) (xy 172.72 107.95))
+    (stroke (width 0) (type default) (color 0 0 0 0))
+  )
   (wire (pts (xy 267.97 20.32) (xy 275.59 20.32))
     (stroke (width 0) (type default) (color 0 0 0 0))
@@
     (stroke (width 0) (type default) (color 0 0 0 0))
   )
+  (wire (pts (xy 172.72 102.87) (xy 173.99 102.87))
+    (stroke (width 0) (type default) (color 0 0 0 0))
+  )
   (wire (pts (xy 231.14 43.18) (xy 232.41 43.18))
     (stroke (width 0) (type default) (color 0 0 0 0))
@@
     (stroke (width 0) (type default) (color 0 0 0 0))
   )
+  (wire (pts (xy 172.72 97.79) (xy 173.99 97.79))
+    (stroke (width 0) (type default) (color 0 0 0 0))
+  )
   (wire (pts (xy 57.15 68.58) (xy 60.96 68.58))
     (stroke (width 0) (type default) (color 0 0 0 0))
@@
     (stroke (width 0) (type default) (color 0 0 0 0))
   )
+  (wire (pts (xy 172.72 110.49) (xy 173.99 110.49))
+    (stroke (width 0) (type default) (color 0 0 0 0))
+  )
   (wire (pts (xy 133.35 87.63) (xy 125.73 87.63))
     (stroke (width 0) (type default) (color 0 0 0 0))
@@
     (stroke (width 0) (type default) (color 0 0 0 0))
   )
+  (wire (pts (xy 172.72 95.25) (xy 173.99 95.25))
+    (stroke (width 0) (type default) (color 0 0 0 0))
+  )
   (wire (pts (xy 69.85 95.25) (xy 73.66 95.25))
     (stroke (width 0) (type default) (color 0 0 0 0))
@@
     (stroke (width 0) (type default) (color 0 0 0 0))
   )
+  (wire (pts (xy 172.72 105.41) (xy 173.99 105.41))
+    (stroke (width 0) (type default) (color 0 0 0 0))
+  )
   (wire (pts (xy 86.36 81.28) (xy 86.36 87.63))
     (stroke (width 0) (type default) (color 0 0 0 0))
@@
     (stroke (width 0) (type default) (color 0 0 0 0))
   )
+  (wire (pts (xy 172.72 100.33) (xy 173.99 100.33))
+    (stroke (width 0) (type default) (color 0 0 0 0))
+  )
   (wire (pts (xy 60.96 81.28) (xy 63.5 81.28))
     (stroke (width 0) (type default) (color 0 0 0 0))
@@
     (effects (font (size 1.27 1.27)) (justify left bottom))
   )
+  (label "APC2AUX" (at 173.99 97.79 0)
+    (effects (font (size 1.27 1.27)) (justify left bottom))
+  )
   (label "CAMTX" (at 269.24 53.34 0)
     (effects (font (size 1.27 1.27)) (justify left bottom))
@@
     (effects (font (size 1.27 1.27)) (justify right bottom))
   )
+  (label "APC2EN" (at 173.99 105.41 0)
+    (effects (font (size 1.27 1.27)) (justify left bottom))
+  )
   (label "CLK2" (at 269.24 58.42 0)
     (effects (font (size 1.27 1.27)) (justify left bottom))
@@
     (effects (font (size 1.27 1.27)) (justify right bottom))
   )
+  (label "APC2TX" (at 173.99 100.33 0)
+    (effects (font (size 1.27 1.27)) (justify left bottom))
+  )
   (label "SW8" (at 101.6 184.15 0)
     (effects (font (size 1.27 1.27)) (justify left bottom))
@@
     (effects (font (size 1.27 1.27)) (justify left bottom))
   )
+  (label "GND2" (at 173.99 110.49 0)
+    (effects (font (size 1.27 1.27)) (justify left bottom))
+  )
   (label "GND1" (at 251.46 40.64 180)
     (effects (font (size 1.27 1.27)) (justify right bottom))
@@
     (effects (font (size 1.27 1.27)) (justify right bottom))
   )
+  (label "APC2SET" (at 173.99 95.25 0)
+    (effects (font (size 1.27 1.27)) (justify left bottom))
+  )
   (label "SW9" (at 101.6 181.61 0)
     (effects (font (size 1.27 1.27)) (justify left bottom))
@@
     (effects (font (size 1.27 1.27)) (justify right bottom))
   )
+  (label "5V4" (at 173.99 107.95 0)
+    (effects (font (size 1.27 1.27)) (justify left bottom))
+  )
   (label "ST" (at 269.24 55.88 0)
+    (effects (font (size 1.27 1.27)) (justify left bottom))
+  )
+  (label "APC2RX" (at 173.99 102.87 0)
     (effects (font (size 1.27 1.27)) (justify left bottom))
   )
@@
     (pin "1")
     (pin "2")
+  )
+  (symbol (lib_id "Connector:Conn_01x07_Female") (at 167.64 102.87 0) (mirror y) (unit 1)
+    (in_bom yes) (on_board yes)
+    (property "Reference" "JAPC-3" (id 0) (at 167.64 92.71 0))
+    (property "Value" "APC220" (id 1) (at 170.18 113.03 0))
+    (property "Footprint" "Connector_PinSocket_2.54mm:PinSocket_1x07_P2.54mm_Vertical" (id 2) (at 165.1 102.87 90)
+      (effects (font (size 1.27 1.27)) hide)
+    )
+    (property "Datasheet" "~" (id 3) (at 167.64 102.87 0)
+      (effects (font (size 1.27 1.27)) hide)
+    )
+    (pin "1")
+    (pin "2")
+    (pin "3")
+    (pin "4")
+    (pin "5")
+    (pin "6")
+    (pin "7")
   )
   (symbol (lib_id "Connector:Conn_01x07_Female") (at 226.06 105.41 0) (mirror y) (unit 1)
@@
       (reference "JAPC-2") (unit 1) (value "APC220") (footprint "Connector_PinSocket_2.54mm:PinSocket_1x07_P2.54mm_Vertical")
     )
+    (path "/6533b2ed-bfe0-455e-a8cc-e29a9b928990"
+      (reference "JAPC-3") (unit 1) (value "APC220") (footprint "Connector_PinSocket_2.54mm:PinSocket_1x07_P2.54mm_Vertical")
+    )
     (path "/82929dde-ddec-49ba-859e-c82cb47ebb15"

Commit message: SpectDrone Development
Parts:
- added JVIN1: Conn_01x01_Male, Connector_PinHeader_2.54mm:PinHeader_1x01_P2.54mm_Vertical, symbol Connector:Conn_01x01_Male
- added TP2, TP3: TestPoint, TestPoint:TestPoint_Keystone_5000-5004_Miniature, symbol Connector:TestPoint
Connections:
- net GND1: now also TP3.1
- net VIN1: now also JVIN1.1 (Pin_1), TP2.1
Changed lines of the file:
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@@
+    (effects (font (size 1.27 1.27)) (justify right bottom))
+  )
+  (label "GND1" (at 50.8 58.42 180)
     (effects (font (size 1.27 1.27)) (justify right bottom))
   )
@@
     (effects (font (size 1.27 1.27)) (justify left bottom))
   )
+  (label "VIN1" (at 45.72 31.75 180)
+    (effects (font (size 1.27 1.27)) (justify right bottom))
+  )
   (label "GND1" (at 251.46 68.58 180)
     (effects (font (size 1.27 1.27)) (justify right bottom))
@@
   (label "D12" (at 267.97 60.96 180)
     (effects (font (size 1.27 1.27)) (justify right bottom))
+  )
+  (symbol (lib_id "Connector:TestPoint") (at 45.72 31.75 270) (unit 1)
+    (in_bom yes) (on_board yes)
+    (property "Reference" "TP2" (id 0) (at 49.53 25.4 90)
+      (effects (font (size 1.27 1.27)) (justify left))
+    )
+    (property "Value" "TestPoint" (id 1) (at 49.53 27.94 90)
+      (effects (font (size 1.27 1.27)) (justify left))
+    )
+    (property "Footprint" "TestPoint:TestPoint_Keystone_5000-5004_Miniature" (id 2) (at 45.72 36.83 0)
+      (effects (font (size 1.27 1.27)) hide)
+    )
+    (property "Datasheet" "~" (id 3) (at 45.72 36.83 0)
+      (effects (font (size 1.27 1.27)) hide)
+    )
+    (pin "1")
   )
   (symbol (lib_id "Mechanical:MountingHole") (at 19.05 69.85 0) (unit 1)
@@
     (pin "2")
   )
+  (symbol (lib_id "Connector:Conn_01x01_Male") (at 45.72 36.83 270) (mirror x) (unit 1)
+    (in_bom yes) (on_board yes)
+    (property "Reference" "JVIN1" (id 0) (at 43.1799 38.1 0)
+      (effects (font (size 1.27 1.27)) (justify right))
+    )
+    (property "Value" "Conn_01x01_Male" (id 1) (at 45.7199 38.1 90)
+      (effects (font (size 1.27 1.27)) (justify right) hide)
+    )
+    (property "Footprint" "Connector_PinHeader_2.54mm:PinHeader_1x01_P2.54mm_Vertical" (id 2) (at 45.72 36.83 0)
+      (effects (font (size 1.27 1.27)) hide)
+    )
+    (property "Datasheet" "~" (id 3) (at 45.72 36.83 0)
+      (effects (font (size 1.27 1.27)) hide)
+    )
+    (pin "1")
+  )
   (symbol (lib_id "Device:Battery_Cell") (at 162.56 71.12 0) (unit 1)
     (in_bom yes) (on_board yes) (fields_autoplaced)
@@
     (pin "1")
     (pin "2")
+  )
+  (symbol (lib_id "Connector:TestPoint") (at 50.8 58.42 270) (unit 1)
+    (in_bom yes) (on_board yes)
+    (property "Reference" "TP3" (id 0) (at 54.61 52.07 90)
+      (effects (font (size 1.27 1.27)) (justify left))
+    )
+    (property "Value" "TestPoint" (id 1) (at 54.61 54.61 90)
+      (effects (font (size 1.27 1.27)) (justify left))
+    )
+    (property "Footprint" "TestPoint:TestPoint_Keystone_5000-5004_Miniature" (id 2) (at 50.8 63.5 0)
+      (effects (font (size 1.27 1.27)) hide)
+    )
+    (property "Datasheet" "~" (id 3) (at 50.8 63.5 0)
+      (effects (font (size 1.27 1.27)) hide)
+    )
+    (pin "1")
   )
   (symbol (lib_id "Mechanical:MountingHole") (at 19.05 115.57 0) (unit 1)
@@
       (reference "JIR1") (unit 1) (value "Conn_01x04_Male") (footprint "Connector_PinHeader_2.54mm:PinHeader_1x04_P2.54mm_Horizontal")
     )
+    (path "/24c3ed88-b44c-461f-a72a-c41465279cde"
+      (reference "JVIN1") (unit 1) (value "Conn_01x01_Male") (footprint "Connector_PinHeader_2.54mm:PinHeader_1x01_P2.54mm_Vertical")
+    )
     (path "/b2849f68-fe47-4de0-b285-7371cb755c79"
       (reference "Q1") (unit 1) (value "FDN340P") (footprint "Package_TO_SOT_SMD:SOT-23")
@@
       (reference "TP1") (unit 1) (value "TestPoint") (footprint "TestPoint:TestPoint_Keystone_5000-5004_Miniature")
     )
+    (path "/05fb8eee-cfcd-467d-a8f4-c70caca5ceaf"
+      (reference "TP2") (unit 1) (value "TestPoint") (footprint "TestPoint:TestPoint_Keystone_5000-5004_Miniature")
+    )
+    (path "/4e443f35-4e24-402e-8626-3841a14370d9"
+      (reference "TP3") (unit 1) (value "TestPoint") (footprint "TestPoint:TestPoint_Keystone_5000-5004_Miniature")
+    )
     (path "/2b83a6cd-a3db-44a5-8cff-1305c7a7d631"

Commit message: SpectDrone Development
Connections:
- net 5V3: now also C4.1, TP1.1, U3.3 (VO); no longer D1.1 (K), Q1.2 (S)
- net VBAT: now also Q1.3 (D); no longer C3.2, U3.1 (VI)
- removed net VOUT: C4.1, Q1.3 (D), TP1.1, U3.3 (VO)
- new net 7-12V: C3.2, D1.1 (K), Q1.2 (S), U3.1 (VI)
Changed lines of the file:
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@@
     (effects (font (size 1.27 1.27)) (justify right bottom))
   )
-  (label "5V3" (at 101.6 20.32 0)
+  (label "7-12V" (at 101.6 20.32 0)
     (effects (font (size 1.27 1.27)) (justify left bottom))
   )
@@
     (effects (font (size 1.27 1.27)) (justify right bottom))
   )
-  (label "VOUT" (at 133.35 31.75 0)
+  (label "5V3" (at 133.35 31.75 0)
     (effects (font (size 1.27 1.27)) (justify left bottom))
   )
@@
     (effects (font (size 1.27 1.27)) (justify right bottom))
   )
-  (label "VBAT" (at 118.11 31.75 180)
+  (label "7-12V" (at 118.11 31.75 180)
     (effects (font (size 1.27 1.27)) (justify right bottom))
   )
@@
     (effects (font (size 1.27 1.27)) (justify right bottom))
   )
-  (label "VOUT" (at 76.2 50.8 0)
-    (effects (font (size 1.27 1.27)) (justify left bottom))
-  )
+  (label "VBAT" (at 76.2 50.8 0)
+    (effects (font (size 1.27 1.27)) (justify left bottom))
+  )

Commit message: SpectDrone Development
Parts:
- added J3: Barrel_Jack, Connector_BarrelJack:BarrelJack_Horizontal, symbol Connector:Barrel_Jack_Switch
- U4, U5: footprint Package_TO_SOT_THT:TO-92_Inline -> Package_TO_SOT_SMD:SOT-89-3
Connections:
- net 5V4: now also C6.1, U6.3 (VO); no longer D2.1 (K), Q2.2 (S)
- net BKL: now also JD1.8 (Pin_8), R3.2
- net D/C: now also U7.7 (5_TX1_PWM); no longer U7.5 (3_TX_PWM)
- net GND2: now also J3.2, J3.3
- net LED: now also U7.6 (4_RX_PWM); no longer U7.21 (14_A0_SCK)
- net VBAT2: now also Q2.3 (D); no longer C5.2, U6.1 (VI)
- net VIN2: now also J3.1
- net 7-12V renamed 7-12V1
- removed net VOUT2: C6.1, Q2.3 (D), U6.3 (VO)
- new net 7-12V2: C5.2, D2.1 (K), Q2.2 (S), U6.1 (VI)
Other:
- moved on the sheet: C3, C4, C5, C6, R3, TP1, U3, U6

Commit message: SpectDrone Development
Parts:
- removed JAPC-3: APC220, Connector_PinSocket_2.54mm:PinSocket_1x07_P2.54mm_Vertical, symbol Connector:Conn_01x07_Female
- JIR1: value Conn_01x04_Male -> Infrared
Connections:
- net VBAT renamed VBAT1
- no-connect marks 54 -> 51
Other:
- moved on the sheet: BT1, C1, C2, D3, J1, J2, J3, J4, J5-1, J5-2, JA1, JAPC-1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

Commit message: SpectDrone Development
Parts:
- added H21, H22, H23, H24: MountingHole, MountingHole:MountingHole_2.5mm, symbol Mechanical:MountingHole
- added JCAM1, JD1: Conn_01x04_Male, Connector_PinHeader_2.54mm:PinHeader_1x04_P2.54mm_Vertical, symbol Connector:Conn_01x04_Male
- added JCAM3: Camera, Connector_JST:JST_XH_B4B-XH-A_1x04_P2.50mm_Vertical, symbol Connector:Conn_01x04_Male
- renumbered J1 to JCAM2, JD1 to JDIS1, JD2 to JDIS2
Connections:
- net 5V3: now also JCAM3.1 (Pin_1)
- net A1: now also JA1.2 (Pin_2); no longer JA1.1 (Pin_1)
- net A2: now also JA1.3 (Pin_3); no longer JA1.2 (Pin_2)
- net CLK1: now also JD1.1 (Pin_1); no longer JAUX1.11 (Pin_11)
- net CLK2: now also JD1.4 (Pin_4); no longer JAUX1.10 (Pin_10)
- net GAIN: now also JD1.3 (Pin_3); no longer JA1.3 (Pin_3)
- net GND1: now also JCAM3.2 (Pin_2)
- net ST: now also JD1.2 (Pin_2); no longer JAUX1.9 (Pin_9)
- net CAMRX renamed CAM1RX
- net CAM1RX: now also JCAM1.2 (Pin_2); no longer JAUX1.4 (Pin_4)
- net CAMTX renamed CAM1TX
- net CAM1TX: now also JCAM1.1 (Pin_1); no longer JAUX1.8 (Pin_8)
- new net CAM2RX: JCAM1.4 (Pin_4), JCAM3.3 (Pin_3)
- new net CAM2TX: JCAM1.3 (Pin_3), JCAM3.4 (Pin_4)
- new net D12: JAUX1.11 (Pin_11)
- new net OPT_EXT: JAUX1.10 (Pin_10)
- new net SS_AUX: JAUX1.4 (Pin_4)
- new net XCL: JAUX1.8 (Pin_8)
- new net XDA: JAUX1.9 (Pin_9)
- no-connect marks 51 -> 56

Commit message: SpectDrone Development
Parts:
- added D4, D5: S1336-18BK, Package_TO_SOT_THT:TO-18-4_Lens, symbol Sensor_Optical:S13360-3025CS
- added R4, R5, R6: R, Resistor_SMD:R_0603_1608Metric_Pad0.98x0.95mm_HandSolder, symbol Device:R
- added RV1: R_Potentiometer, Potentiometer_THT:Potentiometer_Bourns_3296W_Vertical, symbol Device:R_Potentiometer
- added TP4: TestPoint, TestPoint:TestPoint_Keystone_5000-5004_Miniature, symbol Connector:TestPoint
- added U8: ADR510, Package_TO_SOT_SMD:SOT-23, symbol Reference_Voltage:CJ432
- added U9: AD8620, Package_DIP:DIP-8_W7.62mm, symbol Amplifier_Operational:AD8620
Connections:
- net 5V3: now also R6.1
- net GND1: now also R4.2, R5.2, RV1.3, U8.3 (A), U9.4 (V-)
- net PD1: now reaches JA1.1 (Pin_1)
- net PD1: now also D4.1 (A), R4.1, U9.1, U9.2 (-)
- net PD2: now reaches JA1.4 (Pin_4)
- net PD2: now also D5.1 (A), R5.1, U9.6 (-), U9.7
- new net: RV1.2, U8.1 (REF)
- new net 1.0V: D4.2 (K), D5.2 (K), R6.2, RV1.1, TP4.1, U8.2 (K), U9.3 (+), U9.5 (+), U9.8 (V+)
- no-connect marks 56 -> 54
Other:
- moved on the sheet: J2, J4, J5-1, J5-2, JCAM2, JCAM3, JIR1, RSW1, SW0, SW1, SW10, SW2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

Commit message: SpectDrone Development
Parts:
- added R10, R9: R, Resistor_SMD:R_0603_1608Metric_Pad0.98x0.95mm_HandSolder, symbol Device:R
- U9: value AD8620 -> MIC863; footprint Package_DIP:DIP-8_W7.62mm -> Package_TO_SOT_SMD:SOT-23-8
Connections:
- net 1.0V: now also D4.3 (K), D5.3 (K); no longer D4.2 (K), D5.2 (K)
- net PD1: no longer names the net of D4.1 (A), R4.1, U9.2 (-)
- net PD1: now also R9.2; no longer JA1.1 (Pin_1), U9.1
- net PD2: no longer names the net of D5.1 (A), R5.1, U9.6 (-)
- net PD2: now also R10.1; no longer JA1.4 (Pin_4), U9.7
- new net S1: JA1.4 (Pin_4), R9.1, U9.1
- new net S2: JA1.1 (Pin_1), R10.2, U9.7
Other:
- moved on the sheet: R4, R5, U9A, U9B, U9C
