File: SpectDrone/SpectDrone.kicad_sch (KiCad schematic)
At the start: 93 parts, among them J2 GPS, J3 Barrel_Jack, J4 BME280, J5-1 BNO055-1, J5-2 BNO055-2, Q1 FDN340P, Q2 FDN340P, SW0 SW_Push, SW1 SW_Push, SW10 SW_Push, SW2 SW_Push, SW3 SW_Push, SW4 SW_Push, SW5 SW_Push, SW6 SW_Push, SW7 SW_Push, SW8 SW_Push, SW9 SW_Push, U1 C12666MA, U2 C12666MA, U3 LM7805_TO220, U4 MCP112-300E/TO, U5 MCP112-300E/TO, U6 LM7805_TO220, U7 Teensy3.2, U8 ADR510, U9 MIC863

Commit message: SpectDrone development
Parts:
- renumbered D5 to PD1, D4 to PD2
Connections:
- net S1: now also JA1.1 (Pin_1), R10.2, U9.7; no longer JA1.4 (Pin_4), R9.1, U9.1
- net S2: now also JA1.4 (Pin_4), R9.1, U9.1; no longer JA1.1 (Pin_1), R10.2, U9.7
Changed lines of the file:
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@@
     (effects (font (size 1.27 1.27)) (justify right bottom))
   )
-  (label "S2" (at 185.42 152.4 0)
+  (label "S1" (at 185.42 152.4 0)
     (effects (font (size 1.27 1.27)) (justify left bottom))
   )
@@
     (effects (font (size 1.27 1.27)) (justify right bottom))
   )
-  (label "S2" (at 222.25 16.51 180)
+  (label "S2" (at 222.25 24.13 180)
     (effects (font (size 1.27 1.27)) (justify right bottom))
   )
@@
     (effects (font (size 1.27 1.27)) (justify right bottom))
   )
-  (label "S1" (at 185.42 119.38 0)
+  (label "S2" (at 185.42 119.38 0)
     (effects (font (size 1.27 1.27)) (justify left bottom))
   )
@@
     (effects (font (size 1.27 1.27)) (justify right bottom))
   )
-  (label "S1" (at 222.25 24.13 180)
+  (label "S1" (at 222.25 16.51 180)
     (effects (font (size 1.27 1.27)) (justify right bottom))
   )
@@
   (symbol (lib_id "Sensor_Optical:S13360-3025CS") (at 146.05 116.84 270) (unit 1)
     (in_bom yes) (on_board yes)
-    (property "Reference" "D4" (id 0) (at 149.86 113.03 90))
+    (property "Reference" "PD2" (id 0) (at 149.86 113.03 90))
     (property "Value" "S1336-18BK" (id 1) (at 147.32 107.95 90))
     (property "Footprint" "Package_TO_SOT_THT:TO-18-4_Lens" (id 2) (at 144.78 121.285 0)
@@
   (symbol (lib_name "S13360-3025CS_1") (lib_id "Sensor_Optical:S13360-3025CS") (at 146.05 149.86 270) (unit 1)
     (in_bom yes) (on_board yes)
-    (property "Reference" "D5" (id 0) (at 149.86 146.05 90))
+    (property "Reference" "PD1" (id 0) (at 149.86 146.05 90))
     (property "Value" "S1336-18BK" (id 1) (at 147.32 140.97 90))
     (property "Footprint" "Package_TO_SOT_THT:TO-18-4_Lens" (id 2) (at 144.78 154.305 0)
@@
       (reference "D3") (unit 1) (value "Ge") (footprint "Diode_THT:D_T-1_P5.08mm_Horizontal")
     )
-    (path "/9c3344ad-2b12-4670-9290-da422ffdbe3c"
-      (reference "D4") (unit 1) (value "S1336-18BK") (footprint "Package_TO_SOT_THT:TO-18-4_Lens")
-    )
-    (path "/c1de7c16-0fb5-4855-9c92-9e6b4b6586a6"
-      (reference "D5") (unit 1) (value "S1336-18BK") (footprint "Package_TO_SOT_THT:TO-18-4_Lens")
-    )
     (path "/ca03f054-8c98-4670-99f2-ac2394c6b901"
       (reference "H1") (unit 1) (value "MountingHole") (footprint "MountingHole:MountingHole_2.2mm_M2_ISO14580_Pad_TopBottom")
@@
       (reference "JVIN1") (unit 1) (value "Conn_01x01_Male") (footprint "Connector_PinHeader_2.54mm:PinHeader_1x01_P2.54mm_Vertical")
     )
+    (path "/c1de7c16-0fb5-4855-9c92-9e6b4b6586a6"
+      (reference "PD1") (unit 1) (value "S1336-18BK") (footprint "Package_TO_SOT_THT:TO-18-4_Lens")
+    )
+    (path "/9c3344ad-2b12-4670-9290-da422ffdbe3c"
+      (reference "PD2") (unit 1) (value "S1336-18BK") (footprint "Package_TO_SOT_THT:TO-18-4_Lens")
+    )
     (path "/b2849f68-fe47-4de0-b285-7371cb755c79"

Commit message: SpectDrone Development
Parts:
- removed JCAM1: Conn_01x04_Male, Connector_PinHeader_2.54mm:PinHeader_1x04_P2.54mm_Vertical, symbol Connector:Conn_01x04_Male
- added J1: Conn_01x01_Male, Connector_PinHeader_2.54mm:PinHeader_1x01_P2.54mm_Vertical, symbol Connector:Conn_01x01_Male
- added JI2C1, JI2C3-1: Conn_01x04_Male, Connector_PinHeader_2.54mm:PinHeader_1x04_P2.54mm_Vertical, symbol Connector:Conn_01x04_Male
- added U10: PCA9306DC, Package_SO:VSSOP-8_2.3x2mm_P0.5mm, symbol Interface:PCA9306DC
- JAUX1: footprint Connector_PinHeader_2.54mm:PinHeader_1x11_P2.54mm_Vertical -> Connector_PinHeader_2.54mm:PinHeader_1x12_P2.54mm_Vertical; symbol Connector:Conn_01x11_Male -> Connector:Conn_01x12_Male
- renumbered JCAM3 to JCAM2, JCAM2 to JCAM3
Connections:
- net OPT_EXT is gone; now on net CAM2TX: JAUX1.10 (Pin_10)
- net XCL is gone; now on net CAM1TX: JAUX1.8 (Pin_8)
- net XDA is gone; now on net CAM1RX: JAUX1.9 (Pin_9)
- net 5V3: now also JI2C1.3 (Pin_3), U10.7 (VREF2)
- net BMESCK: now also JI2C1.1 (Pin_1), U10.6 (SCL2)
- net BMESDI: now also JI2C1.2 (Pin_2), U10.5 (SDA2)
- net CAM1RX: now also JCAM3.4 (Pin_4); no longer JCAM3.3 (Pin_3)
- net CAM1TX: now also JCAM3.3 (Pin_3); no longer JCAM3.4 (Pin_4)
- net CAM2RX: now also JAUX1.11 (Pin_11), JCAM2.4 (Pin_4); no longer JCAM2.3 (Pin_3)
- net CAM2TX: now also JCAM2.3 (Pin_3); no longer JCAM2.4 (Pin_4)
- net D12: now also JAUX1.12 (Pin_12); no longer JAUX1.11 (Pin_11)
- net GND1: now also JI2C1.4 (Pin_4), JI2C3-1.4 (Pin_4), U10.4 (GND)
- net 3V renamed 3V2
- new net 3V1: J1.1 (Pin_1), JI2C3-1.3 (Pin_3), U10.1 (VREF1)
- new net SCL3: JI2C3-1.1 (Pin_1), U10.2 (SCL1)
- new net SDA3: JI2C3-1.2 (Pin_2), U10.3 (SDA1)
Other:
- moved on the sheet: PD1, PD2, R10, R4, R5, R6, R9, RV1, TP4, U8, U9A, U9B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

Commit message: SpectDrone Development
Parts:
- added TP5: TestPoint, TestPoint:TestPoint_Keystone_5000-5004_Miniature, symbol Connector:TestPoint
Connections:
- net 3V1: now also TP5.1
Changed lines of the file:
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@@
+    (stroke (width 0) (type default) (color 0 0 0 0))
+  )
+  (wire (pts (xy 139.7 162.56) (xy 139.7 163.83))
     (stroke (width 0) (type default) (color 0 0 0 0))
   )
@@
     (stroke (width 0) (type default) (color 0 0 0 0))
   )
-  (wire (pts (xy 149.86 163.83) (xy 156.21 163.83))
+  (wire (pts (xy 139.7 163.83) (xy 156.21 163.83))
     (stroke (width 0) (type default) (color 0 0 0 0))
   )
@@
     (pin "1")
     (pin "2")
+  )
+  (symbol (lib_id "Connector:TestPoint") (at 139.7 162.56 270) (unit 1)
+    (in_bom yes) (on_board yes)
+    (property "Reference" "TP5" (id 0) (at 142.24 157.48 90)
+      (effects (font (size 1.27 1.27)) (justify left))
+    )
+    (property "Value" "TestPoint" (id 1) (at 142.24 160.02 90)
+      (effects (font (size 1.27 1.27)) (justify left))
+    )
+    (property "Footprint" "TestPoint:TestPoint_Keystone_5000-5004_Miniature" (id 2) (at 139.7 167.64 0)
+      (effects (font (size 1.27 1.27)) hide)
+    )
+    (property "Datasheet" "~" (id 3) (at 139.7 167.64 0)
+      (effects (font (size 1.27 1.27)) hide)
+    )
+    (pin "1")
   )
   (symbol (lib_id "Connector:Conn_01x04_Male") (at 232.41 34.29 0) (mirror y) (unit 1)
@@
       (reference "TP4") (unit 1) (value "TestPoint") (footprint "TestPoint:TestPoint_Keystone_5000-5004_Miniature")
     )
+    (path "/6c900bf0-cac7-4987-a689-121ebc5161e1"
+      (reference "TP5") (unit 1) (value "TestPoint") (footprint "TestPoint:TestPoint_Keystone_5000-5004_Miniature")
+    )
     (path "/2b83a6cd-a3db-44a5-8cff-1305c7a7d631"

Commit message: SpectDrone Development
Connections:
- net APCRX: now also JAPC1.1 (Pin_1); no longer JAPC1.2 (Pin_2)
- net APCTX: now also JAPC1.2 (Pin_2); no longer JAPC1.1 (Pin_1)
- net CAM1RX: now also JAUX1.8 (Pin_8); no longer JAUX1.9 (Pin_9)
- net CAM1TX: now also JAUX1.9 (Pin_9); no longer JAUX1.8 (Pin_8)
- net CAM2RX: now also JAUX1.10 (Pin_10); no longer JAUX1.11 (Pin_11)
- net CAM2TX: now also JAUX1.11 (Pin_11); no longer JAUX1.10 (Pin_10)
Changed lines of the file:
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@@
     (effects (font (size 1.27 1.27)) (justify right bottom))
   )
-  (label "CAM2TX" (at 267.97 39.37 180)
+  (label "CAM2TX" (at 267.97 41.91 180)
     (effects (font (size 1.27 1.27)) (justify right bottom))
   )
@@
     (effects (font (size 1.27 1.27)) (justify right bottom))
   )
-  (label "APCRX" (at 241.3 19.05 0)
+  (label "APCRX" (at 241.3 16.51 0)
     (effects (font (size 1.27 1.27)) (justify left bottom))
   )
@@
     (effects (font (size 1.27 1.27)) (justify right bottom))
   )
-  (label "APCTX" (at 241.3 16.51 0)
+  (label "APCTX" (at 241.3 19.05 0)
     (effects (font (size 1.27 1.27)) (justify left bottom))
   )
@@
     (effects (font (size 1.27 1.27)) (justify right bottom))
   )
-  (label "CAM1RX" (at 267.97 36.83 180)
-    (effects (font (size 1.27 1.27)) (justify right bottom))
-  )
-  (label "CAM2RX" (at 267.97 41.91 180)
+  (label "CAM1RX" (at 267.97 34.29 180)
+    (effects (font (size 1.27 1.27)) (justify right bottom))
+  )
+  (label "CAM2RX" (at 267.97 39.37 180)
     (effects (font (size 1.27 1.27)) (justify right bottom))
   )
@@
     (effects (font (size 1.27 1.27)) (justify right bottom))
   )
-  (label "CAM1TX" (at 267.97 34.29 180)
-    (effects (font (size 1.27 1.27)) (justify right bottom))
-  )
+  (label "CAM1TX" (at 267.97 36.83 180)
+    (effects (font (size 1.27 1.27)) (justify right bottom))
+  )

Commit message: SpectDrone development
Parts:
- added JP1: SolderJumper_3_Bridged12, Jumper:SolderJumper-3_P1.3mm_Bridged12_RoundedPad1.0x1.5mm, symbol Jumper:SolderJumper_3_Bridged12
- added JUT1: Conn_01x04_Male, Connector_PinHeader_2.54mm:PinHeader_1x04_P2.54mm_Vertical, symbol Connector:Conn_01x04_Male
- added UT1, UT2: TSIC506F-TO92, Package_TO_SOT_THT:TO-92_Inline, symbol Sensor_Temperature:TSIC506F-TO92
- renumbered J1 to J3V3
Connections:
- net 1.0V: no longer U9.8 (V+)
- net 3V1: now also JP1.3 (B)
- net 5V3: now also JP1.1 (A), UT1.1 (GND), UT2.1 (GND)
- net GND1: now also UT1.3 (V+), UT2.3 (V+)
- net SIG2: now reaches PD2.1 (A), R4.1, R9.2, U9.2 (-)
- net SIG1: now reaches PD1.1 (A), R10.1, R5.1, U9.6 (-)
- new net AREF: JP1.2 (C), U9.8 (V+)
- new net UT1: JUT1.1 (Pin_1), UT1.2 (Signal)
- new net UT2: JUT1.2 (Pin_2), UT2.2 (Signal)
- no-connect marks 54 -> 56
Other:
- moved on the sheet: JI2C3-1, TP5, U9C

Commit message: SpectDrone Development
Parts:
- added JGPS2: GPS, Connector_PinSocket_2.54mm:PinSocket_1x05_P2.54mm_Vertical, symbol Connector:Conn_01x05_Female
- renumbered JI2C3-1 to JI2C3v-1
Connections:
- net 5V3: now also J2.2 (Pin_2), JGPS2.1 (Pin_1)
- net GND1: now also J2.1 (Pin_1), J2.5 (Pin_5), JGPS2.2 (Pin_2)
- net GPSRX: now also J2.3 (Pin_3), JGPS2.3 (Pin_3); no longer J2.4 (Pin_4)
- net GPSTX: now also J2.4 (Pin_4), JGPS2.4 (Pin_4); no longer J2.5 (Pin_5)
- net PPS: now also J2.6 (Pin_6), JGPS2.5 (Pin_5); no longer J2.1 (Pin_1)
- removed net 5V2: J2.2 (Pin_2), J2.3 (Pin_3), JGPS1.1 (Pin_1)
- net GND renamed GPS_GND
- net GPS_GND: no longer J2.6 (Pin_6)
- new net GPS_5V: JGPS1.1 (Pin_1)
- no-connect marks 56 -> 57
Other:
- moved on the sheet: J3V3
Changed lines of the file:
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@@
   (no_connect (at 19.05 80.01))
   (no_connect (at 29.21 115.57))
+  (no_connect (at 200.66 146.05))
   (no_connect (at 207.01 34.29))
   (no_connect (at 170.18 34.29))
@@
     (stroke (width 0) (type default) (color 0 0 0 0))
   )
+  (wire (pts (xy 241.3 58.42) (xy 247.65 58.42))
+    (stroke (width 0) (type default) (color 0 0 0 0))
+  )
   (wire (pts (xy 237.49 67.31) (xy 231.14 67.31))
     (stroke (width 0) (type default) (color 0 0 0 0))
@@
     (stroke (width 0) (type default) (color 0 0 0 0))
   )
+  (wire (pts (xy 241.3 55.88) (xy 247.65 55.88))
+    (stroke (width 0) (type default) (color 0 0 0 0))
+  )
   (wire (pts (xy 219.71 69.85) (xy 213.36 69.85))
     (stroke (width 0) (type default) (color 0 0 0 0))
@@
     (stroke (width 0) (type default) (color 0 0 0 0))
   )
+  (wire (pts (xy 241.3 48.26) (xy 247.65 48.26))
+    (stroke (width 0) (type default) (color 0 0 0 0))
+  )
   (wire (pts (xy 265.43 55.88) (xy 271.78 55.88))
     (stroke (width 0) (type default) (color 0 0 0 0))
@@
     (stroke (width 0) (type default) (color 0 0 0 0))
   )
+  (wire (pts (xy 241.3 53.34) (xy 247.65 53.34))
+    (stroke (width 0) (type default) (color 0 0 0 0))
+  )
   (wire (pts (xy 60.96 33.02) (xy 63.5 33.02))
     (stroke (width 0) (type default) (color 0 0 0 0))
@@
     (stroke (width 0) (type default) (color 0 0 0 0))
   )
+  (wire (pts (xy 241.3 50.8) (xy 247.65 50.8))
+    (stroke (width 0) (type default) (color 0 0 0 0))
+  )
   (wire (pts (xy 60.96 81.28) (xy 63.5 81.28))
     (stroke (width 0) (type default) (color 0 0 0 0))
@@
     (effects (font (size 1.27 1.27)) (justify right bottom))
   )
-  (label "3V1" (at 240.03 52.07 0)
+  (label "3V1" (at 224.79 52.07 0)
     (effects (font (size 1.27 1.27)) (justify left bottom))
   )
@@
     (effects (font (size 1.27 1.27)) (justify left bottom))
   )
-  (label "5V2" (at 241.3 31.75 0)
+  (label "GPS_5V" (at 241.3 31.75 0)
     (effects (font (size 1.27 1.27)) (justify left bottom))
   )
-  (label "PPS" (at 219.71 62.23 180)
+  (label "PPS" (at 219.71 74.93 180)
     (effects (font (size 1.27 1.27)) (justify right bottom))
   )
@@
     (effects (font (size 1.27 1.27)) (justify left bottom))
   )
+  (label "GND1" (at 241.3 50.8 0)
+    (effects (font (size 1.27 1.27)) (justify left bottom))
+  )
+  (label "GPSRX" (at 241.3 53.34 0)
+    (effects (font (size 1.27 1.27)) (justify left bottom))
+  )
   (label "GND2" (at 279.4 137.16 180)
     (effects (font (size 1.27 1.27)) (justify right bottom))
@@
     (effects (font (size 1.27 1.27)) (justify right bottom))
   )
-  (label "GND" (at 241.3 34.29 0)
+  (label "GPS_GND" (at 241.3 34.29 0)
     (effects (font (size 1.27 1.27)) (justify left bottom))
   )
@@
     (effects (font (size 1.27 1.27)) (justify right bottom))
   )
+  (label "PPS" (at 241.3 58.42 0)
+    (effects (font (size 1.27 1.27)) (justify left bottom))
+  )
   (label "APCAUX" (at 279.4 85.09 180)
     (effects (font (size 1.27 1.27)) (justify right bottom))
@@
     (effects (font (size 1.27 1.27)) (justify left bottom))
   )
-  (label "GPSRX" (at 219.71 69.85 180)
+  (label "GPSRX" (at 219.71 67.31 180)
     (effects (font (size 1.27 1.27)) (justify right bottom))
   )
@@
     (effects (font (size 1.27 1.27)) (justify right bottom))
   )
-  (label "5V2" (at 219.71 67.31 180)
-    (effects (font (size 1.27 1.27)) (justify right bottom))
-  )
   (label "SW4" (at 77.47 172.72 0)
     (effects (font (size 1.27 1.27)) (justify left bottom))
@@
     (effects (font (size 1.27 1.27)) (justify right bottom))
   )
-  (label "GPSTX" (at 219.71 72.39 180)
+  (label "GPSTX" (at 219.71 69.85 180)
     (effects (font (size 1.27 1.27)) (justify right bottom))
   )
@@
     (effects (font (size 1.27 1.27)) (justify right bottom))
   )
-  (label "GND" (at 219.71 74.93 180)
+  (label "GND1" (at 219.71 62.23 180)
     (effects (font (size 1.27 1.27)) (justify right bottom))
   )
@@
     (effects (font (size 1.27 1.27)) (justify right bottom))
   )
+  (label "GND1" (at 219.71 72.39 180)
+    (effects (font (size 1.27 1.27)) (justify right bottom))
+  )
   (label "SDA" (at 217.17 91.44 180)
     (effects (font (size 1.27 1.27)) (justify right bottom))
@@
     (effects (font (size 1.27 1.27)) (justify right bottom))
   )
+  (label "GPSTX" (at 241.3 55.88 0)
+    (effects (font (size 1.27 1.27)) (justify left bottom))
+  )
   (label "1.0V" (at 156.21 125.73 180)
     (effects (font (size 1.27 1.27)) (justify right bottom))
@@
     (effects (font (size 1.27 1.27)) (justify left bottom))
   )
+  (label "5V3" (at 241.3 48.26 0)
+    (effects (font (size 1.27 1.27)) (justify left bottom))
+  )
   (label "BKL" (at 270.51 163.83 0)
     (effects (font (size 1.27 1.27)) (justify left bottom))
@@
     (effects (font (size 1.27 1.27)) (justify right bottom))
   )
-  (label "5V2" (at 219.71 64.77 180)
+  (label "5V3" (at 219.71 64.77 180)
     (effects (font (size 1.27 1.27)) (justify right bottom))
   )
@@
     (effects (font (size 1.27 1.27)) (justify right bottom))
   )
+  (symbol (lib_id "Connector:Conn_01x05_Female") (at 252.73 53.34 0) (unit 1)
+    (in_bom yes) (on_board yes)
+    (property "Reference" "JGPS2" (id 0) (at 254 55.88 90)
+      (effects (font (size 1.27 1.27)) (justify left))
+    )
+    (property "Value" "GPS" (id 1) (at 251.46 57.15 90)
+      (effects (font (size 1.27 1.27)) (justify left) hide)
+    )
+    (property "Footprint" "Connector_PinSocket_2.54mm:PinSocket_1x05_P2.54mm_Vertical" (id 2) (at 252.73 53.34 0)
+      (effects (font (size 1.27 1.27)) hide)
+    )
+    (property "Datasheet" "~" (id 3) (at 252.73 53.34 0)
+      (effects (font (size 1.27 1.27)) hide)
+    )
+    (pin "1")
+    (pin "2")
+    (pin "3")
+    (pin "4")
+    (pin "5")
+  )
   (symbol (lib_id "Device:R") (at 143.51 68.58 90) (unit 1)
     (in_bom yes) (on_board yes) (fields_autoplaced)
@@
   (symbol (lib_id "Connector:Conn_01x04_Male") (at 171.45 190.5 0) (mirror y) (unit 1)
     (in_bom yes) (on_board yes)
-    (property "Reference" "JI2C3-1" (id 0) (at 172.72 191.77 90))
+    (property "Reference" "JI2C3v-1" (id 0) (at 172.72 191.77 90))
     (property "Value" "Conn_01x04_Male" (id 1) (at 161.29 191.77 0)
       (effects (font (size 1.27 1.27)) hide)
@@
       (effects (font (size 1.27 1.27)) hide)
     )
-    (pin "3")
-    (pin "2")
     (pin "1")
+    (pin "2")
+    (pin "3")
   )
   (symbol (lib_id "Mechanical:MountingHole") (at 19.05 110.49 0) (unit 1)
@@
     )
   )
-  (symbol (lib_id "Connector:Conn_01x01_Male") (at 234.95 52.07 0) (unit 1)
+  (symbol (lib_id "Connector:Conn_01x01_Male") (at 219.71 52.07 0) (unit 1)
     (in_bom yes) (on_board yes) (fields_autoplaced)
-    (property "Reference" "J3V3" (id 0) (at 235.585 46.99 0))
-    (property "Value" "Conn_01x01_Male" (id 1) (at 235.585 49.53 0))
-    (property "Footprint" "Connector_PinHeader_2.54mm:PinHeader_1x01_P2.54mm_Vertical" (id 2) (at 234.95 52.07 0)
+    (property "Reference" "J3V3" (id 0) (at 220.345 46.99 0))
+    (property "Value" "Conn_01x01_Male" (id 1) (at 220.345 49.53 0))
+    (property "Footprint" "Connector_PinHeader_2.54mm:PinHeader_1x01_P2.54mm_Vertical" (id 2) (at 219.71 52.07 0)
       (effects (font (size 1.27 1.27)) hide)
     )
-    (property "Datasheet" "~" (id 3) (at 234.95 52.07 0)
+    (property "Datasheet" "~" (id 3) (at 219.71 52.07 0)
       (effects (font (size 1.27 1.27)) hide)
     )
@@
       (reference "JGPS1") (unit 1) (value "GPS") (footprint "Connector_PinHeader_2.54mm:PinHeader_1x05_P2.54mm_Vertical")
     )
+    (path "/011a5828-4c3c-4dde-9bdb-284a3f3c4a43"
+      (reference "JGPS2") (unit 1) (value "GPS") (footprint "Connector_PinSocket_2.54mm:PinSocket_1x05_P2.54mm_Vertical")
+    )
     (path "/a6b26d49-3511-4379-b51c-29b09d1a74f5"
       (reference "JI2C1") (unit 1) (value "Conn_01x04_Male") (footprint "Connector_PinHeader_2.54mm:PinHeader_1x04_P2.54mm_Vertical")
     )
     (path "/3303bd17-726e-4fee-8519-8e88505aac59"
-      (reference "JI2C3-1") (unit 1) (value "Conn_01x04_Male") (footprint "Connector_PinHeader_2.54mm:PinHeader_1x04_P2.54mm_Vertical")
+      (reference "JI2C3v-1") (unit 1) (value "Conn_01x04_Male") (footprint "Connector_PinHeader_2.54mm:PinHeader_1x04_P2.54mm_Vertical")
     )
     (path "/72e4d4c2-74b3-4f9a-8d71-bbda38e5099c"

Commit message: SpectDrone Development
Parts:
- added R11, R8: 2K2, Resistor_SMD:R_0402_1005Metric, symbol Device:R
- added R7: 200K, Resistor_SMD:R_0402_1005Metric, symbol Device:R
- BT1: footprint Battery:BatteryHolder_Keystone_500 -> Battery:BatteryHolder_Keystone_103_1x20mm
- H1, H10, H11, H12, H13, H14, H15, H16, H17, H18, H19, H2, H20, H21, H22, H23, H24, H3, H4, H5, H6, H7, H8, H9: now left out of the parts list
- U4, U5: value MCP112-300E/TO -> MCP112-450E/TO
Connections:
- net 3V1: now also R11.1, R8.1
- net 5V3: now also R7.2; no longer U10.7 (VREF2)
- net SCL3: now also R8.2
- net SDA3: now also R11.2
- net at U10.8 (EN): now also U10.7 (VREF2), R7.1
- no-connect marks 57 -> 56
Other:
- moved on the sheet: H1, H10, H11, H12, H13, H14, H15, H16, H17, H18, H19, H2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

Commit message: SpectDrone Development
Parts:
- removed H21, H22, H23, H24: MountingHole, MountingHole:MountingHole_2.5mm, symbol Mechanical:MountingHole
- added C7, C8: 0.1uF, Capacitor_THT:C_Disc_D5.0mm_W2.5mm_P2.50mm, symbol Device:C_Small
Connections:
- net GND1: now also R1.1, C7.1; no longer R1.2
- net GND2: now also R2.1, C8.1; no longer R2.2
- net VIN1: now also R1.2, C7.2; no longer R1.1
- net VIN2: now also R2.2, C8.2; no longer R2.1
- no-connect marks 56 -> 52
Other:
- moved on the sheet: R1, R2
