File: SpectDrone/SpectDrone.kicad_sch (KiCad schematic)
At the start: 118 parts, among them J1 Conn_02x03_Counter_Clockwise, J1-1 Conn_01x04_Male, J1-2 Conn_01x04_Male, J2 GPS, J3 Barrel_Jack, J3V3 Conn_01x01_Male, J4 BME280, J5-1 BNO055-1, J5-2 BNO055-2, Q1 FDN340P, Q2 FDN340P, SW0 SW_Push, SW1 SW_Push, SW10 SW_Push, SW2 SW_Push, SW3 SW_Push, SW4 SW_Push, SW5 SW_Push, SW6 SW_Push, SW7 SW_Push, SW8 SW_Push, SW9 SW_Push, U1 C12666MA, U10 TXS0102DCUR, U11 PCA9306DC, U12 AD799x, U2 C12666MA, U3 LM7805_TO220, U4 MCP112-450E/TO, U5 MCP112-450E/TO, U6 LM7805_TO220, U7 Teensy4.0

Commit message: SpectDrone Development
Parts:
- added C15: 0.1uF, Capacitor_SMD:C_0805_2012Metric, symbol Device:C_Small
- added J1V0-1, J3V1-1, J5V3-1, J5V3-2, JGND1-1, JGND1-2, JVIN1-1: Conn_01x01_Male, Connector_PinHeader_2.54mm:PinHeader_1x01_P2.54mm_Vertical, symbol Connector:Conn_01x01_Male
- added J5: RFShield_OnePiece, RF_Shielding:Laird_Technologies_BMI-S-101_13.66x12.70mm, symbol Device:RFShield_OnePiece
- added R13: 1M, Capacitor_SMD:C_0805_2012Metric, symbol Device:R
Connections:
- net 3V1: now also J3V1-1.1 (Pin_1)
- net 3v_RX: now also JALT1.6 (Pin_6); no longer JALT1.5 (Pin_5)
- net 3v_TX: now also JALT1.5 (Pin_5); no longer JALT1.6 (Pin_6)
- net 5V3: now also J5V3-1.1 (Pin_1), J5V3-2.1 (Pin_1); no longer C13.1, C14.1, R6.2, U12.8 (VDD)
- net GND1: now also C15.2, JGND1-1.1 (Pin_1), JGND1-2.1 (Pin_1), R13.2
- net VIN1: now also JVIN1-1.1 (Pin_1)
- new net 1V2: J1V0-1.1 (Pin_1)
- new net 5V_{RF}: C13.1, C14.1, R6.2, U12.8 (VDD)
- new net GND_RF: C15.1, J5.1 (Shield), R13.1
Other:
- added sheet Band-stop (Band-stop.kicad_sch)
- note added: "U10 & U12"
- moved on the sheet: C13, C14, U12

Commit message: SpectDrone Development
Other:
- moved on the sheet: C10, C15, C9, J1V0-1, J2, J3V1-1, J4, J5, J5-1, J5-2, J5V3-1, J5V3-2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

Commit message: SpectDrone Development
Parts:
- removed C4, C6: 10uF, Capacitor_SMD:C_0805_2012Metric, symbol Device:C_Small
- added C4, C6: 10uF, Capacitor_SMD:CP_Elec_3x5.4, symbol Device:C_Polarized_Small_US
- C13: Part Number (none) -> F381A106MMAAH1
- C14: footprint Capacitor_SMD:C_0603_1608Metric -> Capacitor_SMD:C_0805_2012Metric
- C2: footprint Capacitor_SMD:C_0603_1608Metric -> Capacitor_SMD:CP_Elec_3x5.4
Connections:
- net 5V3: now also C4.1
- net 5V4: now also C6.1
- net GND1: now also C4.2
- net GND2: now also C6.2
Changed lines of the file:
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@@
   (junction (at 248.92 80.01) (diameter 0) (color 0 0 0 0)
   )
-  (junction (at 241.3 21.59) (diameter 0) (color 0 0 0 0)
-  )
   (junction (at 219.71 21.59) (diameter 0) (color 0 0 0 0)
   )
@@
   (junction (at 215.9 80.01) (diameter 0) (color 0 0 0 0)
   )
-  (junction (at 77.47 21.59) (diameter 0) (color 0 0 0 0)
-  )
   (junction (at 70.485 82.55) (diameter 0) (color 0 0 0 0)
   )
@@
   (junction (at 37.465 82.55) (diameter 0) (color 0 0 0 0)
   )
+  (junction (at 241.3 21.59) (diameter 0) (color 0 0 0 0)
+  )
   (junction (at 215.9 69.85) (diameter 0) (color 0 0 0 0)
   )
@@
   (junction (at 34.925 55.88) (diameter 0) (color 0 0 0 0)
   )
+  (junction (at 77.47 21.59) (diameter 0) (color 0 0 0 0)
+  )
   (junction (at 48.26 140.97) (diameter 0) (color 0 0 0 0)
   )
@@
     (pin "3")
   )
+  (symbol (lib_id "Device:C_Polarized_Small_US") (at 241.3 24.13 0) (unit 1)
+    (in_bom yes) (on_board yes)
+    (property "Reference" "C6" (id 0) (at 245.11 25.4 0))
+    (property "Value" "10uF" (id 1) (at 245.11 27.94 0))
+    (property "Footprint" "Capacitor_SMD:CP_Elec_3x5.4" (id 2) (at 241.3 24.13 0)
+      (effects (font (size 1.27 1.27)) hide)
+    )
+    (property "Datasheet" "~" (id 3) (at 241.3 24.13 0)
+      (effects (font (size 1.27 1.27)) hide)
+    )
+    (pin "1")
+    (pin "2")
+  )
   (symbol (lib_id "Device:C_Polarized_Small_US") (at 126.365 67.31 270) (unit 1)
     (in_bom yes) (on_board yes)
     (property "Reference" "C14" (id 0) (at 130.175 67.31 0))
     (property "Value" "0.1uF" (id 1) (at 126.365 69.85 90))
-    (property "Footprint" "Capacitor_SMD:C_0603_1608Metric" (id 2) (at 126.365 67.31 0)
+    (property "Footprint" "Capacitor_SMD:C_0805_2012Metric" (id 2) (at 126.365 67.31 0)
       (effects (font (size 1.27 1.27)) hide)
     )
-    (property "Datasheet" "~" (id 3) (at 126.365 67.31 0)
+    (property "Datasheet" "https://www.vishay.com/docs/40179/tmcp.pdf" (id 3) (at 126.365 67.31 0)
       (effects (font (size 1.27 1.27)) hide)
     )
@@
     )
   )
-  (symbol (lib_id "Device:C_Small") (at 77.47 24.13 0) (unit 1)
-    (in_bom yes) (on_board yes)
-    (property "Reference" "C4" (id 0) (at 78.105 26.035 0)
-      (effects (font (size 1.27 1.27)) (justify left))
-    )
-    (property "Value" "10uF" (id 1) (at 78.105 27.94 0)
-      (effects (font (size 1.27 1.27)) (justify left))
-    )
-    (property "Footprint" "Capacitor_SMD:C_0805_2012Metric" (id 2) (at 77.47 24.13 0)
-      (effects (font (size 1.27 1.27)) hide)
-    )
-    (property "Datasheet" "~" (id 3) (at 77.47 24.13 0)
-      (effects (font (size 1.27 1.27)) hide)
-    )
-    (pin "1")
-    (pin "2")
-  )
   (symbol (lib_id "Connector:Conn_01x01_Male") (at 142.875 165.1 0) (mirror x) (unit 1)
     (in_bom yes) (on_board yes)
@@
     )
   )
-  (symbol (lib_id "Device:C_Small") (at 241.3 24.13 0) (unit 1)
-    (in_bom yes) (on_board yes)
-    (property "Reference" "C6" (id 0) (at 241.935 26.035 0)
-      (effects (font (size 1.27 1.27)) (justify left))
-    )
-    (property "Value" "10uF" (id 1) (at 241.935 27.94 0)
-      (effects (font (size 1.27 1.27)) (justify left))
-    )
-    (property "Footprint" "Capacitor_SMD:C_0805_2012Metric" (id 2) (at 241.3 24.13 0)
-      (effects (font (size 1.27 1.27)) hide)
-    )
-    (property "Datasheet" "~" (id 3) (at 241.3 24.13 0)
-      (effects (font (size 1.27 1.27)) hide)
-    )
-    (pin "1")
-    (pin "2")
-  )
   (symbol (lib_id "Device:C_Small") (at 119.38 111.76 270) (mirror x) (unit 1)
     (in_bom yes) (on_board yes)
@@
       (effects (font (size 1.27 1.27)) hide)
     )
-    (property "Datasheet" "~" (id 3) (at 126.365 62.865 0)
+    (property "Datasheet" "https://datasheets.kyocera-avx.com/F38.pdf" (id 3) (at 126.365 62.865 0)
+      (effects (font (size 1.27 1.27)) hide)
+    )
+    (property "Part Number" "F381A106MMAAH1" (id 4) (at 126.365 62.865 0)
       (effects (font (size 1.27 1.27)) hide)
     )
@@
     (pin "6")
   )
+  (symbol (lib_id "Device:C_Polarized_Small_US") (at 77.47 24.13 0) (unit 1)
+    (in_bom yes) (on_board yes)
+    (property "Reference" "C4" (id 0) (at 81.28 25.4 0))
+    (property "Value" "10uF" (id 1) (at 81.28 27.94 0))
+    (property "Footprint" "Capacitor_SMD:CP_Elec_3x5.4" (id 2) (at 77.47 24.13 0)
+      (effects (font (size 1.27 1.27)) hide)
+    )
+    (property "Datasheet" "~" (id 3) (at 77.47 24.13 0)
+      (effects (font (size 1.27 1.27)) hide)
+    )
+    (pin "1")
+    (pin "2")
+  )
   (symbol (lib_id "Connector:Conn_01x08_Female") (at 151.13 30.48 0) (unit 1)
     (in_bom yes) (on_board yes)
@@
     (property "Reference" "C2" (id 0) (at 61.595 58.42 90))
     (property "Value" "10uF" (id 1) (at 61.595 60.96 90))
-    (property "Footprint" "Capacitor_SMD:C_0603_1608Metric" (id 2) (at 64.135 55.88 0)
+    (property "Footprint" "Capacitor_SMD:CP_Elec_3x5.4" (id 2) (at 64.135 55.88 0)
       (effects (font (size 1.27 1.27)) hide)
     )
@@
     )
   )
-  (sheet (at 138.43 54.61) (size 29.21 12.065) (fields_autoplaced)
+  (sheet (at 138.43 53.975) (size 29.21 12.7) (fields_autoplaced)
     (stroke (width 0.1524) (type solid) (color 0 0 0 0))
     (fill (color 0 0 0 0.0000))
-    (property "Sheet name" "Longwave" (id 0) (at 138.43 53.8984 0)
+    (property "Sheet name" "Longwave" (id 0) (at 138.43 53.2634 0)
       (effects (font (size 1.27 1.27)) (justify left bottom))
     )
@@
     )
     (path "/fd26592e-ed64-49ed-a5c3-f3806d596599"
-      (reference "C2") (unit 1) (value "10uF") (footprint "Capacitor_SMD:C_0603_1608Metric")
+      (reference "C2") (unit 1) (value "10uF") (footprint "Capacitor_SMD:CP_Elec_3x5.4")
     )
     (path "/f8132452-240f-4963-b8d2-904a58923946"
       (reference "C3") (unit 1) (value "0.1uF") (footprint "Capacitor_SMD:C_0805_2012Metric")
     )
-    (path "/4c6d1c4f-815d-4b64-9b7b-5a23cd49842e"
-      (reference "C4") (unit 1) (value "10uF") (footprint "Capacitor_SMD:C_0805_2012Metric")
+    (path "/92427811-8c4c-4b31-976f-ec2422783024"
+      (reference "C4") (unit 1) (value "10uF") (footprint "Capacitor_SMD:CP_Elec_3x5.4")
     )
     (path "/7b7c8c7c-0c7c-4246-ae7a-d3e5c762144e"
       (reference "C5") (unit 1) (value "0.1uF") (footprint "Capacitor_SMD:C_0805_2012Metric")
     )
-    (path "/599c6520-8691-4e2c-81c6-9d50c3dd7f68"
-      (reference "C6") (unit 1) (value "10uF") (footprint "Capacitor_SMD:C_0805_2012Metric")
+    (path "/421d8e29-1043-42dc-8abb-351a6f376897"
+      (reference "C6") (unit 1) (value "10uF") (footprint "Capacitor_SMD:CP_Elec_3x5.4")
     )
     (path "/e7239936-2999-46d3-9f65-8bf9c0cc64dd"
@@
     )
     (path "/43122158-74fb-4bff-a206-ea7936e5b044"
-      (reference "C14") (unit 1) (value "0.1uF") (footprint "Capacitor_SMD:C_0603_1608Metric")
+      (reference "C14") (unit 1) (value "0.1uF") (footprint "Capacitor_SMD:C_0805_2012Metric")
     )
     (path "/fd90dac5-f85a-46a5-99b3-070411286b8d"

Commit message: SpectDrone Development
Parts:
- added CAN_H1, CAN_L1: Conn_01x01_Male, Connector_PinHeader_2.54mm:PinHeader_1x01_P2.54mm_Vertical, symbol Connector:Conn_01x01_Male
- added JIF1: Payload, Connector_PinHeader_2.54mm:PinHeader_1x04_P2.54mm_Vertical, symbol Connector:Conn_01x04_Male
- added JIF2: Base, Connector_PinSocket_2.54mm:PinSocket_1x04_P2.54mm_Vertical, symbol Connector:Conn_01x04_Female
Connections:
- net 5V4 is gone; now on net 5V3: C6.1, JAPC-2.6 (Pin_6), JDIS2.1 (Pin_1), TP4.1, U6.3 (VO), U7.33 (Vin)
- net APCRX is gone; now on net APC2TX: JAPC-1.4 (Pin_4), JAPC1.2 (Pin_2)
- net APCTX is gone; now on net APC2RX: JAPC-1.3 (Pin_3), JAPC1.1 (Pin_1)
- net GND2 is gone; now on net GND1: BT1.2 (-), C5.1, C6.2, C8.1, J3.2, J3.3, JAPC-2.7 (Pin_7), JBAT2.2 (Pin_2), JDIS1.2 (Pin_2), JDIS2.3 (Pin_3), R2.1, RSW1.1, U5.3 (VSS), U6.2 (GND), U7.1 (GND), U7.17 (GND)
- net 5V3: now also JIF1.4 (Pin_4), JIF2.4 (Pin_4)
- net APC2RX: now also JIF1.3 (Pin_3), JIF2.3 (Pin_3)
- net APC2TX: now also JIF1.2 (Pin_2), JIF2.2 (Pin_2)
- net CAN_H: now also CAN_H1.1 (Pin_1)
- net CAN_L: now also CAN_L1.1 (Pin_1)
- net GND1: now also JIF1.1 (Pin_1), JIF2.1 (Pin_1)
- no-connect marks 33 -> 31

Commit message: SpectDrone Development
Parts:
- C15: value 0.1uF -> 2.5pF
- R13: value 1M -> 2K
Connections:
- net 5V3: now also R6.2
- net 5V_{RF}: no longer R6.2
- net A1: no longer U12.3 (Vin0)
- net A2: no longer U12.6 (Vin3)
- net GND1: no longer C13.2, C14.2, U12.7 (GND)
- net S1: no longer U12.4 (Vin1)
- net S2: no longer U12.5 (Vin2)
- net GND_RF renamed GND_{RF}
- net GND_{RF}: now also C13.2, C14.2, U12.7 (GND)
- new net A1_{RF}: U12.3 (Vin0)
- new net A2_{RF}: U12.5 (Vin2)
- new net S1_{RF}: U12.4 (Vin1)
- new net S2_{RF}: U12.6 (Vin3)
Other:
- note added: "U12"
- note removed: "U10 & U12"
- moved on the sheet: C13, C14, U12

Commit message: SpectDrone Development
Parts:
- added J6, J7: Conn_02x16_Counter_Clockwise, Gardenuino Custom:PinSocket_4x16_P2.54mm_Vertical, symbol Gardenuino_Custom:Conn_04x16
- added JP11: SolderJumper_2_Bridged, Jumper:SolderJumper-2_P1.3mm_Bridged2Bar_RoundedPad1.0x1.5mm, symbol Jumper:SolderJumper_2_Bridged
- added JP12, JP13, JP14, JP15: SolderJumper_2_Bridged, Gardenuino Custom:BreakableJumper, symbol Jumper:SolderJumper_2_Bridged
- C13: footprint Capacitor_SMD:C_0603_1608Metric -> Capacitor_SMD:C_0805_2012Metric
- C14: footprint Capacitor_SMD:C_0805_2012Metric -> Capacitor_SMD:C_0603_1608Metric
- J1: footprint Connector_PinSocket_2.54mm:PinSocket_2x04_P2.54mm_Vertical -> Gardenuino Custom:PinSocket_2x04_P2.54mm_Vertical_renumber
- U4: renamed from U3; value LM7805_TO220 -> LM7805_SOT223; footprint Package_TO_SOT_THT:TO-220-3_Vertical -> Package_TO_SOT_SMD:SOT-223-3_TabPin2
- U6: value LM7805_TO220 -> LM7805_SOT223; footprint Package_TO_SOT_THT:TO-220-3_Vertical -> Package_TO_SOT_SMD:SOT-223-3_TabPin2
- renumbered U4 to U3
Connections:
- net 5V3: now also JP15.1 (A); no longer C6.1, JAPC-2.6 (Pin_6), JDIS2.1 (Pin_1), JIF2.4 (Pin_4), TP4.1, U6.3 (VO), U7.33 (Vin)
- net A1_{RF}: now also U12.6 (Vin3); no longer U12.3 (Vin0)
- net A2: now also JA1.4 (Pin_4); no longer JA1.3 (Pin_3)
- net A2_{RF}: now also U12.3 (Vin0); no longer U12.5 (Vin2)
- net APC2RX: now also JP14.2 (B); no longer JAPC-1.3 (Pin_3), JAPC1.1 (Pin_1), JIF1.3 (Pin_3)
- net APC2TX: now also JP13.2 (B); no longer JAPC-1.4 (Pin_4), JAPC1.2 (Pin_2), JIF1.2 (Pin_2)
- net GND1: now also JP11.1 (A), JP12.1 (A); no longer BT1.2 (-), C5.1, C6.2, C8.1, J3.2, J3.3, JAPC-2.7 (Pin_7), JBAT2.2 (Pin_2), JDIS1.2 (Pin_2), JDIS2.3 (Pin_3), JIF2.1 (Pin_1), R2.1, RSW1.1, U5.3 (VSS), U6.2 (GND), U7.1 (GND), U7.17 (GND)
- net GND_{RF}: now also JP11.2 (B)
- net MISO: now also J7.15 (Pin_15)
- net MOSI: now also J7.16 (Pin_16)
- net S1_{RF}: now also U12.5 (Vin2); no longer U12.4 (Vin1)
- net S2: now also JA1.3 (Pin_3); no longer JA1.4 (Pin_4)
- net S2_{RF}: now also U12.4 (Vin1); no longer U12.6 (Vin3)
- net SCK: now also J7.14 (Pin_14)
- net SCL: now also J7.64 (Pin_64)
- net SDA: now also J7.48 (Pin_48)
- net VIN2 renamed VDC
- new net 5V4: C6.1, JAPC-2.6 (Pin_6), JDIS2.1 (Pin_1), JIF2.4 (Pin_4), JP15.2 (B), TP4.1, U6.3 (VO), U7.33 (Vin)
- new net APCRX: JAPC-1.4 (Pin_4), JAPC1.2 (Pin_2), JIF1.2 (Pin_2), JP13.1 (A)
- new net APCTX: JAPC-1.3 (Pin_3), JAPC1.1 (Pin_1), JIF1.3 (Pin_3), JP14.1 (A)
- new net GND2: BT1.2 (-), C5.1, C6.2, C8.1, J3.2, J3.3, JAPC-2.7 (Pin_7), JBAT2.2 (Pin_2), JDIS1.2 (Pin_2), JDIS2.3 (Pin_3), JIF2.1 (Pin_1), JP12.2 (B), R2.1, RSW1.1, U5.3 (VSS), U6.2 (GND), U7.1 (GND), U7.17 (GND)
Other:
- moved on the sheet: C10, C13, C14, C15, C9, CAN_H1, CAN_L1, J1V0-1, J2, J3V1-1, J4, J5-1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

Commit message: SpectDrone Development
Parts:
- JP12, JP13, JP14, JP15: symbol Jumper:SolderJumper_2_Bridged -> Jumper:SolderJumper_2_Open
- renumbered J1V0-1 to J4V0-1
Connections:
- net GND1: now also J7.32 (Pin_32)
- net 1V2 renamed 4.096V
Changed lines of the file:
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@@
     (effects (font (size 1.27 1.27)) (justify left bottom))
   )
+  (label "GND1" (at 92.71 254 0)
+    (effects (font (size 1.27 1.27)) (justify left bottom))
+  )
   (label "UT2" (at 76.2 115.57 0)
     (effects (font (size 1.27 1.27)) (justify left bottom))
@@
     (effects (font (size 1.27 1.27)) (justify right bottom))
   )
-  (label "1V2" (at 109.22 155.575 0)
+  (label "4.096V" (at 109.22 155.575 0)
     (effects (font (size 1.27 1.27)) (justify left bottom))
   )
@@
     (effects (font (size 1.27 1.27)) (justify left bottom))
   )
+  (label "5V0" (at 165.1 254.635 180)
+    (effects (font (size 1.27 1.27)) (justify right bottom))
+  )
   (label "SW1" (at 205.74 59.69 180)
     (effects (font (size 1.27 1.27)) (justify right bottom))
@@
     (effects (font (size 1.27 1.27)) (justify left bottom))
   )
-  (label "1V2" (at 166.37 224.155 180)
+  (label "4.096V" (at 162.56 224.155 180)
     (effects (font (size 1.27 1.27)) (justify right bottom))
   )
@@
     )
   )
-  (global_label "1V2" (shape input) (at 166.37 224.155 0) (fields_autoplaced)
+  (global_label "4.096V" (shape input) (at 162.56 224.155 0) (fields_autoplaced)
     (effects (font (size 1.27 1.27)) (justify left))
-    (property "Intersheet References" "${INTERSHEET_REFS}" (id 0) (at 172.2907 224.0756 0)
+    (property "Intersheet References" "${INTERSHEET_REFS}" (id 0) (at 171.5045 224.0756 0)
       (effects (font (size 1.27 1.27)) (justify left) hide)
     )
@@
     )
   )
+  (global_label "5V0" (shape input) (at 165.1 254.635 0) (fields_autoplaced)
+    (effects (font (size 1.27 1.27)) (justify left))
+    (property "Intersheet References" "${INTERSHEET_REFS}" (id 0) (at 171.0207 254.5556 0)
+      (effects (font (size 1.27 1.27)) (justify left) hide)
+    )
+  )
   (global_label "A1" (shape input) (at 153.67 236.855 180) (fields_autoplaced)
     (effects (font (size 1.27 1.27)) (justify right))
@@
     (pin "1")
   )
-  (symbol (lib_id "Jumper:SolderJumper_2_Bridged") (at 118.745 165.1 0) (mirror x) (unit 1)
+  (symbol (lib_id "Jumper:SolderJumper_2_Open") (at 118.745 165.1 0) (mirror x) (unit 1)
     (in_bom yes) (on_board yes)
     (property "Reference" "JP13" (id 0) (at 121.285 164.465 0))
@@
     (pin "2")
   )
-  (symbol (lib_id "Jumper:SolderJumper_2_Bridged") (at 118.745 167.64 0) (mirror x) (unit 1)
+  (symbol (lib_id "Jumper:SolderJumper_2_Open") (at 118.745 167.64 0) (mirror x) (unit 1)
     (in_bom yes) (on_board yes)
     (property "Reference" "JP14" (id 0) (at 121.285 167.005 0))
@@
   (symbol (lib_id "Connector:Conn_01x01_Male") (at 104.14 155.575 0) (mirror x) (unit 1)
     (in_bom yes) (on_board yes)
-    (property "Reference" "J1V0-1" (id 0) (at 105.41 154.305 0)
+    (property "Reference" "J4V0-1" (id 0) (at 105.41 154.305 0)
       (effects (font (size 1.27 1.27)) (justify right))
     )
@@
     (pin "4")
   )
-  (symbol (lib_id "Jumper:SolderJumper_2_Bridged") (at 118.745 170.18 0) (mirror x) (unit 1)
+  (symbol (lib_id "Jumper:SolderJumper_2_Open") (at 118.745 170.18 0) (mirror x) (unit 1)
     (in_bom yes) (on_board yes)
     (property "Reference" "JP15" (id 0) (at 121.285 169.545 0))
@@
     (pin "2")
   )
-  (symbol (lib_id "Jumper:SolderJumper_2_Bridged") (at 118.745 162.56 0) (mirror x) (unit 1)
+  (symbol (lib_id "Jumper:SolderJumper_2_Open") (at 118.745 162.56 0) (mirror x) (unit 1)
     (in_bom yes) (on_board yes)
     (property "Reference" "JP12" (id 0) (at 121.285 161.925 0))
@@
       (reference "J1-2") (unit 1) (value "Conn_01x04_Male") (footprint "Connector_PinHeader_2.54mm:PinHeader_1x04_P2.54mm_Vertical")
     )
-    (path "/aeb40eeb-bd87-4300-87f5-bb1939c50508"
-      (reference "J1V0-1") (unit 1) (value "Conn_01x01_Male") (footprint "Connector_PinHeader_2.54mm:PinHeader_1x01_P2.54mm_Vertical")
-    )
     (path "/79addd4c-94b0-4421-bf1a-9bce80188468"
       (reference "J2") (unit 1) (value "GPS") (footprint "Connector_JST:JST_XH_B6B-XH-A_1x06_P2.50mm_Vertical")
@@
       (reference "J4") (unit 1) (value "BME280") (footprint "Connector_PinSocket_2.54mm:PinSocket_1x07_P2.54mm_Vertical")
     )
+    (path "/aeb40eeb-bd87-4300-87f5-bb1939c50508"
+      (reference "J4V0-1") (unit 1) (value "Conn_01x01_Male") (footprint "Connector_PinHeader_2.54mm:PinHeader_1x01_P2.54mm_Vertical")
+    )
     (path "/6eb86b9e-8bbb-4bf7-9c5a-a6d9b427965e"
       (reference "J5") (unit 1) (value "RFShield_OnePiece") (footprint "RF_Shielding:Laird_Technologies_BMI-S-101_13.66x12.70mm")
@@
       (reference "JP15") (unit 1) (value "SolderJumper_2_Bridged") (footprint "Gardenuino Custom:BreakableJumper")
     )
+    (path "/e2721bc0-0e6a-4575-b0d1-362e0ffdee3c/cc1f75fa-4ecc-42ba-9eca-342b8e1a1619"
+      (reference "JP16") (unit 1) (value "SolderJumper_3_Bridged12") (footprint "Jumper:SolderJumper-3_P1.3mm_Bridged2Bar12_RoundedPad1.0x1.5mm")
+    )
     (path "/e2721bc0-0e6a-4575-b0d1-362e0ffdee3c/f45ed21a-aad0-4820-9e85-b5ee8dd22921"
       (reference "JPV1") (unit 1) (value "SolderJumper_2_Bridged") (footprint "Jumper:SolderJumper-2_P1.3mm_Bridged_RoundedPad1.0x1.5mm")
@@
       (reference "R9") (unit 1) (value "470K") (footprint "Capacitor_SMD:C_0805_2012Metric")
     )
-    (path "/e2721bc0-0e6a-4575-b0d1-362e0ffdee3c/e6266b84-2db1-4be2-a9ea-9d37d2f709be"
-      (reference "R10") (unit 1) (value "470K") (footprint "Capacitor_SMD:C_0805_2012Metric")
+    (path "/e2721bc0-0e6a-4575-b0d1-362e0ffdee3c/a0032689-e541-4f0e-b571-7f4776bbc742"
+      (reference "R10") (unit 1) (value "0") (footprint "Resistor_SMD:R_0603_1608Metric")
     )
     (path "/b830ae61-5cf3-45d7-b837-1eb84500b62b"
@@
     )
     (path "/e2721bc0-0e6a-4575-b0d1-362e0ffdee3c/1876c30c-72b2-4a8d-9f32-bf8b213530b4"
-      (reference "RS2") (unit 1) (value "12K4") (footprint "Capacitor_SMD:C_0805_2012Metric")
+      (reference "RS2") (unit 1) (value "R") (footprint "Capacitor_SMD:C_0805_2012Metric")
     )
     (path "/e2721bc0-0e6a-4575-b0d1-362e0ffdee3c/4ba1327d-cfd3-4cf5-8277-a2b3eec8cfea"
@@
     )
     (path "/e2721bc0-0e6a-4575-b0d1-362e0ffdee3c/653fdf05-7ad5-427f-9ad5-b898b68fc587"
-      (reference "RS5") (unit 1) (value "12K4") (footprint "Capacitor_SMD:C_0805_2012Metric")
+      (reference "RS5") (unit 1) (value "R") (footprint "Capacitor_SMD:C_0805_2012Metric")
     )
     (path "/e2721bc0-0e6a-4575-b0d1-362e0ffdee3c/1e64913e-e481-4166-b792-ef53d04299f2"
@@
       (reference "RV1") (unit 1) (value "10K") (footprint "Potentiometer_THT:Potentiometer_Bourns_3296W_Vertical")
     )
-    (path "/e2721bc0-0e6a-4575-b0d1-362e0ffdee3c/fdb61b3f-be50-4154-9c6e-015949e5994b"
-      (reference "RV2") (unit 1) (value "10K") (footprint "Potentiometer_THT:Potentiometer_Bourns_3296W_Vertical")
-    )
     (path "/e53d234c-34ee-414a-bc81-a886319740b6"
       (reference "SW0") (unit 1) (value "SW_Push") (footprint "Button_Switch_THT:SW_PUSH_6mm_H4.3mm")
@@
       (reference "TP5") (unit 1) (value "TestPoint") (footprint "TestPoint:TestPoint_Keystone_5000-5004_Miniature")
     )
+    (path "/e2721bc0-0e6a-4575-b0d1-362e0ffdee3c/0c011518-ed06-48e0-8b1e-0e106c0f7563"
+      (reference "TP5v0-1") (unit 1) (value "TestPoint") (footprint "TestPoint:TestPoint_Keystone_5000-5004_Miniature")
+    )
     (path "/e2721bc0-0e6a-4575-b0d1-362e0ffdee3c/0017297a-7de7-4b26-ac36-da2a8ebddace"
       (reference "TPv1-1") (unit 1) (value "TestPoint") (footprint "TestPoint:TestPoint_Keystone_5000-5004_Miniature")
@@
     )
     (path "/e2721bc0-0e6a-4575-b0d1-362e0ffdee3c/b15f1833-1c73-492c-922e-ef0f8affc888"
-      (reference "U9") (unit 1) (value "ADR510") (footprint "Package_TO_SOT_SMD:SOT-23")
+      (reference "U9") (unit 1) (value "ADR504") (footprint "Package_TO_SOT_SMD:SOT-23")
     )
     (path "/721b0118-f7ed-41a6-8c66-6d4a657f1174"
@@
       (reference "U12") (unit 1) (value "AD799x") (footprint "Package_TO_SOT_SMD:SOT-23-8")
     )
+    (path "/e2721bc0-0e6a-4575-b0d1-362e0ffdee3c/bed00ef8-7ad5-4aee-8105-bde4dec392a7"
+      (reference "U13") (unit 1) (value "ADR5045B") (footprint "Package_TO_SOT_SMD:SOT-23")
+    )
     (path "/e2721bc0-0e6a-4575-b0d1-362e0ffdee3c/0554bea0-89b2-4e25-9ea3-4c73921c94cb"

Commit message: SpectDrone Development
Other:
- moved on the sheet: JIF1, JIF2, JP12, JP13, JP14, JP15
