File: SpectDrone/Band-stop.kicad_sch (KiCad schematic)
At the start: 4 parts

Commit message: SpectDrone Development
Other:
- moved on the sheet: C16, C17, R14, R15
Changed lines of the file:
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@@
 (kicad_sch (version 20211123) (generator eeschema)
   (paper "A4")
-  (junction (at 142.24 86.36) (diameter 0) (color 0 0 0 0)
+  (junction (at 84.455 97.155) (diameter 0) (color 0 0 0 0)
   )
-  (junction (at 149.86 72.39) (diameter 0) (color 0 0 0 0)
+  (junction (at 89.535 84.455) (diameter 0) (color 0 0 0 0)
   )
-  (junction (at 146.05 66.04) (diameter 0) (color 0 0 0 0)
+  (junction (at 84.455 84.455) (diameter 0) (color 0 0 0 0)
   )
-  (junction (at 138.43 78.74) (diameter 0) (color 0 0 0 0)
+  (junction (at 84.455 71.755) (diameter 0) (color 0 0 0 0)
   )
-  (junction (at 125.73 72.39) (diameter 0) (color 0 0 0 0)
-  )
-  (wire (pts (xy 146.05 86.36) (xy 146.05 73.66))
+  (wire (pts (xy 89.535 94.615) (xy 89.535 97.155))
     (stroke (width 0) (type default) (color 0 0 0 0))
   )
-  (wire (pts (xy 149.86 72.39) (xy 154.94 72.39))
+  (wire (pts (xy 84.455 94.615) (xy 84.455 97.155))
     (stroke (width 0) (type default) (color 0 0 0 0))
   )
-  (wire (pts (xy 138.43 78.74) (xy 149.86 78.74))
+  (wire (pts (xy 89.535 84.455) (xy 92.075 84.455))
     (stroke (width 0) (type default) (color 0 0 0 0))
   )
-  (wire (pts (xy 146.05 66.04) (xy 149.86 66.04))
+  (wire (pts (xy 89.535 84.455) (xy 84.455 84.455))
     (stroke (width 0) (type default) (color 0 0 0 0))
   )
-  (wire (pts (xy 149.86 66.04) (xy 149.86 72.39))
+  (wire (pts (xy 84.455 84.455) (xy 84.455 86.995))
     (stroke (width 0) (type default) (color 0 0 0 0))
   )
-  (wire (pts (xy 142.24 86.36) (xy 142.24 91.44))
+  (wire (pts (xy 84.455 97.155) (xy 81.915 97.155))
     (stroke (width 0) (type default) (color 0 0 0 0))
   )
-  (wire (pts (xy 138.43 86.36) (xy 142.24 86.36))
+  (wire (pts (xy 84.455 97.155) (xy 89.535 97.155))
     (stroke (width 0) (type default) (color 0 0 0 0))
   )
-  (wire (pts (xy 142.24 86.36) (xy 146.05 86.36))
+  (wire (pts (xy 81.915 71.755) (xy 84.455 71.755))
     (stroke (width 0) (type default) (color 0 0 0 0))
   )
-  (wire (pts (xy 125.73 72.39) (xy 125.73 78.74))
+  (wire (pts (xy 89.535 84.455) (xy 89.535 86.995))
     (stroke (width 0) (type default) (color 0 0 0 0))
   )
-  (wire (pts (xy 118.11 72.39) (xy 125.73 72.39))
+  (wire (pts (xy 84.455 81.915) (xy 84.455 84.455))
     (stroke (width 0) (type default) (color 0 0 0 0))
   )
-  (wire (pts (xy 133.35 78.74) (xy 138.43 78.74))
+  (wire (pts (xy 89.535 71.755) (xy 89.535 74.295))
     (stroke (width 0) (type default) (color 0 0 0 0))
   )
-  (wire (pts (xy 125.73 66.04) (xy 125.73 72.39))
+  (wire (pts (xy 84.455 71.755) (xy 89.535 71.755))
     (stroke (width 0) (type default) (color 0 0 0 0))
   )
-  (wire (pts (xy 149.86 72.39) (xy 149.86 78.74))
+  (wire (pts (xy 84.455 71.755) (xy 84.455 74.295))
     (stroke (width 0) (type default) (color 0 0 0 0))
   )
-  (wire (pts (xy 133.35 66.04) (xy 146.05 66.04))
+  (wire (pts (xy 89.535 81.915) (xy 89.535 84.455))
     (stroke (width 0) (type default) (color 0 0 0 0))
   )
-  (global_label "5V_{RF}" (shape input) (at 154.94 72.39 0) (fields_autoplaced)
+  (global_label "5V_{RF}" (shape input) (at 92.075 84.455 0) (fields_autoplaced)
     (effects (font (size 1.27 1.27)) (justify left))
-    (property "Intersheet References" "${INTERSHEET_REFS}" (id 0) (at 161.5381 72.3106 0)
+    (property "Intersheet References" "${INTERSHEET_REFS}" (id 0) (at 98.6731 84.3756 0)
       (effects (font (size 1.27 1.27)) (justify left) hide)
     )
   )
-  (global_label "5V3" (shape input) (at 118.11 72.39 180) (fields_autoplaced)
+  (global_label "5V3" (shape input) (at 81.915 71.755 180) (fields_autoplaced)
     (effects (font (size 1.27 1.27)) (justify right))
-    (property "Intersheet References" "${INTERSHEET_REFS}" (id 0) (at 112.1893 72.4694 0)
+    (property "Intersheet References" "${INTERSHEET_REFS}" (id 0) (at 75.9943 71.8344 0)
       (effects (font (size 1.27 1.27)) (justify right) hide)
     )
   )
-  (global_label "GND1" (shape input) (at 142.24 91.44 0) (fields_autoplaced)
-    (effects (font (size 1.27 1.27)) (justify left))
-    (property "Intersheet References" "${INTERSHEET_REFS}" (id 0) (at 149.7331 91.3606 0)
-      (effects (font (size 1.27 1.27)) (justify left) hide)
+  (global_label "GND1" (shape input) (at 81.915 97.155 180) (fields_autoplaced)
+    (effects (font (size 1.27 1.27)) (justify right))
+    (property "Intersheet References" "${INTERSHEET_REFS}" (id 0) (at 74.4219 97.2344 0)
+      (effects (font (size 1.27 1.27)) (justify right) hide)
     )
   )
-  (symbol (lib_id "Device:C") (at 146.05 69.85 0) (unit 1)
-    (in_bom yes) (on_board yes) (fields_autoplaced)
-    (property "Reference" "C17" (id 0) (at 149.86 68.5799 0)
+  (symbol (lib_id "Device:C") (at 89.535 90.805 0) (unit 1)
+    (in_bom yes) (on_board yes)
+    (property "Reference" "C17" (id 0) (at 92.71 90.17 0)
       (effects (font (size 1.27 1.27)) (justify left))
     )
-    (property "Value" "C" (id 1) (at 149.86 71.1199 0)
+    (property "Value" "C" (id 1) (at 93.98 92.71 0)
       (effects (font (size 1.27 1.27)) (justify left))
     )
-    (property "Footprint" "Capacitor_SMD:C_0603_1608Metric" (id 2) (at 147.0152 73.66 0)
+    (property "Footprint" "Capacitor_SMD:C_0603_1608Metric" (id 2) (at 90.5002 94.615 0)
       (effects (font (size 1.27 1.27)) hide)
     )
-    (property "Datasheet" "~" (id 3) (at 146.05 69.85 0)
+    (property "Datasheet" "~" (id 3) (at 89.535 90.805 0)
       (effects (font (size 1.27 1.27)) hide)
     )
@@
     (pin "2")
   )
-  (symbol (lib_id "Device:R") (at 129.54 66.04 90) (unit 1)
-    (in_bom yes) (on_board yes) (fields_autoplaced)
-    (property "Reference" "R14" (id 0) (at 129.54 60.325 90))
-    (property "Value" "R" (id 1) (at 129.54 62.865 90))
-    (property "Footprint" "Resistor_SMD:R_0603_1608Metric" (id 2) (at 129.54 67.818 90)
+  (symbol (lib_id "Device:R") (at 84.455 78.105 0) (mirror y) (unit 1)
+    (in_bom yes) (on_board yes)
+    (property "Reference" "R14" (id 0) (at 80.01 76.835 0))
+    (property "Value" "R" (id 1) (at 80.01 79.375 0))
+    (property "Footprint" "Resistor_SMD:R_0603_1608Metric" (id 2) (at 86.233 78.105 90)
       (effects (font (size 1.27 1.27)) hide)
     )
-    (property "Datasheet" "~" (id 3) (at 129.54 66.04 0)
+    (property "Datasheet" "~" (id 3) (at 84.455 78.105 0)
       (effects (font (size 1.27 1.27)) hide)
     )
@@
     (pin "2")
   )
-  (symbol (lib_id "Device:C") (at 129.54 78.74 90) (unit 1)
-    (in_bom yes) (on_board yes) (fields_autoplaced)
-    (property "Reference" "C16" (id 0) (at 129.54 71.755 90))
-    (property "Value" "C" (id 1) (at 129.54 74.295 90))
-    (property "Footprint" "Capacitor_SMD:C_0603_1608Metric" (id 2) (at 133.35 77.7748 0)
+  (symbol (lib_id "Device:C") (at 89.535 78.105 0) (mirror y) (unit 1)
+    (in_bom yes) (on_board yes)
+    (property "Reference" "C16" (id 0) (at 94.615 76.835 0))
+    (property "Value" "C" (id 1) (at 94.615 79.375 0))
+    (property "Footprint" "Capacitor_SMD:C_0603_1608Metric" (id 2) (at 88.5698 81.915 0)
       (effects (font (size 1.27 1.27)) hide)
     )
-    (property "Datasheet" "~" (id 3) (at 129.54 78.74 0)
+    (property "Datasheet" "~" (id 3) (at 89.535 78.105 0)
       (effects (font (size 1.27 1.27)) hide)
     )
@@
     (pin "2")
   )
-  (symbol (lib_id "Device:R") (at 138.43 82.55 180) (unit 1)
-    (in_bom yes) (on_board yes) (fields_autoplaced)
-    (property "Reference" "R15" (id 0) (at 140.335 81.2799 0)
+  (symbol (lib_id "Device:R") (at 84.455 90.805 180) (unit 1)
+    (in_bom yes) (on_board yes)
+    (property "Reference" "R15" (id 0) (at 78.105 92.075 0)
       (effects (font (size 1.27 1.27)) (justify right))
     )
-    (property "Value" "R" (id 1) (at 140.335 83.8199 0)
+    (property "Value" "R" (id 1) (at 79.375 89.535 0)
       (effects (font (size 1.27 1.27)) (justify right))
     )
-    (property "Footprint" "Resistor_SMD:R_0603_1608Metric" (id 2) (at 140.208 82.55 90)
+    (property "Footprint" "Resistor_SMD:R_0603_1608Metric" (id 2) (at 86.233 90.805 90)
       (effects (font (size 1.27 1.27)) hide)
     )
-    (property "Datasheet" "~" (id 3) (at 138.43 82.55 0)
+    (property "Datasheet" "~" (id 3) (at 84.455 90.805 0)
       (effects (font (size 1.27 1.27)) hide)
     )

Commit message: SpectDrone Development
Parts:
- added C18, C19, C20, C21, C22, C23, C24, C25: C, Resistor_SMD:R_0402_1005Metric, symbol Device:C
- added R16, R17, R18, R19, R20, R21, R22, R23: R, Resistor_SMD:R_0402_1005Metric, symbol Device:R
- R14: value R -> 0
- R15: value R -> X
Connections:
- net GND1 renamed GND_{RF}
- net GND_{RF}: now also C19.2, C21.2, C23.2, C25.2, R17.1, R19.1, R21.1, R23.1
- new net A1: C18.1, R16.2
- new net A1_{RF}: C18.2, C19.1, R16.1, R17.2
- new net A2: C24.1, R22.2
- new net A2_{RF}: C24.2, C25.1, R22.1, R23.2
- new net S1: C20.1, R18.2
- new net S1_{RF}: C20.2, C21.1, R18.1, R19.2
- new net S2: C22.1, R20.2
- new net S2_{RF}: C22.2, C23.1, R20.1, R21.2

Commit message: SpectDrone Development
Parts:
- added C26: 1pF, Capacitor_SMD:C_0603_1608Metric, symbol Device:C
- added C27: 0.1uF, Capacitor_SMD:C_0603_1608Metric, symbol Device:C
- C16: value C -> X; footprint Capacitor_SMD:C_0603_1608Metric -> Capacitor_Tantalum_SMD:CP_EIA-2012-15_AVX-P; symbol Device:C -> Device:C_Polarized_US
- C17: value C -> X
- C18, C19, C20, C21, C22, C23, C24, C25: value C -> X; footprint Resistor_SMD:R_0402_1005Metric -> Capacitor_SMD:C_0402_1005Metric
- R16, R18, R20, R22: value R -> 0
- R17, R19, R21, R23: value R -> X
Connections:
- net 5V3: now also C26.1, C27.1
- net 5V_{RF}: now also C26.2, C27.2
- net A1: now also C22.1, R20.2; no longer C18.1, R16.2
- net A1_{RF}: now also C22.2, C23.1, R20.1, R21.2; no longer C18.2, C19.1, R16.1, R17.2
- net A2: now also C18.1, R16.2; no longer C24.1, R22.2
- net A2_{RF}: now also C18.2, C19.1, R16.1, R17.2; no longer C24.2, C25.1, R22.1, R23.2
- net S1: now also C24.1, R22.2; no longer C20.1, R18.2
- net S1_{RF}: now also C24.2, C25.1, R22.1, R23.2; no longer C20.2, C21.1, R18.1, R19.2
- net S2: now also C20.1, R18.2; no longer C22.1, R20.2
- net S2_{RF}: now also C20.2, C21.1, R18.1, R19.2; no longer C22.2, C23.1, R20.1, R21.2
Other:
- moved on the sheet: C18, C19, C20, C21, C22, C23, C24, C25, R14, R16, R17, R18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

Commit message: SpectDrone Development
Connections:
- net 5V3 renamed 5VS
Other:
- moved on the sheet: C16, C17, C18, C19, C20, C21, C22, C23, C24, C25, C26, C27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

Commit message: SpectDrone Development
Changed lines of the file:
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@@
   (symbol (lib_id "Device:R") (at 213.995 81.28 180) (unit 1)
     (in_bom yes) (on_board yes)
-    (property "Reference" "R16" (id 0) (at 218.44 82.55 0))
-    (property "Value" "0" (id 1) (at 218.44 80.01 0))
+    (property "Reference" "R16" (id 0) (at 218.44 80.01 0))
+    (property "Value" "0" (id 1) (at 218.44 82.55 0))
     (property "Footprint" "Resistor_SMD:R_0402_1005Metric" (id 2) (at 215.773 81.28 90)
       (effects (font (size 1.27 1.27)) hide)
@@
   (symbol (lib_id "Device:C") (at 132.08 88.265 0) (mirror y) (unit 1)
     (in_bom yes) (on_board yes)
-    (property "Reference" "C27" (id 0) (at 128.905 87.63 0)
+    (property "Reference" "C27" (id 0) (at 129.54 87.63 0)
       (effects (font (size 1.27 1.27)) (justify left))
     )
@@
   (symbol (lib_id "Device:R") (at 208.915 124.46 180) (unit 1)
     (in_bom yes) (on_board yes)
-    (property "Reference" "R19" (id 0) (at 202.565 125.73 0)
-      (effects (font (size 1.27 1.27)) (justify right))
-    )
-    (property "Value" "X" (id 1) (at 203.835 123.19 0)
+    (property "Reference" "R19" (id 0) (at 202.565 121.92 0)
+      (effects (font (size 1.27 1.27)) (justify right))
+    )
+    (property "Value" "X" (id 1) (at 203.835 124.46 0)
       (effects (font (size 1.27 1.27)) (justify right))
     )
@@
   (symbol (lib_id "Device:C") (at 213.995 93.98 0) (unit 1)
     (in_bom yes) (on_board yes)
-    (property "Reference" "C19" (id 0) (at 215.265 91.44 0)
-      (effects (font (size 1.27 1.27)) (justify left))
-    )
-    (property "Value" "X" (id 1) (at 216.535 93.98 0)
+    (property "Reference" "C19" (id 0) (at 216.535 91.44 0)
+      (effects (font (size 1.27 1.27)) (justify left))
+    )
+    (property "Value" "X" (id 1) (at 217.805 93.98 0)
       (effects (font (size 1.27 1.27)) (justify left))
     )
@@
   (symbol (lib_id "Device:R") (at 183.515 111.76 180) (unit 1)
     (in_bom yes) (on_board yes)
-    (property "Reference" "R22" (id 0) (at 187.96 113.03 0))
-    (property "Value" "0" (id 1) (at 187.96 110.49 0))
+    (property "Reference" "R22" (id 0) (at 187.96 110.49 0))
+    (property "Value" "0" (id 1) (at 187.96 113.03 0))
     (property "Footprint" "Resistor_SMD:R_0402_1005Metric" (id 2) (at 185.293 111.76 90)
       (effects (font (size 1.27 1.27)) hide)
@@
   (symbol (lib_id "Device:R") (at 183.515 81.28 180) (unit 1)
     (in_bom yes) (on_board yes)
-    (property "Reference" "R20" (id 0) (at 187.96 82.55 0))
-    (property "Value" "0" (id 1) (at 187.96 80.01 0))
+    (property "Reference" "R20" (id 0) (at 187.96 80.01 0))
+    (property "Value" "0" (id 1) (at 187.96 82.55 0))
     (property "Footprint" "Resistor_SMD:R_0402_1005Metric" (id 2) (at 185.293 81.28 90)
       (effects (font (size 1.27 1.27)) hide)
@@
   (symbol (lib_id "Device:C") (at 122.555 88.265 0) (mirror y) (unit 1)
     (in_bom yes) (on_board yes)
-    (property "Reference" "C26" (id 0) (at 119.38 87.63 0)
+    (property "Reference" "C26" (id 0) (at 120.015 87.63 0)
       (effects (font (size 1.27 1.27)) (justify left))
     )
@@
   (symbol (lib_id "Device:R") (at 178.435 93.98 180) (unit 1)
     (in_bom yes) (on_board yes)
-    (property "Reference" "R21" (id 0) (at 172.085 95.25 0)
-      (effects (font (size 1.27 1.27)) (justify right))
-    )
-    (property "Value" "X" (id 1) (at 173.355 92.71 0)
+    (property "Reference" "R21" (id 0) (at 172.085 91.44 0)
+      (effects (font (size 1.27 1.27)) (justify right))
+    )
+    (property "Value" "X" (id 1) (at 173.355 93.98 0)
       (effects (font (size 1.27 1.27)) (justify right))
     )
@@
   (symbol (lib_id "Device:R") (at 146.685 88.265 0) (unit 1)
     (in_bom yes) (on_board yes)
-    (property "Reference" "R14" (id 0) (at 151.13 86.995 0))
-    (property "Value" "0" (id 1) (at 151.13 89.535 0))
+    (property "Reference" "R14" (id 0) (at 151.13 87.63 0))
+    (property "Value" "0" (id 1) (at 151.13 90.17 0))
     (property "Footprint" "Resistor_SMD:R_0603_1608Metric" (id 2) (at 144.907 88.265 90)
       (effects (font (size 1.27 1.27)) hide)
@@
   (symbol (lib_id "Device:R") (at 178.435 124.46 180) (unit 1)
     (in_bom yes) (on_board yes)
-    (property "Reference" "R23" (id 0) (at 172.085 125.73 0)
-      (effects (font (size 1.27 1.27)) (justify right))
-    )
-    (property "Value" "X" (id 1) (at 173.355 123.19 0)
+    (property "Reference" "R23" (id 0) (at 172.085 121.92 0)
+      (effects (font (size 1.27 1.27)) (justify right))
+    )
+    (property "Value" "X" (id 1) (at 173.355 124.46 0)
       (effects (font (size 1.27 1.27)) (justify right))
     )
@@
   (symbol (lib_id "Device:C") (at 213.995 124.46 0) (unit 1)
     (in_bom yes) (on_board yes)
-    (property "Reference" "C21" (id 0) (at 215.265 121.92 0)
-      (effects (font (size 1.27 1.27)) (justify left))
-    )
-    (property "Value" "X" (id 1) (at 216.535 124.46 0)
+    (property "Reference" "C21" (id 0) (at 216.535 121.92 0)
+      (effects (font (size 1.27 1.27)) (justify left))
+    )
+    (property "Value" "X" (id 1) (at 217.805 124.46 0)
       (effects (font (size 1.27 1.27)) (justify left))
     )
@@
   (symbol (lib_id "Device:R") (at 208.915 93.98 180) (unit 1)
     (in_bom yes) (on_board yes)
-    (property "Reference" "R17" (id 0) (at 202.565 95.25 0)
-      (effects (font (size 1.27 1.27)) (justify right))
-    )
-    (property "Value" "X" (id 1) (at 203.835 92.71 0)
+    (property "Reference" "R17" (id 0) (at 202.565 91.44 0)
+      (effects (font (size 1.27 1.27)) (justify right))
+    )
+    (property "Value" "X" (id 1) (at 203.835 93.98 0)
       (effects (font (size 1.27 1.27)) (justify right))
     )
@@
   (symbol (lib_id "Device:C_Polarized_US") (at 141.605 88.265 0) (unit 1)
     (in_bom yes) (on_board yes)
-    (property "Reference" "C16" (id 0) (at 136.525 86.995 0))
-    (property "Value" "X" (id 1) (at 136.525 89.535 0))
+    (property "Reference" "C16" (id 0) (at 137.16 87.63 0))
+    (property "Value" "X" (id 1) (at 140.335 90.805 0))
     (property "Footprint" "Capacitor_Tantalum_SMD:CP_EIA-2012-15_AVX-P" (id 2) (at 141.605 88.265 0)
       (effects (font (size 1.27 1.27)) hide)
@@
   (symbol (lib_id "Device:R") (at 141.605 100.965 180) (unit 1)
     (in_bom yes) (on_board yes)
-    (property "Reference" "R15" (id 0) (at 135.255 102.235 0)
-      (effects (font (size 1.27 1.27)) (justify right))
-    )
-    (property "Value" "X" (id 1) (at 136.525 99.695 0)
+    (property "Reference" "R15" (id 0) (at 135.255 100.33 0)
+      (effects (font (size 1.27 1.27)) (justify right))
+    )
+    (property "Value" "X" (id 1) (at 136.525 102.87 0)
       (effects (font (size 1.27 1.27)) (justify right))
     )
@@
   (symbol (lib_id "Device:R") (at 213.995 111.76 180) (unit 1)
     (in_bom yes) (on_board yes)
-    (property "Reference" "R18" (id 0) (at 218.44 113.03 0))
-    (property "Value" "0" (id 1) (at 218.44 110.49 0))
+    (property "Reference" "R18" (id 0) (at 218.44 110.49 0))
+    (property "Value" "0" (id 1) (at 218.44 113.03 0))
     (property "Footprint" "Resistor_SMD:R_0402_1005Metric" (id 2) (at 215.773 111.76 90)
       (effects (font (size 1.27 1.27)) hide)
@@
   (symbol (lib_id "Device:C") (at 183.515 124.46 0) (unit 1)
     (in_bom yes) (on_board yes)
-    (property "Reference" "C25" (id 0) (at 185.42 121.92 0)
-      (effects (font (size 1.27 1.27)) (justify left))
-    )
-    (property "Value" "X" (id 1) (at 186.055 124.46 0)
+    (property "Reference" "C25" (id 0) (at 186.055 121.92 0)
+      (effects (font (size 1.27 1.27)) (justify left))
+    )
+    (property "Value" "X" (id 1) (at 187.325 124.46 0)
       (effects (font (size 1.27 1.27)) (justify left))
     )
@@
   (symbol (lib_id "Device:C") (at 183.515 93.98 0) (unit 1)
     (in_bom yes) (on_board yes)
-    (property "Reference" "C23" (id 0) (at 184.785 91.44 0)
-      (effects (font (size 1.27 1.27)) (justify left))
-    )
-    (property "Value" "X" (id 1) (at 186.055 93.98 0)
-      (effects (font (size 1.27 1.27)) (justify left))
-    )
+    (property "Reference" "C23" (id 0) (at 186.055 91.44 0)
+      (effects (font (size 1.27 1.27)) (justify left))
+    )
+    (property "Value" "X" (id 1) (at 187.325 93.98 0)
+      (effects (font (size 1.27 1.27)) (justify left))
+    )

Commit message: SpectDrone Development
Connections:
- net 5VS renamed V_{AREF}
- net 5V_{RF} renamed V_{RF}
Changed lines of the file:
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@@
     )
   )
-  (global_label "5V_{RF}" (shape input) (at 151.13 94.615 0) (fields_autoplaced)
+  (global_label "V_{RF}" (shape input) (at 151.13 94.615 0) (fields_autoplaced)
     (effects (font (size 1.27 1.27)) (justify left))
-    (property "Intersheet References" "${INTERSHEET_REFS}" (id 0) (at 157.7281 94.5356 0)
+    (property "Intersheet References" "${INTERSHEET_REFS}" (id 0) (at 156.5185 94.5356 0)
       (effects (font (size 1.27 1.27)) (justify left) hide)
     )
@@
     )
   )
-  (global_label "5VS" (shape input) (at 116.84 81.915 180) (fields_autoplaced)
+  (global_label "V_{AREF}" (shape input) (at 116.84 81.915 180) (fields_autoplaced)
     (effects (font (size 1.27 1.27)) (justify right))
-    (property "Intersheet References" "${INTERSHEET_REFS}" (id 0) (at 110.9193 81.8356 0)
+    (property "Intersheet References" "${INTERSHEET_REFS}" (id 0) (at 109.6614 81.8356 0)
       (effects (font (size 1.27 1.27)) (justify right) hide)
     )

Commit message: SpectDrone Development
Connections:
- net A1 is gone; now on net S1: C22.1, R20.2
- net A1_{RF} is gone; now on net S1_{RF}: C22.2, C23.1, R20.1, R21.2
- net A2 is gone; now on net S2: C18.1, R16.2
- net A2_{RF} is gone; now on net S2_{RF}: C18.2, C19.1, R16.1, R17.2
- net S1: no longer C24.1, R22.2
- net S1_{RF}: no longer C24.2, C25.1, R22.1, R23.2
- net S2: no longer C20.1, R18.2
- net S2_{RF}: no longer C20.2, C21.1, R18.1, R19.2
- new net P1: C24.1, R22.2
- new net P1_{RF}: C24.2, C25.1, R22.1, R23.2
- new net P2: C20.1, R18.2
- new net P2_{RF}: C20.2, C21.1, R18.1, R19.2
Other:
- moved on the sheet: C16, C17, C18, C19, C20, C21, C22, C23, C24, C25, C26, C27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

Commit message: SpectDrone Development
Parts:
- C26: footprint Capacitor_SMD:C_0603_1608Metric -> Capacitor_SMD:C_0402_1005Metric; Part Number (none) -> CL05C010CB5NNNC
- C27: Part Number (none) -> CL05A104KA5NNNC
Changed lines of the file:
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@@
+      (effects (font (size 1.27 1.27)) hide)
+    )
+    (property "Part Number" "CL05A104KA5NNNC" (id 4) (at 108.585 93.98 0)
       (effects (font (size 1.27 1.27)) hide)
     )
@@
       (effects (font (size 1.27 1.27)) (justify left))
     )
-    (property "Footprint" "Capacitor_SMD:C_0603_1608Metric" (id 2) (at 98.0948 97.79 0)
+    (property "Footprint" "Capacitor_SMD:C_0402_1005Metric" (id 2) (at 98.0948 97.79 0)
       (effects (font (size 1.27 1.27)) hide)
     )
@@
       (effects (font (size 1.27 1.27)) hide)
     )
+    (property "Part Number" "CL05C010CB5NNNC" (id 4) (at 99.06 93.98 0)
+      (effects (font (size 1.27 1.27)) hide)
+    )
