File: SpectDrone/Band-stop.kicad_sch (KiCad schematic)
At the start: 22 parts

Commit message: SpectDrone Development
Parts:
- R14: Part Number (none) -> ERJ-U030R00V
- R16, R18, R20, R22: Part Number (none) -> ERJ-2GE0R00X
Changed lines of the file:
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@@
+      (effects (font (size 1.27 1.27)) hide)
+    )
+    (property "Part Number" "ERJ-2GE0R00X" (id 4) (at 190.5 78.74 0)
       (effects (font (size 1.27 1.27)) hide)
     )
@@
       (effects (font (size 1.27 1.27)) hide)
     )
+    (property "Part Number" "ERJ-2GE0R00X" (id 4) (at 160.02 109.22 0)
+      (effects (font (size 1.27 1.27)) hide)
+    )
     (pin "1")
     (pin "2")
@@
       (effects (font (size 1.27 1.27)) hide)
     )
+    (property "Part Number" "ERJ-2GE0R00X" (id 4) (at 160.02 78.74 0)
+      (effects (font (size 1.27 1.27)) hide)
+    )
     (pin "1")
     (pin "2")
@@
       (effects (font (size 1.27 1.27)) hide)
     )
+    (property "Part Number" "ERJ-U030R00V" (id 4) (at 123.19 93.98 0)
+      (effects (font (size 1.27 1.27)) hide)
+    )
     (pin "1")
     (pin "2")
@@
       (effects (font (size 1.27 1.27)) hide)
     )
+    (property "Part Number" "ERJ-2GE0R00X" (id 4) (at 190.5 109.22 0)
+      (effects (font (size 1.27 1.27)) hide)
+    )

Commit message: SpectDrone Development
Parts:
- C16, C17, C18, C19, C20, C21, C22, C23, C24, C25, R15, R17, R19, R21, R23: now left out of the parts list
Changed lines of the file:
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@@
   )
   (symbol (lib_id "Device:C") (at 123.19 106.68 0) (unit 1)
-    (in_bom yes) (on_board yes)
+    (in_bom no) (on_board yes)
     (property "Reference" "C17" (id 0) (at 126.365 106.045 0)
       (effects (font (size 1.27 1.27)) (justify left))
@@
   )
   (symbol (lib_id "Device:R") (at 185.42 121.92 180) (unit 1)
-    (in_bom yes) (on_board yes)
+    (in_bom no) (on_board yes)
     (property "Reference" "R19" (id 0) (at 179.07 119.38 0)
       (effects (font (size 1.27 1.27)) (justify right))
@@
   )
   (symbol (lib_id "Device:C") (at 154.94 78.74 0) (unit 1)
-    (in_bom yes) (on_board yes)
+    (in_bom no) (on_board yes)
     (property "Reference" "C22" (id 0) (at 150.495 77.47 0))
     (property "Value" "X" (id 1) (at 150.495 80.01 0))
@@
   )
   (symbol (lib_id "Device:C") (at 190.5 91.44 0) (unit 1)
-    (in_bom yes) (on_board yes)
+    (in_bom no) (on_board yes)
     (property "Reference" "C19" (id 0) (at 193.04 88.9 0)
       (effects (font (size 1.27 1.27)) (justify left))
@@
   )
   (symbol (lib_id "Device:R") (at 154.94 91.44 180) (unit 1)
-    (in_bom yes) (on_board yes)
+    (in_bom no) (on_board yes)
     (property "Reference" "R21" (id 0) (at 148.59 88.9 0)
       (effects (font (size 1.27 1.27)) (justify right))
@@
   )
   (symbol (lib_id "Device:R") (at 154.94 121.92 180) (unit 1)
-    (in_bom yes) (on_board yes)
+    (in_bom no) (on_board yes)
     (property "Reference" "R23" (id 0) (at 148.59 119.38 0)
       (effects (font (size 1.27 1.27)) (justify right))
@@
   )
   (symbol (lib_id "Device:C") (at 190.5 121.92 0) (unit 1)
-    (in_bom yes) (on_board yes)
+    (in_bom no) (on_board yes)
     (property "Reference" "C21" (id 0) (at 193.04 119.38 0)
       (effects (font (size 1.27 1.27)) (justify left))
@@
   )
   (symbol (lib_id "Device:C") (at 154.94 109.22 0) (unit 1)
-    (in_bom yes) (on_board yes)
+    (in_bom no) (on_board yes)
     (property "Reference" "C24" (id 0) (at 150.495 107.95 0))
     (property "Value" "X" (id 1) (at 150.495 110.49 0))
@@
   )
   (symbol (lib_id "Device:R") (at 185.42 91.44 180) (unit 1)
-    (in_bom yes) (on_board yes)
+    (in_bom no) (on_board yes)
     (property "Reference" "R17" (id 0) (at 179.07 88.9 0)
       (effects (font (size 1.27 1.27)) (justify right))
@@
   )
   (symbol (lib_id "Device:C") (at 185.42 78.74 0) (unit 1)
-    (in_bom yes) (on_board yes)
+    (in_bom no) (on_board yes)
     (property "Reference" "C18" (id 0) (at 180.975 77.47 0))
     (property "Value" "X" (id 1) (at 180.975 80.01 0))
@@
   )
   (symbol (lib_id "Device:C_Polarized_US") (at 118.11 93.98 0) (unit 1)
-    (in_bom yes) (on_board yes)
+    (in_bom no) (on_board yes)
     (property "Reference" "C16" (id 0) (at 113.665 93.345 0))
     (property "Value" "X" (id 1) (at 116.84 96.52 0))
@@
   )
   (symbol (lib_id "Device:R") (at 118.11 106.68 180) (unit 1)
-    (in_bom yes) (on_board yes)
+    (in_bom no) (on_board yes)
     (property "Reference" "R15" (id 0) (at 111.76 106.045 0)
       (effects (font (size 1.27 1.27)) (justify right))
@@
   )
   (symbol (lib_id "Device:C") (at 160.02 121.92 0) (unit 1)
-    (in_bom yes) (on_board yes)
+    (in_bom no) (on_board yes)
     (property "Reference" "C25" (id 0) (at 162.56 119.38 0)
       (effects (font (size 1.27 1.27)) (justify left))
@@
   )
   (symbol (lib_id "Device:C") (at 160.02 91.44 0) (unit 1)
-    (in_bom yes) (on_board yes)
+    (in_bom no) (on_board yes)
     (property "Reference" "C23" (id 0) (at 162.56 88.9 0)
       (effects (font (size 1.27 1.27)) (justify left))
@@
   )
   (symbol (lib_id "Device:C") (at 185.42 109.22 0) (unit 1)
-    (in_bom yes) (on_board yes)
+    (in_bom no) (on_board yes)
     (property "Reference" "C20" (id 0) (at 180.975 107.95 0))
     (property "Value" "X" (id 1) (at 180.975 110.49 0))
