File: SpectDrone/Conn_Proto.kicad_sch (KiCad schematic)
At the start: 2 parts, among them J6 Conn_02x16_Counter_Clockwise, J7 Conn_02x16_Counter_Clockwise

Commit message: SpectDrone Development
Changed lines of the file:
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@@
+    (effects (font (size 1.27 1.27)) (justify right bottom))
+  )
+  (label "SCL" (at 189.865 144.78 180)
+    (effects (font (size 1.27 1.27)) (justify right bottom))
+  )
+  (label "SCK" (at 175.26 138.43 180)
+    (effects (font (size 1.27 1.27)) (justify right bottom))
+  )
+  (label "MOSI" (at 175.26 144.78 180)
+    (effects (font (size 1.27 1.27)) (justify right bottom))
+  )
+  (label "GND1" (at 189.865 138.43 180)
+    (effects (font (size 1.27 1.27)) (justify right bottom))
+  )
+  (label "MISO" (at 175.26 141.605 180)
+    (effects (font (size 1.27 1.27)) (justify right bottom))
+  )
+  (label "SDA" (at 189.865 141.605 180)
     (effects (font (size 1.27 1.27)) (justify right bottom))
   )
@@
     (effects (font (size 1.27 1.27)) (justify right bottom))
   )
-  (symbol (lib_id "Gardenuino_Custom:Conn_04x16") (at 105.41 100.965 0)
+  (global_label "MISO" (shape input) (at 175.26 141.605 0) (fields_autoplaced)
+    (effects (font (size 1.27 1.27)) (justify left))
+    (property "Intersheet References" "${INTERSHEET_REFS}" (id 0) (at 182.2693 141.5256 0)
+      (effects (font (size 1.27 1.27)) (justify left) hide)
+    )
+  )
+  (global_label "GND1" (shape input) (at 189.865 138.43 0) (fields_autoplaced)
+    (effects (font (size 1.27 1.27)) (justify left))
+    (property "Intersheet References" "${INTERSHEET_REFS}" (id 0) (at 197.3581 138.3506 0)
+      (effects (font (size 1.27 1.27)) (justify left) hide)
+    )
+  )
+  (global_label "SDA" (shape input) (at 189.865 141.605 0) (fields_autoplaced)
+    (effects (font (size 1.27 1.27)) (justify left))
+    (property "Intersheet References" "${INTERSHEET_REFS}" (id 0) (at 195.8462 141.5256 0)
+      (effects (font (size 1.27 1.27)) (justify left) hide)
+    )
+  )
+  (global_label "SCL" (shape input) (at 189.865 144.78 0) (fields_autoplaced)
+    (effects (font (size 1.27 1.27)) (justify left))
+    (property "Intersheet References" "${INTERSHEET_REFS}" (id 0) (at 195.7857 144.7006 0)
+      (effects (font (size 1.27 1.27)) (justify left) hide)
+    )
+  )
+  (global_label "MOSI" (shape input) (at 175.26 144.78 0) (fields_autoplaced)
+    (effects (font (size 1.27 1.27)) (justify left))
+    (property "Intersheet References" "${INTERSHEET_REFS}" (id 0) (at 182.2693 144.7006 0)
+      (effects (font (size 1.27 1.27)) (justify left) hide)
+    )
+  )
+  (global_label "SCK" (shape input) (at 175.26 138.43 0) (fields_autoplaced)
+    (effects (font (size 1.27 1.27)) (justify left))
+    (property "Intersheet References" "${INTERSHEET_REFS}" (id 0) (at 181.4226 138.3506 0)
+      (effects (font (size 1.27 1.27)) (justify left) hide)
+    )
+  )
+  (symbol (lib_id "Gardenuino_Custom:Conn_04x16") (at 105.41 100.965 0) (unit 1)
     (in_bom yes) (on_board yes) (fields_autoplaced)
     (property "Reference" "J6" (id 0) (at 120.65 76.2 0))
@@
     (pin "9")
   )
-  (symbol (lib_id "Gardenuino_Custom:Conn_04x16") (at 166.37 100.965 0)
+  (symbol (lib_id "Gardenuino_Custom:Conn_04x16") (at 166.37 100.965 0) (unit 1)
     (in_bom yes) (on_board yes) (fields_autoplaced)
     (property "Reference" "J7" (id 0) (at 181.61 76.2 0))

Commit message: SpectDrone Development
Parts:
- J6, J7: Part Number (none) -> RS2-08-G; now left out of the parts list
Changed lines of the file:
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@@
   )
   (symbol (lib_id "Gardenuino_Custom:Conn_04x16") (at 105.41 100.965 0) (unit 1)
-    (in_bom yes) (on_board yes) (fields_autoplaced)
+    (in_bom no) (on_board yes) (fields_autoplaced)
     (property "Reference" "J6" (id 0) (at 120.65 76.2 0))
     (property "Value" "Conn_02x16_Counter_Clockwise" (id 1) (at 120.65 78.74 0))
@@
     )
     (property "Datasheet" "~" (id 3) (at 105.41 100.965 0)
+      (effects (font (size 1.27 1.27)) hide)
+    )
+    (property "Part Number" "RS2-08-G" (id 4) (at 105.41 100.965 0)
       (effects (font (size 1.27 1.27)) hide)
     )
@@
   )
   (symbol (lib_id "Gardenuino_Custom:Conn_04x16") (at 166.37 100.965 0) (unit 1)
-    (in_bom yes) (on_board yes) (fields_autoplaced)
+    (in_bom no) (on_board yes) (fields_autoplaced)
     (property "Reference" "J7" (id 0) (at 181.61 76.2 0))
     (property "Value" "Conn_02x16_Counter_Clockwise" (id 1) (at 181.61 78.74 0))
@@
       (effects (font (size 1.27 1.27)) hide)
     )
+    (property "Part Number" "RS2-08-G" (id 4) (at 166.37 100.965 0)
+      (effects (font (size 1.27 1.27)) hide)
+    )

Commit message: SpectDrone Development
Connections:
- net GND1: now also J6.56 (Pin_56)
- net 5V3: now reaches J6.55 (Pin_55)
Changed lines of the file:
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@@
 (kicad_sch (version 20230121) (generator eeschema)
   (paper "A4")
+  (label "5V3" (at 140.97 98.425 0) (fields_autoplaced)
+    (effects (font (size 1.27 1.27)) (justify left bottom))
+  )
   (label "SDA" (at 189.23 121.285 180) (fields_autoplaced)
     (effects (font (size 1.27 1.27)) (justify right bottom))
@@
   (label "SCL" (at 201.93 121.285 0) (fields_autoplaced)
     (effects (font (size 1.27 1.27)) (justify left bottom))
+  )
+  (label "5V3" (at 175.26 147.32 180) (fields_autoplaced)
+    (effects (font (size 1.27 1.27)) (justify right bottom))
   )
   (label "SCK" (at 161.29 116.205 180) (fields_autoplaced)
@@
   (label "MISO" (at 161.29 118.745 180) (fields_autoplaced)
     (effects (font (size 1.27 1.27)) (justify right bottom))
+  )
+  (label "GND1" (at 140.97 100.965 0) (fields_autoplaced)
+    (effects (font (size 1.27 1.27)) (justify left bottom))
   )
   (label "SCL" (at 189.865 144.78 180) (fields_autoplaced)
@@
       (effects (font (size 1.27 1.27)) (justify left) hide)
     )
+  )
+  (global_label "5V3" (shape input) (at 175.26 147.32 0) (fields_autoplaced)
+    (effects (font (size 1.27 1.27)) (justify left))
+    (property "Intersheetrefs" "${INTERSHEET_REFS}" (at 181.1807 147.2406 0)
+      (effects (font (size 1.27 1.27)) (justify left) hide)
+    )

Commit message: SpectDrone Development
Connections:
- net SDA4: now reaches J7.47 (Pin_47)
- net SCL4: now reaches J7.63 (Pin_63)
Changed lines of the file:
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@@
+    (effects (font (size 1.27 1.27)) (justify right bottom))
+  )
+  (label "SDA4" (at 189.865 148.59 180) (fields_autoplaced)
     (effects (font (size 1.27 1.27)) (justify right bottom))
   )
@@
   )
   (label "GND1" (at 140.97 100.965 0) (fields_autoplaced)
+    (effects (font (size 1.27 1.27)) (justify left bottom))
+  )
+  (label "SCL4" (at 201.93 118.745 0) (fields_autoplaced)
     (effects (font (size 1.27 1.27)) (justify left bottom))
   )
@@
   )
   (label "MOSI" (at 161.29 121.285 180) (fields_autoplaced)
+    (effects (font (size 1.27 1.27)) (justify right bottom))
+  )
+  (label "SDA4" (at 189.23 118.745 180) (fields_autoplaced)
+    (effects (font (size 1.27 1.27)) (justify right bottom))
+  )
+  (label "SCL4" (at 189.865 151.765 180) (fields_autoplaced)
     (effects (font (size 1.27 1.27)) (justify right bottom))
   )
@@
       (effects (font (size 1.27 1.27)) (justify left) hide)
     )
+  )
+  (global_label "SCL4" (shape input) (at 189.865 151.765 0) (fields_autoplaced)
+    (effects (font (size 1.27 1.27)) (justify left))
+    (property "Intersheetrefs" "${INTERSHEET_REFS}" (at 197.5673 151.765 0)
+      (effects (font (size 1.27 1.27)) (justify left) hide)
+    )
+  )
+  (global_label "SDA4" (shape input) (at 189.865 148.59 0) (fields_autoplaced)
+    (effects (font (size 1.27 1.27)) (justify left))
+    (property "Intersheetrefs" "${INTERSHEET_REFS}" (at 197.6278 148.59 0)
+      (effects (font (size 1.27 1.27)) (justify left) hide)
+    )
