File: Gardenuino V0.1f/nutrient V0.1f.kicad_pcb (KiCad board)
At the start: 2 copper layers, 99.1 x 71.1 mm, 84 parts, among them J1 Conn_01x04_Female, J2 Conn_01x04_Female, J3 Conn_01x04_Female, J4 Conn_01x04_Female, J5 Conn_01x04_Female, J6 Conn_01x04_Female, J7 Conn_01x03_Male, J8 Conn_01x03_Male, P1 SolderJumper_2_Open, P2 SolderJumper_2_Bridged, P3 SolderJumper_2_Bridged, Q1 Q_NMOS_DGS, Q10 Q_NMOS_DGS, Q2 Q_NMOS_DGS, Q3 Q_NMOS_DGS, Q4 Q_NMOS_DGS, Q5 Q_NMOS_DGS, Q6 Q_NMOS_DGS, Q7 Q_NMOS_DGS, Q8 2N3904, U1 23LC512, U2 DS1307+, Y1 Crystal_Small

Commit message: SpectDrone Development
Other:
- board text added: "Gardeuino v0.1f"
- board text removed: "Gardeuino v0.1e"
Changed lines of the file:
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@@
   (gr_line (start 99.568 34.798) (end 198.628 34.798) (layer "Edge.Cuts") (width 0.05))
   (gr_line (start 99.568 105.918) (end 99.568 34.798) (layer "Edge.Cuts") (width 0.05))
-  (gr_text "Gardeuino v0.1e" (at 168.656 46.228) (layer "B.Cu")
+  (gr_text "Gardeuino v0.1f" (at 168.656 46.228) (layer "B.Cu")
     (effects (font (size 1.5 1.5) (thickness 0.3)) (justify mirror))
   )
@@
     (effects (font (size 0.5 0.5) (thickness 0.1)) (justify mirror))
   )
-  (gr_text "Gardeuino v0.1e" (at 168.656 46.228) (layer "B.SilkS")
+  (gr_text "Gardeuino v0.1f" (at 168.656 46.228) (layer "B.SilkS")
     (effects (font (size 1.5 1.5) (thickness 0.15)) (justify mirror))
   )

Commit message: SpectDrone development
Parts:
- J1, J3, J4, J6: value Conn_01x04_Female -> Conn_01x04_Male; footprint Connector_JST:JST_XH_B4B-XH-A_1x04_P2.50mm_Vertical -> Connector_PinHeader_2.54mm:PinHeader_1x04_P2.54mm_Vertical
- J2, J5: footprint Connector_JST:JST_XH_B4B-XH-A_1x04_P2.50mm_Vertical -> Connector_PinSocket_2.54mm:PinSocket_1x04_P2.54mm_Vertical; moved to B.Cu
- JAUX1: footprint Connector_PinHeader_2.54mm:PinHeader_1x11_P2.54mm_Vertical -> Connector_PinSocket_2.54mm:PinSocket_1x11_P2.54mm_Vertical; moved to B.Cu
- JGPS1: moved to B.Cu
- turned J1 to 0 degrees
- turned J2 to 180 degrees
- turned J3 to 0 degrees
- turned J4 to 0 degrees
- turned J5 to 180 degrees
- turned J6 to 0 degrees
- turned JAUX1 to 0 degrees
- turned JGPS1 to 180 degrees

Commit message: SpectDrone development
Parts:
- added J9: Conn_01x02_Male, Connector_PinHeader_2.54mm:PinHeader_1x02_P2.54mm_Vertical, B.Cu at (113.5, 47.0)
- moved R6 0.95 mm to (110.5, 48.7)
- moved C6 0.80 mm to (117.1, 49.5), turned to -90 degrees
Connections:
- JDC1 pad 3: GND -> Net-(J9-Pad1)
Routing:
- net GND: track 718.0 -> 707.7 mm
- net Net-(J9-Pad1): track 0.00 -> 4.08 mm
- net /VIN1: track 112.6 -> 111.4 mm
- net /VIN: track 208.0 -> 206.8 mm
- net /INT0: track 25.1 -> 24.3 mm
- net Net-(C5-Pad2): track 11.9 -> 11.4 mm
Other:
- board text added: "Gardenuino v0.1f"
- board text removed: "Gardeuino v0.1f"

Commit message: SpectDrone Development
Parts:
- removed J9: Conn_01x02_Male, Connector_PinHeader_2.54mm:PinHeader_1x02_P2.54mm_Vertical
- moved C6 1.52 mm to (115.8, 50.3), turned to 180 degrees
Connections:
- JDC1 pad 3: Net-(J9-Pad1) -> GND
Routing:
- net GND: track 707.7 -> 719.3 mm
- net /VIN1: track 111.4 -> 103.9 mm
- net Net-(J9-Pad1): track 4.08 -> 0.00 mm

Commit message: SpectDrone Development
Parts:
- added J9: Conn_01x01_Male, Connector_PinHeader_2.54mm:PinHeader_1x01_P2.54mm_Vertical, B.Cu at (185.7, 42.9)
- moved C3 0.21 mm to (181.5, 38.9)
Routing:
- net /VIN1: track 103.9 -> 104.8 mm

Commit message: SpectDrone Development
Parts:
- removed JP5: SolderJumper_3_Bridged12, Jumper:SolderJumper-3_P1.3mm_Bridged2Bar12_RoundedPad1.0x1.5mm
- added J10: Conn_01x01_Male, Connector_PinSocket_2.54mm:PinSocket_1x01_P2.54mm_Vertical, B.Cu at (129.3, 58.0)
- J1, J6: footprint Connector_PinHeader_2.54mm:PinHeader_1x04_P2.54mm_Vertical -> Connector_PinSocket_2.54mm:PinSocket_1x04_P2.54mm_Vertical; moved to B.Cu
- JAUX1: footprint Connector_PinSocket_2.54mm:PinSocket_1x11_P2.54mm_Vertical -> Connector_PinSocket_2.54mm:PinSocket_1x12_P2.54mm_Vertical
- moved C1 5.68 mm to (127.1, 53.9), turned to -90 degrees
- moved Q1 1.19 mm to (129.5, 50.2)
- moved RQD7 1.09 mm to (129.9, 73.6)
- moved P1 0.72 mm to (132.8, 81.3)
- moved BT1 0.44 mm to (136.6, 77.0)
- turned J1 to 180 degrees
- turned J6 to 180 degrees
Connections:
- JAUX1 pad 10: /OPT_EXT -> /TX
- JAUX1 pad 11: /D12 -> /OPT_EXT
- JAUX1 pad 8: /XCL -> /AUX_INT
- JAUX1 pad 9: /TX -> /D19
- P3 pad 1: /INT -> /D19
- XA1 pad 3V2: unconnected-(XA1-Pad3V2) -> Net-(XA1-Pad3V2)
- XA1 pad D16: /D16 -> /GPSTX
- XA1 pad D18: /INT -> /AUX_INT
- XA1 pad D19: /GPSTX -> /D19
Routing:
- net /D19: track 0.00 -> 26.3 mm
- net /INT: track 24.0 -> 0.00 mm
- net /5V2: track 122.8 -> 129.4 mm
- net Net-(XA1-Pad3V2): track 0.00 -> 5.01 mm
- net Net-(BT1-Pad1): track 21.5 -> 25.7 mm
- net /AUX_INT: track 0.00 -> 3.88 mm
- net /D12: track 39.9 -> 43.2 mm
- net /GPSTX: track 16.2 -> 19.5 mm
- net /OPT_EXT: track 4.45 -> 6.26 mm
- net /XCL: track 1.69 -> 0.00 mm
- net /D16: track 1.27 -> 0.00 mm
- net Net-(Q1-Pad2): track 5.37 -> 4.18 mm
- net GND: track 719.4 -> 718.7 mm
- net Net-(RQ7-Pad1): track 25.0 -> 25.6 mm
Other:
- board text added: "3.3V"
- board text added: "RX1"
- board text added: "RX2"
- board text added: "RX2_enable"
- board text added: "TX1"
- board text added: "TX2"
- board text removed: "EXT"
- board text removed: "EXT_enable"
- board text removed: "XCL int"
- board text removed: "XDA TX"

Commit message: SpectDrone Development
Parts:
- added P4: SolderJumper_2_Bridged, Jumper:SolderJumper-2_P1.3mm_Bridged2Bar_RoundedPad1.0x1.5mm, B.Cu at (126.1, 84.5)
- J1, J6: footprint Connector_PinSocket_2.54mm:PinSocket_1x04_P2.54mm_Vertical -> Connector_PinHeader_2.54mm:PinHeader_1x04_P2.54mm_Vertical
- J10: footprint Connector_PinSocket_2.54mm:PinSocket_1x01_P2.54mm_Vertical -> Connector_PinHeader_2.54mm:PinHeader_1x01_P2.54mm_Vertical
Connections:
- JAUX1 pad 9: /D19 -> Net-(JAUX1-Pad9)
Routing:
- net /D19: track 26.3 -> 23.3 mm
- net Net-(JAUX1-Pad9): track 0.00 -> 1.95 mm
