File: Gardenuino V0.1f/nutrient V0.1f.kicad_pcb (KiCad board)
At the start: 2 copper layers, 99.1 x 71.1 mm, 86 parts, among them J1 Conn_01x04_Male, J10 Conn_01x01_Male, J2 Conn_01x04_Female, J3 Conn_01x04_Male, J4 Conn_01x04_Male, J5 Conn_01x04_Female, J6 Conn_01x04_Male, J7 Conn_01x03_Male, J8 Conn_01x03_Male, J9 Conn_01x01_Male, P1 SolderJumper_2_Open, P2 SolderJumper_2_Bridged, P3 SolderJumper_2_Bridged, P4 SolderJumper_2_Bridged, Q1 Q_NMOS_DGS, Q10 Q_NMOS_DGS, Q2 Q_NMOS_DGS, Q3 Q_NMOS_DGS, Q4 Q_NMOS_DGS, Q5 Q_NMOS_DGS, Q6 Q_NMOS_DGS, Q7 Q_NMOS_DGS, Q8 2N3904, U1 23LC512, U2 DS1307+, Y1 Crystal_Small

Commit message: SpectDrone Development
Changed lines of the file:
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@@
   (segment locked (start 112.22999 41.85861) (end 113.1946 40.894) (width 1) (layer "B.Cu") (net 27))
   (segment locked (start 120.957482 43.307) (end 125.091471 47.440989) (width 1) (layer "B.Cu") (net 27))
-  (segment (start 112.22999 45.49149) (end 111.76 45.96148) (width 0.75) (layer "B.Cu") (net 27))
   (segment locked (start 107.315 60.024) (end 109.065021 58.273979) (width 0.25) (layer "B.Cu") (net 27))
   (segment (start 111.506 52.206853) (end 111.506 54.687002) (width 0.75) (layer "B.Cu") (net 27))
@@
   (segment locked (start 115.697 55.372) (end 115.57 55.499) (width 0.75) (layer "B.Cu") (net 27))
   (segment (start 116.967 41.783) (end 118.491 43.307) (width 1) (layer "B.Cu") (net 27))
-  (segment (start 111.76 45.96148) (end 111.76 48.065147) (width 0.75) (layer "B.Cu") (net 27))
   (segment locked (start 189.54501 38.82399) (end 189.54501 73.34499) (width 1) (layer "B.Cu") (net 27))
   (segment locked (start 115.57 55.499) (end 115.316 55.753) (width 0.75) (layer "B.Cu") (net 27))
-  (segment (start 112.113489 48.418636) (end 112.113489 49.938511) (width 0.75) (layer "B.Cu") (net 27))
   (segment locked (start 118.237 60.2615) (end 118.237 61.595) (width 0.75) (layer "B.Cu") (net 27))
   (segment (start 116.967 41.148) (end 116.713 40.894) (width 0.75) (layer "B.Cu") (net 27))
@@
   (segment (start 112.113489 51.599364) (end 111.506 52.206853) (width 0.75) (layer "B.Cu") (net 27))
   (segment locked (start 115.57 55.499) (end 115.824 55.499) (width 0.75) (layer "B.Cu") (net 27))
+  (segment (start 112.22999 45.49149) (end 112.113489 45.607991) (width 0.75) (layer "B.Cu") (net 27))
   (segment locked (start 127.539611 47.440989) (end 137.322611 37.657989) (width 1) (layer "B.Cu") (net 27))
   (segment locked (start 115.316 55.753) (end 112.571998 55.753) (width 0.75) (layer "B.Cu") (net 27))
@@
   (segment locked (start 124.46 60.96) (end 123.2 59.7) (width 0.4) (layer "B.Cu") (net 27))
   (segment locked (start 189.611 76.327) (end 189.611 95.227) (width 1) (layer "B.Cu") (net 27))
-  (segment (start 111.76 48.065147) (end 112.113489 48.418636) (width 0.75) (layer "B.Cu") (net 27))
   (segment (start 109.065021 50.954979) (end 110.081489 49.938511) (width 0.25) (layer "B.Cu") (net 27))
   (segment locked (start 112.571998 55.753) (end 111.506 54.687002) (width 0.75) (layer "B.Cu") (net 27))
+  (segment (start 112.113489 45.607991) (end 112.113489 49.938511) (width 0.75) (layer "B.Cu") (net 27))
   (segment locked (start 118.237 59.69) (end 118.7985 59.69) (width 0.75) (layer "B.Cu") (net 27))
   (segment locked (start 189.611 95.227) (end 185.672 95.227) (width 1) (layer "B.Cu") (net 27))

Commit message: SpectDrone Development
Parts:
- J1, J2: moved to F.Cu
- J3: value Conn_01x04_Male -> Conn_01x04_Female; footprint Connector_PinHeader_2.54mm:PinHeader_1x04_P2.54mm_Vertical -> Connector_PinSocket_2.54mm:PinSocket_1x04_P2.54mm_Vertical; moved to B.Cu
- J6: value Conn_01x04_Male -> Conn_01x04_Female; footprint Connector_PinHeader_2.54mm:PinHeader_1x04_P2.54mm_Vertical -> Connector_PinSocket_2.54mm:PinSocket_1x04_P2.54mm_Vertical
- P1: value SolderJumper_2_Open -> SolderJumper_2_Bridged; footprint Jumper:SolderJumper-2_P1.3mm_Open_RoundedPad1.0x1.5mm -> Jumper:SolderJumper-2_P1.3mm_Bridged2Bar_RoundedPad1.0x1.5mm
- moved P3 1.20 mm to (113.2, 100.4), turned to 90 degrees
- moved R1 0.25 mm to (131.1, 103.1)
- moved P1 0.12 mm to (132.7, 81.3), turned to 180 degrees
- moved JP6 0.10 mm to (120.4, 80.0), turned to 90 degrees
- turned P4 to 90 degrees
- turned J1 to 0 degrees
- turned J2 to 0 degrees
- turned J3 to 180 degrees
Connections:
- net /AUX_INT renamed /TX1
- net /D19 renamed /RX1
- net /INT0 renamed /INT4
- net /INT1 renamed /INT5
- net /TX renamed /TX3
- net Net-(JAUX1-Pad9) renamed /RX1_OPT
- JAUX1 pad 11: /OPT_EXT -> /RX3_OPT
- JGPS1 pad 3: /GPSRX -> /TX2
- JGPS1 pad 4: /GPSTX -> /RX2
- JP6 pad 1: /D13 -> /RX
- JP6 pad 3: /RX -> /D13
- P1 pad 1: /OPT_EXT -> /OPT
- P1 pad 2: /OPT -> /RX3_OPT
- XA1 pad D15: /RX -> /RX3
- XA1 pad D16: /GPSTX -> /TX2
- XA1 pad D17: /GPSRX -> /RX2
Routing:
- net /TX2: track 0.00 -> 26.4 mm
- net /GPSTX: track 19.5 -> 0.00 mm
- net /RX2: track 0.00 -> 17.7 mm
- net /GPSRX: track 16.1 -> 0.00 mm
- net /RX3_OPT: track 0.00 -> 6.30 mm
- net /OPT_EXT: track 6.26 -> 0.00 mm
- net /RX1: track 23.3 -> 26.3 mm
- net /RX3: track 0.00 -> 1.98 mm
- net /RX: track 1.98 -> 0.00 mm
- net GND: track 718.7 -> 719.8 mm
- net /SS_MMC: track 69.6 -> 70.5 mm
- net /D51: track 121.0 -> 121.9 mm
- net /SCL: track 181.8 -> 182.6 mm
- net /5V3: track 124.1 -> 124.9 mm
- net /MISDO: track 78.0 -> 78.8 mm
Other:
- board text added: "OPT_enable"
- board text added: "PPS_enable"
- board text added: "RX1_OPT_disable"
- board text added: "RX3"
- board text added: "RX3_disable"
- board text added: "TX3"
- board text added: "d13 RX3"
- board text removed: "D15 rx"
- board text removed: "INT_disable"
- board text removed: "OPT_disable"
- board text removed: "RX2"
- board text removed: "RX2_enable"
- board text removed: "TX2"

Commit message: SpectDrone development
Parts:
- J4: moved to B.Cu
- turned J4 to 180 degrees
Connections:
- net /RX2 renamed /GPSTX
- net /TX2 renamed /GPSRX
- net /VIN renamed /AREF
Other:
- board text added: "AREF="
- board text removed: "VIN="

Commit message: SpectDrone development
Parts:
- J2: value Conn_01x04_Female -> Conn_01x04_Male; footprint Connector_PinSocket_2.54mm:PinSocket_1x04_P2.54mm_Vertical -> Connector_PinHeader_2.54mm:PinHeader_1x04_P2.54mm_Vertical
- J4: footprint Connector_PinHeader_2.54mm:PinHeader_1x04_P2.54mm_Vertical -> Connector_PinSocket_2.54mm:PinSocket_1x04_P2.54mm_Vertical
- moved P1 0.96 mm to (131.8, 81.4)
Connections:
- JP6 pad 1: /RX -> /RX3
Routing:
- net Net-(BT1-Pad1): track 25.7 -> 24.1 mm
- net /RX3_OPT: track 6.30 -> 5.37 mm
- net /RX1: track 26.5 -> 25.8 mm
- net /VIN1: track 104.8 -> 104.1 mm
- net /RX3: track 1.98 -> 1.27 mm
- net /D13: track 1.98 -> 1.27 mm
- net Net-(Q1-Pad2): track 4.18 -> 3.59 mm
Other:
- board text added: "AUX OPT"
- board text added: "AUXOPT_disable"
- board text added: "VIN"
- board text removed: "RX3_disable"
- board text removed: "d13 RX3"

Commit message: SpectDrone development
Routing:
- net (no net): vias 0 -> 1
Changed lines of the file:
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@@
     )
     (pad_to_mask_clearance 0)
-    (aux_axis_origin 196.088 103.378)
-    (grid_origin 196.088 103.378)
+    (aux_axis_origin 196.088 70.358)
+    (grid_origin 196.088 70.358)
     (pcbplotparams
       (layerselection 0x00010fc_ffffffff)
@@
     (fp_line (start 1.029025 -0.762) (end -1.029025 -0.762) (layer "B.SilkS") (width 0.12))
     (fp_line (start -2.0368 0) (end -2.3368 0.3) (layer "B.SilkS") (width 0.12))
-    (fp_arc (start -1.524 0.5588) (mid -1.750184 -0.27911) (end -1.029025 -0.762) (layer "B.SilkS") (width 0.12))
+    (fp_arc (start -1.524 0.5588) (mid -1.750184 -0.279111) (end -1.029025 -0.762) (layer "B.SilkS") (width 0.12))
     (fp_arc (start 1.029025 -0.762) (mid 1.750142 -0.279094) (end 1.524 0.5588) (layer "B.SilkS") (width 0.12))
     (fp_line (start 1.905 -0.889) (end -1.905 -0.889) (layer "B.CrtYd") (width 0.05))
@@
     (effects (font (size 0.5 0.5) (thickness 0.125)))
   )
+  (via (at 196.088 70.358) (size 0.8) (drill 0.4) (layers "F.Cu" "B.Cu") (free) (net 0))
   (segment (start 174.625 93.98) (end 172.085 96.52) (width 0.25) (layer "B.Cu") (net 12))
   (segment locked (start 167.085033 103.297967) (end 172.085 98.298) (width 0.25) (layer "B.Cu") (net 12))

Commit message: SpectDrone Development
Parts:
- moved R2 0.76 mm to (131.6, 96.1)
- moved R9 0.76 mm to (131.6, 89.0)
- moved Q10 0.70 mm to (134.4, 95.1)
- moved R10 0.08 mm to (140.7, 82.5), turned to -140 degrees
Connections:
- JAUX1 pad 4: /SS_AUX -> /D52
Routing:
- net /D52: track 77.0 -> 116.0 mm
- net /SS_AUX: track 23.8 -> 25.1 mm
- net /D51: track 122.0 -> 120.8 mm
- net /GND3: track 23.6 -> 22.7 mm
- net /SS_INV: track 2.32 -> 1.63 mm

Commit message: SpectDrone Development
Parts:
- J1, J2: value Conn_01x04_Male -> Conn_01x04_Female; footprint Connector_PinHeader_2.54mm:PinHeader_1x04_P2.54mm_Vertical -> Connector_PinSocket_2.54mm:PinSocket_1x04_P2.54mm_Vertical; moved to B.Cu
- turned J1 to 180 degrees
- turned J2 to 180 degrees

Commit message: SpectDrone Development
Routing:
- net /RX1: track 25.8 -> 26.4 mm
Changed lines of the file:
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@@
     (fp_line (start 1.029025 -0.762) (end -1.029025 -0.762) (layer "B.SilkS") (width 0.12))
     (fp_line (start -2.0368 0) (end -2.3368 0.3) (layer "B.SilkS") (width 0.12))
-    (fp_arc (start -1.524 0.5588) (mid -1.750184 -0.279111) (end -1.029025 -0.762) (layer "B.SilkS") (width 0.12))
+    (fp_arc (start -1.524 0.5588) (mid -1.750184 -0.27911) (end -1.029025 -0.762) (layer "B.SilkS") (width 0.12))
     (fp_arc (start 1.029025 -0.762) (mid 1.750142 -0.279094) (end 1.524 0.5588) (layer "B.SilkS") (width 0.12))
     (fp_line (start 1.905 -0.889) (end -1.905 -0.889) (layer "B.CrtYd") (width 0.05))
@@
   (segment locked (start 164.737021 60.444913) (end 176.908935 60.444913) (width 0.25) (layer "B.Cu") (net 45))
   (segment locked (start 157.48 68.58) (end 158.75 68.58) (width 0.25) (layer "B.Cu") (net 45))
-  (segment locked (start 180.610106 68.342106) (end 181.864 69.596) (width 0.25) (layer "B.Cu") (net 46))
   (segment locked (start 180.610106 62.874649) (end 180.610106 68.342106) (width 0.25) (layer "B.Cu") (net 46))
   (segment locked (start 177.280348 59.544891) (end 180.610106 62.874649) (width 0.25) (layer "B.Cu") (net 46))
-  (segment locked (start 181.864 69.596) (end 185.568 69.596) (width 0.25) (layer "B.Cu") (net 46))
   (segment locked (start 164.364914 59.544891) (end 177.280348 59.544891) (width 0.25) (layer "B.Cu") (net 46))
-  (segment locked (start 185.568 69.596) (end 185.672 69.7) (width 0.25) (layer "B.Cu") (net 46))
   (segment locked (start 159.31648 64.593325) (end 164.364914 59.544891) (width 0.25) (layer "B.Cu") (net 46))
   (segment locked (start 157.48 66.04) (end 158.75 66.04) (width 0.25) (layer "B.Cu") (net 46))
   (segment locked (start 159.31648 65.47352) (end 159.31648 64.593325) (width 0.25) (layer "B.Cu") (net 46))
+  (segment (start 181.968 69.7) (end 185.672 69.7) (width 0.25) (layer "B.Cu") (net 46))
   (segment locked (start 158.75 66.04) (end 159.31648 65.47352) (width 0.25) (layer "B.Cu") (net 46))
+  (segment (start 180.610106 68.342106) (end 181.968 69.7) (width 0.25) (layer "B.Cu") (net 46))
   (segment locked (start 180.160095 69.289095) (end 180.160095 63.060355) (width 0.25) (layer "B.Cu") (net 47))
   (segment locked (start 159.766 64.779523) (end 159.766 66.294) (width 0.25) (layer "B.Cu") (net 47))
@@
   (segment (start 130.088 77.3195) (end 127.889 75.1205) (width 0.25) (layer "B.Cu") (net 67))
   (segment (start 143.975085 80.17848) (end 143.020502 80.17848) (width 0.25) (layer "B.Cu") (net 67))
-  (segment (start 124.460718 78.74) (end 127.889 75.311718) (width 0.25) (layer "B.Cu") (net 67))
   (segment locked (start 152.908 78.5495) (end 152.908 72.517) (width 0.25) (layer "B.Cu") (net 67))
   (segment locked (start 152.157524 79.299976) (end 152.908 78.5495) (width 0.25) (layer "B.Cu") (net 67))
+  (segment (start 127.889 75.311718) (end 127.889 75.1205) (width 0.25) (layer "B.Cu") (net 67))
+  (segment (start 124.460718 78.74) (end 127.889 75.311718) (width 0.25) (layer "B.Cu") (net 67))
   (segment locked (start 152.908 72.517) (end 151.13 70.739) (width 0.25) (layer "B.Cu") (net 67))
   (segment locked (start 110.363 63.373) (end 112.014 65.024) (width 0.25) (layer "B.Cu") (net 68))
@@
   (segment (start 129.5527 99.2505) (end 129.8067 99.2505) (width 0.25) (layer "B.Cu") (net 76))
   (segment locked (start 116.83232 103.53808) (end 112.171926 103.53808) (width 0.25) (layer "B.Cu") (net 76))
+  (segment (start 131.064 96.597) (end 131.572 96.089) (width 0.25) (layer "B.Cu") (net 76))
   (segment locked (start 127.254 99.2505) (end 129.5527 99.2505) (width 0.25) (layer "B.Cu") (net 76))
   (segment locked (start 110.923479 102.289633) (end 110.923479 73.861521) (width 0.25) (layer "B.Cu") (net 76))
   (segment locked (start 125.857 97.852782) (end 125.857 96.012) (width 0.25) (layer "B.Cu") (net 76))
+  (segment (start 131.064 97.9932) (end 131.064 96.597) (width 0.25) (layer "B.Cu") (net 76))
   (segment (start 129.8067 99.2505) (end 131.064 97.9932) (width 0.25) (layer "B.Cu") (net 76))
   (segment locked (start 110.923479 73.861521) (end 114.3 70.485) (width 0.25) (layer "B.Cu") (net 76))
@@
   (segment locked (start 120.2944 93.0656) (end 120.2944 100.076) (width 0.25) (layer "B.Cu") (net 76))
   (segment locked (start 126.492 98.4885) (end 127.254 99.2505) (width 0.25) (layer "B.Cu") (net 76))
-  (segment (start 131.064 97.9932) (end 131.064 96.343) (width 0.25) (layer "B.Cu") (net 76))
   (segment locked (start 125.857 96.012) (end 125.095 95.25) (width 0.25) (layer "B.Cu") (net 76))
-  (segment (start 131.064 96.343) (end 130.81 96.089) (width 0.25) (layer "B.Cu") (net 76))
   (segment locked (start 123.825 95.25) (end 125.095 95.25) (width 0.25) (layer "B.Cu") (net 76))
   (segment locked (start 148.59 85.9155) (end 148.59 81.915) (width 0.25) (layer "B.Cu") (net 77))
@@
   (segment locked (start 124.46 91.44) (end 125.7935 91.44) (width 0.25) (layer "B.Cu") (net 78))
   (segment (start 121.92 78.74) (end 120.65 78.74) (width 0.25) (layer "B.Cu") (net 79))
+  (segment (start 120.396 78.994) (end 120.65 78.74) (width 0.25) (layer "B.Cu") (net 79))
   (segment (start 152.14188 79.750469) (end 153.670001 81.27859) (width 0.25) (layer "B.Cu") (net 80))
   (segment (start 129.13848 80.42848) (end 130.8536 82.1436) (width 0.25) (layer "B.Cu") (net 80))
@@
   (segment locked (start 120.5865 86.36) (end 118.79344 88.15306) (width 0.25) (layer "B.Cu") (net 98))
   (segment locked (start 118.4656 88.4809) (end 118.4656 99.2632) (width 0.25) (layer "B.Cu") (net 98))
+  (segment (start 121.92 86.36) (end 122.5804 86.36) (width 0.25) (layer "B.Cu") (net 98))
   (segment (start 123.8504 85.09) (end 126.1026 85.09) (width 0.25) (layer "B.Cu") (net 98))
   (segment (start 122.5804 86.36) (end 123.8504 85.09) (width 0.25) (layer "B.Cu") (net 98))
@@
   (segment (start 125.476 81.28) (end 126.8095 81.28) (width 0.25) (layer "B.Cu") (net 99))
   (segment locked (start 124.46 81.28) (end 125.476 81.28) (width 0.25) (layer "B.Cu") (net 99))
+  (segment (start 120.396 81.026) (end 120.65 81.28) (width 0.25) (layer "B.Cu") (net 100))
   (segment (start 121.92 81.28) (end 120.65 81.28) (width 0.25) (layer "B.Cu") (net 100))
   (segment (start 129.588 79.3595) (end 127.889 77.6605) (width 0.25) (layer "B.Cu") (net 101))
