File: Gardenuino V0.1f/nutrient V0.1f.kicad_sch (KiCad schematic)
At the start: 84 parts, among them J1 Conn_01x04_Female, J2 Conn_01x04_Female, J3 Conn_01x04_Female, J4 Conn_01x04_Female, J5 Conn_01x04_Female, J6 Conn_01x04_Female, J7 Conn_01x03_Male, J8 Conn_01x03_Male, P1 SolderJumper_2_Open, P2 SolderJumper_2_Bridged, P3 SolderJumper_2_Bridged, Q1 Q_NMOS_DGS, Q10 Q_NMOS_DGS, Q2 Q_NMOS_DGS, Q3 Q_NMOS_DGS, Q4 Q_NMOS_DGS, Q5 Q_NMOS_DGS, Q6 Q_NMOS_DGS, Q7 Q_NMOS_DGS, Q8 2N3904, U1 23LC512, U2 DS1307+, Y1 Crystal_Small

Commit message: SpectDrone development
Parts:
- J1, J3, J4, J6: value Conn_01x04_Female -> Conn_01x04_Male; footprint Connector_JST:JST_XH_B4B-XH-A_1x04_P2.50mm_Vertical -> Connector_PinHeader_2.54mm:PinHeader_1x04_P2.54mm_Vertical; symbol Connector:Conn_01x04_Female -> Connector:Conn_01x04_Male
- J2, J5: footprint Connector_JST:JST_XH_B4B-XH-A_1x04_P2.50mm_Vertical -> Connector_PinSocket_2.54mm:PinSocket_1x04_P2.54mm_Vertical
- JAUX1: footprint Connector_PinHeader_2.54mm:PinHeader_1x11_P2.54mm_Vertical -> Connector_PinSocket_2.54mm:PinSocket_1x11_P2.54mm_Vertical; symbol Connector:Conn_01x11_Male -> Connector:Conn_01x11_Female
Changed lines of the file:
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@@
     (pin "VIN2")
   )
-  (symbol (lib_id "Connector:Conn_01x04_Female") (at 124.46 36.83 180) (unit 1)
-    (in_bom yes) (on_board yes)
-    (property "Reference" "J1" (id 0) (at 121.92 33.02 0))
-    (property "Value" "Conn_01x04_Female" (id 1) (at 114.3 35.56 0)
-      (effects (font (size 1.27 1.27)) hide)
-    )
-    (property "Footprint" "Connector_JST:JST_XH_B4B-XH-A_1x04_P2.50mm_Vertical" (id 2) (at 124.46 36.83 0)
+  (symbol (lib_id "Connector:Conn_01x04_Male") (at 124.46 36.83 0) (mirror x) (unit 1)
+    (in_bom yes) (on_board yes)
+    (property "Reference" "J1" (id 0) (at 123.19 39.37 0))
+    (property "Value" "Conn_01x04_Male" (id 1) (at 134.62 35.56 0)
+      (effects (font (size 1.27 1.27)) hide)
+    )
+    (property "Footprint" "Connector_PinHeader_2.54mm:PinHeader_1x04_P2.54mm_Vertical" (id 2) (at 124.46 36.83 0)
       (effects (font (size 1.27 1.27)) hide)
     )
@@
   (symbol (lib_id "Connector:Conn_01x04_Female") (at 113.03 26.67 180) (unit 1)
     (in_bom yes) (on_board yes)
-    (property "Reference" "J2" (id 0) (at 110.49 22.86 0))
+    (property "Reference" "J2" (id 0) (at 111.76 29.21 0))
     (property "Value" "Conn_01x04_Female" (id 1) (at 102.87 25.4 0)
       (effects (font (size 1.27 1.27)) hide)
     )
-    (property "Footprint" "Connector_JST:JST_XH_B4B-XH-A_1x04_P2.50mm_Vertical" (id 2) (at 113.03 26.67 0)
+    (property "Footprint" "Connector_PinSocket_2.54mm:PinSocket_1x04_P2.54mm_Vertical" (id 2) (at 113.03 26.67 0)
       (effects (font (size 1.27 1.27)) hide)
     )
@@
     (pin "3")
   )
-  (symbol (lib_id "Connector:Conn_01x04_Female") (at 124.46 46.99 180) (unit 1)
-    (in_bom yes) (on_board yes)
-    (property "Reference" "J4" (id 0) (at 121.92 43.18 0))
-    (property "Value" "Conn_01x04_Female" (id 1) (at 114.3 45.72 0)
-      (effects (font (size 1.27 1.27)) hide)
-    )
-    (property "Footprint" "Connector_JST:JST_XH_B4B-XH-A_1x04_P2.50mm_Vertical" (id 2) (at 124.46 46.99 0)
+  (symbol (lib_id "Connector:Conn_01x04_Male") (at 124.46 46.99 0) (mirror x) (unit 1)
+    (in_bom yes) (on_board yes)
+    (property "Reference" "J4" (id 0) (at 123.19 49.53 0))
+    (property "Value" "Conn_01x04_Male" (id 1) (at 134.62 45.72 0)
+      (effects (font (size 1.27 1.27)) hide)
+    )
+    (property "Footprint" "Connector_PinHeader_2.54mm:PinHeader_1x04_P2.54mm_Vertical" (id 2) (at 124.46 46.99 0)
       (effects (font (size 1.27 1.27)) hide)
     )
@@
     (pin "4")
   )
-  (symbol (lib_id "Connector:Conn_01x04_Female") (at 124.46 57.15 180) (unit 1)
-    (in_bom yes) (on_board yes)
-    (property "Reference" "J3" (id 0) (at 121.92 53.34 0))
-    (property "Value" "Conn_01x04_Female" (id 1) (at 114.3 55.88 0)
-      (effects (font (size 1.27 1.27)) hide)
-    )
-    (property "Footprint" "Connector_JST:JST_XH_B4B-XH-A_1x04_P2.50mm_Vertical" (id 2) (at 124.46 57.15 0)
+  (symbol (lib_id "Connector:Conn_01x04_Male") (at 124.46 57.15 0) (mirror x) (unit 1)
+    (in_bom yes) (on_board yes)
+    (property "Reference" "J3" (id 0) (at 123.19 59.69 0))
+    (property "Value" "Conn_01x04_Male" (id 1) (at 134.62 55.88 0)
+      (effects (font (size 1.27 1.27)) hide)
+    )
+    (property "Footprint" "Connector_PinHeader_2.54mm:PinHeader_1x04_P2.54mm_Vertical" (id 2) (at 124.46 57.15 0)
       (effects (font (size 1.27 1.27)) hide)
     )
@@
     (pin "4")
   )
-  (symbol (lib_id "Connector:Conn_01x04_Female") (at 124.46 67.31 180) (unit 1)
-    (in_bom yes) (on_board yes)
-    (property "Reference" "J6" (id 0) (at 121.92 63.5 0))
-    (property "Value" "Conn_01x04_Female" (id 1) (at 114.3 66.04 0)
-      (effects (font (size 1.27 1.27)) hide)
-    )
-    (property "Footprint" "Connector_JST:JST_XH_B4B-XH-A_1x04_P2.50mm_Vertical" (id 2) (at 124.46 67.31 0)
+  (symbol (lib_id "Connector:Conn_01x04_Male") (at 124.46 67.31 0) (mirror x) (unit 1)
+    (in_bom yes) (on_board yes)
+    (property "Reference" "J6" (id 0) (at 123.19 69.85 0))
+    (property "Value" "Conn_01x04_Male" (id 1) (at 134.62 66.04 0)
+      (effects (font (size 1.27 1.27)) hide)
+    )
+    (property "Footprint" "Connector_PinHeader_2.54mm:PinHeader_1x04_P2.54mm_Vertical" (id 2) (at 124.46 67.31 0)
       (effects (font (size 1.27 1.27)) hide)
     )
@@
   (symbol (lib_id "Connector:Conn_01x04_Female") (at 212.09 59.69 0) (mirror x) (unit 1)
     (in_bom yes) (on_board yes)
-    (property "Reference" "J5" (id 0) (at 212.09 52.07 0))
+    (property "Reference" "J5" (id 0) (at 213.36 62.23 0))
     (property "Value" "Conn_01x04_Female" (id 1) (at 222.25 58.42 0)
       (effects (font (size 1.27 1.27)) hide)
     )
-    (property "Footprint" "Connector_JST:JST_XH_B4B-XH-A_1x04_P2.50mm_Vertical" (id 2) (at 212.09 59.69 0)
+    (property "Footprint" "Connector_PinSocket_2.54mm:PinSocket_1x04_P2.54mm_Vertical" (id 2) (at 212.09 59.69 0)
       (effects (font (size 1.27 1.27)) hide)
     )
@@
     (pin "3")
   )
-  (symbol (lib_id "Connector:Conn_01x11_Male") (at 283.21 152.4 0) (mirror y) (unit 1)
-    (in_bom yes) (on_board yes)
-    (property "Reference" "JAUX1" (id 0) (at 283.21 139.7 90)
-      (effects (font (size 1.27 1.27)) (justify left))
-    )
-    (property "Value" "GPS" (id 1) (at 280.67 138.43 90)
-      (effects (font (size 1.27 1.27)) (justify left))
-    )
-    (property "Footprint" "Connector_PinHeader_2.54mm:PinHeader_1x11_P2.54mm_Vertical" (id 2) (at 283.21 152.4 0)
+  (symbol (lib_id "Connector:Conn_01x11_Female") (at 283.21 152.4 0) (unit 1)
+    (in_bom yes) (on_board yes)
+    (property "Reference" "JAUX1" (id 0) (at 278.13 138.43 90)
+      (effects (font (size 1.27 1.27)) (justify left))
+    )
+    (property "Value" "GPS" (id 1) (at 280.67 137.16 90)
+      (effects (font (size 1.27 1.27)) (justify left))
+    )
+    (property "Footprint" "Connector_PinSocket_2.54mm:PinSocket_1x11_P2.54mm_Vertical" (id 2) (at 283.21 152.4 0)
       (effects (font (size 1.27 1.27)) hide)
     )
@@
     )
     (path "/00000000-0000-0000-0000-000060d781cb"
-      (reference "J1") (unit 1) (value "Conn_01x04_Female") (footprint "Connector_JST:JST_XH_B4B-XH-A_1x04_P2.50mm_Vertical")
+      (reference "J1") (unit 1) (value "Conn_01x04_Male") (footprint "Connector_PinHeader_2.54mm:PinHeader_1x04_P2.54mm_Vertical")
     )
     (path "/00000000-0000-0000-0000-000060d9b0d3"
-      (reference "J2") (unit 1) (value "Conn_01x04_Female") (footprint "Connector_JST:JST_XH_B4B-XH-A_1x04_P2.50mm_Vertical")
+      (reference "J2") (unit 1) (value "Conn_01x04_Female") (footprint "Connector_PinSocket_2.54mm:PinSocket_1x04_P2.54mm_Vertical")
     )
     (path "/00000000-0000-0000-0000-000060e4bcd3"
-      (reference "J3") (unit 1) (value "Conn_01x04_Female") (footprint "Connector_JST:JST_XH_B4B-XH-A_1x04_P2.50mm_Vertical")
+      (reference "J3") (unit 1) (value "Conn_01x04_Male") (footprint "Connector_PinHeader_2.54mm:PinHeader_1x04_P2.54mm_Vertical")
     )
     (path "/00000000-0000-0000-0000-000060e44026"
-      (reference "J4") (unit 1) (value "Conn_01x04_Female") (footprint "Connector_JST:JST_XH_B4B-XH-A_1x04_P2.50mm_Vertical")
+      (reference "J4") (unit 1) (value "Conn_01x04_Male") (footprint "Connector_PinHeader_2.54mm:PinHeader_1x04_P2.54mm_Vertical")
     )
     (path "/00000000-0000-0000-0000-000060e5c760"
-      (reference "J5") (unit 1) (value "Conn_01x04_Female") (footprint "Connector_JST:JST_XH_B4B-XH-A_1x04_P2.50mm_Vertical")
+      (reference "J5") (unit 1) (value "Conn_01x04_Female") (footprint "Connector_PinSocket_2.54mm:PinSocket_1x04_P2.54mm_Vertical")
     )
     (path "/00000000-0000-0000-0000-000060e52515"
-      (reference "J6") (unit 1) (value "Conn_01x04_Female") (footprint "Connector_JST:JST_XH_B4B-XH-A_1x04_P2.50mm_Vertical")
+      (reference "J6") (unit 1) (value "Conn_01x04_Male") (footprint "Connector_PinHeader_2.54mm:PinHeader_1x04_P2.54mm_Vertical")
     )
     (path "/00000000-0000-0000-0000-000061182723"
@@
     )
     (path "/00000000-0000-0000-0000-000062f67074"
-      (reference "JAUX1") (unit 1) (value "GPS") (footprint "Connector_PinHeader_2.54mm:PinHeader_1x11_P2.54mm_Vertical")
+      (reference "JAUX1") (unit 1) (value "GPS") (footprint "Connector_PinSocket_2.54mm:PinSocket_1x11_P2.54mm_Vertical")
     )
     (path "/00000000-0000-0000-0000-000062c0b2fe"

Commit message: SpectDrone development
Parts:
- added J9: Conn_01x02_Male, Connector_PinHeader_2.54mm:PinHeader_1x02_P2.54mm_Vertical, symbol Connector:Conn_01x02_Male
Connections:
- net GND: no longer JDC1.3
- net VIN1: now also J9.2 (Pin_2)
- new net: J9.1 (Pin_1), JDC1.3
Other:
- moved on the sheet: JDC1
Changed lines of the file:
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@@
   (junction (at 267.97 110.49) (diameter 0) (color 0 0 0 0)
   )
+  (junction (at 250.19 17.78) (diameter 0) (color 0 0 0 0)
+  )
   (junction (at 227.33 125.73) (diameter 0) (color 0 0 0 0)
   )
@@
   )
   (junction (at 68.58 115.57) (diameter 0) (color 0 0 0 0)
-  )
-  (junction (at 243.84 31.75) (diameter 0) (color 0 0 0 0)
   )
   (junction (at 83.82 113.03) (diameter 0) (color 0 0 0 0)
@@
     (stroke (width 0) (type default) (color 0 0 0 0))
   )
+  (wire (pts (xy 237.49 31.75) (xy 261.62 31.75))
+    (stroke (width 0) (type default) (color 0 0 0 0))
+  )
   (wire (pts (xy 104.14 157.48) (xy 134.62 157.48))
     (stroke (width 0) (type default) (color 0 0 0 0))
@@
     (stroke (width 0) (type default) (color 0 0 0 0))
   )
-  (wire (pts (xy 243.84 31.75) (xy 237.49 31.75))
-    (stroke (width 0) (type default) (color 0 0 0 0))
-  )
   (wire (pts (xy 273.05 139.7) (xy 278.13 139.7))
     (stroke (width 0) (type default) (color 0 0 0 0))
@@
     (stroke (width 0) (type default) (color 0 0 0 0))
   )
-  (wire (pts (xy 224.79 17.78) (xy 243.84 17.78))
+  (wire (pts (xy 224.79 17.78) (xy 250.19 17.78))
     (stroke (width 0) (type default) (color 0 0 0 0))
   )
@@
     (stroke (width 0) (type default) (color 0 0 0 0))
   )
-  (wire (pts (xy 243.84 17.78) (xy 243.84 26.67))
+  (wire (pts (xy 261.62 17.78) (xy 261.62 26.67))
     (stroke (width 0) (type default) (color 0 0 0 0))
   )
@@
     (stroke (width 0) (type default) (color 0 0 0 0))
   )
+  (wire (pts (xy 250.19 29.21) (xy 261.62 29.21))
+    (stroke (width 0) (type default) (color 0 0 0 0))
+  )
   (wire (pts (xy 146.685 154.305) (xy 146.685 155.575))
     (stroke (width 0) (type default) (color 0 0 0 0))
@@
     (stroke (width 0) (type default) (color 0 0 0 0))
   )
-  (wire (pts (xy 243.84 29.21) (xy 243.84 31.75))
-    (stroke (width 0) (type default) (color 0 0 0 0))
-  )
   (wire (pts (xy 241.3 115.57) (xy 241.3 116.84))
     (stroke (width 0) (type default) (color 0 0 0 0))
@@
     (stroke (width 0) (type default) (color 0 0 0 0))
   )
+  (wire (pts (xy 250.19 17.78) (xy 261.62 17.78))
+    (stroke (width 0) (type default) (color 0 0 0 0))
+  )
   (wire (pts (xy 134.62 133.35) (xy 138.43 133.35))
     (stroke (width 0) (type default) (color 0 0 0 0))
@@
     (stroke (width 0) (type default) (color 0 0 0 0))
   )
+  (wire (pts (xy 250.19 17.78) (xy 250.19 26.67))
+    (stroke (width 0) (type default) (color 0 0 0 0))
+  )
   (wire (pts (xy 168.91 142.24) (xy 168.91 144.78))
     (stroke (width 0) (type default) (color 0 0 0 0))
@@
     (effects (font (size 1.27 1.27)) (justify left bottom))
   )
-  (label "GND2" (at 243.84 31.75 180)
+  (label "GND2" (at 252.73 31.75 180)
     (effects (font (size 1.27 1.27)) (justify right bottom))
   )
@@
     (pin "2")
   )
-  (symbol (lib_id "Connector:Barrel_Jack_Switch") (at 251.46 29.21 0) (mirror y) (unit 1)
-    (in_bom yes) (on_board yes)
-    (property "Reference" "JDC1" (id 0) (at 257.302 27.94 0)
+  (symbol (lib_id "Connector:Barrel_Jack_Switch") (at 269.24 29.21 0) (mirror y) (unit 1)
+    (in_bom yes) (on_board yes)
+    (property "Reference" "JDC1" (id 0) (at 275.082 27.94 0)
       (effects (font (size 1.27 1.27)) (justify right))
     )
-    (property "Value" "Jack-DC" (id 1) (at 257.302 30.2514 0)
+    (property "Value" "Jack-DC" (id 1) (at 275.082 30.2514 0)
       (effects (font (size 1.27 1.27)) (justify right))
     )
-    (property "Footprint" "Connector_BarrelJack:BarrelJack_Horizontal" (id 2) (at 250.19 30.226 0)
-      (effects (font (size 1.27 1.27)) hide)
-    )
-    (property "Datasheet" "~" (id 3) (at 250.19 30.226 0)
+    (property "Footprint" "Connector_BarrelJack:BarrelJack_Horizontal" (id 2) (at 267.97 30.226 0)
+      (effects (font (size 1.27 1.27)) hide)
+    )
+    (property "Datasheet" "~" (id 3) (at 267.97 30.226 0)
       (effects (font (size 1.27 1.27)) hide)
     )
@@
     (pin "2")
   )
+  (symbol (lib_id "Connector:Conn_01x02_Male") (at 245.11 29.21 0) (mirror x) (unit 1)
+    (in_bom yes) (on_board yes)
+    (property "Reference" "J9" (id 0) (at 243.84 26.6699 0)
+      (effects (font (size 1.27 1.27)) (justify right))
+    )
+    (property "Value" "Conn_01x02_Male" (id 1) (at 243.84 29.2099 90)
+      (effects (font (size 1.27 1.27)) (justify right))
+    )
+    (property "Footprint" "Connector_PinHeader_2.54mm:PinHeader_1x02_P2.54mm_Vertical" (id 2) (at 245.11 29.21 0)
+      (effects (font (size 1.27 1.27)) hide)
+    )
+    (property "Datasheet" "~" (id 3) (at 245.11 29.21 0)
+      (effects (font (size 1.27 1.27)) hide)
+    )
+    (pin "1")
+    (pin "2")
+  )
   (symbol (lib_id "Device:R") (at 93.345 33.655 180) (unit 1)
     (in_bom yes) (on_board yes)
@@
       (reference "J8") (unit 1) (value "Conn_01x03_Male") (footprint "Connector_JST:JST_EH_S3B-EH_1x03_P2.50mm_Horizontal")
     )
+    (path "/6c1a8a3c-f787-40e4-8cd3-77048eeb28fc"
+      (reference "J9") (unit 1) (value "Conn_01x02_Male") (footprint "Connector_PinHeader_2.54mm:PinHeader_1x02_P2.54mm_Vertical")
+    )
     (path "/00000000-0000-0000-0000-000062f67074"

Commit message: SpectDrone Development
Connections:
- net GND: now also J9.1 (Pin_1), JDC1.3
Changed lines of the file:
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@@
   (junction (at 224.79 107.95) (diameter 0) (color 0 0 0 0)
   )
+  (junction (at 256.54 29.21) (diameter 0) (color 0 0 0 0)
+  )
   (junction (at 114.3 107.95) (diameter 0) (color 0 0 0 0)
   )
@@
   )
   (junction (at 242.57 123.19) (diameter 0) (color 0 0 0 0)
+  )
+  (junction (at 256.54 31.75) (diameter 0) (color 0 0 0 0)
   )
   (junction (at 257.81 130.81) (diameter 0) (color 0 0 0 0)
@@
     (stroke (width 0) (type default) (color 0 0 0 0))
   )
+  (wire (pts (xy 256.54 29.21) (xy 256.54 31.75))
+    (stroke (width 0) (type default) (color 0 0 0 0))
+  )
   (wire (pts (xy 273.05 160.02) (xy 278.13 160.02))
     (stroke (width 0) (type default) (color 0 0 0 0))
@@
     (stroke (width 0) (type default) (color 0 0 0 0))
   )
-  (wire (pts (xy 237.49 31.75) (xy 261.62 31.75))
+  (wire (pts (xy 237.49 31.75) (xy 256.54 31.75))
     (stroke (width 0) (type default) (color 0 0 0 0))
   )
@@
     (stroke (width 0) (type default) (color 0 0 0 0))
   )
-  (wire (pts (xy 250.19 29.21) (xy 261.62 29.21))
+  (wire (pts (xy 250.19 29.21) (xy 256.54 29.21))
     (stroke (width 0) (type default) (color 0 0 0 0))
   )
@@
     (stroke (width 0) (type default) (color 0 0 0 0))
   )
+  (wire (pts (xy 256.54 31.75) (xy 261.62 31.75))
+    (stroke (width 0) (type default) (color 0 0 0 0))
+  )
   (wire (pts (xy 222.25 59.69) (xy 222.25 69.85))
     (stroke (width 0) (type default) (color 0 0 0 0))
@@
   )
   (wire (pts (xy 137.16 41.91) (xy 129.54 41.91))
+    (stroke (width 0) (type default) (color 0 0 0 0))
+  )
+  (wire (pts (xy 256.54 29.21) (xy 261.62 29.21))
     (stroke (width 0) (type default) (color 0 0 0 0))
   )
@@
     )
     (property "Value" "Conn_01x02_Male" (id 1) (at 243.84 29.2099 90)
-      (effects (font (size 1.27 1.27)) (justify right))
+      (effects (font (size 1.27 1.27)) (justify right) hide)
     )
     (property "Footprint" "Connector_PinHeader_2.54mm:PinHeader_1x02_P2.54mm_Vertical" (id 2) (at 245.11 29.21 0)

Commit message: SpectDrone Development
Parts:
- J9: value Conn_01x02_Male -> Conn_01x01_Male; footprint Connector_PinHeader_2.54mm:PinHeader_1x02_P2.54mm_Vertical -> Connector_PinHeader_2.54mm:PinHeader_1x01_P2.54mm_Vertical; symbol Connector:Conn_01x02_Male -> Connector:Conn_01x01_Male
Connections:
- net GND: no longer J9.1 (Pin_1)
- net VIN1: now also J9.1 (Pin_1); no longer J9.2 (Pin_2)
Changed lines of the file:
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@@
   (junction (at 224.79 107.95) (diameter 0) (color 0 0 0 0)
   )
-  (junction (at 256.54 29.21) (diameter 0) (color 0 0 0 0)
-  )
   (junction (at 114.3 107.95) (diameter 0) (color 0 0 0 0)
   )
@@
     (stroke (width 0) (type default) (color 0 0 0 0))
   )
-  (wire (pts (xy 250.19 29.21) (xy 256.54 29.21))
-    (stroke (width 0) (type default) (color 0 0 0 0))
-  )
   (wire (pts (xy 146.685 154.305) (xy 146.685 155.575))
     (stroke (width 0) (type default) (color 0 0 0 0))
@@
     (stroke (width 0) (type default) (color 0 0 0 0))
   )
-  (wire (pts (xy 250.19 17.78) (xy 250.19 26.67))
+  (wire (pts (xy 250.19 17.78) (xy 250.19 21.59))
     (stroke (width 0) (type default) (color 0 0 0 0))
   )
@@
     (pin "2")
   )
-  (symbol (lib_id "Connector:Conn_01x02_Male") (at 245.11 29.21 0) (mirror x) (unit 1)
+  (symbol (lib_id "Connector:Conn_01x01_Male") (at 250.19 26.67 270) (mirror x) (unit 1)
     (in_bom yes) (on_board yes)
-    (property "Reference" "J9" (id 0) (at 243.84 26.6699 0)
+    (property "Reference" "J9" (id 0) (at 247.6499 27.94 0)
       (effects (font (size 1.27 1.27)) (justify right))
     )
-    (property "Value" "Conn_01x02_Male" (id 1) (at 243.84 29.2099 90)
+    (property "Value" "Conn_01x01_Male" (id 1) (at 250.1899 27.94 90)
       (effects (font (size 1.27 1.27)) (justify right) hide)
     )
-    (property "Footprint" "Connector_PinHeader_2.54mm:PinHeader_1x02_P2.54mm_Vertical" (id 2) (at 245.11 29.21 0)
+    (property "Footprint" "Connector_PinHeader_2.54mm:PinHeader_1x01_P2.54mm_Vertical" (id 2) (at 250.19 26.67 0)
       (effects (font (size 1.27 1.27)) hide)
     )
-    (property "Datasheet" "~" (id 3) (at 245.11 29.21 0)
+    (property "Datasheet" "~" (id 3) (at 250.19 26.67 0)
       (effects (font (size 1.27 1.27)) hide)
     )
     (pin "1")
-    (pin "2")
   )
   (symbol (lib_id "Device:R") (at 93.345 33.655 180) (unit 1)
@@
     )
     (path "/6c1a8a3c-f787-40e4-8cd3-77048eeb28fc"
-      (reference "J9") (unit 1) (value "Conn_01x02_Male") (footprint "Connector_PinHeader_2.54mm:PinHeader_1x02_P2.54mm_Vertical")
+      (reference "J9") (unit 1) (value "Conn_01x01_Male") (footprint "Connector_PinHeader_2.54mm:PinHeader_1x01_P2.54mm_Vertical")
     )
     (path "/00000000-0000-0000-0000-000062f67074"

Commit message: SpectDrone Development
Other:
- moved on the sheet: P3
Changed lines of the file:
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@@
   (junction (at 222.25 102.87) (diameter 0) (color 0 0 0 0)
   )
+  (junction (at 210.82 118.11) (diameter 0) (color 0 0 0 0)
+  )
   (junction (at 134.62 133.35) (diameter 0) (color 0 0 0 0)
   )
@@
   )
   (junction (at 129.54 105.41) (diameter 0) (color 0 0 0 0)
-  )
-  (junction (at 206.375 118.11) (diameter 0) (color 0 0 0 0)
   )
   (junction (at 100.33 85.09) (diameter 0) (color 0 0 0 0)
@@
     (stroke (width 0) (type default) (color 0 0 0 0))
   )
-  (wire (pts (xy 206.375 112.395) (xy 211.455 112.395))
-    (stroke (width 0) (type default) (color 0 0 0 0))
-  )
   (wire (pts (xy 238.76 67.31) (xy 229.87 67.31))
     (stroke (width 0) (type default) (color 0 0 0 0))
@@
     (stroke (width 0) (type default) (color 0 0 0 0))
   )
+  (wire (pts (xy 210.82 118.11) (xy 213.36 118.11))
+    (stroke (width 0) (type default) (color 0 0 0 0))
+  )
   (wire (pts (xy 43.18 118.11) (xy 43.18 142.24))
     (stroke (width 0) (type default) (color 0 0 0 0))
   )
-  (wire (pts (xy 206.375 118.11) (xy 210.185 118.11))
-    (stroke (width 0) (type default) (color 0 0 0 0))
-  )
   (wire (pts (xy 176.53 139.7) (xy 176.53 137.16))
     (stroke (width 0) (type default) (color 0 0 0 0))
@@
     (stroke (width 0) (type default) (color 0 0 0 0))
   )
-  (wire (pts (xy 203.2 118.11) (xy 206.375 118.11))
+  (wire (pts (xy 203.2 118.11) (xy 210.82 118.11))
     (stroke (width 0) (type default) (color 0 0 0 0))
   )
@@
     (stroke (width 0) (type default) (color 0 0 0 0))
   )
-  (wire (pts (xy 206.375 118.11) (xy 206.375 112.395))
+  (wire (pts (xy 210.82 109.22) (xy 210.82 118.11))
     (stroke (width 0) (type default) (color 0 0 0 0))
   )
@@
     (stroke (width 0) (type default) (color 0 0 0 0))
   )
+  (wire (pts (xy 218.44 111.76) (xy 218.44 109.22))
+    (stroke (width 0) (type default) (color 0 0 0 0))
+  )
   (wire (pts (xy 265.43 125.73) (xy 266.7 125.73))
     (stroke (width 0) (type default) (color 0 0 0 0))
@@
     (effects (font (size 1.27 1.27)) (justify right bottom))
   )
-  (label "PPS" (at 219.075 112.395 0)
-    (effects (font (size 1.27 1.27)) (justify left bottom))
+  (label "PPS" (at 218.44 111.76 270)
+    (effects (font (size 1.27 1.27)) (justify right bottom))
   )
   (label "D13" (at 133.35 97.79 180)
@@
     (effects (font (size 1.27 1.27)) (justify right bottom))
   )
-  (label "INT" (at 210.185 118.11 0)
+  (label "INT" (at 213.36 118.11 0)
     (effects (font (size 1.27 1.27)) (justify left bottom))
   )
@@
     (pin "2")
   )
-  (symbol (lib_id "Jumper:SolderJumper_2_Bridged") (at 215.265 112.395 0) (unit 1)
-    (in_bom yes) (on_board yes)
-    (property "Reference" "P3" (id 0) (at 210.185 121.285 90))
-    (property "Value" "SolderJumper_2_Bridged" (id 1) (at 215.9 109.855 0))
-    (property "Footprint" "Library:SolderJumper-2_P1.3mm_Bridged2Bar_RoundedPad1.0x1.5mm_narrow" (id 2) (at 215.265 112.395 0)
-      (effects (font (size 1.27 1.27)) hide)
-    )
-    (property "Datasheet" "~" (id 3) (at 215.265 112.395 0)
-      (effects (font (size 1.27 1.27)) hide)
-    )
+  (symbol (lib_id "Jumper:SolderJumper_2_Bridged") (at 214.63 109.22 0) (unit 1)
+    (in_bom yes) (on_board yes)
+    (property "Reference" "P3" (id 0) (at 213.995 111.125 0))
+    (property "Value" "SolderJumper_2_Bridged" (id 1) (at 215.265 106.68 0)
+      (effects (font (size 1.27 1.27)) hide)
+    )
+    (property "Footprint" "Library:SolderJumper-2_P1.3mm_Bridged2Bar_RoundedPad1.0x1.5mm_narrow" (id 2) (at 214.63 109.22 0)
+      (effects (font (size 1.27 1.27)) hide)
+    )
+    (property "Datasheet" "~" (id 3) (at 214.63 109.22 0)
+      (effects (font (size 1.27 1.27)) hide)
+    )
