File: Gardenuino V0.1f/nutrient V0.1f.kicad_sch (KiCad schematic)
At the start: 85 parts, among them J1 Conn_01x04_Male, J2 Conn_01x04_Female, J3 Conn_01x04_Male, J4 Conn_01x04_Male, J5 Conn_01x04_Female, J6 Conn_01x04_Male, J7 Conn_01x03_Male, J8 Conn_01x03_Male, J9 Conn_01x01_Male, P1 SolderJumper_2_Open, P2 SolderJumper_2_Bridged, P3 SolderJumper_2_Bridged, Q1 Q_NMOS_DGS, Q10 Q_NMOS_DGS, Q2 Q_NMOS_DGS, Q3 Q_NMOS_DGS, Q4 Q_NMOS_DGS, Q5 Q_NMOS_DGS, Q6 Q_NMOS_DGS, Q7 Q_NMOS_DGS, Q8 2N3904, U1 23LC512, U2 DS1307+, Y1 Crystal_Small

Commit message: SpectDrone Development
Parts:
- removed JP5: SolderJumper_3_Bridged12, Jumper:SolderJumper-3_P1.3mm_Bridged2Bar12_RoundedPad1.0x1.5mm, symbol Jumper:SolderJumper_3_Bridged12
- added J10: Conn_01x01_Male, Connector_PinHeader_2.54mm:PinHeader_1x01_P2.54mm_Vertical, symbol Connector:Conn_01x01_Male
- JAUX1: footprint Connector_PinSocket_2.54mm:PinSocket_1x11_P2.54mm_Vertical -> Connector_PinSocket_2.54mm:PinSocket_1x12_P2.54mm_Vertical; symbol Connector:Conn_01x11_Female -> Connector:Conn_01x12_Female
Connections:
- net D16 is gone; now on net GPSTX: XA1.D16 (D16_TX2)
- net XCL is gone; now on net AUX_INT: JAUX1.8 (Pin_8)
- net D12: now also JAUX1.12 (Pin_12); no longer JAUX1.11 (Pin_11)
- net GPSTX: no longer XA1.D19 (D19_RX1_INT2)
- net OPT_EXT: now also JAUX1.11 (Pin_11); no longer JAUX1.10 (Pin_10)
- net TX: now also JAUX1.10 (Pin_10); no longer JAUX1.9 (Pin_9)
- net at XA1.3V2 (3.3V): now also J10.1 (Pin_1)
- net INT renamed AUX_INT
- net AUX_INT: no longer P3.1 (A)
- new net D19: JAUX1.9 (Pin_9), P3.1 (A), XA1.D19 (D19_RX1_INT2)
- no-connect marks 16 -> 15
Other:
- moved on the sheet: P1, P2

Commit message: SpectDrone Development
Parts:
- added P4: SolderJumper_2_Bridged, Jumper:SolderJumper-2_P1.3mm_Bridged2Bar_RoundedPad1.0x1.5mm, symbol Jumper:SolderJumper_2_Bridged
Connections:
- net D19: now also P4.1 (A); no longer JAUX1.9 (Pin_9)
- new net: JAUX1.9 (Pin_9), P4.2 (B)
Changed lines of the file:
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@@
     (effects (font (size 1.27 1.27)) (justify right bottom))
   )
-  (label "D19" (at 273.05 160.02 180)
+  (label "D19" (at 265.43 160.02 180)
     (effects (font (size 1.27 1.27)) (justify right bottom))
   )
@@
     (pin "2")
   )
+  (symbol (lib_id "Jumper:SolderJumper_2_Bridged") (at 269.24 160.02 0) (unit 1)
+    (in_bom yes) (on_board yes)
+    (property "Reference" "P4" (id 0) (at 264.16 168.91 90))
+    (property "Value" "SolderJumper_2_Bridged" (id 1) (at 261.62 165.1 90))
+    (property "Footprint" "Jumper:SolderJumper-2_P1.3mm_Bridged2Bar_RoundedPad1.0x1.5mm" (id 2) (at 269.24 160.02 0)
+      (effects (font (size 1.27 1.27)) hide)
+    )
+    (property "Datasheet" "~" (id 3) (at 269.24 160.02 0)
+      (effects (font (size 1.27 1.27)) hide)
+    )
+    (pin "1")
+    (pin "2")
+  )
   (symbol (lib_id "Connector:Conn_01x01_Male") (at 36.83 90.805 0) (unit 1)
     (in_bom yes) (on_board yes)
@@
       (reference "P3") (unit 1) (value "SolderJumper_2_Bridged") (footprint "Library:SolderJumper-2_P1.3mm_Bridged2Bar_RoundedPad1.0x1.5mm_narrow")
     )
+    (path "/7e9e8112-44fc-4216-ac01-88d07c366d80"
+      (reference "P4") (unit 1) (value "SolderJumper_2_Bridged") (footprint "Jumper:SolderJumper-2_P1.3mm_Bridged2Bar_RoundedPad1.0x1.5mm")
+    )
     (path "/00000000-0000-0000-0000-000060deff9c"
