File: Gardenuino V0.1f/nutrient V0.1f.kicad_sch (KiCad schematic)
At the start: 86 parts, among them J1 Conn_01x04_Male, J10 Conn_01x01_Male, J2 Conn_01x04_Female, J3 Conn_01x04_Male, J4 Conn_01x04_Male, J5 Conn_01x04_Female, J6 Conn_01x04_Male, J7 Conn_01x03_Male, J8 Conn_01x03_Male, J9 Conn_01x01_Male, P1 SolderJumper_2_Open, P2 SolderJumper_2_Bridged, P3 SolderJumper_2_Bridged, P4 SolderJumper_2_Bridged, Q1 Q_NMOS_DGS, Q10 Q_NMOS_DGS, Q2 Q_NMOS_DGS, Q3 Q_NMOS_DGS, Q4 Q_NMOS_DGS, Q5 Q_NMOS_DGS, Q6 Q_NMOS_DGS, Q7 Q_NMOS_DGS, Q8 2N3904, U1 23LC512, U2 DS1307+, Y1 Crystal_Small

Commit message: SpectDrone Development
Parts:
- removed P1: SolderJumper_2_Open, Jumper:SolderJumper-2_P1.3mm_Open_RoundedPad1.0x1.5mm, symbol Jumper:SolderJumper_2_Open
- added P1: SolderJumper_2_Bridged, Jumper:SolderJumper-2_P1.3mm_Bridged2Bar_RoundedPad1.0x1.5mm, symbol Jumper:SolderJumper_2_Bridged
- J3, J6: value Conn_01x04_Male -> Conn_01x04_Female; footprint Connector_PinHeader_2.54mm:PinHeader_1x04_P2.54mm_Vertical -> Connector_PinSocket_2.54mm:PinSocket_1x04_P2.54mm_Vertical; symbol Connector:Conn_01x04_Male -> Connector:Conn_01x04_Female
Connections:
- net D13: now also JP6.3 (B); no longer JP6.1 (A)
- net GPSRX: now also XA1.D16 (D16_TX2); no longer XA1.D17 (D17_RX2)
- net GPSTX: now also XA1.D17 (D17_RX2); no longer XA1.D16 (D16_TX2)
- net OPT: now also P1.1 (A)
- net RX: now also JP6.1 (A); no longer JP6.3 (B), XA1.D15 (D15_RX3)
- net RX1_OPT: now reaches JAUX1.9 (Pin_9), P4.2 (B)
- net AUX_INT renamed TX1
- net D19 renamed RX1
- net INT0 renamed INT4
- net INT1 renamed INT5
- net OPT_EXT renamed RX3_OPT
- net RX3_OPT: now also P1.2 (B)
- net TX renamed TX3
- new net RX3: XA1.D15 (D15_RX3)
Other:
- moved on the sheet: JGPS1, P2, P4

Commit message: SpectDrone development
Connections:
- net VIN renamed AREF
Changed lines of the file:
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@@
     (effects (font (size 1.27 1.27)) (justify left bottom))
   )
-  (label "VIN" (at 72.39 80.01 180)
+  (label "AREF" (at 72.39 80.01 180)
     (effects (font (size 1.27 1.27)) (justify right bottom))
   )
@@
   (label "TX3" (at 203.2 107.95 0)
     (effects (font (size 1.27 1.27)) (justify left bottom))
+  )
+  (label "AREF" (at 203.2 41.91 180)
+    (effects (font (size 1.27 1.27)) (justify right bottom))
   )
   (label "RX2" (at 203.2 115.57 0)
@@
     (effects (font (size 1.27 1.27)) (justify left bottom))
   )
-  (label "VIN" (at 203.2 41.91 0)
-    (effects (font (size 1.27 1.27)) (justify left bottom))
-  )

Commit message: SpectDrone development
Parts:
- J2: value Conn_01x04_Female -> Conn_01x04_Male; footprint Connector_PinSocket_2.54mm:PinSocket_1x04_P2.54mm_Vertical -> Connector_PinHeader_2.54mm:PinHeader_1x04_P2.54mm_Vertical; symbol Connector:Conn_01x04_Female -> Connector:Conn_01x04_Male
- J4: footprint Connector_PinHeader_2.54mm:PinHeader_1x04_P2.54mm_Vertical -> Connector_PinSocket_2.54mm:PinSocket_1x04_P2.54mm_Vertical; symbol Connector:Conn_01x04_Male -> Connector:Conn_01x04_Female
- P3: symbol Jumper:SolderJumper_2_Bridged -> Jumper:SolderJumper_2_Open
Connections:
- net RX is gone; now on net RX3: JP6.1 (A)
Other:
- moved on the sheet: JAUX1, JSPI1, P1, P2, P4, Q8, R3

Commit message: SpectDrone Development
Changed lines of the file:
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@@
+    (stroke (width 0) (type default) (color 0 0 0 0))
+  )
+  (wire (pts (xy 26.67 163.83) (xy 26.67 165.1))
     (stroke (width 0) (type default) (color 0 0 0 0))
   )
@@
     (effects (font (size 1.27 1.27)) (justify left bottom))
   )
-  (label "RX1" (at 26.67 165.1 90)
+  (label "RX1" (at 26.67 163.83 0)
     (effects (font (size 1.27 1.27)) (justify left bottom))
   )

Commit message: SpectDrone Development
Connections:
- net D52: now also JAUX1.4 (Pin_4)
- net SS_AUX: no longer JAUX1.4 (Pin_4)
Changed lines of the file:
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@@
     (effects (font (size 1.27 1.27)) (justify left bottom))
   )
-  (label "SS_AUX" (at 39.37 180.34 90)
+  (label "SCK" (at 39.37 180.34 90)
     (effects (font (size 1.27 1.27)) (justify left bottom))
   )

Commit message: SpectDrone Development
Other:
- moved on the sheet: C2, C6, J9
