File: SpectDrone2/SpectDrone2/SpectDrone2.kicad_sch (KiCad schematic)
At the start: 11 parts

Commit message: SpectDrone Development
Parts:
- added PD? (x2): S1336-18BK, Package_TO_SOT_THT:TO-18-4_Lens, symbol Sensor_Optical:S13360-3025CS
- added R? (x2): 4K0, Resistor_SMD:R_0603_1608Metric_Pad0.98x0.95mm_HandSolder, symbol Device:R
- added R? (x2): 1K0, Resistor_SMD:R_0603_1608Metric_Pad0.98x0.95mm_HandSolder, symbol Device:R
- added U? (x2): MIC863, Package_TO_SOT_SMD:SOT-23-8, symbol Amplifier_Operational:AD8620
Connections:
- net GND1: now also R?.2, R?.2
- new net 1.0V: PD?.2 (K), PD?.3 (K), U?.3 (+), U?.5 (+)
- new net S1: R?.2, U?.7
- new net S2: R?.1, U?.1
- new net SIG1: PD?.1 (A), R?.1, R?.1, U?.6 (-)
- new net SIG2: PD?.1 (A), R?.1, R?.2, U?.2 (-)
