File: Longwave Instrument/Longwave Instrument.kicad_sch (KiCad schematic)
At the start: 18 parts

Commit message: SpectDrone Development
Connections:
- net 1.0V renamed 1.0V1
- net 1.0V1: no longer CS6.1, CS8.1, PD2.2 (K), US2.4 (+)
- new net 1.0V2: CS6.1, CS8.1, PD2.2 (K), US2.4 (+)
Changed lines of the file:
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@@
     )
   )
-  (global_label "1.0V" (shape input) (at 124.46 67.31 180) (fields_autoplaced)
+  (global_label "1.0V1" (shape input) (at 124.46 67.31 180) (fields_autoplaced)
     (effects (font (size 1.27 1.27)) (justify right))
-    (property "Intersheet References" "${INTERSHEET_REFS}" (id 0) (at 117.9345 67.2306 0)
+    (property "Intersheet References" "${INTERSHEET_REFS}" (id 0) (at 116.725 67.2306 0)
       (effects (font (size 1.27 1.27)) (justify right) hide)
     )
@@
     )
   )
-  (global_label "1.0V" (shape input) (at 124.46 102.87 180) (fields_autoplaced)
+  (global_label "1.0V2" (shape input) (at 124.46 102.87 180) (fields_autoplaced)
     (effects (font (size 1.27 1.27)) (justify right))
-    (property "Intersheet References" "${INTERSHEET_REFS}" (id 0) (at 117.9345 102.7906 0)
+    (property "Intersheet References" "${INTERSHEET_REFS}" (id 0) (at 116.725 102.7906 0)
       (effects (font (size 1.27 1.27)) (justify right) hide)
     )

Commit message: SpectDrone Development
Parts:
- added JPV1: SolderJumper_2_Bridged, Jumper:SolderJumper-2_P1.3mm_Bridged_RoundedPad1.0x1.5mm, symbol Jumper:SolderJumper_2_Bridged
- added JPV2: SolderJumper_2_Open, Jumper:SolderJumper-2_P1.3mm_Open_RoundedPad1.0x1.5mm, symbol Jumper:SolderJumper_2_Open
- added R10, R9: 470K, Capacitor_SMD:C_0805_2012Metric, symbol Device:R
- added R4, R5: 402, Capacitor_SMD:C_0805_2012Metric, symbol Device:R
- added RS? (x2): 1K0, Capacitor_SMD:C_0805_2012Metric, symbol Device:R
- added RS? (x2): 4K02, Capacitor_SMD:C_0805_2012Metric, symbol Device:R
- added RV1, RV2: R_Potentiometer, Potentiometer_THT:Potentiometer_Bourns_3296W_Vertical, symbol Device:R_Potentiometer
- added TPv1-1, TPv1-2: TestPoint, TestPoint:TestPoint_Keystone_5000-5004_Miniature, symbol Connector:TestPoint
- added U8, U9: ADR510, Package_TO_SOT_SMD:SOT-23, symbol Reference_Voltage:CJ432
- CS1, CS6: value 10nF -> 17.4pF
- CS2, CS7: value 1nF -> 1.74pF
- CS3, CS8: value 1nF -> 1.7pF
- RS1: value 1K0 -> 833
- RS4: renamed from RS3; value 1K0 -> 833
- renumbered RS4 to RS5
Connections:
- net 1.0V1: now also JPV1.2 (B), R4.2, RS?.1, RV1.1, TPv1-1.1, U8.2 (K); no longer CS1.1, CS3.1, US1.4 (+)
- net 1.0V2: now also JPV1.1 (A), JPV2.2 (B), RS?.1; no longer CS6.1, CS8.1, US2.4 (+)
- net 5V3: now also R4.1, R5.1
- net GND1: now also RV1.3, RV2.3, U8.3 (A), U9.3 (A)
- net at CS6.2, CS7.1, US2.1 (-): now also RS?.2; no longer PD2.1 (A), RS4.1
- net at CS1.2, CS2.1, US1.1 (-): now also RS?.2; no longer PD1.1 (A), RS1.1
- new net: CS6.1, CS8.1, RS?.2, US2.4 (+)
- new net: CS1.1, CS3.1, RS?.2, US1.4 (+)
- new net: R9.1, U8.1 (REF)
- new net: R9.2, RV1.2
- new net: R10.1, U9.1 (REF)
- new net: R10.2, RV2.2
- new net 1V2: JPV2.1 (A), R5.2, RV2.1, TPv1-2.1, U9.2 (K)
- new net INV1: PD2.1 (A), RS4.1, RS?.1
- new net INV2: PD1.1 (A), RS1.1, RS?.1
Other:
- note added: "AD8221: V(lux)_{PD} = 1.0 v - ( I_{PD} * RS1 ) I_{PD} = 1.2 mA RS1 = 833 ohm V = 1.2 mA * 833 ohm = 1 V"
- note added: "ADR510: I_{Q_min} = 0.1 mA I_{L_max (1PD)} = 1.2 mA I_{L_max (2PD)} = 2.4 mA I_{Q_max} = 10.0 mA I_{L_min} = 2.4 pA = 2.4e-9 mA I_{min_1} = 1.3 mA I_{min_2} = 2.5 mA I_{max} = 10.0 mA V_{S} = 5 v V_{out} = 1 v V = 5 v - 1 v = 4 v R_{BIAS}(I_{L_min (1PD)}) = 4 v / 1.3 mA = 3.3 Kohm R_{BIAS}(I_{L_min (2PD)}) = 4 v / 2.5 mA = 1600 ohm R_{BIAS}(I_{L_max}) = 4 v / 10.0 mA = 400 ohm R_{BIAS} = 402 ohm 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"
- note added: "GRM0225C1E180GA02L 18pF GRM0225C1E181JA02L 180pF FF_{Diff} = ( 2 * pi * R * ( 2 * C_{d} + C_{c} ) )^{ -1} R = 484 ohm C_{d} = 180pF C_{c} = 18pF FF_{Diff} = 434.964 MHz FF_{CM} = ( 2 * pi * R * C_{c} )^{ -1} R = 484 ohm C_{c} = 18pF FF_{CM} = 9.13e6 Hz"
- note added: "Photodiode (~320nm - 1100nm) Dark Current: I_{R}(1V) = 18~22 pA I_{sc}(lx)_{uA} = (1.0 / 100) (uA / lx) Estimated 128Klux Maximum 1280 uA = 128000 lx 1280 uA = 1.2 mA per PD 1 PD = 1.2 mA V = 1.2 mA * R ohm = 1.0 V R_{S1&S4} = 833 ohm 2 PD = 2.4 mA V = 2.4 mA * R ohm = 1.0 V R_{S1|S4} = 417 ohm"
- moved on the sheet: CS1, CS10, CS2, CS3, CS4, CS5, CS6, CS7, CS8, CS9, PD1, PD2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

Commit message: SpectDrone Development
Parts:
- CS1, CS6: value 17.4pF -> 11.1pF
- CS2, CS7: value 1.74pF -> 1.11pF
- CS3, CS8: value 1.7pF -> 1.11pF
- RS1, RS4: value 833 -> 845
- RS3, RS6: renamed from RS?; value 1K0 -> 330
- RS7, RS8: renamed from RS?; value 4K02 -> 330
- RV1, RV2: value R_Potentiometer -> 10K
Connections:
- net INV1: now also PD1.1 (A), RS1.1, RS6.1; no longer PD2.1 (A), RS4.1, RS8.1
- net INV2: now also PD2.1 (A), RS4.1, RS8.1; no longer PD1.1 (A), RS1.1, RS6.1
Other:
- note added: "C_{c} = 02011JR35ZBSTR 1.11pF C_{d} = 04023J3R6BBSTR 11.1pF FF_{Diff} = ( 2 * pi * R * ( 2 * C_{d} + C_{c} ) )^{ -1} R = 330 ohm C_{d} = 11.1pF C_{c} = 1.11pF FF_{Diff} = 20.69 MHz FF_{CM} = ( 2 * pi * R * C_{c} )^{ -1} R = 330 ohm C_{c} = 1.11pF FF_{CM} = 434.5 MHz"
- note added: "Photodiode (~320nm - 1100nm) Dark Current: I_{R}(1V) = 18~22 pA I_{sc}(lx)_{uA} = (1.0 / 100) (uA / lx) Estimated 128Klux Maximum I_{sc}(128Klux)_{uA} 1280 uA = 128000 lx 1280 uA = 1.2 mA per PD 1 PD = 1.2 mA V = 1.2 mA * R ohm = 1.0 V R_{S1&S4} = 833 ohm -> 845 ohm 2 PD = 2.4 mA V = 2.4 mA * R ohm = 1.0 V R_{S1|S4} = 417 ohm"
- note removed: "GRM0225C1E180GA02L 18pF GRM0225C1E181JA02L 180pF FF_{Diff} = ( 2 * pi * R * ( 2 * C_{d} + C_{c} ) )^{ -1} R = 484 ohm C_{d} = 180pF C_{c} = 18pF FF_{Diff} = 434.964 MHz FF_{CM} = ( 2 * pi * R * C_{c} )^{ -1} R = 484 ohm C_{c} = 18pF FF_{CM} = 9.13e6 Hz"
- note removed: "Photodiode (~320nm - 1100nm) Dark Current: I_{R}(1V) = 18~22 pA I_{sc}(lx)_{uA} = (1.0 / 100) (uA / lx) Estimated 128Klux Maximum 1280 uA = 128000 lx 1280 uA = 1.2 mA per PD 1 PD = 1.2 mA V = 1.2 mA * R ohm = 1.0 V R_{S1&S4} = 833 ohm 2 PD = 2.4 mA V = 2.4 mA * R ohm = 1.0 V R_{S1|S4} = 417 ohm"
Changed lines of the file:
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@@
-    (stroke (width 0) (type default) (color 0 0 0 0))
-  )
-  (polyline (pts (xy 67.31 154.94) (xy 67.31 179.705))
     (stroke (width 0) (type default) (color 0 0 0 0))
   )
@@
     (stroke (width 0) (type default) (color 0 0 0 0))
   )
+  (polyline (pts (xy 67.31 185.42) (xy 13.97 185.42))
+    (stroke (width 0) (type default) (color 0 0 0 0))
+  )
   (wire (pts (xy 109.22 110.49) (xy 110.49 110.49))
     (stroke (width 0) (type default) (color 0 0 0 0))
@@
     (stroke (width 0) (type default) (color 0 0 0 0))
   )
-  (polyline (pts (xy 13.97 154.94) (xy 67.31 154.94))
-    (stroke (width 0) (type default) (color 0 0 0 0))
-  )
   (wire (pts (xy 161.29 80.01) (xy 161.29 81.28))
     (stroke (width 0) (type default) (color 0 0 0 0))
@@
     (stroke (width 0) (type default) (color 0 0 0 0))
   )
+  (polyline (pts (xy 67.31 154.305) (xy 67.31 185.42))
+    (stroke (width 0) (type default) (color 0 0 0 0))
+  )
   (wire (pts (xy 106.68 114.3) (xy 123.19 114.3))
     (stroke (width 0) (type default) (color 0 0 0 0))
@@
     (stroke (width 0) (type default) (color 0 0 0 0))
   )
+  (polyline (pts (xy 13.97 154.305) (xy 67.31 154.305))
+    (stroke (width 0) (type default) (color 0 0 0 0))
+  )
   (wire (pts (xy 161.29 71.12) (xy 161.29 72.39))
     (stroke (width 0) (type default) (color 0 0 0 0))
@@
     (stroke (width 0) (type default) (color 0 0 0 0))
   )
-  (polyline (pts (xy 67.31 179.705) (xy 13.97 179.705))
-    (stroke (width 0) (type default) (color 0 0 0 0))
-  )
   (wire (pts (xy 161.29 71.12) (xy 163.83 71.12))
     (stroke (width 0) (type default) (color 0 0 0 0))
   )
+  (polyline (pts (xy 13.97 185.42) (xy 13.97 154.305))
+    (stroke (width 0) (type default) (color 0 0 0 0))
+  )
   (wire (pts (xy 182.88 73.66) (xy 185.42 73.66))
     (stroke (width 0) (type default) (color 0 0 0 0))
@@
     (stroke (width 0) (type default) (color 0 0 0 0))
   )
-  (polyline (pts (xy 13.97 179.705) (xy 13.97 154.94))
-    (stroke (width 0) (type default) (color 0 0 0 0))
-  )
   (wire (pts (xy 173.99 106.68) (xy 185.42 106.68))
     (stroke (width 0) (type default) (color 0 0 0 0))
@@
   (wire (pts (xy 193.04 86.36) (xy 199.39 86.36))
     (stroke (width 0) (type default) (color 0 0 0 0))
+  )
+  (text "C_{c} = 02011JR35ZBSTR  1.11pF\nC_{d} = 04023J3R6BBSTR  11.1pF\n\nFF_{Diff} = ( 2 * pi * R * ( 2 * C_{d} + C_{c} ) )^{ -1}\nR = 330 ohm\nC_{d} = 11.1pF\nC_{c} = 1.11pF\nFF_{Diff} = 20.69 MHz\n\nFF_{CM} = ( 2 * pi * R * C_{c} )^{ -1}\nR = 330 ohm\nC_{c} =  1.11pF\nFF_{CM} = 434.5 MHz\n\n"
+    (at 16.51 185.42 0)
+    (effects (font (size 1.27 1.27)) (justify left bottom))
   )
   (text "ADR510:\n\nI_{Q_min} =  0.1 mA\nI_{L_max (1PD)} =  1.2 mA\nI_{L_max (2PD)} =  2.4 mA\n\nI_{Q_max} = 10.0 mA\nI_{L_min} =  2.4 pA = 2.4e-9 mA\n\nI_{min_1} =  1.3 mA\nI_{min_2} =  2.5 mA\nI_{max} = 10.0 mA\n\nV_{S} = 5 v\nV_{out} = 1 v\n\nV = 5 v - 1 v = 4 v\n\nR_{BIAS}(I_{L_min (1PD)}) = 4 v /  1.3 mA = 3.3  Kohm\nR_{BIAS}(I_{L_min (2PD)}) = 4 v /  2.5 mA = 1600  ohm\nR_{BIAS}(I_{L_max}) = 4 v / 10.0 mA = 400 ohm\n\nR_{BIAS} = 402 ohm\nL = 4 V / 402 ohm = 9.95 mA"
@@
     (effects (font (size 1.27 1.27)) (justify left bottom))
   )
-  (text "GRM0225C1E180GA02L   18pF\nGRM0225C1E181JA02L  180pF\n\nFF_{Diff} = ( 2 * pi * R * ( 2 * C_{d} + C_{c} ) )^{ -1}\nR = 484 ohm\nC_{d} = 180pF\nC_{c} =  18pF\nFF_{Diff} = 434.964 MHz\n\nFF_{CM} = ( 2 * pi * R * C_{c} )^{ -1}\nR = 484 ohm\nC_{c} =  18pF\nFF_{CM} = 9.13e6 Hz\n\n"
-    (at 16.51 180.975 0)
-    (effects (font (size 1.27 1.27)) (justify left bottom))
-  )
   (text "AD8221:\n\nV(lux)_{PD} = 1.0 v - ( I_{PD} * RS1 )\n\nI_{PD} = 1.2 mA\nRS1 = 833 ohm\nV = 1.2 mA * 833 ohm = 1 V"
     (at 16.51 144.78 0)
     (effects (font (size 1.27 1.27)) (justify left bottom))
   )
-  (text "Photodiode (~320nm - 1100nm)\n\nDark Current:\nI_{R}(1V) = 18~22 pA\n\nI_{sc}(lx)_{uA} = (1.0 / 100) (uA / lx)\n\nEstimated 128Klux Maximum\n\n1280 uA = 128000 lx\n1280 uA = 1.2 mA per PD\n\n1 PD = 1.2 mA\nV = 1.2 mA * R ohm = 1.0 V\nR_{S1&S4} = 833 ohm\n\n2 PD = 2.4 mA\nV = 2.4 mA * R ohm = 1.0 V\nR_{S1|S4} = 417 ohm"
+  (text "Photodiode (~320nm - 1100nm)\n\nDark Current:\nI_{R}(1V) = 18~22 pA\n\nI_{sc}(lx)_{uA} = (1.0 / 100) (uA / lx)\n\nEstimated 128Klux Maximum\n\nI_{sc}(128Klux)_{uA}\n1280 uA = 128000 lx\n1280 uA = 1.2 mA per PD\n\n1 PD = 1.2 mA\nV = 1.2 mA * R ohm = 1.0 V\nR_{S1&S4} = 833 ohm -> 845 ohm\n\n2 PD = 2.4 mA\nV = 2.4 mA * R ohm = 1.0 V\nR_{S1|S4} = 417 ohm"
     (at 16.51 57.15 0)
     (effects (font (size 1.27 1.27)) (justify left bottom))
   )
-  (label "INV2" (at 161.29 81.28 180)
+  (label "INV2" (at 161.29 116.84 180)
     (effects (font (size 1.27 1.27)) (justify right bottom))
   )
@@
     (effects (font (size 1.27 1.27)) (justify left bottom))
   )
-  (label "INV1" (at 161.29 116.84 180)
+  (label "INV1" (at 161.29 81.28 180)
     (effects (font (size 1.27 1.27)) (justify right bottom))
   )
@@
       (effects (font (size 1.27 1.27)) (justify left))
     )
-    (property "Value" "1.7pF" (id 1) (at 184.15 67.31 90)
+    (property "Value" "1.11pF" (id 1) (at 184.15 67.31 90)
       (effects (font (size 1.27 1.27)) (justify left))
     )
@@
   (symbol (lib_id "Device:R") (at 167.64 81.28 90) (unit 1)
     (in_bom yes) (on_board yes)
-    (property "Reference" "RS?" (id 0) (at 168.91 83.82 90)
-      (effects (font (size 1.27 1.27)) (justify left))
-    )
-    (property "Value" "1K0" (id 1) (at 170.18 81.28 90)
+    (property "Reference" "RS6" (id 0) (at 168.91 83.82 90)
+      (effects (font (size 1.27 1.27)) (justify left))
+    )
+    (property "Value" "330" (id 1) (at 170.18 81.28 90)
       (effects (font (size 1.27 1.27)) (justify left))
     )
@@
       (effects (font (size 1.27 1.27)) (justify left))
     )
-    (property "Value" "833" (id 1) (at 156.21 123.19 0)
+    (property "Value" "845" (id 1) (at 156.21 123.19 0)
       (effects (font (size 1.27 1.27)) (justify left))
     )
@@
       (effects (font (size 1.27 1.27)) (justify left))
     )
-    (property "Value" "1.7pF" (id 1) (at 184.15 102.87 90)
+    (property "Value" "1.11pF" (id 1) (at 184.15 102.87 90)
       (effects (font (size 1.27 1.27)) (justify left))
     )
@@
       (effects (font (size 1.27 1.27)) (justify right))
     )
-    (property "Value" "R_Potentiometer" (id 1) (at 125.73 88.8999 0)
-      (effects (font (size 1.27 1.27)) (justify right) hide)
+    (property "Value" "10K" (id 1) (at 125.73 85.09 90)
+      (effects (font (size 1.27 1.27)) (justify right))
     )
     (property "Footprint" "Potentiometer_THT:Potentiometer_Bourns_3296W_Vertical" (id 2) (at 123.19 87.63 0)
@@
       (effects (font (size 1.27 1.27)) (justify left))
     )
-    (property "Value" "833" (id 1) (at 156.21 87.63 0)
+    (property "Value" "845" (id 1) (at 156.21 87.63 0)
       (effects (font (size 1.27 1.27)) (justify left))
     )
@@
       (effects (font (size 1.27 1.27)) (justify left))
     )
-    (property "Value" "17.4pF" (id 1) (at 173.99 78.105 0)
+    (property "Value" "11.1pF" (id 1) (at 173.99 78.105 0)
       (effects (font (size 1.27 1.27)) (justify left))
     )
@@
   (symbol (lib_id "Device:R") (at 167.64 71.12 90) (unit 1)
     (in_bom yes) (on_board yes)
-    (property "Reference" "RS?" (id 0) (at 168.91 68.58 90)
-      (effects (font (size 1.27 1.27)) (justify left))
-    )
-    (property "Value" "1K0" (id 1) (at 170.18 71.12 90)
+    (property "Reference" "RS3" (id 0) (at 168.91 68.58 90)
+      (effects (font (size 1.27 1.27)) (justify left))
+    )
+    (property "Value" "330" (id 1) (at 170.18 71.12 90)
       (effects (font (size 1.27 1.27)) (justify left))
     )
@@
   (symbol (lib_id "Device:R") (at 167.64 106.68 90) (unit 1)
     (in_bom yes) (on_board yes)
-    (property "Reference" "RS?" (id 0) (at 168.91 104.14 90)
-      (effects (font (size 1.27 1.27)) (justify left))
-    )
-    (property "Value" "4K02" (id 1) (at 170.18 106.68 90)
+    (property "Reference" "RS7" (id 0) (at 168.91 104.14 90)
+      (effects (font (size 1.27 1.27)) (justify left))
+    )
+    (property "Value" "330" (id 1) (at 170.18 106.68 90)
       (effects (font (size 1.27 1.27)) (justify left))
     )
@@
   (symbol (lib_id "Device:R") (at 167.64 116.84 90) (unit 1)
     (in_bom yes) (on_board yes)
-    (property "Reference" "RS?" (id 0) (at 168.91 119.38 90)
-      (effects (font (size 1.27 1.27)) (justify left))
-    )
-    (property "Value" "4K02" (id 1) (at 170.18 116.84 90)
+    (property "Reference" "RS8" (id 0) (at 168.91 119.38 90)
+      (effects (font (size 1.27 1.27)) (justify left))
+    )
+    (property "Value" "330" (id 1) (at 170.18 116.84 90)
       (effects (font (size 1.27 1.27)) (justify left))
     )
@@
       (effects (font (size 1.27 1.27)) (justify left))
     )
-    (property "Value" "17.4pF" (id 1) (at 173.99 114.3 0)
+    (property "Value" "11.1pF" (id 1) (at 173.99 114.3 0)
       (effects (font (size 1.27 1.27)) (justify left))
     )
@@
       (effects (font (size 1.27 1.27)) (justify left))
     )
-    (property "Value" "1.74pF" (id 1) (at 173.99 123.825 0)
+    (property "Value" "1.11pF" (id 1) (at 173.99 123.825 0)
       (effects (font (size 1.27 1.27)) (justify left))
     )
@@
       (effects (font (size 1.27 1.27)) (justify left))
     )
-    (property "Value" "1.74pF" (id 1) (at 173.99 88.265 0)
+    (property "Value" "1.11pF" (id 1) (at 173.99 88.265 0)
       (effects (font (size 1.27 1.27)) (justify left))
     )
@@
       (effects (font (size 1.27 1.27)) (justify right))
     )
-    (property "Value" "R_Potentiometer" (id 1) (at 125.73 111.7599 0)
-      (effects (font (size 1.27 1.27)) (justify right) hide)
+    (property "Value" "10K" (id 1) (at 125.73 107.95 90)
+      (effects (font (size 1.27 1.27)) (justify right))
     )
     (property "Footprint" "Potentiometer_THT:Potentiometer_Bourns_3296W_Vertical" (id 2) (at 123.19 110.49 0)

Commit message: SpectDrone Development
Changed lines of the file:
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@@
     (stroke (width 0) (type default) (color 0 0 0 0))
   )
-  (polyline (pts (xy 67.31 128.27) (xy 67.31 147.32))
+  (polyline (pts (xy 67.31 118.11) (xy 67.31 137.16))
     (stroke (width 0) (type default) (color 0 0 0 0))
   )
@@
     (stroke (width 0) (type default) (color 0 0 0 0))
   )
-  (polyline (pts (xy 13.97 67.31) (xy 67.31 67.31))
+  (polyline (pts (xy 13.97 62.23) (xy 67.31 62.23))
     (stroke (width 0) (type default) (color 0 0 0 0))
   )
@@
     (stroke (width 0) (type default) (color 0 0 0 0))
   )
-  (polyline (pts (xy 67.31 67.31) (xy 67.31 120.65))
+  (polyline (pts (xy 67.31 62.23) (xy 67.31 115.57))
     (stroke (width 0) (type default) (color 0 0 0 0))
   )
@@
     (stroke (width 0) (type default) (color 0 0 0 0))
   )
-  (polyline (pts (xy 67.31 185.42) (xy 13.97 185.42))
+  (polyline (pts (xy 67.31 170.815) (xy 13.97 170.815))
     (stroke (width 0) (type default) (color 0 0 0 0))
   )
@@
     (stroke (width 0) (type default) (color 0 0 0 0))
   )
-  (polyline (pts (xy 67.31 147.32) (xy 13.97 147.32))
+  (polyline (pts (xy 67.31 137.16) (xy 13.97 137.16))
     (stroke (width 0) (type default) (color 0 0 0 0))
   )
@@
     (stroke (width 0) (type default) (color 0 0 0 0))
   )
-  (polyline (pts (xy 67.31 120.65) (xy 13.97 120.65))
+  (polyline (pts (xy 67.31 115.57) (xy 13.97 115.57))
     (stroke (width 0) (type default) (color 0 0 0 0))
   )
@@
     (stroke (width 0) (type default) (color 0 0 0 0))
   )
-  (polyline (pts (xy 67.31 154.305) (xy 67.31 185.42))
+  (polyline (pts (xy 67.31 139.7) (xy 67.31 170.815))
     (stroke (width 0) (type default) (color 0 0 0 0))
   )
@@
     (stroke (width 0) (type default) (color 0 0 0 0))
   )
-  (polyline (pts (xy 13.97 128.27) (xy 67.31 128.27))
+  (polyline (pts (xy 13.97 118.11) (xy 67.31 118.11))
     (stroke (width 0) (type default) (color 0 0 0 0))
   )
@@
     (stroke (width 0) (type default) (color 0 0 0 0))
   )
-  (polyline (pts (xy 13.97 154.305) (xy 67.31 154.305))
+  (polyline (pts (xy 13.97 139.7) (xy 67.31 139.7))
     (stroke (width 0) (type default) (color 0 0 0 0))
   )
@@
     (stroke (width 0) (type default) (color 0 0 0 0))
   )
-  (polyline (pts (xy 13.97 185.42) (xy 13.97 154.305))
+  (polyline (pts (xy 13.97 170.815) (xy 13.97 139.7))
     (stroke (width 0) (type default) (color 0 0 0 0))
   )
@@
     (stroke (width 0) (type default) (color 0 0 0 0))
   )
-  (polyline (pts (xy 13.97 147.32) (xy 13.97 128.27))
+  (polyline (pts (xy 13.97 137.16) (xy 13.97 118.11))
     (stroke (width 0) (type default) (color 0 0 0 0))
   )
@@
     (stroke (width 0) (type default) (color 0 0 0 0))
   )
-  (polyline (pts (xy 13.97 120.65) (xy 13.97 67.31))
+  (polyline (pts (xy 13.97 115.57) (xy 13.97 62.23))
     (stroke (width 0) (type default) (color 0 0 0 0))
   )
@@
   )
   (text "C_{c} = 02011JR35ZBSTR  1.11pF\nC_{d} = 04023J3R6BBSTR  11.1pF\n\nFF_{Diff} = ( 2 * pi * R * ( 2 * C_{d} + C_{c} ) )^{ -1}\nR = 330 ohm\nC_{d} = 11.1pF\nC_{c} = 1.11pF\nFF_{Diff} = 20.69 MHz\n\nFF_{CM} = ( 2 * pi * R * C_{c} )^{ -1}\nR = 330 ohm\nC_{c} =  1.11pF\nFF_{CM} = 434.5 MHz\n\n"
-    (at 16.51 185.42 0)
+    (at 16.51 170.815 0)
     (effects (font (size 1.27 1.27)) (justify left bottom))
   )
   (text "ADR510:\n\nI_{Q_min} =  0.1 mA\nI_{L_max (1PD)} =  1.2 mA\nI_{L_max (2PD)} =  2.4 mA\n\nI_{Q_max} = 10.0 mA\nI_{L_min} =  2.4 pA = 2.4e-9 mA\n\nI_{min_1} =  1.3 mA\nI_{min_2} =  2.5 mA\nI_{max} = 10.0 mA\n\nV_{S} = 5 v\nV_{out} = 1 v\n\nV = 5 v - 1 v = 4 v\n\nR_{BIAS}(I_{L_min (1PD)}) = 4 v /  1.3 mA = 3.3  Kohm\nR_{BIAS}(I_{L_min (2PD)}) = 4 v /  2.5 mA = 1600  ohm\nR_{BIAS}(I_{L_max}) = 4 v / 10.0 mA = 400 ohm\n\nR_{BIAS} = 402 ohm\nL = 4 V / 402 ohm = 9.95 mA"
-    (at 16.51 118.11 0)
+    (at 16.51 113.03 0)
     (effects (font (size 1.27 1.27)) (justify left bottom))
   )
   (text "AD8221:\n\nV(lux)_{PD} = 1.0 v - ( I_{PD} * RS1 )\n\nI_{PD} = 1.2 mA\nRS1 = 833 ohm\nV = 1.2 mA * 833 ohm = 1 V"
-    (at 16.51 144.78 0)
+    (at 16.51 134.62 0)
     (effects (font (size 1.27 1.27)) (justify left bottom))
   )

Commit message: SpectDrone Development
Other:
- moved on the sheet: CS1, CS10, CS2, CS3, CS4, CS5, CS6, CS7, CS8, CS9, JPV1, JPV2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

Commit message: SpectDrone Development
Parts:
- added JPV1: SolderJumper_2_Bridged, Jumper:SolderJumper-2_P1.3mm_Bridged_RoundedPad1.0x1.5mm, symbol Jumper:SolderJumper_2_Bridged
- renumbered JPV1 to JPV2, JPV2 to JPV3
Connections:
- net 1.0V1: now also JPV1.1 (A); no longer R4.2, RV1.1, TPv1-1.1, U8.2 (K)
- new net 1V1: JPV1.2 (B), R4.2, RV1.1, TPv1-1.1, U8.2 (K)
Other:
- note added: "RS1 & RS5: Per datasheet: R_{G} = (49.4 Kohm) / (G-1) ex. R_{G} Gain V_{RF} inf 1.000 5.0 49.9 k 1.990 2.5 12.4 k 4.984 1.0 <--- 5.49 k 9.998 0.5 2.61 k 19.93 1.00 k 50.40 499 100.0 249 199.4 100 495.0 49.9 991.0"
- moved on the sheet: JPV2, R4, R9, RV1, TPv1-1, U8

Commit message: SpectDrone Development
Parts:
- removed RV2: 10K, Potentiometer_THT:Potentiometer_Bourns_3296W_Vertical, symbol Device:R_Potentiometer
- added JP16: SolderJumper_3_Bridged12, Jumper:SolderJumper-3_P1.3mm_Bridged2Bar12_RoundedPad1.0x1.5mm, symbol Jumper:SolderJumper_3_Bridged12
- added TP5v0-1: TestPoint, TestPoint:TestPoint_Keystone_5000-5004_Miniature, symbol Connector:TestPoint
- added U13: ADR5045B, Package_TO_SOT_SMD:SOT-23, symbol Gardenuino_Custom:ADR510
- R10: value 470K -> 0; footprint Capacitor_SMD:C_0805_2012Metric -> Resistor_SMD:R_0603_1608Metric
- RS2, RS5: value 12K4 -> R
- U8: symbol Reference_Voltage:CJ432 -> Gardenuino_Custom:ADR510
- U9: value ADR510 -> ADR504; symbol Reference_Voltage:CJ432 -> Gardenuino_Custom:ADR510
Connections:
- net 1V1: now also U8.1 (K); no longer U8.2 (K)
- net 5V3: now also R10.2, JP16.1 (A); no longer CS10.2, CS4.1, CS5.2, CS9.1, US1.8 (Vs+), US2.8 (Vs+)
- net GND1: now also U8.2 (A), U9.2 (A); no longer U8.3 (A), U9.3 (A)
- net at R9.1: now also U8.3 (REF); no longer U8.1 (REF)
- net 4.096V: now reaches U9.1 (K)
- net 4.096V: now also JPV3.1 (A), R5.2, TPv1-2.1, U9.3 (REF); no longer R10.1
- net 1.0V1 renamed PD1
- net 1.0V2 renamed PD2
- removed net 1V2: JPV3.1 (A), R5.2, TPv1-2.1, U9.2 (K)
- new net 5V0: JP16.3 (B), R10.1, U13.1 (K), U13.3 (REF)
- new net 5VS: CS10.2, CS4.1, CS5.2, CS9.1, JP16.2 (C), TP5v0-1.1, US1.8 (Vs+), US2.8 (Vs+)
- new net GND_{RF}: U13.2 (A)
Other:
- note added: "RS2 & RS5: Per datasheet: R_{G} = (49.4 Kohm) / (G-1) ex. R_{G} Gain V_{RF} inf 1.000 5.0 226 k 1.218 4.096 <--- 49.9 k 1.990 2.5 12.4 k 4.984 1.0 <--- 5.49 k 9.998 0.5 2.61 k 19.93 1.00 k 50.40 499 100.0 249 199.4 100 495.0 49.9 991.0"
- note removed: "RS1 & RS5: Per datasheet: R_{G} = (49.4 Kohm) / (G-1) ex. R_{G} Gain V_{RF} inf 1.000 5.0 49.9 k 1.990 2.5 12.4 k 4.984 1.0 <--- 5.49 k 9.998 0.5 2.61 k 19.93 1.00 k 50.40 499 100.0 249 199.4 100 495.0 49.9 991.0"
