File: Longwave Instrument/Longwave Instrument.kicad_sch (KiCad schematic)
At the start: 37 parts, among them U13 ADR5045B, U8 ADR510, U9 ADR504

Commit message: SpectDrone Development
Parts:
- R10: value 0 -> R
- R4, R5: value 402 -> R_{BIAS}
- RS2, RS5: value R -> R_{G}
- R_{PD}1: renamed from RS1; value 845 -> R_{PD}
- R_{PD}2: renamed from RS4; value 845 -> R_{PD}
Other:
- note added: "1 PD = 1.2 mA V = 1.2 mA * R ohm = 4.0 V R_{S1&S4} = 3.33 Kohm -> 3.32 Kohm 2 PD = 2.4 mA V = 2.4 mA * R ohm = 4.0 V R_{S1|S4} = 1.67 Kohm -> 1.65 Kohm"
- note added: "AD8221: V(lux)_{PD} = 1000 mV - ( I_{PD} * RS1 ) I_{PD} = 1.2 mA R_{PD} = 825 ohm V = 1.2 mA * 833 ohm = 1000 mV V = 1.2 mA * 825 ohm = 990 mV"
- note added: "AD8221: V(lux)_{PD} = 4096 mV - ( I_{PD} * RS1 ) I_{PD} = 1.2 mA R_{PD} = 3K4 ohm V = 1.2 mA * 3413 ohm = 4096 mV V = 1.2 mA * 3400 ohm = 4080 mV"
- note added: "ADR510 / ADR504: I_{Q_min} = 0.1 mA I_{L_max (1PD)} = 1.2 mA I_{L_max (2PD)} = 2.4 mA I_{Q_max} = 10.0 mA I_{L_min} = 2.4 pA = 2.4e-9 mA I_{min_1} = 1.3 mA I_{min_2} = 2.5 mA I_{max} = 10.0 mA V_{S} = 5 v V_{out} = 1 v V = 5 v - 1 v = 4 v R_{BIAS}(I_{L_min (1PD)}) = 4 v / 1.3 mA = 3.3 Kohm R_{BIAS}(I_{L_min (2PD)}) = 4 v / 2.5 mA = 1600 ohm R_{BIAS}(I_{L_max}) = 4 v / 10.0 mA = 400 ohm R_{BIAS} =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"
- note added: "Photodiode (~320nm - 1100nm) Dark Current: I_{R}(1V) = 18~22 pA Short Circuit Current: I_{sc}(lx)_{uA} = (1.0 / 100) (uA / lx) Estimated 128Klux Maximum I_{sc}(128Klux)_{uA} 1280 uA = 128000 lx 1280 uA = 1.2 mA per PD 1 PD = 1.2 mA V = 1.2 mA * R ohm = 1.0 V R_{S1&S4} = 833 ohm -> 845 ohm 2 PD = 2.4 mA V = 2.4 mA * R ohm = 1.0 V R_{S1|S4} = 417 ohm"
- note added: "RS2 & RS5: Per datasheet: R_{G} = (49.4 Kohm) / (G-1) ex. R_{G} Gain V(PD) inf 1.000 5.0 226 k 1.218 4.096 <--- 49.9 k 1.990 2.5 12.4 k 4.984 1.0 <--- 5.49 k 9.998 0.5 2.61 k 19.93 1.00 k 50.40 499 100.0 249 199.4 100 495.0 49.9 991.0"
- note added: "V_{S} = 5 v V_{out} = 4 v V = 5 v - 4 v = 1 v R_{BIAS}(I_{L_min (1PD)}) = 1 v / 1.3 mA = 769 ohm R_{BIAS}(I_{L_min (2PD)}) = 1 v / 2.5 mA = 400 ohm R_{BIAS}(I_{L_max}) = 1 v / 10.0 mA = 100 ohm R_{BIAS} = 100 ohm L = 1 V / 100 ohm = 10 mA R5 = 100 ohm"
- note removed: "AD8221: V(lux)_{PD} = 1.0 v - ( I_{PD} * RS1 ) I_{PD} = 1.2 mA RS1 = 833 ohm V = 1.2 mA * 833 ohm = 1 V"
- note removed: "ADR510: I_{Q_min} = 0.1 mA I_{L_max (1PD)} = 1.2 mA I_{L_max (2PD)} = 2.4 mA I_{Q_max} = 10.0 mA I_{L_min} = 2.4 pA = 2.4e-9 mA I_{min_1} = 1.3 mA I_{min_2} = 2.5 mA I_{max} = 10.0 mA V_{S} = 5 v V_{out} = 1 v V = 5 v - 1 v = 4 v R_{BIAS}(I_{L_min (1PD)}) = 4 v / 1.3 mA = 3.3 Kohm R_{BIAS}(I_{L_min (2PD)}) = 4 v / 2.5 mA = 1600 ohm R_{BIAS}(I_{L_max}) = 4 v / 10.0 mA = 400 ohm R_{BIAS} = 402 ohm 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"
- note removed: "Photodiode (~320nm - 1100nm) Dark Current: I_{R}(1V) = 18~22 pA I_{sc}(lx)_{uA} = (1.0 / 100) (uA / lx) Estimated 128Klux Maximum I_{sc}(128Klux)_{uA} 1280 uA = 128000 lx 1280 uA = 1.2 mA per PD 1 PD = 1.2 mA V = 1.2 mA * R ohm = 1.0 V R_{S1&S4} = 833 ohm -> 845 ohm 2 PD = 2.4 mA V = 2.4 mA * R ohm = 1.0 V R_{S1|S4} = 417 ohm"
- note removed: "RS2 & RS5: Per datasheet: R_{G} = (49.4 Kohm) / (G-1) ex. R_{G} Gain V_{RF} inf 1.000 5.0 226 k 1.218 4.096 <--- 49.9 k 1.990 2.5 12.4 k 4.984 1.0 <--- 5.49 k 9.998 0.5 2.61 k 19.93 1.00 k 50.40 499 100.0 249 199.4 100 495.0 49.9 991.0"
- moved on the sheet: CS1, CS10, CS2, CS3, CS4, CS5, CS6, CS7, CS8, CS9, JP16, JPV1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
