File: Longwave Instrument/Longwave Instrument.kicad_sch (KiCad schematic)
At the start: 37 parts, among them U13 ADR5045B, U8 ADR510, U9 ADR504

Commit message: SpectDrone Development
Parts:
- R4: value R_{BIAS} -> 402
- R5: value R_{BIAS} -> 100
Other:
- note added: "R_{BIAS}"
Changed lines of the file:
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@@
+    (effects (font (size 1.27 1.27)) (justify left bottom))
+  )
+  (text "R_{BIAS}" (at 145.415 124.46 0)
     (effects (font (size 1.27 1.27)) (justify left bottom))
   )
@@
     (effects (font (size 1.27 1.27)) (justify left bottom))
   )
+  (text "R_{BIAS}" (at 145.415 95.25 0)
+    (effects (font (size 1.27 1.27)) (justify left bottom))
+  )
   (text "\nV_{S} = 5 v\nV_{out} = 4 v\n\nV = 5 v - 4 v = 1 v\n\nR_{BIAS}(I_{L_min (1PD)}) = 1 v /  1.3 mA = 769 ohm\nR_{BIAS}(I_{L_min (2PD)}) = 1 v /  2.5 mA = 400 ohm\nR_{BIAS}(I_{L_max}) = 1 v / 10.0 mA = 100 ohm\n\nR_{BIAS} = 100 ohm\nL = 1 V / 100 ohm = 10 mA\nR5 = 100 ohm"
     (at 73.025 121.92 0)
@@
   (global_label "5VS" (shape input) (at 179.07 74.295 0) (fields_autoplaced)
     (effects (font (size 1.27 1.27)) (justify left))
-    (property "Intersheet References" "${INTERSHEET_REFS}" (id 0) (at 184.9907 74.3744 0)
-      (effects (font (size 1.27 1.27)) (justify right) hide)
+    (property "Intersheet References" "${INTERSHEET_REFS}" (id 0) (at 184.9907 74.2156 0)
+      (effects (font (size 1.27 1.27)) (justify left) hide)
     )
   )
@@
     (in_bom yes) (on_board yes)
     (property "Reference" "R5" (id 0) (at 147.955 118.745 90))
-    (property "Value" "R_{BIAS}" (id 1) (at 147.955 121.285 90))
+    (property "Value" "100" (id 1) (at 147.955 121.285 90))
     (property "Footprint" "Capacitor_SMD:C_0805_2012Metric" (id 2) (at 147.955 123.063 90)
       (effects (font (size 1.27 1.27)) hide)
@@
     (in_bom yes) (on_board yes)
     (property "Reference" "R4" (id 0) (at 147.955 89.535 90))
-    (property "Value" "R_{BIAS}" (id 1) (at 147.955 92.075 90))
+    (property "Value" "402" (id 1) (at 147.955 92.075 90))
     (property "Footprint" "Capacitor_SMD:C_0805_2012Metric" (id 2) (at 147.955 93.853 90)
       (effects (font (size 1.27 1.27)) hide)

Commit message: SpectDrone Development
Other:
- moved on the sheet: JP16, R10, TP5v0-1, TPv1-2, U13, U9

Commit message: SpectDrone Development
Parts:
- added R_{PD}2, R_{PD}4: 0, Capacitor_SMD:C_0805_2012Metric, symbol Device:R
- renumbered R_{PD}2 to R_{PD}3
Connections:
- net GND1: now also R_{PD}2.2, R_{PD}4.2; no longer R_{PD}1.2, R_{PD}3.2
- net INV1: now also R_{PD}1.2, R_{PD}2.1; no longer PD1.1 (A), R_{PD}1.1
- net INV2: now also R_{PD}3.2, R_{PD}4.1; no longer PD2.1 (A), R_{PD}3.1
- net PD1: no longer RS3.1
- net PD2: no longer RS7.1
- new net: PD2.1 (A), RS7.1, R_{PD}3.1
- new net: PD1.1 (A), RS3.1, R_{PD}1.1
Other:
- note added: "AD8221: V(lux)_{PD} = 1000 mV - ( I_{PD} * RS1 ) I_{PD} = 1.5 mA R_{PD} = 665 ohm V = 1.5 mA * 666.~{6} ohm = 1000 mV V = 1.5 mA * 665 ohm = 997.5 mV"
- note added: "AD8221: V(lux)_{PD} = 4096 mV - ( I_{PD} * RS1 ) I_{PD} = 1.5 mA R_{PD} = 2k67 ohm V = 1.5 mA * 2730.~{6} ohm = 4096 mV V = 1.5 mA * 2670 ohm = 4005 mV"
- note added: "Photodiode (~320nm - 1100nm) Dark Current: I_{R}(1V) = 18~22 pA Short Circuit Current: I_{sc}(lx)_{uA} = (1.0 / 100) (uA / lx) Estimated 128Klux Maximum I_{sc}(128Klux)_{uA} 1280 uA = 128000 lx 1280 uA = 1.2 mA per PD"
- note removed: "1 PD = 1.2 mA V = 1.2 mA * R ohm = 4.0 V R_{S1&S4} = 3.33 Kohm -> 3.32 Kohm 2 PD = 2.4 mA V = 2.4 mA * R ohm = 4.0 V R_{S1|S4} = 1.67 Kohm -> 1.65 Kohm"
- note removed: "Photodiode (~320nm - 1100nm) Dark Current: I_{R}(1V) = 18~22 pA Short Circuit Current: I_{sc}(lx)_{uA} = (1.0 / 100) (uA / lx) Estimated 128Klux Maximum I_{sc}(128Klux)_{uA} 1280 uA = 128000 lx 1280 uA = 1.2 mA per PD 1 PD = 1.2 mA V = 1.2 mA * R ohm = 1.0 V R_{S1&S4} = 833 ohm -> 845 ohm 2 PD = 2.4 mA V = 2.4 mA * R ohm = 1.0 V R_{S1|S4} = 417 ohm"
- moved on the sheet: CS1, CS10, CS2, CS3, CS4, CS5, CS6, CS7, CS8, CS9, JP16, JPV1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

Commit message: SpectDrone Development
Parts:
- JP16: footprint Jumper:SolderJumper-3_P1.3mm_Bridged2Bar12_RoundedPad1.0x1.5mm -> Gardenuino Custom:SolderJumper-4_P1.3mm_Bridged2Bar12_RoundedPad
Connections:
- net 5VS renamed V_{AREF}
- new net 3V1: JP16.4 (B)
Changed lines of the file:
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@@
+    (stroke (width 0) (type default) (color 0 0 0 0))
+  )
+  (wire (pts (xy 153.035 40.64) (xy 156.21 40.64))
     (stroke (width 0) (type default) (color 0 0 0 0))
   )
@@
     )
   )
-  (global_label "5VS" (shape input) (at 273.685 90.805 0) (fields_autoplaced)
+  (global_label "V_{AREF}" (shape input) (at 273.685 90.805 0) (fields_autoplaced)
     (effects (font (size 1.27 1.27)) (justify left))
-    (property "Intersheet References" "${INTERSHEET_REFS}" (id 0) (at 279.6057 90.7256 0)
-      (effects (font (size 1.27 1.27)) (justify left) hide)
+    (property "Intersheet References" "${INTERSHEET_REFS}" (id 0) (at 280.8636 90.7256 0)
+      (effects (font (size 1.27 1.27)) (justify left) hide)
+    )
+  )
+  (global_label "3V1" (shape input) (at 153.035 40.64 180) (fields_autoplaced)
+    (effects (font (size 1.27 1.27)) (justify right))
+    (property "Intersheet References" "${INTERSHEET_REFS}" (id 0) (at 147.1143 40.5606 0)
+      (effects (font (size 1.27 1.27)) (justify right) hide)
     )
   )
@@
     )
   )
-  (global_label "5VS" (shape input) (at 181.61 40.64 0) (fields_autoplaced)
+  (global_label "V_{AREF}" (shape input) (at 181.61 40.64 0) (fields_autoplaced)
     (effects (font (size 1.27 1.27)) (justify left))
-    (property "Intersheet References" "${INTERSHEET_REFS}" (id 0) (at 187.5307 40.5606 0)
+    (property "Intersheet References" "${INTERSHEET_REFS}" (id 0) (at 188.7886 40.5606 0)
       (effects (font (size 1.27 1.27)) (justify left) hide)
     )
@@
   )
   (symbol (lib_id "Jumper:SolderJumper_3_Bridged12") (at 161.29 40.64 90) (unit 1)
-    (in_bom yes) (on_board yes) (fields_autoplaced)
-    (property "Reference" "JP16" (id 0) (at 158.75 39.3699 90)
-      (effects (font (size 1.27 1.27)) (justify left))
-    )
-    (property "Value" "SolderJumper_3_Bridged12" (id 1) (at 158.75 41.9099 90)
-      (effects (font (size 1.27 1.27)) (justify left))
-    )
-    (property "Footprint" "Jumper:SolderJumper-3_P1.3mm_Bridged2Bar12_RoundedPad1.0x1.5mm" (id 2) (at 161.29 40.64 0)
+    (in_bom yes) (on_board yes)
+    (property "Reference" "JP16" (id 0) (at 156.845 44.45 90)
+      (effects (font (size 1.27 1.27)) (justify left))
+    )
+    (property "Value" "SolderJumper_3_Bridged12" (id 1) (at 168.91 38.1 0)
+      (effects (font (size 1.27 1.27)) (justify left) hide)
+    )
+    (property "Footprint" "Gardenuino Custom:SolderJumper-4_P1.3mm_Bridged2Bar12_RoundedPad" (id 2) (at 166.37 35.56 0)
       (effects (font (size 1.27 1.27)) hide)
     )
@@
     (pin "2")
     (pin "3")
+    (pin "4")
   )
   (symbol (lib_id "Device:C_Small") (at 231.14 80.01 0) (mirror y) (unit 1)

Commit message: SpectDrone Development
Parts:
- U9: value ADR504 -> ADR5043B
Connections:
- net 4.096V is gone; now on net 3V0: JPV3.1 (A), R5.2, TPv1-2.1, U9.1 (K), U9.3 (REF)
- net 3V1 renamed 3V0
Changed lines of the file:
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@@
     )
   )
-  (global_label "4.096V" (shape input) (at 180.34 95.25 0) (fields_autoplaced)
-    (effects (font (size 1.27 1.27)) (justify left))
-    (property "Intersheet References" "${INTERSHEET_REFS}" (id 0) (at 189.2845 95.1706 0)
+  (global_label "3V0" (shape input) (at 180.34 95.25 0) (fields_autoplaced)
+    (effects (font (size 1.27 1.27)) (justify left))
+    (property "Intersheet References" "${INTERSHEET_REFS}" (id 0) (at 186.2607 95.1706 0)
       (effects (font (size 1.27 1.27)) (justify left) hide)
     )
@@
     )
   )
-  (global_label "3V1" (shape input) (at 153.035 40.64 180) (fields_autoplaced)
+  (global_label "3V0" (shape input) (at 153.035 40.64 180) (fields_autoplaced)
     (effects (font (size 1.27 1.27)) (justify right))
     (property "Intersheet References" "${INTERSHEET_REFS}" (id 0) (at 147.1143 40.5606 0)
@@
       (effects (font (size 1.27 1.27)) (justify right))
     )
-    (property "Value" "ADR504" (id 1) (at 154.94 100.33 90)
-      (effects (font (size 1.27 1.27)) (justify right))
-    )
+    (property "Value" "ADR5043B" (id 1) (at 154.94 100.33 90)
+      (effects (font (size 1.27 1.27)) (justify right))
+    )

Commit message: SpectDrone Development
Parts:
- renumbered R_{PD}2 to R_{PD.bias}1, R_{PD}4 to R_{PD.bias}2, R_{PD}3 to R_{PD}2
Other:
- note added: "V_{S} = 5 v V_{out} = 3.3 v V = 5 v - 3.3 v = 1.7 v R_{BIAS}(I_{L_min (1PD)}) = 1.7 v / 1.3 mA = 1308 ohm R_{BIAS}(I_{L_min (2PD)}) = 1.7 v / 2.5 mA = 680 ohm R_{BIAS}(I_{L_max}) = 1.7 v / 10.0 mA = 170 ohm R_{BIAS} = 169 ohm L = 1.7 V / 169 ohm = 10.06 mA R5 = 169 ohm"
Changed lines of the file:
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@@
+    (stroke (width 0) (type default) (color 0 0 0 0))
+  )
+  (polyline (pts (xy 125.73 109.22) (xy 125.73 135.89))
     (stroke (width 0) (type default) (color 0 0 0 0))
   )
@@
     (stroke (width 0) (type default) (color 0 0 0 0))
   )
-  (polyline (pts (xy 72.39 136.525) (xy 125.73 136.525))
+  (polyline (pts (xy 72.39 137.16) (xy 125.73 137.16))
     (stroke (width 0) (type default) (color 0 0 0 0))
   )
@@
     (stroke (width 0) (type default) (color 0 0 0 0))
   )
+  (polyline (pts (xy 72.39 109.22) (xy 125.73 109.22))
+    (stroke (width 0) (type default) (color 0 0 0 0))
+  )
   (wire (pts (xy 179.07 76.2) (xy 179.07 77.47))
     (stroke (width 0) (type default) (color 0 0 0 0))
@@
     (stroke (width 0) (type default) (color 0 0 0 0))
   )
+  (polyline (pts (xy 72.39 135.89) (xy 72.39 109.22))
+    (stroke (width 0) (type default) (color 0 0 0 0))
+  )
   (wire (pts (xy 250.19 78.74) (xy 271.78 78.74))
     (stroke (width 0) (type default) (color 0 0 0 0))
@@
     (stroke (width 0) (type default) (color 0 0 0 0))
   )
-  (polyline (pts (xy 72.39 163.83) (xy 72.39 136.525))
+  (polyline (pts (xy 72.39 163.83) (xy 72.39 137.16))
     (stroke (width 0) (type default) (color 0 0 0 0))
   )
@@
     (stroke (width 0) (type default) (color 0 0 0 0))
   )
-  (polyline (pts (xy 125.73 136.525) (xy 125.73 163.83))
+  (polyline (pts (xy 125.73 137.16) (xy 125.73 163.83))
     (stroke (width 0) (type default) (color 0 0 0 0))
   )
@@
   )
   (wire (pts (xy 213.36 100.33) (xy 218.44 100.33))
+    (stroke (width 0) (type default) (color 0 0 0 0))
+  )
+  (polyline (pts (xy 125.73 135.89) (xy 72.39 135.89))
     (stroke (width 0) (type default) (color 0 0 0 0))
   )
@@
     (effects (font (size 1.27 1.27)) (justify left bottom))
   )
+  (text "\nV_{S} = 5 v\nV_{out} = 4 v\n\nV = 5 v - 4 v = 1 v\n\nR_{BIAS}(I_{L_min (1PD)}) = 1 v /  1.3 mA = 769 ohm\nR_{BIAS}(I_{L_min (2PD)}) = 1 v /  2.5 mA = 400 ohm\nR_{BIAS}(I_{L_max}) = 1 v / 10.0 mA = 100 ohm\n\nR_{BIAS} = 100 ohm\nL = 1 V / 100 ohm = 10 mA\nR5 = 100 ohm"
+    (at 74.93 134.62 0)
+    (effects (font (size 1.27 1.27)) (justify left bottom))
+  )
   (text "AD8221:\n\nV(lux)_{PD} = 1000 mV - ( I_{PD} * RS1 )\n\nI_{PD} = 1.2 mA\nR_{PD} = 825 ohm\nV = 1.2 mA * 833 ohm = 1000 mV\nV = 1.2 mA * 825 ohm =  990 mV"
     (at 19.05 82.55 0)
@@
     (effects (font (size 1.27 1.27)) (justify left bottom))
   )
-  (text "\nV_{S} = 5 v\nV_{out} = 4 v\n\nV = 5 v - 4 v = 1 v\n\nR_{BIAS}(I_{L_min (1PD)}) = 1 v /  1.3 mA = 769 ohm\nR_{BIAS}(I_{L_min (2PD)}) = 1 v /  2.5 mA = 400 ohm\nR_{BIAS}(I_{L_max}) = 1 v / 10.0 mA = 100 ohm\n\nR_{BIAS} = 100 ohm\nL = 1 V / 100 ohm = 10 mA\nR5 = 100 ohm"
+  (text "\nV_{S} = 5 v\nV_{out} = 3.3 v\n\nV = 5 v - 3.3 v = 1.7 v\n\nR_{BIAS}(I_{L_min (1PD)}) = 1.7 v /  1.3 mA = 1308 ohm\nR_{BIAS}(I_{L_min (2PD)}) = 1.7 v /  2.5 mA =  680 ohm\nR_{BIAS}(I_{L_max}) = 1.7 v / 10.0 mA = 170 ohm\n\nR_{BIAS} = 169 ohm\nL = 1.7 V / 169 ohm = 10.06 mA\nR5 = 169 ohm"
     (at 74.93 162.56 0)
     (effects (font (size 1.27 1.27)) (justify left bottom))
@@
   (symbol (lib_id "Device:R") (at 218.44 80.01 0) (unit 1)
     (in_bom yes) (on_board yes)
-    (property "Reference" "R_{PD}2" (id 0) (at 212.725 78.74 0)
+    (property "Reference" "R_{PD.bias}1" (id 0) (at 208.28 78.74 0)
       (effects (font (size 1.27 1.27)) (justify left))
     )
@@
   (symbol (lib_id "Device:R") (at 218.44 105.41 0) (unit 1)
     (in_bom yes) (on_board yes)
-    (property "Reference" "R_{PD}3" (id 0) (at 212.09 104.14 0)
+    (property "Reference" "R_{PD}2" (id 0) (at 212.09 104.14 0)
       (effects (font (size 1.27 1.27)) (justify left))
     )
@@
   (symbol (lib_id "Device:R") (at 218.44 115.57 0) (unit 1)
     (in_bom yes) (on_board yes)
-    (property "Reference" "R_{PD}4" (id 0) (at 212.725 114.3 0)
-      (effects (font (size 1.27 1.27)) (justify left))
-    )
+    (property "Reference" "R_{PD.bias}2" (id 0) (at 208.28 114.3 0)
+      (effects (font (size 1.27 1.27)) (justify left))
+    )

Commit message: SpectDrone Development
Parts:
- added JPD1, JPD3, JPD4, JPD6: SolderJumper_2_Bridged, Jumper:SolderJumper-2_P1.3mm_Bridged_RoundedPad1.0x1.5mm, symbol Jumper:SolderJumper_2_Bridged
- added JPD2, JPD5: SolderJumper_2_Open, Jumper:SolderJumper-2_P1.3mm_Open_RoundedPad1.0x1.5mm, symbol Jumper:SolderJumper_2_Open
- R_{PD}1, R_{PD}2: value R_{PD} -> X
Connections:
- net 1V1: now also JPV3.2 (B); no longer JPV1.2 (B)
- net 3V0: now also JP16.1 (A), JPV1.1 (A); no longer JP16.4 (B), JPV3.1 (A)
- net 5V3: now also JP16.4 (B); no longer JP16.1 (A)
- net INV1: now also JPD3.2 (B)
- net INV2: now also JPD6.2 (B)
- net PD1: now also JPV3.1 (A), JPD1.1 (A); no longer JPV1.1 (A)
- net PD2: now also JPV1.2 (B), JPD4.1 (A); no longer JPV3.2 (B)
- net at RS7.1, R_{PD}2.1: now also JPD4.2 (B), JPD5.2 (B); no longer PD2.1 (A)
- net at RS3.1, R_{PD}1.1: now also JPD1.2 (B), JPD2.2 (B); no longer PD1.1 (A)
- net S1 renamed P1
- net S2 renamed P2
- new net: JPD5.1 (A), JPD6.1 (A), PD2.1 (A)
- new net: JPD2.1 (A), JPD3.1 (A), PD1.1 (A)
Other:
- note added: "* In this configuration, outputs P1 and P2 are inverted in reference to photocurrent. Invert the state of JPD1-6 and place R_{PD} to make the signs the same."
- note added: "1 +/- 0.0035 mV"
- note added: "3 +/- 0.003 mV"
- note added: "AD8221: V(lux)_{PD} = 1000 mV - ( I_{PD} * RS1 ) I_{PD} = 1 mA R_{PD} = 1K0 ohm V = 1 mA * 1000 ohm = 1000 mV"
- note added: "AD8221: V(lux)_{PD} = 3000 mV - ( I_{PD} * RS1 ) I_{PD} = 1 mA R_{PD} = 3K0 ohm V = 1 mA * 3000 ohm = 3000 mV"
- note added: "AD8221: V(lux)_{PD} = 3000 mV - ( I_{PD} * RS1 ) I_{PD} = 1.2 mA R_{PD} = 2K49 ohm V = 1.2 mA * 2500 ohm = 3000 mV V = 1.2 mA * 2490 ohm = 2988 mV"
- note added: "AD8221: V(lux)_{PD} = 3000 mV - ( I_{PD} * RS1 ) I_{PD} = 1.5 mA R_{PD} = 2k ohm V = 1.5 mA * 2000 ohm = 3000 mV"
- note added: "RS2 & RS5: Per datasheet: R_{G} = (49.4 Kohm) / (G-1) G = ((49.4 Kohm) / R_{G}) + 1 ex. R_{G} Gain V(PD) inf 1.000 5.0 226 k 1.218 4.096 49.9 k 1.990 2.5 24.3 k 3.033 1.0 24.9 k 2.984 1.0 <--- 12.4 k 4.984 1.0"
- note added: "V_{S} = 5 v V_{out} = 3.0 v V = 5 v - 3.0 v = 2.0 v R_{BIAS}(I_{L_min (1PD)}) = 2.0 v / 1.3 mA = 1538 ohm R_{BIAS}(I_{L_min (2PD)}) = 2.0 v / 2.5 mA = 800 ohm R_{BIAS}(I_{L_max}) = 2.0 v / 10.0 mA = 200 ohm R_{BIAS} = 200 ohm L = 1.0 V / 200 ohm = 10.00 mA R5 = 200 ohm"
- note removed: "AD8221: V(lux)_{PD} = 4096 mV - ( I_{PD} * RS1 ) I_{PD} = 1.2 mA R_{PD} = 3K4 ohm V = 1.2 mA * 3413 ohm = 4096 mV V = 1.2 mA * 3400 ohm = 4080 mV"
- note removed: "AD8221: V(lux)_{PD} = 4096 mV - ( I_{PD} * RS1 ) I_{PD} = 1.5 mA R_{PD} = 2k67 ohm V = 1.5 mA * 2730.~{6} ohm = 4096 mV V = 1.5 mA * 2670 ohm = 4005 mV"
- note removed: "RS2 & RS5: Per datasheet: R_{G} = (49.4 Kohm) / (G-1) ex. R_{G} Gain V(PD) inf 1.000 5.0 226 k 1.218 4.096 <--- 49.9 k 1.990 2.5 12.4 k 4.984 1.0 <--- 5.49 k 9.998 0.5 2.61 k 19.93 1.00 k 50.40 499 100.0 249 199.4 100 495.0 49.9 991.0"
- note removed: "V_{S} = 5 v V_{out} = 3.3 v V = 5 v - 3.3 v = 1.7 v R_{BIAS}(I_{L_min (1PD)}) = 1.7 v / 1.3 mA = 1308 ohm R_{BIAS}(I_{L_min (2PD)}) = 1.7 v / 2.5 mA = 680 ohm R_{BIAS}(I_{L_max}) = 1.7 v / 10.0 mA = 170 ohm R_{BIAS} = 169 ohm L = 1.7 V / 169 ohm = 10.06 mA R5 = 169 ohm"
- moved on the sheet: CS1, CS10, CS2, CS3, CS4, CS5, CS6, CS7, CS8, CS9, JP16, JPV1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

Commit message: SpectDrone Development
Parts:
- R10: value R -> X
- R5: value 100 -> 174
- U13: value ADR5045B -> X
- U9: value ADR5043B -> LM4040B
Other:
- note added: "3.3 +/- 0.0066 mV"
- note added: "ADR5045B"
- note added: "V_{S} = 5 v V_{out} = 3.0 v V = 5 v - 3.0 v = 2.0 v R_{BIAS}(I_{L_min (1PD)}) = 2.0 v / 1.3 mA = 1538 ohm R_{BIAS}(I_{L_min (2PD)}) = 2.0 v / 2.5 mA = 800 ohm R_{BIAS}(I_{L_max}) = 2.0 v / 10.0 mA = 200 ohm R_{BIAS} = 200 ohm L = 2.0 V / 200 ohm = 10.00 mA R5 = 200 ohm"
- note added: "V_{S} = 5 v V_{out} = 3.3 v V = 5 v - 3.3 v = 1.7 v R_{BIAS}(I_{L_min (1PD)}) = 1.7 v / 1.3 mA = 1308 ohm R_{BIAS}(I_{L_min (2PD)}) = 1.7 v / 2.5 mA = 680 ohm R_{BIAS}(I_{L_max}) = 1.7 v / 10.0 mA = 170 ohm R_{BIAS} = 170 ohm L = 1.7 V / 174 ohm = 9.77 mA R5 = 174 ohm"
- note removed: "3 +/- 0.003 mV"
- note removed: "V_{S} = 5 v V_{out} = 3.0 v V = 5 v - 3.0 v = 2.0 v R_{BIAS}(I_{L_min (1PD)}) = 2.0 v / 1.3 mA = 1538 ohm R_{BIAS}(I_{L_min (2PD)}) = 2.0 v / 2.5 mA = 800 ohm R_{BIAS}(I_{L_max}) = 2.0 v / 10.0 mA = 200 ohm R_{BIAS} = 200 ohm L = 1.0 V / 200 ohm = 10.00 mA R5 = 200 ohm"
Changed lines of the file:
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@@
     (stroke (width 0) (type default) (color 0 0 0 0))
   )
-  (polyline (pts (xy 97.79 46.355) (xy 97.79 102.235))
+  (polyline (pts (xy 98.425 46.355) (xy 98.425 102.235))
     (stroke (width 0) (type default) (color 0 0 0 0))
   )
@@
     (stroke (width 0) (type default) (color 0 0 0 0))
   )
+  (polyline (pts (xy 215.265 151.765) (xy 215.265 125.095))
+    (stroke (width 0) (type default) (color 0 0 0 0))
+  )
   (wire (pts (xy 224.155 40.005) (xy 226.695 40.005))
     (stroke (width 0) (type default) (color 0 0 0 0))
@@
     (stroke (width 0) (type default) (color 0 0 0 0))
   )
+  (polyline (pts (xy 268.605 125.095) (xy 215.265 151.765))
+    (stroke (width 0) (type default) (color 0 0 0 0))
+  )
   (wire (pts (xy 79.375 59.055) (xy 86.995 59.055))
     (stroke (width 0) (type default) (color 0 0 0 0))
@@
     (stroke (width 0) (type default) (color 0 0 0 0))
   )
+  (polyline (pts (xy 268.605 125.095) (xy 268.605 151.765))
+    (stroke (width 0) (type default) (color 0 0 0 0))
+  )
   (wire (pts (xy 238.125 46.355) (xy 238.125 47.625))
     (stroke (width 0) (type default) (color 0 0 0 0))
@@
     (stroke (width 0) (type default) (color 0 0 0 0))
   )
+  (polyline (pts (xy 268.605 151.765) (xy 215.265 151.765))
+    (stroke (width 0) (type default) (color 0 0 0 0))
+  )
   (wire (pts (xy 128.27 43.815) (xy 133.35 43.815))
     (stroke (width 0) (type default) (color 0 0 0 0))
@@
     (stroke (width 0) (type default) (color 0 0 0 0))
   )
-  (polyline (pts (xy 97.79 102.235) (xy 71.12 102.235))
+  (polyline (pts (xy 98.425 102.235) (xy 71.12 102.235))
     (stroke (width 0) (type default) (color 0 0 0 0))
   )
@@
     (stroke (width 0) (type default) (color 0 0 0 0))
   )
+  (polyline (pts (xy 215.265 125.095) (xy 268.605 125.095))
+    (stroke (width 0) (type default) (color 0 0 0 0))
+  )
   (wire (pts (xy 234.315 69.215) (xy 238.125 69.215))
     (stroke (width 0) (type default) (color 0 0 0 0))
@@
     (stroke (width 0) (type default) (color 0 0 0 0))
   )
+  (polyline (pts (xy 215.265 125.095) (xy 268.605 151.765))
+    (stroke (width 0) (type default) (color 0 0 0 0))
+  )
   (polyline (pts (xy 95.885 128.27) (xy 95.885 147.32))
     (stroke (width 0) (type default) (color 0 0 0 0))
@@
     (stroke (width 0) (type default) (color 0 0 0 0))
   )
-  (polyline (pts (xy 71.12 46.355) (xy 97.79 46.355))
+  (polyline (pts (xy 71.12 46.355) (xy 98.425 46.355))
     (stroke (width 0) (type default) (color 0 0 0 0))
   )
@@
     (effects (font (size 1.27 1.27)) (justify left bottom))
   )
-  (text "1 +/- 0.0035 mV" (at 262.255 38.1 0)
-    (effects (font (size 1.27 1.27)) (justify left bottom))
-  )
-  (text "3 +/- 0.003 mV" (at 261.62 73.025 0)
+  (text "ADR5045B" (at 239.395 88.9 0)
+    (effects (font (size 1.27 1.27)) (justify left bottom))
+  )
+  (text "1 +/- 0.0035 mV" (at 257.175 38.1 0)
+    (effects (font (size 1.27 1.27)) (justify left bottom))
+  )
+  (text "3.3 +/- 0.0066 mV" (at 257.175 73.025 0)
     (effects (font (size 1.27 1.27)) (justify left bottom))
   )
@@
     (effects (font (size 1.27 1.27)) (justify left bottom))
   )
+  (text "\nV_{S} = 5 v\nV_{out} = 3.0 v\n\nV = 5 v - 3.0 v = 2.0 v\n\nR_{BIAS}(I_{L_min (1PD)}) = 2.0 v /  1.3 mA = 1538 ohm\nR_{BIAS}(I_{L_min (2PD)}) = 2.0 v /  2.5 mA =  800 ohm\nR_{BIAS}(I_{L_max}) = 2.0 v / 10.0 mA = 200 ohm\n\nR_{BIAS} = 200 ohm\nL = 2.0 V / 200 ohm = 10.00 mA\nR5 = 200 ohm"
+    (at 217.805 150.495 0)
+    (effects (font (size 1.27 1.27)) (justify left bottom))
+  )
   (text "AD8221:\n\nV(lux)_{PD} = 1000 mV - ( I_{PD} * RS1 )\n\nI_{PD} = 1 mA\nR_{PD} = 1K0 ohm\nV = 1 mA * 1000 ohm = 1000 mV\n "
     (at 19.05 124.46 0)
@@
     (effects (font (size 1.27 1.27)) (justify left bottom))
   )
-  (text "\nV_{S} = 5 v\nV_{out} = 3.0 v\n\nV = 5 v - 3.0 v = 2.0 v\n\nR_{BIAS}(I_{L_min (1PD)}) = 2.0 v /  1.3 mA = 1538 ohm\nR_{BIAS}(I_{L_min (2PD)}) = 2.0 v /  2.5 mA =  800 ohm\nR_{BIAS}(I_{L_max}) = 2.0 v / 10.0 mA = 200 ohm\n\nR_{BIAS} = 200 ohm\nL = 1.0 V / 200 ohm = 10.00 mA\nR5 = 200 ohm"
+  (text "\nV_{S} = 5 v\nV_{out} = 3.3 v\n\nV = 5 v - 3.3 v = 1.7 v\n\nR_{BIAS}(I_{L_min (1PD)}) = 1.7 v /  1.3 mA = 1308 ohm\nR_{BIAS}(I_{L_min (2PD)}) = 1.7 v /  2.5 mA =  680 ohm\nR_{BIAS}(I_{L_max}) = 1.7 v / 10.0 mA = 170 ohm\n\nR_{BIAS} = 170 ohm\nL = 1.7 V / 174 ohm = 9.77 mA\nR5 = 174 ohm"
     (at 162.56 118.745 0)
     (effects (font (size 1.27 1.27)) (justify left bottom))
@@
     (in_bom yes) (on_board yes)
     (property "Reference" "R5" (id 0) (at 230.505 65.405 90))
-    (property "Value" "100" (id 1) (at 230.505 69.215 90))
+    (property "Value" "174" (id 1) (at 230.505 69.215 90))
     (property "Footprint" "Capacitor_SMD:C_0805_2012Metric" (id 2) (at 230.505 70.993 90)
       (effects (font (size 1.27 1.27)) hide)
@@
   (symbol (lib_id "Device:R") (at 96.52 84.455 0) (unit 1)
     (in_bom yes) (on_board yes)
-    (property "Reference" "R_{PD}2" (id 0) (at 97.79 84.455 0)
+    (property "Reference" "R_{PD}2" (id 0) (at 90.805 81.28 0)
       (effects (font (size 1.27 1.27)) (justify left))
     )
@@
   (symbol (lib_id "Device:R") (at 96.52 53.975 0) (unit 1)
     (in_bom yes) (on_board yes)
-    (property "Reference" "R_{PD}1" (id 0) (at 97.79 53.975 0)
+    (property "Reference" "R_{PD}1" (id 0) (at 90.805 50.8 0)
       (effects (font (size 1.27 1.27)) (justify left))
     )
@@
     (in_bom yes) (on_board yes)
     (property "Reference" "R10" (id 0) (at 230.505 80.01 90))
-    (property "Value" "R" (id 1) (at 230.505 82.55 90))
+    (property "Value" "X" (id 1) (at 230.505 82.55 90))
     (property "Footprint" "Resistor_SMD:R_0603_1608Metric" (id 2) (at 230.505 84.328 90)
       (effects (font (size 1.27 1.27)) hide)
@@
       (effects (font (size 1.27 1.27)) (justify right))
     )
-    (property "Value" "ADR5043B" (id 1) (at 235.585 74.295 90)
+    (property "Value" "LM4040B" (id 1) (at 235.585 74.295 90)
       (effects (font (size 1.27 1.27)) (justify right))
     )
@@
       (effects (font (size 1.27 1.27)) (justify right))
     )
-    (property "Value" "ADR5045B" (id 1) (at 236.22 88.265 90)
-      (effects (font (size 1.27 1.27)) (justify right))
-    )
+    (property "Value" "X" (id 1) (at 236.22 88.265 90)
+      (effects (font (size 1.27 1.27)) (justify right))
+    )
