File: Longwave Instrument/Longwave Instrument.kicad_sch (KiCad schematic)
At the start: 45 parts, among them U13 X, U8 ADR510, U9 LM4040B

Commit message: SpectDrone Development
Parts:
- RV1: footprint Potentiometer_THT:Potentiometer_Bourns_3296W_Vertical -> Potentiometer_THT:Potentiometer_Bourns_3296P_Horizontal
Changed lines of the file:
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@@
       (effects (font (size 1.27 1.27)) (justify right))
     )
-    (property "Footprint" "Potentiometer_THT:Potentiometer_Bourns_3296W_Vertical" (id 2) (at 254.635 43.815 0)
+    (property "Footprint" "Potentiometer_THT:Potentiometer_Bourns_3296P_Horizontal" (id 2) (at 254.635 43.815 0)
       (effects (font (size 1.27 1.27)) hide)
     )

Commit message: SpectDrone Development
Parts:
- CS1, CS6: footprint Capacitor_SMD:C_0805_2012Metric -> Capacitor_SMD:C_0603_1608Metric; Part Number (none) -> CL10C110JB8NNNC
- CS10, CS5: Part Number (none) -> CL21B104KACNNNC
- CS2, CS3, CS7, CS8: footprint Capacitor_SMD:C_0805_2012Metric -> Capacitor_SMD:C_0402_1005Metric; Part Number (none) -> CL05C010CB5NNNC
- CS4, CS9: Part Number (none) -> CL21A106KACLRNC
- JP16, JPD1, JPD2, JPD3, JPD4, JPD5, JPD6, JPV1, JPV2, JPV3, PD1, PD2, TP5v0-1, TPv1-1, TPv1-2: now left out of the parts list
- R4, R5, R9, RS2, RS3, RS5, RS6, RS7, RS8, R_{PD.bias}1, R_{PD.bias}2, R_{PD}1, R_{PD}2: footprint Capacitor_SMD:C_0805_2012Metric -> Resistor_SMD:R_0805_2012Metric

Commit message: SpectDrone Development
Parts:
- CS1, CS6: Part Number CL10C110JB8NNNC -> 06035J100FBTTR
- CS2, CS3, CS7, CS8: Part Number CL05C010CB5NNNC -> 04023J1R1PBSTR
- R4: Part Number (none) -> ERJ-6ENF4020V
- R5: Part Number (none) -> ERJ-6ENF1740V
- R9: Part Number (none) -> ERA-6AEB474V
- RS2, RS5: value R_{G} -> R_{G}=X
- RS3, RS6, RS7, RS8: Part Number (none) -> ERJ-U6RD3300V
- RV1: Part Number (none) -> 3296P-1-103LF
- R_{PD.bias}1, R_{PD.bias}2: Part Number (none) -> ERJ-6GEY0R00V
- U13: Part Number (none) -> ADR5045BRTZ-REEL7
- U8: Part Number (none) -> ADR510ARTZ-REEL7
- U9: Part Number (none) -> LM4040B33FTA
- US1, US2: Part Number (none) -> AD8221ARMZ
Changed lines of the file:
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@@
+      (effects (font (size 1.27 1.27)) hide)
+    )
+    (property "Part Number" "AD8221ARMZ" (id 4) (at 130.81 84.455 0)
       (effects (font (size 1.27 1.27)) hide)
     )
@@
       (effects (font (size 1.27 1.27)) hide)
     )
+    (property "Part Number" "AD8221ARMZ" (id 4) (at 130.81 53.975 0)
+      (effects (font (size 1.27 1.27)) hide)
+    )
     (pin "1")
     (pin "2")
@@
       (effects (font (size 1.27 1.27)) hide)
     )
-    (property "Part Number" "CL05C010CB5NNNC" (id 4) (at 111.76 43.815 0)
+    (property "Part Number" "04023J1R1PBSTR" (id 4) (at 111.76 43.815 0)
       (effects (font (size 1.27 1.27)) hide)
     )
@@
       (effects (font (size 1.27 1.27)) hide)
     )
+    (property "Part Number" "ERJ-6ENF1740V" (id 4) (at 230.505 69.215 0)
+      (effects (font (size 1.27 1.27)) hide)
+    )
     (pin "1")
     (pin "2")
@@
       (effects (font (size 1.27 1.27)) (justify left))
     )
-    (property "Value" "R_{G}" (id 1) (at 115.57 54.61 0)
+    (property "Value" "R_{G}=X" (id 1) (at 115.57 54.61 0)
       (effects (font (size 1.27 1.27)) (justify left))
     )
@@
       (effects (font (size 1.27 1.27)) hide)
     )
+    (property "Part Number" "ERJ-U6RD3300V" (id 4) (at 102.87 59.055 0)
+      (effects (font (size 1.27 1.27)) hide)
+    )
     (pin "1")
     (pin "2")
@@
     )
     (property "Datasheet" "~" (id 3) (at 96.52 64.135 0)
+      (effects (font (size 1.27 1.27)) hide)
+    )
+    (property "Part Number" "ERJ-6GEY0R00V" (id 4) (at 96.52 64.135 0)
       (effects (font (size 1.27 1.27)) hide)
     )
@@
       (effects (font (size 1.27 1.27)) hide)
     )
+    (property "Part Number" "ERA-6AEB474V" (id 4) (at 245.5301 43.815 0)
+      (effects (font (size 1.27 1.27)) hide)
+    )
     (pin "1")
     (pin "2")
@@
       (effects (font (size 1.27 1.27)) hide)
     )
+    (property "Part Number" "ERJ-6ENF4020V" (id 4) (at 230.505 40.005 0)
+      (effects (font (size 1.27 1.27)) hide)
+    )
     (pin "1")
     (pin "2")
@@
       (effects (font (size 1.27 1.27)) hide)
     )
-    (property "Part Number" "CL05C010CB5NNNC" (id 4) (at 111.76 74.295 0)
+    (property "Part Number" "04023J1R1PBSTR" (id 4) (at 111.76 74.295 0)
       (effects (font (size 1.27 1.27)) hide)
     )
@@
       (effects (font (size 1.27 1.27)) hide)
     )
+    (property "Part Number" "3296P-1-103LF" (id 4) (at 254.635 43.815 0)
+      (effects (font (size 1.27 1.27)) hide)
+    )
     (pin "1")
     (pin "2")
@@
       (effects (font (size 1.27 1.27)) hide)
     )
-    (property "Part Number" "CL10C110JB8NNNC" (id 4) (at 109.22 53.975 0)
+    (property "Part Number" "06035J100FBTTR" (id 4) (at 109.22 53.975 0)
       (effects (font (size 1.27 1.27)) hide)
     )
@@
       (effects (font (size 1.27 1.27)) hide)
     )
+    (property "Part Number" "ERJ-U6RD3300V" (id 4) (at 102.87 48.895 0)
+      (effects (font (size 1.27 1.27)) hide)
+    )
     (pin "1")
     (pin "2")
@@
     )
     (property "Datasheet" "~" (id 3) (at 102.87 79.375 0)
+      (effects (font (size 1.27 1.27)) hide)
+    )
+    (property "Part Number" "ERJ-U6RD3300V" (id 4) (at 102.87 79.375 0)
       (effects (font (size 1.27 1.27)) hide)
     )
@@
       (effects (font (size 1.27 1.27)) (justify left))
     )
-    (property "Value" "R_{G}" (id 1) (at 115.57 85.09 0)
+    (property "Value" "R_{G}=X" (id 1) (at 115.57 85.09 0)
       (effects (font (size 1.27 1.27)) (justify left))
     )
@@
       (effects (font (size 1.27 1.27)) hide)
     )
+    (property "Part Number" "ERJ-U6RD3300V" (id 4) (at 102.87 89.535 0)
+      (effects (font (size 1.27 1.27)) hide)
+    )
     (pin "1")
     (pin "2")
@@
       (effects (font (size 1.27 1.27)) hide)
     )
-    (property "Part Number" "CL10C110JB8NNNC" (id 4) (at 109.22 84.455 0)
+    (property "Part Number" "06035J100FBTTR" (id 4) (at 109.22 84.455 0)
       (effects (font (size 1.27 1.27)) hide)
     )
@@
     )
     (property "Datasheet" "~" (id 3) (at 96.52 94.615 0)
+      (effects (font (size 1.27 1.27)) hide)
+    )
+    (property "Part Number" "ERJ-6GEY0R00V" (id 4) (at 96.52 94.615 0)
       (effects (font (size 1.27 1.27)) hide)
     )
@@
       (effects (font (size 1.27 1.27)) hide)
     )
-    (property "Part Number" "CL05C010CB5NNNC" (id 4) (at 109.22 94.615 0)
+    (property "Part Number" "04023J1R1PBSTR" (id 4) (at 109.22 94.615 0)
       (effects (font (size 1.27 1.27)) hide)
     )
@@
     (property "Datasheet" "http://www.cj-elec.com/txUpfile/20134181474991806.pdf" (id 3) (at 238.125 73.025 0)
       (effects (font (size 1.27 1.27) italic) hide)
+    )
+    (property "Part Number" "LM4040B33FTA" (id 4) (at 238.125 73.025 0)
+      (effects (font (size 1.27 1.27)) hide)
     )
     (pin "1")
@@
       (effects (font (size 1.27 1.27) italic) hide)
     )
+    (property "Part Number" "ADR510ARTZ-REEL7" (id 4) (at 238.125 43.815 0)
+      (effects (font (size 1.27 1.27)) hide)
+    )
     (pin "1")
     (pin "2")
@@
       (effects (font (size 1.27 1.27) italic) hide)
     )
+    (property "Part Number" "ADR5045BRTZ-REEL7" (id 4) (at 238.125 86.995 0)
+      (effects (font (size 1.27 1.27)) hide)
+    )
     (pin "1")
     (pin "2")
@@
       (effects (font (size 1.27 1.27)) hide)
     )
-    (property "Part Number" "CL05C010CB5NNNC" (id 4) (at 109.22 64.135 0)
-      (effects (font (size 1.27 1.27)) hide)
-    )
+    (property "Part Number" "04023J1R1PBSTR" (id 4) (at 109.22 64.135 0)
+      (effects (font (size 1.27 1.27)) hide)
+    )

Commit message: SpectDrone Development
Parts:
- U9: value LM4040B -> ADR5043BRTZ; Part Number LM4040B33FTA -> ADR5043BRTZ
Changed lines of the file:
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@@
       (effects (font (size 1.27 1.27)) (justify right))
     )
-    (property "Value" "LM4040B" (id 1) (at 235.585 74.295 90)
+    (property "Value" "ADR5043BRTZ" (id 1) (at 235.585 74.295 90)
       (effects (font (size 1.27 1.27)) (justify right))
     )
@@
       (effects (font (size 1.27 1.27) italic) hide)
     )
-    (property "Part Number" "LM4040B33FTA" (id 4) (at 238.125 73.025 0)
+    (property "Part Number" "ADR5043BRTZ" (id 4) (at 238.125 73.025 0)
       (effects (font (size 1.27 1.27)) hide)
     )

Commit message: SpectDrone Development
Parts:
- R5: value 174 -> 200
Other:
- note added: "3.0 +/- 0.0030 mV"
- note removed: "3.3 +/- 0.0066 mV"
Changed lines of the file:
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@@
     (stroke (width 0) (type default) (color 0 0 0 0))
   )
-  (polyline (pts (xy 268.605 125.095) (xy 215.265 151.765))
+  (polyline (pts (xy 213.36 93.345) (xy 160.02 120.015))
     (stroke (width 0) (type default) (color 0 0 0 0))
   )
@@
     (stroke (width 0) (type default) (color 0 0 0 0))
   )
-  (polyline (pts (xy 215.265 125.095) (xy 268.605 151.765))
+  (polyline (pts (xy 160.02 93.345) (xy 213.36 120.015))
     (stroke (width 0) (type default) (color 0 0 0 0))
   )
@@
     (effects (font (size 1.27 1.27)) (justify left bottom))
   )
-  (text "3.3 +/- 0.0066 mV" (at 257.175 73.025 0)
+  (text "3.0 +/- 0.0030 mV" (at 257.175 73.025 0)
     (effects (font (size 1.27 1.27)) (justify left bottom))
   )
@@
     (in_bom yes) (on_board yes)
     (property "Reference" "R5" (id 0) (at 230.505 65.405 90))
-    (property "Value" "174" (id 1) (at 230.505 69.215 90))
+    (property "Value" "200" (id 1) (at 230.505 69.215 90))
     (property "Footprint" "Resistor_SMD:R_0805_2012Metric" (id 2) (at 230.505 70.993 90)
       (effects (font (size 1.27 1.27)) hide)
@@
       (effects (font (size 1.27 1.27) italic) hide)
     )
-    (property "Datasheet" "http://www.cj-elec.com/txUpfile/20134181474991806.pdf" (id 3) (at 238.125 73.025 0)
+    (property "Datasheet" "https://www.analog.com/media/en/technical-documentation/data-sheets/ADR5040_5041_5043_5044_5045.pdf" (id 3) (at 238.125 73.025 0)
       (effects (font (size 1.27 1.27) italic) hide)
     )

Commit message: SpectDrone Development
Parts:
- R5: value 200 -> 174
- U9: value ADR5043BRTZ -> LM4040B
Changed lines of the file:
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@@
     (in_bom yes) (on_board yes)
     (property "Reference" "R5" (id 0) (at 230.505 65.405 90))
-    (property "Value" "200" (id 1) (at 230.505 69.215 90))
+    (property "Value" "174" (id 1) (at 230.505 69.215 90))
     (property "Footprint" "Resistor_SMD:R_0805_2012Metric" (id 2) (at 230.505 70.993 90)
       (effects (font (size 1.27 1.27)) hide)
@@
       (effects (font (size 1.27 1.27)) (justify right))
     )
-    (property "Value" "ADR5043BRTZ" (id 1) (at 235.585 74.295 90)
-      (effects (font (size 1.27 1.27)) (justify right))
-    )
+    (property "Value" "LM4040B" (id 1) (at 235.585 74.295 90)
+      (effects (font (size 1.27 1.27)) (justify right))
+    )

Commit message: SpectDrone Development
Parts:
- R10, RS2, RS5, R_{PD}1, R_{PD}2, U13: now left out of the parts list
Changed lines of the file:
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@@
   )
   (symbol (lib_id "Device:R") (at 114.3 53.975 0) (unit 1)
-    (in_bom yes) (on_board yes)
+    (in_bom no) (on_board yes)
     (property "Reference" "RS2" (id 0) (at 115.57 52.705 0)
       (effects (font (size 1.27 1.27)) (justify left))
@@
   )
   (symbol (lib_id "Device:R") (at 96.52 84.455 0) (unit 1)
-    (in_bom yes) (on_board yes)
+    (in_bom no) (on_board yes)
     (property "Reference" "R_{PD}2" (id 0) (at 90.805 81.28 0)
       (effects (font (size 1.27 1.27)) (justify left))
@@
   )
   (symbol (lib_id "Device:R") (at 96.52 53.975 0) (unit 1)
-    (in_bom yes) (on_board yes)
+    (in_bom no) (on_board yes)
     (property "Reference" "R_{PD}1" (id 0) (at 90.805 50.8 0)
       (effects (font (size 1.27 1.27)) (justify left))
@@
   )
   (symbol (lib_id "Device:R") (at 114.3 84.455 0) (unit 1)
-    (in_bom yes) (on_board yes)
+    (in_bom no) (on_board yes)
     (property "Reference" "RS5" (id 0) (at 115.57 83.185 0)
       (effects (font (size 1.27 1.27)) (justify left))
@@
   )
   (symbol (lib_id "Device:R") (at 230.505 82.55 270) (mirror x) (unit 1)
-    (in_bom yes) (on_board yes)
+    (in_bom no) (on_board yes)
     (property "Reference" "R10" (id 0) (at 230.505 80.01 90))
     (property "Value" "X" (id 1) (at 230.505 82.55 90))
@@
   )
   (symbol (lib_id "Gardenuino_Custom:ADR510") (at 238.125 86.995 270) (mirror x) (unit 1)
-    (in_bom yes) (on_board yes)
+    (in_bom no) (on_board yes)
     (property "Reference" "U13" (id 0) (at 236.22 85.725 90)
       (effects (font (size 1.27 1.27)) (justify right))

Commit message: SpectDrone Development
Parts:
- R4: value 402 -> 250; Part Number ERJ-6ENF4020V -> ERJ-PB6B2490V
- R5: value 174 -> 91; Part Number ERJ-6ENF1740V -> CRCW080591R0FKEAHP
- U8: value ADR510 -> ADR5041B
- U9: value LM4040B -> ADR5044B
Connections:
- net 5V0: now also JP16.4 (B); no longer JP16.3 (B)
- net 5V3: no longer JP16.4 (B)
- net 1V1 renamed 2V5
- net 2V5: now also JP16.3 (B)
- net 3V0 renamed 4V0
Other:
- note added: "2.500V +/- 2.5mV"
- note added: "4.096V +/- 4.1mV"
- note added: "5.000V +/- 5.0mV"
- note removed: "1 +/- 0.0035 mV"
- note removed: "3.0 +/- 0.0030 mV"
- moved on the sheet: CS1, CS10, CS2, CS3, CS4, CS5, CS6, CS7, CS8, CS9, JP16, JPD1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
