File: SpectDroneControl/SpectDroneControl.kicad_pcb (KiCad board)
At the start: 2 copper layers, 101.7 x 73.7 mm, 24 parts, among them J1 Conn_02x03_Counter_Clockwise, J1-1 Conn_01x04_Male, J1-2 Conn_01x04_Male, U1 Teensy4.1, U2 Teensy4.0

Commit message: SpectDrone Development
Parts:
- added R1: 10K, Resistor_SMD:R_0603_1608Metric, F.Cu at (172.3, 93.3)
- added SW1: SW_SPDT, Button_Switch_SMD:SW_SPDT_CK-JS102011SAQN, F.Cu at (172.3, 82.2)
- U2: footprint Teensy:Teensy30_31_32_LC -> Teensy:Teensy40
Connections:
- U1 pad 10: /RX -> /APCRX
- U1 pad 11: /APCTX -> /TX
- U1 pad 12: /APCRX -> /RX
- U1 pad 17: /UT1 -> unconnected-(U1-Pad17)
- U1 pad 26: unconnected-(U1-Pad26) -> /RX8
- U1 pad 27: unconnected-(U1-Pad27) -> /TX8
- U1 pad 28: unconnected-(U1-Pad28) -> /CS3
- U1 pad 29: unconnected-(U1-Pad29) -> /CS2
- U1 pad 34: unconnected-(U1-Pad34) -> /GND
- U1 pad 5: /GAIN -> /ST
- U1 pad 6: /ST -> /CLK1
- U1 pad 7: /CLK1 -> /UT2
- U1 pad 8: /UT2 -> /UT1
- U1 pad 9: /TX -> /APCTX
- U2 pad 10: /RX -> /APCRX
- U2 pad 11: /APCTX -> /TX
- U2 pad 12: /APCRX -> /RX
- U2 pad 17: unconnected-(U2-Pad17) -> /GND
- U2 pad 34: unconnected-(U2-Pad34) -> (no net)
- U2 pad 5: /GAIN -> /ST
- U2 pad 6: /ST -> /CLK1
- U2 pad 7: /CLK1 -> /UT2
- U2 pad 8: /UT2 -> /UT1
- U2 pad 9: /TX -> /APCTX
Routing:
- net /GND: track 13.4 -> 60.8 mm, vias 0 -> 1
- net /GAIN: track 44.6 -> 6.90 mm
- net /UT1: track 74.9 -> 58.2 mm
- net /TX: track 10.7 -> 21.1 mm
- net Net-(SW1-Pad2): track 0.00 -> 7.60 mm
- net /RX: track 16.5 -> 23.7 mm
- net /PPS: track 56.9 -> 64.0 mm
- net /VBat: track 74.5 -> 71.6 mm
- net /SCK: track 40.7 -> 38.7 mm
- net /APCRX: track 16.8 -> 18.4 mm
- net /ST: track 45.7 -> 47.1 mm
- net /APCTX: track 10.7 -> 12.0 mm
- net /UT2: track 26.0 -> 25.3 mm
- net /A2: track 41.9 -> 41.3 mm
Other:
- board text added: "5V"
- board text added: "CS"
- board text added: "GND"
- board text added: "MISO"
- board text added: "MOSI"
- board text added: "RX"
- board text added: "SCK"
- board text added: "TX"

Commit message: SpectDrone Development
Routing:
- net /TX: track 21.1 -> 20.5 mm
- net /APCRX: track 18.4 -> 17.8 mm

Commit message: SpectDrone Development
Parts:
- added R10: R, Resistor_SMD:R_0805_2012Metric, F.Cu at (210.4, 103.4)
- added R11: R, Resistor_SMD:R_0805_2012Metric, F.Cu at (210.4, 98.4)
- added R12: R, Resistor_SMD:R_0805_2012Metric, F.Cu at (210.4, 93.3)
- added R13: R, Resistor_SMD:R_0805_2012Metric, F.Cu at (210.4, 88.3)
- added R14: R, Resistor_SMD:R_0805_2012Metric, B.Cu at (184.8, 104.5)
- added R15: R, Resistor_SMD:R_0805_2012Metric, B.Cu at (182.8, 104.5)
- added R16: R, Resistor_SMD:R_0805_2012Metric, B.Cu at (180.7, 104.5)
- added R17: R, Resistor_SMD:R_0805_2012Metric, B.Cu at (173.6, 112.9)
- added R18: R, Resistor_SMD:R_0805_2012Metric, B.Cu at (171.6, 112.9)
- added R19: R, Resistor_SMD:R_0805_2012Metric, B.Cu at (163.2, 106.6)
- added R2: R, Resistor_SMD:R_0805_2012Metric, B.Cu at (189.0, 112.6)
- added R20: R, Resistor_SMD:R_0805_2012Metric, B.Cu at (165.2, 106.6)
- added R21: R, Resistor_SMD:R_0805_2012Metric, B.Cu at (165.2, 110.1)
- added R22: R, Resistor_SMD:R_0805_2012Metric, B.Cu at (163.2, 110.1)
- added R23: R, Resistor_SMD:R_0805_2012Metric, F.Cu at (210.4, 83.2)
- added R24: R, Resistor_SMD:R_0805_2012Metric, F.Cu at (210.4, 78.1)
- added R25: R, Resistor_SMD:R_0805_2012Metric, F.Cu at (210.4, 73.0)
- added R26: R, Resistor_SMD:R_0805_2012Metric, F.Cu at (181.0, 41.5)
- added R27: R, Resistor_SMD:R_0805_2012Metric, F.Cu at (186.1, 41.5)
- added R28: R, Resistor_SMD:R_0805_2012Metric, F.Cu at (191.1, 41.5)
- added R29: R, Resistor_SMD:R_0805_2012Metric, F.Cu at (196.2, 41.5)
- added R3: R, Resistor_SMD:R_0805_2012Metric, B.Cu at (191.6, 92.8)
- added R30: R, Resistor_SMD:R_0805_2012Metric, F.Cu at (201.3, 41.7)
- added R31: R, Resistor_SMD:R_0805_2012Metric, F.Cu at (206.4, 41.5)
- added R32: R, Resistor_SMD:R_0805_2012Metric, B.Cu at (196.2, 84.2)
- added R33: R, Resistor_SMD:R_0805_2012Metric, B.Cu at (194.2, 84.2)
- added R34: R, Resistor_SMD:R_0805_2012Metric, B.Cu at (192.2, 84.2)
- added R35: R, Resistor_SMD:R_0805_2012Metric, B.Cu at (190.1, 84.2)
- added R36: R, Resistor_SMD:R_0805_2012Metric, B.Cu at (188.1, 84.2)
- added R37: R, Resistor_SMD:R_0805_2012Metric, B.Cu at (186.1, 84.2)
- added R38: R, Resistor_SMD:R_0805_2012Metric, B.Cu at (184.0, 84.2)
- added R39: R, Resistor_SMD:R_0805_2012Metric, B.Cu at (182.0, 84.2)
- added R4: R, Resistor_SMD:R_0805_2012Metric, B.Cu at (133.7, 110.5)
- added R40: R, Resistor_SMD:R_0805_2012Metric, B.Cu at (180.0, 84.2)
- added R41: R, Resistor_SMD:R_0805_2012Metric, F.Cu at (89.9, 105.7)
- added R42: R, Resistor_SMD:R_0805_2012Metric, F.Cu at (89.9, 110.7)
- added R43: R, Resistor_SMD:R_0805_2012Metric, F.Cu at (89.9, 115.8)
- added R44: R, Resistor_SMD:R_0805_2012Metric, F.Cu at (89.9, 120.9)
- added R45: R, Resistor_SMD:R_0805_2012Metric, F.Cu at (89.9, 126.0)
- added R46: R, Resistor_SMD:R_0805_2012Metric, F.Cu at (89.9, 131.1)
- added R47: R, Resistor_SMD:R_0805_2012Metric, F.Cu at (89.9, 136.1)
- added R48: R, Resistor_SMD:R_0805_2012Metric, F.Cu at (131.2, 146.2)
- added R49: R, Resistor_SMD:R_0805_2012Metric, F.Cu at (136.3, 146.2)
- added R5: R, Resistor_SMD:R_0805_2012Metric, F.Cu at (210.4, 128.8)
- added R50: R, Resistor_SMD:R_0805_2012Metric, F.Cu at (141.4, 146.2)
- added R51: R, Resistor_SMD:R_0805_2012Metric, B.Cu at (125.9, 105.3)
- added R52: R, Resistor_SMD:R_0805_2012Metric, B.Cu at (125.9, 107.8)
- added R53: R, Resistor_SMD:R_0805_2012Metric, B.Cu at (125.9, 110.4)
- added R54: R, Resistor_SMD:R_0805_2012Metric, B.Cu at (125.9, 112.9)
- added R55: R, Resistor_SMD:R_0805_2012Metric, B.Cu at (125.9, 115.4)
- added R56: R, Resistor_SMD:R_0805_2012Metric, B.Cu at (125.9, 118.0)
- added R57: R, Resistor_SMD:R_0805_2012Metric, B.Cu at (125.9, 120.5)
- added R58: R, Resistor_SMD:R_0805_2012Metric, B.Cu at (125.9, 123.1)
- added R59: R, Resistor_SMD:R_0805_2012Metric, B.Cu at (125.9, 125.6)
- added R6: R, Resistor_SMD:R_0805_2012Metric, F.Cu at (210.4, 123.7)
- added R60: R, Resistor_SMD:R_0805_2012Metric, B.Cu at (125.9, 128.1)
- added R7: R, Resistor_SMD:R_0805_2012Metric, F.Cu at (210.4, 118.6)
- added R8: R, Resistor_SMD:R_0805_2012Metric, F.Cu at (210.4, 113.5)
- added R9: R, Resistor_SMD:R_0805_2012Metric, F.Cu at (210.4, 108.5)
- added U3: NVT2010PW, Package_SO:TSSOP-24_4.4x7.8mm_P0.65mm, B.Cu at (183.8, 112.6)
- added U4: NVT2010PW, Package_SO:TSSOP-24_4.4x7.8mm_P0.65mm, B.Cu at (186.3, 98.2)
- added U5: NVT2010PW, Package_SO:TSSOP-24_4.4x7.8mm_P0.65mm, B.Cu at (136.5, 116.7)
- moved R1 20.6 mm to (172.3, 72.8)
- moved SW1 16.5 mm to (172.3, 65.7)
Connections:
- net /GAIN renamed /GAIN_5V
- JAPC1 pad 1: /APCTX -> /APCTX_5V
- JAPC1 pad 2: /APCRX -> /APCRX_5V
- JAPC1 pad 3: /TX -> /TX_5V
- JAPC1 pad 4: /RX -> /RX_5V
- JAUX1 pad 10: /CAM1RX -> /CAM1RX_5V
- JAUX1 pad 11: /CAM1TX -> /CAM1TX_5V
- JAUX1 pad 12: /TXS_{E} -> /TXS_{E}_5V
- JAUX1 pad 3: /MOSI -> /MOSI_5V
- JAUX1 pad 4: /SCK -> /SCK_5V
- JAUX1 pad 5: /MISO -> /MISO_5V
- JAUX1 pad 6: /SCL -> /SCL_5V
- JAUX1 pad 7: /SDA -> /SDA_5V
- JAUX1 pad 8: /CAM2RX -> /CAM2RX_5V
- JAUX1 pad 9: /CAM2TX -> /CAM2TX_5V
- JD1 pad 1: /CLK1 -> /CLK1_5V
- JD1 pad 2: /ST -> /ST_5V
- JD1 pad 4: /CLK2 -> /CLK2_5V
- JGPS1 pad 3: /GPSRX -> /GPSRX_5V
- JGPS1 pad 4: /GPSTX -> /GPSTX_5V
- JGPS1 pad 5: /PPS -> /PPS_5V
- JP5 pad 1: /SCK1 -> /CS1_5V
- JP6 pad 1: /CS1 -> /SCK1_5V
- JP7 pad 1: /MOSI1 -> /MISO1_5V
- JP8 pad 1: /MISO1 -> /MOSI1_5V
- JUT1 pad 1: /UT1 -> /UT1_5V
- JUT1 pad 2: /UT2 -> /UT2_5V
- JUT1 pad 3: unconnected-(JUT1-Pad3) -> /CAN_H_5V
- JUT1 pad 4: unconnected-(JUT1-Pad4) -> /CAN_L_5V
- U1 pad 15: unconnected-(U1-Pad15) -> /TXS_{E}
- U1 pad 33: /TXS_{E} -> unconnected-(U1-Pad33)
- U1 pad 46: unconnected-(U1-Pad46) -> /3V
- U2 pad 16: unconnected-(U2-Pad16) -> /TXS_{E}
- U2 pad 19: /TXS_{E} -> unconnected-(U2-Pad19)
- U2 pad 31: unconnected-(U2-Pad31) -> /3V
- U2 pad 34: (no net) -> unconnected-(U2-Pad34)
Routing:
- net /5V: track 23.4 -> 105.5 mm, vias 0 -> 4
- net /PPS: track 64.0 -> 0.00 mm
- net /CS1_5V: track 0.00 -> 59.2 mm
- net /SCK1_5V: track 0.00 -> 57.1 mm
- net /MISO1_5V: track 0.00 -> 56.1 mm
- net /CS3: track 0.00 -> 55.8 mm
- net /MOSI1_5V: track 0.00 -> 55.1 mm
- net /CS2: track 0.00 -> 53.8 mm
- net /GPSTX: track 42.9 -> 0.00 mm
- net /GPSRX: track 42.9 -> 0.00 mm
- net /SCK1: track 66.8 -> 35.4 mm
- net /UT1: track 58.2 -> 28.8 mm
- net /RX_5V: track 0.00 -> 27.4 mm
- net /APCTX_5V: track 0.00 -> 26.3 mm
- net /CS1: track 77.8 -> 52.3 mm
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
Commit message: SpectDrone Development
Parts:
- added R15: R, Resistor_SMD:R_0805_2012Metric, B.Cu at (186.6, 104.3)
- added R25: R, Resistor_SMD:R_0805_2012Metric, B.Cu at (193.7, 108.0)
- added R35: R, Resistor_SMD:R_0805_2012Metric, B.Cu at (196.2, 84.2)
- added R5: R, Resistor_SMD:R_0805_2012Metric, B.Cu at (185.3, 119.5)
- R10: renamed from R9; moved to B.Cu
- R11: renamed from R10; moved to B.Cu
- R12: renamed from R11; moved to B.Cu
- R13: renamed from R12; moved to B.Cu
- R14: renamed from R13; moved to B.Cu
- R26: renamed from R23; moved to B.Cu
- R27: renamed from R24; moved to B.Cu
- R28: renamed from R25; moved to B.Cu
- R29: renamed from R26; moved to B.Cu
- R30: renamed from R27; moved to B.Cu
- R31: renamed from R28; moved to B.Cu
- R32: renamed from R29; moved to B.Cu
- R33: renamed from R30; moved to B.Cu
- R34: renamed from R31; moved to B.Cu
- R45: renamed from R41; moved to B.Cu
- R46: renamed from R42; moved to B.Cu
- R47: renamed from R43; moved to B.Cu
- R48: renamed from R44; moved to B.Cu
- R49: renamed from R45; moved to B.Cu
- R50: renamed from R46; moved to B.Cu
- R51: renamed from R47; moved to B.Cu
- R52: renamed from R48; moved to B.Cu
- R53: renamed from R49; moved to B.Cu
- R54: renamed from R50; moved to B.Cu
- R6: renamed from R5; moved to B.Cu
- R7: renamed from R6; moved to B.Cu
- R8: renamed from R7; moved to B.Cu
- R9: renamed from R8; moved to B.Cu
- moved R33 78.4 mm to (139.8, 90.3), turned to 180 degrees
- moved R32 73.1 mm to (139.8, 88.0), turned to 180 degrees
- moved R34 71.1 mm to (155.1, 90.7), turned to 180 degrees
- moved R31 67.7 mm to (139.8, 85.7), turned to 180 degrees
- moved R45 63.9 mm to (153.3, 97.2), turned to 90 degrees
- moved R30 62.2 mm to (139.8, 83.2), turned to 180 degrees
- moved R51 59.7 mm to (145.9, 115.6), turned to 0 degrees
- moved R50 58.8 mm to (145.9, 113.0), turned to 0 degrees
- moved R49 58.1 mm to (145.9, 110.5), turned to 0 degrees
- moved R14 57.7 mm to (155.6, 106.0), turned to 180 degrees
- moved R47 57.5 mm to (145.9, 102.9), turned to 0 degrees
- moved R48 57.5 mm to (145.9, 108.0), turned to 0 degrees
- moved R13 56.9 mm to (155.6, 108.6), turned to 180 degrees
- moved R29 56.8 mm to (139.8, 80.6), turned to 180 degrees
- moved R12 56.3 mm to (155.6, 111.1), turned to 180 degrees
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- renumbered R14 to R16, R15 to R17, R16 to R18, R17 to R19, R18 to R20, R19 to R21, R20 to R22, R21 to R23, R22 to R24, R32 to R36, R33 to R37, R34 to R38, R35 to R39, R36 to R40, R37 to R41, R38 to R42, R39 to R43, R40 to R44, R51 to R55, R52 to R56, R53 to R57, R54 to R58, R55 to R59, R56 to R60, R57 to R61, R58 to R62, R59 to R63, R60 to R64
Connections:
- R26 pad 1: Net-(U4-Pad4) -> unconnected-(R26-Pad1)
- R27 pad 1: Net-(U4-Pad5) -> unconnected-(R27-Pad1)
- R28 pad 1: Net-(U4-Pad6) -> unconnected-(R28-Pad1)
- R36 pad 1: Net-(U4-Pad21) -> unconnected-(R36-Pad1)
- R37 pad 1: Net-(U4-Pad20) -> unconnected-(R37-Pad1)
- R38 pad 1: Net-(U4-Pad19) -> unconnected-(R38-Pad1)
- U4 pad 19: Net-(U4-Pad19) -> unconnected-(R38-Pad1)
- U4 pad 20: Net-(U4-Pad20) -> unconnected-(R37-Pad1)
- U4 pad 21: Net-(U4-Pad21) -> unconnected-(R36-Pad1)
- U4 pad 4: Net-(U4-Pad4) -> unconnected-(R26-Pad1)
- U4 pad 5: Net-(U4-Pad5) -> unconnected-(R27-Pad1)
- U4 pad 6: Net-(U4-Pad6) -> unconnected-(R28-Pad1)
Routing:
- net /3V: track 20.0 -> 209.3 mm, vias 0 -> 5
- net /TXS_{E}: track 31.3 -> 55.7 mm
- net /SCK1: track 35.4 -> 55.6 mm
- net /CLK2_5V: track 17.8 -> 35.7 mm
- net /5V: track 105.5 -> 122.6 mm, vias 4 -> 5
- net Net-(U4-Pad21): track 13.6 -> 0.00 mm
- net unconnected-(U4-Pad22): track 0.00 -> 13.4 mm
- net Net-(U4-Pad20): track 13.1 -> 0.00 mm
- net unconnected-(R36-Pad1): track 0.00 -> 12.8 mm
- net Net-(U4-Pad19): track 12.5 -> 0.00 mm
- net /GND: track 71.0 -> 83.2 mm, vias 5 -> 4
- net unconnected-(R37-Pad1): track 0.00 -> 12.2 mm
- net unconnected-(R38-Pad1): track 0.00 -> 11.6 mm
- net unconnected-(U4-Pad3): track 0.00 -> 11.6 mm
- net unconnected-(R26-Pad1): track 0.00 -> 11.1 mm
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
Commit message: SpectDrone Development
Parts:
- added C1: 0.1uF, Capacitor_SMD:C_0805_2012Metric, F.Cu at (117.5, 87.8)
- added C2: 0.1uF, Capacitor_SMD:C_0805_2012Metric, F.Cu at (117.5, 89.8)
- added C3: 10uF, Capacitor_SMD:CP_Elec_3x5.4, F.Cu at (117.4, 81.7)
- added D1: D, Diode_SMD:Nexperia_CFP3_SOD-123W, F.Cu at (109.4, 84.2)
- added J3-1: Conn_01x01_Female, Connector_Wire:SolderWire-0.1sqmm_1x01_D0.4mm_OD1mm, F.Cu at (183.0, 121.0)
- added J3-2: Conn_01x01_Female, Connector_Wire:SolderWire-0.1sqmm_1x01_D0.4mm_OD1mm, F.Cu at (188.2, 103.5)
- added J3-3: Conn_01x01_Female, Connector_Wire:SolderWire-0.1sqmm_1x01_D0.4mm_OD1mm, F.Cu at (188.2, 105.9)
- added J3-4: Conn_01x01_Female, Connector_Wire:SolderWire-0.1sqmm_1x01_D0.4mm_OD1mm, F.Cu at (185.7, 105.9)
- added J3-5: Conn_01x01_Female, Connector_Wire:SolderWire-0.1sqmm_1x01_D0.4mm_OD1mm, F.Cu at (183.1, 103.4)
- added J3V1: Conn_01x01_Male, Connector_PinHeader_2.54mm:PinHeader_1x01_P2.54mm_Vertical, B.Cu at (130.9, 87.6)
- added J5-1: Conn_01x01_Female, Connector_Wire:SolderWire-0.1sqmm_1x01_D0.4mm_OD1mm, F.Cu at (183.1, 105.9)
- added J5-2: Conn_01x01_Female, Connector_Wire:SolderWire-0.1sqmm_1x01_D0.4mm_OD1mm, F.Cu at (195.2, 87.2)
- added J5-3: Conn_01x01_Female, Connector_Wire:SolderWire-0.1sqmm_1x01_D0.4mm_OD1mm, F.Cu at (193.2, 87.2)
- added J5-4: Conn_01x01_Female, Connector_Wire:SolderWire-0.1sqmm_1x01_D0.4mm_OD1mm, F.Cu at (191.1, 87.2)
- added J5-5: Conn_01x01_Female, Connector_Wire:SolderWire-0.1sqmm_1x01_D0.4mm_OD1mm, F.Cu at (189.1, 87.2)
- added JAX1: Conn_01x01_Female, Connector_Wire:SolderWire-0.1sqmm_1x01_D0.4mm_OD1mm, F.Cu at (162.1, 75.1)
- added JAX2: Conn_01x01_Female, Connector_Wire:SolderWire-0.1sqmm_1x01_D0.4mm_OD1mm, F.Cu at (139.4, 75.1)
- added JAX3: Conn_01x01_Female, Connector_Wire:SolderWire-0.1sqmm_1x01_D0.4mm_OD1mm, F.Cu at (139.4, 95.4)
- added JBAT1: Conn_01x02_Female, Connector_Molex:Molex_Micro-Fit_3.0_43045-0200_2x01_P3.00mm_Horizontal, F.Cu at (125.3, 74.2)
- added JCRX3: Conn_01x01_Female, Connector_Wire:SolderWire-0.1sqmm_1x01_D0.4mm_OD1mm, F.Cu at (162.1, 80.1)
- added JCTX3: Conn_01x01_Female, Connector_Wire:SolderWire-0.1sqmm_1x01_D0.4mm_OD1mm, F.Cu at (162.1, 77.6)
- added JDC1: Barrel_Jack, Connector_BarrelJack:BarrelJack_Horizontal, F.Cu at (113.4, 77.1)
- added JPPS1: Conn_01x01_Female, Connector_Wire:SolderWire-0.1sqmm_1x01_D0.4mm_OD1mm, F.Cu at (139.4, 92.8)
- added JPPS2: Conn_01x01_Female, Connector_Wire:SolderWire-0.1sqmm_1x01_D0.4mm_OD1mm, F.Cu at (120.1, 130.2)
- added JRX6: Conn_01x01_Female, Connector_Wire:SolderWire-0.1sqmm_1x01_D0.4mm_OD1mm, F.Cu at (162.1, 92.8)
- added JRX8: Conn_01x01_Female, Connector_Wire:SolderWire-0.1sqmm_1x01_D0.4mm_OD1mm, F.Cu at (139.4, 77.6)
- added JTX6: Conn_01x01_Female, Connector_Wire:SolderWire-0.1sqmm_1x01_D0.4mm_OD1mm, F.Cu at (162.1, 95.4)
- added JTX8: Conn_01x01_Female, Connector_Wire:SolderWire-0.1sqmm_1x01_D0.4mm_OD1mm, F.Cu at (139.4, 80.1)
- added JVIN1: Conn_01x01_Male, Connector_PinHeader_2.54mm:PinHeader_1x01_P2.54mm_Vertical, B.Cu at (187.3, 72.5)
- added Q1: FDN340P, Package_TO_SOT_SMD:SOT-23, F.Cu at (113.5, 82.4)
- added R65: 100K, Capacitor_SMD:C_0805_2012Metric, F.Cu at (117.5, 85.7)
- added TP1: TestPoint, TestPoint:TestPoint_Keystone_5000-5004_Miniature, F.Cu at (131.1, 67.4)
- added TP2: TestPoint, TestPoint:TestPoint_Keystone_5000-5004_Miniature, F.Cu at (131.1, 71.4)
- added TP3: TestPoint, TestPoint:TestPoint_Keystone_5000-5004_Miniature, F.Cu at (131.1, 75.2)
- added TP4: TestPoint, TestPoint:TestPoint_Keystone_5000-5004_Miniature, F.Cu at (131.2, 79.1)
- added U6: MCP112-450E/TO, Package_TO_SOT_SMD:SOT-89-3, F.Cu at (113.2, 86.7)
- added U7: LM7805_SOT223, Package_TO_SOT_SMD:SOT-223-3_TabPin2, F.Cu at (123.8, 84.5)
- BT1: footprint Battery:BatteryHolder_Keystone_103_1x20mm -> Battery:BatteryHolder_Keystone_3000_1x12mm
- moved R16 12.9 mm to (172.6, 99.4), turned to 180 degrees
- moved R18 12.7 mm to (172.6, 94.4), turned to 180 degrees
- moved R17 12.3 mm to (172.6, 96.9), turned to 180 degrees
- moved BT1 8.53 mm to (109.9, 99.9), turned to -90 degrees
- moved R15 3.64 mm to (187.3, 107.8), turned to 0 degrees
- moved R3 1.53 mm to (191.5, 94.4)
- moved R29 1.52 mm to (139.8, 82.2)
- moved R30 1.02 mm to (139.8, 84.2)
- moved R21 0.71 mm to (163.8, 106.2)
- moved R24 0.71 mm to (163.8, 109.8)
- moved R22 0.71 mm to (165.9, 106.2)
- moved R23 0.71 mm to (165.9, 109.8)
- moved R31 0.51 mm to (139.8, 86.2)
- moved R32 0.25 mm to (139.8, 88.3)
- renumbered R47 to R46, R46 to R47
Connections:
- BT1 pad 2: /GND -> GND1
- JAUX1 pad 2: /GND -> GND1
- JGPS1 pad 2: /GND -> GND1
- JP1 pad 1: /GND -> GND1
- R15 pad 1: unconnected-(U3-Pad22) -> Net-(R15-Pad1)
- R25 pad 1: unconnected-(U4-Pad3) -> /CAN_H
- R26 pad 1: unconnected-(R26-Pad1) -> /CAN_L
- R27 pad 1: unconnected-(R27-Pad1) -> /TX6
- R28 pad 1: unconnected-(R28-Pad1) -> /RX6
- R35 pad 1: unconnected-(U4-Pad22) -> /CAN_H_5V
- R36 pad 1: unconnected-(R36-Pad1) -> /CAN_L_5V
- R37 pad 1: unconnected-(R37-Pad1) -> /TX6_5V
- R38 pad 1: unconnected-(R38-Pad1) -> /RX6_5V
- R5 pad 1: unconnected-(U3-Pad3) -> Net-(R5-Pad1)
- SW1 pad 3: /GND -> GND1
- U1 pad 1: /GND -> GND1
- U1 pad 16: unconnected-(U1-Pad16) -> /TX6
- U1 pad 17: unconnected-(U1-Pad17) -> /RX6
- U1 pad 22: unconnected-(U1-Pad22) -> /CAN_H
- U1 pad 23: unconnected-(U1-Pad23) -> /CAN_L
- U1 pad 24: unconnected-(U1-Pad24) -> Net-(U1-Pad24)
- U1 pad 25: unconnected-(U1-Pad25) -> Net-(U1-Pad25)
- U1 pad 33: unconnected-(U1-Pad33) -> Net-(U1-Pad33)
- U1 pad 34: /GND -> GND1
- U1 pad 47: /GND -> GND1
- U1 pad 52: unconnected-(U1-Pad52) -> GND1
- U2 pad 1: /GND -> GND1
- U2 pad 17: /GND -> GND1
- U2 pad 32: /GND -> GND1
- U3 pad 1: /GND -> GND1
- U3 pad 22: unconnected-(U3-Pad22) -> Net-(R15-Pad1)
- U3 pad 3: unconnected-(U3-Pad3) -> Net-(R5-Pad1)
- U4 pad 1: /GND -> GND1
- U4 pad 19: unconnected-(R38-Pad1) -> /RX6_5V
- U4 pad 20: unconnected-(R37-Pad1) -> /TX6_5V
- U4 pad 21: unconnected-(R36-Pad1) -> /CAN_L_5V
- U4 pad 22: unconnected-(U4-Pad22) -> /CAN_H_5V
- U4 pad 3: unconnected-(U4-Pad3) -> /CAN_H
- U4 pad 4: unconnected-(R26-Pad1) -> /CAN_L
- U4 pad 5: unconnected-(R27-Pad1) -> /TX6
- U4 pad 6: unconnected-(R28-Pad1) -> /RX6
- U5 pad 1: /GND -> GND1
Routing:
- net GND1: track 0.00 -> 111.3 mm, vias 0 -> 2
- net /VDC: track 0.00 -> 94.3 mm
- net /GND: track 83.2 -> 0.00 mm, vias 4 -> 0
- net /CAN_L: track 0.00 -> 64.1 mm, vias 0 -> 1
- net /CAN_H: track 0.00 -> 60.7 mm
- net /5V: track 122.6 -> 183.2 mm
- net /TX6: track 0.00 -> 55.2 mm
- net /3V: track 209.3 -> 259.5 mm, vias 5 -> 4
- net /RX6: track 0.00 -> 48.3 mm
- net /CAN_L_5V: track 0.00 -> 46.6 mm, vias 0 -> 1
- net /CAN_H_5V: track 0.00 -> 42.9 mm, vias 0 -> 1
- net /VBat: track 71.6 -> 109.1 mm
- net /7-12V1: track 0.00 -> 30.6 mm, vias 0 -> 2
- net /VBAT1: track 0.00 -> 20.4 mm
- net /CLK2_5V: track 35.7 -> 16.7 mm
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- added copper zone on B.Cu, net /5V
- added copper zone on F.Cu, net GND1
- removed copper zone on F.Cu, net /5V
- removed copper zone on B.Cu, net /GND
Other:
- board text added: "(3V!)"
- board text added: "(5V!)"
- board text added: "3V"
- board text added: "VDC"

Commit message: SpectDrone Development
Parts:
- added D2: HPZR-C7V0X, Diode_SMD:D_SOD-123F, F.Cu at (107.3, 78.5)
- added JCS2: Conn_01x01_Female, Connector_Wire:SolderWire-0.1sqmm_1x01_D0.4mm_OD1mm, F.Cu at (90.0, 83.8)
- added JCS3: Conn_01x01_Female, Connector_Wire:SolderWire-0.1sqmm_1x01_D0.4mm_OD1mm, F.Cu at (93.7, 83.8)
- added Q2: Q_NPN_EBC, Package_TO_SOT_SMD:SOT-323_SC-70, F.Cu at (106.3, 84.2)
- added R66: 1K, Capacitor_SMD:C_0805_2012Metric, F.Cu at (106.3, 81.8)
- added REF**: PinHeader_Corner, Gardenuino Custom:PinHeader_Corner, B.Cu at (199.0, 116.5)
- added TP5: TestPoint, TestPoint:TestPoint_Keystone_5000-5004_Miniature, F.Cu at (131.2, 83.7)
- added TP6: TestPoint, TestPoint:TestPoint_Keystone_5000-5004_Miniature, F.Cu at (131.2, 75.6)
- J1: moved to F.Cu
- moved R1 17.1 mm to (174.9, 90.9)
- moved TP1 4.19 mm to (135.3, 67.4)
- moved TP2 3.94 mm to (131.2, 67.4)
- moved TP3 3.69 mm to (131.2, 71.5)
- moved SW1 2.67 mm to (174.8, 66.9)
- moved R6 2.44 mm to (155.6, 128.8)
- moved J1 2.43 mm to (173.6, 123.6), turned to 0 degrees
- moved R10 2.41 mm to (155.6, 118.6)
- moved R12 2.41 mm to (155.6, 113.5)
- moved R13 2.41 mm to (155.6, 111.0)
- moved R14 2.41 mm to (155.6, 108.5)
- moved R7 2.41 mm to (155.6, 126.2)
- moved R8 2.41 mm to (155.6, 123.7)
- moved R9 2.41 mm to (155.6, 121.2)
- moved R11 2.41 mm to (155.6, 116.1)
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- renumbered C3 to C1, C1 to C2, C2 to C3
Connections:
- C2 pad 2: /VDC -> /7VDC
- D1 pad 2: /VDC -> /7VDC
- J1 pad 1: Net-(J1-1-Pad1) -> Net-(J1-2-Pad1)
- J1 pad 2: Net-(J1-1-Pad2) -> Net-(J1-Pad2)
- J1 pad 3: Net-(J1-1-Pad3) -> Net-(J1-Pad3)
- J1 pad 4: Net-(J1-1-Pad4) -> Net-(J1-2-Pad4)
- J1 pad 5: Net-(J1-2-Pad4) -> Net-(J1-1-Pad4)
- J1 pad 6: Net-(J1-2-Pad3) -> Net-(J1-1-Pad3)
- J1 pad 7: Net-(J1-2-Pad2) -> Net-(J1-1-Pad2)
- J1 pad 8: Net-(J1-2-Pad1) -> Net-(J1-1-Pad1)
- J1-2 pad 2: Net-(J1-2-Pad2) -> Net-(J1-Pad2)
- J1-2 pad 3: Net-(J1-2-Pad3) -> Net-(J1-Pad3)
- JP6 pad 2: Net-(J1-2-Pad3) -> Net-(J1-Pad3)
- JP7 pad 2: Net-(J1-2-Pad2) -> Net-(J1-Pad2)
- JVIN1 pad 1: /VDC -> /VIN
- R65 pad 2: /VDC -> /7VDC
- TP3 pad 1: /5V3 -> /VIN
- TP4 pad 1: /3V -> /5V3
- U6 pad 2: /VDC -> /7VDC
Routing:
- net /VIN: track 0.00 -> 61.6 mm
- net /VDC: track 94.3 -> 35.7 mm
- net GND1: track 111.3 -> 56.0 mm
- net /7VDC: track 0.00 -> 37.4 mm
- net /GAIN_5V: track 26.3 -> 8.26 mm
- net Net-(R1-Pad2): track 3.54 -> 20.5 mm
- net /3V: track 259.5 -> 253.0 mm
- net Net-(J1-Pad3): track 0.00 -> 5.68 mm
- net Net-(J1-Pad2): track 0.00 -> 5.68 mm
- net Net-(J1-2-Pad3): track 5.61 -> 0.00 mm
- net Net-(J1-2-Pad2): track 5.61 -> 0.00 mm
- net Net-(D2-Pad1): track 0.00 -> 4.01 mm
- net /VBAT1: track 20.4 -> 17.9 mm
- net /A2: track 44.2 -> 42.3 mm
- net /MOSI: track 43.9 -> 42.1 mm
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Other:
- board text added: "(3.3V!)"
- board text added: "3.3V"
- board text added: "7V"
- board text added: "Design by: Shawn L. Jaker shawn.jaker@nrel.gov National Renewable Energy Laboratory Solar Radiation Research Laboratory Golden, Colorado, USA"
- board text added: "Logic level voltage conversion (5v<->3.3v)"
- board text added: "VIN"
- board text removed: "(3V!)"
- board text removed: "3V"

Commit message: SpectDrone Development
Parts:
- JCS2, JCS3: moved to B.Cu
- moved JCS2 104.2 mm to (181.2, 134.2), turned to 180 degrees
- moved JCS3 98.8 mm to (178.7, 134.2), turned to 180 degrees
Routing:
- net /CS2_5V: track 10.5 -> 69.9 mm, vias 0 -> 1
- net /CS3_5V: track 11.1 -> 70.4 mm, vias 0 -> 1
- net /VIN: track 61.6 -> 62.4 mm
- net /CAN_L_5V: track 46.7 -> 46.2 mm
Other:
- board text added: "J2"
