File: SpectDroneControl/SpectDroneControl.kicad_pcb (KiCad board)
At the start: 2 copper layers, 101.7 x 73.7 mm, 137 parts, among them J1 Conn_02x03_Counter_Clockwise, J1-1 Conn_01x04_Male, J1-2 Conn_01x04_Male, J3-1 Conn_01x01_Female, J3-2 Conn_01x01_Female, J3-3 Conn_01x01_Female, J3-4 Conn_01x01_Female, J3-5 Conn_01x01_Female, J3V1 Conn_01x01_Male, J5-1 Conn_01x01_Female, J5-2 Conn_01x01_Female, J5-3 Conn_01x01_Female, J5-4 Conn_01x01_Female, J5-5 Conn_01x01_Female, Q1 FDN340P, Q2 Q_NPN_EBC, SW1 SW_SPDT, U1 Teensy4.1, U2 Teensy4.0, U3 NVT2010PW, U4 NVT2010PW, U5 NVT2010PW, U6 MCP112-450E/TO, U7 LM7805_SOT223

Commit message: SpectDrone Development
Parts:
- added JCAN_{H}1: Conn_01x01_Female, Connector_Wire:SolderWire-0.1sqmm_1x01_D0.4mm_OD1mm, F.Cu at (171.2, 116.6)
- added JCAN_{L}1: locked, Connector_Wire:SolderWire-0.1sqmm_1x01_D0.4mm_OD1mm, F.Cu at (173.7, 116.6)
- JCR1: renamed from REF**; value PinHeader_Corner -> Conn_01x37_Female
- moved J1 0.11 mm to (173.7, 123.6)
Connections:
- net /CAN_H renamed /CRX
- net /CAN_L renamed /CTX
- J5-2 pad 1: /CAN_H_5V -> /CRX_5V
- J5-3 pad 1: /CAN_L_5V -> /CTX_5V
- JCR1 pad 1: (no net) -> GND1
- JCR1 pad 10: (no net) -> unconnected-(JCR1-Pad10)
- JCR1 pad 11: (no net) -> unconnected-(JCR1-Pad11)
- JCR1 pad 12: (no net) -> unconnected-(JCR1-Pad12)
- JCR1 pad 13: (no net) -> unconnected-(JCR1-Pad13)
- JCR1 pad 14: (no net) -> unconnected-(JCR1-Pad14)
- JCR1 pad 15: (no net) -> unconnected-(JCR1-Pad15)
- JCR1 pad 16: (no net) -> unconnected-(JCR1-Pad16)
- JCR1 pad 17: (no net) -> unconnected-(JCR1-Pad17)
- JCR1 pad 18: (no net) -> unconnected-(JCR1-Pad18)
- JCR1 pad 19: (no net) -> unconnected-(JCR1-Pad19)
- JCR1 pad 2: (no net) -> /3V
- JCR1 pad 20: (no net) -> unconnected-(JCR1-Pad20)
- JCR1 pad 21: (no net) -> unconnected-(JCR1-Pad21)
- JCR1 pad 22: (no net) -> unconnected-(JCR1-Pad22)
- JCR1 pad 23: (no net) -> unconnected-(JCR1-Pad23)
- JCR1 pad 24: (no net) -> unconnected-(JCR1-Pad24)
- JCR1 pad 25: (no net) -> unconnected-(JCR1-Pad25)
- JCR1 pad 26: (no net) -> unconnected-(JCR1-Pad26)
- JCR1 pad 27: (no net) -> unconnected-(JCR1-Pad27)
- JCR1 pad 28: (no net) -> unconnected-(JCR1-Pad28)
- JCR1 pad 29: (no net) -> unconnected-(JCR1-Pad29)
- JCR1 pad 3: (no net) -> /5V
- JCR1 pad 30: (no net) -> unconnected-(JCR1-Pad30)
- JCR1 pad 31: (no net) -> unconnected-(JCR1-Pad31)
- JCR1 pad 32: (no net) -> unconnected-(JCR1-Pad32)
- JCR1 pad 33: (no net) -> unconnected-(JCR1-Pad33)
- JCR1 pad 34: (no net) -> unconnected-(JCR1-Pad34)
- JCR1 pad 35: (no net) -> /MOSI1_5V
- JCR1 pad 36: (no net) -> /MISO1_5V
- JCR1 pad 37: (no net) -> /SCK1_5V
- JCR1 pad 4: (no net) -> unconnected-(JCR1-Pad4)
- JCR1 pad 5: (no net) -> unconnected-(JCR1-Pad5)
- JCR1 pad 6: (no net) -> unconnected-(JCR1-Pad6)
- JCR1 pad 7: (no net) -> unconnected-(JCR1-Pad7)
- JCR1 pad 8: (no net) -> unconnected-(JCR1-Pad8)
- JCR1 pad 9: (no net) -> unconnected-(JCR1-Pad9)
- R35 pad 1: /CAN_H_5V -> /CRX_5V
- R36 pad 1: /CAN_L_5V -> /CTX_5V
- U4 pad 21: /CAN_L_5V -> /CTX_5V
- U4 pad 22: /CAN_H_5V -> /CRX_5V
Routing:
- net /CAN_L_5V: track 46.2 -> 2.54 mm, vias 1 -> 0
- net /CTX_5V: track 0.00 -> 39.3 mm, vias 0 -> 1
- net /CRX_5V: track 0.00 -> 37.0 mm, vias 0 -> 1
- net /CAN_H_5V: track 42.9 -> 6.13 mm, vias 1 -> 0
- net /CS3_5V: track 70.4 -> 80.5 mm
- net /MISO1_5V: track 59.5 -> 68.3 mm, vias 0 -> 1
- net /SCK1_5V: track 60.7 -> 68.7 mm, vias 0 -> 1
- net /CS2_5V: track 69.9 -> 76.4 mm
- net /MOSI1_5V: track 58.3 -> 64.3 mm, vias 0 -> 1
- net /5V: track 182.1 -> 183.3 mm
- net /VIN: track 62.4 -> 61.6 mm
- net (no net): vias 0 -> 1
Other:
- board text added: "CAN_{H}"
- board text added: "CAN_{L}"
- board text added: "CS1"
- board text added: "CS2"
- board text added: "CS3"
- board text added: "MISO_{B}"
- board text added: "MOSI_{B}"
- board text added: "SCK_{B}"
- board text removed: "CS"
- board text removed: "MISO"
- board text removed: "MOSI"
- board text removed: "SCK"
