File: SpectDroneControl/SpectDroneControl.kicad_pcb (KiCad board)
At the start: 2 copper layers, 101.7 x 73.7 mm, 139 parts, among them J1 Conn_02x03_Counter_Clockwise, J1-1 Conn_01x04_Male, J1-2 Conn_01x04_Male, J3-1 Conn_01x01_Female, J3-2 Conn_01x01_Female, J3-3 Conn_01x01_Female, J3-4 Conn_01x01_Female, J3-5 Conn_01x01_Female, J3V1 Conn_01x01_Male, J5-1 Conn_01x01_Female, J5-2 Conn_01x01_Female, J5-3 Conn_01x01_Female, J5-4 Conn_01x01_Female, J5-5 Conn_01x01_Female, Q1 FDN340P, Q2 Q_NPN_EBC, SW1 SW_SPDT, U1 Teensy4.1, U2 Teensy4.0, U3 NVT2010PW, U4 NVT2010PW, U5 NVT2010PW, U6 MCP112-450E/TO, U7 LM7805_SOT223

Commit message: SpectDrone Development
Parts:
- added C4: 0.1uF, Capacitor_SMD:C_0805_2012Metric, B.Cu at (112.8, 127.7)
- added C5: 0.1uF, Capacitor_SMD:C_0805_2012Metric, B.Cu at (119.8, 121.5)
- added R67: 200K, Capacitor_SMD:C_0805_2012Metric, B.Cu at (112.9, 119.9)
- added R68: 200K, Capacitor_SMD:C_0805_2012Metric, B.Cu at (112.8, 129.8)
- added U8: TXS0102DCUR, Package_SO:SSOP-8_2.95x2.8mm_P0.65mm, B.Cu at (112.8, 123.9)
- R45: value R -> X
- renumbered J1-2 to J2-1, J1-1 to J2-2
Connections:
- C1 pad 1: /5V3 -> /5V
- JCR1 pad 2: /3V -> unconnected-(JCR1-Pad2)
- JCR1 pad 3: /5V -> unconnected-(JCR1-Pad3)
- JP2 pad 1: /JRX -> /JTX
- JP3 pad 1: /JTX -> /JRX
- TP4 pad 1: /5V3 -> /5V
- U1 pad 20: /JTX -> /JRX
- U1 pad 21: /JRX -> /JTX
- U7 pad 3: /5V3 -> /5V
Routing:
- net /GPSRX: track 0.00 -> 59.8 mm
- net /GPSTX: track 0.00 -> 52.0 mm, vias 0 -> 1
- net /3V: track 253.0 -> 290.5 mm
- net /CTX_5V: track 39.3 -> 12.8 mm, vias 1 -> 0
- net /CRX_5V: track 37.0 -> 13.4 mm, vias 1 -> 0
- net GND1: track 56.0 -> 74.4 mm
- net /5V3: track 17.1 -> 0.00 mm
- net /5V: track 183.3 -> 200.3 mm
- net Net-(C5-Pad1): track 0.00 -> 9.68 mm
- net Net-(R68-Pad2): track 0.00 -> 9.09 mm
- net /GPSRX_5V: track 0.00 -> 4.21 mm
- net /GPSTX_5V: track 0.00 -> 3.85 mm
- net (no net): vias 1 -> 0

Commit message: SpectDrone Development
Parts:
- moved R45 4.44 mm to (155.6, 93.3), turned to 180 degrees
- moved BT1 3.59 mm to (106.3, 99.4)
- moved R28 1.40 mm to (193.7, 103.2)
- moved R27 1.14 mm to (193.7, 105.0)
- moved R34 0.92 mm to (155.6, 91.4)
- moved R26 0.89 mm to (193.7, 106.8)
- moved R25 0.63 mm to (193.7, 108.6)
- moved R5 0.51 mm to (185.3, 119.0), turned to 45 degrees
- moved J3-1 0.13 mm to (183.3, 121.0)
Connections:
- net Net-(J3-1-Pad1) renamed /J3_1
- net Net-(J5-1-Pad1) renamed /J5_1
Routing:
- net /VBat: track 108.6 -> 85.3 mm
- net /TXS_{E}: track 55.6 -> 62.0 mm
- net /CS2_5V: track 76.4 -> 73.0 mm
- net /MISO1_5V: track 68.3 -> 64.9 mm
- net /CS3_5V: track 80.5 -> 77.7 mm
- net /GPSTX: track 52.0 -> 53.9 mm
- net /SCK1_5V: track 68.7 -> 67.1 mm
- net /MOSI1: track 34.8 -> 33.5 mm
- net /5V: track 200.3 -> 199.0 mm
- net /MISO1: track 51.6 -> 50.5 mm
- net /CS3: track 57.5 -> 56.4 mm
- net /CS2: track 55.9 -> 54.7 mm
- net /CS1: track 55.0 -> 53.8 mm
- net /SCK1: track 54.7 -> 53.6 mm
- net /RX: track 34.6 -> 33.5 mm
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Other:
- board text added: "Spectroradiometer GAIN <-HIGH|LOW->"
- board text added: "X"

Commit message: SpectDrone Development
Parts:
- added C6: 0.1uF, Capacitor_SMD:C_0805_2012Metric, B.Cu at (190.1, 109.2)
- added C7: 0.1uF, Capacitor_SMD:C_0805_2012Metric, B.Cu at (193.3, 91.7)
- added C8: 0.1uF, Capacitor_SMD:C_0805_2012Metric, B.Cu at (134.2, 123.3)
- R10, R11, R12, R13, R14, R25, R26, R27, R28, R29, R30, R31, R32, R33, R34, R46, R47, R48, R49, R5, R50, R51, R52, R53, R54, R6, R7, R8, R9: value R -> 6K8
- R15, R16, R17, R18, R19, R20, R21, R22, R23, R24, R35, R36, R37, R38, R39, R40, R41, R42, R43, R44, R55, R56, R57, R58, R59, R60, R61, R62, R63, R64: value R -> 10K
- R2, R3, R4: value R -> 200K
- moved R15 9.96 mm to (178.7, 112.8), turned to -90 degrees
- moved C5 5.64 mm to (114.4, 123.4)
- moved JCS2 2.54 mm to (178.7, 134.2)
- moved JCS3 2.54 mm to (181.2, 134.2)
- moved R3 1.93 mm to (193.3, 93.6), turned to 0 degrees
- moved C4 1.45 mm to (111.4, 127.7)
- moved R67 1.45 mm to (111.4, 119.9)
- moved R68 1.45 mm to (111.4, 129.8)
- moved U8 1.45 mm to (111.4, 123.9)
Connections:
- R68 pad 2: Net-(R68-Pad2) -> /TXS_{E}_5V
- U8 pad 6: Net-(R68-Pad2) -> /TXS_{E}_5V
Routing:
- net /TXS_{E}_5V: track 14.0 -> 71.8 mm
- net /TXS_{E}: track 62.0 -> 41.2 mm
- net /5V: track 199.0 -> 179.1 mm
- net Net-(R4-Pad1): track 2.39 -> 12.4 mm
- net Net-(R68-Pad2): track 9.09 -> 0.00 mm
- net GND1: track 74.4 -> 83.4 mm, vias 2 -> 3
- net /J5_1: track 6.18 -> 14.0 mm
- net /CS3_5V: track 77.7 -> 72.1 mm, vias 1 -> 2
- net /GPSTX: track 53.9 -> 58.5 mm
- net Net-(C5-Pad1): track 9.68 -> 5.94 mm
- net Net-(R3-Pad1): track 2.30 -> 5.78 mm
- net /3V: track 291.5 -> 293.8 mm
- net /GPSRX: track 59.3 -> 61.6 mm
- net /S1: track 43.8 -> 41.7 mm
- net Net-(R2-Pad1): track 2.77 -> 4.42 mm
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
Commit message: SpectDrone Development
Parts:
- removed the U2 at (150.7, 116.9)
- added J5V1: Conn_01x01_Female, Gardenuino Custom:SolderWire-0.1sqmm_1x01_D0.4mm_OD1mm, F.Cu at (126.2, 133.3)
- added JA1: Conn_01x01_Female, Gardenuino Custom:SolderWire-0.1sqmm_1x01_D0.4mm_OD1mm, F.Cu at (165.2, 96.9)
- added JA2: Conn_01x01_Female, Gardenuino Custom:SolderWire-0.1sqmm_1x01_D0.4mm_OD1mm, F.Cu at (165.2, 102.0)
- added JCMR1: Conn_01x01_Female, Gardenuino Custom:SolderWire-0.1sqmm_1x01_D0.4mm_OD1mm, F.Cu at (126.2, 110.4)
- added JCMR2: Conn_01x01_Female, Gardenuino Custom:SolderWire-0.1sqmm_1x01_D0.4mm_OD1mm, F.Cu at (126.2, 115.5)
- added JCMT1: Conn_01x01_Female, Gardenuino Custom:SolderWire-0.1sqmm_1x01_D0.4mm_OD1mm, F.Cu at (126.2, 107.9)
- added JCMT2: Conn_01x01_Female, Gardenuino Custom:SolderWire-0.1sqmm_1x01_D0.4mm_OD1mm, F.Cu at (126.2, 113.0)
- added JGND1: Conn_01x01_Female, Gardenuino Custom:SolderWire-0.1sqmm_1x01_D0.4mm_OD1mm, F.Cu at (126.2, 130.7)
- added JMISO1: Conn_01x01_Female, Gardenuino Custom:SolderWire-0.1sqmm_1x01_D0.4mm_OD1mm, F.Cu at (126.2, 123.1)
- added JMOSI1: Conn_01x01_Female, Gardenuino Custom:SolderWire-0.1sqmm_1x01_D0.4mm_OD1mm, F.Cu at (126.2, 128.2)
- added JPAX1: SolderJumper, Jumper:SolderJumper-3_P1.3mm_Bridged12_RoundedPad1.0x1.5mm, F.Cu at (174.9, 88.3)
- added JS1: Conn_01x01_Female, Gardenuino Custom:SolderWire-0.1sqmm_1x01_D0.4mm_OD1mm, F.Cu at (165.2, 94.4)
- added JS2: Conn_01x01_Female, Gardenuino Custom:SolderWire-0.1sqmm_1x01_D0.4mm_OD1mm, F.Cu at (165.2, 99.4)
- added JSCK1: Conn_01x01_Female, Gardenuino Custom:SolderWire-0.1sqmm_1x01_D0.4mm_OD1mm, F.Cu at (126.2, 125.7)
- added JSCL1: Conn_01x01_Female, Gardenuino Custom:SolderWire-0.1sqmm_1x01_D0.4mm_OD1mm, F.Cu at (126.2, 120.6)
- added JSDA1: Conn_01x01_Female, Gardenuino Custom:SolderWire-0.1sqmm_1x01_D0.4mm_OD1mm, F.Cu at (126.2, 118.0)
- added JTXSE1: Conn_01x01_Female, Gardenuino Custom:SolderWire-0.1sqmm_1x01_D0.4mm_OD1mm, F.Cu at (126.2, 105.3)
- J3-1, J3-2, J3-3, J3-4, J3-5, J5-1, J5-2, J5-3, J5-4, J5-5, JAX1, JAX2, JAX3, JCAN_{H}1, JCAN_{L}1, JCRX3, JCS2, JCS3, JCTX3, JPPS1, JPPS2, JRX6, JRX8, JTX6, JTX8: footprint Connector_Wire:SolderWire-0.1sqmm_1x01_D0.4mm_OD1mm -> Gardenuino Custom:SolderWire-0.1sqmm_1x01_D0.4mm_OD1mm
- R2: renamed from R66; footprint Capacitor_SMD:C_0805_2012Metric -> Resistor_SMD:R_0805_2012Metric
- R28: renamed from R45; value X -> 6K8
- R3: renamed from R65; footprint Capacitor_SMD:C_0805_2012Metric -> Resistor_SMD:R_0805_2012Metric
- R7-1: renamed from R67; footprint Capacitor_SMD:C_0805_2012Metric -> Resistor_SMD:R_0805_2012Metric
- R7-2: renamed from R68; footprint Capacitor_SMD:C_0805_2012Metric -> Resistor_SMD:R_0805_2012Metric
- U1: footprint Teensy:Teensy41 -> Gardenuino Custom:Teensy4.0-1
- moved R38 11.6 mm to (179.5, 101.2), turned to 90 degrees
- moved R28 5.73 mm to (152.0, 97.8)
- moved R27 3.56 mm to (152.0, 91.4)
- moved R58 2.54 mm to (123.3, 105.3)
- moved R59 2.54 mm to (123.3, 107.8)
- moved R60 2.54 mm to (123.3, 110.4)
- moved R61 2.54 mm to (123.3, 112.9)
- moved R62 2.54 mm to (123.3, 115.4)
- moved R63 2.54 mm to (123.3, 118.0)
- moved R64 2.54 mm to (123.3, 120.5)
- moved R65 2.54 mm to (123.3, 123.1)
- moved R66 2.54 mm to (123.3, 125.6)
- moved R67 2.54 mm to (123.3, 128.1)
- moved R29 2.54 mm to (145.9, 102.9)
- moved R30 2.54 mm to (145.9, 105.4)
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- renumbered C1 to C2-1, C3 to C2-2, C2 to C3, C6 to C4, C7 to C5, C8 to C6, C4 to C7-1, C5 to C7-2, JA1 to JADC1, R7 to R10, R8 to R11, R9 to R12, R10 to R13, R11 to R14, R12 to R15, R13 to R16, R14 to R17, R25 to R18, R26 to R19, R27 to R20, R28 to R21, R29 to R22, R30 to R23, R31 to R24, R32 to R25, R33 to R26, R34 to R27, R47 to R29, R46 to R30, R48 to R31, R49 to R32, R50 to R33, R51 to R34, R52 to R35, R53 to R36, R54 to R37, R15 to R38, R16 to R39, R2 to R4, R17 to R40, R18 to R41, R19 to R42, R20 to R43, R21 to R44, R22 to R45, R23 to R46, R24 to R47, R35 to R48, R36 to R49, R3 to R5, R37 to R50, R38 to R51, R39 to R52, R40 to R53, R41 to R54, R42 to R55, R43 to R56, R44 to R57, R55 to R58, R56 to R59, R4 to R6, R57 to R60, R58 to R61, R59 to R62, R60 to R63, R61 to R64, R62 to R65, R63 to R66, R64 to R67, R5 to R8, R6 to R9, U7 to U2, U6 to U3, U3 to U4, U4 to U5, U5 to U6, U8 to U7
Connections:
- net Net-(JAX1-Pad1) renamed /AX1
- net Net-(JAX2-Pad1) renamed /AX2
- R1 pad 2: Net-(R1-Pad2) -> Net-(JPAX1-Pad2)
- R28 pad 2: /3V -> Net-(R28-Pad2)
- SW1 pad 2: Net-(R1-Pad2) -> Net-(SW1-Pad2)
- U6 pad 3: /TXS_{E} -> Net-(R28-Pad2)
Routing:
- net /TXS_{E}: track 41.2 -> 10.9 mm
- net Net-(R28-Pad2): track 0.00 -> 27.6 mm, vias 0 -> 2
- net Net-(R1-Pad2): track 20.5 -> 0.00 mm
- net /5V: track 179.1 -> 159.6 mm
- net Net-(SW1-Pad2): track 0.00 -> 19.1 mm
- net /3V: track 293.8 -> 274.8 mm, vias 3 -> 4
- net /AX1: track 3.72 -> 22.3 mm
- net /VBat: track 85.2 -> 92.3 mm
- net /MOSI1: track 33.5 -> 37.1 mm
- net /J5_1: track 14.0 -> 11.0 mm
- net /GPSTX: track 58.5 -> 55.7 mm
- net /CAM2TX_5V: track 8.34 -> 10.7 mm
- net /CAM1TX_5V: track 12.1 -> 14.5 mm
- net /CAM1RX_5V: track 10.2 -> 12.6 mm
- net /CAM1RX: track 18.8 -> 21.0 mm
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Other:
- board text added: "(3.3V max analog signal)"
- board text added: "(Soft/Hard)-ware Gain control"
- board text added: "CAM1RX"
- board text added: "CAM1TX"
- board text added: "CAM2RX"
- board text added: "CAM2TX"
- board text added: "MISO"
- board text added: "MOSI"
- board text added: "SCK"
- board text added: "SCL"
- board text added: "SDA"
- board text added: "TXS_{e}"

Commit message: SpectDrone Development
Parts:
- moved C7-2 0.13 mm to (114.0, 123.3)
- moved JPAX1 0.13 mm to (174.9, 88.1)
- turned C7-1 to 180 degrees
- turned R7-2 to 0 degrees
- renumbered JS1 to JPD1, JS2 to JPD2, JA1 to JSR1, JA2 to JSR2, TP6 to TP4, TP4 to TP5, TP5 to TP6
Connections:
- JADC1 pad 1: /S1 -> /P1
- JADC1 pad 2: /A1 -> /S1
- JADC1 pad 3: /S2 -> /P2
- JADC1 pad 4: /A2 -> /S2
- JPD1 pad 1: /S1 -> /P1
- JPD2 pad 1: /S2 -> /P2
- JSR1 pad 1: /A1 -> /S1
- JSR2 pad 1: /A2 -> /S2
- U1 pad 42: /S1 -> /P1
- U1 pad 43: /A1 -> /S1
- U1 pad 44: /S2 -> /P2
- U1 pad 45: /A2 -> /S2
Routing:
- net /P1: track 0.00 -> 41.7 mm
- net /A2: track 41.5 -> 0.00 mm
- net /A1: track 40.9 -> 0.00 mm
- net /P2: track 0.00 -> 40.9 mm
- net GND1: track 83.0 -> 87.8 mm
- net /TXS_{E}_5V: track 71.5 -> 76.2 mm
- net /3V: track 274.8 -> 272.3 mm
- net /S1: track 41.7 -> 40.9 mm
- net /S2: track 40.9 -> 41.5 mm
- net /MISO: track 37.4 -> 37.9 mm

Commit message: SpectDrone Development
Parts:
- added JP10: SolderJumper_2_Open, Jumper:SolderJumper-2_P1.3mm_Open_RoundedPad1.0x1.5mm, B.Cu at (168.5, 134.2)
- added JP9: SolderJumper_2_Open, Jumper:SolderJumper-2_P1.3mm_Open_RoundedPad1.0x1.5mm, B.Cu at (171.8, 134.2)
- moved BT1 3.30 mm to (109.6, 99.9)
- moved R9 0.15 mm to (155.6, 128.7)
- moved R10 0.12 mm to (155.6, 126.1)
- moved R11 0.12 mm to (155.6, 123.6)
- moved R12 0.12 mm to (155.6, 121.0)
- moved R13 0.12 mm to (155.6, 118.5)
- moved R14 0.12 mm to (155.6, 116.0)
- moved R15 0.12 mm to (155.6, 113.4)
- moved R16 0.12 mm to (155.6, 110.9)
- moved R17 0.12 mm to (155.6, 108.3)
- renumbered J2-2 to J2-1, J2-1 to J2-2
Connections:
- JP1 pad 1: GND1 -> /5V
- JP4 pad 1: /5V -> GND1
Routing:
- net /SDA: track 8.68 -> 63.2 mm, vias 0 -> 1
- net /SCL: track 7.28 -> 54.3 mm, vias 0 -> 1
- net /5V: track 159.6 -> 201.3 mm
- net GND1: track 87.8 -> 81.3 mm
- net Net-(J1-Pad6): track 5.61 -> 11.7 mm
- net Net-(JP4-Pad2): track 5.61 -> 8.88 mm
- net /VBat: track 92.3 -> 89.3 mm
- net /3V: track 272.3 -> 270.4 mm
- net /GPSTX: track 55.7 -> 57.3 mm
- net /VDC: track 35.7 -> 36.4 mm
- net /SCK: track 28.9 -> 28.2 mm
Other:
- board text added: "J2-1-3 SDA3v"
- board text added: "J2-1-4 SCL3v"

Commit message: SpectDrone Development
Parts:
- moved SW1 1.52 mm to (174.9, 68.5)
Routing:
- net /VBat: track 89.3 -> 85.8 mm
- net /5V: track 201.3 -> 198.4 mm
- net Net-(JPAX1-Pad3): track 19.0 -> 17.5 mm
Other:
- board size 101.7 x 73.7 mm -> 101.6 x 73.7 mm
- board text added: "SpectDroneControl version 0.1a"

Commit message: SpectDrone Development
Parts:
- J2-1, J2-2, JADC1, JAPC1, JUT1: footprint Connector_PinHeader_2.54mm:PinHeader_1x04_P2.54mm_Vertical -> Connector_PinSocket_2.54mm:PinSocket_1x04_P2.54mm_Vertical
- J3V1, JVIN1: footprint Connector_PinHeader_2.54mm:PinHeader_1x01_P2.54mm_Vertical -> Connector_PinSocket_2.54mm:PinSocket_1x01_P2.54mm_Vertical
- JAUX1: footprint Connector_PinHeader_2.54mm:PinHeader_1x12_P2.54mm_Vertical -> Connector_PinSocket_2.54mm:PinSocket_1x12_P2.54mm_Vertical
- JD1: value Conn_01x04_Male -> Conn_01x04_Female; footprint Connector_PinHeader_2.54mm:PinHeader_1x04_P2.54mm_Vertical -> Connector_PinSocket_2.54mm:PinSocket_1x04_P2.54mm_Vertical
- JGPS1: footprint Connector_PinHeader_2.54mm:PinHeader_1x05_P2.54mm_Vertical -> Connector_PinSocket_2.54mm:PinSocket_1x05_P2.54mm_Vertical
