File: SpectDroneControl/SpectDroneControl.kicad_pcb (KiCad board)
At the start: 2 copper layers, 101.6 x 73.7 mm, 166 parts, among them J1 Conn_02x03_Counter_Clockwise, J2-1 Conn_01x04_Female, J2-2 Conn_01x04_Female, J3-1 Conn_01x01_Female, J3-2 Conn_01x01_Female, J3-3 Conn_01x01_Female, J3-4 Conn_01x01_Female, J3-5 Conn_01x01_Female, J3V1 Conn_01x01_Female, J5-1 Conn_01x01_Female, J5-2 Conn_01x01_Female, J5-3 Conn_01x01_Female, J5-4 Conn_01x01_Female, J5-5 Conn_01x01_Female, J5V1 Conn_01x01_Female, Q1 FDN340P, Q2 NPN 50V 1A NPN_BEC, SW1 SW_SPDT, U1 Teensy4.1, U2 LM7805_SOT223, U3 MCP112-450E/TO, U4 NVT2010PW, U5 NVT2010PW, U6 NVT2010PW, U7 TXS0102DCUR

Commit message: SpectDrone Development
Routing:
- net /5V: track 202.4 -> 246.3 mm, vias 5 -> 7
- net GND1: track 81.1 -> 108.4 mm, vias 3 -> 5
- net /MOSI: track 41.1 -> 41.7 mm
- net /P2: track 40.9 -> 41.6 mm
- net /P1: track 40.9 -> 41.6 mm
- net /MISO: track 37.7 -> 38.3 mm
- net /S2: track 41.5 -> 42.2 mm
- added copper zone on In2.Cu, net /5V
- added copper zone on In1.Cu, net GND1
- removed copper zone on B.Cu, net /5V
- removed copper zone on F.Cu, net GND1
Other:
- copper layers 2 -> 4
- board text added: "CAM1RX/CS2"
- board text added: "CAM1TX/CS1"
- board text added: "CAM2/ALT_{RX}"
- board text added: "CAM2/ALT_{TX}"
- board text removed: "CAM1RX"
- board text removed: "CAM1TX"
- board text removed: "CAM2RX"
- board text removed: "CAM2TX"

Commit message: SpectDrone Development
Parts:
- D2: value HPZR-C7V0X -> HPZR-C5V6X
Connections:
- net /7-12V1 renamed Net-(D1-K)
- net /7VDC renamed Net-(D1-A)
Changed lines of the file:
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@@
   (net 86 "Net-(J1-Pin_5)")
   (net 87 "GND1")
-  (net 88 "/7-12V1")
+  (net 88 "Net-(D1-K)")
   (net 89 "/VBAT1")
   (net 90 "Net-(J1-Pin_6)")
   (net 91 "/VDC")
   (net 92 "/VIN")
-  (net 93 "/7VDC")
+  (net 93 "Net-(D1-A)")
   (net 94 "Net-(J1-Pin_7)")
   (net 95 "/CRX")
@@
         (effects (font (size 1 1) (thickness 0.15)))
     )
-    (fp_text value "HPZR-C7V0X" (at 6.478051 0.051354 90) (layer "F.Fab")
+    (fp_text value "HPZR-C5V6X" (at 6.478051 0.051354 90) (layer "F.Fab")
         (effects (font (size 1 1) (thickness 0.15)))
     )
@@
       (net 35 "Net-(D2-K)") (pinfunction "B") (pintype "passive"))
     (pad "2" smd rect (at -1 0.65 90) (size 0.45 0.7) (layers "F.Cu" "F.Paste" "F.Mask")
-      (net 93 "/7VDC") (pinfunction "E") (pintype "passive"))
+      (net 93 "Net-(D1-A)") (pinfunction "E") (pintype "passive"))
     (pad "3" smd rect (at 1 0 90) (size 0.45 0.7) (layers "F.Cu" "F.Paste" "F.Mask")
       (net 91 "/VDC") (pinfunction "C") (pintype "passive"))
@@
       (stroke (width 0.1) (type solid)) (layer "F.Fab"))
     (pad "1" smd rect (at -3.15 -2.3 180) (size 2 1.5) (layers "F.Cu" "F.Paste" "F.Mask")
-      (net 88 "/7-12V1") (pinfunction "VI") (pintype "power_in"))
+      (net 88 "Net-(D1-K)") (pinfunction "VI") (pintype "power_in"))
     (pad "2" smd rect (at -3.15 0 180) (size 2 1.5) (layers "F.Cu" "F.Paste" "F.Mask")
       (net 87 "GND1") (pinfunction "GND") (pintype "power_in"))
@@
       (stroke (width 0.15) (type solid)) (fill none) (layer "F.Fab"))
     (pad "1" thru_hole circle (at 0 0 180) (size 2 2) (drill 1) (layers "*.Cu" "*.Mask")
-      (net 93 "/7VDC") (pinfunction "1") (pintype "passive"))
+      (net 93 "Net-(D1-A)") (pinfunction "1") (pintype "passive"))
     (model "${KICAD6_3DMODEL_DIR}/TestPoint.3dshapes/TestPoint_Keystone_5000-5004_Miniature.wrl"
       (offset (xyz 0 0 0))
@@
       (net 87 "GND1") (pintype "passive"))
     (pad "2" smd roundrect (at 0.95 0) (size 1 1.45) (layers "F.Cu" "F.Paste" "F.Mask") (roundrect_rratio 0.25)
-      (net 88 "/7-12V1") (pintype "passive"))
+      (net 88 "Net-(D1-K)") (pintype "passive"))
     (model "${KICAD6_3DMODEL_DIR}/Capacitor_SMD.3dshapes/C_0805_2012Metric.wrl"
       (offset (xyz 0 0 0))
@@
       (net 87 "GND1") (pintype "passive"))
     (pad "2" smd roundrect (at 0.95 0 180) (size 1 1.45) (layers "F.Cu" "F.Paste" "F.Mask") (roundrect_rratio 0.25)
-      (net 93 "/7VDC") (pintype "passive"))
+      (net 93 "Net-(D1-A)") (pintype "passive"))
     (model "${KICAD6_3DMODEL_DIR}/Capacitor_SMD.3dshapes/C_0805_2012Metric.wrl"
       (offset (xyz 0 0 0))
@@
       (net 136 "Net-(Q1-G)") (pinfunction "OUT") (pintype "power_out"))
     (pad "2" smd custom (at -1.5625 0) (size 1.475 0.9) (layers "F.Cu" "F.Paste" "F.Mask")
-      (net 93 "/7VDC") (pinfunction "VDD") (pintype "power_in") (zone_connect 2) (thermal_bridge_angle 45)
+      (net 93 "Net-(D1-A)") (pinfunction "VDD") (pintype "power_in") (zone_connect 2) (thermal_bridge_angle 45)
       (options (clearance outline) (anchor rect))
       (primitives
@@
       (stroke (width 0.1) (type solid)) (layer "F.Fab"))
     (pad "1" smd rect (at -1.4 0 270) (size 1.2 1.2) (layers "F.Cu" "F.Paste" "F.Mask")
-      (net 88 "/7-12V1") (pinfunction "K") (pintype "passive"))
+      (net 88 "Net-(D1-K)") (pinfunction "K") (pintype "passive"))
     (pad "2" smd rect (at 1.4 0 270) (size 1.2 1.2) (layers "F.Cu" "F.Paste" "F.Mask")
-      (net 93 "/7VDC") (pinfunction "A") (pintype "passive"))
+      (net 93 "Net-(D1-A)") (pinfunction "A") (pintype "passive"))
     (model "${KICAD6_3DMODEL_DIR}/Diode_SMD.3dshapes/Nexperia_CFP3_SOD-123W.wrl"
       (offset (xyz 0 0 0))
@@
       (net 87 "GND1") (pintype "passive"))
     (pad "2" smd roundrect (at 0.9125 0 180) (size 1.025 1.4) (layers "F.Cu" "F.Paste" "F.Mask") (roundrect_rratio 0.243902439)
-      (net 93 "/7VDC") (pintype "passive"))
+      (net 93 "Net-(D1-A)") (pintype "passive"))
     (model "${KICAD6_3DMODEL_DIR}/Resistor_SMD.3dshapes/R_0805_2012Metric.wrl"
       (offset (xyz 0 0 0))
@@
       (net 136 "Net-(Q1-G)") (pinfunction "G") (pintype "input"))
     (pad "2" smd roundrect (at -0.9375 0.95 180) (size 1.475 0.6) (layers "F.Cu" "F.Paste" "F.Mask") (roundrect_rratio 0.25)
-      (net 88 "/7-12V1") (pinfunction "S") (pintype "passive"))
+      (net 88 "Net-(D1-K)") (pinfunction "S") (pintype "passive"))
     (pad "3" smd roundrect (at 0.9375 0 180) (size 1.475 0.6) (layers "F.Cu" "F.Paste" "F.Mask") (roundrect_rratio 0.25)
       (net 89 "/VBAT1") (pinfunction "D") (pintype "passive"))

Commit message: SpectDrone Development
Parts:
- removed JAX3: Conn_01x01_Female, Gardenuino Custom:SolderWire-0.1sqmm_1x01_D0.4mm_OD1mm
- added JP11: SolderJumper_2_Bridged, Jumper:SolderJumper-2_P1.3mm_Bridged_RoundedPad1.0x1.5mm, B.Cu at (145.7, 118.1)
- added JP12: SolderJumper_2_Bridged, Jumper:SolderJumper-2_P1.3mm_Bridged_RoundedPad1.0x1.5mm, B.Cu at (145.7, 120.7)
- added JP13: SolderJumper_2_Bridged, Jumper:SolderJumper-2_P1.3mm_Bridged_RoundedPad1.0x1.5mm, B.Cu at (145.7, 123.2)
- added JP14: SolderJumper_2_Bridged, Jumper:SolderJumper-2_P1.3mm_Bridged_RoundedPad1.0x1.5mm, B.Cu at (145.7, 125.8)
- added R68: 100K, Resistor_SMD:R_0805_2012Metric, B.Cu at (135.5, 93.5)
- added R69: 100K, Resistor_SMD:R_0805_2012Metric, B.Cu at (135.5, 97.1)
- BT1, JGAIN1, JPAX1, SW1: moved to B.Cu
- C1-1: renamed from C2-1; moved to B.Cu
- C1-2: renamed from C2-2; moved to B.Cu
- C2: renamed from C3; moved to B.Cu
- D1: renamed from D2; value HPZR-C5V6X -> D; moved to B.Cu
- D2: renamed from D1; moved to B.Cu
- Q1: renamed from Q2; moved to B.Cu
- Q2: renamed from Q1; moved to B.Cu
- R1: renamed from R2; value 1K -> 10K; moved to B.Cu
- R2: renamed from R3; moved to B.Cu
- R38: renamed from R1; moved to B.Cu
- U1: renamed from U2; moved to B.Cu
- U2: renamed from U3; moved to B.Cu
- moved R1 27.3 mm to (125.7, 101.0), turned to -90 degrees
- moved D1 24.9 mm to (120.0, 99.9)
- moved Q1 23.2 mm to (122.8, 101.0), turned to -90 degrees
- moved D2 20.5 mm to (123.9, 98.0), turned to 180 degrees
- moved Q2 16.3 mm to (125.0, 93.8), turned to -90 degrees
- moved C1-1 11.8 mm to (125.8, 89.9), turned to 180 degrees
- moved R38 11.4 mm to (172.6, 102.5), turned to 180 degrees
- moved U2 10.6 mm to (120.7, 94.2), turned to 90 degrees
- moved JPAX1 7.71 mm to (172.6, 80.9)
- moved R2 5.83 mm to (121.7, 89.8), turned to -90 degrees
- moved C2 2.96 mm to (119.7, 89.8), turned to -90 degrees
- moved JGAIN1 2.29 mm to (172.6, 74.3), turned to 180 degrees
- moved SW1 2.29 mm to (172.6, 68.5), turned to 0 degrees
- moved R48 1.77 mm to (197.6, 83.1)
- moved R49 1.77 mm to (195.6, 83.1)
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- renumbered U1 to A1, C4 to C3, C5 to C4, C6 to C5, C7-1 to C6-1, C7-2 to C6-2, R11 to R10, R12 to R11, R13 to R12, R14 to R13, R15 to R14, R16 to R15, R17 to R16, R18 to R17, R19 to R18, R20 to R19, R21 to R20, R22 to R21, R23 to R22, R24 to R23, R25 to R24, R26 to R25, R27 to R26, R28 to R27, R29 to R28, R30 to R29, R4 to R3, R31 to R30, R32 to R31, R33 to R32, R34 to R33, R35 to R34, R36 to R35, R37 to R36, R38 to R37, R5 to R4, R6 to R5, R7-1 to R6-1, R7-2 to R6-2, R8 to R7, R9 to R8, R10 to R9, U4 to U3, U5 to U4, U6 to U5, U7 to U6
Connections:
- net /VBAT1 renamed /BAT_{V}
- net Net-(D1-A) renamed /6.7V
- A1 pad 33: Net-(JAX3-Pin_1) -> /A17
- A1 pad 42: /S1 -> Net-(A1-20_A6_TX5_LRCLK1)
- A1 pad 43: /P1 -> Net-(A1-21_A7_RX5_BCLK1)
- A1 pad 44: /P2 -> Net-(A1-22_A8_CTX1)
- A1 pad 45: /S2 -> Net-(A1-23_A9_CRX1_MCLK1)
- C1-2 pad 2: Net-(D1-K) (its old number) -> /6V
- D2 pad 1: Net-(D1-K) (its old number) -> /6V
- Q2 pad 2: Net-(D1-K) (its old number) -> /6V
- U1 pad 1: Net-(D1-K) (its old number) -> /6V
Routing:
- net /6V: track 0.00 -> 30.4 mm, vias 0 -> 2
- net Net-(D1-K) (its old number): track 30.3 -> 0.00 mm, vias 2 -> 0
- net /5V: track 246.3 -> 217.9 mm, vias 7 -> 9
- net /BAT_{V}: track 17.9 -> 39.2 mm, vias 0 -> 1
- net /VDC: track 37.0 -> 56.9 mm, vias 0 -> 1
- net Net-(JPAX1-C): track 2.14 -> 22.0 mm, vias 0 -> 2
- net /A17: track 0.00 -> 10.6 mm
- net Net-(JGAIN1-C): track 17.6 -> 10.2 mm
- net /AX1: track 22.3 -> 15.5 mm
- net /CRX: track 61.2 -> 67.8 mm
- net /6.7V: track 38.1 -> 43.3 mm, vias 0 -> 1
- net /3V: track 270.3 -> 274.9 mm
- net /VBat: track 85.8 -> 90.3 mm, vias 0 -> 1
- net /CTX: track 63.9 -> 67.8 mm
- net Net-(JAX3-Pin_1): track 3.70 -> 0.00 mm
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Other:
- board text added: "6.7V"
- board text added: "7.0 Vdc MAX"
- board text added: "Enable"
- board text added: "GAIN"
- board text removed: "7V"
- board text removed: "TXS_{e}"

Commit message: SpectDrone Development
Parts:
- JBAT1: moved to B.Cu
- JDC1: footprint Connector_BarrelJack:BarrelJack_Horizontal -> Connector_BarrelJack:BarrelJack_CUI_PJ-063AH_Horizontal; moved to B.Cu
- moved JDC1 2.87 mm to (112.3, 74.4), turned to 90 degrees
- turned JBAT1 to 180 degrees
Routing:
- net /VDC: track 56.9 -> 62.7 mm
- net GND1: track 109.0 -> 110.5 mm
