File: SpectDroneControl/SpectDroneControl.kicad_sch (KiCad schematic)
At the start: 20 parts, among them J1 Conn_02x03_Counter_Clockwise, J1-1 Conn_01x04_Male, J1-2 Conn_01x04_Male, U1 Teensy4.1, U2 Teensy4.0

Commit message: SpectDrone Development
Parts:
- added R1: 10K, Resistor_SMD:R_0603_1608Metric, symbol Device:R
- added SW1: SW_SPDT, Button_Switch_SMD:SW_SPDT_CK-JS102011SAQN, symbol Switch:SW_SPDT
- U2: footprint Teensy:Teensy30_31_32_LC -> Teensy:Teensy40
Connections:
- net 5V: now also SW1.1 (A)
- net APCRX: now also U1.10 (8_TX2_IN1), U2.10 (8_TX2_DIN_PWM); no longer U1.12 (10_CS_MQSR), U2.12 (10_TX2_CS_PWM)
- net APCTX: now also U1.9 (7_RX2_OUT1A), U2.9 (7_RX2_DOUT_PWM); no longer U1.11 (9_OUT1C), U2.11 (9_RX2_CS_PWM)
- net CLK1: now also U1.6 (4_BCLK2), U2.6 (4_PWM); no longer U1.7 (5_IN2), U2.7 (5_TX1_PWM)
- net GAIN: now also R1.1; no longer U1.5 (3_LRCLK2), U2.5 (3_TX_PWM)
- net GND: now also U1.34 (GND), U2.17 (GND), SW1.3 (C)
- net RX: now also U1.12 (10_CS_MQSR), U2.12 (10_CS_PWM); no longer U1.10 (8_TX2_IN1), U2.10 (8_TX3_DIN)
- net ST: now also U1.5 (3_LRCLK2), U2.5 (3_PWM); no longer U1.6 (4_BCLK2), U2.6 (4_RX_PWM)
- net TX: now also U1.11 (9_OUT1C), U2.11 (9_PWM); no longer U1.9 (7_RX2_OUT1A), U2.9 (7_RX3_DOUT)
- net UT1: now also U1.8 (6_OUT1D), U2.8 (6_PWM); no longer U1.17 (25_A11_RX6_SDA2), U2.36 (A10)
- net UT2: now also U1.7 (5_IN2), U2.7 (5_PWM); no longer U1.8 (6_OUT1D), U2.8 (6_PWM)
- net RX8: now reaches U1.26 (34_RX8)
- net TX8: now reaches U1.27 (35_TX8)
- net CS3: now reaches U1.28 (36_CS)
- net CS2: now reaches U1.29 (37_CS)
- new net: R1.2, SW1.2 (B)
- no-connect marks 4 -> 6
Other:
- moved on the sheet: BT1

Commit message: SpectDrone Development
Parts:
- added R10, R11, R12, R13, R14, R15, R16, R17, R18, R19, R2, R20, R21, R22, R23, R24, R25, R26, R27, R28, R29, R3, R30, R31, R32, R33, R34, R35, R36, R37, R38, R39, R4, R40, R41, R42, R43, R44, R45, R46, R47, R48, R49, R5, R50, R51, R52, R53, R54, R55, R56, R57, R58, R59, R6, R60, R7, R8, R9: R, Resistor_SMD:R_0805_2012Metric, symbol Device:R
- added U3, U4, U5: NVT2010PW, Package_SO:TSSOP-24_4.4x7.8mm_P0.65mm, symbol Logic_LevelTranslator:TXS0108EPW
Connections:
- net 5V: now also R14.2, R15.2, R16.2, R17.2, R18.2, R19.2, R2.2, R20.2, R21.2, R22.2, R3.2, R32.2, R33.2, R34.2, R35.2, R36.2, R37.2, R38.2, R39.2, R4.2, R40.2, R51.2, R52.2, R53.2, R54.2, R55.2, R56.2, R57.2, R58.2, R59.2, R60.2
- net APCRX: now also R11.1, U3.10 (A8); no longer JAPC1.2 (Pin_2)
- net APCTX: now also R10.1, U3.9 (A7); no longer JAPC1.1 (Pin_1)
- net CAM1RX: now also R43.1, U5.5 (A3); no longer JAUX1.10 (Pin_10)
- net CAM1TX: now also R42.1, U5.4 (A2); no longer JAUX1.11 (Pin_11)
- net CAM2RX: now also R45.1, U5.7 (A5); no longer JAUX1.8 (Pin_8)
- net CAM2TX: now also R44.1, U5.6 (A4); no longer JAUX1.9 (Pin_9)
- net CLK1: now also R7.1, U3.6 (A4); no longer JD1.1 (Pin_1)
- net CLK2: now also R5.1, U3.4 (A2); no longer JD1.4 (Pin_4)
- net CS1: now also R28.1, U4.9 (A7); no longer JP6.1 (A)
- net CS2: now also R27.1, U4.8 (A6)
- net CS3: now also R26.1, U4.7 (A5)
- net GND: now also U3.1 (GND), U4.1 (GND), U5.1 (GND)
- net GPSRX: no longer JGPS1.3 (Pin_3)
- net GPSTX: no longer JGPS1.4 (Pin_4)
- net MISO: now also R48.1, U5.10 (A8); no longer JAUX1.5 (Pin_5)
- net MISO1: now also R30.1, U4.11 (A9); no longer JP8.1 (A)
- net MOSI: now also R50.1, U5.12 (A10); no longer JAUX1.3 (Pin_3)
- net MOSI1: now also R31.1, U4.12 (A10); no longer JP7.1 (A)
- net PPS: no longer JGPS1.5 (Pin_5)
- net RX: now also R13.1, U3.12 (A10); no longer JAPC1.4 (Pin_4)
- net SCK: now also R49.1, U5.11 (A9); no longer JAUX1.4 (Pin_4)
- net SCK1: now also R29.1, U4.10 (A8); no longer JP5.1 (A)
- net SCL: now also R47.1, U5.9 (A7); no longer JAUX1.6 (Pin_6)
- net SDA: now also R46.1, U5.8 (A6); no longer JAUX1.7 (Pin_7)
- net ST: now also R6.1, U3.5 (A3); no longer JD1.2 (Pin_2)
- net TX: now also R12.1, U3.11 (A9); no longer JAPC1.3 (Pin_3)
- net TXS_{E}: now also U1.15 (3V3), U2.16 (3.3V), R41.1, U5.3 (A1); no longer JAUX1.12 (Pin_12), U1.33 (41_A17), U2.19 (ON/OFF)
- net UT1: now also R9.1, U3.8 (A6); no longer JUT1.1 (Pin_1)
- net UT2: now also R8.1, U3.7 (A5); no longer JUT1.2 (Pin_2)
- net 3V: now reaches U2.31 (3.3V)
- net 3V: now also U1.46 (3V3), R10.2, R11.2, R12.2, R13.2, R23.2, R24.2, R25.2, R26.2, R27.2, R28.2, R29.2, R30.2, R31.2, R41.2, R42.2, R43.2, R44.2, R45.2, R46.2, R47.2, R48.2, R49.2, R5.2, R50.2, R6.2, R7.2, R8.2, R9.2, U3.2 (VREFA), U4.2 (VREFA), U5.2 (VREFA)
- net CAN_H_5V: now reaches JUT1.3 (Pin_3)
- net CAN_L_5V: now reaches JUT1.4 (Pin_4)
- net GAIN renamed GAIN_5V
- new net: R24.1, U4.5 (A3)
- new net: R4.1, U5.23 (VREFB), U5.24 (EN)
- new net: R33.1, U4.20 (B3)
- new net: R32.1, U4.21 (B2)
- new net: R34.1, U4.19 (B4)
- new net: R23.1, U4.4 (A2)
- new net: R25.1, U4.6 (A4)
- new net: R3.1, U4.23 (VREFB), U4.24 (EN)
- new net: R2.1, U3.23 (VREFB), U3.24 (EN)
- new net APCRX_5V: JAPC1.2 (Pin_2), R20.1, U3.15 (B8)
- new net APCTX_5V: JAPC1.1 (Pin_1), R19.1, U3.16 (B7)
- new net CAM1RX_5V: JAUX1.10 (Pin_10), R53.1, U5.20 (B3)
- new net CAM1TX_5V: JAUX1.11 (Pin_11), R52.1, U5.21 (B2)
- new net CAM2RX_5V: JAUX1.8 (Pin_8), R55.1, U5.18 (B5)
- new net CAM2TX_5V: JAUX1.9 (Pin_9), R54.1, U5.19 (B4)
- new net CLK1_5V: JD1.1 (Pin_1), R16.1, U3.19 (B4)
- new net CLK2_5V: JD1.4 (Pin_4), R14.1, U3.21 (B2)
- new net CS1_5V: JP5.1 (A), R37.1, U4.16 (B7)
- new net CS2_5V: R36.1, U4.17 (B6)
- new net CS3_5V: R35.1, U4.18 (B5)
- new net GPSRX_5V: JGPS1.3 (Pin_3)
- new net GPSTX_5V: JGPS1.4 (Pin_4)
- new net MISO1_5V: JP7.1 (A), R39.1, U4.14 (B9)
- new net MISO_5V: JAUX1.5 (Pin_5), R58.1, U5.15 (B8)
- new net MOSI1_5V: JP8.1 (A), R40.1, U4.13 (B10)
- new net MOSI_5V: JAUX1.3 (Pin_3), R60.1, U5.13 (B10)
- new net PPS_5V: JGPS1.5 (Pin_5)
- new net RX_5V: JAPC1.4 (Pin_4), R22.1, U3.13 (B10)
- new net SCK1_5V: JP6.1 (A), R38.1, U4.15 (B8)
- new net SCK_5V: JAUX1.4 (Pin_4), R59.1, U5.14 (B9)
- new net SCL_5V: JAUX1.6 (Pin_6), R57.1, U5.16 (B7)
- new net SDA_5V: JAUX1.7 (Pin_7), R56.1, U5.17 (B6)
- new net ST_5V: JD1.2 (Pin_2), R15.1, U3.20 (B3)
- new net TXS_{E}_5V: JAUX1.12 (Pin_12), R51.1, U5.22 (B1)
- new net TX_5V: JAPC1.3 (Pin_3), R21.1, U3.14 (B9)
- new net UT1_5V: JUT1.1 (Pin_1), R18.1, U3.17 (B6)
- new net UT2_5V: JUT1.2 (Pin_2), R17.1, U3.18 (B5)
- no-connect marks 6 -> 14
Other:
- moved on the sheet: BT1, JA1, JAPC1, JAUX1, JD1, JGPS1, JUT1, R1, SW1

Commit message: SpectDrone Development
Parts:
- added R15, R25, R35, R5: R, Resistor_SMD:R_0805_2012Metric, symbol Device:R
- renumbered R9 to R10, R10 to R11, R11 to R12, R12 to R13, R13 to R14, R14 to R16, R15 to R17, R16 to R18, R17 to R19, R18 to R20, R19 to R21, R20 to R22, R21 to R23, R22 to R24, R23 to R26, R24 to R27, R25 to R28, R26 to R29, R27 to R30, R28 to R31, R29 to R32, R30 to R33, R31 to R34, R32 to R36, R33 to R37, R34 to R38, R35 to R39, R36 to R40, R37 to R41, R38 to R42, R39 to R43, R40 to R44, R41 to R45, R42 to R46, R43 to R47, R44 to R48, R45 to R49, R46 to R50, R47 to R51, R48 to R52, R49 to R53, R50 to R54, R51 to R55, R52 to R56, R53 to R57, R54 to R58, R55 to R59, R5 to R6, R56 to R60, R57 to R61, R58 to R62, R59 to R63, R60 to R64, R6 to R7, R7 to R8, R8 to R9
Connections:
- net 3V: now also R25.2, R5.2
- net 5V: now also R15.2, R35.2
- net at U3.22 (B1): now also R15.1
- net at U3.3 (A1): now also R5.1
- net at U4.22 (B1): now also R35.1
- net at U4.3 (A1): now also R25.1
- no-connect marks 14 -> 24
Other:
- moved on the sheet: JGPS1, JUT1, R10, R11, R12, R13, R14, R16, R17, R18, R19, R2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

Commit message: SpectDrone Development
Parts:
- added C1, C2: 0.1uF, Capacitor_SMD:C_0805_2012Metric, symbol Device:C_Small
- added C3: 10uF, Capacitor_SMD:CP_Elec_3x5.4, symbol Device:C_Polarized_Small_US
- added D1: D, Diode_SMD:Nexperia_CFP3_SOD-123W, symbol Device:D
- added J3-1, J3-2, J3-3, J3-4, J3-5, J5-1, J5-2, J5-3, J5-4, J5-5, JAX1, JAX2, JAX3, JCRX3, JCTX3, JPPS1, JPPS2, JRX6, JRX8, JTX6, JTX8: Conn_01x01_Female, Connector_Wire:SolderWire-0.1sqmm_1x01_D0.4mm_OD1mm, symbol Connector:Conn_01x01_Female
- added J3V1, JVIN1: Conn_01x01_Male, Connector_PinHeader_2.54mm:PinHeader_1x01_P2.54mm_Vertical, symbol Connector:Conn_01x01_Male
- added JBAT1: Conn_01x02_Female, Connector_Molex:Molex_Micro-Fit_3.0_43045-0200_2x01_P3.00mm_Horizontal, symbol Connector:Conn_01x02_Female
- added JDC1: Barrel_Jack, Connector_BarrelJack:BarrelJack_Horizontal, symbol Connector:Barrel_Jack_Switch
- added Q1: FDN340P, Package_TO_SOT_SMD:SOT-23, symbol Transistor_FET:FDN340P
- added R65: 100K, Capacitor_SMD:C_0805_2012Metric, symbol Device:R
- added TP1, TP2, TP3, TP4: TestPoint, TestPoint:TestPoint_Keystone_5000-5004_Miniature, symbol Connector:TestPoint
- added U6: MCP112-450E/TO, Package_TO_SOT_SMD:SOT-89-3, symbol Power_Supervisor:MCP120-xxxDxTO
- added U7: LM7805_SOT223, Package_TO_SOT_SMD:SOT-223-3_TabPin2, symbol Regulator_Linear:LM7805_TO220
- BT1: footprint Battery:BatteryHolder_Keystone_103_1x20mm -> Battery:BatteryHolder_Keystone_3000_1x12mm
Connections:
- net GND is gone; now on net GND1: BT1.2 (-), JAUX1.2 (Pin_2), JGPS1.2 (Pin_2), JP1.1 (A), SW1.3 (C), U1.1 (GND), U1.34 (GND), U1.47 (GND), U2.1 (GND), U2.17 (GND), U2.32 (AGND), U3.1 (GND), U4.1 (GND), U5.1 (GND)
- net 3V: now also J3V1.1 (Pin_1), TP4.1
- net CAM1RX: now also R46.1; no longer R47.1
- net CAM1TX: now also R47.1; no longer R46.1
- net CAN_H: now also R25.1, U1.22 (30_CRX3), U4.3 (A1), J3-2.1 (Pin_1), JCRX3.1 (Pin_1)
- net CAN_H_5V: now also R35.1, U4.22 (B1), J5-2.1 (Pin_1)
- net CAN_L: now also R26.1, U1.23 (31_CTX3), U4.4 (A2), J3-3.1 (Pin_1), JCTX3.1 (Pin_1)
- net CAN_L_5V: now also R36.1, U4.21 (B2), J5-3.1 (Pin_1)
- net PPS: now also JPPS1.1 (Pin_1)
- net PPS_5V: now also JPPS2.1 (Pin_1)
- net RX8: now also JRX8.1 (Pin_1)
- net TX8: now also JTX8.1 (Pin_1)
- net at R15.1, U3.22 (B1): now also J5-1.1 (Pin_1)
- net TX6: now reaches R27.1, U4.5 (A3)
- net TX6: now also U1.16 (24_A10_TX6_SCL2), J3-4.1 (Pin_1), JTX6.1 (Pin_1)
- net at R5.1, U3.3 (A1): now also J3-1.1 (Pin_1)
- net TX6_5V: now reaches R37.1, U4.20 (B3)
- net TX6_5V: now also J5-4.1 (Pin_1)
- net RX6_5V: now reaches R38.1, U4.19 (B4)
- net RX6_5V: now also J5-5.1 (Pin_1)
- net RX6: now reaches R28.1, U4.6 (A4)
- net RX6: now also U1.17 (25_A11_RX6_SDA2), J3-5.1 (Pin_1), JRX6.1 (Pin_1)
- net at U1.24 (32_OUT1B): now also JAX1.1 (Pin_1)
- net at U1.25 (33_MCLK2): now also JAX2.1 (Pin_1)
- net at U1.33 (41_A17): now also JAX3.1 (Pin_1)
- net GND1: now reaches U1.52 (GND)
- net GND1: now also C1.1, C2.1, C3.2, JBAT1.2 (Pin_2), JDC1.2, JDC1.3, R65.1, TP1.1, U6.3 (VSS), U7.2 (GND)
- new net: Q1.1 (G), U6.1 (OUT)
- new net 5V3: C3.1, TP3.1, U7.3 (VO)
- new net 7-12V1: C2.2, D1.1 (K), Q1.2 (S), U7.1 (VI)
- new net VBAT1: JBAT1.1 (Pin_1), Q1.3 (D)
- new net VDC: C1.2, D1.2 (A), JDC1.1, JVIN1.1 (Pin_1), R65.2, TP2.1, U6.2 (VDD)
- no-connect marks 24 -> 7
Other:
- moved on the sheet: R10, R11, R12, R13, R14, R15, R16, R17, R18, R19, R2, R20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

Commit message: SpectDrone Development
Parts:
- added D2: HPZR-C7V0X, Diode_SMD:D_SOD-123F, symbol Device:D
- added JCS2, JCS3: Conn_01x01_Female, Connector_Wire:SolderWire-0.1sqmm_1x01_D0.4mm_OD1mm, symbol Connector:Conn_01x01_Female
- added Q2: Q_NPN_EBC, Package_TO_SOT_SMD:SOT-323_SC-70, symbol Device:Q_NPN_EBC
- added R66: 1K, Capacitor_SMD:C_0805_2012Metric, symbol Device:R
- added TP2, TP6: TestPoint, TestPoint:TestPoint_Keystone_5000-5004_Miniature, symbol Connector:TestPoint
- renumbered C3 to C1, C1 to C2, C2 to C3, TP2 to TP3, TP3 to TP4, TP4 to TP5
Connections:
- net CS2_5V: now also JCS2.1 (Pin_1)
- net CS3_5V: now also JCS3.1 (Pin_1)
- net GND1: now also D2.2 (A)
- net VDC: now also Q2.3 (C), R66.2, TP2.1; no longer C2.2, D1.2 (A), JVIN1.1 (Pin_1), R65.2, TP3.1, U6.2 (VDD)
- net at J1-1.3 (Pin_3), JP3.2 (B): now also J1.6 (Pin_6); no longer J1.3 (Pin_3)
- net at J1-1.1 (Pin_1), JP1.2 (B): now also J1.8 (Pin_8); no longer J1.1 (Pin_1)
- net at J1-1.2 (Pin_2), JP2.2 (B): now also J1.7 (Pin_7); no longer J1.2 (Pin_2)
- net at J1-1.4 (Pin_4), JP4.2 (B): now also J1.5 (Pin_5); no longer J1.4 (Pin_4)
- net at J1-2.4 (Pin_4), JP5.2 (B): now also J1.4 (Pin_4); no longer J1.5 (Pin_5)
- net at J1-2.3 (Pin_3), JP6.2 (B): now also J1.3 (Pin_3); no longer J1.6 (Pin_6)
- net at J1-2.2 (Pin_2), JP7.2 (B): now also J1.2 (Pin_2); no longer J1.7 (Pin_7)
- net at J1-2.1 (Pin_1), JP8.2 (B): now also J1.1 (Pin_1); no longer J1.8 (Pin_8)
- new net: D2.1 (K), Q2.2 (B), R66.1
- new net 7VDC: C2.2, D1.2 (A), Q2.1 (E), R65.2, TP6.1, U6.2 (VDD)
- new net VIN: JVIN1.1 (Pin_1), TP3.1
Other:
- moved on the sheet: BT1, C1, C2, C3, D1, J1, J1-1, J1-2, J3V1, JA1, JAPC1, JAUX1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

Commit message: SpectDrone Development
Other:
- moved on the sheet: D2, JAX1, JAX2, JAX3, JCRX3, JCTX3, JDC1, JPPS1, JRX6, JRX8, JTX6, JTX8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

Commit message: SpectDrone Development
Parts:
- added JCAN_{H}1, JCAN_{L}1: Conn_01x01_Female, Connector_Wire:SolderWire-0.1sqmm_1x01_D0.4mm_OD1mm, symbol Connector:Conn_01x01_Female
- added JCR1: Conn_01x37_Female, Gardenuino Custom:PinHeader_Corner, symbol Connector:Conn_01x37_Female
Connections:
- net 3V: now also JCR1.2 (Pin_2)
- net 5V: now also JCR1.3 (Pin_3)
- net CAN_H_5V: now also JCAN_{H}1.1 (Pin_1); no longer J5-2.1 (Pin_1), R35.1, U4.22 (B1)
- net CAN_L_5V: now also JCAN_{L}1.1 (Pin_1); no longer J5-3.1 (Pin_1), R36.1, U4.21 (B2)
- net GND1: now also JCR1.1 (Pin_1)
- net MISO1_5V: now also JCR1.36 (Pin_36)
- net MOSI1_5V: now also JCR1.35 (Pin_35)
- net SCK1_5V: now also JCR1.37 (Pin_37)
- net CAN_H renamed CRX
- net CAN_L renamed CTX
- new net CRX_5V: J5-2.1 (Pin_1), R35.1, U4.22 (B1)
- new net CTX_5V: J5-3.1 (Pin_1), R36.1, U4.21 (B2)
Changed lines of the file:
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@@
     (stroke (width 0) (type default) (color 0 0 0 0))
   )
-  (polyline (pts (xy 127.635 53.34) (xy 127.635 19.05))
+  (polyline (pts (xy 138.43 53.34) (xy 138.43 19.05))
     (stroke (width 0) (type default) (color 0 0 0 0))
   )
@@
     (stroke (width 0) (type default) (color 0 0 0 0))
   )
-  (polyline (pts (xy 21.59 53.34) (xy 127.635 53.34))
+  (polyline (pts (xy 21.59 53.34) (xy 138.43 53.34))
     (stroke (width 0) (type default) (color 0 0 0 0))
   )
@@
     (stroke (width 0) (type default) (color 0 0 0 0))
   )
-  (polyline (pts (xy 127.635 19.05) (xy 21.59 19.05))
+  (polyline (pts (xy 138.43 19.05) (xy 21.59 19.05))
     (stroke (width 0) (type default) (color 0 0 0 0))
   )
@@
     (effects (font (size 1.27 1.27)) (justify left bottom))
   )
+  (label "GND" (at 148.59 100.965 180)
+    (effects (font (size 1.27 1.27)) (justify right bottom))
+  )
   (label "A2" (at 212.09 29.21 0)
     (effects (font (size 1.27 1.27)) (justify left bottom))
@@
     (effects (font (size 1.27 1.27)) (justify right bottom))
   )
-  (label "CAN_H" (at 29.21 130.175 180)
+  (label "CRX" (at 29.21 130.175 180)
     (effects (font (size 1.27 1.27)) (justify right bottom))
   )
@@
     (effects (font (size 1.27 1.27)) (justify right bottom))
   )
+  (label "MOSI1_5V" (at 148.59 187.325 180)
+    (effects (font (size 1.27 1.27)) (justify right bottom))
+  )
   (label "TX6" (at 156.21 59.69 180)
     (effects (font (size 1.27 1.27)) (justify right bottom))
@@
     (effects (font (size 1.27 1.27)) (justify left bottom))
   )
-  (label "CAN_H_5V" (at 122.555 130.175 180)
+  (label "CRX_5V" (at 122.555 130.175 180)
     (effects (font (size 1.27 1.27)) (justify right bottom))
   )
-  (label "CAN_L" (at 156.21 77.47 180)
+  (label "CTX" (at 156.21 77.47 180)
     (effects (font (size 1.27 1.27)) (justify right bottom))
   )
@@
     (effects (font (size 1.27 1.27)) (justify left bottom))
   )
+  (label "SCK1_5V" (at 148.59 192.405 180)
+    (effects (font (size 1.27 1.27)) (justify right bottom))
+  )
   (label "MISO" (at 230.505 50.8 180)
     (effects (font (size 1.27 1.27)) (justify right bottom))
@@
     (effects (font (size 1.27 1.27)) (justify right bottom))
   )
+  (label "3V" (at 148.59 103.505 180)
+    (effects (font (size 1.27 1.27)) (justify right bottom))
+  )
   (label "3V" (at 281.305 81.28 0)
     (effects (font (size 1.27 1.27)) (justify left bottom))
@@
     (effects (font (size 1.27 1.27)) (justify right bottom))
   )
-  (label "CAN_L" (at 29.21 132.715 180)
+  (label "CTX" (at 29.21 132.715 180)
     (effects (font (size 1.27 1.27)) (justify right bottom))
   )
@@
     (effects (font (size 1.27 1.27)) (justify right bottom))
   )
+  (label "5V" (at 148.59 106.045 180)
+    (effects (font (size 1.27 1.27)) (justify right bottom))
+  )
   (label "VDC" (at 266.7 122.555 180)
     (effects (font (size 1.27 1.27)) (justify right bottom))
@@
     (effects (font (size 1.27 1.27)) (justify right bottom))
   )
-  (label "CAN_L_5V" (at 122.555 132.715 180)
+  (label "CTX_5V" (at 122.555 132.715 180)
     (effects (font (size 1.27 1.27)) (justify right bottom))
   )
@@
     (effects (font (size 1.27 1.27)) (justify left bottom))
   )
+  (label "MISO1_5V" (at 148.59 189.865 180)
+    (effects (font (size 1.27 1.27)) (justify right bottom))
+  )
   (label "CLK2_5V" (at 114.935 90.805 0)
     (effects (font (size 1.27 1.27)) (justify left bottom))
@@
     (effects (font (size 1.27 1.27)) (justify right bottom))
   )
-  (label "CAN_H" (at 156.21 74.93 180)
+  (label "CRX" (at 156.21 74.93 180)
     (effects (font (size 1.27 1.27)) (justify right bottom))
   )
@@
     (pin "2")
   )
+  (symbol (lib_id "Connector:Conn_01x37_Female") (at 153.67 146.685 0) (unit 1)
+    (in_bom yes) (on_board yes) (fields_autoplaced)
+    (property "Reference" "JCR1" (id 0) (at 154.94 145.4149 0)
+      (effects (font (size 1.27 1.27)) (justify left))
+    )
+    (property "Value" "Conn_01x37_Female" (id 1) (at 154.94 147.9549 0)
+      (effects (font (size 1.27 1.27)) (justify left))
+    )
+    (property "Footprint" "Gardenuino Custom:PinHeader_Corner" (id 2) (at 153.67 146.685 0)
+      (effects (font (size 1.27 1.27)) hide)
+    )
+    (property "Datasheet" "~" (id 3) (at 153.67 146.685 0)
+      (effects (font (size 1.27 1.27)) hide)
+    )
+    (pin "1")
+    (pin "10")
+    (pin "11")
+    (pin "12")
+    (pin "13")
+    (pin "14")
+    (pin "15")
+    (pin "16")
+    (pin "17")
+    (pin "18")
+    (pin "19")
+    (pin "2")
+    (pin "20")
+    (pin "21")
+    (pin "22")
+    (pin "23")
+    (pin "24")
+    (pin "25")
+    (pin "26")
+    (pin "27")
+    (pin "28")
+    (pin "29")
+    (pin "3")
+    (pin "30")
+    (pin "31")
+    (pin "32")
+    (pin "33")
+    (pin "34")
+    (pin "35")
+    (pin "36")
+    (pin "37")
+    (pin "4")
+    (pin "5")
+    (pin "6")
+    (pin "7")
+    (pin "8")
+    (pin "9")
+  )
   (symbol (lib_id "Connector:Conn_01x01_Female") (at 128.27 130.175 0) (unit 1)
     (in_bom yes) (on_board yes)
@@
     (pin "2")
   )
+  (symbol (lib_id "Connector:Conn_01x01_Female") (at 130.175 33.655 0) (unit 1)
+    (in_bom yes) (on_board yes)
+    (property "Reference" "JCAN_{L}1" (id 0) (at 130.81 33.655 0)
+      (effects (font (size 1.27 1.27)) (justify left))
+    )
+    (property "Value" "Conn_01x01_Female" (id 1) (at 129.54 36.195 0)
+      (effects (font (size 1.27 1.27)) hide)
+    )
+    (property "Footprint" "Connector_Wire:SolderWire-0.1sqmm_1x01_D0.4mm_OD1mm" (id 2) (at 130.175 33.655 0)
+      (effects (font (size 1.27 1.27)) hide)
+    )
+    (property "Datasheet" "~" (id 3) (at 130.175 33.655 0)
+      (effects (font (size 1.27 1.27)) hide)
+    )
+    (pin "1")
+  )
   (symbol (lib_id "Connector:Conn_01x04_Male") (at 110.49 28.575 0) (unit 1)
     (in_bom yes) (on_board yes)
@@
     (pin "2")
   )
+  (symbol (lib_id "Connector:Conn_01x01_Female") (at 130.175 31.115 0) (unit 1)
+    (in_bom yes) (on_board yes)
+    (property "Reference" "JCAN_{H}1" (id 0) (at 130.81 31.115 0)
+      (effects (font (size 1.27 1.27)) (justify left))
+    )
+    (property "Value" "Conn_01x01_Female" (id 1) (at 129.54 33.655 0)
+      (effects (font (size 1.27 1.27)) hide)
+    )
+    (property "Footprint" "Connector_Wire:SolderWire-0.1sqmm_1x01_D0.4mm_OD1mm" (id 2) (at 130.175 31.115 0)
+      (effects (font (size 1.27 1.27)) hide)
+    )
+    (property "Datasheet" "~" (id 3) (at 130.175 31.115 0)
+      (effects (font (size 1.27 1.27)) hide)
+    )
+    (pin "1")
+  )
   (symbol (lib_id "Jumper:SolderJumper_2_Open") (at 43.815 48.26 0) (unit 1)
     (in_bom yes) (on_board yes)
@@
       (reference "JBAT1") (unit 1) (value "Conn_01x02_Female") (footprint "Connector_Molex:Molex_Micro-Fit_3.0_43045-0200_2x01_P3.00mm_Horizontal")
     )
+    (path "/cb122ac4-cab1-4e41-9397-1c87b93e8255"
+      (reference "JCAN_{H}1") (unit 1) (value "Conn_01x01_Female") (footprint "Connector_Wire:SolderWire-0.1sqmm_1x01_D0.4mm_OD1mm")
+    )
+    (path "/94dcc620-a87a-403e-b579-f56fb04fc4df"
+      (reference "JCAN_{L}1") (unit 1) (value "Conn_01x01_Female") (footprint "Connector_Wire:SolderWire-0.1sqmm_1x01_D0.4mm_OD1mm")
+    )
+    (path "/828b4ec8-f926-4823-95c9-3c582d5f4d49"
+      (reference "JCR1") (unit 1) (value "Conn_01x37_Female") (footprint "Gardenuino Custom:PinHeader_Corner")
+    )
     (path "/008f154a-6349-4fd5-b138-2a3e4ec8b643"

Commit message: SpectDrone Development
Parts:
- added C4, C5: 0.1uF, Capacitor_SMD:C_0805_2012Metric, symbol Device:C_Small
- added R67, R68: 200K, Capacitor_SMD:C_0805_2012Metric, symbol Device:R
- added U8: TXS0102DCUR, Package_SO:SSOP-8_2.95x2.8mm_P0.65mm, symbol Logic_LevelTranslator:TXS0102DCT
- R45: value R -> X
- renumbered J1-2 to J2-1, J1-1 to J2-2
Connections:
- net 5V3 is gone; now on net 5V: C1.1, TP4.1, U7.3 (VO)
- net 3V: now also C4.1, U8.3 (VCCA); no longer JCR1.2 (Pin_2)
- net 5V: now also R67.2; no longer JCR1.3 (Pin_3)
- net GND1: now also C4.2, C5.2, R68.1, U8.2 (GND)
- net GPSRX: now also U8.5 (A1)
- net GPSRX_5V: now also U8.8 (B1)
- net GPSTX: now also U8.4 (A2)
- net GPSTX_5V: now also U8.1 (B2)
- net JRX: now also JP3.1 (A), U1.20 (28_RX7); no longer JP2.1 (A), U1.21 (29_TX7)
- net JTX: now also JP2.1 (A), U1.21 (29_TX7); no longer JP3.1 (A), U1.20 (28_RX7)
- new net: R68.2, U8.6 (OE)
- new net: C5.1, R67.1, U8.7 (VCCB)
Other:
- moved on the sheet: JCR1
