File: SpectDroneControl/SpectDroneControl.kicad_sch (KiCad schematic)
At the start: 140 parts, among them J1 Conn_02x03_Counter_Clockwise, J2-1 Conn_01x04_Male, J2-2 Conn_01x04_Male, J3-1 Conn_01x01_Female, J3-2 Conn_01x01_Female, J3-3 Conn_01x01_Female, J3-4 Conn_01x01_Female, J3-5 Conn_01x01_Female, J3V1 Conn_01x01_Male, J5-1 Conn_01x01_Female, J5-2 Conn_01x01_Female, J5-3 Conn_01x01_Female, J5-4 Conn_01x01_Female, J5-5 Conn_01x01_Female, Q1 FDN340P, Q2 Q_NPN_EBC, SW1 SW_SPDT, U1 Teensy4.1, U2 Teensy4.0, U3 NVT2010PW, U4 NVT2010PW, U5 NVT2010PW, U6 MCP112-450E/TO, U7 LM7805_SOT223, U8 TXS0102DCUR

Commit message: SpectDrone Development
Connections:
- net J5_1: now reaches J5-1.1 (Pin_1), R15.1, U3.22 (B1)
- net J3_1: now reaches J3-1.1 (Pin_1), R5.1, U3.3 (A1)
Changed lines of the file:
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@@
+    (effects (font (size 1.27 1.27)) (justify left bottom))
+  )
+  (label "J5_1" (at 114.935 88.265 0)
     (effects (font (size 1.27 1.27)) (justify left bottom))
   )
@@
     (effects (font (size 1.27 1.27)) (justify left bottom))
   )
+  (label "J3_1" (at 29.21 88.265 180)
+    (effects (font (size 1.27 1.27)) (justify right bottom))
+  )
   (label "SCL_5V" (at 114.935 187.325 0)
     (effects (font (size 1.27 1.27)) (justify left bottom))
@@
     (effects (font (size 1.27 1.27)) (justify left bottom))
   )
-  (label "TXS_{E}" (at 161.29 145.415 180)
+  (label "TXS_{E}" (at 162.56 147.32 180)
     (effects (font (size 1.27 1.27)) (justify right bottom))
   )

Commit message: SpectDrone Development
Parts:
- added C6, C7, C8: 0.1uF, Capacitor_SMD:C_0805_2012Metric, symbol Device:C_Small
- R10, R11, R12, R13, R14, R25, R26, R27, R28, R29, R30, R31, R32, R33, R34, R46, R47, R48, R49, R5, R50, R51, R52, R53, R54, R6, R7, R8, R9: value R -> 6K8
- R15, R16, R17, R18, R19, R20, R21, R22, R23, R24, R35, R36, R37, R38, R39, R40, R41, R42, R43, R44, R55, R56, R57, R58, R59, R60, R61, R62, R63, R64: value R -> 10K
- R2, R3, R4: value R -> 200K
Connections:
- net GND1: now also C6.1, C7.1, C8.1
- net TXS_{E}_5V: now also R68.2, U8.6 (OE)
- net at R4.1, U5.23 (VREFB), U5.24 (EN): now also C8.2
- net at R3.1, U4.23 (VREFB), U4.24 (EN): now also C7.2
- net at R2.1, U3.23 (VREFB), U3.24 (EN): now also C6.2
Other:
- moved on the sheet: BT1, J3-1, J3-2, J3-3, J3-4, J3-5, J5-1, J5-2, J5-3, J5-4, J5-5, JCS2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

Commit message: SpectDrone Development
Parts:
- added J5V1, JA1, JA2, JCMR1, JCMR2, JCMT1, JCMT2, JGND1, JMISO1, JMOSI1, JS1, JS2, JSCK1, JSCL1, JSDA1, JTXSE1: Conn_01x01_Female, Gardenuino Custom:SolderWire-0.1sqmm_1x01_D0.4mm_OD1mm, symbol Connector:Conn_01x01_Female
- added JPAX1: SolderJumper, Jumper:SolderJumper-3_P1.3mm_Bridged12_RoundedPad1.0x1.5mm, symbol Jumper:SolderJumper_3_Bridged12
- added R28: 6K8, Resistor_SMD:R_0805_2012Metric, symbol Device:R
- J3-1, J3-2, J3-3, J3-4, J3-5, J5-1, J5-2, J5-3, J5-4, J5-5, JAX1, JAX2, JAX3, JCAN_{H}1, JCAN_{L}1, JCRX3, JCS2, JCS3, JCTX3, JPPS1, JPPS2, JRX6, JRX8, JTX6, JTX8: footprint Connector_Wire:SolderWire-0.1sqmm_1x01_D0.4mm_OD1mm -> Gardenuino Custom:SolderWire-0.1sqmm_1x01_D0.4mm_OD1mm
- R2: renamed from R66; footprint Capacitor_SMD:C_0805_2012Metric -> Resistor_SMD:R_0805_2012Metric
- R3: renamed from R65; footprint Capacitor_SMD:C_0805_2012Metric -> Resistor_SMD:R_0805_2012Metric
- R68: renamed from R45; value X -> 200K
- R7-1: renamed from R67; footprint Capacitor_SMD:C_0805_2012Metric -> Resistor_SMD:R_0805_2012Metric
- R7-2: renamed from R68; footprint Capacitor_SMD:C_0805_2012Metric -> Resistor_SMD:R_0805_2012Metric
- U1: footprint Teensy:Teensy41 -> Gardenuino Custom:Teensy4.0-1
- renumbered C1 to C2-1, C3 to C2-2, C2 to C3, C6 to C4, C7 to C5, C8 to C6, C4 to C7-1, C5 to C7-2, JA1 to JADC1, R7 to R10, R8 to R11, R9 to R12, R10 to R13, R11 to R14, R12 to R15, R13 to R16, R14 to R17, R25 to R18, R26 to R19, R27 to R20, R28 to R21, R29 to R22, R30 to R23, R31 to R24, R32 to R25, R33 to R26, R34 to R27, R47 to R29, R46 to R30, R48 to R31, R49 to R32, R50 to R33, R51 to R34, R52 to R35, R53 to R36, R54 to R37, R15 to R38, R16 to R39, R2 to R4, R17 to R40, R18 to R41, R19 to R42, R20 to R43, R21 to R44, R22 to R45, R23 to R46, R24 to R47, R35 to R48, R36 to R49, R3 to R5, R37 to R50, R38 to R51, R39 to R52, R40 to R53, R41 to R54, R42 to R55, R43 to R56, R44 to R57, R55 to R58, R56 to R59, R4 to R6, R57 to R60, R58 to R61, R59 to R62, R60 to R63, R61 to R64, R62 to R65, R63 to R66, R64 to R67, R5 to R8, R6 to R9, U2 to U1-2, U7 to U2, U6 to U3, U3 to U4, U4 to U5, U5 to U6, U8 to U7
Connections:
- net 3V: no longer R68.2
- net 5V: now also J5V1.1 (Pin_1)
- net A1: now also JA1.1 (Pin_1)
- net A2: now also JA2.1 (Pin_1)
- net CAM1RX_5V: now also JCMR1.1 (Pin_1)
- net CAM1TX_5V: now also JCMT1.1 (Pin_1)
- net CAM2RX_5V: now also JCMR2.1 (Pin_1)
- net CAM2TX_5V: now also JCMT2.1 (Pin_1)
- net GND1: now also R68.1, U1.0-17 (GND), JGND1.1 (Pin_1)
- net MISO_5V: now also JMISO1.1 (Pin_1)
- net MOSI_5V: now also JMOSI1.1 (Pin_1)
- net S1: now also JS1.1 (Pin_1)
- net S2: now also JS2.1 (Pin_1)
- net SCK_5V: now also JSCK1.1 (Pin_1)
- net SCL_5V: now also JSCL1.1 (Pin_1)
- net SDA_5V: now also JSDA1.1 (Pin_1)
- net TXS_{E}: now also U1.0-16 (TXS_{e}), R28.1; no longer R68.1, U6.3 (A1)
- net TXS_{E}_5V: now also JTXSE1.1 (Pin_1)
- net VBat: now also U1.0-15 (VBAT)
- net AX1: now reaches JAX1.1 (Pin_1), U1.24 (32_OUT1B)
- net AX1: now also JPAX1.1 (A)
- net AX2: now reaches JAX2.1 (Pin_1), U1.25 (33_MCLK2)
- net at R1.2: now also JPAX1.2 (C); no longer SW1.2 (B)
- new net: R28.2, R68.2, U6.3 (A1)
- new net: JPAX1.3 (B), SW1.2 (B)
- no-connect marks 7 -> 42
Other:
- moved on the sheet: JADC1, JAPC1, JAUX1, JCAN_{H}1, JCAN_{L}1, JGPS1, JUT1, R1, R68, SW1

Commit message: SpectDrone Development
Parts:
- renumbered JS1 to JPD1, JS2 to JPD2, JA1 to JSR1, JA2 to JSR2, TP6 to TP4, TP4 to TP5, TP5 to TP6
Connections:
- net A1 is gone; now on net S1: JADC1.2 (Pin_2), JSR1.1 (Pin_1), U1-2.28 (21_A7_RX1_CS_PWM), U1.43 (21_A7_RX5_BCLK1)
- net A2 is gone; now on net S2: JADC1.4 (Pin_4), JSR2.1 (Pin_1), U1-2.30 (23_A9_Touch_PWM), U1.45 (23_A9_CRX1_MCLK1)
- net S1: no longer JADC1.1 (Pin_1), JPD1.1 (Pin_1), U1-2.27 (20_A6_CS_PWM), U1.42 (20_A6_TX5_LRCLK1)
- net S2: no longer JADC1.3 (Pin_3), JPD2.1 (Pin_1), U1-2.29 (22_A8_Touch_PWM), U1.44 (22_A8_CTX1)
- new net P1: JADC1.1 (Pin_1), JPD1.1 (Pin_1), U1-2.27 (20_A6_CS_PWM), U1.42 (20_A6_TX5_LRCLK1)
- new net P2: JADC1.3 (Pin_3), JPD2.1 (Pin_1), U1-2.29 (22_A8_Touch_PWM), U1.44 (22_A8_CTX1)
Changed lines of the file:
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@@
     (effects (font (size 1.27 1.27)) (justify right bottom))
   )
-  (label "A1" (at 52.07 26.67 0)
+  (label "S1" (at 52.07 26.67 0)
     (effects (font (size 1.27 1.27)) (justify left bottom))
   )
@@
     (effects (font (size 1.27 1.27)) (justify right bottom))
   )
-  (label "A1" (at 212.09 34.29 0)
+  (label "S1" (at 212.09 34.29 0)
     (effects (font (size 1.27 1.27)) (justify left bottom))
   )
@@
     (effects (font (size 1.27 1.27)) (justify right bottom))
   )
-  (label "S1" (at 212.09 36.83 0)
+  (label "P1" (at 212.09 36.83 0)
     (effects (font (size 1.27 1.27)) (justify left bottom))
   )
@@
     (effects (font (size 1.27 1.27)) (justify left bottom))
   )
-  (label "A1" (at 230.505 86.36 180)
+  (label "S1" (at 230.505 86.36 180)
     (effects (font (size 1.27 1.27)) (justify right bottom))
   )
@@
     (effects (font (size 1.27 1.27)) (justify right bottom))
   )
-  (label "A2" (at 212.09 29.21 0)
+  (label "S2" (at 212.09 29.21 0)
     (effects (font (size 1.27 1.27)) (justify left bottom))
   )
@@
     (effects (font (size 1.27 1.27)) (justify right bottom))
   )
-  (label "S2" (at 281.305 86.36 0)
+  (label "P2" (at 281.305 86.36 0)
     (effects (font (size 1.27 1.27)) (justify left bottom))
   )
-  (label "A2" (at 52.07 31.75 0)
+  (label "S2" (at 52.07 31.75 0)
     (effects (font (size 1.27 1.27)) (justify left bottom))
   )
@@
     (effects (font (size 1.27 1.27)) (justify left bottom))
   )
-  (label "S2" (at 212.09 31.75 0)
+  (label "P2" (at 212.09 31.75 0)
     (effects (font (size 1.27 1.27)) (justify left bottom))
   )
@@
     (effects (font (size 1.27 1.27)) (justify left bottom))
   )
-  (label "S2" (at 52.07 29.21 0)
+  (label "P2" (at 52.07 29.21 0)
     (effects (font (size 1.27 1.27)) (justify left bottom))
   )
@@
     (effects (font (size 1.27 1.27)) (justify left bottom))
   )
-  (label "A2" (at 281.305 83.82 0)
+  (label "S2" (at 281.305 83.82 0)
     (effects (font (size 1.27 1.27)) (justify left bottom))
   )
@@
     (effects (font (size 1.27 1.27)) (justify left bottom))
   )
-  (label "S1" (at 230.505 83.82 180)
+  (label "P1" (at 230.505 83.82 180)
     (effects (font (size 1.27 1.27)) (justify right bottom))
   )
@@
     (effects (font (size 1.27 1.27)) (justify right bottom))
   )
-  (label "S1" (at 52.07 24.13 0)
+  (label "P1" (at 52.07 24.13 0)
     (effects (font (size 1.27 1.27)) (justify left bottom))
   )
@@
   (symbol (lib_id "Connector:Conn_01x01_Female") (at 46.99 31.75 180) (unit 1)
     (in_bom yes) (on_board yes)
-    (property "Reference" "JA2" (id 0) (at 46.355 31.75 0)
+    (property "Reference" "JSR2" (id 0) (at 46.355 31.75 0)
       (effects (font (size 1.27 1.27)) (justify left))
     )
@@
   (symbol (lib_id "Connector:Conn_01x01_Female") (at 46.99 24.13 180) (unit 1)
     (in_bom yes) (on_board yes)
-    (property "Reference" "JS1" (id 0) (at 46.355 24.13 0)
+    (property "Reference" "JPD1" (id 0) (at 46.355 24.13 0)
       (effects (font (size 1.27 1.27)) (justify left))
     )
@@
   (symbol (lib_id "Connector:TestPoint") (at 264.795 160.02 270) (unit 1)
     (in_bom yes) (on_board yes)
-    (property "Reference" "TP5" (id 0) (at 269.875 158.75 90)
+    (property "Reference" "TP6" (id 0) (at 269.875 158.75 90)
       (effects (font (size 1.27 1.27)) (justify left))
     )
@@
   (symbol (lib_id "Connector:Conn_01x01_Female") (at 46.99 26.67 180) (unit 1)
     (in_bom yes) (on_board yes)
-    (property "Reference" "JA1" (id 0) (at 46.355 26.67 0)
+    (property "Reference" "JSR1" (id 0) (at 46.355 26.67 0)
       (effects (font (size 1.27 1.27)) (justify left))
     )
@@
   (symbol (lib_id "Connector:Conn_01x01_Female") (at 46.99 29.21 180) (unit 1)
     (in_bom yes) (on_board yes)
-    (property "Reference" "JS2" (id 0) (at 46.355 29.21 0)
+    (property "Reference" "JPD2" (id 0) (at 46.355 29.21 0)
       (effects (font (size 1.27 1.27)) (justify left))
     )
@@
       (effects (font (size 1.27 1.27)) hide)
     )
+    (pin "0-15")
+    (pin "0-16")
+    (pin "0-17")
+    (pin "0-18")
+    (pin "0-19")
     (pin "10")
     (pin "11")
@@
     (pin "23")
     (pin "24")
-    (pin "0-15")
     (pin "25")
-    (pin "0-16")
     (pin "26")
-    (pin "0-17")
     (pin "27")
-    (pin "0-18")
     (pin "28")
-    (pin "0-19")
     (pin "29")
     (pin "30")
@@
   (symbol (lib_id "Connector:TestPoint") (at 212.725 133.985 0) (unit 1)
     (in_bom yes) (on_board yes)
-    (property "Reference" "TP6" (id 0) (at 213.36 129.54 90)
+    (property "Reference" "TP4" (id 0) (at 213.36 129.54 90)
       (effects (font (size 1.27 1.27)) (justify left))
     )
@@
   (symbol (lib_id "Connector:TestPoint") (at 274.955 137.16 270) (unit 1)
     (in_bom yes) (on_board yes)
-    (property "Reference" "TP4" (id 0) (at 278.13 132.715 0)
+    (property "Reference" "TP5" (id 0) (at 278.13 132.715 0)
       (effects (font (size 1.27 1.27)) (justify left))
     )
@@
       (reference "J5V1") (unit 1) (value "Conn_01x01_Female") (footprint "Gardenuino Custom:SolderWire-0.1sqmm_1x01_D0.4mm_OD1mm")
     )
-    (path "/95f1e658-6de5-4ff6-b5e1-43b103874ec7"
-      (reference "JA1") (unit 1) (value "Conn_01x01_Female") (footprint "Gardenuino Custom:SolderWire-0.1sqmm_1x01_D0.4mm_OD1mm")
-    )
-    (path "/02dfd111-9da1-4721-9efe-b45bafeb5be8"
-      (reference "JA2") (unit 1) (value "Conn_01x01_Female") (footprint "Gardenuino Custom:SolderWire-0.1sqmm_1x01_D0.4mm_OD1mm")
-    )
     (path "/da546d77-4b03-4562-8fc6-837fd68e7691"
       (reference "JADC1") (unit 1) (value "Conn_01x04_Male") (footprint "Connector_PinHeader_2.54mm:PinHeader_1x04_P2.54mm_Vertical")
@@
       (reference "JPAX1") (unit 1) (value "SolderJumper") (footprint "Jumper:SolderJumper-3_P1.3mm_Bridged12_RoundedPad1.0x1.5mm")
     )
+    (path "/11f43f8c-faee-4437-9aa5-4367e18bf9bf"
+      (reference "JPD1") (unit 1) (value "Conn_01x01_Female") (footprint "Gardenuino Custom:SolderWire-0.1sqmm_1x01_D0.4mm_OD1mm")
+    )
+    (path "/d65aadf7-f352-40e1-a5fb-c8fddd193a24"
+      (reference "JPD2") (unit 1) (value "Conn_01x01_Female") (footprint "Gardenuino Custom:SolderWire-0.1sqmm_1x01_D0.4mm_OD1mm")
+    )
     (path "/3dd62eeb-7427-4721-89d0-49d4fb70bc68"
       (reference "JPPS1") (unit 1) (value "Conn_01x01_Female") (footprint "Gardenuino Custom:SolderWire-0.1sqmm_1x01_D0.4mm_OD1mm")
@@
       (reference "JRX8") (unit 1) (value "Conn_01x01_Female") (footprint "Gardenuino Custom:SolderWire-0.1sqmm_1x01_D0.4mm_OD1mm")
     )
-    (path "/11f43f8c-faee-4437-9aa5-4367e18bf9bf"
-      (reference "JS1") (unit 1) (value "Conn_01x01_Female") (footprint "Gardenuino Custom:SolderWire-0.1sqmm_1x01_D0.4mm_OD1mm")
-    )
-    (path "/d65aadf7-f352-40e1-a5fb-c8fddd193a24"
-      (reference "JS2") (unit 1) (value "Conn_01x01_Female") (footprint "Gardenuino Custom:SolderWire-0.1sqmm_1x01_D0.4mm_OD1mm")
-    )
     (path "/52464f5b-4071-4bee-952b-593875b54674"
       (reference "JSCK1") (unit 1) (value "Conn_01x01_Female") (footprint "Gardenuino Custom:SolderWire-0.1sqmm_1x01_D0.4mm_OD1mm")
@@
       (reference "JSDA1") (unit 1) (value "Conn_01x01_Female") (footprint "Gardenuino Custom:SolderWire-0.1sqmm_1x01_D0.4mm_OD1mm")
     )
+    (path "/95f1e658-6de5-4ff6-b5e1-43b103874ec7"
+      (reference "JSR1") (unit 1) (value "Conn_01x01_Female") (footprint "Gardenuino Custom:SolderWire-0.1sqmm_1x01_D0.4mm_OD1mm")
+    )
+    (path "/02dfd111-9da1-4721-9efe-b45bafeb5be8"
+      (reference "JSR2") (unit 1) (value "Conn_01x01_Female") (footprint "Gardenuino Custom:SolderWire-0.1sqmm_1x01_D0.4mm_OD1mm")
+    )
     (path "/3ac49f90-4050-4836-babd-2e934b6ad582"
       (reference "JTX6") (unit 1) (value "Conn_01x01_Female") (footprint "Gardenuino Custom:SolderWire-0.1sqmm_1x01_D0.4mm_OD1mm")
@@
       (reference "TP3") (unit 1) (value "TestPoint") (footprint "TestPoint:TestPoint_Keystone_5000-5004_Miniature")
     )
-    (path "/f5ff370a-f300-4577-b18d-5c4bec424748"
+    (path "/e7952da8-ed6d-40d6-bf3d-dd81f122ea3f"
       (reference "TP4") (unit 1) (value "TestPoint") (footprint "TestPoint:TestPoint_Keystone_5000-5004_Miniature")
     )
-    (path "/7d077e44-a436-402c-9cb4-20f8503d2301"
+    (path "/f5ff370a-f300-4577-b18d-5c4bec424748"
       (reference "TP5") (unit 1) (value "TestPoint") (footprint "TestPoint:TestPoint_Keystone_5000-5004_Miniature")
     )
-    (path "/e7952da8-ed6d-40d6-bf3d-dd81f122ea3f"
+    (path "/7d077e44-a436-402c-9cb4-20f8503d2301"
       (reference "TP6") (unit 1) (value "TestPoint") (footprint "TestPoint:TestPoint_Keystone_5000-5004_Miniature")
     )

Commit message: SpectDrone Development
Parts:
- added JP10, JP9: SolderJumper_2_Open, Jumper:SolderJumper-2_P1.3mm_Open_RoundedPad1.0x1.5mm, symbol Jumper:SolderJumper_2_Open
- renumbered J2-2 to J2-1, J2-1 to J2-2
Connections:
- net 5V: now also JP1.1 (A); no longer JP4.1 (A)
- net GND1: now also JP4.1 (A); no longer JP1.1 (A)
- net SCL: now also JP10.1 (A)
- net SDA: now also JP9.1 (A)
- net at J1.6 (Pin_6), J2-1.3 (Pin_3), JP3.2 (B): now also JP9.2 (B)
- net at J1.5 (Pin_5), J2-1.4 (Pin_4), JP4.2 (B): now also JP10.2 (B)
Other:
- moved on the sheet: J1, J2-1, J2-2, JP1, JP2, JP3, JP4, JP5, JP6, JP7, JP8

Commit message: SpectDrone Development
Parts:
- J2-1, J2-2, JADC1, JAPC1, JUT1: footprint Connector_PinHeader_2.54mm:PinHeader_1x04_P2.54mm_Vertical -> Connector_PinSocket_2.54mm:PinSocket_1x04_P2.54mm_Vertical; symbol Connector:Conn_01x04_Male -> Connector:Conn_01x04_Female
- J3V1, JVIN1: footprint Connector_PinHeader_2.54mm:PinHeader_1x01_P2.54mm_Vertical -> Connector_PinSocket_2.54mm:PinSocket_1x01_P2.54mm_Vertical; symbol Connector:Conn_01x01_Male -> Connector:Conn_01x01_Female
- JAUX1: footprint Connector_PinHeader_2.54mm:PinHeader_1x12_P2.54mm_Vertical -> Connector_PinSocket_2.54mm:PinSocket_1x12_P2.54mm_Vertical; symbol Connector:Conn_01x12_Male -> Connector:Conn_01x12_Female
- JD1: value Conn_01x04_Male -> Conn_01x04_Female; footprint Connector_PinHeader_2.54mm:PinHeader_1x04_P2.54mm_Vertical -> Connector_PinSocket_2.54mm:PinSocket_1x04_P2.54mm_Vertical; symbol Connector:Conn_01x04_Male -> Connector:Conn_01x04_Female
- JGPS1: footprint Connector_PinHeader_2.54mm:PinHeader_1x05_P2.54mm_Vertical -> Connector_PinSocket_2.54mm:PinSocket_1x05_P2.54mm_Vertical; symbol Connector:Conn_01x05_Male -> Connector:Conn_01x05_Female

Commit message: SpectDrone Development
Parts:
- added JGAIN1: SolderJumper, Jumper:SolderJumper-3_P1.3mm_Bridged12_RoundedPad1.0x1.5mm, symbol Jumper:SolderJumper_3_Bridged12
- BT1: Part Number (none) -> 3000
- C2-1: Part Number (none) -> 865090368008
- C2-2, C3, C4, C5, C6, C7-1, C7-2: Part Number (none) -> CL21B104KACNNNC
- D1: Part Number (none) -> PMEG10010ELRX
- D2: Part Number (none) -> HPZR-C7V0X
- J1: Part Number (none) -> RS2-08-G
- J2-1, J2-2, JADC1, JAPC1, JUT1: value Conn_01x04_Male -> Conn_01x04_Female; Part Number (none) -> PH1-04-UA
- J3-1, J3-2, J3-3, J3-4, J3-5: Part Number (none) -> RS1-01G; now left out of the parts list
- J3V1, JVIN1: value Conn_01x01_Male -> Conn_01x01_Female; Part Number (none) -> SSW-101-01-G-S
- J5-1, J5-2, J5-3, J5-4, J5-5, J5V1, JAX1, JAX2, JAX3, JCAN_{H}1, JCAN_{L}1, JCMR1, JCMR2, JCMT1, JCMT2, JCR1, JCRX3, JCS2, JCS3, JCTX3, JGND1, JMISO1, JMOSI1, JP1, JP10, JP2, JP3, JP4, JP5, JP6, JP7, JP8, JP9, JPAX1, JPD1, JPD2, JPPS1, JPPS2, JRX6, JRX8, JSCK1, JSCL1, JSDA1, JSR1, JSR2, JTX6, JTX8, JTXSE1, TP1, TP2, TP3, TP4, TP5, TP6: now left out of the parts list
- JAUX1: Part Number (none) -> RS1-12-G
- JD1: Part Number (none) -> PH1-04-UA
- JGPS1: Part Number (none) -> PH1-05-UA
- Q1: Part Number (none) -> FDN340P
- Q2: value Q_NPN_EBC -> NPN 50V 1A NPN_BEC; Part Number (none) -> ZUMT618
- R1: footprint Resistor_SMD:R_0603_1608Metric -> Resistor_SMD:R_0805_2012Metric; Part Number (none) -> ERJ-6ENF1002V
- R10, R11, R12, R13, R14, R15, R16, R17, R18, R19, R20, R21, R22, R23, R24, R25, R26, R27, R28, R29, R30, R31, R32, R33, R34, R35, R36, R37, R8, R9: Part Number (none) -> ERJ-6ENF6801V
- R2: Part Number (none) -> ERJ-6ENF1001V
- R3: Part Number (none) -> ERJ-6ENF1003V
- R38, R39, R40, R41, R42, R43, R44, R45, R46, R47, R48, R49, R50, R51, R52, R53, R54, R55, R56, R57, R58, R59, R60, R61, R62, R63, R64, R65, R66, R67: Part Number (none) -> ERJ-6ENF1002V
- R4, R5, R6, R68, R7-1, R7-2: Part Number (none) -> ERJ-6ENF2003V
- SW1: Part Number (none) -> JS102011SAQN
- U2: Part Number (none) -> LM7805_SOT223
- U3: Part Number (none) -> MCP112T-450E/MB
- U4, U5, U6: Part Number (none) -> NVT2010PW
- U7: Part Number (none) -> TXS0102DCUR
Connections:
- net 5V: now also JGAIN1.3 (B)
- net 7VDC: now also Q2.2 (E); no longer Q2.1 (E)
- net GND1: now also JGAIN1.1 (A)
- net at D2.1 (K), R2.1: now also Q2.1 (B); no longer Q2.2 (B)
- net at JPAX1.3 (B), SW1.2 (B): now also JGAIN1.2 (C)
Other:
- moved on the sheet: JPAX1, R1, SW1

Commit message: SpectDrone Development
Parts:
- JBAT1, JDC1, U1, U1-2: now left out of the parts list
Changed lines of the file:
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@@
   )
   (symbol (lib_id "Teensy:Teensy3.2") (at 255.905 52.07 0) (unit 1)
-    (in_bom yes) (on_board no)
+    (in_bom no) (on_board no)
     (property "Reference" "U1-2" (id 0) (at 255.905 13.97 0)
       (effects (font (size 1.524 1.524)))
@@
   )
   (symbol (lib_id "Connector:Conn_01x02_Female") (at 231.775 162.56 270) (unit 1)
-    (in_bom yes) (on_board yes)
+    (in_bom no) (on_board yes)
     (property "Reference" "JBAT1" (id 0) (at 232.41 160.655 90)
       (effects (font (size 1.27 1.27)) (justify left))
@@
   )
   (symbol (lib_id "Connector:Barrel_Jack_Switch") (at 274.32 125.095 0) (mirror y) (unit 1)
-    (in_bom yes) (on_board yes)
+    (in_bom no) (on_board yes)
     (property "Reference" "JDC1" (id 0) (at 269.24 118.11 0)
       (effects (font (size 1.27 1.27)) (justify right))
@@
   )
   (symbol (lib_id "Teensy:Teensy4.1") (at 184.15 76.2 0) (unit 1)
-    (in_bom yes) (on_board yes)
+    (in_bom no) (on_board yes)
     (property "Reference" "U1" (id 0) (at 184.15 13.97 0))
     (property "Value" "Teensy4.1" (id 1) (at 184.15 16.51 0))
@@
       (effects (font (size 1.27 1.27)) hide)
     )
-    (pin "2")
-    (pin "1")
+    (pin "1")
+    (pin "2")
     (pin "3")
   )
