File: SpectDroneControl/SpectDroneControl.kicad_sch (KiCad schematic)
At the start: 164 parts, among them J1 Conn_02x03_Counter_Clockwise, J2-1 Conn_01x04_Female, J2-2 Conn_01x04_Female, J3-1 Conn_01x01_Female, J3-2 Conn_01x01_Female, J3-3 Conn_01x01_Female, J3-4 Conn_01x01_Female, J3-5 Conn_01x01_Female, J3V1 Conn_01x01_Female, J5-1 Conn_01x01_Female, J5-2 Conn_01x01_Female, J5-3 Conn_01x01_Female, J5-4 Conn_01x01_Female, J5-5 Conn_01x01_Female, J5V1 Conn_01x01_Female, Q1 FDN340P, Q2 NPN 50V 1A NPN_BEC, SW1 SW_SPDT, U1 Teensy4.1, U1-2 Teensy4.0, U2 LM7805_SOT223, U3 MCP112-450E/TO, U4 NVT2010PW, U5 NVT2010PW, U6 NVT2010PW, U7 TXS0102DCUR

Commit message: SpectDrone Development
Connections:
- net P1: now also JADC1.2 (Pin_2), U1-2.28 (21_A7_RX1_CS_PWM), U1.43 (21_A7_RX5_BCLK1); no longer JADC1.1 (Pin_1), U1-2.27 (20_A6_CS_PWM), U1.42 (20_A6_TX5_LRCLK1)
- net S1: now also JADC1.1 (Pin_1), U1-2.27 (20_A6_CS_PWM), U1.42 (20_A6_TX5_LRCLK1); no longer JADC1.2 (Pin_2), U1-2.28 (21_A7_RX1_CS_PWM), U1.43 (21_A7_RX5_BCLK1)
Other:
- moved on the sheet: JPD1, JSR1

Commit message: SpectDrone Development
Parts:
- D2: value HPZR-C7V0X -> HPZR-C5V6X
Connections:
- net 7-12V1: no longer names the net of C2-2.2, D1.1 (K), Q1.2 (S), U2.1 (VI)
- net 7VDC: no longer names the net of C3.2, D1.2 (A), Q2.2 (E), R3.2, TP4.1, U3.2 (VDD)
Changed lines of the file:
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@@
     (stroke (width 0) (type default))
   )
-  (wire (pts (xy 248.285 133.985) (xy 248.285 137.16))
-    (stroke (width 0) (type default))
-  )
   (wire (pts (xy 266.065 105.41) (xy 266.065 107.315))
     (stroke (width 0) (type default))
@@
     (effects (font (size 1.27 1.27)) (justify right bottom))
   )
-  (label "7VDC" (at 216.535 137.16 0) (fields_autoplaced)
-    (effects (font (size 1.27 1.27)) (justify left bottom))
-  )
   (label "VBAT1" (at 231.775 157.48 0) (fields_autoplaced)
     (effects (font (size 1.27 1.27)) (justify left bottom))
@@
     (effects (font (size 1.27 1.27)) (justify right bottom))
   )
-  (label "7-12V1" (at 248.285 133.985 90) (fields_autoplaced)
-    (effects (font (size 1.27 1.27)) (justify left bottom))
-  )
   (label "APCRX_5V" (at 62.23 26.67 0) (fields_autoplaced)
     (effects (font (size 1.27 1.27)) (justify left bottom))
@@
       (effects (font (size 1.27 1.27)) (justify left))
     )
-    (property "Value" "HPZR-C7V0X" (at 231.14 118.11 0)
+    (property "Value" "HPZR-C5V6X" (at 231.14 118.11 0)
       (effects (font (size 1.27 1.27)) (justify left))
     )

Commit message: SpectDrone Development
Parts:
- removed JAX3: Conn_01x01_Female, Gardenuino Custom:SolderWire-0.1sqmm_1x01_D0.4mm_OD1mm, symbol Connector:Conn_01x01_Female
- added JP11, JP12, JP13, JP14: SolderJumper_2_Bridged, Jumper:SolderJumper-2_P1.3mm_Bridged_RoundedPad1.0x1.5mm, symbol Jumper:SolderJumper_2_Bridged
- added R68, R69: 100K, Resistor_SMD:R_0805_2012Metric, symbol Device:R
- D1: renamed from D2; value HPZR-C5V6X -> D; Part Number HPZR-C7V0X -> HPZR-C6V7X
- R1: renamed from R2; value 1K -> 10K
- renumbered U1 to A1, C2-1 to C1-1, C2-2 to C1-2, C3 to C2, C4 to C3, C5 to C4, C6 to C5, C7-1 to C6-1, C7-2 to C6-2, D1 to D2, Q2 to Q1, Q1 to Q2, R11 to R10, R12 to R11, R13 to R12, R14 to R13, R15 to R14, R16 to R15, R17 to R16, R18 to R17, R19 to R18, R20 to R19, R3 to R2, R21 to R20, R22 to R21, R23 to R22, R24 to R23, R25 to R24, R26 to R25, R27 to R26, R28 to R27, R29 to R28, R30 to R29, R4 to R3, R31 to R30, R32 to R31, R33 to R32, R34 to R33, R35 to R34, R36 to R35, R37 to R36, R38 to R37, R1 to R38, R5 to R4, R6 to R5, R7-1 to R6-1, R7-2 to R6-2, R8 to R7, R68 to R70, R9 to R8, R10 to R9, U2 to U1, U3 to U2, U4 to U3, U5 to U4, U6 to U5, U7 to U6
Connections:
- net GND1: now also R69.1
- net P1: now also JP12.2 (B); no longer A1.43 (21_A7_RX5_BCLK1)
- net P2: now also JP13.2 (B); no longer A1.44 (22_A8_CTX1)
- net S1: now also JP11.2 (B); no longer A1.42 (20_A6_TX5_LRCLK1)
- net S2: now also JP14.2 (B); no longer A1.45 (23_A9_CRX1_MCLK1)
- net 6V: now reaches C1-2.2, D2.1 (K), Q2.2 (S), U1.1 (VI)
- net 6.7V: now reaches C2.2, D2.2 (A), Q1.2 (E), R2.2, TP4.1, U2.2 (VDD)
- net A17: now reaches A1.33 (41_A17)
- net A17: now also R68.1, R69.2
- net VBAT1 renamed BAT_{V}
- net BAT_{V}: now also R68.2
- new net: A1.43 (21_A7_RX5_BCLK1), JP12.1 (A)
- new net: A1.44 (22_A8_CTX1), JP13.1 (A)
- new net: A1.42 (20_A6_TX5_LRCLK1), JP11.1 (A)
- new net: A1.45 (23_A9_CRX1_MCLK1), JP14.1 (A)
Other:
- moved on the sheet: A1, JAX1, JAX2, JCRX3, JCTX3, JP10, JP9, JPPS1, JRX6, JRX8, JTX6, JTX8

Commit message: SpectDrone Development
Parts:
- J1, J2-1, J2-2, J3V1, JADC1, JAPC1, JAUX1, JD1, JGPS1, JUT1, JVIN1: now left out of the parts list
- JDC1: footprint Connector_BarrelJack:BarrelJack_Horizontal -> Connector_BarrelJack:BarrelJack_CUI_PJ-063AH_Horizontal; symbol Connector:Barrel_Jack_Switch -> Connector:Barrel_Jack
Connections:
- net GND1: no longer JDC1.3
Changed lines of the file:
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@@
     (stroke (width 0) (type default))
   )
-  (wire (pts (xy 266.7 125.095) (xy 266.7 127.635))
-    (stroke (width 0) (type default))
-  )
   (wire (pts (xy 34.925 130.175) (xy 60.325 130.175))
     (stroke (width 0) (type default))
@@
   )
   (symbol (lib_id "Connector:Conn_01x12_Female") (at 113.03 35.56 0) (unit 1)
-    (in_bom yes) (on_board yes) (dnp no)
+    (in_bom no) (on_board yes) (dnp no)
     (property "Reference" "JAUX1" (at 111.76 38.1 90)
       (effects (font (size 1.27 1.27)) (justify left))
@@
   )
   (symbol (lib_id "Connector:Conn_01x01_Female") (at 257.175 160.02 0) (mirror y) (unit 1)
-    (in_bom yes) (on_board yes) (dnp no)
+    (in_bom no) (on_board yes) (dnp no)
     (property "Reference" "J3V1" (at 258.445 158.75 0)
       (effects (font (size 1.27 1.27)))
@@
   )
   (symbol (lib_id "Connector_Generic:Conn_02x04_Counter_Clockwise") (at 63.5 -31.75 0) (unit 1)
-    (in_bom yes) (on_board yes) (dnp no)
+    (in_bom no) (on_board yes) (dnp no)
     (property "Reference" "J1" (at 64.77 -38.1 0)
       (effects (font (size 1.27 1.27)))
@@
   )
   (symbol (lib_id "Connector:Conn_01x01_Female") (at 257.175 154.94 180) (unit 1)
-    (in_bom yes) (on_board yes) (dnp no)
+    (in_bom no) (on_board yes) (dnp no)
     (property "Reference" "JVIN1" (at 255.905 153.67 0)
       (effects (font (size 1.27 1.27)) (justify right))
@@
   )
   (symbol (lib_id "Connector:Conn_01x05_Female") (at 118.11 42.545 0) (mirror y) (unit 1)
-    (in_bom yes) (on_board yes) (dnp no)
+    (in_bom no) (on_board yes) (dnp no)
     (property "Reference" "JGPS1" (at 119.38 45.085 90)
       (effects (font (size 1.27 1.27)) (justify left))
@@
   )
   (symbol (lib_id "Connector:Conn_01x04_Female") (at 76.2 -31.75 0) (unit 1)
-    (in_bom yes) (on_board yes) (dnp no)
+    (in_bom no) (on_board yes) (dnp no)
     (property "Reference" "J2-1" (at 75.565 -27.94 0)
       (effects (font (size 1.27 1.27)))
@@
   )
   (symbol (lib_id "Connector:Conn_01x04_Female") (at 118.11 28.575 0) (mirror y) (unit 1)
-    (in_bom yes) (on_board yes) (dnp no)
+    (in_bom no) (on_board yes) (dnp no)
     (property "Reference" "JUT1" (at 119.38 29.845 90)
       (effects (font (size 1.27 1.27)))
@@
   )
   (symbol (lib_id "Connector:Conn_01x04_Female") (at 53.34 -31.75 0) (mirror y) (unit 1)
-    (in_bom yes) (on_board yes) (dnp no)
+    (in_bom no) (on_board yes) (dnp no)
     (property "Reference" "J2-2" (at 53.975 -27.94 0)
       (effects (font (size 1.27 1.27)))
@@
   )
   (symbol (lib_id "Connector:Conn_01x04_Female") (at 40.005 26.67 0) (unit 1)
-    (in_bom yes) (on_board yes) (dnp no)
+    (in_bom no) (on_board yes) (dnp no)
     (property "Reference" "JD1" (at 38.735 27.94 90)
       (effects (font (size 1.27 1.27)))
@@
   )
   (symbol (lib_id "Connector:Conn_01x04_Female") (at 76.835 26.67 0) (unit 1)
-    (in_bom yes) (on_board yes) (dnp no)
+    (in_bom no) (on_board yes) (dnp no)
     (property "Reference" "JAPC1" (at 75.565 27.94 90)
       (effects (font (size 1.27 1.27)))
@@
     )
   )
-  (symbol (lib_id "Connector:Barrel_Jack_Switch") (at 274.32 125.095 0) (mirror y) (unit 1)
+  (symbol (lib_id "Connector:Barrel_Jack") (at 274.32 125.095 0) (mirror y) (unit 1)
     (in_bom no) (on_board yes) (dnp no)
     (property "Reference" "JDC1" (at 269.24 118.11 0)
@@
       (effects (font (size 1.27 1.27)) (justify right))
     )
-    (property "Footprint" "Connector_BarrelJack:BarrelJack_Horizontal" (at 273.05 126.111 0)
+    (property "Footprint" "Connector_BarrelJack:BarrelJack_CUI_PJ-063AH_Horizontal" (at 273.05 126.111 0)
       (effects (font (size 1.27 1.27)) hide)
     )
@@
     (pin "1")
     (pin "2")
-    (pin "3")
     (instances
       (project "SpectDroneControl"
@@
   )
   (symbol (lib_id "Connector:Conn_01x04_Female") (at 59.055 26.67 0) (unit 1)
-    (in_bom yes) (on_board yes) (dnp no)
+    (in_bom no) (on_board yes) (dnp no)
     (property "Reference" "JADC1" (at 57.785 27.94 90)
       (effects (font (size 1.27 1.27)))

Commit message: SpectDrone Development
Parts:
- removed J3-1, J5-1, JRX6, JTX6: Conn_01x01_Female, Gardenuino Custom:SolderWire-0.1sqmm_1x01_D0.4mm_OD1mm, symbol Connector:Conn_01x01_Female
- removed JP10, JP9: SolderJumper_2_Open, Jumper:SolderJumper-2_P1.3mm_Open_RoundedPad1.0x1.5mm, symbol Jumper:SolderJumper_2_Open
- removed TP2: TestPoint, TestPoint:TestPoint_Keystone_5000-5004_Miniature, symbol Connector:TestPoint
- added JBAT2: Conn_01x02_Female, Connector_PinSocket_2.54mm:PinSocket_1x02_P2.54mm_Vertical, symbol Connector:Conn_01x02_Female
- JBAT1: footprint Connector_Molex:Molex_Micro-Fit_3.0_43045-0200_2x01_P3.00mm_Horizontal -> Gardenuino Custom:Molex_Micro-Fit_3.0_43045-0200_2x01_P3.00mm_Horizontal
- JDC1: symbol Connector:Barrel_Jack -> Connector:Barrel_Jack_MountingPin
- JP2, JP3: footprint Jumper:SolderJumper-2_P1.3mm_Open_RoundedPad1.0x1.5mm -> Jumper:SolderJumper-2_P1.3mm_Bridged_RoundedPad1.0x1.5mm; symbol Jumper:SolderJumper_2_Open -> Jumper:SolderJumper_2_Bridged; now in the parts list
- R38: value 10K -> 0
- SW1: now left out of the parts list
- TP1: footprint TestPoint:TestPoint_Keystone_5000-5004_Miniature -> Gardenuino Custom:TestPoint_Keystone_5000-5004_Miniature
- TP2: renamed from TP3; footprint TestPoint:TestPoint_Keystone_5000-5004_Miniature -> Gardenuino Custom:TestPoint_Keystone_5000-5004_Miniature
- TP3: renamed from TP4; footprint TestPoint:TestPoint_Keystone_5000-5004_Miniature -> Gardenuino Custom:TestPoint_Keystone_5000-5004_Miniature
- TP4: renamed from TP5; footprint TestPoint:TestPoint_Keystone_5000-5004_Miniature -> Gardenuino Custom:TestPoint_Keystone_5000-5004_Miniature
- TP5: renamed from TP6; footprint TestPoint:TestPoint_Keystone_5000-5004_Miniature -> Gardenuino Custom:TestPoint_Keystone_5000-5004_Miniature
- renumbered JVIN1 to JDCOUT1, J3-4 to JSCL-3, J5-4 to JSCL-5, J3-5 to JSDA-3, J5-5 to JSDA-5
Connections:
- net CAM1RX_5V is gone; now on net CS2_5V: JAUX1.10 (Pin_10), JCMR1.1 (Pin_1), R60.1, U5.20 (B3)
- net CAM1TX_5V is gone; now on net CS1_5V: JAUX1.11 (Pin_11), JCMT1.1 (Pin_1), R59.1, U5.21 (B2)
- net J5_1 is gone; now on net GAIN_5V: R37.1, U3.22 (B1)
- net VIN is gone; now on net VDC: JDCOUT1.1 (Pin_1), TP2.1
- net 3V: now also JGAIN1.3 (B), SW1.1 (A)
- net 5V: no longer JGAIN1.3 (B), SW1.1 (A)
- net BAT_{V}: now also JBAT2.1 (Pin_1)
- net CS1_5V: no longer JP5.1 (A), R54.1, U4.16 (B7)
- net CS2_5V: no longer JCS2.1 (Pin_1), R53.1, U4.17 (B6)
- net GAIN_5V: no longer R38.1
- net GND1: now also JBAT2.2 (Pin_2)
- net JRX: now also A1.12 (10_CS_MQSR); no longer A1.20 (28_RX7), JP3.1 (A)
- net JTX: now also A1.11 (9_OUT1C); no longer A1.21 (29_TX7), JP2.1 (A)
- net RX: now also A1.21 (29_TX7); no longer A1.12 (10_CS_MQSR)
- net TX: now also A1.20 (28_RX7); no longer A1.11 (9_OUT1C)
- net CAM1RX renamed CS2_3V
- net CAM1TX renamed CS1_3V
- net CAM2RX renamed ALT_RX_3V
- net CAM2RX_5V renamed ALT_RX_5V
- net CAM2TX renamed ALT_TX_3V
- net CAM2TX_5V renamed ALT_TX_5V
- net CS3_5V renamed CS3_5
- net J3_1 renamed GAIN_3V
- net GAIN_3V: now also R38.1
- net RX6 renamed SDA2
- net SDA2: now also JP2.1 (A)
- net RX6_5V renamed SDA2_5V
- net TX6 renamed SCL2
- net SCL2: now also JP3.1 (A)
- net TX6_5V renamed SCL2_5V
- new net CS1_5: JP5.1 (A), R54.1, U4.16 (B7)
- new net CS2_5: JCS2.1 (Pin_1), R53.1, U4.17 (B6)
- no-connect marks 42 -> 43
Other:
- moved on the sheet: J1, J2-1, J2-2, J5V1, JADC1, JAPC1, JAUX1, JCAN_{H}1, JCAN_{L}1, JCMR1, JCMR2, JCMT1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

Commit message: SpectDrone Development
Parts:
- removed J3V1, JDCOUT1: Conn_01x01_Female, Connector_PinSocket_2.54mm:PinSocket_1x01_P2.54mm_Vertical, symbol Connector:Conn_01x01_Female
- removed JBAT2: Conn_01x02_Female, Connector_PinSocket_2.54mm:PinSocket_1x02_P2.54mm_Vertical, symbol Connector:Conn_01x02_Female
- added J2: Conn_01x03_Socket, Connector_PinSocket_2.54mm:PinSocket_1x03_P2.54mm_Vertical, symbol Connector:Conn_01x03_Socket
Connections:
- net 3V: now also J2.3 (Pin_3)
- net BAT_{V}: now also J2.2 (Pin_2)
- net VDC: now also J2.1 (Pin_1)
Other:
- moved on the sheet: TP2, TP5
