File: SpectDroneControl/_autosave-SpectDroneControl.kicad_pcb (KiCad board)
At the start: 2 copper layers, 101.6 x 73.7 mm, 166 parts, among them J1 Conn_02x03_Counter_Clockwise, J2-1 Conn_01x04_Female, J2-2 Conn_01x04_Female, J3-1 Conn_01x01_Female, J3-2 Conn_01x01_Female, J3-3 Conn_01x01_Female, J3-4 Conn_01x01_Female, J3-5 Conn_01x01_Female, J3V1 Conn_01x01_Female, J5-1 Conn_01x01_Female, J5-2 Conn_01x01_Female, J5-3 Conn_01x01_Female, J5-4 Conn_01x01_Female, J5-5 Conn_01x01_Female, J5V1 Conn_01x01_Female, Q1 FDN340P, Q2 NPN 50V 1A NPN_BEC, SW1 SW_SPDT, U1 Teensy4.1, U2 LM7805_SOT223, U3 MCP112-450E/TO, U4 NVT2010PW, U5 NVT2010PW, U6 NVT2010PW, U7 TXS0102DCUR

Commit message: SpectDrone Development
Routing:
- net /5V: track 202.4 -> 246.3 mm, vias 5 -> 7
- net GND1: track 81.1 -> 108.4 mm, vias 3 -> 5
- added copper zone on In2.Cu, net /5V
- added copper zone on In1.Cu, net GND1
- removed copper zone on B.Cu, net /5V
- removed copper zone on F.Cu, net GND1
Other:
- copper layers 2 -> 4
