File: TestComponents/InsturmentationsAmps.kicad_sch (KiCad schematic)
At the start: 30 parts

Commit message: SpectDrone Development
Parts:
- added CS11, CS13: 0.1uF, Capacitor_SMD:C_0805_2012Metric, symbol Device:C_Small
- added CS12: 10uF, Capacitor_SMD:C_0805_2012Metric, symbol Device:C_Small
- added R1: 10K, symbol Device:R
- added R2: 2K67, symbol Device:R
- added SW2: SW_SPDT, Button_Switch_SMD:SW_SPDT_CK-JS102011SAQN, symbol Switch:SW_SPDT
- added SW3: SW_DPDT_x2, Button_Switch_THT:SW_CuK_JS202011AQN_DPDT_Angled, symbol Switch:SW_DPDT_x2
- added U2: REF200AU, Package_SO:SOIC-8_3.9x4.9mm_P1.27mm, symbol Reference_Current:REF200AU
- added U3: MCP6L01x-xLT, Package_TO_SOT_SMD:SOT-353_SC-70-5, symbol Amplifier_Operational:MCP6L01x-xLT
Connections:
- net GND1: now also CS12.2, CS13.1, SW3.6 (C), U3.2 (V-)
- net V_{AREF}: now also CS12.1, CS13.2, U3.5 (V+)
- net PD1_{TEST}: now reaches JPD2.1 (A), JPD3.1 (A), PD1.1 (A)
- net PD1_{TEST}: now also SW2.1 (A)
- net PD2_{TEST}: now reaches JPD5.1 (A), JPD6.1 (A), PD2.1 (A)
- net PD2_{TEST}: now also SW2.3 (C)
- new net: CS11.2, R1.1, U2.3, U3.3 (+)
- new net: CS11.1, R1.2, R2.2, U3.1
- new net: U2.1, U2.2, U2.5
- new net: U2.6 (S), U2.6 (S), U2.6 (S)
- new net -I_{const}: R2.1, SW3.5 (B), U3.4 (-)
- new net 5V3: SW3.1 (A)
- new net I_{input}: SW3.2 (B), U2.4, U2.7, U2.8
- new net PD_{TEST}: SW2.2 (B), SW3.3 (C), SW3.4 (A)
Other:
- note added: "I_{C}=400.0uA ↓"
- note added: "I_{out} = N * I_{C} I_{C} = 400uA I_{out} = 1500uA N = I_{out} / I_{C} = 1500uA / 400uA = 3.75 R_{1} = N * R_{2} R_{1} = 10K R_{2} = R_{1} / N = 10Kohm / 3.75 = 2.~{6}Kohm"
- note added: "I_{out}=1500.0uA ↓"
- moved on the sheet: CS1, CS10, CS2, CS3, CS4, CS5, CS6, CS7, CS8, CS9, JPD1, JPD2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

Commit message: SpectDrone Development
Parts:
- renumbered U2 to U3, U3 to U4
Other:
- note added: "Calibration currents 400uA and 1500uA if V_{AREF} = 3.00V and I_{"PD"} = 400uA then"
Changed lines of the file:
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@@
     (effects (font (size 1.27 1.27)) (justify right bottom))
+  )
+  (text "Calibration currents 400uA and 1500uA\n\nif V_{AREF} = 3.00V and I_{\"PD\"} = 400uA then "
+    (at 135.89 38.735 0)
+    (effects (font (size 1.27 1.27)) (justify left bottom))
   )
   (label "PD1_{TEST}" (at 33.655 66.675 180)
@@
   (symbol (lib_id "Reference_Current:REF200AU") (at 101.6 82.55 0) (unit 3)
     (in_bom yes) (on_board yes) (fields_autoplaced)
-    (property "Reference" "U2" (id 0) (at 112.395 81.2799 0)
-      (effects (font (size 1.27 1.27)) (justify left))
-    )
-    (property "Value" "REF200AU" (id 1) (at 112.395 83.8199 0)
+    (property "Reference" "U3" (id 0) (at 111.76 81.2799 0)
+      (effects (font (size 1.27 1.27)) (justify left))
+    )
+    (property "Value" "REF200AU" (id 1) (at 111.76 83.8199 0)
       (effects (font (size 1.27 1.27) italic) (justify left))
     )
@@
   (symbol (lib_id "Reference_Current:REF200AU") (at 104.775 63.5 0) (unit 2)
     (in_bom yes) (on_board yes) (fields_autoplaced)
-    (property "Reference" "U2" (id 0) (at 109.855 62.2299 0)
-      (effects (font (size 1.27 1.27)) (justify left))
-    )
-    (property "Value" "REF200AU" (id 1) (at 109.855 64.7699 0)
+    (property "Reference" "U3" (id 0) (at 110.49 62.2299 0)
+      (effects (font (size 1.27 1.27)) (justify left))
+    )
+    (property "Value" "REF200AU" (id 1) (at 110.49 64.7699 0)
       (effects (font (size 1.27 1.27) italic) (justify left))
     )
@@
   (symbol (lib_id "Reference_Current:REF200AU") (at 98.425 63.5 0) (mirror y) (unit 1)
     (in_bom yes) (on_board yes)
-    (property "Reference" "U2" (id 0) (at 88.9 62.865 0)
+    (property "Reference" "U3" (id 0) (at 88.9 62.865 0)
       (effects (font (size 1.27 1.27)) (justify right))
     )
@@
   (symbol (lib_id "Amplifier_Operational:MCP6L01x-xLT") (at 109.855 111.76 0) (unit 1)
     (in_bom yes) (on_board yes)
-    (property "Reference" "U3" (id 0) (at 93.98 110.49 0))
+    (property "Reference" "U4" (id 0) (at 93.98 110.49 0))
     (property "Value" "MCP6L01x-xLT" (id 1) (at 93.98 113.03 0))
     (property "Footprint" "Package_TO_SOT_SMD:SOT-353_SC-70-5" (id 2) (at 107.315 116.84 0)

Commit message: SpectDrone Development
Parts:
- R1, R2: footprint (none) -> Resistor_SMD:R_0805_2012Metric
- SW2: value SW_SPDT -> SW_SP3T; footprint Button_Switch_SMD:SW_SPDT_CK-JS102011SAQN -> Button_Switch_SMD:SW_SP3T_PCM13; symbol Switch:SW_SPDT -> Switch:SW_SP3T
Connections:
- net PD2_{TEST}: now also SW2.4; no longer SW2.3 (C)
- net PD_{TEST}: now also SW2.3; no longer SW2.2 (B)
- no-connect marks 0 -> 1
Changed lines of the file:
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@@
   (junction (at 248.92 85.09) (diameter 0) (color 0 0 0 0)
   )
+  (no_connect (at 33.655 69.215))
   (wire (pts (xy 200.025 80.01) (xy 207.645 80.01))
     (stroke (width 0) (type default) (color 0 0 0 0))
@@
     (property "Reference" "R1" (id 0) (at 111.125 96.52 90))
     (property "Value" "10K" (id 1) (at 111.125 99.06 90))
-    (property "Footprint" "" (id 2) (at 111.125 100.838 90)
+    (property "Footprint" "Resistor_SMD:R_0805_2012Metric" (id 2) (at 111.125 100.838 90)
       (effects (font (size 1.27 1.27)) hide)
     )
@@
     (pin "2")
   )
-  (symbol (lib_id "Switch:SW_SPDT") (at 38.735 69.215 0) (mirror y) (unit 1)
+  (symbol (lib_id "Switch:SW_SP3T") (at 38.735 69.215 0) (mirror y) (unit 1)
     (in_bom yes) (on_board yes) (fields_autoplaced)
     (property "Reference" "SW2" (id 0) (at 38.735 60.96 0))
-    (property "Value" "SW_SPDT" (id 1) (at 38.735 63.5 0))
-    (property "Footprint" "Button_Switch_SMD:SW_SPDT_CK-JS102011SAQN" (id 2) (at 38.735 69.215 0)
-      (effects (font (size 1.27 1.27)) hide)
-    )
-    (property "Datasheet" "~" (id 3) (at 38.735 69.215 0)
+    (property "Value" "SW_SP3T" (id 1) (at 38.735 63.5 0))
+    (property "Footprint" "Button_Switch_SMD:SW_SP3T_PCM13" (id 2) (at 54.61 64.77 0)
+      (effects (font (size 1.27 1.27)) hide)
+    )
+    (property "Datasheet" "~" (id 3) (at 54.61 64.77 0)
       (effects (font (size 1.27 1.27)) hide)
     )
@@
     (pin "2")
     (pin "3")
+    (pin "4")
   )
   (symbol (lib_id "Device:R") (at 106.68 124.46 90) (mirror x) (unit 1)
@@
     (property "Reference" "R2" (id 0) (at 106.68 121.92 90))
     (property "Value" "2K67" (id 1) (at 106.68 124.46 90))
-    (property "Footprint" "" (id 2) (at 106.68 122.682 90)
-      (effects (font (size 1.27 1.27)) hide)
-    )
+    (property "Footprint" "Resistor_SMD:R_0805_2012Metric" (id 2) (at 106.68 122.682 90)
+      (effects (font (size 1.27 1.27)) hide)
+    )

Commit message: SpectDrone Development
Parts:
- removed SW3: SW_DPDT_x2, Button_Switch_THT:SW_CuK_JS202011AQN_DPDT_Angled, symbol Switch:SW_DPDT_x2
- added SW3: SW_SP3T, Button_Switch_SMD:SW_SP3T_PCM13, symbol Switch:SW_SP3T
- R_{PD}1, R_{PD}2: value X -> 2K
Connections:
- net PD2 is gone; now on net PD(V)_{BIAS}: JPD4.1 (A), PD2.2 (K)
- net PD1_{TEST}: now also JPD1.2 (B), JPD2.2 (B), RS3.1, R_{PD}1.1; no longer JPD2.1 (A), JPD3.1 (A), PD1.1 (A)
- net PD2_{TEST}: now also JPD4.2 (B), JPD5.2 (B), RS7.1, R_{PD}2.1; no longer JPD5.1 (A), JPD6.1 (A), PD2.1 (A)
- net PD_{TEST}: now also SW3.3
- net -I_{const} renamed -I_{const}=1.5mA
- net -I_{const}=1.5mA: now also SW3.4
- net I_{input} renamed -I_{const}=0.4mA
- net -I_{const}=0.4mA: now also SW3.1
- net PD1 renamed PD(V)_{BIAS}
- new net: JPD2.1 (A), JPD3.1 (A), PD1.1 (A)
- new net: JPD5.1 (A), JPD6.1 (A), PD2.1 (A)
- no-connect marks 1 -> 2
Other:
- note added: "Calibration currents 400uA and 1500uA"
- note added: "V = IR V = PD(V)_{BIAS} = [ 1.00 | 3.00V ] I = I_{C} = [ 0.4mA | 1.5mA ] PD(V)_{BIAS} = I_{C} * R R = PD(V)_{BIAS} / I_{C} "Dark" current = ~ 5.0pA R = 1.00V / 5.0pA = 0.2Tohm ~= 1Gohm R = 3.00V / 5.0pA = 0.6Tohm ~= 1Gohm "Mid-zenith" current = 400uA R = 1.00V / 0.4mA = 2.5Kohm R = 3.00V / 0.4mA = 7.5Kohm "High-zenith" current = 1500uA R = 1.00V / 1.5mA = 667ohm R = 3.00V / 1.5mA = 2.0Kohm"
- note added: "if V_{AREF} = 1.00V, I_{"PD"} = 0.400mA, R_{PD} = 100 ohm if V_{AREF} = 1.00V, I_{"PD"} = 1.500mA, R_{PD} = 100 ohm if V_{AREF} = 3.00V, I_{"PD"} = 0.400mA, R_{PD} = 100 ohm if V_{AREF} = 3.00V, I_{"PD"} = 1.500mA, R_{PD} = 100 ohm"
- note added: "↓ I_{C}=400.0uA"
- note added: "↓ I_{out}=1500.0uA"
- note removed: "Calibration currents 400uA and 1500uA if V_{AREF} = 3.00V and I_{"PD"} = 400uA then"
- note removed: "I_{C}=400.0uA ↓"
- note removed: "I_{out}=1500.0uA ↓"
- moved on the sheet: CS1, CS10, CS11, CS12, CS13, CS2, CS3, CS4, CS5, CS6, CS7, CS8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
