File: TestComponents/InsturmentationsAmps.kicad_sch (KiCad schematic)
At the start: 39 parts, among them SW2 SW_SP3T, SW3 SW_SP3T, U3 REF200AU, U4 MCP6L01x-xLT

Commit message: SpectDrone Development
Parts:
- added R_{PD}1.1, R_{PD}2.1: 2K, Capacitor_SMD:C_0805_2012Metric, symbol Device:R
- R_{PD}1, R_{PD}2: value 2K -> 1M
Connections:
- net PD1_{TEST}: now also R_{PD}1.1.2; no longer JPD1.2 (B), JPD2.2 (B)
- net PD2_{TEST}: now also R_{PD}2.1.2; no longer JPD4.2 (B), JPD5.2 (B)
- new net: JPD4.2 (B), JPD5.2 (B), R_{PD}2.1.1
- new net: JPD1.2 (B), JPD2.2 (B), R_{PD}1.1.1
Other:
- note added: "R = 666.6 ohm | V_{in} | I_{C} | PD_{V} | Gain | PD_{OUT} | Ratio | Digital_{1024} | Digital_{4096} | Digital_{262K} | Digital_{16M} | ------------------------------------------------------------------------------ | 3.000 | 0.400 | 2.730 | 1.00 | 2.730 | 0.910 | 932 | 3727 | 238551 | 15267267 | | 1.000 | 0.400 | 0.733 | 3.00 | 2.199 | 0.733 | 751 | 3002 | 192152 | 12297699 | | 3.000 | 1.500 | 2.0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"
Changed lines of the file:
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@@
     (stroke (width 0) (type default) (color 0 0 0 0))
   )
-  (wire (pts (xy 211.455 54.61) (xy 220.98 54.61))
+  (wire (pts (xy 211.455 54.61) (xy 212.725 54.61))
     (stroke (width 0) (type default) (color 0 0 0 0))
   )
@@
     (stroke (width 0) (type default) (color 0 0 0 0))
   )
+  (wire (pts (xy 220.345 54.61) (xy 220.98 54.61))
+    (stroke (width 0) (type default) (color 0 0 0 0))
+  )
   (polyline (pts (xy 283.21 77.47) (xy 243.205 77.47))
     (stroke (width 0) (type default) (color 0 0 0 0))
@@
     (stroke (width 0) (type default) (color 0 0 0 0))
   )
+  (wire (pts (xy 220.345 24.13) (xy 220.98 24.13))
+    (stroke (width 0) (type default) (color 0 0 0 0))
+  )
   (wire (pts (xy 72.39 104.14) (xy 76.835 104.14))
     (stroke (width 0) (type default) (color 0 0 0 0))
@@
     (stroke (width 0) (type default) (color 0 0 0 0))
   )
-  (wire (pts (xy 211.455 24.13) (xy 220.98 24.13))
+  (wire (pts (xy 211.455 24.13) (xy 212.725 24.13))
     (stroke (width 0) (type default) (color 0 0 0 0))
   )
@@
   )
   (text "↓ I_{C}=400.0uA" (at 90.805 69.215 0)
+    (effects (font (size 1.27 1.27)) (justify left bottom))
+  )
+  (text "R = 666.6 ohm\n\n|   V_{in}     |   I_{C}     |   PD_{V}   |  Gain  |  PD_{OUT}  | Ratio |  Digital_{1024}  |  Digital_{4096}   |  Digital_{262K}  |  Digital_{16M}   |\n------------------------------------------------------------------------------\n|  3.000   |  0.400  |  2.730  |  1.00  |  2.730  | 0.910 |         932  |       3727  |     238551  |   15267267  |\n|  1.000   |  0.400  |  0.733  |  3.00  |  2.199  | 0.733 |         751  |       3002  |     192152  |   12297699  |\n|  3.000   |  1.500  |  2.000  |  1.00  |  2.000  | 0.666 |         683  |       2728  |     174588  |   11173626  |\n|  1.000   |  0.400  |  0.733  |  1.00  |  0.733  | 0.244 |         250  |       1001  |      64051  |    4099233  |\n|  1.000   |  1.500  |  0.000  |  1.00  |  0.000  | 0.000 |"
+    (at 120.65 98.425 0)
     (effects (font (size 1.27 1.27)) (justify left bottom))
   )
@@
       (effects (font (size 1.27 1.27)) (justify right) hide)
     )
+  )
+  (symbol (lib_id "Device:R") (at 216.535 54.61 90) (unit 1)
+    (in_bom yes) (on_board yes)
+    (property "Reference" "R_{PD}2.1" (id 0) (at 219.075 52.705 90)
+      (effects (font (size 1.27 1.27)) (justify left))
+    )
+    (property "Value" "2K" (id 1) (at 218.44 54.61 90)
+      (effects (font (size 1.27 1.27)) (justify left))
+    )
+    (property "Footprint" "Capacitor_SMD:C_0805_2012Metric" (id 2) (at 216.535 56.388 90)
+      (effects (font (size 1.27 1.27)) hide)
+    )
+    (property "Datasheet" "~" (id 3) (at 216.535 54.61 0)
+      (effects (font (size 1.27 1.27)) hide)
+    )
+    (pin "1")
+    (pin "2")
   )
   (symbol (lib_id "Switch:SW_SP3T") (at 143.51 59.69 0) (mirror y) (unit 1)
@@
   (symbol (lib_id "Device:R") (at 220.98 29.21 0) (unit 1)
     (in_bom yes) (on_board yes)
-    (property "Reference" "R_{PD}1" (id 0) (at 215.265 26.035 0)
-      (effects (font (size 1.27 1.27)) (justify left))
-    )
-    (property "Value" "2K" (id 1) (at 220.98 31.115 90)
+    (property "Reference" "R_{PD}1" (id 0) (at 215.265 27.94 0)
+      (effects (font (size 1.27 1.27)) (justify left))
+    )
+    (property "Value" "1M" (id 1) (at 220.98 31.115 90)
       (effects (font (size 1.27 1.27)) (justify left))
     )
@@
     (pin "2")
   )
+  (symbol (lib_id "Device:R") (at 216.535 24.13 90) (unit 1)
+    (in_bom yes) (on_board yes)
+    (property "Reference" "R_{PD}1.1" (id 0) (at 219.075 22.225 90)
+      (effects (font (size 1.27 1.27)) (justify left))
+    )
+    (property "Value" "2K" (id 1) (at 218.44 24.13 90)
+      (effects (font (size 1.27 1.27)) (justify left))
+    )
+    (property "Footprint" "Capacitor_SMD:C_0805_2012Metric" (id 2) (at 216.535 25.908 90)
+      (effects (font (size 1.27 1.27)) hide)
+    )
+    (property "Datasheet" "~" (id 3) (at 216.535 24.13 0)
+      (effects (font (size 1.27 1.27)) hide)
+    )
+    (pin "1")
+    (pin "2")
+  )
   (symbol (lib_id "Device:C_Small") (at 59.69 95.25 0) (mirror x) (unit 1)
     (in_bom yes) (on_board yes)
@@
   (symbol (lib_id "Device:R") (at 220.98 59.69 0) (unit 1)
     (in_bom yes) (on_board yes)
-    (property "Reference" "R_{PD}2" (id 0) (at 215.265 56.515 0)
-      (effects (font (size 1.27 1.27)) (justify left))
-    )
-    (property "Value" "2K" (id 1) (at 220.98 61.595 90)
-      (effects (font (size 1.27 1.27)) (justify left))
-    )
+    (property "Reference" "R_{PD}2" (id 0) (at 215.265 58.42 0)
+      (effects (font (size 1.27 1.27)) (justify left))
+    )
+    (property "Value" "1M" (id 1) (at 220.98 61.595 90)
+      (effects (font (size 1.27 1.27)) (justify left))
+    )

Commit message: SpectDrone Development
Parts:
- removed SW2, SW3: SW_SP3T, Button_Switch_SMD:SW_SP3T_PCM13, symbol Switch:SW_SP3T
- added R_{C}1: 500, Capacitor_SMD:C_0805_2012Metric, symbol Device:R
- added SW2: SW_DP3T, Gardenuino Custom:SW_DP3T_CK_JS203011JAQN, symbol Switch:SW_DP3T
- added SW3: SW_DPDT, Gardenuino Custom:SW_DPDT_CK_JS202011JAQN, symbol Switch:SW_DPDT_x2
Connections:
- net -I_{const}=0.4mA: now also SW3.3 (C), SW3.4 (A)
- net -I_{const}=1.5mA: now also SW3.1 (A)
- net PD(V)_{BIAS}: now also R_{C}1.2
- net PD1_{TEST}: now also SW2.1
- net PD2_{TEST}: now also SW2.4
- net PD_{TEST}: now also SW2.3, SW3.2 (B)
- new net: R_{C}1.1, SW3.5 (B)
- no-connect marks 2 -> 6
Other:
- note added: "R = 666.6 ohm | V_{in} | I_{C} | PD_{V} | Gain | PD_{OUT} | Ratio | Digital_{1024} | Digital_{4096} | Digital_{262K} | Digital_{16M} | ------------------------------------------------------------------------------ | 3.000 | 0.400 | 2.730 | 1.00 | 2.730 | 0.910 | 932 | 3727 | 238551 | 15267267 | | 3.000 | 1.500 | 2.000 | 1.00 | 2.000 | 0.666 | 683 | 2728 | 174588 | 11173626 | | 1.000 | 0.400 | 0.7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"
- note removed: "Calibration currents 400uA and 1500uA"
- note removed: "R = 666.6 ohm | V_{in} | I_{C} | PD_{V} | Gain | PD_{OUT} | Ratio | Digital_{1024} | Digital_{4096} | Digital_{262K} | Digital_{16M} | ------------------------------------------------------------------------------ | 3.000 | 0.400 | 2.730 | 1.00 | 2.730 | 0.910 | 932 | 3727 | 238551 | 15267267 | | 1.000 | 0.400 | 0.733 | 3.00 | 2.199 | 0.733 | 751 | 3002 | 192152 | 12297699 | | 3.000 | 1.500 | 2.0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"
- note removed: "if V_{AREF} = 1.00V, I_{"PD"} = 0.400mA, R_{PD} = 100 ohm if V_{AREF} = 1.00V, I_{"PD"} = 1.500mA, R_{PD} = 100 ohm if V_{AREF} = 3.00V, I_{"PD"} = 0.400mA, R_{PD} = 100 ohm if V_{AREF} = 3.00V, I_{"PD"} = 1.500mA, R_{PD} = 100 ohm"
- moved on the sheet: CS1, CS10, CS11, CS12, CS13, CS2, CS3, CS4, CS5, CS6, CS7, CS8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

Commit message: SpectDrone Development
Parts:
- RS3, RS6, RS7, RS8, R_{C}1, R_{PD}1, R_{PD}1.1, R_{PD}2, R_{PD}2.1: footprint Capacitor_SMD:C_0805_2012Metric -> Resistor_SMD:R_0805_2012Metric
Changed lines of the file:
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@@
       (effects (font (size 1.27 1.27)) (justify left))
     )
-    (property "Footprint" "Capacitor_SMD:C_0805_2012Metric" (id 2) (at 195.58 81.788 90)
+    (property "Footprint" "Resistor_SMD:R_0805_2012Metric" (id 2) (at 195.58 81.788 90)
       (effects (font (size 1.27 1.27)) hide)
     )
@@
       (effects (font (size 1.27 1.27)) (justify left))
     )
-    (property "Footprint" "Capacitor_SMD:C_0805_2012Metric" (id 2) (at 208.28 61.468 90)
+    (property "Footprint" "Resistor_SMD:R_0805_2012Metric" (id 2) (at 208.28 61.468 90)
       (effects (font (size 1.27 1.27)) hide)
     )
@@
       (effects (font (size 1.27 1.27)) (justify left))
     )
-    (property "Footprint" "Capacitor_SMD:C_0805_2012Metric" (id 2) (at 198.247 54.61 90)
+    (property "Footprint" "Resistor_SMD:R_0805_2012Metric" (id 2) (at 198.247 54.61 90)
       (effects (font (size 1.27 1.27)) hide)
     )
@@
       (effects (font (size 1.27 1.27)) (justify left))
     )
-    (property "Footprint" "Capacitor_SMD:C_0805_2012Metric" (id 2) (at 125.73 58.928 90)
+    (property "Footprint" "Resistor_SMD:R_0805_2012Metric" (id 2) (at 125.73 58.928 90)
       (effects (font (size 1.27 1.27)) hide)
     )
@@
       (effects (font (size 1.27 1.27)) (justify left))
     )
-    (property "Footprint" "Capacitor_SMD:C_0805_2012Metric" (id 2) (at 208.28 91.948 90)
+    (property "Footprint" "Resistor_SMD:R_0805_2012Metric" (id 2) (at 208.28 91.948 90)
       (effects (font (size 1.27 1.27)) hide)
     )
@@
       (effects (font (size 1.27 1.27)) (justify left))
     )
-    (property "Footprint" "Capacitor_SMD:C_0805_2012Metric" (id 2) (at 195.58 51.308 90)
+    (property "Footprint" "Resistor_SMD:R_0805_2012Metric" (id 2) (at 195.58 51.308 90)
       (effects (font (size 1.27 1.27)) hide)
     )
@@
       (effects (font (size 1.27 1.27)) (justify left))
     )
-    (property "Footprint" "Capacitor_SMD:C_0805_2012Metric" (id 2) (at 208.28 81.788 90)
+    (property "Footprint" "Resistor_SMD:R_0805_2012Metric" (id 2) (at 208.28 81.788 90)
       (effects (font (size 1.27 1.27)) hide)
     )
@@
       (effects (font (size 1.27 1.27)) (justify left))
     )
-    (property "Footprint" "Capacitor_SMD:C_0805_2012Metric" (id 2) (at 198.247 85.09 90)
+    (property "Footprint" "Resistor_SMD:R_0805_2012Metric" (id 2) (at 198.247 85.09 90)
       (effects (font (size 1.27 1.27)) hide)
     )
@@
       (effects (font (size 1.27 1.27)) (justify left))
     )
-    (property "Footprint" "Capacitor_SMD:C_0805_2012Metric" (id 2) (at 208.28 51.308 90)
-      (effects (font (size 1.27 1.27)) hide)
-    )
+    (property "Footprint" "Resistor_SMD:R_0805_2012Metric" (id 2) (at 208.28 51.308 90)
+      (effects (font (size 1.27 1.27)) hide)
+    )

Commit message: SpectDrone Development
Connections:
- net -I_{const}=1.5mA: now also SW3.6 (C)
- no-connect marks 6 -> 5
Other:
- note added: "* In order for 1.5mA to work, 0.4mA must have source also."
- note added: "<-- Current"
- note added: "Current -->"
Changed lines of the file:
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@@
   (no_connect (at 157.48 54.61))
   (no_connect (at 147.32 57.15))
-  (no_connect (at 110.49 59.69))
   (no_connect (at 157.48 59.69))
   (no_connect (at 157.48 57.15))
@@
     (stroke (width 0) (type default) (color 0 0 0 0))
   )
+  (wire (pts (xy 109.22 59.69) (xy 110.49 59.69))
+    (stroke (width 0) (type default) (color 0 0 0 0))
+  )
   (polyline (pts (xy 31.75 85.725) (xy 90.805 85.725))
     (stroke (width 0) (type default) (color 0 0 0 0))
@@
     (effects (font (size 1.27 1.27)) (justify left bottom))
   )
+  (text "Current -->" (at 168.91 67.945 0)
+    (effects (font (size 1.27 1.27)) (justify left bottom))
+  )
   (text "↓ I_{C}=400.0uA" (at 72.39 88.9 0)
     (effects (font (size 1.27 1.27)) (justify left bottom))
@@
     (effects (font (size 1.27 1.27)) (justify left bottom))
   )
+  (text "<-- Current" (at 130.175 55.245 0)
+    (effects (font (size 1.27 1.27)) (justify left bottom))
+  )
   (text "↓ I_{C}=400.0uA" (at 73.025 43.18 0)
     (effects (font (size 1.27 1.27)) (justify left bottom))
+  )
+  (text "* In order for 1.5mA to work,\n0.4mA must have source also."
+    (at 92.71 70.485 0)
+    (effects (font (size 1.27 1.27) italic) (justify left bottom))
   )
   (text "↓ I_{out}=1500.0uA" (at 73.025 123.825 0)
@@
       (effects (font (size 1.27 1.27)) (justify right) hide)
     )
+  )
+  (global_label "-I_{const}=1.5mA" (shape input) (at 109.22 59.69 180) (fields_autoplaced)
+    (effects (font (size 1.27 1.27)) (justify right))
+    (property "Intersheet References" "${INTERSHEET_REFS}" (id 0) (at 93.1393 59.7694 0)
+      (effects (font (size 1.27 1.27)) (justify right) hide)
+    )

Commit message: SpectDrone Development
Parts:
- CS1, CS6: footprint Capacitor_SMD:C_0805_2012Metric -> Capacitor_SMD:C_0603_1608Metric; Part Number (none) -> 06035J100FBTTR
- CS2, CS3, CS7, CS8: footprint Capacitor_SMD:C_0805_2012Metric -> Capacitor_SMD:C_0402_1005Metric; Part Number (none) -> 04023J1R1PBSTR
Changed lines of the file:
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@@
       (effects (font (size 1.27 1.27)) (justify left))
     )
-    (property "Footprint" "Capacitor_SMD:C_0805_2012Metric" (id 2) (at 217.17 44.45 0)
+    (property "Footprint" "Capacitor_SMD:C_0402_1005Metric" (id 2) (at 217.17 44.45 0)
       (effects (font (size 1.27 1.27)) hide)
     )
     (property "Datasheet" "~" (id 3) (at 217.17 44.45 0)
+      (effects (font (size 1.27 1.27)) hide)
+    )
+    (property "Part Number" "04023J1R1PBSTR" (id 4) (at 217.17 44.45 0)
       (effects (font (size 1.27 1.27)) hide)
     )
@@
       (effects (font (size 1.27 1.27)) (justify left))
     )
-    (property "Footprint" "Capacitor_SMD:C_0805_2012Metric" (id 2) (at 214.63 54.61 0)
+    (property "Footprint" "Capacitor_SMD:C_0603_1608Metric" (id 2) (at 214.63 54.61 0)
       (effects (font (size 1.27 1.27)) hide)
     )
     (property "Datasheet" "~" (id 3) (at 214.63 54.61 0)
+      (effects (font (size 1.27 1.27)) hide)
+    )
+    (property "Part Number" "06035J100FBTTR" (id 4) (at 214.63 54.61 0)
       (effects (font (size 1.27 1.27)) hide)
     )
@@
       (effects (font (size 1.27 1.27)) (justify left))
     )
-    (property "Footprint" "Capacitor_SMD:C_0805_2012Metric" (id 2) (at 214.63 85.09 0)
+    (property "Footprint" "Capacitor_SMD:C_0603_1608Metric" (id 2) (at 214.63 85.09 0)
       (effects (font (size 1.27 1.27)) hide)
     )
     (property "Datasheet" "~" (id 3) (at 214.63 85.09 0)
+      (effects (font (size 1.27 1.27)) hide)
+    )
+    (property "Part Number" "06035J100FBTTR" (id 4) (at 214.63 85.09 0)
       (effects (font (size 1.27 1.27)) hide)
     )
@@
       (effects (font (size 1.27 1.27)) (justify left))
     )
-    (property "Footprint" "Capacitor_SMD:C_0805_2012Metric" (id 2) (at 214.63 95.25 0)
+    (property "Footprint" "Capacitor_SMD:C_0402_1005Metric" (id 2) (at 214.63 95.25 0)
       (effects (font (size 1.27 1.27)) hide)
     )
@@
       (effects (font (size 1.27 1.27)) hide)
     )
+    (property "Part Number" "04023J1R1PBSTR" (id 4) (at 214.63 95.25 0)
+      (effects (font (size 1.27 1.27)) hide)
+    )
     (pin "1")
     (pin "2")
@@
       (effects (font (size 1.27 1.27)) (justify left))
     )
-    (property "Footprint" "Capacitor_SMD:C_0805_2012Metric" (id 2) (at 214.63 64.77 0)
+    (property "Footprint" "Capacitor_SMD:C_0402_1005Metric" (id 2) (at 214.63 64.77 0)
       (effects (font (size 1.27 1.27)) hide)
     )
@@
       (effects (font (size 1.27 1.27)) hide)
     )
+    (property "Part Number" "04023J1R1PBSTR" (id 4) (at 214.63 64.77 0)
+      (effects (font (size 1.27 1.27)) hide)
+    )
     (pin "1")
     (pin "2")
@@
       (effects (font (size 1.27 1.27)) (justify left))
     )
-    (property "Footprint" "Capacitor_SMD:C_0805_2012Metric" (id 2) (at 217.17 74.93 0)
+    (property "Footprint" "Capacitor_SMD:C_0402_1005Metric" (id 2) (at 217.17 74.93 0)
       (effects (font (size 1.27 1.27)) hide)
     )
@@
       (effects (font (size 1.27 1.27)) hide)
     )
+    (property "Part Number" "04023J1R1PBSTR" (id 4) (at 217.17 74.93 0)
+      (effects (font (size 1.27 1.27)) hide)
+    )
