File: TestComponents/InsturmentationsAmps.kicad_sch (KiCad schematic)
At the start: 41 parts, among them SW2 SW_DP3T, SW3 SW_DP3T, U3 REF200AU, U4 MCP6L01x-xLT

Commit message: SpectDrone Development
Parts:
- added D1: D_Small, Diode_SMD:D_0805_2012Metric, symbol Device:D_Small
- added JP1: SolderJumper_2_Bridged, Jumper:SolderJumper-2_P1.3mm_Bridged_RoundedPad1.0x1.5mm, symbol Jumper:SolderJumper_2_Bridged
- added JP16: SolderJumper_3_Bridged12, Gardenuino Custom:SolderJumper-4_P1.3mm_Bridged2Bar12_RoundedPad, symbol Jumper:SolderJumper_3_Bridged12
- added R10: X, Resistor_SMD:R_0603_1608Metric, symbol Device:R
- added R4: 250, Resistor_SMD:R_0805_2012Metric, symbol Device:R
- added R5: 91, Resistor_SMD:R_0805_2012Metric, symbol Device:R
- added R9: 470K, Resistor_SMD:R_0805_2012Metric, symbol Device:R
- added RV1: 10K, Potentiometer_THT:Potentiometer_Bourns_3296P_Horizontal, symbol Device:R_Potentiometer
- added SW1: SW_DPDT, Gardenuino Custom:SW_DPDT_CK_JS202011JAQN, symbol Switch:SW_DPDT_x2
- added SW4: SW_DP3T, Gardenuino Custom:SW_DP3T_CK_JS203011JAQN, symbol Switch:SW_DP3T
- added TPGND-1, TPV1, TPV3, TPV5: TestPoint, TestPoint:TestPoint_Keystone_5000-5004_Miniature, symbol Connector:TestPoint
- added U13: X, Package_TO_SOT_SMD:SOT-23, symbol Gardenuino_Custom:ADR510
- added U8: ADR5041B, Package_TO_SOT_SMD:SOT-23, symbol Gardenuino_Custom:ADR510
- added U9: ADR5044B, Package_TO_SOT_SMD:SOT-23, symbol Gardenuino_Custom:ADR510
Connections:
- net -I_{const}=0.4mA: now also SW4.3; no longer U3.4, U3.7
- net GND1: now also RV1.3, TPGND-1.1, U8.2 (A), U9.2 (A)
- net PD(V)_{BIAS}: now also JP16.1 (A), SW1.2 (B)
- net V_{AREF}: now also JP16.2 (C), TPV5.1
- net I_{C}out: now reaches CS11.2, R1.1, U3.3, U4.4 (-)
- net I_{C}out: now also SW4.6
- net I_{C}in: now reaches U3.1, U3.5
- net I_{C}in: now also SW4.5, SW4.8; no longer U3.2
- new net: JP1.1 (A), R9.1, U8.3 (REF)
- new net: R9.2, RV1.2
- new net 2V5: JP1.2 (B), R4.2, RV1.1, SW1.3 (C), TPV1.1, U8.1 (K)
- new net 4V0: JP16.4, R5.2, SW1.1 (A), TPV3.1, U9.1 (K), U9.3 (REF)
- new net 5V0: JP16.3 (B), R10.1, U13.1 (K), U13.3 (REF)
- new net 5V3: R10.2, R4.1, R5.1
- new net GND_{RF}: U13.2 (A)
- new net I_{C}1: D1.1 (K), SW4.1, U3.7
- new net I_{C}1out: SW4.7, U3.2
- new net I_{Mirror}_{IN}: D1.2 (A), SW4.2, SW4.4, U3.4
- no-connect marks 7 -> 10
Other:
- note added: "2.500V +/- 2.5mV"
- note added: "4.096V +/- 4.1mV"
- note added: "5.000V +/- 5.0mV"
- note added: "ADR5045B"
- note added: "R_{BIAS}"
- note added: "SW4A/B Position 1: 0.200mA and 0.750mA Position 2: 0.300mA and 1.125mA Position 3: 0.400mA and 1.500mA"
- moved on the sheet: U3A, U3B

Commit message: SpectDrone Development
Parts:
- R_{PD.bias}1, R_{PD.bias}2: value 0 -> 1K; Part Number ERJ-6GEY0R00V -> (none)
Connections:
- net I_{C}1: now also SW4.4; no longer SW4.1
- net I_{Mirror}_{IN}: now also SW4.1; no longer SW4.4
Other:
- note added: "Config 1: SW1-PD_{V}-2.500V SW2-PD1_{TEST} SW3-1.500mA SW4-1.00x ==> I_{C}out=401.04mA ==> 1.5039mA ==> V_{DROP}=1.504V ==> PD1_{TEST} = 0.996V ==> Ratio = 39.85% Config 2: SW1-PD_{V}-2.500V SW2-PD1_{TEST} SW3-1.500mA SW4-0.75x ==> I_{C}out=300.78mA ==> 1.1279mA ==> V_{DROP}=1.128V ==> PD1_{TEST} = 1.372V ==> Ratio = 54.88% Config 3: SW1-PD_{V}-2.500V SW2-PD1_{TEST} SW3-1.500mA SW4-0.50x ==> I_{C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"
- note added: "R = 666.6 ohm | V_{in} | I_{C} | PD_{V} | Gain | PD_{OUT} | Ratio | Digital_{1024} | Digital_{4096} | Digital_{262K} | Digital_{16M} | --------------------------------------------------------------------------------------------------------------------- | 3.000 | 0.400 | 2.730 | 1.00 | 2.730 | 0.910 | 932 | 3727 | 238551 | 15267267 | | 3.000 | 1.500 | 2.000 | 1.00 | 2.000 | 0.666 | 683 | 2728 | 17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"
- note added: "SW4A/B Position 1: 0.400mA and 1.500mA Position 2: 0.300mA and 1.125mA Position 3: 0.200mA and 0.750mA"
- note added: "V = IR V = PD(V)_{BIAS} = [ 2.5 V | 4.096 V ] I = I_{C} = [ 0.4 mA | 1.5 mA ] PD(V)_{BIAS} = I_{C} * R R = PD(V)_{BIAS} / I_{C} "Dark" current for 2.5 V = ~ 10.9 pA "Dark" current for 4.096 V = ~ 11.2 pA Effective Resistance of Photodiode R = 2.5 V / 10.9 pA = 0.229 Tohm ~= 1 Gohm R = 4.096 V / 11.2 pA = 0.366 Tohm ~= 1 Gohm If R = 1 Gohm: I(2.5 V) = 2.5 nA I(4.096 V) = 4.096 nA "Mid-zenith" curr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"
- note added: "V_{S} = 5 v V_{out} = 2.5 v V = 5 v - 2.5 v = 2.5 v R_{BIAS}(I_{L_min (1PD)}) = 2.5 v / 1.3 mA = 1923 ohm R_{BIAS}(I_{L_min (2PD)}) = 2.5 v / 2.5 mA = 1000 ohm R_{BIAS}(I_{L_max}) = 2.5 v / 10.0 mA = 250 ohm R_{BIAS} = 250 ohm L = 2.5 V / 250 ohm = 10.00 mA R4 = 250 ohm"
- note added: "V_{S} = 5 v V_{out} = 4.096 v V = 5 v - 4.096 v = .904 v R_{BIAS}(I_{L_min (1PD)}) = 0.904 v / 1.3 mA = 769 ohm R_{BIAS}(I_{L_min (2PD)}) = 0.904 v / 2.5 mA = 400 ohm R_{BIAS}(I_{L_max}) = 0.904 v / 10.0 mA = 90.4 ohm R_{BIAS} = 91 ohm L = 0.904 V / 0.091 Kohm = 9.93 mA R5 = 91 ohm"
- note removed: "I=0.4mA V=IR=0.4mA*0.25kohm=0.10V I=1.5mA V=IR=1.5mA*0.25kohm=0.375V I=0.4mA V=IR=1.5mA*66.7ohm=0.10V I=0.4mA V=IR=0.4mA*0.5kohm=0.20V I=1.5mA V=IR=1.5mA*0.5kohm=0.75V"
- note removed: "I=0.4mA V=IR=0.4mA*1.0kohm=0.4V I=1.5mA V=IR=1.5mA*1.0kohm=1.5V"
- note removed: "R = 666.6 ohm | V_{in} | I_{C} | PD_{V} | Gain | PD_{OUT} | Ratio | Digital_{1024} | Digital_{4096} | Digital_{262K} | Digital_{16M} | ------------------------------------------------------------------------------ | 3.000 | 0.400 | 2.730 | 1.00 | 2.730 | 0.910 | 932 | 3727 | 238551 | 15267267 | | 3.000 | 1.500 | 2.000 | 1.00 | 2.000 | 0.666 | 683 | 2728 | 174588 | 11173626 | | 1.000 | 0.400 | 0.7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"
- note removed: "SW4A/B Position 1: 0.200mA and 0.750mA Position 2: 0.300mA and 1.125mA Position 3: 0.400mA and 1.500mA"
- note removed: "V = IR V = PD(V)_{BIAS} = [ 2.5 V | 4.096 V ] I = I_{C} = [ 0.4 mA | 1.5 mA ] PD(V)_{BIAS} = I_{C} * R R = PD(V)_{BIAS} / I_{C} "Dark" current for 2.5 V = ~ 10.9 pA "Dark" current for 4.096 V = ~ 11.2 pA R = 2.5 V / 10.9 pA = 0.229 Tohm ~= 1 Gohm R = 4.096 V / 11.2 pA = 0.366 Tohm ~= 1 Gohm If R = 1 Gohm: I(2.5 V) = 2.5 nA I(4.096 V) = 4.096 nA "Mid-zenith" current = 400 uA R = 2.5 V / 0.4 mA = 6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"
- moved on the sheet: CS1, CS10, CS11, CS12, CS13, CS2, CS3, CS4, CS5, CS6, CS7, CS8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

Commit message: SpectDrone Development
Parts:
- RS2, RS5: footprint Capacitor_SMD:C_0805_2012Metric -> Resistor_SMD:R_0805_2012Metric
Other:
- note added: "SIM-PASS"
Changed lines of the file:
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@@
     (effects (font (size 1.27 1.27)) (justify left bottom))
+  )
+  (text "SIM-PASS" (at 184.15 160.655 0)
+    (effects (font (size 1.27 1.27) (color 255 0 0 1)) (justify left bottom))
   )
   (label "I_{C}in" (at 50.8 89.535 90) (fields_autoplaced)
@@
       (effects (font (size 1.27 1.27)) hide)
     )
+    (property "Sim.Device" "XSPICE" (at 257.175 112.395 0)
+      (effects (font (size 1.27 1.27)) hide)
+    )
     (pin "1")
     (pin "2")
@@
       (effects (font (size 1.27 1.27)) (justify left))
     )
-    (property "Footprint" "Capacitor_SMD:C_0805_2012Metric" (at 240.792 112.395 90)
+    (property "Footprint" "Resistor_SMD:R_0805_2012Metric" (at 240.792 112.395 90)
       (effects (font (size 1.27 1.27)) hide)
     )
@@
       (effects (font (size 1.27 1.27)) (justify left))
     )
-    (property "Footprint" "Capacitor_SMD:C_0805_2012Metric" (at 240.792 142.875 90)
-      (effects (font (size 1.27 1.27)) hide)
-    )
+    (property "Footprint" "Resistor_SMD:R_0805_2012Metric" (at 240.792 142.875 90)
+      (effects (font (size 1.27 1.27)) hide)
+    )

Commit message: SpectDrone Development
Parts:
- added JBAT2: Conn_01x02_Female, Connector_PinHeader_2.54mm:PinHeader_1x02_P2.54mm_Vertical, symbol Connector:Conn_01x02_Female
- R10: value X -> 24R9
- U13: value X -> ADR5045B; Part Number (none) -> ADR5045B
Connections:
- net 4V0: now also JP16.3 (B); no longer JP16.4
- net 5V0: now also CS10.2, CS4.1, CS5.2, CS9.1, JP16.4, US1.8 (Vs+), US2.8 (Vs+), JBAT2.1 (Pin_1); no longer JP16.3 (B)
- net GND1: now also JBAT2.2 (Pin_2)
- net V_{AREF}: no longer CS10.2, CS4.1, CS5.2, CS9.1, US1.8 (Vs+), US2.8 (Vs+)

Commit message: SpectDrone Development
Parts:
- removed JBAT2: Conn_01x02_Female, Connector_PinHeader_2.54mm:PinHeader_1x02_P2.54mm_Vertical, symbol Connector:Conn_01x02_Female
Changed lines of the file:
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@@
-    )
-  )
-  (global_label "5V0" (shape input) (at 199.39 52.07 0) (fields_autoplaced)
-    (effects (font (size 1.27 1.27)) (justify left))
-    (property "Intersheetrefs" "${INTERSHEET_REFS}" (at 205.8828 52.07 0)
-      (effects (font (size 1.27 1.27)) (justify left) hide)
-    )
-  )
-  (global_label "GND1" (shape input) (at 196.85 52.07 180) (fields_autoplaced)
-    (effects (font (size 1.27 1.27)) (justify right))
-    (property "Intersheetrefs" "${INTERSHEET_REFS}" (at 189.3569 51.9906 0)
-      (effects (font (size 1.27 1.27)) (justify right) hide)
     )
   )
@@
         )
       )
-    )
-  )
-  (symbol (lib_id "Connector:Conn_01x02_Female") (at 199.39 57.15 270) (unit 1)
-    (in_bom no) (on_board yes) (dnp no)
-    (property "Reference" "JBAT2" (at 200.025 55.245 90)
-      (effects (font (size 1.27 1.27)) (justify left))
-    )
-    (property "Value" "Conn_01x02_Female" (at 196.8501 58.42 0)
-      (effects (font (size 1.27 1.27)) (justify left) hide)
-    )
-    (property "Footprint" "Connector_PinHeader_2.54mm:PinHeader_1x02_P2.54mm_Vertical" (at 199.39 57.15 0)
-      (effects (font (size 1.27 1.27)) hide)
-    )
-    (property "Datasheet" "~" (at 199.39 57.15 0)
-      (effects (font (size 1.27 1.27)) hide)
-    )
-    (pin "1")
-    (pin "2")
-    (instances
-      (project "TestComponents"
-        (path "/e63e39d7-6ac0-4ffd-8aa3-1841a4541b55"
-          (reference "JBAT2") (unit 1)
-        )
-        (path "/e63e39d7-6ac0-4ffd-8aa3-1841a4541b55/fcc3e372-6be4-4e20-89ea-15d74da3ea1f"
-          (reference "JBAT1") (unit 1)
-        )
-      )
