File: TestComponents/TestComponents.kicad_sch (KiCad schematic)
At the start: 9 parts, among them J5 RFShield_OnePiece, U1 AD7991

Commit message: SpectDrone Development
Parts:
- added C38: 2.5pF, Capacitor_SMD:C_0805_2012Metric, symbol Device:C_Small
- added C39: 10uF, Capacitor_SMD:C_0805_2012Metric, symbol Device:C_Polarized_Small_US
- added C40: 0.1uF, Capacitor_SMD:C_0603_1608Metric, symbol Device:C_Polarized_Small_US
- added J6: RFShield_OnePiece, RF_Shielding:Laird_Technologies_BMI-S-101_13.66x12.70mm, symbol Device:RFShield_OnePiece
- added JP12: SolderJumper_2_Bridged, Jumper:SolderJumper-2_P1.3mm_Bridged2Bar_RoundedPad1.0x1.5mm, symbol Jumper:SolderJumper_2_Bridged
- added R34: 2K, Capacitor_SMD:C_0805_2012Metric, symbol Device:R
Connections:
- net GND1: now also C38.2, JP12.1 (A), R34.2
- net GND_{RF}: now also C38.1, C39.2, C40.2, J6.1 (Shield), JP12.2 (B), R34.1
- net V_{RF}: now also C39.1, C40.1
Other:
- moved on the sheet: C15, JP11, R13

Commit message: SpectDrone Development
Parts:
- added C3, C4: 100nF, Capacitor_SMD:C_0805_2012Metric, symbol Device:C_Small
- added J3V1: Conn_01x01_Male, symbol Connector:Conn_01x01_Male
- added R3, R6: 10K, symbol Device:R
- added U2: ADS1219, Package_SO:TSSOP-16_4.4x5mm_P0.65mm, symbol ads1219:ADS1219
Connections:
- net GND1: now also C3.1, R6.2, U2.1 (A0), U2.2 (A1), U2.5 (AGND)
- net GND_{RF}: now also C4.1, U2.4 (DGND), U2.8 (REFN)
- net P1_{RF}: now also U2.6 (AIN3)
- net P2_{RF}: now also U2.10 (AIN1)
- net S1_{RF}: now also U2.7 (AIN2)
- net S2_{RF}: now also U2.11 (AIN0)
- net SCL_{RF}: now also U2.16 (SCL)
- net SDA_{RF}: now also U2.15 (SDA)
- net V_{RF}: now also C4.2, U2.13 (DVDD), U2.9 (REFP)
- new net: R3.1, U2.14 (~{DRDY})
- new net: R6.1, U2.3 (~{RESET})
- new net 3V1: C3.2, J3V1.1 (Pin_1), R3.2, U2.12 (AVDD)
Other:
- moved on the sheet: C1, C13, C14, C15, C2, C38, C39, C40, JP11, JP12, R13, R34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

Commit message: SpectDrone Development
Parts:
- removed C39: 10uF, Capacitor_SMD:C_0805_2012Metric, symbol Device:C_Polarized_Small_US
- removed C4: 100nF, Capacitor_SMD:C_0805_2012Metric, symbol Device:C_Small
- removed C40: 0.1uF, Capacitor_SMD:C_0603_1608Metric, symbol Device:C_Polarized_Small_US
- removed R3: 10K, symbol Device:R
- R13, R34: footprint Capacitor_SMD:C_0805_2012Metric -> Resistor_SMD:R_0805_2012Metric
- R6: footprint (none) -> Resistor_SMD:R_0805_2012Metric
- U2: symbol ads1219:ADS1219 -> ADS1219:ADS1219
Connections:
- net 3V1: now also R6.2, U2.13 (DVDD); no longer U2.12 (AVDD)
- net GND1: now also U2.4 (DGND); no longer R6.2, U2.5 (AGND)
- net GND_{RF}: now also U2.5 (AGND); no longer U2.4 (DGND)
- net P1_{RF}: no longer U2.6 (AIN3)
- net P2_{RF}: no longer U2.10 (AIN1)
- net S1_{RF}: no longer U2.7 (AIN2)
- net S2_{RF}: no longer U2.11 (AIN0)
- net V_{RF}: now also U2.12 (AVDD); no longer U2.13 (DVDD)
- net at U2.14 (~{DRDY}): now also R6.1, U2.3 (~{RESET})
- new net P1_{RF}-2: U2.6 (AIN3)
- new net P2_{RF}-2: U2.10 (AIN1)
- new net S1_{RF}-2: U2.7 (AIN2)
- new net S2_{RF}-2: U2.11 (AIN0)
Other:
- note removed: "U12"
- moved on the sheet: C15, C3, C38, J5, JP11, JP12, R34, R6, U2

Commit message: SpectDrone Development
Parts:
- added JVIN1: Conn_01x01_Male, Connector_PinHeader_2.54mm:PinHeader_1x01_P2.54mm_Vertical, symbol Connector:Conn_01x01_Male
- J3V1: footprint (none) -> Connector_PinHeader_2.54mm:PinHeader_1x01_P2.54mm_Vertical
Connections:
- new net VIN: JVIN1.1 (Pin_1)
Other:
- moved on the sheet: C3, J6
Changed lines of the file:
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@@
+    (stroke (width 0) (type default) (color 0 0 0 0))
+  )
+  (wire (pts (xy 137.16 114.3) (xy 131.445 114.3))
     (stroke (width 0) (type default) (color 0 0 0 0))
   )
@@
     (stroke (width 0) (type default) (color 0 0 0 0))
   )
-  (wire (pts (xy 36.83 35.56) (xy 41.91 35.56))
+  (wire (pts (xy 36.83 35.56) (xy 41.275 35.56))
     (stroke (width 0) (type default) (color 0 0 0 0))
   )
@@
     (effects (font (size 1.27 1.27)) (justify left bottom))
   )
-  (label "GND1" (at 54.61 66.04 0)
+  (label "GND1" (at 55.88 63.5 0)
     (effects (font (size 1.27 1.27)) (justify left bottom))
   )
@@
     (effects (font (size 1.27 1.27)) (justify left bottom))
   )
+  (label "GND1" (at 67.945 78.105 0)
+    (effects (font (size 1.27 1.27)) (justify left bottom))
+  )
   (label "GND_{RF}" (at 38.1 40.64 0)
     (effects (font (size 1.27 1.27)) (justify left bottom))
@@
     (effects (font (size 1.27 1.27)) (justify right bottom))
   )
-  (label "3V1" (at 49.53 66.04 180)
+  (label "3V1" (at 50.8 63.5 180)
     (effects (font (size 1.27 1.27)) (justify right bottom))
   )
@@
   )
   (label "S2_{RF}" (at 207.01 96.52 180)
+    (effects (font (size 1.27 1.27)) (justify right bottom))
+  )
+  (label "VIN1" (at 136.525 114.3 180)
     (effects (font (size 1.27 1.27)) (justify right bottom))
   )
@@
     )
   )
+  (global_label "GND1" (shape input) (at 67.945 78.105 180) (fields_autoplaced)
+    (effects (font (size 1.27 1.27)) (justify right))
+    (property "Intersheet References" "${INTERSHEET_REFS}" (id 0) (at 60.4519 78.0256 0)
+      (effects (font (size 1.27 1.27)) (justify right) hide)
+    )
+  )
   (global_label "P2" (shape input) (at 196.215 105.41 180) (fields_autoplaced)
     (effects (font (size 1.27 1.27)) (justify right))
@@
     )
   )
+  (global_label "VIN" (shape input) (at 137.16 114.3 0) (fields_autoplaced)
+    (effects (font (size 1.27 1.27)) (justify left))
+    (property "Intersheet References" "${INTERSHEET_REFS}" (id 0) (at 142.5969 114.2206 0)
+      (effects (font (size 1.27 1.27)) (justify left) hide)
+    )
+  )
   (global_label "5V3" (shape input) (at 196.215 87.63 180) (fields_autoplaced)
     (effects (font (size 1.27 1.27)) (justify right))
@@
     )
   )
-  (symbol (lib_id "Device:C_Small") (at 52.07 66.04 270) (mirror x) (unit 1)
-    (in_bom yes) (on_board yes)
-    (property "Reference" "C3" (id 0) (at 50.8 67.31 90)
+  (symbol (lib_id "Device:C_Small") (at 53.34 63.5 270) (mirror x) (unit 1)
+    (in_bom yes) (on_board yes)
+    (property "Reference" "C3" (id 0) (at 52.07 64.77 90)
       (effects (font (size 1.27 1.27)) (justify right))
     )
-    (property "Value" "100nF" (id 1) (at 53.34 67.31 90)
+    (property "Value" "100nF" (id 1) (at 54.61 64.77 90)
       (effects (font (size 1.27 1.27)) (justify left))
     )
-    (property "Footprint" "Capacitor_SMD:C_0805_2012Metric" (id 2) (at 52.07 66.04 0)
-      (effects (font (size 1.27 1.27)) hide)
-    )
-    (property "Datasheet" "~" (id 3) (at 52.07 66.04 0)
-      (effects (font (size 1.27 1.27)) hide)
-    )
-    (pin "1")
-    (pin "2")
-  )
-  (symbol (lib_name "RFShield_OnePiece_2") (lib_id "Device:RFShield_OnePiece") (at 52.07 35.56 270)
-    (in_bom yes) (on_board yes)
-    (property "Reference" "J6" (id 0) (at 45.085 21.59 90)
+    (property "Footprint" "Capacitor_SMD:C_0805_2012Metric" (id 2) (at 53.34 63.5 0)
+      (effects (font (size 1.27 1.27)) hide)
+    )
+    (property "Datasheet" "~" (id 3) (at 53.34 63.5 0)
+      (effects (font (size 1.27 1.27)) hide)
+    )
+    (pin "1")
+    (pin "2")
+  )
+  (symbol (lib_name "RFShield_OnePiece_2") (lib_id "Device:RFShield_OnePiece") (at 51.435 35.56 270) (unit 1)
+    (in_bom yes) (on_board yes)
+    (property "Reference" "J6" (id 0) (at 44.45 21.59 90)
       (effects (font (size 1.27 1.27)) (justify left))
     )
-    (property "Value" "RFShield_OnePiece" (id 1) (at 49.53 21.59 90)
+    (property "Value" "RFShield_OnePiece" (id 1) (at 48.895 21.59 90)
       (effects (font (size 1.27 1.27)) (justify left))
     )
-    (property "Footprint" "RF_Shielding:Laird_Technologies_BMI-S-101_13.66x12.70mm" (id 2) (at 52.07 38.1 0)
-      (effects (font (size 1.27 1.27)) hide)
-    )
-    (property "Datasheet" "~" (id 3) (at 52.07 38.1 0)
+    (property "Footprint" "RF_Shielding:Laird_Technologies_BMI-S-101_13.66x12.70mm" (id 2) (at 51.435 38.1 0)
+      (effects (font (size 1.27 1.27)) hide)
+    )
+    (property "Datasheet" "~" (id 3) (at 51.435 38.1 0)
       (effects (font (size 1.27 1.27)) hide)
     )
@@
     (property "Reference" "J3V1" (id 0) (at 127 100.33 0))
     (property "Value" "Conn_01x01_Male" (id 1) (at 127 102.87 0))
-    (property "Footprint" "" (id 2) (at 126.365 106.045 0)
+    (property "Footprint" "Connector_PinHeader_2.54mm:PinHeader_1x01_P2.54mm_Vertical" (id 2) (at 126.365 106.045 0)
       (effects (font (size 1.27 1.27)) hide)
     )
@@
     (pin "1")
   )
+  (symbol (lib_id "Connector:Conn_01x01_Male") (at 126.365 114.3 0) (unit 1)
+    (in_bom yes) (on_board yes) (fields_autoplaced)
+    (property "Reference" "JVIN1" (id 0) (at 127 109.22 0))
+    (property "Value" "Conn_01x01_Male" (id 1) (at 127 111.76 0))
+    (property "Footprint" "Connector_PinHeader_2.54mm:PinHeader_1x01_P2.54mm_Vertical" (id 2) (at 126.365 114.3 0)
+      (effects (font (size 1.27 1.27)) hide)
+    )
+    (property "Datasheet" "~" (id 3) (at 126.365 114.3 0)
+      (effects (font (size 1.27 1.27)) hide)
+    )
+    (pin "1")
+  )
   (symbol (lib_id "Device:R") (at 110.49 30.48 270) (unit 1)
     (in_bom yes) (on_board yes)
@@
     )
     (path "/21f0c995-97eb-43ed-8e0f-a133d3e4b10f"
-      (reference "J3V1") (unit 1) (value "Conn_01x01_Male") (footprint "")
+      (reference "J3V1") (unit 1) (value "Conn_01x01_Male") (footprint "Connector_PinHeader_2.54mm:PinHeader_1x01_P2.54mm_Vertical")
     )
     (path "/f1a9fb80-4cc4-410f-9616-e19c969dcab5"
@@
       (reference "JUT1") (unit 1) (value "Conn_01x04_Male") (footprint "Connector_PinHeader_2.54mm:PinHeader_1x04_P2.54mm_Vertical")
     )
+    (path "/f686aee0-011d-49d4-b9f1-91a248d4901a"
+      (reference "JVIN1") (unit 1) (value "Conn_01x01_Male") (footprint "Connector_PinHeader_2.54mm:PinHeader_1x01_P2.54mm_Vertical")
+    )
     (path "/fcc3e372-6be4-4e20-89ea-15d74da3ea1f/35afb089-9fdf-4674-9ec7-76a0c05da5b2"
       (reference "PD1") (unit 1) (value "S1336-18BK") (footprint "Gardenuino Custom:S1336")
@@
     )
     (path "/b2a165aa-ab09-4352-b1f3-7ca3517b67aa/38fab12b-3a44-45bc-898e-d40ab088c5ca"
-      (reference "R5") (unit 1) (value "174") (footprint "Capacitor_SMD:C_0805_2012Metric")
+      (reference "R5") (unit 1) (value "200") (footprint "Capacitor_SMD:C_0805_2012Metric")
     )
     (path "/e4add989-3502-4243-878f-d4babef5c9f6"
@@
     )
     (path "/fcc3e372-6be4-4e20-89ea-15d74da3ea1f/1bef5b1c-5aba-4e23-8748-ea44cb5e23bb"
-      (reference "R_{PD}1") (unit 1) (value "X") (footprint "Capacitor_SMD:C_0805_2012Metric")
+      (reference "R_{PD}1") (unit 1) (value "2K") (footprint "Capacitor_SMD:C_0805_2012Metric")
     )
     (path "/fcc3e372-6be4-4e20-89ea-15d74da3ea1f/941744c3-43df-4c8c-89c7-828cc479a95d"
-      (reference "R_{PD}2") (unit 1) (value "X") (footprint "Capacitor_SMD:C_0805_2012Metric")
+      (reference "R_{PD}2") (unit 1) (value "2K") (footprint "Capacitor_SMD:C_0805_2012Metric")
     )
     (path "/b2a165aa-ab09-4352-b1f3-7ca3517b67aa/11a85d83-ca23-4a66-9a7a-3b010acc3da7"
@@
       (reference "SW2") (unit 1) (value "SW_SP3T") (footprint "Button_Switch_SMD:SW_SP3T_PCM13")
     )
-    (path "/fcc3e372-6be4-4e20-89ea-15d74da3ea1f/00383856-7ba1-45d0-a65d-5461545f05b2"
-      (reference "SW3") (unit 1) (value "SW_DPDT_x2") (footprint "Button_Switch_THT:SW_CuK_JS202011AQN_DPDT_Angled")
-    )
-    (path "/fcc3e372-6be4-4e20-89ea-15d74da3ea1f/2453cafe-798d-494d-9534-38604e842a32"
-      (reference "SW3") (unit 2) (value "SW_DPDT_x2") (footprint "")
+    (path "/fcc3e372-6be4-4e20-89ea-15d74da3ea1f/1175f0f4-71a1-40e9-8071-75f5dbc0b5f1"
+      (reference "SW3") (unit 1) (value "SW_SP3T") (footprint "Button_Switch_SMD:SW_SP3T_PCM13")
     )
     (path "/b2a165aa-ab09-4352-b1f3-7ca3517b67aa/50a66564-4ba6-42ac-a9d9-7efe41dfbb5a"

Commit message: SpectDrone Development
Parts:
- J3V1, JVIN1: footprint Connector_PinHeader_2.54mm:PinHeader_1x01_P2.54mm_Vertical -> Connector_PinSocket_2.54mm:PinSocket_1x01_P2.54mm_Vertical
Changed lines of the file:
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@@
     (property "Reference" "J3V1" (id 0) (at 127 100.33 0))
     (property "Value" "Conn_01x01_Male" (id 1) (at 127 102.87 0))
-    (property "Footprint" "Connector_PinHeader_2.54mm:PinHeader_1x01_P2.54mm_Vertical" (id 2) (at 126.365 106.045 0)
+    (property "Footprint" "Connector_PinSocket_2.54mm:PinSocket_1x01_P2.54mm_Vertical" (id 2) (at 126.365 106.045 0)
       (effects (font (size 1.27 1.27)) hide)
     )
@@
     (property "Reference" "JVIN1" (id 0) (at 127 109.22 0))
     (property "Value" "Conn_01x01_Male" (id 1) (at 127 111.76 0))
-    (property "Footprint" "Connector_PinHeader_2.54mm:PinHeader_1x01_P2.54mm_Vertical" (id 2) (at 126.365 114.3 0)
+    (property "Footprint" "Connector_PinSocket_2.54mm:PinSocket_1x01_P2.54mm_Vertical" (id 2) (at 126.365 114.3 0)
       (effects (font (size 1.27 1.27)) hide)
     )
@@
     )
     (path "/6476e233-d260-45fe-84d2-9ade7d0003a0/92cf4db4-2dba-4763-9cd8-3c7f8aff8f24"
-      (reference "J2-1") (unit 1) (value "Conn_01x04_Male") (footprint "Connector_PinHeader_2.54mm:PinHeader_1x04_P2.54mm_Vertical")
+      (reference "J2-1") (unit 1) (value "Conn_01x04_Male") (footprint "Connector_PinSocket_2.54mm:PinSocket_1x04_P2.54mm_Vertical")
     )
     (path "/6476e233-d260-45fe-84d2-9ade7d0003a0/6f75ea3e-6135-44f5-9313-1aad839ab6f6"
-      (reference "J2-2") (unit 1) (value "Conn_01x04_Male") (footprint "Connector_PinHeader_2.54mm:PinHeader_1x04_P2.54mm_Vertical")
+      (reference "J2-2") (unit 1) (value "Conn_01x04_Male") (footprint "Connector_PinSocket_2.54mm:PinSocket_1x04_P2.54mm_Vertical")
     )
     (path "/21f0c995-97eb-43ed-8e0f-a133d3e4b10f"
-      (reference "J3V1") (unit 1) (value "Conn_01x01_Male") (footprint "Connector_PinHeader_2.54mm:PinHeader_1x01_P2.54mm_Vertical")
+      (reference "J3V1") (unit 1) (value "Conn_01x01_Male") (footprint "Connector_PinSocket_2.54mm:PinSocket_1x01_P2.54mm_Vertical")
     )
     (path "/f1a9fb80-4cc4-410f-9616-e19c969dcab5"
@@
     )
     (path "/6476e233-d260-45fe-84d2-9ade7d0003a0/815a0815-7930-45ec-8d6e-dc110f979c75"
-      (reference "JADC1") (unit 1) (value "Conn_01x04_Male") (footprint "Connector_PinHeader_2.54mm:PinHeader_1x04_P2.54mm_Vertical")
+      (reference "JADC1") (unit 1) (value "Conn_01x04_Male") (footprint "Connector_PinSocket_2.54mm:PinSocket_1x04_P2.54mm_Vertical")
     )
     (path "/6476e233-d260-45fe-84d2-9ade7d0003a0/7d4fcb23-c914-48df-941d-94cf5f1f85b5"
-      (reference "JAPC1") (unit 1) (value "Conn_01x04_Male") (footprint "Connector_PinHeader_2.54mm:PinHeader_1x04_P2.54mm_Vertical")
+      (reference "JAPC1") (unit 1) (value "Conn_01x04_Male") (footprint "Connector_PinSocket_2.54mm:PinSocket_1x04_P2.54mm_Vertical")
     )
     (path "/6476e233-d260-45fe-84d2-9ade7d0003a0/95a40d19-41c6-4680-9b37-9cb1bed1a413"
-      (reference "JAUX1") (unit 1) (value "AUX") (footprint "Connector_PinHeader_2.54mm:PinHeader_1x12_P2.54mm_Vertical")
+      (reference "JAUX1") (unit 1) (value "AUX") (footprint "Connector_PinSocket_2.54mm:PinSocket_1x12_P2.54mm_Vertical")
     )
     (path "/6476e233-d260-45fe-84d2-9ade7d0003a0/0df376e0-b3b8-4926-8318-ef70bcc43326"
-      (reference "JD1") (unit 1) (value "Conn_01x04_Male") (footprint "Connector_PinHeader_2.54mm:PinHeader_1x04_P2.54mm_Vertical")
+      (reference "JD1") (unit 1) (value "Conn_01x04_Male") (footprint "Connector_PinSocket_2.54mm:PinSocket_1x04_P2.54mm_Vertical")
     )
     (path "/6476e233-d260-45fe-84d2-9ade7d0003a0/70b53718-ed58-494c-b8a6-19eb974c07c4"
-      (reference "JGPS1") (unit 1) (value "GPS") (footprint "Connector_PinHeader_2.54mm:PinHeader_1x05_P2.54mm_Vertical")
+      (reference "JGPS1") (unit 1) (value "GPS") (footprint "Connector_PinSocket_2.54mm:PinSocket_1x05_P2.54mm_Vertical")
     )
     (path "/6f675e5f-8fe6-4148-baf1-da97afc770f8"
@@
     )
     (path "/6476e233-d260-45fe-84d2-9ade7d0003a0/24cb67fc-f0c9-4f6e-88c1-7636ab854c5e"
-      (reference "JUT1") (unit 1) (value "Conn_01x04_Male") (footprint "Connector_PinHeader_2.54mm:PinHeader_1x04_P2.54mm_Vertical")
+      (reference "JUT1") (unit 1) (value "Conn_01x04_Male") (footprint "Connector_PinSocket_2.54mm:PinSocket_1x04_P2.54mm_Vertical")
     )
     (path "/f686aee0-011d-49d4-b9f1-91a248d4901a"
-      (reference "JVIN1") (unit 1) (value "Conn_01x01_Male") (footprint "Connector_PinHeader_2.54mm:PinHeader_1x01_P2.54mm_Vertical")
+      (reference "JVIN1") (unit 1) (value "Conn_01x01_Male") (footprint "Connector_PinSocket_2.54mm:PinSocket_1x01_P2.54mm_Vertical")
     )
     (path "/fcc3e372-6be4-4e20-89ea-15d74da3ea1f/35afb089-9fdf-4674-9ec7-76a0c05da5b2"
@@
     )
     (path "/b2a165aa-ab09-4352-b1f3-7ca3517b67aa/81975237-87d0-4ccf-948f-3491e3cf30f9"
-      (reference "RV1") (unit 1) (value "10K") (footprint "Potentiometer_THT:Potentiometer_Bourns_3296W_Vertical")
+      (reference "RV1") (unit 1) (value "10K") (footprint "Potentiometer_THT:Potentiometer_Bourns_3296P_Horizontal")
+    )
+    (path "/fcc3e372-6be4-4e20-89ea-15d74da3ea1f/25915a5f-4800-4383-a1d4-70417d5200b6"
+      (reference "R_{C}1") (unit 1) (value "500") (footprint "Capacitor_SMD:C_0805_2012Metric")
     )
     (path "/fcc3e372-6be4-4e20-89ea-15d74da3ea1f/d890e3ce-0d5d-49bd-a448-e1b7e92c15f8"
@@
       (reference "SW1") (unit 1) (value "SW_SPDT") (footprint "Button_Switch_SMD:SW_SPDT_CK-JS102011SAQN")
     )
-    (path "/fcc3e372-6be4-4e20-89ea-15d74da3ea1f/7c9345d3-5ddc-475b-b1b4-0007c3029eac"
-      (reference "SW2") (unit 1) (value "SW_SP3T") (footprint "Button_Switch_SMD:SW_SP3T_PCM13")
-    )
-    (path "/fcc3e372-6be4-4e20-89ea-15d74da3ea1f/1175f0f4-71a1-40e9-8071-75f5dbc0b5f1"
-      (reference "SW3") (unit 1) (value "SW_SP3T") (footprint "Button_Switch_SMD:SW_SP3T_PCM13")
+    (path "/fcc3e372-6be4-4e20-89ea-15d74da3ea1f/2f3c1326-d3aa-454b-a6fd-3e9f6ecf7423"
+      (reference "SW2") (unit 1) (value "SW_DP3T") (footprint "Gardenuino Custom:SW_DP3T_CK_JS203011JAQN")
+    )
+    (path "/fcc3e372-6be4-4e20-89ea-15d74da3ea1f/b6c14fc4-0ee3-4260-a55d-aa7b944a260e"
+      (reference "SW2") (unit 2) (value "SW_DP3T") (footprint "Gardenuino Custom:SW_DP3T_CK_JS203011JAQN")
+    )
+    (path "/fcc3e372-6be4-4e20-89ea-15d74da3ea1f/b9465500-820c-4a81-b13b-d156e8995357"
+      (reference "SW3") (unit 1) (value "SW_DPDT") (footprint "Gardenuino Custom:SW_DPDT_CK_JS202011JAQN")
+    )
+    (path "/fcc3e372-6be4-4e20-89ea-15d74da3ea1f/b37bacae-9217-4ba2-884a-61ed1df647ae"
+      (reference "SW3") (unit 2) (value "SW_DPDT") (footprint "Gardenuino Custom:SW_DPDT_CK_JS202011JAQN")
     )
     (path "/b2a165aa-ab09-4352-b1f3-7ca3517b67aa/50a66564-4ba6-42ac-a9d9-7efe41dfbb5a"
