File: TestComponents/TestComponents.kicad_sch (KiCad schematic)
At the start: 18 parts, among them J3V1 Conn_01x01_Male, J5 RFShield_OnePiece, J6 RFShield_OnePiece, U1 AD7991, U2 ADS1219

Commit message: SpectDrone Development
Parts:
- J3V1, JVIN1: footprint Connector_PinSocket_2.54mm:PinSocket_1x01_P2.54mm_Vertical -> Connector_PinHeader_2.54mm:PinHeader_1x01_P2.54mm_Vertical
Changed lines of the file:
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@@
     (property "Reference" "J3V1" (id 0) (at 127 100.33 0))
     (property "Value" "Conn_01x01_Male" (id 1) (at 127 102.87 0))
-    (property "Footprint" "Connector_PinSocket_2.54mm:PinSocket_1x01_P2.54mm_Vertical" (id 2) (at 126.365 106.045 0)
+    (property "Footprint" "Connector_PinHeader_2.54mm:PinHeader_1x01_P2.54mm_Vertical" (id 2) (at 126.365 106.045 0)
       (effects (font (size 1.27 1.27)) hide)
     )
@@
     (property "Reference" "JVIN1" (id 0) (at 127 109.22 0))
     (property "Value" "Conn_01x01_Male" (id 1) (at 127 111.76 0))
-    (property "Footprint" "Connector_PinSocket_2.54mm:PinSocket_1x01_P2.54mm_Vertical" (id 2) (at 126.365 114.3 0)
+    (property "Footprint" "Connector_PinHeader_2.54mm:PinHeader_1x01_P2.54mm_Vertical" (id 2) (at 126.365 114.3 0)
       (effects (font (size 1.27 1.27)) hide)
     )
@@
     )
     (path "/6476e233-d260-45fe-84d2-9ade7d0003a0/92cf4db4-2dba-4763-9cd8-3c7f8aff8f24"
-      (reference "J2-1") (unit 1) (value "Conn_01x04_Male") (footprint "Connector_PinSocket_2.54mm:PinSocket_1x04_P2.54mm_Vertical")
+      (reference "J2-1") (unit 1) (value "Conn_01x04_Male") (footprint "Connector_PinHeader_2.54mm:PinHeader_1x04_P2.54mm_Vertical")
     )
     (path "/6476e233-d260-45fe-84d2-9ade7d0003a0/6f75ea3e-6135-44f5-9313-1aad839ab6f6"
-      (reference "J2-2") (unit 1) (value "Conn_01x04_Male") (footprint "Connector_PinSocket_2.54mm:PinSocket_1x04_P2.54mm_Vertical")
+      (reference "J2-2") (unit 1) (value "Conn_01x04_Male") (footprint "Connector_PinHeader_2.54mm:PinHeader_1x04_P2.54mm_Vertical")
     )
     (path "/21f0c995-97eb-43ed-8e0f-a133d3e4b10f"
-      (reference "J3V1") (unit 1) (value "Conn_01x01_Male") (footprint "Connector_PinSocket_2.54mm:PinSocket_1x01_P2.54mm_Vertical")
+      (reference "J3V1") (unit 1) (value "Conn_01x01_Male") (footprint "Connector_PinHeader_2.54mm:PinHeader_1x01_P2.54mm_Vertical")
     )
     (path "/f1a9fb80-4cc4-410f-9616-e19c969dcab5"
@@
     )
     (path "/6476e233-d260-45fe-84d2-9ade7d0003a0/815a0815-7930-45ec-8d6e-dc110f979c75"
-      (reference "JADC1") (unit 1) (value "Conn_01x04_Male") (footprint "Connector_PinSocket_2.54mm:PinSocket_1x04_P2.54mm_Vertical")
+      (reference "JADC1") (unit 1) (value "Conn_01x04_Male") (footprint "Connector_PinHeader_2.54mm:PinHeader_1x04_P2.54mm_Vertical")
     )
     (path "/6476e233-d260-45fe-84d2-9ade7d0003a0/7d4fcb23-c914-48df-941d-94cf5f1f85b5"
-      (reference "JAPC1") (unit 1) (value "Conn_01x04_Male") (footprint "Connector_PinSocket_2.54mm:PinSocket_1x04_P2.54mm_Vertical")
+      (reference "JAPC1") (unit 1) (value "Conn_01x04_Male") (footprint "Connector_PinHeader_2.54mm:PinHeader_1x04_P2.54mm_Vertical")
     )
     (path "/6476e233-d260-45fe-84d2-9ade7d0003a0/95a40d19-41c6-4680-9b37-9cb1bed1a413"
-      (reference "JAUX1") (unit 1) (value "AUX") (footprint "Connector_PinSocket_2.54mm:PinSocket_1x12_P2.54mm_Vertical")
+      (reference "JAUX1") (unit 1) (value "AUX") (footprint "Connector_PinHeader_2.54mm:PinHeader_1x12_P2.54mm_Vertical")
     )
     (path "/6476e233-d260-45fe-84d2-9ade7d0003a0/bf74c99b-6291-4cef-a3b3-a7e4ae401405"
@@
     )
     (path "/6476e233-d260-45fe-84d2-9ade7d0003a0/0df376e0-b3b8-4926-8318-ef70bcc43326"
-      (reference "JD1") (unit 1) (value "Conn_01x04_Male") (footprint "Connector_PinSocket_2.54mm:PinSocket_1x04_P2.54mm_Vertical")
+      (reference "JD1") (unit 1) (value "Conn_01x04_Male") (footprint "Connector_PinHeader_2.54mm:PinHeader_1x04_P2.54mm_Vertical")
     )
     (path "/6476e233-d260-45fe-84d2-9ade7d0003a0/70b53718-ed58-494c-b8a6-19eb974c07c4"
-      (reference "JGPS1") (unit 1) (value "GPS") (footprint "Connector_PinSocket_2.54mm:PinSocket_1x05_P2.54mm_Vertical")
+      (reference "JGPS1") (unit 1) (value "GPS") (footprint "Connector_PinHeader_2.54mm:PinHeader_1x05_P2.54mm_Vertical")
     )
     (path "/6f675e5f-8fe6-4148-baf1-da97afc770f8"
@@
     )
     (path "/6476e233-d260-45fe-84d2-9ade7d0003a0/24cb67fc-f0c9-4f6e-88c1-7636ab854c5e"
-      (reference "JUT1") (unit 1) (value "Conn_01x04_Male") (footprint "Connector_PinSocket_2.54mm:PinSocket_1x04_P2.54mm_Vertical")
+      (reference "JUT1") (unit 1) (value "Conn_01x04_Male") (footprint "Connector_PinHeader_2.54mm:PinHeader_1x04_P2.54mm_Vertical")
     )
     (path "/f686aee0-011d-49d4-b9f1-91a248d4901a"
-      (reference "JVIN1") (unit 1) (value "Conn_01x01_Male") (footprint "Connector_PinSocket_2.54mm:PinSocket_1x01_P2.54mm_Vertical")
+      (reference "JVIN1") (unit 1) (value "Conn_01x01_Male") (footprint "Connector_PinHeader_2.54mm:PinHeader_1x01_P2.54mm_Vertical")
     )
     (path "/fcc3e372-6be4-4e20-89ea-15d74da3ea1f/35afb089-9fdf-4674-9ec7-76a0c05da5b2"

Commit message: SpectDrone Development
Parts:
- C1, C14: Part Number (none) -> CL05A104KA5NNNC
- C13: footprint Capacitor_SMD:C_0805_2012Metric -> Capacitor_SMD:C_0603_1608Metric
- C15, C38: footprint Capacitor_SMD:C_0805_2012Metric -> Capacitor_SMD:C_0402_1005Metric; Part Number (none) -> CL05C2R5CB5NNNC
- C2: Part Number (none) -> 865090368008
- C3: value 100nF -> 0.1uF; footprint Capacitor_SMD:C_0805_2012Metric -> Capacitor_SMD:C_0603_1608Metric; Part Number (none) -> CL05A104KA5NNNC
Changed lines of the file:
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@@
       (effects (font (size 1.27 1.27)) (justify right))
     )
-    (property "Value" "100nF" (id 1) (at 54.61 64.77 90)
-      (effects (font (size 1.27 1.27)) (justify left))
-    )
-    (property "Footprint" "Capacitor_SMD:C_0805_2012Metric" (id 2) (at 53.34 63.5 0)
+    (property "Value" "0.1uF" (id 1) (at 54.61 64.77 90)
+      (effects (font (size 1.27 1.27)) (justify left))
+    )
+    (property "Footprint" "Capacitor_SMD:C_0603_1608Metric" (id 2) (at 53.34 63.5 0)
       (effects (font (size 1.27 1.27)) hide)
     )
     (property "Datasheet" "~" (id 3) (at 53.34 63.5 0)
+      (effects (font (size 1.27 1.27)) hide)
+    )
+    (property "Part Number" "CL05A104KA5NNNC" (id 4) (at 53.34 63.5 0)
       (effects (font (size 1.27 1.27)) hide)
     )
@@
       (effects (font (size 1.27 1.27)) (justify left))
     )
-    (property "Footprint" "Capacitor_SMD:C_0805_2012Metric" (id 2) (at 33.02 35.56 0)
+    (property "Footprint" "Capacitor_SMD:C_0402_1005Metric" (id 2) (at 33.02 35.56 0)
       (effects (font (size 1.27 1.27)) hide)
     )
     (property "Datasheet" "~" (id 3) (at 33.02 35.56 0)
+      (effects (font (size 1.27 1.27)) hide)
+    )
+    (property "Part Number" "CL05C2R5CB5NNNC" (id 4) (at 33.02 35.56 0)
       (effects (font (size 1.27 1.27)) hide)
     )
@@
       (effects (font (size 1.27 1.27)) (justify left))
     )
-    (property "Footprint" "Capacitor_SMD:C_0805_2012Metric" (id 2) (at 111.76 35.56 0)
+    (property "Footprint" "Capacitor_SMD:C_0402_1005Metric" (id 2) (at 111.76 35.56 0)
       (effects (font (size 1.27 1.27)) hide)
     )
     (property "Datasheet" "~" (id 3) (at 111.76 35.56 0)
+      (effects (font (size 1.27 1.27)) hide)
+    )
+    (property "Part Number" "CL05C2R5CB5NNNC" (id 4) (at 111.76 35.56 0)
       (effects (font (size 1.27 1.27)) hide)
     )
@@
       (effects (font (size 1.27 1.27)) hide)
     )
+    (property "Part Number" "865090368008 " (id 4) (at 197.485 34.29 0)
+      (effects (font (size 1.27 1.27)) hide)
+    )
     (pin "1")
     (pin "2")
@@
     )
     (property "Datasheet" "~" (id 3) (at 189.23 34.29 0)
+      (effects (font (size 1.27 1.27)) hide)
+    )
+    (property "Part Number" "CL05A104KA5NNNC" (id 4) (at 189.23 34.29 0)
       (effects (font (size 1.27 1.27)) hide)
     )
@@
     (property "Reference" "C13" (id 0) (at 161.29 29.845 90))
     (property "Value" "10uF" (id 1) (at 161.29 32.385 90))
-    (property "Footprint" "Capacitor_SMD:C_0805_2012Metric" (id 2) (at 161.925 35.56 0)
+    (property "Footprint" "Capacitor_SMD:C_0603_1608Metric" (id 2) (at 161.925 35.56 0)
       (effects (font (size 1.27 1.27)) hide)
     )
@@
       (effects (font (size 1.27 1.27)) hide)
     )
+    (property "Part Number" "CL05A104KA5NNNC" (id 4) (at 161.925 40.005 0)
+      (effects (font (size 1.27 1.27)) hide)
+    )
     (pin "1")
     (pin "2")
@@
     )
     (path "/0b67e92a-4dac-47c1-a2bb-8f4e3cd3cef2"
-      (reference "C3") (unit 1) (value "100nF") (footprint "Capacitor_SMD:C_0805_2012Metric")
+      (reference "C3") (unit 1) (value "0.1uF") (footprint "Capacitor_SMD:C_0603_1608Metric")
     )
     (path "/a5be2cb8-c68d-4180-8412-69a6b4c5b1d4"
-      (reference "C13") (unit 1) (value "10uF") (footprint "Capacitor_SMD:C_0805_2012Metric")
+      (reference "C13") (unit 1) (value "10uF") (footprint "Capacitor_SMD:C_0603_1608Metric")
     )
     (path "/c9b9e62d-dede-4d1a-9a05-275614f8bdb2"
@@
     )
     (path "/2891767f-251c-48c4-91c0-deb1b368f45c"
-      (reference "C15") (unit 1) (value "2.5pF") (footprint "Capacitor_SMD:C_0805_2012Metric")
+      (reference "C15") (unit 1) (value "2.5pF") (footprint "Capacitor_SMD:C_0402_1005Metric")
     )
     (path "/c2d24be9-0a91-4ad8-a6f8-4f606bd871ac/414df5d7-f19b-4687-a4de-327c40e73e20"
@@
     )
     (path "/132b9d29-514e-4bcb-9704-58af6ef66ac0"
-      (reference "C38") (unit 1) (value "2.5pF") (footprint "Capacitor_SMD:C_0805_2012Metric")
+      (reference "C38") (unit 1) (value "2.5pF") (footprint "Capacitor_SMD:C_0402_1005Metric")
     )
     (path "/fcc3e372-6be4-4e20-89ea-15d74da3ea1f/8b9633a8-dd12-495b-8c38-4879c9a2181e"
@@
       (reference "JADC1") (unit 1) (value "Conn_01x04_Male") (footprint "Connector_PinHeader_2.54mm:PinHeader_1x04_P2.54mm_Vertical")
     )
+    (path "/6476e233-d260-45fe-84d2-9ade7d0003a0/c5e053bf-12a3-4339-9020-ec8a06217732"
+      (reference "JADC2") (unit 1) (value "Term_Block_01x08_Female") (footprint "Gardenuino Custom:Term_Block_1x08_Female")
+    )
     (path "/6476e233-d260-45fe-84d2-9ade7d0003a0/7d4fcb23-c914-48df-941d-94cf5f1f85b5"

Commit message: SpectDrone Development
Other:
- moved on the sheet: C13, C14, U1

Commit message: SpectDrone Development
Parts:
- J3V1, JVIN1: Part Number (none) -> PH1-01-UA
- J5, J6: Part Number (none) -> BMI-S-101
- JP11, JP12: now left out of the parts list
- R13, R34: Part Number (none) -> ERJ-6ENF2001V
- R6: Part Number (none) -> ERA-6VRW1002V
- U1: Part Number (none) -> AD7991YRJZ-1500RL7
- U2: Part Number (none) -> ADS1219
Changed lines of the file:
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@@
+      (effects (font (size 1.27 1.27)) hide)
+    )
+    (property "Part Number" "BMI-S-101" (id 4) (at 51.435 35.56 0)
       (effects (font (size 1.27 1.27)) hide)
     )
@@
   )
   (symbol (lib_id "Jumper:SolderJumper_2_Bridged") (at 31.75 40.64 0) (mirror x) (unit 1)
-    (in_bom yes) (on_board yes)
+    (in_bom no) (on_board yes)
     (property "Reference" "JP12" (id 0) (at 31.75 43.18 0))
     (property "Value" "SolderJumper_2_Bridged" (id 1) (at 31.75 44.45 0)
@@
       (effects (font (size 1.27 1.27)) hide)
     )
+    (property "Part Number" "PH1-01-UA" (id 4) (at 126.365 106.045 0)
+      (effects (font (size 1.27 1.27)) hide)
+    )
     (pin "1")
   )
@@
   )
   (symbol (lib_id "Jumper:SolderJumper_2_Bridged") (at 110.49 40.64 0) (mirror x) (unit 1)
-    (in_bom yes) (on_board yes)
+    (in_bom no) (on_board yes)
     (property "Reference" "JP11" (id 0) (at 110.49 43.18 0))
     (property "Value" "SolderJumper_2_Bridged" (id 1) (at 110.49 44.45 0)
@@
       (effects (font (size 1.27 1.27)) hide)
     )
+    (property "Part Number" "ERJ-6ENF2001V" (id 4) (at 31.75 30.48 0)
+      (effects (font (size 1.27 1.27)) hide)
+    )
     (pin "1")
     (pin "2")
@@
     )
     (property "Datasheet" "https://www.analog.com/media/en/technical-documentation/data-sheets/AD7991_7995_7999.pdf" (id 3) (at 149.86 26.67 0)
+      (effects (font (size 1.27 1.27)) hide)
+    )
+    (property "Part Number" "AD7991YRJZ-1500RL7" (id 4) (at 149.86 26.67 0)
       (effects (font (size 1.27 1.27)) hide)
     )
@@
     )
     (property "Datasheet" "http://www.ti.com/lit/ds/symlink/ads1219.pdf" (id 3) (at 72.39 57.15 0)
+      (effects (font (size 1.27 1.27)) hide)
+    )
+    (property "Part Number" "ADS1219" (id 4) (at 72.39 46.99 0)
       (effects (font (size 1.27 1.27)) hide)
     )
@@
       (effects (font (size 1.27 1.27)) hide)
     )
+    (property "Part Number" "ERA-6VRW1002V" (id 4) (at 80.01 30.48 0)
+      (effects (font (size 1.27 1.27)) hide)
+    )
     (pin "1")
     (pin "2")
@@
     )
     (property "Datasheet" "~" (id 3) (at 134.62 35.56 0)
+      (effects (font (size 1.27 1.27)) hide)
+    )
+    (property "Part Number" "BMI-S-101" (id 4) (at 132.08 35.56 0)
       (effects (font (size 1.27 1.27)) hide)
     )
@@
       (effects (font (size 1.27 1.27)) hide)
     )
+    (property "Part Number" "PH1-01-UA" (id 4) (at 126.365 114.3 0)
+      (effects (font (size 1.27 1.27)) hide)
+    )
     (pin "1")
   )
@@
       (effects (font (size 1.27 1.27)) hide)
     )
+    (property "Part Number" "ERJ-6ENF2001V" (id 4) (at 110.49 30.48 0)
+      (effects (font (size 1.27 1.27)) hide)
+    )
