File: TestComponents/TestComponents.kicad_pcb (KiCad board)
At the start: 2 copper layers, 101.7 x 73.7 mm, 117 parts, among them J2-1 Conn_01x04_Male, J2-2 Conn_01x04_Male, J3V1 Conn_01x01_Male, J5 RFShield_OnePiece, J6 RFShield_OnePiece, SW1 SW_SPDT, SW2 SW_SP3T, SW3 SW_SP3T, U1 AD7991, U13 X, U2 ADS1219, U3 REF200AU, U4 MCP6L01x-xLT, U8 ADR510, U9 LM4040B

Commit message: SpectDrone Development
Parts:
- added R_{PD}1.1: 2K, Capacitor_SMD:C_0805_2012Metric, F.Cu at (156.5, 105.0)
- added R_{PD}2.1: 2K, Capacitor_SMD:C_0805_2012Metric, F.Cu at (138.7, 105.0)
- R5: value 174 -> 200
- R_{PD}1, R_{PD}2: value X -> 1M
- moved JPD4 0.40 mm to (136.1, 107.7)
- moved JPD5 0.40 mm to (138.7, 107.7)
- moved JPD6 0.40 mm to (141.2, 107.7)
- moved JPD1 0.38 mm to (153.9, 107.7)
- moved JPD2 0.38 mm to (156.5, 107.7)
- moved JPD3 0.38 mm to (159.0, 107.7)
Connections:
- JPD2 pad 1: /InsturmentationsAmps/PD1_{TEST} -> Net-(JPD2-Pad1)
- JPD3 pad 1: /InsturmentationsAmps/PD1_{TEST} -> Net-(JPD2-Pad1)
- JPD5 pad 1: /InsturmentationsAmps/PD2_{TEST} -> Net-(JPD5-Pad1)
- JPD6 pad 1: /InsturmentationsAmps/PD2_{TEST} -> Net-(JPD5-Pad1)
- PD1 pad 1: /InsturmentationsAmps/PD1_{TEST} -> Net-(JPD2-Pad1)
- PD2 pad 1: /InsturmentationsAmps/PD2_{TEST} -> Net-(JPD5-Pad1)
- RS3 pad 1: Net-(JPD1-Pad2) -> /InsturmentationsAmps/PD1_{TEST}
- RS7 pad 1: Net-(JPD4-Pad2) -> /InsturmentationsAmps/PD2_{TEST}
- R_{PD}1 pad 1: Net-(JPD1-Pad2) -> /InsturmentationsAmps/PD1_{TEST}
- R_{PD}2 pad 1: Net-(JPD4-Pad2) -> /InsturmentationsAmps/PD2_{TEST}
Routing:
- net Net-(JPD5-Pad1): track 0.00 -> 16.9 mm
- net /InsturmentationsAmps/PD1_{TEST}: track 49.7 -> 62.3 mm, vias 1 -> 3
- net Net-(JPD2-Pad1): track 0.00 -> 9.72 mm
- net Net-(JPD1-Pad2): track 16.1 -> 6.45 mm
- net /InsturmentationsAmps/PD2_{TEST}: track 61.0 -> 69.8 mm, vias 1 -> 3
- net Net-(JPD4-Pad2): track 16.1 -> 7.32 mm
- net V_{AREF}: track 120.9 -> 125.0 mm
- net /InsturmentationsAmps/INV2: track 10.3 -> 13.5 mm
- net /InsturmentationsAmps/INV1: track 10.3 -> 13.5 mm
- net P2: track 62.9 -> 65.5 mm
- net PD(V)_{BIAS}: track 59.2 -> 61.4 mm
- net P1: track 70.8 -> 71.5 mm

Commit message: SpectDrone Development
Parts:
- renumbered J2-2 to J2-1, J2-1 to J2-2
Connections:
- J2-1 pad 3: unconnected-(J2-2-Pad3) -> SDA_{RF}
- J2-1 pad 4: unconnected-(J2-2-Pad4) -> SCL_{RF}
- J2-2 pad 3: SDA_{RF} -> unconnected-(J2-2-Pad3)
- J2-2 pad 4: SCL_{RF} -> unconnected-(J2-2-Pad4)
Routing:
- net GND1: track 107.6 -> 82.4 mm
- net SDA_{RF}: track 109.1 -> 97.8 mm
- net SCL_{RF}: track 106.7 -> 97.1 mm
- net P1: track 71.5 -> 68.0 mm
- net -I_{const}=0.4mA: track 13.5 -> 14.7 mm
- net /InsturmentationsAmps/PD1_{TEST}: track 62.3 -> 61.8 mm
Other:
- board text added: "Analog to Digital Expansion, Evaluation, & Calibration Board version 0.1a"
- board text added: "Design by: Shawn L. Jaker shawn.jaker@nrel.gov National Renewable Energy Laboratory Solar Radiation Research Laboratory Golden, Colorado, USA"

Commit message: SpectDrone Development
Parts:
- added REF**: TestPoint_THTPad_D2.0mm_Drill1.0mm, TestPoint:TestPoint_THTPad_D2.0mm_Drill1.0mm, F.Cu at (105.4, 73.7)
- added REF**: TestPoint_THTPad_D2.0mm_Drill1.0mm, TestPoint:TestPoint_THTPad_D2.0mm_Drill1.0mm, F.Cu at (184.3, 87.1)
- added REF**1: TestPoint_THTPad_D2.0mm_Drill1.0mm, TestPoint:TestPoint_THTPad_D2.0mm_Drill1.0mm, F.Cu at (108.0, 73.7)
- added REF**10: TestPoint_THTPad_D2.0mm_Drill1.0mm, TestPoint:TestPoint_THTPad_D2.0mm_Drill1.0mm, F.Cu at (105.4, 76.2)
- added REF**100: TestPoint_THTPad_D2.0mm_Drill1.0mm, TestPoint:TestPoint_THTPad_D2.0mm_Drill1.0mm, F.Cu at (105.4, 99.1)
- added REF**101: TestPoint_THTPad_D2.0mm_Drill1.0mm, TestPoint:TestPoint_THTPad_D2.0mm_Drill1.0mm, F.Cu at (108.0, 99.1)
- added REF**102: TestPoint_THTPad_D2.0mm_Drill1.0mm, TestPoint:TestPoint_THTPad_D2.0mm_Drill1.0mm, F.Cu at (110.5, 99.1)
- added REF**103: TestPoint_THTPad_D2.0mm_Drill1.0mm, TestPoint:TestPoint_THTPad_D2.0mm_Drill1.0mm, F.Cu at (113.0, 99.1)
- added REF**104: TestPoint_THTPad_D2.0mm_Drill1.0mm, TestPoint:TestPoint_THTPad_D2.0mm_Drill1.0mm, F.Cu at (115.6, 99.1)
- added REF**105: TestPoint_THTPad_D2.0mm_Drill1.0mm, TestPoint:TestPoint_THTPad_D2.0mm_Drill1.0mm, F.Cu at (118.1, 99.1)
- added REF**106: TestPoint_THTPad_D2.0mm_Drill1.0mm, TestPoint:TestPoint_THTPad_D2.0mm_Drill1.0mm, F.Cu at (120.7, 99.1)
- added REF**107: TestPoint_THTPad_D2.0mm_Drill1.0mm, TestPoint:TestPoint_THTPad_D2.0mm_Drill1.0mm, F.Cu at (123.2, 99.1)
- added REF**108: TestPoint_THTPad_D2.0mm_Drill1.0mm, TestPoint:TestPoint_THTPad_D2.0mm_Drill1.0mm, F.Cu at (125.7, 99.1)
- added REF**109: TestPoint_THTPad_D2.0mm_Drill1.0mm, TestPoint:TestPoint_THTPad_D2.0mm_Drill1.0mm, F.Cu at (128.3, 99.1)
- added REF**11: TestPoint_THTPad_D2.0mm_Drill1.0mm, TestPoint:TestPoint_THTPad_D2.0mm_Drill1.0mm, F.Cu at (108.0, 76.2)
- added REF**110: TestPoint_THTPad_D2.0mm_Drill1.0mm, TestPoint:TestPoint_THTPad_D2.0mm_Drill1.0mm, F.Cu at (105.4, 101.6)
- added REF**111: TestPoint_THTPad_D2.0mm_Drill1.0mm, TestPoint:TestPoint_THTPad_D2.0mm_Drill1.0mm, F.Cu at (108.0, 101.6)
- added REF**112: TestPoint_THTPad_D2.0mm_Drill1.0mm, TestPoint:TestPoint_THTPad_D2.0mm_Drill1.0mm, F.Cu at (110.5, 101.6)
- added REF**113: TestPoint_THTPad_D2.0mm_Drill1.0mm, TestPoint:TestPoint_THTPad_D2.0mm_Drill1.0mm, F.Cu at (113.0, 101.6)
- added REF**114: TestPoint_THTPad_D2.0mm_Drill1.0mm, TestPoint:TestPoint_THTPad_D2.0mm_Drill1.0mm, F.Cu at (115.6, 101.6)
- added REF**115: TestPoint_THTPad_D2.0mm_Drill1.0mm, TestPoint:TestPoint_THTPad_D2.0mm_Drill1.0mm, F.Cu at (118.1, 101.6)
- added REF**116: TestPoint_THTPad_D2.0mm_Drill1.0mm, TestPoint:TestPoint_THTPad_D2.0mm_Drill1.0mm, F.Cu at (120.7, 101.6)
- added REF**117: TestPoint_THTPad_D2.0mm_Drill1.0mm, TestPoint:TestPoint_THTPad_D2.0mm_Drill1.0mm, F.Cu at (123.2, 101.6)
- added REF**118: TestPoint_THTPad_D2.0mm_Drill1.0mm, TestPoint:TestPoint_THTPad_D2.0mm_Drill1.0mm, F.Cu at (125.7, 101.6)
- added REF**119: TestPoint_THTPad_D2.0mm_Drill1.0mm, TestPoint:TestPoint_THTPad_D2.0mm_Drill1.0mm, F.Cu at (128.3, 101.6)
- added REF**12: TestPoint_THTPad_D2.0mm_Drill1.0mm, TestPoint:TestPoint_THTPad_D2.0mm_Drill1.0mm, F.Cu at (110.5, 76.2)
- added REF**120: TestPoint_THTPad_D2.0mm_Drill1.0mm, TestPoint:TestPoint_THTPad_D2.0mm_Drill1.0mm, F.Cu at (105.4, 104.1)
- added REF**121: TestPoint_THTPad_D2.0mm_Drill1.0mm, TestPoint:TestPoint_THTPad_D2.0mm_Drill1.0mm, F.Cu at (108.0, 104.1)
- added REF**122: TestPoint_THTPad_D2.0mm_Drill1.0mm, TestPoint:TestPoint_THTPad_D2.0mm_Drill1.0mm, F.Cu at (110.5, 104.1)
- added REF**123: TestPoint_THTPad_D2.0mm_Drill1.0mm, TestPoint:TestPoint_THTPad_D2.0mm_Drill1.0mm, F.Cu at (113.0, 104.1)
- added REF**124: TestPoint_THTPad_D2.0mm_Drill1.0mm, TestPoint:TestPoint_THTPad_D2.0mm_Drill1.0mm, F.Cu at (115.6, 104.1)
- added REF**125: TestPoint_THTPad_D2.0mm_Drill1.0mm, TestPoint:TestPoint_THTPad_D2.0mm_Drill1.0mm, F.Cu at (118.1, 104.1)
- added REF**126: TestPoint_THTPad_D2.0mm_Drill1.0mm, TestPoint:TestPoint_THTPad_D2.0mm_Drill1.0mm, F.Cu at (120.7, 104.1)
- added REF**127: TestPoint_THTPad_D2.0mm_Drill1.0mm, TestPoint:TestPoint_THTPad_D2.0mm_Drill1.0mm, F.Cu at (123.2, 104.1)
- added REF**128: TestPoint_THTPad_D2.0mm_Drill1.0mm, TestPoint:TestPoint_THTPad_D2.0mm_Drill1.0mm, F.Cu at (125.7, 104.1)
- added REF**129: TestPoint_THTPad_D2.0mm_Drill1.0mm, TestPoint:TestPoint_THTPad_D2.0mm_Drill1.0mm, F.Cu at (128.3, 104.1)
- added REF**13: TestPoint_THTPad_D2.0mm_Drill1.0mm, TestPoint:TestPoint_THTPad_D2.0mm_Drill1.0mm, F.Cu at (113.0, 76.2)
- added REF**130: TestPoint_THTPad_D2.0mm_Drill1.0mm, TestPoint:TestPoint_THTPad_D2.0mm_Drill1.0mm, F.Cu at (105.4, 106.7)
- added REF**131: TestPoint_THTPad_D2.0mm_Drill1.0mm, TestPoint:TestPoint_THTPad_D2.0mm_Drill1.0mm, F.Cu at (108.0, 106.7)
- added REF**132: TestPoint_THTPad_D2.0mm_Drill1.0mm, TestPoint:TestPoint_THTPad_D2.0mm_Drill1.0mm, F.Cu at (110.5, 106.7)
- added REF**133: TestPoint_THTPad_D2.0mm_Drill1.0mm, TestPoint:TestPoint_THTPad_D2.0mm_Drill1.0mm, F.Cu at (113.0, 106.7)
- added REF**134: TestPoint_THTPad_D2.0mm_Drill1.0mm, TestPoint:TestPoint_THTPad_D2.0mm_Drill1.0mm, F.Cu at (115.6, 106.7)
- added REF**135: TestPoint_THTPad_D2.0mm_Drill1.0mm, TestPoint:TestPoint_THTPad_D2.0mm_Drill1.0mm, F.Cu at (118.1, 106.7)
- added REF**136: TestPoint_THTPad_D2.0mm_Drill1.0mm, TestPoint:TestPoint_THTPad_D2.0mm_Drill1.0mm, F.Cu at (120.7, 106.7)
- added REF**137: TestPoint_THTPad_D2.0mm_Drill1.0mm, TestPoint:TestPoint_THTPad_D2.0mm_Drill1.0mm, F.Cu at (123.2, 106.7)
- added REF**138: TestPoint_THTPad_D2.0mm_Drill1.0mm, TestPoint:TestPoint_THTPad_D2.0mm_Drill1.0mm, F.Cu at (125.7, 106.7)
- added REF**139: TestPoint_THTPad_D2.0mm_Drill1.0mm, TestPoint:TestPoint_THTPad_D2.0mm_Drill1.0mm, F.Cu at (128.3, 106.7)
- added REF**14: TestPoint_THTPad_D2.0mm_Drill1.0mm, TestPoint:TestPoint_THTPad_D2.0mm_Drill1.0mm, F.Cu at (115.6, 76.2)
- added REF**140: TestPoint_THTPad_D2.0mm_Drill1.0mm, TestPoint:TestPoint_THTPad_D2.0mm_Drill1.0mm, F.Cu at (105.4, 109.2)
- added REF**141: TestPoint_THTPad_D2.0mm_Drill1.0mm, TestPoint:TestPoint_THTPad_D2.0mm_Drill1.0mm, F.Cu at (108.0, 109.2)
- added REF**142: TestPoint_THTPad_D2.0mm_Drill1.0mm, TestPoint:TestPoint_THTPad_D2.0mm_Drill1.0mm, F.Cu at (110.5, 109.2)
- added REF**143: TestPoint_THTPad_D2.0mm_Drill1.0mm, TestPoint:TestPoint_THTPad_D2.0mm_Drill1.0mm, F.Cu at (113.0, 109.2)
- added REF**144: TestPoint_THTPad_D2.0mm_Drill1.0mm, TestPoint:TestPoint_THTPad_D2.0mm_Drill1.0mm, F.Cu at (115.6, 109.2)
- added REF**145: TestPoint_THTPad_D2.0mm_Drill1.0mm, TestPoint:TestPoint_THTPad_D2.0mm_Drill1.0mm, F.Cu at (118.1, 109.2)
- added REF**146: TestPoint_THTPad_D2.0mm_Drill1.0mm, TestPoint:TestPoint_THTPad_D2.0mm_Drill1.0mm, F.Cu at (120.7, 109.2)
- added REF**147: TestPoint_THTPad_D2.0mm_Drill1.0mm, TestPoint:TestPoint_THTPad_D2.0mm_Drill1.0mm, F.Cu at (123.2, 109.2)
- added REF**148: TestPoint_THTPad_D2.0mm_Drill1.0mm, TestPoint:TestPoint_THTPad_D2.0mm_Drill1.0mm, F.Cu at (125.7, 109.2)
- added REF**149: TestPoint_THTPad_D2.0mm_Drill1.0mm, TestPoint:TestPoint_THTPad_D2.0mm_Drill1.0mm, F.Cu at (128.3, 109.2)
- added REF**15: TestPoint_THTPad_D2.0mm_Drill1.0mm, TestPoint:TestPoint_THTPad_D2.0mm_Drill1.0mm, F.Cu at (118.1, 76.2)
- added REF**150: TestPoint_THTPad_D2.0mm_Drill1.0mm, TestPoint:TestPoint_THTPad_D2.0mm_Drill1.0mm, F.Cu at (105.4, 111.8)
- added REF**151: TestPoint_THTPad_D2.0mm_Drill1.0mm, TestPoint:TestPoint_THTPad_D2.0mm_Drill1.0mm, F.Cu at (108.0, 111.8)
- added REF**152: TestPoint_THTPad_D2.0mm_Drill1.0mm, TestPoint:TestPoint_THTPad_D2.0mm_Drill1.0mm, F.Cu at (110.5, 111.8)
- added REF**153: TestPoint_THTPad_D2.0mm_Drill1.0mm, TestPoint:TestPoint_THTPad_D2.0mm_Drill1.0mm, F.Cu at (113.0, 111.8)
- added REF**154: TestPoint_THTPad_D2.0mm_Drill1.0mm, TestPoint:TestPoint_THTPad_D2.0mm_Drill1.0mm, F.Cu at (115.6, 111.8)
- added REF**155: TestPoint_THTPad_D2.0mm_Drill1.0mm, TestPoint:TestPoint_THTPad_D2.0mm_Drill1.0mm, F.Cu at (118.1, 111.8)
- added REF**156: TestPoint_THTPad_D2.0mm_Drill1.0mm, TestPoint:TestPoint_THTPad_D2.0mm_Drill1.0mm, F.Cu at (120.7, 111.8)
- added REF**157: TestPoint_THTPad_D2.0mm_Drill1.0mm, TestPoint:TestPoint_THTPad_D2.0mm_Drill1.0mm, F.Cu at (123.2, 111.8)
- added REF**158: TestPoint_THTPad_D2.0mm_Drill1.0mm, TestPoint:TestPoint_THTPad_D2.0mm_Drill1.0mm, F.Cu at (125.7, 111.8)
- added REF**159: TestPoint_THTPad_D2.0mm_Drill1.0mm, TestPoint:TestPoint_THTPad_D2.0mm_Drill1.0mm, F.Cu at (128.3, 111.8)
- added REF**16: TestPoint_THTPad_D2.0mm_Drill1.0mm, TestPoint:TestPoint_THTPad_D2.0mm_Drill1.0mm, F.Cu at (120.7, 76.2)
- added REF**160: TestPoint_THTPad_D2.0mm_Drill1.0mm, TestPoint:TestPoint_THTPad_D2.0mm_Drill1.0mm, F.Cu at (186.8, 87.1)
- added REF**161: TestPoint_THTPad_D2.0mm_Drill1.0mm, TestPoint:TestPoint_THTPad_D2.0mm_Drill1.0mm, F.Cu at (189.4, 87.1)
- added REF**162: TestPoint_THTPad_D2.0mm_Drill1.0mm, TestPoint:TestPoint_THTPad_D2.0mm_Drill1.0mm, F.Cu at (191.9, 87.1)
- added REF**163: TestPoint_THTPad_D2.0mm_Drill1.0mm, TestPoint:TestPoint_THTPad_D2.0mm_Drill1.0mm, F.Cu at (194.4, 87.1)
- added REF**164: TestPoint_THTPad_D2.0mm_Drill1.0mm, TestPoint:TestPoint_THTPad_D2.0mm_Drill1.0mm, F.Cu at (197.0, 87.1)
- added REF**165: TestPoint_THTPad_D2.0mm_Drill1.0mm, TestPoint:TestPoint_THTPad_D2.0mm_Drill1.0mm, F.Cu at (199.5, 87.1)
- added REF**166: TestPoint_THTPad_D2.0mm_Drill1.0mm, TestPoint:TestPoint_THTPad_D2.0mm_Drill1.0mm, F.Cu at (202.1, 87.1)
- added REF**167: TestPoint_THTPad_D2.0mm_Drill1.0mm, TestPoint:TestPoint_THTPad_D2.0mm_Drill1.0mm, F.Cu at (184.3, 89.7)
- added REF**168: TestPoint_THTPad_D2.0mm_Drill1.0mm, TestPoint:TestPoint_THTPad_D2.0mm_Drill1.0mm, F.Cu at (186.8, 89.7)
- added REF**169: TestPoint_THTPad_D2.0mm_Drill1.0mm, TestPoint:TestPoint_THTPad_D2.0mm_Drill1.0mm, F.Cu at (189.4, 89.7)
- added REF**17: TestPoint_THTPad_D2.0mm_Drill1.0mm, TestPoint:TestPoint_THTPad_D2.0mm_Drill1.0mm, F.Cu at (123.2, 76.2)
- added REF**170: TestPoint_THTPad_D2.0mm_Drill1.0mm, TestPoint:TestPoint_THTPad_D2.0mm_Drill1.0mm, F.Cu at (191.9, 89.7)
- added REF**171: TestPoint_THTPad_D2.0mm_Drill1.0mm, TestPoint:TestPoint_THTPad_D2.0mm_Drill1.0mm, F.Cu at (194.4, 89.7)
- added REF**172: TestPoint_THTPad_D2.0mm_Drill1.0mm, TestPoint:TestPoint_THTPad_D2.0mm_Drill1.0mm, F.Cu at (197.0, 89.7)
- added REF**173: TestPoint_THTPad_D2.0mm_Drill1.0mm, TestPoint:TestPoint_THTPad_D2.0mm_Drill1.0mm, F.Cu at (199.5, 89.7)
- added REF**174: TestPoint_THTPad_D2.0mm_Drill1.0mm, TestPoint:TestPoint_THTPad_D2.0mm_Drill1.0mm, F.Cu at (202.1, 89.7)
- added REF**175: TestPoint_THTPad_D2.0mm_Drill1.0mm, TestPoint:TestPoint_THTPad_D2.0mm_Drill1.0mm, F.Cu at (184.3, 92.2)
- added REF**176: TestPoint_THTPad_D2.0mm_Drill1.0mm, TestPoint:TestPoint_THTPad_D2.0mm_Drill1.0mm, F.Cu at (186.8, 92.2)
- added REF**177: TestPoint_THTPad_D2.0mm_Drill1.0mm, TestPoint:TestPoint_THTPad_D2.0mm_Drill1.0mm, F.Cu at (189.4, 92.2)
- added REF**178: TestPoint_THTPad_D2.0mm_Drill1.0mm, TestPoint:TestPoint_THTPad_D2.0mm_Drill1.0mm, F.Cu at (191.9, 92.2)
- added REF**179: TestPoint_THTPad_D2.0mm_Drill1.0mm, TestPoint:TestPoint_THTPad_D2.0mm_Drill1.0mm, F.Cu at (194.4, 92.2)
- added REF**18: TestPoint_THTPad_D2.0mm_Drill1.0mm, TestPoint:TestPoint_THTPad_D2.0mm_Drill1.0mm, F.Cu at (125.7, 76.2)
- added REF**180: TestPoint_THTPad_D2.0mm_Drill1.0mm, TestPoint:TestPoint_THTPad_D2.0mm_Drill1.0mm, F.Cu at (197.0, 92.2)
- added REF**181: TestPoint_THTPad_D2.0mm_Drill1.0mm, TestPoint:TestPoint_THTPad_D2.0mm_Drill1.0mm, F.Cu at (199.5, 92.2)
- added REF**182: TestPoint_THTPad_D2.0mm_Drill1.0mm, TestPoint:TestPoint_THTPad_D2.0mm_Drill1.0mm, F.Cu at (202.1, 92.2)
- added REF**183: TestPoint_THTPad_D2.0mm_Drill1.0mm, TestPoint:TestPoint_THTPad_D2.0mm_Drill1.0mm, F.Cu at (184.3, 94.7)
- added REF**184: TestPoint_THTPad_D2.0mm_Drill1.0mm, TestPoint:TestPoint_THTPad_D2.0mm_Drill1.0mm, F.Cu at (186.8, 94.7)
- added REF**185: TestPoint_THTPad_D2.0mm_Drill1.0mm, TestPoint:TestPoint_THTPad_D2.0mm_Drill1.0mm, F.Cu at (189.4, 94.7)
- added REF**186: TestPoint_THTPad_D2.0mm_Drill1.0mm, TestPoint:TestPoint_THTPad_D2.0mm_Drill1.0mm, F.Cu at (191.9, 94.7)
- added REF**187: TestPoint_THTPad_D2.0mm_Drill1.0mm, TestPoint:TestPoint_THTPad_D2.0mm_Drill1.0mm, F.Cu at (194.4, 94.7)
- added REF**188: TestPoint_THTPad_D2.0mm_Drill1.0mm, TestPoint:TestPoint_THTPad_D2.0mm_Drill1.0mm, F.Cu at (197.0, 94.7)
- added REF**189: TestPoint_THTPad_D2.0mm_Drill1.0mm, TestPoint:TestPoint_THTPad_D2.0mm_Drill1.0mm, F.Cu at (199.5, 94.7)
- added REF**19: TestPoint_THTPad_D2.0mm_Drill1.0mm, TestPoint:TestPoint_THTPad_D2.0mm_Drill1.0mm, F.Cu at (128.3, 76.2)
- added REF**190: TestPoint_THTPad_D2.0mm_Drill1.0mm, TestPoint:TestPoint_THTPad_D2.0mm_Drill1.0mm, F.Cu at (202.1, 94.7)
- added REF**191: TestPoint_THTPad_D2.0mm_Drill1.0mm, TestPoint:TestPoint_THTPad_D2.0mm_Drill1.0mm, F.Cu at (184.3, 97.3)
- added REF**192: TestPoint_THTPad_D2.0mm_Drill1.0mm, TestPoint:TestPoint_THTPad_D2.0mm_Drill1.0mm, F.Cu at (186.8, 97.3)
- added REF**193: TestPoint_THTPad_D2.0mm_Drill1.0mm, TestPoint:TestPoint_THTPad_D2.0mm_Drill1.0mm, F.Cu at (189.4, 97.3)
- added REF**194: TestPoint_THTPad_D2.0mm_Drill1.0mm, TestPoint:TestPoint_THTPad_D2.0mm_Drill1.0mm, F.Cu at (191.9, 97.3)
- added REF**195: TestPoint_THTPad_D2.0mm_Drill1.0mm, TestPoint:TestPoint_THTPad_D2.0mm_Drill1.0mm, F.Cu at (194.4, 97.3)
- added REF**196: TestPoint_THTPad_D2.0mm_Drill1.0mm, TestPoint:TestPoint_THTPad_D2.0mm_Drill1.0mm, F.Cu at (197.0, 97.3)
- added REF**197: TestPoint_THTPad_D2.0mm_Drill1.0mm, TestPoint:TestPoint_THTPad_D2.0mm_Drill1.0mm, F.Cu at (199.5, 97.3)
- added REF**198: TestPoint_THTPad_D2.0mm_Drill1.0mm, TestPoint:TestPoint_THTPad_D2.0mm_Drill1.0mm, F.Cu at (202.1, 97.3)
- added REF**199: TestPoint_THTPad_D2.0mm_Drill1.0mm, TestPoint:TestPoint_THTPad_D2.0mm_Drill1.0mm, F.Cu at (184.3, 99.8)
- added REF**2: TestPoint_THTPad_D2.0mm_Drill1.0mm, TestPoint:TestPoint_THTPad_D2.0mm_Drill1.0mm, F.Cu at (110.5, 73.7)
- added REF**20: TestPoint_THTPad_D2.0mm_Drill1.0mm, TestPoint:TestPoint_THTPad_D2.0mm_Drill1.0mm, F.Cu at (105.4, 78.7)
- added REF**200: TestPoint_THTPad_D2.0mm_Drill1.0mm, TestPoint:TestPoint_THTPad_D2.0mm_Drill1.0mm, F.Cu at (186.8, 99.8)
- added REF**201: TestPoint_THTPad_D2.0mm_Drill1.0mm, TestPoint:TestPoint_THTPad_D2.0mm_Drill1.0mm, F.Cu at (189.4, 99.8)
- added REF**202: TestPoint_THTPad_D2.0mm_Drill1.0mm, TestPoint:TestPoint_THTPad_D2.0mm_Drill1.0mm, F.Cu at (191.9, 99.8)
- added REF**203: TestPoint_THTPad_D2.0mm_Drill1.0mm, TestPoint:TestPoint_THTPad_D2.0mm_Drill1.0mm, F.Cu at (194.4, 99.8)
- added REF**204: TestPoint_THTPad_D2.0mm_Drill1.0mm, TestPoint:TestPoint_THTPad_D2.0mm_Drill1.0mm, F.Cu at (197.0, 99.8)
- added REF**205: TestPoint_THTPad_D2.0mm_Drill1.0mm, TestPoint:TestPoint_THTPad_D2.0mm_Drill1.0mm, F.Cu at (199.5, 99.8)
- added REF**206: TestPoint_THTPad_D2.0mm_Drill1.0mm, TestPoint:TestPoint_THTPad_D2.0mm_Drill1.0mm, F.Cu at (202.1, 99.8)
- added REF**207: TestPoint_THTPad_D2.0mm_Drill1.0mm, TestPoint:TestPoint_THTPad_D2.0mm_Drill1.0mm, F.Cu at (184.3, 102.4)
- added REF**208: TestPoint_THTPad_D2.0mm_Drill1.0mm, TestPoint:TestPoint_THTPad_D2.0mm_Drill1.0mm, F.Cu at (186.8, 102.4)
- added REF**209: TestPoint_THTPad_D2.0mm_Drill1.0mm, TestPoint:TestPoint_THTPad_D2.0mm_Drill1.0mm, F.Cu at (189.4, 102.4)
- added REF**21: TestPoint_THTPad_D2.0mm_Drill1.0mm, TestPoint:TestPoint_THTPad_D2.0mm_Drill1.0mm, F.Cu at (108.0, 78.7)
- added REF**210: TestPoint_THTPad_D2.0mm_Drill1.0mm, TestPoint:TestPoint_THTPad_D2.0mm_Drill1.0mm, F.Cu at (191.9, 102.4)
- added REF**211: TestPoint_THTPad_D2.0mm_Drill1.0mm, TestPoint:TestPoint_THTPad_D2.0mm_Drill1.0mm, F.Cu at (194.4, 102.4)
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Connections:
- JGPS1 pad 1: /TestConnectors/5V -> /TestConnectors/GPS_5V
- JGPS1 pad 2: /TestConnectors/GND -> /TestConnectors/GPS_GND
- SW3 pad 1: -I_{const}=0.4mA -> -I_{const}=1.5mA
- SW3 pad 2: unconnected-(SW3-Pad2) -> /InsturmentationsAmps/PD_{TEST}
- SW3 pad 3: /InsturmentationsAmps/PD_{TEST} -> -I_{const}=0.4mA
- SW3 pad 4: -I_{const}=1.5mA -> -I_{const}=0.4mA
Routing:
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Other:
- board size 101.7 x 73.7 mm -> 101.6 x 73.7 mm
- board text added: "TEST CURRENT 1.5mA <- | -> 400uA"
- board text added: "TEST PD CHANNEL 1 <- nc -> 2"
- board text removed: "TEST CURRENT 0.400 <- 0 -> 1.50 mA"
- board text removed: "TEST PD CHANNEL 2 <- nc -> 1"

Commit message: SpectDrone Development
Parts:
- removed the REF** at (105.4, 73.7)
- removed the REF** at (184.3, 87.1)
- removed REF**1, REF**10, REF**100, REF**101, REF**102, REF**103, REF**104, REF**105, REF**106, REF**107, REF**108, REF**109, REF**11, REF**110, REF**111, REF**112, REF**113, REF**114, REF**115, REF**116, REF**117, REF**118, REF**119, REF**12, REF**120, REF**121, REF**122, REF**123, REF**124, REF**125, REF**126, REF**127, REF**128, REF**129, REF**13, REF**130, REF**131, REF**132, REF**133, REF**134, REF**135, REF**136, REF**137, REF**138, REF**139, REF**14, REF**140, REF**141, REF**142, REF**143, REF**144, REF**145, REF**146, REF**147, REF**148, REF**149, REF**15, REF**150, REF**151, REF**152, REF**153, REF**154, REF**155, REF**156, REF**157, REF**158, REF**159, REF**16, REF**160, REF**161, REF**162, REF**163, REF**164, REF**165, REF**166, REF**167, REF**168, REF**169, REF**17, REF**170, REF**171, REF**172, REF**173, REF**174, REF**175, REF**176, REF**177, REF**178, REF**179, REF**18, REF**180, REF**181, REF**182, REF**183, REF**184, REF**185, REF**186, REF**187, REF**188, REF**189, REF**19, REF**190, REF**191, REF**192, REF**193, REF**194, REF**195, REF**196, REF**197, REF**198, REF**199, REF**2, REF**20, REF**200, REF**201, REF**202, REF**203, REF**204, REF**205, REF**206, REF**207, REF**208, REF**209, REF**21, REF**210, REF**211, REF**212, REF**213, REF**214, REF**215, REF**216, REF**217, REF**218, REF**219, REF**22, REF**220, REF**221, REF**222, REF**223, REF**224, REF**225, REF**226, REF**227, REF**228, REF**229, REF**23, REF**230, REF**231, REF**232, REF**233, REF**234, REF**235, REF**236, REF**237, REF**238, REF**239, REF**24, REF**240, REF**241, REF**242, REF**243, REF**244, REF**245, REF**246, REF**247, REF**248, REF**249, REF**25, REF**250, REF**251, REF**252, REF**253, REF**254, REF**255, REF**256, REF**257, REF**258, REF**259, REF**26, REF**260, REF**261, REF**262, REF**263, REF**264, REF**265, REF**266, REF**267, REF**268, REF**269, REF**27, REF**270, REF**271, REF**272, REF**273, REF**274, REF**275, REF**276, REF**277, REF**278, REF**279, REF**28, REF**280, REF**281, REF**282, REF**283, REF**284, REF**285, REF**286, REF**287, REF**288, REF**289, REF**29, REF**290, REF**291, REF**292, REF**293, REF**294, REF**295, REF**296, REF**297, REF**298, REF**299, REF**3, REF**30, REF**300, REF**301, REF**302, REF**303, REF**304, REF**305, REF**306, REF**307, REF**308, REF**309, REF**31, REF**310, REF**32, REF**33, REF**34, REF**35, REF**36, REF**37, REF**38, REF**39, REF**4, REF**40, REF**41, REF**42, REF**43, REF**44, REF**45, REF**46, REF**47, REF**48, REF**49, REF**5, REF**50, REF**51, REF**52, REF**53, REF**54, REF**55, REF**56, REF**57, REF**58, REF**59, REF**6, REF**60, REF**61, REF**62, REF**63, REF**64, REF**65, REF**66, REF**67, REF**68, REF**69, REF**7, REF**70, REF**71, REF**72, REF**73, REF**74, REF**75, REF**76, REF**77, REF**78, REF**79, REF**8, REF**80, REF**81, REF**82, REF**83, REF**84, REF**85, REF**86, REF**87, REF**88, REF**89, REF**9, REF**90, REF**91, REF**92, REF**93, REF**94, REF**95, REF**96, REF**97, REF**98, REF**99: TestPoint_THTPad_D2.0mm_Drill1.0mm, TestPoint:TestPoint_THTPad_D2.0mm_Drill1.0mm
- added JAUX2: AUX, Connector_PinSocket_2.54mm:PinSocket_1x12_P2.54mm_Vertical, F.Cu at (128.7, 136.2)
- added REF**: PinHeader_Corner, Gardenuino Custom:PinHeader_Corner, F.Cu at (184.2, 137.2)
- added REF**: PinHeader_Corner, Gardenuino Custom:PinHeader_Corner, F.Cu at (133.3, 68.6)
- SW1: value SW_SPDT -> SW_DPDT; footprint Button_Switch_SMD:SW_SPDT_CK-JS102011SAQN -> Gardenuino Custom:SW_DPDT_CK_JS202011JAQN
- moved U3 1.28 mm to (183.9, 80.1)
- moved CS11 1.28 mm to (176.0, 78.3)
- moved CS12 1.28 mm to (173.2, 80.9)
- moved CS13 1.28 mm to (173.2, 82.9)
- moved R1 1.28 mm to (178.1, 78.3)
- moved R2 1.28 mm to (180.1, 78.3)
- moved U4 1.28 mm to (173.2, 78.3)
- moved SW1 0.76 mm to (152.7, 133.6)
- moved RV1 0.50 mm to (160.5, 130.3)
- moved SW2 0.25 mm to (172.0, 72.0)
Routing:
- net /TestConnectors/TXS_{E}_5V: track 0.00 -> 3.81 mm
- net /TestConnectors/SDA_5V: track 0.00 -> 3.81 mm
- net /TestConnectors/SCL_5V: track 0.00 -> 3.81 mm
- net /TestConnectors/SCK_5V: track 0.00 -> 3.81 mm
- net /TestConnectors/MOSI_5V: track 0.00 -> 3.81 mm
- net /TestConnectors/MISO_5V: track 0.00 -> 3.81 mm
- net /TestConnectors/GND: track 0.00 -> 3.81 mm
- net /TestConnectors/CAM2TX_5V: track 0.00 -> 3.81 mm
- net /TestConnectors/CAM2RX_5V: track 0.00 -> 3.81 mm
- net /TestConnectors/CAM1TX_5V: track 0.00 -> 3.81 mm
- net /TestConnectors/CAM1RX_5V: track 0.00 -> 3.81 mm
- net /TestConnectors/5V: track 0.00 -> 3.81 mm
- net PD(V)_{BIAS}: track 110.1 -> 113.8 mm
- net /InsturmentationsAmps/PD1_{TEST}: track 58.5 -> 62.0 mm
- net 1V1: track 30.6 -> 33.2 mm
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Other:
- board text added: "CAM1RX"
- board text added: "CAM1TX"
- board text added: "CAM2RX"
- board text added: "CAM2TX"
- board text added: "GND"
- board text added: "MISO"
- board text added: "MOSI"
- board text added: "P1"
- board text added: "P2"
- board text added: "S1"
- board text added: "S2"
- board text added: "SCK"
- board text added: "SCL_{3V}"
- board text added: "SCL_{5V}"
- board text added: "SDA_{3V}"
- board text added: "SDA_{5V}"
- board text added: "TXSe"

Commit message: SpectDrone Development
Parts:
- B1: renamed from REF**; value PinHeader_Corner -> Conn_02x20_Top_Bottom; footprint Gardenuino Custom:PinHeader_Corner -> Gardenuino Custom:PinHeader_CornerB1
- B2: renamed from REF**; value PinHeader_Corner -> Conn_02x20_Top_Bottom; footprint Gardenuino Custom:PinHeader_Corner -> Gardenuino Custom:PinHeader_CornerB2
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Connections:
- B1 pad 1: (no net) -> 5V3
- B1 pad 10: (no net) -> unconnected-(B1-Pad10)
- B1 pad 100: (no net) -> unconnected-(B1-Pad100)
- B1 pad 101: (no net) -> /TestConnectors/UT1_5V
- B1 pad 102: (no net) -> unconnected-(B1-Pad102)
- B1 pad 103: (no net) -> unconnected-(B1-Pad103)
- B1 pad 104: (no net) -> unconnected-(B1-Pad104)
- B1 pad 105: (no net) -> unconnected-(B1-Pad105)
- B1 pad 106: (no net) -> unconnected-(B1-Pad106)
- B1 pad 107: (no net) -> unconnected-(B1-Pad107)
- B1 pad 108: (no net) -> unconnected-(B1-Pad108)
- B1 pad 109: (no net) -> /TestConnectors/RX_5V
- B1 pad 11: (no net) -> unconnected-(B1-Pad11)
- B1 pad 110: (no net) -> unconnected-(B1-Pad110)
- B1 pad 111: (no net) -> unconnected-(B1-Pad111)
- B1 pad 112: (no net) -> unconnected-(B1-Pad112)
- B1 pad 113: (no net) -> unconnected-(B1-Pad113)
- B1 pad 114: (no net) -> unconnected-(B1-Pad114)
- B1 pad 115: (no net) -> unconnected-(B1-Pad115)
- B1 pad 116: (no net) -> unconnected-(B1-Pad116)
- B1 pad 117: (no net) -> /TestConnectors/TX_5V
- B1 pad 118: (no net) -> unconnected-(B1-Pad118)
- B1 pad 119: (no net) -> unconnected-(B1-Pad119)
- B1 pad 12: (no net) -> unconnected-(B1-Pad12)
- B1 pad 120: (no net) -> unconnected-(B1-Pad120)
- B1 pad 121: (no net) -> unconnected-(B1-Pad121)
- B1 pad 122: (no net) -> unconnected-(B1-Pad122)
- B1 pad 123: (no net) -> unconnected-(B1-Pad123)
- B1 pad 124: (no net) -> unconnected-(B1-Pad124)
- B1 pad 125: (no net) -> /TestConnectors/APCRX_5V
- B1 pad 126: (no net) -> unconnected-(B1-Pad126)
- B1 pad 127: (no net) -> unconnected-(B1-Pad127)
- B1 pad 128: (no net) -> unconnected-(B1-Pad128)
- B1 pad 129: (no net) -> unconnected-(B1-Pad129)
- B1 pad 13: (no net) -> J-2-4
- B1 pad 130: (no net) -> unconnected-(B1-Pad130)
- B1 pad 131: (no net) -> unconnected-(B1-Pad131)
- B1 pad 132: (no net) -> unconnected-(B1-Pad132)
- B1 pad 133: (no net) -> /TestConnectors/GAIN_5V
- B1 pad 134: (no net) -> /TestConnectors/ST_5V
- B1 pad 135: (no net) -> unconnected-(B1-Pad135)
- B1 pad 136: (no net) -> /TestConnectors/APCTX_5V
- B1 pad 137: (no net) -> unconnected-(B1-Pad137)
- B1 pad 138: (no net) -> unconnected-(B1-Pad138)
- B1 pad 139: (no net) -> unconnected-(B1-Pad139)
- B1 pad 14: (no net) -> unconnected-(B1-Pad14)
- B1 pad 140: (no net) -> unconnected-(B1-Pad140)
- B1 pad 141: (no net) -> unconnected-(B1-Pad141)
- B1 pad 142: (no net) -> unconnected-(B1-Pad142)
- B1 pad 143: (no net) -> unconnected-(B1-Pad143)
- B1 pad 144: (no net) -> /TestConnectors/CLK2_5V
- B1 pad 145: (no net) -> /TestConnectors/CLK1_5V
- B1 pad 146: (no net) -> unconnected-(B1-Pad146)
- B1 pad 147: (no net) -> unconnected-(B1-Pad147)
- B1 pad 148: (no net) -> unconnected-(B1-Pad148)
- B1 pad 149: (no net) -> unconnected-(B1-Pad149)
- B1 pad 15: (no net) -> unconnected-(B1-Pad15)
- B1 pad 150: (no net) -> unconnected-(B1-Pad150)
- B1 pad 151: (no net) -> unconnected-(B1-Pad151)
- B1 pad 152: (no net) -> unconnected-(B1-Pad152)
- B1 pad 153: (no net) -> unconnected-(B1-Pad153)
- B1 pad 154: (no net) -> unconnected-(B1-Pad154)
- B1 pad 155: (no net) -> unconnected-(B1-Pad155)
- B1 pad 156: (no net) -> unconnected-(B1-Pad156)
- B1 pad 157: (no net) -> unconnected-(B1-Pad157)
- B1 pad 158: (no net) -> unconnected-(B1-Pad158)
- B1 pad 159: (no net) -> unconnected-(B1-Pad159)
- B1 pad 16: (no net) -> unconnected-(B1-Pad16)
- B1 pad 160: (no net) -> unconnected-(B1-Pad160)
- B1 pad 161: (no net) -> unconnected-(B1-Pad161)
- B1 pad 162: (no net) -> unconnected-(B1-Pad162)
- B1 pad 163: (no net) -> unconnected-(B1-Pad163)
- B1 pad 164: (no net) -> unconnected-(B1-Pad164)
- B1 pad 165: (no net) -> unconnected-(B1-Pad165)
- B1 pad 166: (no net) -> unconnected-(B1-Pad166)
- B1 pad 167: (no net) -> unconnected-(B1-Pad167)
- B1 pad 168: (no net) -> unconnected-(B1-Pad168)
- B1 pad 169: (no net) -> unconnected-(B1-Pad169)
- B1 pad 17: (no net) -> unconnected-(B1-Pad17)
- B1 pad 170: (no net) -> unconnected-(B1-Pad170)
- B1 pad 171: (no net) -> unconnected-(B1-Pad171)
- B1 pad 172: (no net) -> unconnected-(B1-Pad172)
- B1 pad 173: (no net) -> unconnected-(B1-Pad173)
- B1 pad 174: (no net) -> unconnected-(B1-Pad174)
- B1 pad 175: (no net) -> unconnected-(B1-Pad175)
- B1 pad 176: (no net) -> unconnected-(B1-Pad176)
- B1 pad 177: (no net) -> unconnected-(B1-Pad177)
- B1 pad 178: (no net) -> unconnected-(B1-Pad178)
- B1 pad 179: (no net) -> unconnected-(B1-Pad179)
- B1 pad 18: (no net) -> unconnected-(B1-Pad18)
- B1 pad 180: (no net) -> unconnected-(B1-Pad180)
- B1 pad 181: (no net) -> unconnected-(B1-Pad181)
- B1 pad 182: (no net) -> unconnected-(B1-Pad182)
- B1 pad 183: (no net) -> unconnected-(B1-Pad183)
- B1 pad 184: (no net) -> unconnected-(B1-Pad184)
- B1 pad 185: (no net) -> unconnected-(B1-Pad185)
- B1 pad 186: (no net) -> unconnected-(B1-Pad186)
- B1 pad 187: (no net) -> unconnected-(B1-Pad187)
- B1 pad 188: (no net) -> unconnected-(B1-Pad188)
- B1 pad 189: (no net) -> unconnected-(B1-Pad189)
- B1 pad 19: (no net) -> unconnected-(B1-Pad19)
- B1 pad 190: (no net) -> unconnected-(B1-Pad190)
- B1 pad 191: (no net) -> unconnected-(B1-Pad191)
- B1 pad 192: (no net) -> unconnected-(B1-Pad192)
- B1 pad 193: (no net) -> unconnected-(B1-Pad193)
- B1 pad 194: (no net) -> unconnected-(B1-Pad194)
- B1 pad 195: (no net) -> unconnected-(B1-Pad195)
- B1 pad 196: (no net) -> unconnected-(B1-Pad196)
- B1 pad 197: (no net) -> unconnected-(B1-Pad197)
- B1 pad 2: (no net) -> unconnected-(B1-Pad2)
- B1 pad 20: (no net) -> unconnected-(B1-Pad20)
- B1 pad 21: (no net) -> J-2-3
- B1 pad 22: (no net) -> unconnected-(B1-Pad22)
- B1 pad 23: (no net) -> unconnected-(B1-Pad23)
- B1 pad 24: (no net) -> unconnected-(B1-Pad24)
- B1 pad 25: (no net) -> unconnected-(B1-Pad25)
- B1 pad 26: (no net) -> unconnected-(B1-Pad26)
- B1 pad 27: (no net) -> unconnected-(B1-Pad27)
- B1 pad 28: (no net) -> unconnected-(B1-Pad28)
- B1 pad 29: (no net) -> J-2-2
- B1 pad 3: (no net) -> unconnected-(B1-Pad3)
- B1 pad 30: (no net) -> unconnected-(B1-Pad30)
- B1 pad 31: (no net) -> unconnected-(B1-Pad31)
- B1 pad 32: (no net) -> unconnected-(B1-Pad32)
- B1 pad 33: (no net) -> unconnected-(B1-Pad33)
- B1 pad 34: (no net) -> unconnected-(B1-Pad34)
- B1 pad 35: (no net) -> unconnected-(B1-Pad35)
- B1 pad 36: (no net) -> unconnected-(B1-Pad36)
- B1 pad 37: (no net) -> J-2-1
- B1 pad 38: (no net) -> unconnected-(B1-Pad38)
- B1 pad 39: (no net) -> unconnected-(B1-Pad39)
- B1 pad 4: (no net) -> unconnected-(B1-Pad4)
- B1 pad 40: (no net) -> unconnected-(B1-Pad40)
- B1 pad 41: (no net) -> unconnected-(B1-Pad41)
- B1 pad 42: (no net) -> unconnected-(B1-Pad42)
- B1 pad 43: (no net) -> unconnected-(B1-Pad43)
- B1 pad 44: (no net) -> unconnected-(B1-Pad44)
- B1 pad 45: (no net) -> J-1-4
- B1 pad 46: (no net) -> unconnected-(B1-Pad46)
- B1 pad 47: (no net) -> unconnected-(B1-Pad47)
- B1 pad 48: (no net) -> unconnected-(B1-Pad48)
- B1 pad 49: (no net) -> unconnected-(B1-Pad49)
- B1 pad 5: (no net) -> unconnected-(B1-Pad5)
- B1 pad 50: (no net) -> unconnected-(B1-Pad50)
- B1 pad 51: (no net) -> unconnected-(B1-Pad51)
- B1 pad 52: (no net) -> unconnected-(B1-Pad52)
- B1 pad 53: (no net) -> J-1-3
- B1 pad 54: (no net) -> unconnected-(B1-Pad54)
- B1 pad 55: (no net) -> unconnected-(B1-Pad55)
- B1 pad 56: (no net) -> unconnected-(B1-Pad56)
- B1 pad 57: (no net) -> unconnected-(B1-Pad57)
- B1 pad 58: (no net) -> unconnected-(B1-Pad58)
- B1 pad 59: (no net) -> unconnected-(B1-Pad59)
- B1 pad 6: (no net) -> unconnected-(B1-Pad6)
- B1 pad 60: (no net) -> unconnected-(B1-Pad60)
- B1 pad 61: (no net) -> J-1-2
- B1 pad 62: (no net) -> unconnected-(B1-Pad62)
- B1 pad 63: (no net) -> unconnected-(B1-Pad63)
- B1 pad 64: (no net) -> unconnected-(B1-Pad64)
- B1 pad 65: (no net) -> unconnected-(B1-Pad65)
- B1 pad 66: (no net) -> unconnected-(B1-Pad66)
- B1 pad 67: (no net) -> unconnected-(B1-Pad67)
- B1 pad 68: (no net) -> unconnected-(B1-Pad68)
- B1 pad 69: (no net) -> J-1-1
- B1 pad 7: (no net) -> GND1
- B1 pad 70: (no net) -> unconnected-(B1-Pad70)
- B1 pad 71: (no net) -> unconnected-(B1-Pad71)
- B1 pad 72: (no net) -> unconnected-(B1-Pad72)
- B1 pad 73: (no net) -> unconnected-(B1-Pad73)
- B1 pad 74: (no net) -> unconnected-(B1-Pad74)
- B1 pad 75: (no net) -> unconnected-(B1-Pad75)
- B1 pad 76: (no net) -> unconnected-(B1-Pad76)
- B1 pad 77: (no net) -> /TestConnectors/CAN_L_5V
- B1 pad 78: (no net) -> unconnected-(B1-Pad78)
- B1 pad 79: (no net) -> unconnected-(B1-Pad79)
- B1 pad 8: (no net) -> unconnected-(B1-Pad8)
- B1 pad 80: (no net) -> unconnected-(B1-Pad80)
- B1 pad 81: (no net) -> unconnected-(B1-Pad81)
- B1 pad 82: (no net) -> unconnected-(B1-Pad82)
- B1 pad 83: (no net) -> unconnected-(B1-Pad83)
- B1 pad 84: (no net) -> unconnected-(B1-Pad84)
- B1 pad 85: (no net) -> /TestConnectors/CAN_H_5V
- B1 pad 86: (no net) -> unconnected-(B1-Pad86)
- B1 pad 87: (no net) -> unconnected-(B1-Pad87)
- B1 pad 88: (no net) -> unconnected-(B1-Pad88)
- B1 pad 89: (no net) -> unconnected-(B1-Pad89)
- B1 pad 9: (no net) -> unconnected-(B1-Pad9)
- B1 pad 90: (no net) -> unconnected-(B1-Pad90)
- B1 pad 91: (no net) -> unconnected-(B1-Pad91)
- B1 pad 92: (no net) -> unconnected-(B1-Pad92)
- B1 pad 93: (no net) -> /TestConnectors/UT2_5V
- B1 pad 94: (no net) -> unconnected-(B1-Pad94)
- B1 pad 95: (no net) -> unconnected-(B1-Pad95)
- B1 pad 96: (no net) -> unconnected-(B1-Pad96)
- B1 pad 97: (no net) -> unconnected-(B1-Pad97)
- B1 pad 98: (no net) -> unconnected-(B1-Pad98)
- B1 pad 99: (no net) -> unconnected-(B1-Pad99)
- B2 pad 1: (no net) -> 5V3
- B2 pad 10: (no net) -> unconnected-(B2-Pad10)
- B2 pad 100: (no net) -> unconnected-(B2-Pad100)
- B2 pad 101: (no net) -> unconnected-(B2-Pad101)
- B2 pad 102: (no net) -> unconnected-(B2-Pad102)
- B2 pad 103: (no net) -> unconnected-(B2-Pad103)
- B2 pad 104: (no net) -> unconnected-(B2-Pad104)
- B2 pad 105: (no net) -> unconnected-(B2-Pad105)
- B2 pad 106: (no net) -> unconnected-(B2-Pad106)
- B2 pad 107: (no net) -> unconnected-(B2-Pad107)
- B2 pad 108: (no net) -> unconnected-(B2-Pad108)
- B2 pad 109: (no net) -> unconnected-(B2-Pad109)
- B2 pad 11: (no net) -> GND1
- B2 pad 110: (no net) -> unconnected-(B2-Pad110)
- B2 pad 111: (no net) -> unconnected-(B2-Pad111)
- B2 pad 112: (no net) -> unconnected-(B2-Pad112)
- B2 pad 113: (no net) -> unconnected-(B2-Pad113)
- B2 pad 114: (no net) -> unconnected-(B2-Pad114)
- B2 pad 115: (no net) -> unconnected-(B2-Pad115)
- B2 pad 116: (no net) -> unconnected-(B2-Pad116)
- B2 pad 117: (no net) -> unconnected-(B2-Pad117)
- B2 pad 118: (no net) -> unconnected-(B2-Pad118)
- B2 pad 119: (no net) -> unconnected-(B2-Pad119)
- B2 pad 12: (no net) -> unconnected-(B2-Pad12)
- B2 pad 120: (no net) -> unconnected-(B2-Pad120)
- B2 pad 121: (no net) -> unconnected-(B2-Pad121)
- B2 pad 122: (no net) -> unconnected-(B2-Pad122)
- B2 pad 123: (no net) -> unconnected-(B2-Pad123)
- B2 pad 124: (no net) -> unconnected-(B2-Pad124)
- B2 pad 125: (no net) -> unconnected-(B2-Pad125)
- B2 pad 126: (no net) -> unconnected-(B2-Pad126)
- B2 pad 127: (no net) -> unconnected-(B2-Pad127)
- B2 pad 128: (no net) -> unconnected-(B2-Pad128)
- B2 pad 129: (no net) -> unconnected-(B2-Pad129)
- B2 pad 13: (no net) -> unconnected-(B2-Pad13)
- B2 pad 130: (no net) -> unconnected-(B2-Pad130)
- B2 pad 131: (no net) -> unconnected-(B2-Pad131)
- B2 pad 132: (no net) -> unconnected-(B2-Pad132)
- B2 pad 133: (no net) -> unconnected-(B2-Pad133)
- B2 pad 134: (no net) -> unconnected-(B2-Pad134)
- B2 pad 135: (no net) -> unconnected-(B2-Pad135)
- B2 pad 136: (no net) -> unconnected-(B2-Pad136)
- B2 pad 137: (no net) -> unconnected-(B2-Pad137)
- B2 pad 138: (no net) -> unconnected-(B2-Pad138)
- B2 pad 139: (no net) -> unconnected-(B2-Pad139)
- B2 pad 14: (no net) -> unconnected-(B2-Pad14)
- B2 pad 140: (no net) -> unconnected-(B2-Pad140)
- B2 pad 141: (no net) -> unconnected-(B2-Pad141)
- B2 pad 142: (no net) -> unconnected-(B2-Pad142)
- B2 pad 143: (no net) -> unconnected-(B2-Pad143)
- B2 pad 144: (no net) -> unconnected-(B2-Pad144)
- B2 pad 145: (no net) -> unconnected-(B2-Pad145)
- B2 pad 146: (no net) -> unconnected-(B2-Pad146)
- B2 pad 147: (no net) -> unconnected-(B2-Pad147)
- B2 pad 148: (no net) -> unconnected-(B2-Pad148)
- B2 pad 149: (no net) -> unconnected-(B2-Pad149)
- B2 pad 15: (no net) -> unconnected-(B2-Pad15)
- B2 pad 150: (no net) -> unconnected-(B2-Pad150)
- B2 pad 151: (no net) -> unconnected-(B2-Pad151)
- B2 pad 152: (no net) -> unconnected-(B2-Pad152)
- B2 pad 153: (no net) -> unconnected-(B2-Pad153)
- B2 pad 154: (no net) -> unconnected-(B2-Pad154)
- B2 pad 155: (no net) -> unconnected-(B2-Pad155)
- B2 pad 156: (no net) -> unconnected-(B2-Pad156)
- B2 pad 157: (no net) -> unconnected-(B2-Pad157)
- B2 pad 158: (no net) -> unconnected-(B2-Pad158)
- B2 pad 159: (no net) -> unconnected-(B2-Pad159)
- B2 pad 16: (no net) -> unconnected-(B2-Pad16)
- B2 pad 160: (no net) -> unconnected-(B2-Pad160)
- B2 pad 161: (no net) -> unconnected-(B2-Pad161)
- B2 pad 162: (no net) -> unconnected-(B2-Pad162)
- B2 pad 163: (no net) -> unconnected-(B2-Pad163)
- B2 pad 164: (no net) -> unconnected-(B2-Pad164)
- B2 pad 165: (no net) -> unconnected-(B2-Pad165)
- B2 pad 166: (no net) -> unconnected-(B2-Pad166)
- B2 pad 167: (no net) -> unconnected-(B2-Pad167)
- B2 pad 168: (no net) -> unconnected-(B2-Pad168)
- B2 pad 169: (no net) -> unconnected-(B2-Pad169)
- B2 pad 17: (no net) -> unconnected-(B2-Pad17)
- B2 pad 170: (no net) -> unconnected-(B2-Pad170)
- B2 pad 171: (no net) -> unconnected-(B2-Pad171)
- B2 pad 172: (no net) -> unconnected-(B2-Pad172)
- B2 pad 173: (no net) -> unconnected-(B2-Pad173)
- B2 pad 174: (no net) -> unconnected-(B2-Pad174)
- B2 pad 175: (no net) -> unconnected-(B2-Pad175)
- B2 pad 176: (no net) -> unconnected-(B2-Pad176)
- B2 pad 177: (no net) -> unconnected-(B2-Pad177)
- B2 pad 178: (no net) -> unconnected-(B2-Pad178)
- B2 pad 179: (no net) -> unconnected-(B2-Pad179)
- B2 pad 18: (no net) -> unconnected-(B2-Pad18)
- B2 pad 180: (no net) -> unconnected-(B2-Pad180)
- B2 pad 181: (no net) -> unconnected-(B2-Pad181)
- B2 pad 182: (no net) -> unconnected-(B2-Pad182)
- B2 pad 183: (no net) -> unconnected-(B2-Pad183)
- B2 pad 184: (no net) -> unconnected-(B2-Pad184)
- B2 pad 185: (no net) -> unconnected-(B2-Pad185)
- B2 pad 186: (no net) -> unconnected-(B2-Pad186)
- B2 pad 187: (no net) -> unconnected-(B2-Pad187)
- B2 pad 188: (no net) -> unconnected-(B2-Pad188)
- B2 pad 189: (no net) -> /TestConnectors/GPS_5V
- B2 pad 19: (no net) -> unconnected-(B2-Pad19)
- B2 pad 190: (no net) -> /TestConnectors/GPS_GND
- B2 pad 191: (no net) -> /TestConnectors/GPSRX_5V
- B2 pad 192: (no net) -> /TestConnectors/GPSTX_5V
- B2 pad 193: (no net) -> /TestConnectors/PPS_5V
- B2 pad 194: (no net) -> unconnected-(B2-Pad194)
- B2 pad 195: (no net) -> unconnected-(B2-Pad195)
- B2 pad 2: (no net) -> unconnected-(B2-Pad2)
- B2 pad 20: (no net) -> unconnected-(B2-Pad20)
- B2 pad 21: (no net) -> 3V1
- B2 pad 22: (no net) -> unconnected-(B2-Pad22)
- B2 pad 23: (no net) -> unconnected-(B2-Pad23)
- B2 pad 24: (no net) -> unconnected-(B2-Pad24)
- B2 pad 25: (no net) -> unconnected-(B2-Pad25)
- B2 pad 26: (no net) -> unconnected-(B2-Pad26)
- B2 pad 27: (no net) -> unconnected-(B2-Pad27)
- B2 pad 28: (no net) -> unconnected-(B2-Pad28)
- B2 pad 29: (no net) -> unconnected-(B2-Pad29)
- B2 pad 3: (no net) -> unconnected-(B2-Pad3)
- B2 pad 30: (no net) -> unconnected-(B2-Pad30)
- B2 pad 31: (no net) -> unconnected-(B2-Pad31)
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Routing:
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Other:
- board text added: "3V3"
- board text added: "APCRX"
- board text added: "APCTX"
- board text added: "CAN_H"
- board text added: "CAN_L"
- board text added: "CLK1"
- board text added: "CLK2"
- board text added: "GAIN"
- board text added: "GPSRX"
- board text added: "GPSTX"
- board text added: "GPS_5V"
- board text added: "GPS_GND"
- board text added: "J2-1-1"
- board text added: "J2-1-2"
- board text added: "J2-2-1"
- board text added: "J2-2-2"
- board text added: "J2-2-3"
- board text added: "J2-2-4"
- board text added: "PPS"
- board text added: "RX"
- board text added: "ST"
- board text added: "TX"
- board text added: "UT1"
- board text added: "UT2"
