File: TestComponents/TestComponents.kicad_pcb (KiCad board)
At the start: 2 copper layers, 101.6 x 73.7 mm, 123 parts, among them J2-1 Conn_01x04_Male, J2-2 Conn_01x04_Male, J3V1 Conn_01x01_Male, J5 RFShield_OnePiece, J6 RFShield_OnePiece, SW1 SW_DPDT, SW2 SW_DP3T, SW3 SW_DPDT, U1 AD7991, U13 X, U2 ADS1219, U3 REF200AU, U4 MCP6L01x-xLT, U8 ADR510, U9 LM4040B

Commit message: SpectDrone Development
Routing:
- net V_{RF}: track 45.7 -> 44.4 mm
- net S2_{RF}: track 5.85 -> 5.20 mm
Changed lines of the file:
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@@
     (effects (font (size 0.5 0.5) (thickness 0.075)))
   )
-  (gr_text "0" (at 139.6891 95.0566 180) (layer "F.SilkS")
+  (gr_text "0" (at 139.6891 94.7166 180) (layer "F.SilkS")
     (effects (font (size 0.5 0.5) (thickness 0.1) italic) (justify mirror))
   )
@@
     (effects (font (size 0.5 0.5) (thickness 0.125)))
   )
-  (gr_text "0" (at 145.2751 91.7546) (layer "F.SilkS")
+  (gr_text "0" (at 145.2751 91.4654) (layer "F.SilkS")
     (effects (font (size 0.5 0.5) (thickness 0.1) italic) (justify mirror))
   )
@@
     (effects (font (size 1 1) (thickness 0.15)) (justify left))
   )
-  (gr_text "0" (at 145.4529 95.0566 180) (layer "F.SilkS")
+  (gr_text "0" (at 145.4603 94.7166 180) (layer "F.SilkS")
     (effects (font (size 0.5 0.5) (thickness 0.1) italic) (justify mirror))
   )
@@
     (effects (font (size 1 1) (thickness 0.15)) (justify right))
   )
+  (segment (start 145.7447 86.2174) (end 144.1849 86.2174) (width 0.4) (layer "F.Cu") (net 1))
+  (segment (start 146.4697 88.2138) (end 146.4697 89.7131) (width 0.4) (layer "F.Cu") (net 1))
   (segment (start 161.417 82.931) (end 161.417 83.439) (width 0.4) (layer "F.Cu") (net 1))
   (segment (start 142.6581 86.2702) (end 142.6081 86.2202) (width 0.4) (layer "F.Cu") (net 1))
-  (segment (start 146.2418 87.9859) (end 145.4158 87.1599) (width 0.4) (layer "F.Cu") (net 1))
   (segment (start 141.0971 86.2202) (end 141.0841 86.2332) (width 0.4) (layer "F.Cu") (net 1))
-  (segment (start 145.4529 86.7762) (end 145.4529 87.1228) (width 0.4) (layer "F.Cu") (net 1))
-  (segment (start 144.5046 86.6427) (end 144.1321 86.2702) (width 0.4) (layer "F.Cu") (net 1))
   (segment (start 155.2956 86.741) (end 155.6056 87.051) (width 0.25) (layer "F.Cu") (net 1))
   (segment (start 142.6081 86.2202) (end 141.0971 86.2202) (width 0.4) (layer "F.Cu") (net 1))
   (segment (start 144.1321 86.2702) (end 142.6581 86.2702) (width 0.4) (layer "F.Cu") (net 1))
-  (segment (start 145.3194 86.6427) (end 145.4529 86.7762) (width 0.4) (layer "F.Cu") (net 1))
-  (segment (start 146.4697 88.2138) (end 146.4697 89.7131) (width 0.4) (layer "F.Cu") (net 1))
   (segment (start 156.3955 85.101) (end 155.6148 85.101) (width 0.25) (layer "F.Cu") (net 1))
+  (segment (start 146.2418 87.9859) (end 145.7447 87.4888) (width 0.4) (layer "F.Cu") (net 1))
   (segment (start 155.6056 87.051) (end 156.3955 87.051) (width 0.25) (layer "F.Cu") (net 1))
-  (segment (start 145.4529 87.1228) (end 145.4158 87.1599) (width 0.4) (layer "F.Cu") (net 1))
   (segment (start 145.7447 87.4888) (end 145.7447 86.2174) (width 0.4) (layer "F.Cu") (net 1))
   (segment (start 139.2201 88.694417) (end 139.2201 89.4487) (width 0.4) (layer "F.Cu") (net 1))
   (segment (start 141.0841 86.830417) (end 139.2201 88.694417) (width 0.4) (layer "F.Cu") (net 1))
+  (segment (start 144.1849 86.2174) (end 144.1321 86.2702) (width 0.4) (layer "F.Cu") (net 1))
   (segment (start 139.4681 86.2332) (end 139.3061 86.3952) (width 0.4) (layer "F.Cu") (net 1))
   (segment (start 141.0841 86.2332) (end 141.0841 86.830417) (width 0.4) (layer "F.Cu") (net 1))
   (segment (start 157.647889 83.848611) (end 156.3955 85.101) (width 0.4) (layer "F.Cu") (net 1))
+  (segment (start 146.2418 87.9859) (end 146.4697 88.2138) (width 0.4) (layer "F.Cu") (net 1))
   (segment (start 145.7447 84.6839) (end 145.7447 83.2363) (width 0.4) (layer "F.Cu") (net 1))
   (segment (start 161.007389 83.848611) (end 157.647889 83.848611) (width 0.4) (layer "F.Cu") (net 1))
   (segment (start 141.0841 86.2332) (end 139.4681 86.2332) (width 0.4) (layer "F.Cu") (net 1))
   (segment (start 161.417 83.439) (end 161.007389 83.848611) (width 0.4) (layer "F.Cu") (net 1))
-  (segment (start 146.2418 87.9859) (end 146.4697 88.2138) (width 0.4) (layer "F.Cu") (net 1))
   (segment (start 155.6148 85.101) (end 155.2956 85.4202) (width 0.25) (layer "F.Cu") (net 1))
-  (segment (start 145.3194 86.6427) (end 145.7447 86.2174) (width 0.4) (layer "F.Cu") (net 1))
   (segment (start 155.2956 85.4202) (end 155.2956 86.741) (width 0.25) (layer "F.Cu") (net 1))
   (segment (start 145.7447 86.2174) (end 145.7447 84.6839) (width 0.4) (layer "F.Cu") (net 1))
-  (segment (start 145.3194 86.6427) (end 144.5046 86.6427) (width 0.4) (layer "F.Cu") (net 1))
   (segment (start 145.7447 83.2363) (end 146.05 82.931) (width 0.4) (layer "F.Cu") (net 1))
   (via (at 146.05 82.931) (size 0.8) (drill 0.4) (layers "F.Cu" "B.Cu") (net 1))
@@
   (segment (start 154.94 91.948) (end 154.94 92.972614) (width 0.25) (layer "B.Cu") (net 5))
   (segment (start 153.932614 93.98) (end 153.924 93.98) (width 0.25) (layer "B.Cu") (net 5))
-  (segment (start 140.7311 94.0734) (end 140.7797 94.0734) (width 0.25) (layer "F.Cu") (net 6))
-  (segment (start 141.1271 93.726) (end 141.028044 93.726) (width 0.25) (layer "F.Cu") (net 6))
-  (segment (start 140.903872 93.900628) (end 140.7311 94.0734) (width 0.25) (layer "F.Cu") (net 6))
-  (segment (start 140.5201 92.8162) (end 140.903872 93.199972) (width 0.25) (layer "F.Cu") (net 6))
-  (segment (start 140.7797 94.0734) (end 141.1271 93.726) (width 0.25) (layer "F.Cu") (net 6))
-  (segment (start 140.5201 91.7237) (end 140.5201 92.8162) (width 0.25) (layer "F.Cu") (net 6))
-  (segment (start 141.0971 94.742) (end 140.1991 94.742) (width 0.25) (layer "F.Cu") (net 6))
-  (segment (start 141.028044 93.726) (end 140.903872 93.850172) (width 0.25) (layer "F.Cu") (net 6))
-  (segment (start 141.1271 93.726) (end 141.1271 94.712) (width 0.25) (layer "F.Cu") (net 6))
-  (segment (start 140.1991 94.0734) (end 140.7311 94.0734) (width 0.25) (layer "F.Cu") (net 6))
-  (segment (start 141.1271 94.712) (end 141.0971 94.742) (width 0.25) (layer "F.Cu") (net 6))
-  (segment (start 140.903872 93.900628) (end 140.903872 93.199972) (width 0.25) (layer "F.Cu") (net 6))
+  (segment (start 140.1991 94.742) (end 141.0971 94.742) (width 0.25) (layer "F.Cu") (net 6))
+  (segment (start 140.18 93.726) (end 140.18 94.7229) (width 0.25) (layer "F.Cu") (net 6))
+  (segment (start 140.79455 93.39345) (end 141.1271 93.726) (width 0.25) (layer "F.Cu") (net 6))
+  (segment (start 140.787 93.3859) (end 140.79455 93.39345) (width 0.25) (layer "F.Cu") (net 6))
+  (segment (start 140.5201 93.119) (end 140.5201 93.3859) (width 0.25) (layer "F.Cu") (net 6))
+  (segment (start 140.5201 91.7237) (end 140.5201 93.119) (width 0.25) (layer "F.Cu") (net 6))
+  (segment (start 140.5201 93.3859) (end 140.18 93.726) (width 0.25) (layer "F.Cu") (net 6))
+  (segment (start 140.18 94.7229) (end 140.1991 94.742) (width 0.25) (layer "F.Cu") (net 6))
+  (segment (start 140.5201 93.3859) (end 140.787 93.3859) (width 0.25) (layer "F.Cu") (net 6))
+  (segment (start 140.5201 93.119) (end 140.79455 93.39345) (width 0.25) (layer "F.Cu") (net 6))
   (segment (start 163.1305 110.871) (end 163.1715 110.912) (width 0.4) (layer "F.Cu") (net 7))
   (segment (start 147.2947 86.2174) (end 147.2947 84.6839) (width 0.4) (layer "F.Cu") (net 7))
@@
   (segment (start 183.261 82.58502) (end 183.261 83.6695) (width 0.4) (layer "F.Cu") (net 63))
   (segment (start 181.991 82.58502) (end 183.261 82.58502) (width 0.4) (layer "F.Cu") (net 63))
-  (segment (start 155.6704 94.0405) (end 156.5984 94.0405) (width 0.25) (layer "F.Cu") (net 65))
+  (segment (start 156.083 91.937079) (end 158.496 89.524079) (width 0.25) (layer "F.Cu") (net 65))
+  (segment (start 156.5984 94.0405) (end 156.24695 93.68905) (width 0.25) (layer "F.Cu") (net 65))
+  (segment (start 155.6704 95.0565) (end 156.5684 95.0565) (width 0.25) (layer "F.Cu") (net 65))
+  (segment (start 156.083 93.5979) (end 155.95545 93.72545) (width 0.25) (layer "F.Cu") (net 65))
+  (segment (start 156.083 93.5251) (end 156.083 91.937079) (width 0.25) (layer "F.Cu") (net 65))
+  (segment (start 155.6404 94.0405) (end 155.6404 95.0265) (width 0.25) (layer "F.Cu") (net 65))
+  (segment (start 156.083 93.5251) (end 156.083 93.5979) (width 0.25) (layer "F.Cu") (net 65))
+  (segment (start 158.496 87.5538) (end 157.3432 86.401) (width 0.25) (layer "F.Cu") (net 65))
+  (segment (start 157.3432 86.401) (end 156.3955 86.401) (width 0.25) (layer "F.Cu") (net 65))
+  (segment (start 156.24695 93.68905) (end 156.083 93.5251) (width 0.25) (layer "F.Cu") (net 65))
+  (segment (start 155.95545 93.72545) (end 155.6404 94.0405) (width 0.25) (layer "F.Cu") (net 65))
+  (segment (start 155.95545 93.72545) (end 156.21055 93.72545) (width 0.25) (layer "F.Cu") (net 65))
+  (segment (start 155.6404 95.0265) (end 155.6704 95.0565) (width 0.25) (layer "F.Cu") (net 65))
   (segment (start 158.496 89.524079) (end 158.496 87.5538) (width 0.25) (layer "F.Cu") (net 65))
-  (segment (start 156.5684 95.0565) (end 155.6704 95.0565) (width 0.25) (layer "F.Cu") (net 65))
-  (segment (start 158.496 87.5538) (end 157.3432 86.401) (width 0.25) (layer "F.Cu") (net 65))
-  (segment (start 156.5984 94.0405) (end 156.5984 95.0265) (width 0.25) (layer "F.Cu") (net 65))
-  (segment (start 156.5984 94.0405) (end 156.337 93.7791) (width 0.25) (layer "F.Cu") (net 65))
-  (segment (start 156.5984 95.0265) (end 156.5684 95.0565) (width 0.25) (layer "F.Cu") (net 65))
-  (segment (start 156.337 93.7791) (end 156.337 91.683079) (width 0.25) (layer "F.Cu") (net 65))
-  (segment (start 157.3432 86.401) (end 156.3955 86.401) (width 0.25) (layer "F.Cu") (net 65))
-  (segment (start 156.337 91.683079) (end 158.496 89.524079) (width 0.25) (layer "F.Cu") (net 65))
+  (segment (start 156.21055 93.72545) (end 156.24695 93.68905) (width 0.25) (layer "F.Cu") (net 65))
   (segment (start 157.4552 85.751) (end 159.004 87.2998) (width 0.25) (layer "F.Cu") (net 66))
   (segment (start 159.5256 95.0469) (end 160.4236 95.0469) (width 0.25) (layer "F.Cu") (net 66))

Commit message: SpectDrone Development
Parts:
- J2-1, J2-2, JADC1, JAPC1, JD1, JUT1: footprint Connector_PinSocket_2.54mm:PinSocket_1x04_P2.54mm_Vertical -> Connector_PinHeader_2.54mm:PinHeader_1x04_P2.54mm_Vertical
- J3V1, JVIN1: footprint Connector_PinSocket_2.54mm:PinSocket_1x01_P2.54mm_Vertical -> Connector_PinHeader_2.54mm:PinHeader_1x01_P2.54mm_Vertical
- JAUX1: footprint Connector_PinSocket_2.54mm:PinSocket_1x12_P2.54mm_Vertical -> Connector_PinHeader_2.54mm:PinHeader_1x12_P2.54mm_Vertical
- JGPS1: footprint Connector_PinSocket_2.54mm:PinSocket_1x05_P2.54mm_Vertical -> Connector_PinHeader_2.54mm:PinHeader_1x05_P2.54mm_Vertical
- moved JVIN1 0.89 mm to (190.2, 75.4)
- moved SW3 0.64 mm to (183.5, 72.0)
Connections:
- B1 pad 199: unconnected-(B1-Pad199) -> GND1
- B1 pad 200: unconnected-(B1-Pad200) -> VIN
- JAUX1 pad 1: 5V3 -> unconnected-(JAUX1-Pad1)
- JAUX1 pad 10: /TestConnectors/CAM1RX_5V -> unconnected-(JAUX1-Pad10)
- JAUX1 pad 11: /TestConnectors/CAM1TX_5V -> unconnected-(JAUX1-Pad11)
- JAUX1 pad 12: /TestConnectors/TXS_{E}_5V -> unconnected-(JAUX1-Pad12)
- JAUX1 pad 2: GND1 -> unconnected-(JAUX1-Pad2)
- JAUX1 pad 3: /TestConnectors/MOSI_5V -> unconnected-(JAUX1-Pad3)
- JAUX1 pad 4: /TestConnectors/SCK_5V -> unconnected-(JAUX1-Pad4)
- JAUX1 pad 5: /TestConnectors/MISO_5V -> unconnected-(JAUX1-Pad5)
- JAUX1 pad 6: /TestConnectors/SCL_5V -> unconnected-(JAUX1-Pad6)
- JAUX1 pad 7: /TestConnectors/SDA_5V -> unconnected-(JAUX1-Pad7)
- JAUX1 pad 8: /TestConnectors/CAM2RX_5V -> unconnected-(JAUX1-Pad8)
- JAUX1 pad 9: /TestConnectors/CAM2TX_5V -> unconnected-(JAUX1-Pad9)
Routing:
- net unconnected-(JAUX1-Pad2): track 0.00 -> 16.6 mm, vias 0 -> 1
- net GND1: track 100.8 -> 84.2 mm, vias 6 -> 5
- net VIN: track 0.00 -> 14.2 mm
- net unconnected-(JAUX1-Pad8): track 0.00 -> 3.81 mm
- net unconnected-(JAUX1-Pad7): track 0.00 -> 3.81 mm
- net unconnected-(JAUX1-Pad6): track 0.00 -> 3.81 mm
- net unconnected-(JAUX1-Pad5): track 0.00 -> 3.81 mm
- net unconnected-(JAUX1-Pad11): track 0.00 -> 3.81 mm
- net /TestConnectors/SDA_5V: track 3.81 -> 0.00 mm
- net /TestConnectors/SCL_5V: track 3.81 -> 0.00 mm
- net /TestConnectors/MISO_5V: track 3.81 -> 0.00 mm
- net /TestConnectors/CAM2RX_5V: track 3.81 -> 0.00 mm
- net /TestConnectors/CAM1TX_5V: track 3.81 -> 0.00 mm
- net -I_{const}=1.5mA: track 17.1 -> 16.5 mm
- net /InsturmentationsAmps/PD_{TEST}: track 15.3 -> 14.7 mm

Commit message: SpectDrone Development
Parts:
- removed JAUX2: AUX, Connector_PinSocket_2.54mm:PinSocket_1x12_P2.54mm_Vertical
- added TPGND-1: TestPoint, TestPoint:TestPoint_Keystone_5000-5004_Miniature, F.Cu at (149.2, 70.5)
- added TPV1: TestPoint, TestPoint:TestPoint_Keystone_5000-5004_Miniature, F.Cu at (155.6, 117.1)
- added TPV3: TestPoint, TestPoint:TestPoint_Keystone_5000-5004_Miniature, F.Cu at (149.2, 117.1)
- added TPV5: TestPoint, TestPoint:TestPoint_Keystone_5000-5004_Miniature, F.Cu at (155.6, 70.5)
- moved SW1 0.72 mm to (152.7, 132.9)
- moved RV1 0.57 mm to (160.3, 129.8)
Connections:
- B2 pad 115: unconnected-(B2-Pad115) -> /TestConnectors/TXS_{E}_5V
- B2 pad 127: unconnected-(B2-Pad127) -> /TestConnectors/CAM1TX_5V
- B2 pad 139: unconnected-(B2-Pad139) -> /TestConnectors/CAM1RX_5V
- B2 pad 151: unconnected-(B2-Pad151) -> /TestConnectors/CAM2TX_5V
- B2 pad 163: unconnected-(B2-Pad163) -> /TestConnectors/CAM2RX_5V
- B2 pad 185: unconnected-(B2-Pad185) -> /TestConnectors/SDA_5V
- B2 pad 186: unconnected-(B2-Pad186) -> /TestConnectors/SCL_5V
- B2 pad 187: unconnected-(B2-Pad187) -> /TestConnectors/MISO_5V
- B2 pad 188: unconnected-(B2-Pad188) -> /TestConnectors/SCK_5V
- B2 pad 189: /TestConnectors/GPS_5V -> /TestConnectors/MOSI_5V
- B2 pad 190: /TestConnectors/GPS_GND -> unconnected-(B2-Pad190)
- B2 pad 191: /TestConnectors/GPSRX_5V -> /TestConnectors/GPS_5V
- B2 pad 192: /TestConnectors/GPSTX_5V -> unconnected-(B2-Pad192)
- B2 pad 193: /TestConnectors/PPS_5V -> unconnected-(B2-Pad193)
- JAUX1 pad 1: unconnected-(JAUX1-Pad1) -> 5V3
- JAUX1 pad 10: unconnected-(JAUX1-Pad10) -> /TestConnectors/CAM1RX_5V
- JAUX1 pad 11: unconnected-(JAUX1-Pad11) -> /TestConnectors/CAM1TX_5V
- JAUX1 pad 12: unconnected-(JAUX1-Pad12) -> /TestConnectors/TXS_{E}_5V
- JAUX1 pad 2: unconnected-(JAUX1-Pad2) -> GND1
- JAUX1 pad 3: unconnected-(JAUX1-Pad3) -> /TestConnectors/MOSI_5V
- JAUX1 pad 4: unconnected-(JAUX1-Pad4) -> /TestConnectors/SCK_5V
- JAUX1 pad 5: unconnected-(JAUX1-Pad5) -> /TestConnectors/MISO_5V
- JAUX1 pad 6: unconnected-(JAUX1-Pad6) -> /TestConnectors/SCL_5V
- JAUX1 pad 7: unconnected-(JAUX1-Pad7) -> /TestConnectors/SDA_5V
- JAUX1 pad 8: unconnected-(JAUX1-Pad8) -> /TestConnectors/CAM2RX_5V
- JAUX1 pad 9: unconnected-(JAUX1-Pad9) -> /TestConnectors/CAM2TX_5V
Routing:
- net /TestConnectors/MOSI_5V: track 3.81 -> 31.1 mm
- net /TestConnectors/SCK_5V: track 3.81 -> 26.5 mm
- net /TestConnectors/MISO_5V: track 0.00 -> 21.6 mm
- net /TestConnectors/SCL_5V: track 0.00 -> 17.1 mm
- net unconnected-(JAUX1-Pad2): track 16.6 -> 0.00 mm, vias 1 -> 0
- net GND1: track 84.2 -> 100.8 mm, vias 5 -> 6
- net /TestConnectors/CAM2RX_5V: track 0.00 -> 16.4 mm
- net /TestConnectors/CAM1TX_5V: track 0.00 -> 15.7 mm
- net /TestConnectors/CAM1RX_5V: track 3.81 -> 19.3 mm
- net /TestConnectors/SDA_5V: track 0.00 -> 13.5 mm
- net /TestConnectors/CAM2TX_5V: track 3.81 -> 16.4 mm
- net V_{AREF}: track 125.8 -> 137.8 mm
- net /TestConnectors/TXS_{E}_5V: track 3.81 -> 15.0 mm
- net /TestConnectors/PPS_5V: track 25.1 -> 31.4 mm
- net /TestConnectors/GPSTX_5V: track 21.5 -> 26.8 mm
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Other:
- board text added: "1 <- nc -> 2"
- board text added: "1.00V"
- board text added: "1.5mA <-|-> 400uA"
- board text added: "3.00V <-|-> 1.00V"
- board text added: "PD TEST CHANNEL"
- board text added: "REVERSE BIAS AND REFERENCE VOLTAGE"
- board text added: "TEST CURRENT"
- board text added: "TPGND"
- board text added: "VOLTAGE ADJUST"
- board text removed: "REVERSE BIAS AND REFERENCE VOLTAGE <-- 3.00V | 1.00V -->"
- board text removed: "TEST CURRENT 1.5mA <- | -> 400uA"
- board text removed: "TEST PD CHANNEL 1 <- nc -> 2"
