File: TestComponents/TestComponents.kicad_pcb (KiCad board)
At the start: 2 copper layers, 101.6 x 73.7 mm, 126 parts, among them J2-1 Conn_01x04_Male, J2-2 Conn_01x04_Male, J3V1 Conn_01x01_Male, J5 RFShield_OnePiece, J6 RFShield_OnePiece, SW1 SW_DPDT, SW2 SW_DP3T, SW3 SW_DPDT, U1 AD7991, U13 X, U2 ADS1219, U3 REF200AU, U4 MCP6L01x-xLT, U8 ADR510, U9 LM4040B

Commit message: SpectDrone Development
Parts:
- added JADC2: Term_Block_01x08_Female, Gardenuino Custom:Term_Block_1x08_Female, B.Cu at (180.3, 86.4)
- C13: footprint Capacitor_SMD:C_0805_2012Metric -> Capacitor_SMD:C_0603_1608Metric
- C15, C38: footprint Capacitor_SMD:C_0805_2012Metric -> Capacitor_SMD:C_0402_1005Metric
- C3: value 100nF -> 0.1uF; footprint Capacitor_SMD:C_0805_2012Metric -> Capacitor_SMD:C_0603_1608Metric
- moved C38 5.47 mm to (158.5, 80.3), turned to 90 degrees
- moved C3 1.71 mm to (154.2, 77.7)
- moved R13 0.15 mm to (137.9, 81.0)
Connections:
- B1 pad 133: /TestConnectors/GAIN_5V -> unconnected-(B1-Pad133)
- B1 pad 134: /TestConnectors/ST_5V -> unconnected-(B1-Pad134)
- B1 pad 144: /TestConnectors/CLK2_5V -> unconnected-(B1-Pad144)
- B1 pad 145: /TestConnectors/CLK1_5V -> unconnected-(B1-Pad145)
- B1 pad 170: unconnected-(B1-Pad170) -> P1
- B1 pad 171: unconnected-(B1-Pad171) -> S1
- B1 pad 172: unconnected-(B1-Pad172) -> P2
- B1 pad 173: unconnected-(B1-Pad173) -> S2
- B1 pad 174: unconnected-(B1-Pad174) -> /TestConnectors/CLK2_5V
- B1 pad 175: unconnected-(B1-Pad175) -> /TestConnectors/GAIN_5V
- B1 pad 176: unconnected-(B1-Pad176) -> /TestConnectors/ST_5V
- B1 pad 177: unconnected-(B1-Pad177) -> /TestConnectors/CLK1_5V
Routing:
- net S2: track 46.5 -> 69.0 mm
- net P2: track 64.6 -> 84.3 mm
- net S1: track 42.7 -> 60.4 mm
- net /TestConnectors/ST_5V: track 6.95 -> 20.4 mm
- net P1: track 67.8 -> 80.2 mm
- net /TestConnectors/GAIN_5V: track 9.49 -> 21.4 mm
- net /TestConnectors/CLK2_5V: track 16.7 -> 24.6 mm
- net /TestConnectors/CLK1_5V: track 11.5 -> 17.4 mm
- net /InsturmentationsAmps/PD2_{TEST}: track 72.5 -> 75.1 mm
- net /InsturmentationsAmps/PD1_{TEST}: track 59.5 -> 60.9 mm
- net Net-(U3-Pad1): track 12.7 -> 11.8 mm
- net GND1: track 100.8 -> 100.1 mm
- net GND_{RF}: track 129.7 -> 129.1 mm
Other:
- board text added: "TPV1"
- board text added: "TPV3"
- board text added: "TPV5"

Commit message: SpectDrone Development
Parts:
- removed JADC2: Term_Block_01x08_Female, Gardenuino Custom:Term_Block_1x08_Female
- added JMISO5: SolderJumper_2_Bridged, Jumper:SolderJumper-2_P1.3mm_Bridged_RoundedPad1.0x1.5mm, F.Cu at (128.8, 126.0)
- added JMOSI5: SolderJumper_2_Bridged, Jumper:SolderJumper-2_P1.3mm_Bridged_RoundedPad1.0x1.5mm, F.Cu at (128.8, 131.1)
- added JSCK5: SolderJumper_2_Bridged, Jumper:SolderJumper-2_P1.3mm_Bridged_RoundedPad1.0x1.5mm, F.Cu at (128.8, 128.6)
- added JSCL5: SolderJumper_2_Bridged, Jumper:SolderJumper-2_P1.3mm_Bridged_RoundedPad1.0x1.5mm, F.Cu at (128.8, 123.5)
- added JSDA5: SolderJumper_2_Bridged, Jumper:SolderJumper-2_P1.3mm_Bridged_RoundedPad1.0x1.5mm, F.Cu at (128.8, 121.0)
- R4, R5, R9, RS3, RS6, RS7, RS8, R_{C}1, R_{PD}1, R_{PD}1.1, R_{PD}2, R_{PD}2.1: footprint Capacitor_SMD:C_0805_2012Metric -> Resistor_SMD:R_0805_2012Metric
- moved JP11 0.13 mm to (141.0, 80.3)
- moved JP12 0.10 mm to (156.5, 80.3)
Connections:
- B2 pad 185: /TestConnectors/SDA_5V -> Net-(B2-Pad185)
- B2 pad 186: /TestConnectors/SCL_5V -> Net-(B2-Pad186)
- B2 pad 187: /TestConnectors/MISO_5V -> Net-(B2-Pad187)
- B2 pad 188: /TestConnectors/SCK_5V -> Net-(B2-Pad188)
- B2 pad 189: /TestConnectors/MOSI_5V -> Net-(B2-Pad189)
Routing:
- net Net-(B2-Pad189): track 0.00 -> 28.3 mm
- net /TestConnectors/MOSI_5V: track 31.1 -> 3.03 mm
- net Net-(B2-Pad188): track 0.00 -> 23.6 mm
- net /TestConnectors/SCK_5V: track 26.5 -> 3.03 mm
- net Net-(B2-Pad187): track 0.00 -> 18.9 mm
- net /TestConnectors/MISO_5V: track 21.6 -> 3.03 mm
- net Net-(B2-Pad186): track 0.00 -> 15.3 mm
- net /TestConnectors/SCL_5V: track 17.1 -> 3.03 mm
- net Net-(B2-Pad185): track 0.00 -> 13.4 mm
- net /TestConnectors/SDA_5V: track 13.5 -> 3.03 mm
- net /TestConnectors/TXS_{E}_5V: track 15.0 -> 18.3 mm
- net /TestConnectors/CAM2TX_5V: track 16.4 -> 18.0 mm
- net /TestConnectors/CAM1TX_5V: track 15.7 -> 17.0 mm
- net /TestConnectors/CAM1RX_5V: track 19.3 -> 18.1 mm
- net /TestConnectors/GPSTX_5V: track 26.8 -> 25.7 mm
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
Commit message: SpectDrone Development
Parts:
- U9: value LM4040B -> ADR5043B
Connections:
- SW3 pad 6: unconnected-(SW3-Pad6) -> -I_{const}=1.5mA
Routing:
- net -I_{const}=1.5mA: track 16.5 -> 24.8 mm
- net -I_{const}=0.4mA: track 23.9 -> 28.0 mm
- net /InsturmentationsAmps/PD_{TEST}: track 14.7 -> 16.0 mm
- net Net-(R_{C}1-Pad1): track 62.7 -> 63.8 mm
- net /InsturmentationsAmps/PD1_{TEST}: track 61.0 -> 60.4 mm

Commit message: SpectDrone Development
Parts:
- CS1, CS6: footprint Capacitor_SMD:C_0805_2012Metric -> Capacitor_SMD:C_0603_1608Metric
- CS2, CS3, CS7, CS8: footprint Capacitor_SMD:C_0805_2012Metric -> Capacitor_SMD:C_0402_1005Metric
- U9: value ADR5043B -> ADR5043BRTZ
- moved J6 0.11 mm to (158.8, 89.7)
Routing:
- net V_{RF}: track 44.3 -> 34.7 mm
- net 3V0: track 72.5 -> 76.6 mm
- net GND_{RF}: track 129.1 -> 131.1 mm
- net Net-(CS6-Pad2): track 9.33 -> 10.3 mm
- net Net-(CS1-Pad2): track 9.33 -> 10.3 mm
- net Net-(CS6-Pad1): track 9.34 -> 10.3 mm
- net Net-(CS1-Pad1): track 9.45 -> 10.3 mm

Commit message: SpectDrone Development
Connections:
- B1 pad 157: unconnected-(B1-Pad157) -> P1
- B1 pad 158: unconnected-(B1-Pad158) -> S1
- B1 pad 159: unconnected-(B1-Pad159) -> P2
- B1 pad 160: unconnected-(B1-Pad160) -> S2
- B1 pad 161: unconnected-(B1-Pad161) -> /TestConnectors/CLK2_5V
- B1 pad 162: unconnected-(B1-Pad162) -> /TestConnectors/GAIN_5V
- B1 pad 163: unconnected-(B1-Pad163) -> /TestConnectors/ST_5V
- B1 pad 164: unconnected-(B1-Pad164) -> /TestConnectors/CLK1_5V
Routing:
- net GND_{RF}: track 131.1 -> 88.0 mm, vias 17 -> 15
- net GND1: track 99.8 -> 83.2 mm, vias 6 -> 5
- net J-1-4: track 120.1 -> 117.4 mm
- net J-1-3: track 118.6 -> 115.9 mm
- net P2: track 84.3 -> 82.9 mm
- net -I_{const}=0.4mA: track 28.0 -> 29.1 mm
- net V_{AREF}: track 137.8 -> 136.9 mm
- net -I_{const}=1.5mA: track 24.8 -> 25.7 mm
- net Net-(R_{C}1-Pad1): track 63.8 -> 64.5 mm
- net S1: track 60.2 -> 60.7 mm

Commit message: SpectDrone Development
Routing:
- net GND_{RF}: track 88.0 -> 126.5 mm, vias 15 -> 17

Commit message: SpectDrone Development
Parts:
- moved TPV5 0.38 mm to (155.2, 70.5)
Connections:
- SW1 pad 4: (no net) -> unconnected-(SW1-Pad4)
- SW1 pad 5: (no net) -> unconnected-(SW1-Pad5)
- SW1 pad 6: (no net) -> unconnected-(SW1-Pad6)
Routing:
- net J-1-4: track 117.4 -> 111.3 mm, vias 2 -> 3
- net J-1-3: track 115.9 -> 110.7 mm, vias 2 -> 3
- net 3V1: track 54.0 -> 51.4 mm
