File: TestComponents/TestComponents.kicad_pcb (KiCad board)
At the start: 2 copper layers, 101.6 x 73.7 mm, 131 parts, among them J2-1 Conn_01x04_Male, J2-2 Conn_01x04_Male, J3V1 Conn_01x01_Male, J5 RFShield_OnePiece, J6 RFShield_OnePiece, SW1 SW_DPDT, SW2 SW_DP3T, SW3 SW_DPDT, U1 AD7991, U13 X, U2 ADS1219, U3 REF200AU, U4 MCP6L01x-xLT, U8 ADR510, U9 ADR5043BRTZ

Commit message: SpectDrone Development
Parts:
- added JP1: SolderJumper_2_Bridged, Jumper:SolderJumper-2_P1.3mm_Bridged_RoundedPad1.0x1.5mm, F.Cu at (165.7, 117.5)
- R4: value 402 -> 250
- R5: value 200 -> 91
- SW3: value SW_DPDT -> SW_DP3T; footprint Gardenuino Custom:SW_DPDT_CK_JS202011JAQN -> Gardenuino Custom:SW_DP3T_CK_JS203011JAQN
- U8: value ADR510 -> ADR5041B
- U9: value ADR5043BRTZ -> ADR5044B
- moved SW2 4.66 mm to (167.3, 72.0)
- moved SW3 3.21 mm to (180.3, 72.0)
- moved C2 0.51 mm to (140.7, 75.2)
- moved R5 0.38 mm to (140.8, 116.5)
Connections:
- net 1V1 renamed 2V5
- net 3V0 renamed 4V0
- B2 pad 104: unconnected-(B2-Pad104) -> 3V1
- B2 pad 21: 3V1 -> unconnected-(B2-Pin_21-Pad21)
- CS11 pad 2: Net-(CS11-Pad2) -> Net-(U4--)
- R1 pad 1: Net-(CS11-Pad2) -> Net-(U4--)
- SW3 pad 2: /InsturmentationsAmps/PD_{TEST} -> unconnected-(SW3-Pad2)
- SW3 pad 3: -I_{const}=0.4mA -> /InsturmentationsAmps/PD_{TEST}
- SW3 pad 5: Net-(R_{C}1-Pad1) -> -I_{const}=0.4mA
- SW3 pad 6: -I_{const}=1.5mA -> unconnected-(SW3-Pad6)
- U3 pad 3: Net-(CS11-Pad2) -> Net-(U4--)
- U4 pad 3: Net-(CS11-Pad2) -> -I_{const}=1.5mA
- U4 pad 4: -I_{const}=1.5mA -> Net-(U4--)
Routing:
- net V_{AREF}: track 137.2 -> 120.2 mm
- net Net-(U4--): track 0.00 -> 15.2 mm
- net Net-(CS11-Pad2): track 13.0 -> 0.00 mm
- net -I_{const}=1.5mA: track 25.7 -> 31.3 mm
- net 3V1: track 51.4 -> 46.5 mm, vias 1 -> 2
- net 4V0: track 76.3 -> 81.0 mm, vias 2 -> 1
- net /InsturmentationsAmps/PD2_{TEST}: track 75.1 -> 79.4 mm
- net /InsturmentationsAmps/PD1_{TEST}: track 60.4 -> 64.2 mm
- net 2V5: track 32.5 -> 35.0 mm
- net Net-(R9-Pad2): track 30.9 -> 32.8 mm
- net -I_{const}=0.4mA: track 29.1 -> 30.8 mm
- net Net-(JP1-A): track 5.95 -> 7.10 mm
- net Net-(R_{C}1-Pad1): track 64.5 -> 65.6 mm
- net P2: track 82.9 -> 81.9 mm
Other:
- board text added: "1.5mA <- nc -> 400uA"
- board text added: "4.096V <-|-> 2.50V"
- board text removed: "1.00V"
- board text removed: "1.5mA <-|-> 400uA"
- board text removed: "3.00V <-|-> 1.00V"
- board text removed: "VOLTAGE ADJUST"

Commit message: SpectDrone Development
Parts:
- removed R_{C}1: 500, Resistor_SMD:R_0805_2012Metric
- added D1: D_Small, Diode_SMD:D_0805_2012Metric, F.Cu at (183.8, 74.7)
- added SW4: SW_DP3T, Gardenuino Custom:SW_DP3T_CK_JS203011JAQN, F.Cu at (190.0, 71.3)
- R_{PD}1, R_{PD}2: value 1M -> 1G
- R_{PD}1.1, R_{PD}2.1: value 2K -> 1K
- moved SW2 3.37 mm to (164.0, 71.3)
- moved SW3 3.37 mm to (177.0, 71.3)
- moved CS11 3.37 mm to (172.7, 77.6)
- moved R2 3.37 mm to (176.8, 77.6)
- moved CS12 3.37 mm to (169.9, 80.2)
- moved CS13 3.37 mm to (169.9, 82.2)
- moved U3 3.37 mm to (180.6, 79.4)
- moved R1 3.37 mm to (174.8, 77.6)
- moved U4 3.37 mm to (169.9, 77.6)
- moved R10 1.36 mm to (145.3, 75.7), turned to 180 degrees
- moved U13 0.56 mm to (149.4, 76.5)
- moved C1 0.38 mm to (143.6, 77.7)
- moved R_{PD}1.1 0.38 mm to (156.5, 105.0)
- moved R_{PD}2.1 0.38 mm to (138.7, 105.0)
- moved PD1 0.25 mm to (156.3, 100.7)
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Connections:
- net Net-(U4--) renamed /InsturmentationsAmps/I_{C}out
- B1 pad 157: P1 -> S1
- B1 pad 158: S1 -> P1
- B1 pad 170: P1 -> S1
- B1 pad 171: S1 -> P1
- JADC1 pad 1: P1 -> S1
- JADC1 pad 2: S1 -> P1
- JP16 pad 1: 4V0 -> PD(V)_{BIAS}
- JP16 pad 4: 5V3 -> 4V0
- SW3 pad 7: Net-(R_{C}1-Pad1) -> PD(V)_{BIAS}
- U2 pad 6: P1_{RF}-2 -> S1_{RF}-2
- U2 pad 7: S1_{RF}-2 -> P1_{RF}-2
- U3 pad 1: Net-(U3-Pad1) -> /InsturmentationsAmps/I_{C}in
- U3 pad 2: Net-(U3-Pad1) -> /InsturmentationsAmps/I_{C}1out
- U3 pad 4: -I_{const}=0.4mA -> /InsturmentationsAmps/I_{Mirror}_{IN}
- U3 pad 5: Net-(U3-Pad1) -> /InsturmentationsAmps/I_{C}in
- U3 pad 7: -I_{const}=0.4mA -> /InsturmentationsAmps/I_{C}1
Routing:
- net Net-(R_{C}1-Pad1): track 65.6 -> 0.00 mm
- net PD(V)_{BIAS}: track 112.3 -> 139.1 mm, vias 0 -> 2
- net /InsturmentationsAmps/I_{C}1: track 0.00 -> 25.1 mm
- net /InsturmentationsAmps/I_{C}in: track 0.00 -> 23.9 mm
- net /InsturmentationsAmps/I_{C}out: track 15.2 -> 37.4 mm
- net /InsturmentationsAmps/I_{Mirror}_{IN}: track 0.00 -> 19.9 mm, vias 0 -> 3
- net /InsturmentationsAmps/I_{C}1out: track 0.00 -> 16.4 mm
- net P1: track 80.3 -> 95.6 mm, vias 1 -> 2
- net S1: track 60.7 -> 46.9 mm
- net Net-(R9-Pad2): track 32.8 -> 19.4 mm
- net Net-(U3-Pad1): track 11.8 -> 0.00 mm
- net /InsturmentationsAmps/PD1_{TEST}: track 64.2 -> 54.7 mm
- net V_{AREF}: track 120.2 -> 111.4 mm
- net 5V3: track 0.00 -> 8.54 mm, vias 0 -> 3
- net GND_{RF}: track 126.5 -> 119.7 mm
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- added copper zone on In2.Cu, net 5V3
- added copper zone on In1.Cu, net GND1
- added copper zone on In1.Cu, net GND_{RF}
- removed copper zone on F.Cu, net 5V3
- removed copper zone on B.Cu, net GND1
- removed copper zone on B.Cu, net GND_{RF}
Other:
- copper layers 2 -> 4
- board text added: "0.5 | 0.75 | 1.0"
- board text added: "4.0V"
- board text added: "PD(V)_{BIAS}"
- board text added: "TEST CURRENT MULTIPLIER"
- board text removed: "3.000V"

Commit message: SpectDrone Development
Parts:
- removed TPV3: TestPoint, TestPoint:TestPoint_Keystone_5000-5004_Miniature
- added TPV2: TestPoint, TestPoint:TestPoint_Keystone_5000-5004_Miniature, F.Cu at (149.7, 119.6)
- R_{PD.bias}1, R_{PD.bias}2: value 0 -> 1K
- moved R34 5.72 mm to (159.1, 80.0), turned to 90 degrees
- moved JP12 4.95 mm to (161.4, 80.0)
- moved PD1 3.63 mm to (159.3, 102.9)
- moved PD2 3.33 mm to (150.6, 102.9)
- moved R13 2.74 mm to (140.5, 80.0), turned to 90 degrees
- moved C13 2.54 mm to (141.8, 85.4)
- moved C18 2.54 mm to (142.2, 93.7)
- moved C20 2.54 mm to (147.9, 93.7)
- moved C21 2.54 mm to (146.0, 93.7)
- moved C29 2.54 mm to (159.6, 94.0)
- moved C32 2.54 mm to (165.3, 93.9)
- moved C33 2.54 mm to (165.3, 91.9)
- moved C35 2.54 mm to (161.4, 92.7)
- moved JP16 2.54 mm to (149.8, 80.8)
- moved R18 2.54 mm to (148.0, 94.7)
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Connections:
- B1 pad 161: /TestConnectors/CLK2_5V -> /TestConnectors/GAIN_5V
- B1 pad 162: /TestConnectors/GAIN_5V -> /TestConnectors/ST_5V
- B1 pad 163: /TestConnectors/ST_5V -> /TestConnectors/CLK2_5V
- B1 pad 174: /TestConnectors/CLK2_5V -> /TestConnectors/GAIN_5V
- B1 pad 175: /TestConnectors/GAIN_5V -> /TestConnectors/ST_5V
- B1 pad 176: /TestConnectors/ST_5V -> /TestConnectors/CLK2_5V
- JD1 pad 2: /TestConnectors/ST_5V -> /TestConnectors/CLK2_5V
- JD1 pad 3: /TestConnectors/GAIN_5V -> /TestConnectors/ST_5V
- JD1 pad 4: /TestConnectors/CLK2_5V -> /TestConnectors/GAIN_5V
- SW4 pad 1: /InsturmentationsAmps/I_{C}1 -> /InsturmentationsAmps/I_{Mirror}_{IN}
- SW4 pad 4: /InsturmentationsAmps/I_{Mirror}_{IN} -> /InsturmentationsAmps/I_{C}1
Routing:
- net GND_{RF}: track 119.7 -> 193.1 mm, vias 17 -> 24
- net /InsturmentationsAmps/PD1_{TEST}: track 54.7 -> 99.0 mm
- net V_{AREF}: track 111.4 -> 154.1 mm
- net S1: track 46.9 -> 79.1 mm
- net P2: track 78.4 -> 107.8 mm
- net S2: track 65.1 -> 87.1 mm
- net /InsturmentationsAmps/I_{C}1: track 25.1 -> 10.4 mm, vias 0 -> 2
- net /InsturmentationsAmps/PD2_{TEST}: track 77.7 -> 90.5 mm
- net 4V0: track 79.8 -> 90.8 mm
- net 5V0: track 8.67 -> 16.4 mm
- net J-1-3: track 110.5 -> 103.4 mm
- net J-1-4: track 111.0 -> 104.8 mm
- net /TestConnectors/CLK2_5V: track 24.7 -> 20.0 mm
- net PD(V)_{BIAS}: track 139.1 -> 142.7 mm
- net /TestConnectors/GAIN_5V: track 21.6 -> 24.4 mm
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- added copper zone on F.Cu, net GND_{RF}

Commit message: SpectDrone Development
Parts:
- RS2, RS5: footprint Capacitor_SMD:C_0805_2012Metric -> Resistor_SMD:R_0805_2012Metric
- moved JP16 1.43 mm to (149.8, 79.4)
- moved U13 1.40 mm to (149.5, 74.8)
Routing:
- net J-1-3: track 103.4 -> 101.7 mm
- net 3V1: track 48.7 -> 47.1 mm
- net 5V0: track 16.4 -> 17.7 mm
- net PD(V)_{BIAS}: track 142.7 -> 141.6 mm
- net V_{AREF}: track 154.1 -> 155.1 mm
- net GND_{RF}: track 193.1 -> 192.1 mm
- net 4V0: track 90.8 -> 91.4 mm

Commit message: SpectDrone Development
Other:
- board text added: "CAM1RX/CS2"
- board text added: "CAM1TX/CS1"
- board text added: "CS1/CAM1TX"
- board text added: "CS2/CAM1RX"
- board text removed: "CAM1RX"
- board text removed: "CAM1TX"
Changed lines of the file:
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@@
     (effects (font (size 0.5 0.5) (thickness 0.125)) (justify left mirror))
   )
-  (gr_text "3V3" (at 134.62 73.66) (layer "B.SilkS")
+  (gr_text "3V3" (at 131.826 91.948) (layer "B.SilkS")
     (effects (font (size 0.5 0.5) (thickness 0.125)) (justify right mirror))
   )
@@
     (effects (font (size 1 1) (thickness 0.15)) (justify mirror))
   )
-  (gr_text "CAM2RX" (at 140.39357 102.108) (layer "B.SilkS")
-    (effects (font (size 1 0.75) (thickness 0.15)) (justify left mirror))
+  (gr_text "CAM2RX" (at 135.89 102.108) (layer "B.SilkS")
+    (effects (font (size 1 0.75) (thickness 0.15)) (justify right mirror))
   )
   (gr_text "TX" (at 182.88 99.06) (layer "B.SilkS")
@@
     (effects (font (size 0.5 0.5) (thickness 0.125)) (justify right mirror))
   )
-  (gr_text "S1" (at 173.99 85.09) (layer "B.SilkS")
+  (gr_text "S1" (at 171.45 85.09) (layer "B.SilkS")
     (effects (font (size 0.5 0.5) (thickness 0.125)) (justify mirror))
   )
@@
     (effects (font (size 0.5 0.35) (thickness 0.0625)) (justify left mirror))
   )
-  (gr_text "S1" (at 179.07 85.09) (layer "B.SilkS")
+  (gr_text "S2" (at 179.07 85.09) (layer "B.SilkS")
     (effects (font (size 0.5 0.5) (thickness 0.125)) (justify mirror))
   )
@@
     (effects (font (size 0.5 0.5) (thickness 0.125)) (justify mirror))
   )
-  (gr_text "CAM1RX" (at 140.39357 99.568) (layer "B.SilkS")
-    (effects (font (size 1 0.75) (thickness 0.15)) (justify left mirror))
-  )
-  (gr_text "GAIN" (at 184.15 85.09) (layer "B.SilkS")
+  (gr_text "CS2/CAM1RX" (at 135.89 99.568) (layer "B.SilkS")
+    (effects (font (size 1 0.75) (thickness 0.15)) (justify right mirror))
+  )
+  (gr_text "ST" (at 184.15 85.09) (layer "B.SilkS")
     (effects (font (size 0.5 0.5) (thickness 0.125)) (justify mirror))
   )
@@
     (effects (font (size 0.5 0.4) (thickness 0.1)) (justify mirror))
   )
-  (gr_text "CLK2" (at 181.61 85.09) (layer "B.SilkS")
+  (gr_text "GAIN" (at 181.61 85.09) (layer "B.SilkS")
     (effects (font (size 0.5 0.5) (thickness 0.125)) (justify mirror))
   )
@@
     (effects (font (size 1 1) (thickness 0.15)) (justify left mirror))
   )
-  (gr_text "CAM1TX" (at 140.39357 98.298) (layer "B.SilkS")
-    (effects (font (size 1 0.75) (thickness 0.15)) (justify left mirror))
-  )
-  (gr_text "CAM2TX" (at 140.39357 100.838) (layer "B.SilkS")
-    (effects (font (size 1 0.75) (thickness 0.15)) (justify left mirror))
+  (gr_text "CS1/CAM1TX" (at 135.89 98.298) (layer "B.SilkS")
+    (effects (font (size 1 0.75) (thickness 0.15)) (justify right mirror))
+  )
+  (gr_text "CAM2TX" (at 135.89 100.838) (layer "B.SilkS")
+    (effects (font (size 1 0.75) (thickness 0.15)) (justify right mirror))
   )
   (gr_text "CLK1" (at 187.706 84.836 -45) (layer "B.SilkS")
@@
     (effects (font (size 0.5 0.4) (thickness 0.1)) (justify mirror))
   )
-  (gr_text "ST" (at 186.69 85.09) (layer "B.SilkS")
+  (gr_text "CLK2" (at 186.182 85.09) (layer "B.SilkS")
     (effects (font (size 0.5 0.5) (thickness 0.125)) (justify mirror))
   )
@@
     (effects (font (size 0.5 0.5) (thickness 0.125)) (justify left mirror))
   )
-  (gr_text "P1" (at 171.45 85.09) (layer "B.SilkS")
+  (gr_text "P1" (at 173.99 85.09) (layer "B.SilkS")
     (effects (font (size 0.5 0.5) (thickness 0.125)) (justify mirror))
   )
@@
     (effects (font (size 0.5 0.4) (thickness 0.1)))
   )
-  (gr_text "CAM1RX" (at 135.89 99.568) (layer "F.SilkS")
+  (gr_text "CAM1RX/CS2" (at 135.89 99.568) (layer "F.SilkS")
     (effects (font (size 1 0.75) (thickness 0.15)) (justify left))
   )
@@
     (effects (font (size 1 0.55) (thickness 0.1375)) (justify right))
   )
+  (gr_text "TXSe" (at 134.366 93.98) (layer "F.SilkS")
+    (effects (font (size 1 0.5) (thickness 0.125)) (justify right mirror))
+  )
   (gr_text "S1" (at 173.228 97.282) (layer "F.SilkS")
     (effects (font (size 1 1) (thickness 0.15)) (justify left))
@@
     (effects (font (size 0.5 0.5) (thickness 0.125)))
   )
-  (gr_text "CAM1TX" (at 135.89 98.298) (layer "F.SilkS")
+  (gr_text "CAM1TX/CS1" (at 135.89 98.298) (layer "F.SilkS")
     (effects (font (size 1 0.75) (thickness 0.15)) (justify left))
   )

Commit message: SpectDrone Development
Parts:
- added JBAT1: Conn_01x02_Female, Connector_PinHeader_2.54mm:PinHeader_1x02_P2.54mm_Vertical, F.Cu at (132.5, 98.1)
- added U5: LCC110, Package_DIP:DIP-8_W8.89mm_SMDSocket_LongPads, F.Cu at (142.2, 128.9)
- R10: value X -> 24R9
- U13: value X -> ADR5045B
- moved TPV1 1.71 mm to (154.4, 120.9)
- moved TPV2 1.71 mm to (150.9, 120.9)
- moved TPGND-1 1.65 mm to (150.9, 70.5)
- moved JP16 0.77 mm to (149.8, 80.1)
- moved TPV5 0.76 mm to (154.4, 70.5)
Connections:
- B1 pad 161: /TestConnectors/GAIN_5V -> /TestConnectors/CLK2_5V
- B1 pad 162: /TestConnectors/ST_5V -> /TestConnectors/GAIN_5V
- B1 pad 163: /TestConnectors/CLK2_5V -> /TestConnectors/ST_5V
- B1 pad 174: /TestConnectors/GAIN_5V -> /TestConnectors/CLK2_5V
- B1 pad 175: /TestConnectors/ST_5V -> /TestConnectors/GAIN_5V
- B1 pad 176: /TestConnectors/CLK2_5V -> /TestConnectors/ST_5V
- CS10 pad 2: V_{AREF} -> 5V0
- CS4 pad 1: V_{AREF} -> 5V0
- CS5 pad 2: V_{AREF} -> 5V0
- CS9 pad 1: V_{AREF} -> 5V0
- JAUX1 pad 10: /TestConnectors/CAM1RX_5V -> /TestConnectors/CS2
- JAUX1 pad 11: /TestConnectors/CAM1TX_5V -> /TestConnectors/CS1
- JAUX1 pad 12: /TestConnectors/TXS_{E}_5V -> PWM
- JAUX1 pad 8: /TestConnectors/CAM2RX_5V -> /TestConnectors/Alt_{RX}
- JAUX1 pad 9: /TestConnectors/CAM2TX_5V -> /TestConnectors/Alt_{TX}
- JD1 pad 2: /TestConnectors/CLK2_5V -> /TestConnectors/ST_5V
- JD1 pad 3: /TestConnectors/ST_5V -> /TestConnectors/GAIN_5V
- JD1 pad 4: /TestConnectors/GAIN_5V -> /TestConnectors/CLK2_5V
- JP16 pad 3: 5V0 -> 4V0
- JP16 pad 4: 4V0 -> 5V0
- US1 pad 8: V_{AREF} -> 5V0
- US2 pad 8: V_{AREF} -> 5V0
Routing:
- net V_{AREF}: track 155.1 -> 48.2 mm, vias 4 -> 1
- net 5V0: track 17.7 -> 103.3 mm, vias 0 -> 4
- net PD(V)_{BIAS}: track 141.6 -> 175.6 mm
- net PWM: track 0.00 -> 28.6 mm, vias 0 -> 1
- net 2V5: track 32.5 -> 53.5 mm
- net /TestConnectors/TXS_{E}_5V: track 18.3 -> 0.00 mm
- net /TestConnectors/CAM1RX_5V: track 18.1 -> 0.00 mm
- net /TestConnectors/CAM2TX_5V: track 18.0 -> 0.00 mm
- net /TestConnectors/CAM1TX_5V: track 17.0 -> 0.00 mm
- net /TestConnectors/CAM2RX_5V: track 16.7 -> 0.00 mm
- net /TestConnectors/CLK2_5V: track 20.0 -> 24.4 mm
- net GND1: track 84.7 -> 89.0 mm, vias 6 -> 7
- net 4V0: track 91.4 -> 95.6 mm
- net /TestConnectors/GAIN_5V: track 24.4 -> 21.3 mm
- net /InsturmentationsAmps/PD2_{TEST}: track 90.3 -> 92.1 mm
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Other:
- board text added: "2.500V"
- board text added: "4.096V"
- board text added: "4.096V <-|-> 2.500V"
- board text added: "4V"
- board text added: "=R_{BIAS}"
- board text added: "SCL2_{3V}"
- board text added: "SDA2_{3V}"
- board text added: "V_{AREF}"
- board text removed: "4.096V <-|-> 2.50V"
- board text removed: "4.0V"
- board text removed: "5.0V"
- board text removed: "APCRX"
- board text removed: "APCTX"
- board text removed: "CAM1RX/CS2"
- board text removed: "CAM1TX/CS1"
- board text removed: "CAM2RX"
- board text removed: "CAM2TX"
- board text removed: "CAN_H"
- board text removed: "CAN_L"
- board text removed: "CS1/CAM1TX"
- board text removed: "CS2/CAM1RX"
- board text removed: "GPSRX"
- board text removed: "GPSTX"
- board text removed: "GPS_5V"
- board text removed: "GPS_GND"
- board text removed: "J2-1-1"
- board text removed: "J2-1-2"
- board text removed: "J2-2-1"
- board text removed: "J2-2-2"
- board text removed: "J2-2-3"
- board text removed: "J2-2-4"
- board text removed: "PPS"
- board text removed: "RX"
- board text removed: "R_{BIAS}"
- board text removed: "SCL_{3V}"
- board text removed: "SDA_{3V}"
- board text removed: "TPV1"
- board text removed: "TPV3"
- board text removed: "TPV5"
- board text removed: "TX"
- board text removed: "TXSe"
- board text removed: "UT1"
- board text removed: "UT2"
