File: TestComponents/TestConnectors.kicad_sch (KiCad schematic)
At the start: 8 parts, among them J2-1 Conn_01x04_Male, J2-2 Conn_01x04_Male

Commit message: SpectDrone Development
Changed lines of the file:
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@@
     (effects (font (size 1.27 1.27)) (justify right bottom))
+  )
+  (global_label "S1" (shape input) (at 125.095 90.805 180) (fields_autoplaced)
+    (effects (font (size 1.27 1.27)) (justify right))
+    (property "Intersheet References" "${INTERSHEET_REFS}" (id 0) (at 120.2629 90.7256 0)
+      (effects (font (size 1.27 1.27)) (justify right) hide)
+    )
+  )
+  (global_label "P1" (shape input) (at 125.095 88.265 180) (fields_autoplaced)
+    (effects (font (size 1.27 1.27)) (justify right))
+    (property "Intersheet References" "${INTERSHEET_REFS}" (id 0) (at 120.2024 88.1856 0)
+      (effects (font (size 1.27 1.27)) (justify right) hide)
+    )
+  )
+  (global_label "P2" (shape input) (at 125.095 93.345 180) (fields_autoplaced)
+    (effects (font (size 1.27 1.27)) (justify right))
+    (property "Intersheet References" "${INTERSHEET_REFS}" (id 0) (at 120.2024 93.2656 0)
+      (effects (font (size 1.27 1.27)) (justify right) hide)
+    )
   )
   (global_label "SDA_{RF}" (shape input) (at 121.92 107.95 0) (fields_autoplaced)
@@
     )
   )
+  (global_label "S2" (shape input) (at 125.095 95.885 180) (fields_autoplaced)
+    (effects (font (size 1.27 1.27)) (justify right))
+    (property "Intersheet References" "${INTERSHEET_REFS}" (id 0) (at 120.2629 95.8056 0)
+      (effects (font (size 1.27 1.27)) (justify right) hide)
+    )
+  )

Commit message: SpectDrone Development
Parts:
- renumbered J2-2 to J2-1, J2-1 to J2-2
Connections:
- net SCL_{RF}: now also J2-1.4 (Pin_4); no longer J2-2.4 (Pin_4)
- net SDA_{RF}: now also J2-1.3 (Pin_3); no longer J2-2.3 (Pin_3)
Changed lines of the file:
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@@
     )
   )
-  (global_label "SDA_{RF}" (shape input) (at 121.92 107.95 0) (fields_autoplaced)
-    (effects (font (size 1.27 1.27)) (justify left))
-    (property "Intersheet References" "${INTERSHEET_REFS}" (id 0) (at 129.7881 108.0294 0)
-      (effects (font (size 1.27 1.27)) (justify left) hide)
+  (global_label "SDA_{RF}" (shape input) (at 134.62 107.95 180) (fields_autoplaced)
+    (effects (font (size 1.27 1.27)) (justify right))
+    (property "Intersheet References" "${INTERSHEET_REFS}" (id 0) (at 126.7519 108.0294 0)
+      (effects (font (size 1.27 1.27)) (justify right) hide)
     )
   )
-  (global_label "SCL_{RF}" (shape input) (at 121.92 110.49 0) (fields_autoplaced)
-    (effects (font (size 1.27 1.27)) (justify left))
-    (property "Intersheet References" "${INTERSHEET_REFS}" (id 0) (at 129.7276 110.5694 0)
-      (effects (font (size 1.27 1.27)) (justify left) hide)
+  (global_label "SCL_{RF}" (shape input) (at 134.62 110.49 180) (fields_autoplaced)
+    (effects (font (size 1.27 1.27)) (justify right))
+    (property "Intersheet References" "${INTERSHEET_REFS}" (id 0) (at 126.8124 110.5694 0)
+      (effects (font (size 1.27 1.27)) (justify right) hide)
     )
   )
@@
   (symbol (lib_id "Connector:Conn_01x04_Male") (at 116.84 105.41 0) (unit 1)
     (in_bom yes) (on_board yes)
-    (property "Reference" "J2-1" (id 0) (at 116.205 109.22 0))
+    (property "Reference" "J2-2" (id 0) (at 116.205 109.22 0))
     (property "Value" "Conn_01x04_Male" (id 1) (at 127 106.68 0)
       (effects (font (size 1.27 1.27)) hide)
@@
   (symbol (lib_id "Connector:Conn_01x04_Male") (at 139.7 105.41 0) (mirror y) (unit 1)
     (in_bom yes) (on_board yes)
-    (property "Reference" "J2-2" (id 0) (at 140.335 109.22 0))
+    (property "Reference" "J2-1" (id 0) (at 140.335 109.22 0))
     (property "Value" "Conn_01x04_Male" (id 1) (at 129.54 106.68 0)
       (effects (font (size 1.27 1.27)) hide)

Commit message: SpectDrone Development
Parts:
- J2-1, J2-2, JADC1, JAPC1, JD1, JUT1: footprint Connector_PinHeader_2.54mm:PinHeader_1x04_P2.54mm_Vertical -> Connector_PinSocket_2.54mm:PinSocket_1x04_P2.54mm_Vertical
- JAUX1: footprint Connector_PinHeader_2.54mm:PinHeader_1x12_P2.54mm_Vertical -> Connector_PinSocket_2.54mm:PinSocket_1x12_P2.54mm_Vertical
- JGPS1: footprint Connector_PinHeader_2.54mm:PinHeader_1x05_P2.54mm_Vertical -> Connector_PinSocket_2.54mm:PinSocket_1x05_P2.54mm_Vertical
Connections:
- net 5V: no longer JGPS1.1 (Pin_1)
- net GND: no longer JGPS1.2 (Pin_2)
- new net GPS_5V: JGPS1.1 (Pin_1)
- new net GPS_GND: JGPS1.2 (Pin_2)
Changed lines of the file:
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@@
     (effects (font (size 1.27 1.27)) (justify left bottom))
   )
-  (label "5V" (at 205.74 101.6 180)
+  (label "GPS_5V" (at 205.74 101.6 180)
     (effects (font (size 1.27 1.27)) (justify right bottom))
   )
@@
     (effects (font (size 1.27 1.27)) (justify left bottom))
   )
-  (label "GND" (at 205.74 104.14 180)
+  (label "GPS_GND" (at 205.74 104.14 180)
     (effects (font (size 1.27 1.27)) (justify right bottom))
   )
@@
       (effects (font (size 1.27 1.27)) hide)
     )
-    (property "Footprint" "Connector_PinHeader_2.54mm:PinHeader_1x04_P2.54mm_Vertical" (id 2) (at 113.03 90.805 0)
+    (property "Footprint" "Connector_PinSocket_2.54mm:PinSocket_1x04_P2.54mm_Vertical" (id 2) (at 113.03 90.805 0)
       (effects (font (size 1.27 1.27)) hide)
     )
@@
       (effects (font (size 1.27 1.27)) hide)
     )
-    (property "Footprint" "Connector_PinHeader_2.54mm:PinHeader_1x04_P2.54mm_Vertical" (id 2) (at 191.135 92.71 0)
+    (property "Footprint" "Connector_PinSocket_2.54mm:PinSocket_1x04_P2.54mm_Vertical" (id 2) (at 191.135 92.71 0)
       (effects (font (size 1.27 1.27)) hide)
     )
@@
       (effects (font (size 1.27 1.27)) hide)
     )
-    (property "Footprint" "Connector_PinHeader_2.54mm:PinHeader_1x04_P2.54mm_Vertical" (id 2) (at 116.84 105.41 0)
+    (property "Footprint" "Connector_PinSocket_2.54mm:PinSocket_1x04_P2.54mm_Vertical" (id 2) (at 116.84 105.41 0)
       (effects (font (size 1.27 1.27)) hide)
     )
@@
       (effects (font (size 1.27 1.27)) (justify left) hide)
     )
-    (property "Footprint" "Connector_PinHeader_2.54mm:PinHeader_1x05_P2.54mm_Vertical" (id 2) (at 191.135 106.68 0)
+    (property "Footprint" "Connector_PinSocket_2.54mm:PinSocket_1x05_P2.54mm_Vertical" (id 2) (at 191.135 106.68 0)
       (effects (font (size 1.27 1.27)) hide)
     )
@@
       (effects (font (size 1.27 1.27)) hide)
     )
-    (property "Footprint" "Connector_PinHeader_2.54mm:PinHeader_1x04_P2.54mm_Vertical" (id 2) (at 149.86 90.805 0)
+    (property "Footprint" "Connector_PinSocket_2.54mm:PinSocket_1x04_P2.54mm_Vertical" (id 2) (at 149.86 90.805 0)
       (effects (font (size 1.27 1.27)) hide)
     )
@@
       (effects (font (size 1.27 1.27)) hide)
     )
-    (property "Footprint" "Connector_PinHeader_2.54mm:PinHeader_1x04_P2.54mm_Vertical" (id 2) (at 132.08 90.805 0)
+    (property "Footprint" "Connector_PinSocket_2.54mm:PinSocket_1x04_P2.54mm_Vertical" (id 2) (at 132.08 90.805 0)
       (effects (font (size 1.27 1.27)) hide)
     )
@@
       (effects (font (size 1.27 1.27)) hide)
     )
-    (property "Footprint" "Connector_PinHeader_2.54mm:PinHeader_1x04_P2.54mm_Vertical" (id 2) (at 139.7 105.41 0)
+    (property "Footprint" "Connector_PinSocket_2.54mm:PinSocket_1x04_P2.54mm_Vertical" (id 2) (at 139.7 105.41 0)
       (effects (font (size 1.27 1.27)) hide)
     )
@@
       (effects (font (size 1.27 1.27)) (justify left) hide)
     )
-    (property "Footprint" "Connector_PinHeader_2.54mm:PinHeader_1x12_P2.54mm_Vertical" (id 2) (at 186.055 99.695 0)
-      (effects (font (size 1.27 1.27)) hide)
-    )
+    (property "Footprint" "Connector_PinSocket_2.54mm:PinSocket_1x12_P2.54mm_Vertical" (id 2) (at 186.055 99.695 0)
+      (effects (font (size 1.27 1.27)) hide)
+    )

Commit message: SpectDrone Development
Parts:
- added JAUX2: AUX, Connector_PinSocket_2.54mm:PinSocket_1x12_P2.54mm_Vertical, symbol Connector:Conn_01x12_Female
Connections:
- net 5V: now also JAUX2.1 (Pin_1)
- net CAM1RX_5V: now also JAUX2.10 (Pin_10)
- net CAM1TX_5V: now also JAUX2.11 (Pin_11)
- net CAM2RX_5V: now also JAUX2.8 (Pin_8)
- net CAM2TX_5V: now also JAUX2.9 (Pin_9)
- net GND: now also JAUX2.2 (Pin_2)
- net MISO_5V: now also JAUX2.5 (Pin_5)
- net MOSI_5V: now also JAUX2.3 (Pin_3)
- net SCK_5V: now also JAUX2.4 (Pin_4)
- net SCL_5V: now also JAUX2.6 (Pin_6)
- net SDA_5V: now also JAUX2.7 (Pin_7)
- net TXS_{E}_5V: now also JAUX2.12 (Pin_12)
Changed lines of the file:
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@@
+    (pin "9")
+  )
+  (symbol (lib_id "Connector:Conn_01x12_Female") (at 163.195 99.695 0) (mirror y) (unit 1)
+    (in_bom yes) (on_board yes)
+    (property "Reference" "JAUX2" (id 0) (at 161.925 102.235 90)
+      (effects (font (size 1.27 1.27)) (justify left))
+    )
+    (property "Value" "AUX" (id 1) (at 165.735 100.965 90)
+      (effects (font (size 1.27 1.27)) (justify left) hide)
+    )
+    (property "Footprint" "Connector_PinSocket_2.54mm:PinSocket_1x12_P2.54mm_Vertical" (id 2) (at 163.195 99.695 0)
+      (effects (font (size 1.27 1.27)) hide)
+    )
+    (property "Datasheet" "~" (id 3) (at 163.195 99.695 0)
+      (effects (font (size 1.27 1.27)) hide)
+    )
+    (pin "1")
+    (pin "10")
+    (pin "11")
+    (pin "12")
+    (pin "2")
+    (pin "3")
+    (pin "4")
+    (pin "5")
+    (pin "6")
+    (pin "7")
+    (pin "8")
     (pin "9")
   )

Commit message: SpectDrone Development
Parts:
- added B1: Conn_02x20_Top_Bottom, Gardenuino Custom:PinHeader_CornerB1, symbol Connector_Generic:Conn_02x20_Top_Bottom
- added B2: Conn_02x20_Top_Bottom, Gardenuino Custom:PinHeader_CornerB2, symbol Connector_Generic:Conn_02x20_Top_Bottom
Connections:
- net APCRX_5V: now also B1.125 (Pin_125)
- net APCTX_5V: now also B1.136 (Pin_136)
- net CAN_H_5V: now also B1.85 (Pin_85)
- net CAN_L_5V: now also B1.77 (Pin_77)
- net CLK1_5V: now also B1.145 (Pin_145)
- net CLK2_5V: now also B1.144 (Pin_144)
- net GAIN_5V: now also B1.133 (Pin_133)
- net GPSRX_5V: now also B2.191 (Pin_191)
- net GPSTX_5V: now also B2.192 (Pin_192)
- net GPS_5V: now also B2.189 (Pin_189)
- net GPS_GND: now also B2.190 (Pin_190)
- net PPS_5V: now also B2.193 (Pin_193)
- net RX_5V: now also B1.109 (Pin_109)
- net ST_5V: now also B1.134 (Pin_134)
- net TX_5V: now also B1.117 (Pin_117)
- net UT1_5V: now also B1.101 (Pin_101)
- net UT2_5V: now also B1.93 (Pin_93)
- net J-2-1: now reaches J2-2.1 (Pin_1)
- net J-2-1: now also B1.37 (Pin_37)
- net J-2-2: now reaches J2-2.2 (Pin_2)
- net J-2-2: now also B1.29 (Pin_29)
- net J-2-3: now reaches J2-2.3 (Pin_3)
- net J-2-3: now also B1.21 (Pin_21)
- net J-2-4: now reaches J2-2.4 (Pin_4)
- net J-2-4: now also B1.13 (Pin_13)
- net J-1-1: now reaches J2-1.1 (Pin_1)
- net J-1-1: now also B1.69 (Pin_69)
- net J-1-2: now reaches J2-1.2 (Pin_2)
- net J-1-2: now also B1.61 (Pin_61)
- net 5V renamed 5V3
- net 5V3: now also B1.1 (Pin_1), B2.1 (Pin_1)
- net GND renamed GND1
- net GND1: now also B1.7 (Pin_7), B2.11 (Pin_11)
- net SCL_{RF} renamed J-1-4
- net J-1-4: now also B1.45 (Pin_45)
- net SDA_{RF} renamed J-1-3
- net J-1-3: now also B1.53 (Pin_53)
- new net 3V1: B2.21 (Pin_21)
Other:
- moved on the sheet: J2-1, J2-2, JADC1, JAPC1, JAUX1, JAUX2, JD1, JGPS1, JUT1

Commit message: SpectDrone Development
Parts:
- J2-1, J2-2, JADC1, JAPC1, JD1, JUT1: footprint Connector_PinSocket_2.54mm:PinSocket_1x04_P2.54mm_Vertical -> Connector_PinHeader_2.54mm:PinHeader_1x04_P2.54mm_Vertical
- JAUX1: footprint Connector_PinSocket_2.54mm:PinSocket_1x12_P2.54mm_Vertical -> Connector_PinHeader_2.54mm:PinHeader_1x12_P2.54mm_Vertical
- JGPS1: footprint Connector_PinSocket_2.54mm:PinSocket_1x05_P2.54mm_Vertical -> Connector_PinHeader_2.54mm:PinHeader_1x05_P2.54mm_Vertical
Connections:
- net 5V3: no longer JAUX1.1 (Pin_1)
- net CAM1RX_5V: no longer JAUX1.10 (Pin_10)
- net CAM1TX_5V: no longer JAUX1.11 (Pin_11)
- net CAM2RX_5V: no longer JAUX1.8 (Pin_8)
- net CAM2TX_5V: no longer JAUX1.9 (Pin_9)
- net GND1: now also B1.199 (Pin_199); no longer JAUX1.2 (Pin_2)
- net MISO_5V: no longer JAUX1.5 (Pin_5)
- net MOSI_5V: no longer JAUX1.3 (Pin_3)
- net SCK_5V: no longer JAUX1.4 (Pin_4)
- net SCL_5V: no longer JAUX1.6 (Pin_6)
- net SDA_5V: no longer JAUX1.7 (Pin_7)
- net TXS_{E}_5V: no longer JAUX1.12 (Pin_12)
- net VIN: now reaches B1.200 (Pin_200)
Other:
- moved on the sheet: JAUX1
Changed lines of the file:
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@@
+    )
+  )
+  (global_label "GND1" (shape input) (at 130.175 96.52 0) (fields_autoplaced)
+    (effects (font (size 1.27 1.27)) (justify left))
+    (property "Intersheet References" "${INTERSHEET_REFS}" (id 0) (at 137.6681 96.4406 0)
+      (effects (font (size 1.27 1.27)) (justify left) hide)
     )
   )
@@
     (property "Intersheet References" "${INTERSHEET_REFS}" (id 0) (at 196.6624 152.4794 0)
       (effects (font (size 1.27 1.27)) (justify right) hide)
+    )
+  )
+  (global_label "VIN" (shape input) (at 130.175 99.06 0) (fields_autoplaced)
+    (effects (font (size 1.27 1.27)) (justify left))
+    (property "Intersheet References" "${INTERSHEET_REFS}" (id 0) (at 135.6119 99.1394 0)
+      (effects (font (size 1.27 1.27)) (justify left) hide)
     )
   )
@@
       (effects (font (size 1.27 1.27)) hide)
     )
-    (property "Footprint" "Connector_PinSocket_2.54mm:PinSocket_1x04_P2.54mm_Vertical" (id 2) (at 173.99 127 0)
+    (property "Footprint" "Connector_PinHeader_2.54mm:PinHeader_1x04_P2.54mm_Vertical" (id 2) (at 173.99 127 0)
       (effects (font (size 1.27 1.27)) hide)
     )
@@
       (effects (font (size 1.27 1.27)) hide)
     )
-    (property "Footprint" "Connector_PinSocket_2.54mm:PinSocket_1x04_P2.54mm_Vertical" (id 2) (at 253.365 128.905 0)
+    (property "Footprint" "Connector_PinHeader_2.54mm:PinHeader_1x04_P2.54mm_Vertical" (id 2) (at 253.365 128.905 0)
       (effects (font (size 1.27 1.27)) hide)
     )
@@
       (effects (font (size 1.27 1.27)) hide)
     )
-    (property "Footprint" "Connector_PinSocket_2.54mm:PinSocket_1x04_P2.54mm_Vertical" (id 2) (at 173.99 141.605 0)
+    (property "Footprint" "Connector_PinHeader_2.54mm:PinHeader_1x04_P2.54mm_Vertical" (id 2) (at 173.99 141.605 0)
       (effects (font (size 1.27 1.27)) hide)
     )
@@
       (effects (font (size 1.27 1.27)) (justify left) hide)
     )
-    (property "Footprint" "Connector_PinSocket_2.54mm:PinSocket_1x05_P2.54mm_Vertical" (id 2) (at 253.365 142.875 0)
+    (property "Footprint" "Connector_PinHeader_2.54mm:PinHeader_1x05_P2.54mm_Vertical" (id 2) (at 253.365 142.875 0)
       (effects (font (size 1.27 1.27)) hide)
     )
@@
       (effects (font (size 1.27 1.27)) hide)
     )
-    (property "Footprint" "Connector_PinSocket_2.54mm:PinSocket_1x04_P2.54mm_Vertical" (id 2) (at 212.09 127 0)
+    (property "Footprint" "Connector_PinHeader_2.54mm:PinHeader_1x04_P2.54mm_Vertical" (id 2) (at 212.09 127 0)
       (effects (font (size 1.27 1.27)) hide)
     )
@@
       (effects (font (size 1.27 1.27)) hide)
     )
-    (property "Footprint" "Connector_PinSocket_2.54mm:PinSocket_1x04_P2.54mm_Vertical" (id 2) (at 191.77 127 0)
+    (property "Footprint" "Connector_PinHeader_2.54mm:PinHeader_1x04_P2.54mm_Vertical" (id 2) (at 191.77 127 0)
       (effects (font (size 1.27 1.27)) hide)
     )
@@
       (effects (font (size 1.27 1.27)) hide)
     )
-    (property "Footprint" "Connector_PinSocket_2.54mm:PinSocket_1x04_P2.54mm_Vertical" (id 2) (at 212.09 141.605 0)
+    (property "Footprint" "Connector_PinHeader_2.54mm:PinHeader_1x04_P2.54mm_Vertical" (id 2) (at 212.09 141.605 0)
       (effects (font (size 1.27 1.27)) hide)
     )
@@
     (pin "4")
   )
-  (symbol (lib_id "Connector:Conn_01x12_Male") (at 248.285 135.89 0) (mirror y) (unit 1)
-    (in_bom yes) (on_board yes)
-    (property "Reference" "JAUX1" (id 0) (at 249.555 138.43 90)
+  (symbol (lib_id "Connector:Conn_01x12_Male") (at 248.285 135.89 0) (unit 1)
+    (in_bom yes) (on_board yes)
+    (property "Reference" "JAUX1" (id 0) (at 247.015 138.43 90)
       (effects (font (size 1.27 1.27)) (justify left))
     )
-    (property "Value" "AUX" (id 1) (at 250.825 137.16 90)
+    (property "Value" "AUX" (id 1) (at 245.745 137.16 90)
       (effects (font (size 1.27 1.27)) (justify left) hide)
     )
-    (property "Footprint" "Connector_PinSocket_2.54mm:PinSocket_1x12_P2.54mm_Vertical" (id 2) (at 248.285 135.89 0)
-      (effects (font (size 1.27 1.27)) hide)
-    )
+    (property "Footprint" "Connector_PinHeader_2.54mm:PinHeader_1x12_P2.54mm_Vertical" (id 2) (at 248.285 135.89 0)
+      (effects (font (size 1.27 1.27)) hide)
+    )

Commit message: SpectDrone Development
Parts:
- removed JAUX2: AUX, Connector_PinSocket_2.54mm:PinSocket_1x12_P2.54mm_Vertical, symbol Connector:Conn_01x12_Female
Connections:
- net 5V3: now also JAUX1.1 (Pin_1)
- net CAM1RX_5V: now also B2.139 (Pin_139), JAUX1.10 (Pin_10)
- net CAM1TX_5V: now also B2.127 (Pin_127), JAUX1.11 (Pin_11)
- net CAM2RX_5V: now also B2.163 (Pin_163), JAUX1.8 (Pin_8)
- net CAM2TX_5V: now also B2.151 (Pin_151), JAUX1.9 (Pin_9)
- net GND1: now also JAUX1.2 (Pin_2)
- net GPSRX_5V: now also B2.202 (Pin_202); no longer B2.191 (Pin_191)
- net GPSTX_5V: now also B2.203 (Pin_203); no longer B2.192 (Pin_192)
- net GPS_5V: now also B2.191 (Pin_191); no longer B2.189 (Pin_189)
- net GPS_GND: now also B2.201 (Pin_201); no longer B2.190 (Pin_190)
- net MISO_5V: now also B2.187 (Pin_187), JAUX1.5 (Pin_5)
- net MOSI_5V: now also B2.189 (Pin_189), JAUX1.3 (Pin_3)
- net PPS_5V: now also B2.204 (Pin_204); no longer B2.193 (Pin_193)
- net SCK_5V: now also B2.188 (Pin_188), JAUX1.4 (Pin_4)
- net SCL_5V: now also B2.186 (Pin_186), JAUX1.6 (Pin_6)
- net SDA_5V: now also B2.185 (Pin_185), JAUX1.7 (Pin_7)
- net TXS_{E}_5V: now also B2.115 (Pin_115), JAUX1.12 (Pin_12)
- no-connect marks 0 -> 11
Other:
- moved on the sheet: JAUX1
Changed lines of the file:
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@@
   (junction (at 205.74 146.685) (diameter 0) (color 0 0 0 0)
   )
+  (no_connect (at 130.175 168.91))
+  (no_connect (at 130.175 171.45))
+  (no_connect (at 130.175 173.99))
+  (no_connect (at 117.475 173.99))
+  (no_connect (at 130.175 113.03))
+  (no_connect (at 130.175 115.57))
+  (no_connect (at 130.175 118.11))
+  (no_connect (at 130.175 120.65))
+  (no_connect (at 130.175 123.19))
+  (no_connect (at 130.175 166.37))
+  (no_connect (at 130.175 163.83))
   (wire (pts (xy 184.785 129.54) (xy 186.69 129.54))
     (stroke (width 0) (type default) (color 0 0 0 0))
@@
     (effects (font (size 1.27 1.27)) (justify left bottom))
   )
+  (label "MOSI_5V" (at 130.175 146.05 0)
+    (effects (font (size 1.27 1.27)) (justify left bottom))
+  )
   (label "GND1" (at 240.03 114.3 0)
     (effects (font (size 1.27 1.27)) (justify left bottom))
@@
     (effects (font (size 1.27 1.27)) (justify left bottom))
   )
+  (label "CAM1TX_5V" (at 104.775 115.57 0)
+    (effects (font (size 1.27 1.27)) (justify left bottom))
+  )
   (label "MOSI_5V" (at 230.505 128.27 0)
     (effects (font (size 1.27 1.27)) (justify left bottom))
@@
     (effects (font (size 1.27 1.27)) (justify right bottom))
   )
+  (label "MISO_5V" (at 130.175 140.97 0)
+    (effects (font (size 1.27 1.27)) (justify left bottom))
+  )
   (label "RX_5V" (at 197.485 132.08 0)
     (effects (font (size 1.27 1.27)) (justify left bottom))
@@
     (effects (font (size 1.27 1.27)) (justify left bottom))
   )
-  (label "GPSRX_5V" (at 130.175 151.13 0)
-    (effects (font (size 1.27 1.27)) (justify left bottom))
-  )
-  (label "PPS_5V" (at 130.175 156.21 0)
+  (label "GPSRX_5V" (at 130.175 179.07 0)
+    (effects (font (size 1.27 1.27)) (justify left bottom))
+  )
+  (label "PPS_5V" (at 130.175 184.15 0)
     (effects (font (size 1.27 1.27)) (justify left bottom))
   )
@@
     (effects (font (size 1.27 1.27)) (justify left bottom))
   )
+  (label "TXS_{E}_5V" (at 92.075 148.59 180)
+    (effects (font (size 1.27 1.27)) (justify right bottom))
+  )
+  (label "SCK_5V" (at 130.175 143.51 0)
+    (effects (font (size 1.27 1.27)) (justify left bottom))
+  )
   (label "CAN_H_5V" (at 79.375 60.96 0)
     (effects (font (size 1.27 1.27)) (justify left bottom))
@@
     (effects (font (size 1.27 1.27)) (justify left bottom))
   )
+  (label "CAM2RX_5V" (at 117.475 143.51 180)
+    (effects (font (size 1.27 1.27)) (justify right bottom))
+  )
   (label "S1" (at 184.785 127 0)
     (effects (font (size 1.27 1.27)) (justify left bottom))
   )
+  (label "SCL_5V" (at 130.175 138.43 0)
+    (effects (font (size 1.27 1.27)) (justify left bottom))
+  )
+  (label "CAM1RX_5V" (at 104.775 146.05 0)
+    (effects (font (size 1.27 1.27)) (justify left bottom))
+  )
   (label "ST_5V" (at 104.775 58.42 0)
     (effects (font (size 1.27 1.27)) (justify left bottom))
@@
     (effects (font (size 1.27 1.27)) (justify right bottom))
   )
+  (label "CAM2TX_5V" (at 117.475 113.03 180)
+    (effects (font (size 1.27 1.27)) (justify right bottom))
+  )
   (label "ST_5V" (at 160.655 127 0)
     (effects (font (size 1.27 1.27)) (justify left bottom))
@@
     (effects (font (size 1.27 1.27)) (justify left bottom))
   )
-  (label "GPSTX_5V" (at 130.175 153.67 0)
-    (effects (font (size 1.27 1.27)) (justify left bottom))
-  )
-  (label "GPS_5V" (at 130.175 146.05 0)
-    (effects (font (size 1.27 1.27)) (justify left bottom))
-  )
-  (label "GPS_GND" (at 130.175 148.59 0)
+  (label "GPSTX_5V" (at 130.175 181.61 0)
+    (effects (font (size 1.27 1.27)) (justify left bottom))
+  )
+  (label "GPS_5V" (at 130.175 151.13 0)
+    (effects (font (size 1.27 1.27)) (justify left bottom))
+  )
+  (label "GPS_GND" (at 130.175 176.53 0)
     (effects (font (size 1.27 1.27)) (justify left bottom))
   )
   (label "GPS_GND" (at 267.97 140.335 180)
     (effects (font (size 1.27 1.27)) (justify right bottom))
+  )
+  (label "SDA_5V" (at 130.175 135.89 0)
+    (effects (font (size 1.27 1.27)) (justify left bottom))
   )
   (label "RX_5V" (at 92.075 58.42 180)
@@
     (pin "194")
     (pin "195")
+    (pin "196")
+    (pin "197")
+    (pin "198")
+    (pin "199")
     (pin "2")
     (pin "20")
+    (pin "200")
+    (pin "201")
+    (pin "202")
+    (pin "203")
+    (pin "204")
     (pin "21")
     (pin "22")
@@
     (pin "4")
   )
-  (symbol (lib_id "Connector:Conn_01x12_Male") (at 248.285 135.89 0) (unit 1)
+  (symbol (lib_id "Connector:Conn_01x12_Male") (at 248.285 135.89 0) (mirror y) (unit 1)
     (in_bom yes) (on_board yes)
-    (property "Reference" "JAUX1" (id 0) (at 247.015 138.43 90)
+    (property "Reference" "JAUX1" (id 0) (at 249.555 138.43 90)
       (effects (font (size 1.27 1.27)) (justify left))
     )
-    (property "Value" "AUX" (id 1) (at 245.745 137.16 90)
+    (property "Value" "AUX" (id 1) (at 250.825 137.16 90)
       (effects (font (size 1.27 1.27)) (justify left) hide)
     )
@@
       (effects (font (size 1.27 1.27)) hide)
     )
-    (pin "1")
-    (pin "10")
-    (pin "11")
-    (pin "12")
-    (pin "2")
-    (pin "3")
-    (pin "4")
-    (pin "5")
-    (pin "6")
-    (pin "7")
-    (pin "8")
-    (pin "9")
-  )
-  (symbol (lib_id "Connector:Conn_01x12_Female") (at 225.425 135.89 0) (mirror y) (unit 1)
-    (in_bom yes) (on_board yes)
-    (property "Reference" "JAUX2" (id 0) (at 224.155 138.43 90)
-      (effects (font (size 1.27 1.27)) (justify left))
-    )
-    (property "Value" "AUX" (id 1) (at 227.965 137.16 90)
-      (effects (font (size 1.27 1.27)) (justify left) hide)
-    )
-    (property "Footprint" "Connector_PinSocket_2.54mm:PinSocket_1x12_P2.54mm_Vertical" (id 2) (at 225.425 135.89 0)
-      (effects (font (size 1.27 1.27)) hide)
-    )
-    (property "Datasheet" "~" (id 3) (at 225.425 135.89 0)
-      (effects (font (size 1.27 1.27)) hide)
-    )
