File: TestComponents/TestConnectors.kicad_sch (KiCad schematic)
At the start: 10 parts, among them J2-1 Conn_01x04_Male, J2-2 Conn_01x04_Male

Commit message: SpectDrone Development
Parts:
- added JADC2: Term_Block_01x08_Female, Gardenuino Custom:Term_Block_1x08_Female, symbol CustomParts:Terminal_Block_1x08
Connections:
- net CLK1_5V: now also B1.177 (Pin_177), JADC2.1; no longer B1.145 (Pin_145)
- net CLK2_5V: now also B1.174 (Pin_174), JADC2.4; no longer B1.144 (Pin_144)
- net GAIN_5V: now also B1.175 (Pin_175), JADC2.3; no longer B1.133 (Pin_133)
- net P1: now also B1.170 (Pin_170), JADC2.8
- net P2: now also B1.172 (Pin_172), JADC2.6
- net S1: now also B1.171 (Pin_171), JADC2.7
- net S2: now also B1.173 (Pin_173), JADC2.5
- net ST_5V: now also B1.176 (Pin_176), JADC2.2; no longer B1.134 (Pin_134)
Changed lines of the file:
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@@
+    (stroke (width 0) (type default) (color 0 0 0 0))
+  )
+  (wire (pts (xy 182.88 56.515) (xy 191.135 56.515))
     (stroke (width 0) (type default) (color 0 0 0 0))
   )
@@
     (stroke (width 0) (type default) (color 0 0 0 0))
   )
+  (wire (pts (xy 182.88 53.975) (xy 191.135 53.975))
+    (stroke (width 0) (type default) (color 0 0 0 0))
+  )
   (wire (pts (xy 230.505 151.13) (xy 243.205 151.13))
     (stroke (width 0) (type default) (color 0 0 0 0))
@@
     (stroke (width 0) (type default) (color 0 0 0 0))
   )
+  (wire (pts (xy 182.88 51.435) (xy 191.135 51.435))
+    (stroke (width 0) (type default) (color 0 0 0 0))
+  )
   (wire (pts (xy 267.97 147.955) (xy 258.445 147.955))
     (stroke (width 0) (type default) (color 0 0 0 0))
@@
     (stroke (width 0) (type default) (color 0 0 0 0))
   )
+  (wire (pts (xy 182.88 59.055) (xy 191.135 59.055))
+    (stroke (width 0) (type default) (color 0 0 0 0))
+  )
   (wire (pts (xy 197.485 129.54) (xy 207.01 129.54))
     (stroke (width 0) (type default) (color 0 0 0 0))
@@
     (stroke (width 0) (type default) (color 0 0 0 0))
   )
+  (wire (pts (xy 182.88 43.815) (xy 191.135 43.815))
+    (stroke (width 0) (type default) (color 0 0 0 0))
+  )
+  (wire (pts (xy 182.88 46.355) (xy 191.135 46.355))
+    (stroke (width 0) (type default) (color 0 0 0 0))
+  )
   (wire (pts (xy 230.505 128.27) (xy 243.205 128.27))
     (stroke (width 0) (type default) (color 0 0 0 0))
@@
     (stroke (width 0) (type default) (color 0 0 0 0))
   )
+  (wire (pts (xy 182.88 41.275) (xy 191.135 41.275))
+    (stroke (width 0) (type default) (color 0 0 0 0))
+  )
   (wire (pts (xy 205.74 152.4) (xy 205.74 146.685))
     (stroke (width 0) (type default) (color 0 0 0 0))
@@
     (stroke (width 0) (type default) (color 0 0 0 0))
   )
+  (wire (pts (xy 182.88 48.895) (xy 191.135 48.895))
+    (stroke (width 0) (type default) (color 0 0 0 0))
+  )
   (wire (pts (xy 203.2 141.605) (xy 207.01 141.605))
     (stroke (width 0) (type default) (color 0 0 0 0))
@@
     (effects (font (size 1.27 1.27)) (justify left bottom))
   )
+  (label "P2" (at 182.88 53.975 0)
+    (effects (font (size 1.27 1.27)) (justify left bottom))
+  )
+  (label "P1" (at 182.88 59.055 0)
+    (effects (font (size 1.27 1.27)) (justify left bottom))
+  )
   (label "TXS_{E}_5V" (at 230.505 151.13 0)
     (effects (font (size 1.27 1.27)) (justify left bottom))
   )
+  (label "CLK2_5V" (at 182.88 48.895 0)
+    (effects (font (size 1.27 1.27)) (justify left bottom))
+  )
   (label "TX_5V" (at 92.075 78.74 180)
     (effects (font (size 1.27 1.27)) (justify right bottom))
@@
     (effects (font (size 1.27 1.27)) (justify right bottom))
   )
-  (label "CLK2_5V" (at 104.775 83.82 0)
-    (effects (font (size 1.27 1.27)) (justify left bottom))
-  )
   (label "CAM1TX_5V" (at 230.505 148.59 0)
     (effects (font (size 1.27 1.27)) (justify left bottom))
@@
     (effects (font (size 1.27 1.27)) (justify right bottom))
   )
+  (label "P2" (at 117.475 91.44 180)
+    (effects (font (size 1.27 1.27)) (justify right bottom))
+  )
   (label "UT1_5V" (at 92.075 38.1 180)
     (effects (font (size 1.27 1.27)) (justify right bottom))
@@
     (effects (font (size 1.27 1.27)) (justify left bottom))
   )
-  (label "CLK1_5V" (at 104.775 86.36 0)
-    (effects (font (size 1.27 1.27)) (justify left bottom))
-  )
   (label "GPSRX_5V" (at 130.175 179.07 0)
     (effects (font (size 1.27 1.27)) (justify left bottom))
@@
     (effects (font (size 1.27 1.27)) (justify left bottom))
   )
+  (label "S1" (at 182.88 56.515 0)
+    (effects (font (size 1.27 1.27)) (justify left bottom))
+  )
   (label "PPS_5V" (at 267.97 147.955 180)
     (effects (font (size 1.27 1.27)) (justify right bottom))
   )
+  (label "S2" (at 182.88 51.435 0)
+    (effects (font (size 1.27 1.27)) (justify left bottom))
+  )
   (label "SCL_5V" (at 230.505 135.89 0)
     (effects (font (size 1.27 1.27)) (justify left bottom))
@@
     (effects (font (size 1.27 1.27)) (justify right bottom))
   )
+  (label "ST_5V" (at 182.88 43.815 0)
+    (effects (font (size 1.27 1.27)) (justify left bottom))
+  )
   (label "5V3" (at 230.505 123.19 0)
     (effects (font (size 1.27 1.27)) (justify left bottom))
@@
     (effects (font (size 1.27 1.27)) (justify left bottom))
   )
-  (label "ST_5V" (at 104.775 58.42 0)
-    (effects (font (size 1.27 1.27)) (justify left bottom))
-  )
   (label "CAM2RX_5V" (at 230.505 140.97 0)
     (effects (font (size 1.27 1.27)) (justify left bottom))
@@
     (effects (font (size 1.27 1.27)) (justify right bottom))
   )
+  (label "CLK2_5V" (at 117.475 96.52 180)
+    (effects (font (size 1.27 1.27)) (justify right bottom))
+  )
+  (label "S2" (at 117.475 93.98 180)
+    (effects (font (size 1.27 1.27)) (justify right bottom))
+  )
   (label "CAM2TX_5V" (at 117.475 113.03 180)
     (effects (font (size 1.27 1.27)) (justify right bottom))
@@
     (effects (font (size 1.27 1.27)) (justify left bottom))
   )
+  (label "GAIN_5V" (at 182.88 46.355 0)
+    (effects (font (size 1.27 1.27)) (justify left bottom))
+  )
   (label "CAN_L_5V" (at 79.375 40.64 0)
     (effects (font (size 1.27 1.27)) (justify left bottom))
   )
+  (label "GAIN_5V" (at 117.475 99.06 180)
+    (effects (font (size 1.27 1.27)) (justify right bottom))
+  )
+  (label "S1" (at 117.475 88.9 180)
+    (effects (font (size 1.27 1.27)) (justify right bottom))
+  )
   (label "CLK1_5V" (at 160.655 124.46 0)
     (effects (font (size 1.27 1.27)) (justify left bottom))
@@
     (effects (font (size 1.27 1.27)) (justify right bottom))
   )
+  (label "CLK1_5V" (at 130.175 40.64 0)
+    (effects (font (size 1.27 1.27)) (justify left bottom))
+  )
   (label "SDA_5V" (at 130.175 135.89 0)
     (effects (font (size 1.27 1.27)) (justify left bottom))
   )
+  (label "ST_5V" (at 130.175 38.1 0)
+    (effects (font (size 1.27 1.27)) (justify left bottom))
+  )
   (label "RX_5V" (at 92.075 58.42 180)
     (effects (font (size 1.27 1.27)) (justify right bottom))
   )
-  (label "GAIN_5V" (at 104.775 55.88 0)
-    (effects (font (size 1.27 1.27)) (justify left bottom))
+  (label "P1" (at 117.475 86.36 180)
+    (effects (font (size 1.27 1.27)) (justify right bottom))
   )
   (label "P2" (at 184.785 129.54 0)
+    (effects (font (size 1.27 1.27)) (justify left bottom))
+  )
+  (label "CLK1_5V" (at 182.88 41.275 0)
     (effects (font (size 1.27 1.27)) (justify left bottom))
   )
@@
     (pin "9")
   )
+  (symbol (lib_id "CustomParts:Terminal_Block_1x08") (at 196.215 50.165 270) (unit 1)
+    (in_bom yes) (on_board yes)
+    (property "Reference" "JADC2" (id 0) (at 202.565 50.165 90))
+    (property "Value" "Term_Block_01x08_Female" (id 1) (at 194.945 60.325 0)
+      (effects (font (size 1.27 1.27)) hide)
+    )
+    (property "Footprint" "Gardenuino Custom:Term_Block_1x08_Female" (id 2) (at 196.215 50.165 0)
+      (effects (font (size 1.27 1.27)) hide)
+    )
+    (property "Datasheet" "~" (id 3) (at 196.215 50.165 0)
+      (effects (font (size 1.27 1.27)) hide)
+    )
+    (pin "1")
+    (pin "2")
+    (pin "3")
+    (pin "4")
+    (pin "5")
+    (pin "6")
+    (pin "7")
+    (pin "8")
+  )
 )

Commit message: SpectDrone Development
Parts:
- removed JADC2: Term_Block_01x08_Female, Gardenuino Custom:Term_Block_1x08_Female, symbol CustomParts:Terminal_Block_1x08
- added JMISO5, JMOSI5, JSCK5, JSCL5, JSDA5: SolderJumper_2_Bridged, Jumper:SolderJumper-2_P1.3mm_Bridged_RoundedPad1.0x1.5mm, symbol Jumper:SolderJumper_2_Bridged
Connections:
- net MISO_5V: now also JMISO5.1 (A); no longer B2.187 (Pin_187)
- net MOSI_5V: now also JMOSI5.1 (A); no longer B2.189 (Pin_189)
- net SCK_5V: now also JSCK5.1 (A); no longer B2.188 (Pin_188)
- net SCL_5V: now also JSCL5.1 (A); no longer B2.186 (Pin_186)
- net SDA_5V: now also JSDA5.1 (A); no longer B2.185 (Pin_185)
- new net: B2.188 (Pin_188), JSCK5.2 (B)
- new net: B2.185 (Pin_185), JSDA5.2 (B)
- new net: B2.186 (Pin_186), JSCL5.2 (B)
- new net: B2.187 (Pin_187), JMISO5.2 (B)
- new net: B2.189 (Pin_189), JMOSI5.2 (B)

Commit message: SpectDrone Development
Connections:
- net CLK1_5V: now also B1.164 (Pin_164)
- net CLK2_5V: now also B1.161 (Pin_161)
- net GAIN_5V: now also B1.162 (Pin_162)
- net P1: now also B1.157 (Pin_157)
- net P2: now also B1.159 (Pin_159)
- net S1: now also B1.158 (Pin_158)
- net S2: now also B1.160 (Pin_160)
- net ST_5V: now also B1.163 (Pin_163)
Changed lines of the file:
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@@
     (effects (font (size 1.27 1.27)) (justify left bottom))
+  )
+  (label "GAIN_5V" (at 117.475 66.04 180)
+    (effects (font (size 1.27 1.27)) (justify right bottom))
   )
   (label "GAIN_5V" (at 160.655 129.54 0)
@@
   )
   (label "UT1_5V" (at 267.97 126.365 180)
+    (effects (font (size 1.27 1.27)) (justify right bottom))
+  )
+  (label "P1" (at 117.475 53.34 180)
     (effects (font (size 1.27 1.27)) (justify right bottom))
   )
@@
     (effects (font (size 1.27 1.27)) (justify right bottom))
   )
+  (label "S2" (at 117.475 60.96 180)
+    (effects (font (size 1.27 1.27)) (justify right bottom))
+  )
   (label "MISO_5V" (at 143.51 140.97 0)
     (effects (font (size 1.27 1.27)) (justify left bottom))
@@
     (effects (font (size 1.27 1.27)) (justify left bottom))
   )
+  (label "P2" (at 117.475 58.42 180)
+    (effects (font (size 1.27 1.27)) (justify right bottom))
+  )
   (label "CAM2RX_5V" (at 230.505 140.97 0)
     (effects (font (size 1.27 1.27)) (justify left bottom))
@@
     (effects (font (size 1.27 1.27)) (justify right bottom))
   )
+  (label "ST_5V" (at 117.475 68.58 180)
+    (effects (font (size 1.27 1.27)) (justify right bottom))
+  )
   (label "S2" (at 117.475 93.98 180)
+    (effects (font (size 1.27 1.27)) (justify right bottom))
+  )
+  (label "CLK2_5V" (at 117.475 63.5 180)
     (effects (font (size 1.27 1.27)) (justify right bottom))
   )
@@
     (effects (font (size 1.27 1.27)) (justify right bottom))
   )
+  (label "CLK1_5V" (at 117.475 71.12 180)
+    (effects (font (size 1.27 1.27)) (justify right bottom))
+  )
   (label "S1" (at 117.475 88.9 180)
     (effects (font (size 1.27 1.27)) (justify right bottom))
@@
     (effects (font (size 1.27 1.27)) (justify left bottom))
   )
+  (label "S1" (at 117.475 55.88 180)
+    (effects (font (size 1.27 1.27)) (justify right bottom))
+  )
   (label "GPS_GND" (at 130.175 176.53 0)

Commit message: SpectDrone Development
Parts:
- B1, B2, JMISO5, JMOSI5, JSCK5, JSCL5, JSDA5: now left out of the parts list
- J2-1, J2-2, JADC1, JAPC1, JD1, JUT1: Part Number (none) -> PH1-04-UA
- JAUX1: Part Number (none) -> PH1-12-UA
- JGPS1: Part Number (none) -> PH1-05-UA
Changed lines of the file:
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@@
+      (effects (font (size 1.27 1.27)) hide)
+    )
+    (property "Part Number" "PH1-04-UA" (id 4) (at 173.99 127 0)
       (effects (font (size 1.27 1.27)) hide)
     )
@@
       (effects (font (size 1.27 1.27)) hide)
     )
+    (property "Part Number" "PH1-04-UA" (id 4) (at 253.365 128.905 0)
+      (effects (font (size 1.27 1.27)) hide)
+    )
     (pin "1")
     (pin "2")
@@
   )
   (symbol (lib_id "Jumper:SolderJumper_2_Bridged") (at 133.985 143.51 0) (mirror y) (unit 1)
-    (in_bom yes) (on_board yes)
+    (in_bom no) (on_board yes)
     (property "Reference" "JSCK5" (id 0) (at 140.335 142.24 0))
     (property "Value" "SolderJumper_2_Bridged" (id 1) (at 127.635 146.05 0)
@@
   )
   (symbol (lib_name "Conn_02x20_Top_Bottom_1") (lib_id "Connector_Generic:Conn_02x20_Top_Bottom") (at 46.355 135.89 0) (unit 1)
-    (in_bom yes) (on_board yes) (fields_autoplaced)
+    (in_bom no) (on_board yes) (fields_autoplaced)
     (property "Reference" "B2" (id 0) (at 85.725 106.045 0))
     (property "Value" "Conn_02x20_Top_Bottom" (id 1) (at 85.725 108.585 0))
@@
   )
   (symbol (lib_id "Connector_Generic:Conn_02x20_Top_Bottom") (at 46.355 60.96 0) (unit 1)
-    (in_bom yes) (on_board yes) (fields_autoplaced)
+    (in_bom no) (on_board yes) (fields_autoplaced)
     (property "Reference" "B1" (id 0) (at 85.725 31.115 0))
     (property "Value" "Conn_02x20_Top_Bottom" (id 1) (at 85.725 33.655 0))
@@
       (effects (font (size 1.27 1.27)) hide)
     )
+    (property "Part Number" "PH1-04-UA" (id 4) (at 173.99 141.605 0)
+      (effects (font (size 1.27 1.27)) hide)
+    )
     (pin "1")
     (pin "2")
@@
       (effects (font (size 1.27 1.27)) hide)
     )
+    (property "Part Number" "PH1-05-UA" (id 4) (at 253.365 142.875 0)
+      (effects (font (size 1.27 1.27)) hide)
+    )
     (pin "1")
     (pin "2")
@@
       (effects (font (size 1.27 1.27)) hide)
     )
+    (property "Part Number" "PH1-04-UA" (id 4) (at 212.09 127 0)
+      (effects (font (size 1.27 1.27)) hide)
+    )
     (pin "1")
     (pin "2")
@@
   )
   (symbol (lib_id "Jumper:SolderJumper_2_Bridged") (at 133.985 146.05 0) (mirror y) (unit 1)
-    (in_bom yes) (on_board yes)
+    (in_bom no) (on_board yes)
     (property "Reference" "JMOSI5" (id 0) (at 140.335 144.78 0))
     (property "Value" "SolderJumper_2_Bridged" (id 1) (at 127.635 148.59 0)
@@
       (effects (font (size 1.27 1.27)) hide)
     )
+    (property "Part Number" "PH1-04-UA" (id 4) (at 191.77 127 0)
+      (effects (font (size 1.27 1.27)) hide)
+    )
     (pin "1")
     (pin "2")
@@
   )
   (symbol (lib_id "Jumper:SolderJumper_2_Bridged") (at 133.985 135.89 0) (mirror y) (unit 1)
-    (in_bom yes) (on_board yes)
+    (in_bom no) (on_board yes)
     (property "Reference" "JSDA5" (id 0) (at 140.335 134.62 0))
     (property "Value" "SolderJumper_2_Bridged" (id 1) (at 127.635 138.43 0)
@@
       (effects (font (size 1.27 1.27)) hide)
     )
+    (property "Part Number" "PH1-04-UA" (id 4) (at 212.09 141.605 0)
+      (effects (font (size 1.27 1.27)) hide)
+    )
     (pin "1")
     (pin "2")
@@
   )
   (symbol (lib_id "Jumper:SolderJumper_2_Bridged") (at 133.985 138.43 0) (mirror y) (unit 1)
-    (in_bom yes) (on_board yes)
+    (in_bom no) (on_board yes)
     (property "Reference" "JSCL5" (id 0) (at 140.335 137.16 0))
     (property "Value" "SolderJumper_2_Bridged" (id 1) (at 127.635 140.97 0)
@@
     )
     (property "Datasheet" "~" (id 3) (at 248.285 135.89 0)
+      (effects (font (size 1.27 1.27)) hide)
+    )
+    (property "Part Number" "PH1-12-UA" (id 4) (at 248.285 135.89 0)
       (effects (font (size 1.27 1.27)) hide)
     )
@@
   )
   (symbol (lib_id "Jumper:SolderJumper_2_Bridged") (at 133.985 140.97 0) (mirror y) (unit 1)
-    (in_bom yes) (on_board yes)
+    (in_bom no) (on_board yes)
     (property "Reference" "JMISO5" (id 0) (at 140.335 139.7 0))
     (property "Value" "SolderJumper_2_Bridged" (id 1) (at 127.635 143.51 0)

Commit message: SpectDrone Development
Connections:
- net 3V1: now also B2.104 (Pin_104); no longer B2.21 (Pin_21)

Commit message: SpectDrone Development
Connections:
- net P1: now also B1.158 (Pin_158), B1.171 (Pin_171), JADC1.2 (Pin_2); no longer B1.157 (Pin_157), B1.170 (Pin_170), JADC1.1 (Pin_1)
- net S1: now also B1.157 (Pin_157), B1.170 (Pin_170), JADC1.1 (Pin_1); no longer B1.158 (Pin_158), B1.171 (Pin_171), JADC1.2 (Pin_2)
Changed lines of the file:
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@@
     (effects (font (size 1.27 1.27)) (justify right bottom))
   )
-  (label "P1" (at 117.475 53.34 180) (fields_autoplaced)
+  (label "P1" (at 117.475 55.88 180) (fields_autoplaced)
     (effects (font (size 1.27 1.27)) (justify right bottom))
   )
@@
     (effects (font (size 1.27 1.27)) (justify right bottom))
   )
-  (label "P1" (at 184.785 124.46 0) (fields_autoplaced)
+  (label "P1" (at 184.785 127 0) (fields_autoplaced)
     (effects (font (size 1.27 1.27)) (justify left bottom))
   )
@@
     (effects (font (size 1.27 1.27)) (justify right bottom))
   )
-  (label "S1" (at 184.785 127 0) (fields_autoplaced)
+  (label "S1" (at 184.785 124.46 0) (fields_autoplaced)
     (effects (font (size 1.27 1.27)) (justify left bottom))
   )
@@
     (effects (font (size 1.27 1.27)) (justify right bottom))
   )
-  (label "S1" (at 117.475 88.9 180) (fields_autoplaced)
+  (label "S1" (at 117.475 86.36 180) (fields_autoplaced)
     (effects (font (size 1.27 1.27)) (justify right bottom))
   )
@@
     (effects (font (size 1.27 1.27)) (justify left bottom))
   )
-  (label "S1" (at 117.475 55.88 180) (fields_autoplaced)
+  (label "S1" (at 117.475 53.34 180) (fields_autoplaced)
     (effects (font (size 1.27 1.27)) (justify right bottom))
   )
@@
     (effects (font (size 1.27 1.27)) (justify right bottom))
   )
-  (label "P1" (at 117.475 86.36 180) (fields_autoplaced)
+  (label "P1" (at 117.475 88.9 180) (fields_autoplaced)
     (effects (font (size 1.27 1.27)) (justify right bottom))
   )
@@
     )
   )
-  (global_label "S1" (shape input) (at 184.785 127 180) (fields_autoplaced)
-    (effects (font (size 1.27 1.27)) (justify right))
-    (property "Intersheetrefs" "${INTERSHEET_REFS}" (at 179.9529 126.9206 0)
+  (global_label "S1" (shape input) (at 184.785 124.46 180) (fields_autoplaced)
+    (effects (font (size 1.27 1.27)) (justify right))
+    (property "Intersheetrefs" "${INTERSHEET_REFS}" (at 179.9529 124.5394 0)
       (effects (font (size 1.27 1.27)) (justify right) hide)
     )
@@
     )
   )
-  (global_label "P1" (shape input) (at 184.785 124.46 180) (fields_autoplaced)
-    (effects (font (size 1.27 1.27)) (justify right))
-    (property "Intersheetrefs" "${INTERSHEET_REFS}" (at 179.8924 124.3806 0)
-      (effects (font (size 1.27 1.27)) (justify right) hide)
-    )
+  (global_label "P1" (shape input) (at 184.785 127 180) (fields_autoplaced)
+    (effects (font (size 1.27 1.27)) (justify right))
+    (property "Intersheetrefs" "${INTERSHEET_REFS}" (at 179.8924 127.0794 0)
+      (effects (font (size 1.27 1.27)) (justify right) hide)
+    )

Commit message: SpectDrone Development
Connections:
- net CLK2_5V: now also B1.163 (Pin_163), B1.176 (Pin_176), JD1.2 (Pin_2); no longer B1.161 (Pin_161), B1.174 (Pin_174), JD1.4 (Pin_4)
- net GAIN_5V: now also B1.161 (Pin_161), B1.174 (Pin_174), JD1.4 (Pin_4); no longer B1.162 (Pin_162), B1.175 (Pin_175), JD1.3 (Pin_3)
- net ST_5V: now also B1.162 (Pin_162), B1.175 (Pin_175), JD1.3 (Pin_3); no longer B1.163 (Pin_163), B1.176 (Pin_176), JD1.2 (Pin_2)
Changed lines of the file:
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@@
     (effects (font (size 1.27 1.27)) (justify left bottom))
   )
-  (label "GAIN_5V" (at 117.475 66.04 180) (fields_autoplaced)
-    (effects (font (size 1.27 1.27)) (justify right bottom))
-  )
-  (label "GAIN_5V" (at 160.655 129.54 0) (fields_autoplaced)
+  (label "GAIN_5V" (at 117.475 63.5 180) (fields_autoplaced)
+    (effects (font (size 1.27 1.27)) (justify right bottom))
+  )
+  (label "GAIN_5V" (at 160.655 132.08 0) (fields_autoplaced)
     (effects (font (size 1.27 1.27)) (justify left bottom))
   )
@@
     (effects (font (size 1.27 1.27)) (justify left bottom))
   )
-  (label "CLK2_5V" (at 160.655 132.08 0) (fields_autoplaced)
+  (label "CLK2_5V" (at 160.655 127 0) (fields_autoplaced)
     (effects (font (size 1.27 1.27)) (justify left bottom))
   )
@@
     (effects (font (size 1.27 1.27)) (justify right bottom))
   )
-  (label "CLK2_5V" (at 117.475 96.52 180) (fields_autoplaced)
-    (effects (font (size 1.27 1.27)) (justify right bottom))
-  )
-  (label "ST_5V" (at 117.475 68.58 180) (fields_autoplaced)
+  (label "CLK2_5V" (at 130.175 38.1 0) (fields_autoplaced)
+    (effects (font (size 1.27 1.27)) (justify left bottom))
+  )
+  (label "ST_5V" (at 117.475 66.04 180) (fields_autoplaced)
     (effects (font (size 1.27 1.27)) (justify right bottom))
   )
@@
     (effects (font (size 1.27 1.27)) (justify right bottom))
   )
-  (label "CLK2_5V" (at 117.475 63.5 180) (fields_autoplaced)
+  (label "CLK2_5V" (at 117.475 68.58 180) (fields_autoplaced)
     (effects (font (size 1.27 1.27)) (justify right bottom))
   )
@@
     (effects (font (size 1.27 1.27)) (justify right bottom))
   )
-  (label "ST_5V" (at 160.655 127 0) (fields_autoplaced)
+  (label "ST_5V" (at 160.655 129.54 0) (fields_autoplaced)
     (effects (font (size 1.27 1.27)) (justify left bottom))
   )
@@
     (effects (font (size 1.27 1.27)) (justify left bottom))
   )
-  (label "GAIN_5V" (at 117.475 99.06 180) (fields_autoplaced)
+  (label "GAIN_5V" (at 117.475 96.52 180) (fields_autoplaced)
     (effects (font (size 1.27 1.27)) (justify right bottom))
   )
@@
     (effects (font (size 1.27 1.27)) (justify left bottom))
   )
-  (label "ST_5V" (at 130.175 38.1 0) (fields_autoplaced)
-    (effects (font (size 1.27 1.27)) (justify left bottom))
+  (label "ST_5V" (at 117.475 99.06 180) (fields_autoplaced)
+    (effects (font (size 1.27 1.27)) (justify right bottom))
   )
   (label "RX_5V" (at 92.075 58.42 180) (fields_autoplaced)
@@
     (pin "55")
     (pin "56")
-    (pin "57")
     (pin "58")
     (pin "59")
@@
     (pin "67")
     (pin "68")
-    (pin "69")
     (pin "7")
     (pin "70")
@@
     (pin "8")
     (pin "80")
-    (pin "81")
     (pin "82")
     (pin "83")
