File: TestComponents/TestConnectors.kicad_sch (KiCad schematic)
At the start: 15 parts, among them J2-1 Conn_01x04_Male, J2-2 Conn_01x04_Male

Commit message: SpectDrone Development
Connections:
- net CLK2_5V: now also B1.161 (Pin_161), B1.174 (Pin_174), JD1.4 (Pin_4); no longer B1.163 (Pin_163), B1.176 (Pin_176), JD1.2 (Pin_2)
- net GAIN_5V: now also B1.162 (Pin_162), B1.175 (Pin_175), JD1.3 (Pin_3); no longer B1.161 (Pin_161), B1.174 (Pin_174), JD1.4 (Pin_4)
- net ST_5V: now also B1.163 (Pin_163), B1.176 (Pin_176), JD1.2 (Pin_2); no longer B1.162 (Pin_162), B1.175 (Pin_175), JD1.3 (Pin_3)
- net CAM1RX_5V renamed CS2
- net CAM1TX_5V renamed CS1
- net CAM2RX_5V renamed Alt_{RX}
- net CAM2TX_5V renamed Alt_{TX}
- net TXS_{E}_5V renamed PWM
Changed lines of the file:
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@@
     (effects (font (size 1.27 1.27)) (justify left bottom))
   )
-  (label "GAIN_5V" (at 117.475 63.5 180) (fields_autoplaced)
-    (effects (font (size 1.27 1.27)) (justify right bottom))
-  )
-  (label "GAIN_5V" (at 160.655 132.08 0) (fields_autoplaced)
+  (label "GAIN_5V" (at 117.475 66.04 180) (fields_autoplaced)
+    (effects (font (size 1.27 1.27)) (justify right bottom))
+  )
+  (label "GAIN_5V" (at 160.655 129.54 0) (fields_autoplaced)
     (effects (font (size 1.27 1.27)) (justify left bottom))
   )
@@
     (effects (font (size 1.27 1.27)) (justify left bottom))
   )
-  (label "TXS_{E}_5V" (at 230.505 151.13 0) (fields_autoplaced)
-    (effects (font (size 1.27 1.27)) (justify left bottom))
-  )
   (label "TX_5V" (at 92.075 78.74 180) (fields_autoplaced)
     (effects (font (size 1.27 1.27)) (justify right bottom))
@@
     (effects (font (size 1.27 1.27)) (justify left bottom))
   )
-  (label "CAM1RX_5V" (at 230.505 146.05 0) (fields_autoplaced)
+  (label "CS2" (at 230.505 146.05 0) (fields_autoplaced)
     (effects (font (size 1.27 1.27)) (justify left bottom))
   )
@@
     (effects (font (size 1.27 1.27)) (justify right bottom))
   )
-  (label "CAM1TX_5V" (at 230.505 148.59 0) (fields_autoplaced)
-    (effects (font (size 1.27 1.27)) (justify left bottom))
-  )
-  (label "CLK2_5V" (at 160.655 127 0) (fields_autoplaced)
+  (label "CS1" (at 230.505 148.59 0) (fields_autoplaced)
+    (effects (font (size 1.27 1.27)) (justify left bottom))
+  )
+  (label "CLK2_5V" (at 160.655 132.08 0) (fields_autoplaced)
     (effects (font (size 1.27 1.27)) (justify left bottom))
   )
@@
     (effects (font (size 1.27 1.27)) (justify left bottom))
   )
-  (label "CAM1TX_5V" (at 104.775 115.57 0) (fields_autoplaced)
+  (label "CS1" (at 104.775 115.57 0) (fields_autoplaced)
     (effects (font (size 1.27 1.27)) (justify left bottom))
   )
@@
     (effects (font (size 1.27 1.27)) (justify left bottom))
   )
-  (label "TXS_{E}_5V" (at 92.075 148.59 180) (fields_autoplaced)
+  (label "PWM" (at 92.075 148.59 180) (fields_autoplaced)
     (effects (font (size 1.27 1.27)) (justify right bottom))
   )
@@
     (effects (font (size 1.27 1.27)) (justify left bottom))
   )
-  (label "CAM2RX_5V" (at 117.475 143.51 180) (fields_autoplaced)
+  (label "Alt_{RX}" (at 117.475 143.51 180) (fields_autoplaced)
     (effects (font (size 1.27 1.27)) (justify right bottom))
   )
@@
     (effects (font (size 1.27 1.27)) (justify left bottom))
   )
-  (label "CAM1RX_5V" (at 104.775 146.05 0) (fields_autoplaced)
+  (label "CS2" (at 104.775 146.05 0) (fields_autoplaced)
     (effects (font (size 1.27 1.27)) (justify left bottom))
   )
@@
     (effects (font (size 1.27 1.27)) (justify right bottom))
   )
-  (label "CAM2RX_5V" (at 230.505 140.97 0) (fields_autoplaced)
+  (label "Alt_{RX}" (at 230.505 140.97 0) (fields_autoplaced)
     (effects (font (size 1.27 1.27)) (justify left bottom))
   )
@@
     (effects (font (size 1.27 1.27)) (justify right bottom))
   )
-  (label "CLK2_5V" (at 130.175 38.1 0) (fields_autoplaced)
-    (effects (font (size 1.27 1.27)) (justify left bottom))
-  )
-  (label "ST_5V" (at 117.475 66.04 180) (fields_autoplaced)
+  (label "CLK2_5V" (at 117.475 96.52 180) (fields_autoplaced)
+    (effects (font (size 1.27 1.27)) (justify right bottom))
+  )
+  (label "ST_5V" (at 117.475 68.58 180) (fields_autoplaced)
     (effects (font (size 1.27 1.27)) (justify right bottom))
   )
@@
     (effects (font (size 1.27 1.27)) (justify right bottom))
   )
-  (label "CLK2_5V" (at 117.475 68.58 180) (fields_autoplaced)
-    (effects (font (size 1.27 1.27)) (justify right bottom))
-  )
-  (label "CAM2TX_5V" (at 117.475 113.03 180) (fields_autoplaced)
-    (effects (font (size 1.27 1.27)) (justify right bottom))
-  )
-  (label "ST_5V" (at 160.655 129.54 0) (fields_autoplaced)
-    (effects (font (size 1.27 1.27)) (justify left bottom))
-  )
-  (label "CAM2TX_5V" (at 230.505 143.51 0) (fields_autoplaced)
+  (label "CLK2_5V" (at 117.475 63.5 180) (fields_autoplaced)
+    (effects (font (size 1.27 1.27)) (justify right bottom))
+  )
+  (label "Alt_{TX}" (at 117.475 113.03 180) (fields_autoplaced)
+    (effects (font (size 1.27 1.27)) (justify right bottom))
+  )
+  (label "ST_5V" (at 160.655 127 0) (fields_autoplaced)
+    (effects (font (size 1.27 1.27)) (justify left bottom))
+  )
+  (label "Alt_{TX}" (at 230.505 143.51 0) (fields_autoplaced)
     (effects (font (size 1.27 1.27)) (justify left bottom))
   )
@@
     (effects (font (size 1.27 1.27)) (justify left bottom))
   )
-  (label "GAIN_5V" (at 117.475 96.52 180) (fields_autoplaced)
+  (label "GAIN_5V" (at 117.475 99.06 180) (fields_autoplaced)
     (effects (font (size 1.27 1.27)) (justify right bottom))
   )
@@
     (effects (font (size 1.27 1.27)) (justify left bottom))
   )
-  (label "ST_5V" (at 117.475 99.06 180) (fields_autoplaced)
-    (effects (font (size 1.27 1.27)) (justify right bottom))
+  (label "ST_5V" (at 130.175 38.1 0) (fields_autoplaced)
+    (effects (font (size 1.27 1.27)) (justify left bottom))
   )
   (label "RX_5V" (at 92.075 58.42 180) (fields_autoplaced)
@@
       (effects (font (size 1.27 1.27)) (justify right) hide)
     )
+  )
+  (global_label "PWM" (shape input) (at 230.505 151.13 180) (fields_autoplaced)
+    (effects (font (size 1.27 1.27)) (justify right))
+    (property "Intersheetrefs" "${INTERSHEET_REFS}" (at 223.347 151.13 0)
+      (effects (font (size 1.27 1.27)) (justify right) hide)
+    )
