File: TestComponents/References.kicad_sch (KiCad schematic)
At the start: 14 parts, among them SW1 SW_DPDT, U13 X, U8 ADR510, U9 ADR5043BRTZ

Commit message: SpectDrone Development
Parts:
- JP16, TPGND-1, TPV1, TPV3, TPV5: now left out of the parts list
- R4: Part Number (none) -> ERJ-PB6B4020V
- R9: Part Number (none) -> ERJ-PB6B4703V
- RV1: Part Number (none) -> 3296P-1-103LF
- SW1: Part Number (none) -> JS202011JAQN
- U8: Part Number (none) -> ADR510ARTZ-REEL7
Changed lines of the file:
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@@
+      (effects (font (size 1.27 1.27)) hide)
+    )
+    (property "Part Number" "ERJ-PB6B4020V" (id 4) (at 126.365 90.17 0)
       (effects (font (size 1.27 1.27)) hide)
     )
@@
       (effects (font (size 1.27 1.27)) hide)
     )
+    (property "Part Number" "JS202011JAQN" (id 4) (at 160.655 98.425 0)
+      (effects (font (size 1.27 1.27)) hide)
+    )
     (pin "1")
     (pin "2")
@@
       (effects (font (size 1.27 1.27)) hide)
     )
+    (property "Part Number" "ERJ-PB6B4703V" (id 4) (at 141.3901 93.98 0)
+      (effects (font (size 1.27 1.27)) hide)
+    )
     (pin "1")
     (pin "2")
   )
   (symbol (lib_id "Connector:TestPoint") (at 214.63 115.57 180) (unit 1)
-    (in_bom yes) (on_board yes)
+    (in_bom no) (on_board yes)
     (property "Reference" "TPV5" (id 0) (at 224.79 119.38 0)
       (effects (font (size 1.27 1.27)) (justify left))
@@
     (property "Datasheet" "http://www.cj-elec.com/txUpfile/20134181474991806.pdf" (id 3) (at 133.985 93.98 0)
       (effects (font (size 1.27 1.27) italic) hide)
+    )
+    (property "Part Number" "ADR510ARTZ-REEL7" (id 4) (at 133.985 93.98 0)
+      (effects (font (size 1.27 1.27)) hide)
     )
     (pin "1")
@@
   )
   (symbol (lib_id "Jumper:SolderJumper_3_Bridged12") (at 209.55 113.665 90) (mirror x) (unit 1)
-    (in_bom yes) (on_board yes)
+    (in_bom no) (on_board yes)
     (property "Reference" "JP16" (id 0) (at 207.645 111.76 90)
       (effects (font (size 1.27 1.27)) (justify left))
@@
       (effects (font (size 1.27 1.27)) hide)
     )
+    (property "Part Number" "3296P-1-103LF" (id 4) (at 150.495 93.98 0)
+      (effects (font (size 1.27 1.27)) hide)
+    )
     (pin "1")
     (pin "2")
@@
   )
   (symbol (lib_id "Connector:TestPoint") (at 150.495 90.17 0) (unit 1)
-    (in_bom yes) (on_board yes)
+    (in_bom no) (on_board yes)
     (property "Reference" "TPV1" (id 0) (at 140.335 86.36 0)
       (effects (font (size 1.27 1.27)) (justify left))
@@
   )
   (symbol (lib_id "Connector:TestPoint") (at 214.63 103.505 180) (unit 1)
-    (in_bom yes) (on_board yes)
+    (in_bom no) (on_board yes)
     (property "Reference" "TPGND-1" (id 0) (at 224.79 107.315 0)
       (effects (font (size 1.27 1.27)) (justify left))
@@
   )
   (symbol (lib_id "Connector:TestPoint") (at 150.495 106.045 0) (unit 1)
-    (in_bom yes) (on_board yes)
+    (in_bom no) (on_board yes)
     (property "Reference" "TPV3" (id 0) (at 140.335 102.235 0)
       (effects (font (size 1.27 1.27)) (justify left))

Commit message: SpectDrone Development
Parts:
- added unit 2 of SW1
- SW1: symbol Switch:SW_SPDT -> Switch:SW_DPDT_x2
Connections:
- no-connect marks 0 -> 3
Changed lines of the file:
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@@
   (junction (at 133.985 90.17) (diameter 0) (color 0 0 0 0)
   )
+  (no_connect (at 155.575 111.125))
+  (no_connect (at 155.575 116.205))
+  (no_connect (at 165.735 113.665))
   (wire (pts (xy 133.985 119.38) (xy 133.985 121.285))
     (stroke (width 0) (type default) (color 0 0 0 0))
@@
     (effects (font (size 1.27 1.27)) (justify left bottom))
   )
-  (label "GND1" (at 182.88 102.235 0)
+  (label "GND1" (at 214.63 103.505 0)
     (effects (font (size 1.27 1.27)) (justify left bottom))
   )
@@
     (pin "2")
   )
-  (symbol (lib_id "Switch:SW_SPDT") (at 160.655 98.425 180) (unit 1)
+  (symbol (lib_id "Switch:SW_DPDT_x2") (at 160.655 98.425 180) (unit 1)
     (in_bom yes) (on_board yes)
     (property "Reference" "SW1" (id 0) (at 163.83 93.98 0))
@@
     (pin "3")
   )
+  (symbol (lib_id "Switch:SW_DPDT_x2") (at 160.655 113.665 180) (unit 2)
+    (in_bom yes) (on_board yes)
+    (property "Reference" "SW1" (id 0) (at 163.83 109.855 0))
+    (property "Value" "SW_DPDT" (id 1) (at 163.83 111.76 0))
+    (property "Footprint" "" (id 2) (at 160.655 113.665 0)
+      (effects (font (size 1.27 1.27)) hide)
+    )
+    (property "Datasheet" "~" (id 3) (at 160.655 113.665 0)
+      (effects (font (size 1.27 1.27)) hide)
+    )
+    (pin "4")
+    (pin "5")
+    (pin "6")
+  )
   (symbol (lib_id "Device:R") (at 126.365 106.045 90) (unit 1)

Commit message: SpectDrone Development
Parts:
- R10, U13: now left out of the parts list
Changed lines of the file:
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@@
   )
   (symbol (lib_id "Device:R") (at 126.365 119.38 270) (mirror x) (unit 1)
-    (in_bom yes) (on_board yes)
+    (in_bom no) (on_board yes)
     (property "Reference" "R10" (id 0) (at 126.365 116.84 90))
     (property "Value" "X" (id 1) (at 126.365 119.38 90))
@@
   )
   (symbol (lib_id "Gardenuino_Custom:ADR510") (at 133.985 123.825 270) (mirror x) (unit 1)
-    (in_bom yes) (on_board yes)
+    (in_bom no) (on_board yes)
     (property "Reference" "U13" (id 0) (at 132.08 122.555 90)
       (effects (font (size 1.27 1.27)) (justify right))

Commit message: SpectDrone Development
Parts:
- added JP1: SolderJumper_2_Bridged, Jumper:SolderJumper-2_P1.3mm_Bridged_RoundedPad1.0x1.5mm, symbol Jumper:SolderJumper_2_Bridged
- R4: value 402 -> 250
- R5: value 200 -> 91
- R9, RV1: now left out of the parts list
- U8: value ADR510 -> ADR5041B
- U9: value ADR5043BRTZ -> ADR5044B
Connections:
- net at R9.1, U8.3 (REF): now also JP1.1 (A)
- net 1V1 renamed 2V5
- net 2V5: now also JP1.2 (B)
- net 3V0 renamed 4V0
Other:
- note added: "2.500V +/- 2.5mV"
- note added: "4.096V +/- 4.1mV"
- note added: "V_{S} = 5 v V_{out} = 2.5 v V = 5 v - 2.5 v = 2.5 v R_{BIAS}(I_{L_min (1PD)}) = 2.5 v / 1.3 mA = 1923 ohm R_{BIAS}(I_{L_min (2PD)}) = 2.5 v / 2.5 mA = 1000 ohm R_{BIAS}(I_{L_max}) = 2.5 v / 10.0 mA = 250 ohm R_{BIAS} = 250 ohm L = 2.5 V / 250 ohm = 10.00 mA R4 = 250 ohm"
- note added: "V_{S} = 5 v V_{out} = 4.096 v V = 5 v - 4.096 v = .904 v R_{BIAS}(I_{L_min (1PD)}) = 0.904 v / 1.3 mA = 769 ohm R_{BIAS}(I_{L_min (2PD)}) = 0.904 v / 2.5 mA = 400 ohm R_{BIAS}(I_{L_max}) = 0.904 v / 10.0 mA = 90.4 ohm R_{BIAS} = 91 ohm L = 0.904 V / 0.091 Kohm = 9.93 mA R5 = 91 ohm"
- note removed: "1.000V +/- 3.5mV"
- note removed: "3.000V +/- 3.0mV"
- note removed: "V_{S} = 5 v V_{out} = 1.0 v V = 5 v - 1.0 v = 4.0 v R_{BIAS}(I_{L_min (1PD)}) = 4.0 v / 1.3 mA = 3077 ohm R_{BIAS}(I_{L_min (2PD)}) = 4.0 v / 2.5 mA = 1600 ohm R_{BIAS}(I_{L_max}) = 4.0 v / 10.0 mA = 400 ohm R_{BIAS} = 400 ohm L = 4.0 V / 402 ohm = 9.95 mA R4 = 402 ohm"
- note removed: "V_{S} = 5 v V_{out} = 3.0 v V = 5 v - 3.0 v = 2.0 v R_{BIAS}(I_{L_min (1PD)}) = 2.0 v / 1.3 mA = 1528 ohm R_{BIAS}(I_{L_min (2PD)}) = 2.0 v / 2.5 mA = 800 ohm R_{BIAS}(I_{L_max}) = 2.0 v / 10.0 mA = 200 ohm R_{BIAS} = 200 ohm L = 2.0 V / 0.200Kohm = 10.0 mA R5 = 200 ohm"
- moved on the sheet: JP16, R10, R4, R5, SW1A, SW1B, TPGND-1, TPV5, U13, U8, U9

Commit message: SpectDrone Development
Parts:
- removed JP1: SolderJumper_2_Bridged, Jumper:SolderJumper-2_P1.3mm_Bridged_RoundedPad1.0x1.5mm, symbol Jumper:SolderJumper_2_Bridged
- removed JP16: SolderJumper_3_Bridged12, Gardenuino Custom:SolderJumper-4_P1.3mm_Bridged2Bar12_RoundedPad, symbol Jumper:SolderJumper_3_Bridged12
- removed R10: X, Resistor_SMD:R_0603_1608Metric, symbol Device:R
- removed R4: 250, Resistor_SMD:R_0805_2012Metric, symbol Device:R
- removed R5: 91, Resistor_SMD:R_0805_2012Metric, symbol Device:R
- removed R9: 470K, Resistor_SMD:R_0805_2012Metric, symbol Device:R
- removed RV1: 10K, Potentiometer_THT:Potentiometer_Bourns_3296P_Horizontal, symbol Device:R_Potentiometer
- removed SW1: SW_DPDT, Gardenuino Custom:SW_DPDT_CK_JS202011JAQN, symbol Switch:SW_DPDT_x2
- removed TPGND-1, TPV1, TPV3, TPV5: TestPoint, TestPoint:TestPoint_Keystone_5000-5004_Miniature, symbol Connector:TestPoint
- removed U13: X, Package_TO_SOT_SMD:SOT-23, symbol Gardenuino_Custom:ADR510
- removed U8: ADR5041B, Package_TO_SOT_SMD:SOT-23, symbol Gardenuino_Custom:ADR510
- removed U9: ADR5044B, Package_TO_SOT_SMD:SOT-23, symbol Gardenuino_Custom:ADR510
Connections:
- no-connect marks 3 -> 0
Other:
- note removed: "2.500V +/- 2.5mV"
- note removed: "4.096V +/- 4.1mV"
- note removed: "5.000V +/- 5.0mV"
- note removed: "ADR5045B"
- note removed: "Current -->"
- note removed: "R_{BIAS}"

Commit message: SpectDrone Development
Other:
- note removed: "V_{S} = 5 v V_{out} = 2.5 v V = 5 v - 2.5 v = 2.5 v R_{BIAS}(I_{L_min (1PD)}) = 2.5 v / 1.3 mA = 1923 ohm R_{BIAS}(I_{L_min (2PD)}) = 2.5 v / 2.5 mA = 1000 ohm R_{BIAS}(I_{L_max}) = 2.5 v / 10.0 mA = 250 ohm R_{BIAS} = 250 ohm L = 2.5 V / 250 ohm = 10.00 mA R4 = 250 ohm"
- note removed: "V_{S} = 5 v V_{out} = 4.096 v V = 5 v - 4.096 v = .904 v R_{BIAS}(I_{L_min (1PD)}) = 0.904 v / 1.3 mA = 769 ohm R_{BIAS}(I_{L_min (2PD)}) = 0.904 v / 2.5 mA = 400 ohm R_{BIAS}(I_{L_max}) = 0.904 v / 10.0 mA = 90.4 ohm R_{BIAS} = 91 ohm L = 0.904 V / 0.091 Kohm = 9.93 mA R5 = 91 ohm"
- note removed: "V_{drop} = IR -> I = V_{drop} / R R4 I = (5-1)V / .402Kohm = 9.95mA = ~10.0mA R5 I = (5-3)V / .200Kohm = 10.0mA R5 I = (5-3.3)V / .174Kohm = 9.77mA"
Changed lines of the file:
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@@
 (kicad_sch (version 20230121) (generator eeschema)
   (paper "A4")
-  (polyline (pts (xy 159.385 24.13) (xy 207.01 24.13))
-    (stroke (width 0) (type default))
-  )
-  (polyline (pts (xy 159.385 24.13) (xy 159.385 29.845))
-    (stroke (width 0) (type default))
-  )
-  (polyline (pts (xy 207.01 24.13) (xy 207.01 29.845))
-    (stroke (width 0) (type default))
-  )
-  (polyline (pts (xy 207.01 29.845) (xy 159.385 29.845))
-    (stroke (width 0) (type default))
-  )
-  (text "V_{drop} = IR -> I = V_{drop} / R\n\nR4\nI = (5-1)V / .402Kohm = 9.95mA = ~10.0mA\n\nR5\nI = (5-3)V / .200Kohm = 10.0mA\n\nR5\nI = (5-3.3)V / .174Kohm = 9.77mA"
-    (at 160.02 34.925 0)
-    (effects (font (size 1.27 1.27)) (justify left bottom))
-  )
-  (text "\nV_{S} = 5 v\nV_{out} = 2.5 v\n\nV = 5 v - 2.5 v = 2.5 v\n\nR_{BIAS}(I_{L_min (1PD)}) = 2.5 v /  1.3 mA = 1923 ohm\nR_{BIAS}(I_{L_min (2PD)}) = 2.5 v /  2.5 mA = 1000 ohm\nR_{BIAS}(I_{L_max}) = 2.5 v / 10.0 mA = 250 ohm\n\nR_{BIAS} = 250 ohm\nL = 2.5 V / 250 ohm = 10.00 mA\nR4 = 250 ohm"
-    (at 230.505 59.69 0)
-    (effects (font (size 1.27 1.27)) (justify left bottom))
-  )
-  (text "\nV_{S} = 5 v\nV_{out} = 4.096 v\n\nV = 5 v - 4.096 v = .904 v\n\nR_{BIAS}(I_{L_min (1PD)}) = 0.904 v /  1.3 mA =  769 ohm\nR_{BIAS}(I_{L_min (2PD)}) = 0.904 v /  2.5 mA =  400 ohm\nR_{BIAS}(I_{L_max}) = 0.904 v / 10.0 mA = 90.4 ohm\n\nR_{BIAS} = 91 ohm\nL = 0.904 V / 0.091 Kohm = 9.93 mA\nR5 = 91 ohm"
-    (at 231.14 109.855 0)
-    (effects (font (size 1.27 1.27)) (justify left bottom))
-  )
 )
