File: TestComponents/BandStop.kicad_sch (KiCad schematic)
At the start: 22 parts

Commit message: SpectDrone Development
Parts:
- added C26: X, Capacitor_Tantalum_SMD:CP_EIA-2012-15_AVX-P, symbol Device:C_Polarized_US
- added C27: X, Capacitor_SMD:C_0603_1608Metric, symbol Device:C
- added C28, C29, C30, C31, C32, C33, C34, C35: X, Capacitor_SMD:C_0402_1005Metric, symbol Device:C
- added C36: 1pF, Capacitor_SMD:C_0603_1608Metric, symbol Device:C
- added C37: 0.1uF, Capacitor_SMD:C_0603_1608Metric, symbol Device:C
- added R24: 0, Resistor_SMD:R_0603_1608Metric, symbol Device:R
- added R25: X, Resistor_SMD:R_0603_1608Metric, symbol Device:R
- added R26, R28, R30, R32: 0, Resistor_SMD:R_0402_1005Metric, symbol Device:R
- added R27, R29, R31, R33: X, Resistor_SMD:R_0402_1005Metric, symbol Device:R
Connections:
- net GND_{RF}: now also C27.2, C29.2, C31.2, C33.2, C35.2, R25.1, R27.1, R29.1, R31.1, R33.1
- net P1: now also C34.1, R32.2
- net P1_{RF}: now also C34.2, C35.1, R32.1, R33.2
- net P2: now also C30.1, R28.2
- net P2_{RF}: now also C30.2, C31.1, R28.1, R29.2
- net S1: now also C32.1, R30.2
- net S1_{RF}: now also C32.2, C33.1, R30.1, R31.2
- net S2: now also C28.1, R26.2
- net S2_{RF}: now also C28.2, C29.1, R26.1, R27.2
- net V_{AREF}: now also C26.1, C36.1, C37.1, R24.1
- net V_{RF}: now also C26.2, C27.1, C36.2, C37.2, R24.2, R25.2
Other:
- moved on the sheet: C16, C17, C18, C19, C20, C21, C22, C23, C24, C25, C26, C27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

Commit message: SpectDrone Development
Parts:
- renumbered C26 to C41, C27 to C42
Changed lines of the file:
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@@
   (symbol (lib_id "Device:C") (at 110.49 136.525 0) (unit 1)
     (in_bom yes) (on_board yes)
-    (property "Reference" "C27" (id 0) (at 113.665 135.89 0)
+    (property "Reference" "C42" (id 0) (at 113.665 135.89 0)
       (effects (font (size 1.27 1.27)) (justify left))
     )
@@
   (symbol (lib_id "Device:C_Polarized_US") (at 105.41 123.825 0) (unit 1)
     (in_bom yes) (on_board yes)
-    (property "Reference" "C26" (id 0) (at 100.965 123.19 0))
+    (property "Reference" "C41" (id 0) (at 100.965 123.19 0))
     (property "Value" "X" (id 1) (at 104.14 126.365 0))
     (property "Footprint" "Capacitor_Tantalum_SMD:CP_EIA-2012-15_AVX-P" (id 2) (at 105.41 123.825 0)

Commit message: SpectDrone Development
Parts:
- removed C36: 1pF, Capacitor_SMD:C_0603_1608Metric, symbol Device:C
- removed C37: 0.1uF, Capacitor_SMD:C_0603_1608Metric, symbol Device:C
- removed C41: X, Capacitor_Tantalum_SMD:CP_EIA-2012-15_AVX-P, symbol Device:C_Polarized_US
- removed C42: X, Capacitor_SMD:C_0603_1608Metric, symbol Device:C
- removed R24: 0, Resistor_SMD:R_0603_1608Metric, symbol Device:R
- removed R25: X, Resistor_SMD:R_0603_1608Metric, symbol Device:R
Connections:
- net P1_{RF}: no longer C34.2, C35.1, R32.1, R33.2
- net P2_{RF}: no longer C30.2, C31.1, R28.1, R29.2
- net S1_{RF}: no longer C32.2, C33.1, R30.1, R31.2
- net S2_{RF}: no longer C28.2, C29.1, R26.1, R27.2
- new net P1_{RF}-2: C34.2, C35.1, R32.1, R33.2
- new net P2_{RF}-2: C30.2, C31.1, R28.1, R29.2
- new net S1_{RF}-2: C32.2, C33.1, R30.1, R31.2
- new net S2_{RF}-2: C28.2, C29.1, R26.1, R27.2

Commit message: SpectDrone Development
Parts:
- C26, C27: Part Number (none) -> CL05A104KA5NNNC
Changed lines of the file:
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@@
+      (effects (font (size 1.27 1.27)) hide)
+    )
+    (property "Part Number" "CL05A104KA5NNNC" (id 4) (at 95.885 42.545 0)
       (effects (font (size 1.27 1.27)) hide)
     )
@@
       (effects (font (size 1.27 1.27)) hide)
     )
+    (property "Part Number" "CL05A104KA5NNNC" (id 4) (at 86.36 42.545 0)
+      (effects (font (size 1.27 1.27)) hide)
+    )

Commit message: SpectDrone Development
Parts:
- R14: Part Number (none) -> ERJ-U030R00V
- R16, R18, R20, R22, R26, R28, R30, R32: Part Number (none) -> ERJ-2GE0R00X
Changed lines of the file:
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@@
+      (effects (font (size 1.27 1.27)) hide)
+    )
+    (property "Part Number" "ERJ-2GE0R00X" (id 4) (at 147.32 108.585 0)
       (effects (font (size 1.27 1.27)) hide)
     )
@@
       (effects (font (size 1.27 1.27)) hide)
     )
+    (property "Part Number" "ERJ-2GE0R00X" (id 4) (at 147.32 27.305 0)
+      (effects (font (size 1.27 1.27)) hide)
+    )
     (pin "1")
     (pin "2")
@@
       (effects (font (size 1.27 1.27)) hide)
     )
+    (property "Part Number" "ERJ-2GE0R00X" (id 4) (at 177.8 27.305 0)
+      (effects (font (size 1.27 1.27)) hide)
+    )
     (pin "1")
     (pin "2")
@@
       (effects (font (size 1.27 1.27)) hide)
     )
+    (property "Part Number" "ERJ-2GE0R00X" (id 4) (at 147.32 57.785 0)
+      (effects (font (size 1.27 1.27)) hide)
+    )
     (pin "1")
     (pin "2")
@@
       (effects (font (size 1.27 1.27)) hide)
     )
+    (property "Part Number" "ERJ-2GE0R00X" (id 4) (at 147.32 139.065 0)
+      (effects (font (size 1.27 1.27)) hide)
+    )
     (pin "1")
     (pin "2")
@@
       (effects (font (size 1.27 1.27)) hide)
     )
+    (property "Part Number" "ERJ-U030R00V" (id 4) (at 110.49 42.545 0)
+      (effects (font (size 1.27 1.27)) hide)
+    )
     (pin "1")
     (pin "2")
@@
       (effects (font (size 1.27 1.27)) hide)
     )
+    (property "Part Number" "ERJ-2GE0R00X" (id 4) (at 177.8 139.065 0)
+      (effects (font (size 1.27 1.27)) hide)
+    )
     (pin "1")
     (pin "2")
@@
       (effects (font (size 1.27 1.27)) hide)
     )
+    (property "Part Number" "ERJ-2GE0R00X" (id 4) (at 177.8 108.585 0)
+      (effects (font (size 1.27 1.27)) hide)
+    )
     (pin "1")
     (pin "2")
@@
       (effects (font (size 1.27 1.27)) hide)
     )
+    (property "Part Number" "ERJ-2GE0R00X" (id 4) (at 177.8 57.785 0)
+      (effects (font (size 1.27 1.27)) hide)
+    )

Commit message: SpectDrone Development
Parts:
- C16, C17, C18, C19, C20, C21, C22, C23, C24, C25, C28, C29, C30, C31, C32, C33, C34, C35, R15, R17, R19, R21, R23, R27, R29, R31, R33: now left out of the parts list
Changed lines of the file:
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@@
   )
   (symbol (lib_id "Device:R") (at 142.24 121.285 180) (unit 1)
-    (in_bom yes) (on_board yes)
+    (in_bom no) (on_board yes)
     (property "Reference" "R31" (id 0) (at 135.89 118.745 0)
       (effects (font (size 1.27 1.27)) (justify right))
@@
   )
   (symbol (lib_id "Device:C") (at 142.24 139.065 0) (unit 1)
-    (in_bom yes) (on_board yes)
+    (in_bom no) (on_board yes)
     (property "Reference" "C34" (id 0) (at 137.795 137.795 0))
     (property "Value" "X" (id 1) (at 137.795 140.335 0))
@@
   )
   (symbol (lib_id "Device:C") (at 172.72 139.065 0) (unit 1)
-    (in_bom yes) (on_board yes)
+    (in_bom no) (on_board yes)
     (property "Reference" "C30" (id 0) (at 168.275 137.795 0))
     (property "Value" "X" (id 1) (at 168.275 140.335 0))
@@
   )
   (symbol (lib_id "Device:R") (at 172.72 121.285 180) (unit 1)
-    (in_bom yes) (on_board yes)
+    (in_bom no) (on_board yes)
     (property "Reference" "R27" (id 0) (at 166.37 118.745 0)
       (effects (font (size 1.27 1.27)) (justify right))
@@
   )
   (symbol (lib_id "Device:R") (at 142.24 151.765 180) (unit 1)
-    (in_bom yes) (on_board yes)
+    (in_bom no) (on_board yes)
     (property "Reference" "R33" (id 0) (at 135.89 149.225 0)
       (effects (font (size 1.27 1.27)) (justify right))
@@
   )
   (symbol (lib_id "Device:C") (at 177.8 121.285 0) (unit 1)
-    (in_bom yes) (on_board yes)
+    (in_bom no) (on_board yes)
     (property "Reference" "C29" (id 0) (at 180.34 118.745 0)
       (effects (font (size 1.27 1.27)) (justify left))
@@
   )
   (symbol (lib_id "Device:C") (at 177.8 70.485 0) (unit 1)
-    (in_bom yes) (on_board yes)
+    (in_bom no) (on_board yes)
     (property "Reference" "C21" (id 0) (at 180.34 67.945 0)
       (effects (font (size 1.27 1.27)) (justify left))
@@
   )
   (symbol (lib_id "Device:C") (at 172.72 108.585 0) (unit 1)
-    (in_bom yes) (on_board yes)
+    (in_bom no) (on_board yes)
     (property "Reference" "C28" (id 0) (at 168.275 107.315 0))
     (property "Value" "X" (id 1) (at 168.275 109.855 0))
@@
   )
   (symbol (lib_id "Device:C") (at 142.24 27.305 0) (unit 1)
-    (in_bom yes) (on_board yes)
+    (in_bom no) (on_board yes)
     (property "Reference" "C22" (id 0) (at 137.795 26.035 0))
     (property "Value" "X" (id 1) (at 137.795 28.575 0))
@@
   )
   (symbol (lib_id "Device:R") (at 172.72 151.765 180) (unit 1)
-    (in_bom yes) (on_board yes)
+    (in_bom no) (on_board yes)
     (property "Reference" "R29" (id 0) (at 166.37 149.225 0)
       (effects (font (size 1.27 1.27)) (justify right))
@@
   )
   (symbol (lib_id "Device:C") (at 172.72 27.305 0) (unit 1)
-    (in_bom yes) (on_board yes)
+    (in_bom no) (on_board yes)
     (property "Reference" "C18" (id 0) (at 168.275 26.035 0))
     (property "Value" "X" (id 1) (at 168.275 28.575 0))
@@
   )
   (symbol (lib_id "Device:R") (at 142.24 40.005 180) (unit 1)
-    (in_bom yes) (on_board yes)
+    (in_bom no) (on_board yes)
     (property "Reference" "R21" (id 0) (at 135.89 37.465 0)
       (effects (font (size 1.27 1.27)) (justify right))
@@
   )
   (symbol (lib_id "Device:C_Polarized_US") (at 105.41 42.545 0) (unit 1)
-    (in_bom yes) (on_board yes)
+    (in_bom no) (on_board yes)
     (property "Reference" "C16" (id 0) (at 100.965 41.91 0))
     (property "Value" "X" (id 1) (at 104.14 45.085 0))
@@
   )
   (symbol (lib_id "Device:C") (at 147.32 40.005 0) (unit 1)
-    (in_bom yes) (on_board yes)
+    (in_bom no) (on_board yes)
     (property "Reference" "C23" (id 0) (at 149.86 37.465 0)
       (effects (font (size 1.27 1.27)) (justify left))
@@
   )
   (symbol (lib_id "Device:R") (at 105.41 55.245 180) (unit 1)
-    (in_bom yes) (on_board yes)
+    (in_bom no) (on_board yes)
     (property "Reference" "R15" (id 0) (at 99.06 54.61 0)
       (effects (font (size 1.27 1.27)) (justify right))
@@
   )
   (symbol (lib_id "Device:R") (at 172.72 70.485 180) (unit 1)
-    (in_bom yes) (on_board yes)
+    (in_bom no) (on_board yes)
     (property "Reference" "R19" (id 0) (at 166.37 67.945 0)
       (effects (font (size 1.27 1.27)) (justify right))
@@
   )
   (symbol (lib_id "Device:C") (at 177.8 151.765 0) (unit 1)
-    (in_bom yes) (on_board yes)
+    (in_bom no) (on_board yes)
     (property "Reference" "C31" (id 0) (at 180.34 149.225 0)
       (effects (font (size 1.27 1.27)) (justify left))
@@
   )
   (symbol (lib_id "Device:C") (at 177.8 40.005 0) (unit 1)
-    (in_bom yes) (on_board yes)
+    (in_bom no) (on_board yes)
     (property "Reference" "C19" (id 0) (at 180.34 37.465 0)
       (effects (font (size 1.27 1.27)) (justify left))
@@
   )
   (symbol (lib_id "Device:C") (at 147.32 151.765 0) (unit 1)
-    (in_bom yes) (on_board yes)
+    (in_bom no) (on_board yes)
     (property "Reference" "C35" (id 0) (at 149.86 149.225 0)
       (effects (font (size 1.27 1.27)) (justify left))
@@
   )
   (symbol (lib_id "Device:C") (at 147.32 70.485 0) (unit 1)
-    (in_bom yes) (on_board yes)
+    (in_bom no) (on_board yes)
     (property "Reference" "C25" (id 0) (at 149.86 67.945 0)
       (effects (font (size 1.27 1.27)) (justify left))
@@
   )
   (symbol (lib_id "Device:C") (at 147.32 121.285 0) (unit 1)
-    (in_bom yes) (on_board yes)
+    (in_bom no) (on_board yes)
     (property "Reference" "C33" (id 0) (at 149.86 118.745 0)
       (effects (font (size 1.27 1.27)) (justify left))
@@
   )
   (symbol (lib_id "Device:R") (at 172.72 40.005 180) (unit 1)
-    (in_bom yes) (on_board yes)
+    (in_bom no) (on_board yes)
     (property "Reference" "R17" (id 0) (at 166.37 37.465 0)
       (effects (font (size 1.27 1.27)) (justify right))
@@
   )
   (symbol (lib_id "Device:C") (at 172.72 57.785 0) (unit 1)
-    (in_bom yes) (on_board yes)
+    (in_bom no) (on_board yes)
     (property "Reference" "C20" (id 0) (at 168.275 56.515 0))
     (property "Value" "X" (id 1) (at 168.275 59.055 0))
@@
   )
   (symbol (lib_id "Device:C") (at 142.24 108.585 0) (unit 1)
-    (in_bom yes) (on_board yes)
+    (in_bom no) (on_board yes)
     (property "Reference" "C32" (id 0) (at 137.795 107.315 0))
     (property "Value" "X" (id 1) (at 137.795 109.855 0))
@@
   )
   (symbol (lib_id "Device:C") (at 110.49 55.245 0) (unit 1)
-    (in_bom yes) (on_board yes)
+    (in_bom no) (on_board yes)
     (property "Reference" "C17" (id 0) (at 113.665 54.61 0)
       (effects (font (size 1.27 1.27)) (justify left))
@@
   )
   (symbol (lib_id "Device:C") (at 142.24 57.785 0) (unit 1)
-    (in_bom yes) (on_board yes)
+    (in_bom no) (on_board yes)
     (property "Reference" "C24" (id 0) (at 137.795 56.515 0))
     (property "Value" "X" (id 1) (at 137.795 59.055 0))
@@
   )
   (symbol (lib_id "Device:R") (at 142.24 70.485 180) (unit 1)
-    (in_bom yes) (on_board yes)
+    (in_bom no) (on_board yes)
     (property "Reference" "R23" (id 0) (at 135.89 67.945 0)
       (effects (font (size 1.27 1.27)) (justify right))
