File: Simulations/_autosave-Simulations.kicad_sch (KiCad schematic)
At the start: 10 parts

Commit message: SpectDrone Development
Parts:
- added V2, V4, V5: VSIN, symbol Simulation_SPICE:VSIN
- RPD1.1: value 15G -> 15
Connections:
- net GND: now also V5.2; no longer V3.2
- net NI_input_RF: now also V2.1; no longer V1.1
- net at V1.2: now also V5.1; no longer V3.1
- new net: V1.1, V4.2
- new net: V2.2, V3.1
- new net: V3.2, V4.1
Other:
- moved on the sheet: V1, V3
